File: board/hardware/t1-main-board/buttons.kicad_sch (KiCad schematic)
At the start: 9 parts, among them SW5501 PTS815, SW5502 PTS815, SW5503 PTS815, SW5504 Action (part open)

Commit message: Board: capture blk.current-monitors
Five INA236 on I2C1 (0x40-0x43, 0x48) with their shunts, per power tree
§4.12 and BOM v1 lines 54 and 136. The measured branches are rails of
their own (VSYS_SRC, VSYS_LV_AUDIO, VSYS_AUDIO, VSYS_LV_BL, VSYS_P5V1),
fed through the shunts on this sheet; the charger, audio, backlight and
5.1 V sheets take them. The root's layout may leave a stack level empty,
so the block sits under the notes; IC bboxes hold turned rail values;
passive rows hold a bottom rail's text.

Co-Authored-By: Claude Opus 5.5 <noreply@anthropic.com>
Claude-Session: https://claude.ai/code/session_01Ei262h3TpgY9vyfNLMi5Mn
Parts:
- removed D5501, D5502, D5503, D5504: TPD1E10B06, Package_SON:Texas_DPY0002A_0.6x1mm_P0.65mm, symbol Device:D_TVS
- removed R5501: 100 kΩ, Resistor_SMD:R_0402_1005Metric, symbol Device:R
- removed SW5501, SW5502, SW5503: PTS815, T1_Main_Board:SW_CK_PTS815, symbol Switch:SW_Push
- removed SW5504: Action (part open), Button_Switch_SMD:SW_Push_1P1T_NO_CK_KMR2, symbol Switch:SW_Push
- added D5601, D5602, D5603, D5604: TPD1E10B06, Package_SON:Texas_DPY0002A_0.6x1mm_P0.65mm, symbol Device:D_TVS
- added R5601: 100 kΩ, Resistor_SMD:R_0402_1005Metric, symbol Device:R
- added SW5601, SW5602, SW5603: PTS815, T1_Main_Board:SW_CK_PTS815, symbol Switch:SW_Push
- added SW5604: Action (part open), Button_Switch_SMD:SW_Push_1P1T_NO_CK_KMR2, symbol Switch:SW_Push
Connections:
- net ACTION_BTN_N: now also D5604.2 (A2), SW5604.1
- net GND: now also D5601.1 (A1), D5602.1 (A1), D5603.1 (A1), D5604.1 (A1), SW5601.2, SW5602.2, SW5603.2, SW5604.2
- net PWRON_N: now also D5601.2 (A2), SW5601.1
- net SARADC_VOLUP: now also D5602.2 (A2), SW5602.1
- net VOLDN_N: now also D5603.2 (A2), R5601.2, SW5603.1
- net vcca1v8_pmu: now also R5601.1
Changed lines of the file:
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@@
 (title_block (title "Side buttons") (date "2026-10-25") (rev "A") (company "The OpenDAP Project") (comment 1 "blk.buttons") (comment 2 "Power, Action, Vol+ and Vol-, each with its ESD diode"))
 (symbol (lib_id "Switch:SW_Push") (at 30.48 60.96 270) (unit 1) (body_style 1) (exclude_from_sim no) (in_bom yes) (on_board yes) (dnp no)
-  (property "Reference" "SW5501" (at 36.83 59.69 270) (effects (font (size 1.27 1.27))))
+  (property "Reference" "SW5601" (at 36.83 59.69 270) (effects (font (size 1.27 1.27))))
   (property "Value" "PTS815" (at 36.83 62.23 270) (effects (font (size 1.27 1.27))))
   (property "Footprint" "T1_Main_Board:SW_CK_PTS815" (at 30.48 60.96 0) (effects (font (size 1.27 1.27))) (hide yes))
@@
   (pin "1")
   (pin "2")
-  (instances (project "t1-main-board" (path "/7746052e-d7f9-59ad-ba73-bd2b74439529/afc5e553-cbff-5b60-bd19-e1f58e5228b5" (reference "SW5501") (unit 1))))
+  (instances (project "t1-main-board" (path "/7746052e-d7f9-59ad-ba73-bd2b74439529/afc5e553-cbff-5b60-bd19-e1f58e5228b5" (reference "SW5601") (unit 1))))
 )
 (wire (pts (xy 30.48 55.88) (xy 30.48 53.34)) (stroke (width 0) (type default)))
@@
 )
 (symbol (lib_id "Switch:SW_Push") (at 60.96 60.96 270) (unit 1) (body_style 1) (exclude_from_sim no) (in_bom yes) (on_board yes) (dnp no)
-  (property "Reference" "SW5502" (at 67.31 59.69 270) (effects (font (size 1.27 1.27))))
+  (property "Reference" "SW5602" (at 67.31 59.69 270) (effects (font (size 1.27 1.27))))
   (property "Value" "PTS815" (at 67.31 62.23 270) (effects (font (size 1.27 1.27))))
   (property "Footprint" "T1_Main_Board:SW_CK_PTS815" (at 60.96 60.96 0) (effects (font (size 1.27 1.27))) (hide yes))
@@
   (pin "1")
   (pin "2")
-  (instances (project "t1-main-board" (path "/7746052e-d7f9-59ad-ba73-bd2b74439529/afc5e553-cbff-5b60-bd19-e1f58e5228b5" (reference "SW5502") (unit 1))))
+  (instances (project "t1-main-board" (path "/7746052e-d7f9-59ad-ba73-bd2b74439529/afc5e553-cbff-5b60-bd19-e1f58e5228b5" (reference "SW5602") (unit 1))))
 )
 (wire (pts (xy 60.96 55.88) (xy 60.96 53.34)) (stroke (width 0) (type default)))
@@
 )
 (symbol (lib_id "Switch:SW_Push") (at 91.44 60.96 270) (unit 1) (body_style 1) (exclude_from_sim no) (in_bom yes) (on_board yes) (dnp no)
-  (property "Reference" "SW5503" (at 97.79 59.69 270) (effects (font (size 1.27 1.27))))
+  (property "Reference" "SW5603" (at 97.79 59.69 270) (effects (font (size 1.27 1.27))))
   (property "Value" "PTS815" (at 97.79 62.23 270) (effects (font (size 1.27 1.27))))
   (property "Footprint" "T1_Main_Board:SW_CK_PTS815" (at 91.44 60.96 0) (effects (font (size 1.27 1.27))) (hide yes))
@@
   (pin "1")
   (pin "2")
-  (instances (project "t1-main-board" (path "/7746052e-d7f9-59ad-ba73-bd2b74439529/afc5e553-cbff-5b60-bd19-e1f58e5228b5" (reference "SW5503") (unit 1))))
+  (instances (project "t1-main-board" (path "/7746052e-d7f9-59ad-ba73-bd2b74439529/afc5e553-cbff-5b60-bd19-e1f58e5228b5" (reference "SW5603") (unit 1))))
 )
 (wire (pts (xy 91.44 55.88) (xy 91.44 53.34)) (stroke (width 0) (type default)))
@@
 )
 (symbol (lib_id "Switch:SW_Push") (at 121.92 60.96 270) (unit 1) (body_style 1) (exclude_from_sim no) (in_bom yes) (on_board yes) (dnp no)
-  (property "Reference" "SW5504" (at 128.27 59.69 270) (effects (font (size 1.27 1.27))))
+  (property "Reference" "SW5604" (at 128.27 59.69 270) (effects (font (size 1.27 1.27))))
   (property "Value" "Action (part open)" (at 135.89 62.23 270) (effects (font (size 1.27 1.27))))
   (property "Footprint" "Button_Switch_SMD:SW_Push_1P1T_NO_CK_KMR2" (at 121.92 60.96 0) (effects (font (size 1.27 1.27))) (hide yes))
@@
   (pin "1")
   (pin "2")
-  (instances (project "t1-main-board" (path "/7746052e-d7f9-59ad-ba73-bd2b74439529/afc5e553-cbff-5b60-bd19-e1f58e5228b5" (reference "SW5504") (unit 1))))
+  (instances (project "t1-main-board" (path "/7746052e-d7f9-59ad-ba73-bd2b74439529/afc5e553-cbff-5b60-bd19-e1f58e5228b5" (reference "SW5604") (unit 1))))
 )
 (wire (pts (xy 121.92 55.88) (xy 121.92 53.34)) (stroke (width 0) (type default)))
@@
 (text "Buttons (BOM v1 lines 76, 77)" (exclude_from_sim no) (at 24.13 34.29 0) (effects (font (size 2.54 2.54)) (justify left bottom)))
 (symbol (lib_id "Device:R") (at 176.53 48.26 0) (unit 1) (body_style 1) (exclude_from_sim no) (in_bom yes) (on_board yes) (dnp no)
-  (property "Reference" "R5501" (at 177.8 46.99 0) (effects (font (size 1.27 1.27)) (justify left)))
+  (property "Reference" "R5601" (at 177.8 46.99 0) (effects (font (size 1.27 1.27)) (justify left)))
   (property "Value" "100 kΩ" (at 177.8 49.53 0) (effects (font (size 1.27 1.27)) (justify left)))
   (property "Footprint" "Resistor_SMD:R_0402_1005Metric" (at 176.53 48.26 0) (effects (font (size 1.27 1.27))) (hide yes))
@@
   (pin "1")
   (pin "2")
-  (instances (project "t1-main-board" (path "/7746052e-d7f9-59ad-ba73-bd2b74439529/afc5e553-cbff-5b60-bd19-e1f58e5228b5" (reference "R5501") (unit 1))))
+  (instances (project "t1-main-board" (path "/7746052e-d7f9-59ad-ba73-bd2b74439529/afc5e553-cbff-5b60-bd19-e1f58e5228b5" (reference "R5601") (unit 1))))
 )
 (wire (pts (xy 176.53 44.45) (xy 176.53 41.91)) (stroke (width 0) (type default)))
@@
 (text "Vol- pull-up 100 kΩ (pinout v1 §4)" (exclude_from_sim no) (at 165.1 34.29 0) (effects (font (size 2.54 2.54)) (justify left bottom)))
 (symbol (lib_id "Device:D_TVS") (at 30.48 113.03 90) (unit 1) (body_style 1) (exclude_from_sim no) (in_bom yes) (on_board yes) (dnp no)
-  (property "Reference" "D5501" (at 35.92 111.76 90) (effects (font (size 1.27 1.27))))
+  (property "Reference" "D5601" (at 35.92 111.76 90) (effects (font (size 1.27 1.27))))
   (property "Value" "TPD1E10B06" (at 38.82 114.3 90) (effects (font (size 1.27 1.27))))
   (property "Footprint" "Package_SON:Texas_DPY0002A_0.6x1mm_P0.65mm" (at 30.48 113.03 0) (effects (font (size 1.27 1.27))) (hide yes))
@@
   (pin "1")
   (pin "2")
-  (instances (project "t1-main-board" (path "/7746052e-d7f9-59ad-ba73-bd2b74439529/afc5e553-cbff-5b60-bd19-e1f58e5228b5" (reference "D5501") (unit 1))))
+  (instances (project "t1-main-board" (path "/7746052e-d7f9-59ad-ba73-bd2b74439529/afc5e553-cbff-5b60-bd19-e1f58e5228b5" (reference "D5601") (unit 1))))
 )
 (wire (pts (xy 30.48 109.22) (xy 30.48 106.68)) (stroke (width 0) (type default)))
@@
 )
 (symbol (lib_id "Device:D_TVS") (at 53.34 113.03 90) (unit 1) (body_style 1) (exclude_from_sim no) (in_bom yes) (on_board yes) (dnp no)
-  (property "Reference" "D5502" (at 58.78 111.76 90) (effects (font (size 1.27 1.27))))
+  (property "Reference" "D5602" (at 58.78 111.76 90) (effects (font (size 1.27 1.27))))
   (property "Value" "TPD1E10B06" (at 61.68 114.3 90) (effects (font (size 1.27 1.27))))
   (property "Footprint" "Package_SON:Texas_DPY0002A_0.6x1mm_P0.65mm" (at 53.34 113.03 0) (effects (font (size 1.27 1.27))) (hide yes))
@@
   (pin "1")
   (pin "2")
-  (instances (project "t1-main-board" (path "/7746052e-d7f9-59ad-ba73-bd2b74439529/afc5e553-cbff-5b60-bd19-e1f58e5228b5" (reference "D5502") (unit 1))))
+  (instances (project "t1-main-board" (path "/7746052e-d7f9-59ad-ba73-bd2b74439529/afc5e553-cbff-5b60-bd19-e1f58e5228b5" (reference "D5602") (unit 1))))
 )
 (wire (pts (xy 53.34 109.22) (xy 53.34 106.68)) (stroke (width 0) (type default)))
@@
 )
 (symbol (lib_id "Device:D_TVS") (at 76.2 113.03 90) (unit 1) (body_style 1) (exclude_from_sim no) (in_bom yes) (on_board yes) (dnp no)
-  (property "Reference" "D5503" (at 81.64 111.76 90) (effects (font (size 1.27 1.27))))
+  (property "Reference" "D5603" (at 81.64 111.76 90) (effects (font (size 1.27 1.27))))
   (property "Value" "TPD1E10B06" (at 84.54 114.3 90) (effects (font (size 1.27 1.27))))
   (property "Footprint" "Package_SON:Texas_DPY0002A_0.6x1mm_P0.65mm" (at 76.2 113.03 0) (effects (font (size 1.27 1.27))) (hide yes))
@@
   (pin "1")
   (pin "2")
-  (instances (project "t1-main-board" (path "/7746052e-d7f9-59ad-ba73-bd2b74439529/afc5e553-cbff-5b60-bd19-e1f58e5228b5" (reference "D5503") (unit 1))))
+  (instances (project "t1-main-board" (path "/7746052e-d7f9-59ad-ba73-bd2b74439529/afc5e553-cbff-5b60-bd19-e1f58e5228b5" (reference "D5603") (unit 1))))
 )
 (wire (pts (xy 76.2 109.22) (xy 76.2 106.68)) (stroke (width 0) (type default)))
@@
 )
 (symbol (lib_id "Device:D_TVS") (at 99.06 113.03 90) (unit 1) (body_style 1) (exclude_from_sim no) (in_bom yes) (on_board yes) (dnp no)
-  (property "Reference" "D5504" (at 104.5 111.76 90) (effects (font (size 1.27 1.27))))
+  (property "Reference" "D5604" (at 104.5 111.76 90) (effects (font (size 1.27 1.27))))
   (property "Value" "TPD1E10B06" (at 107.4 114.3 90) (effects (font (size 1.27 1.27))))
   (property "Footprint" "Package_SON:Texas_DPY0002A_0.6x1mm_P0.65mm" (at 99.06 113.03 0) (effects (font (size 1.27 1.27))) (hide yes))
@@
   (pin "1")
   (pin "2")
-  (instances (project "t1-main-board" (path "/7746052e-d7f9-59ad-ba73-bd2b74439529/afc5e553-cbff-5b60-bd19-e1f58e5228b5" (reference "D5504") (unit 1))))
+  (instances (project "t1-main-board" (path "/7746052e-d7f9-59ad-ba73-bd2b74439529/afc5e553-cbff-5b60-bd19-e1f58e5228b5" (reference "D5604") (unit 1))))
 )
 (wire (pts (xy 99.06 109.22) (xy 99.06 106.68)) (stroke (width 0) (type default)))

Commit message: Board: capture blk.status-led
LP5521 at 0x32 on I2C2 (BOM v1 line 105) with its charge-pump
capacitors, EN on vcca1v8_pmu, VDD from VSYS_LV through link #22;
LED_R/G/B reach the faceplate connector as the LED bus alias. The
faceplate row of the root is re-packed so five full columns sit left of
the title block.

Co-Authored-By: Claude Opus 5.5 <noreply@anthropic.com>
Claude-Session: https://claude.ai/code/session_01Ei262h3TpgY9vyfNLMi5Mn
Parts:
- removed D5601, D5602, D5603, D5604: TPD1E10B06, Package_SON:Texas_DPY0002A_0.6x1mm_P0.65mm, symbol Device:D_TVS
- removed R5601: 100 kΩ, Resistor_SMD:R_0402_1005Metric, symbol Device:R
- removed SW5601, SW5602, SW5603: PTS815, T1_Main_Board:SW_CK_PTS815, symbol Switch:SW_Push
- removed SW5604: Action (part open), Button_Switch_SMD:SW_Push_1P1T_NO_CK_KMR2, symbol Switch:SW_Push
- added D6501, D6502, D6503, D6504: TPD1E10B06, Package_SON:Texas_DPY0002A_0.6x1mm_P0.65mm, symbol Device:D_TVS
- added R6501: 100 kΩ, Resistor_SMD:R_0402_1005Metric, symbol Device:R
- added SW6501, SW6502, SW6503: PTS815, T1_Main_Board:SW_CK_PTS815, symbol Switch:SW_Push
- added SW6504: Action (part open), Button_Switch_SMD:SW_Push_1P1T_NO_CK_KMR2, symbol Switch:SW_Push
Connections:
- net ACTION_BTN_N: now also D6504.2 (A2), SW6504.1
- net GND: now also D6501.1 (A1), D6502.1 (A1), D6503.1 (A1), D6504.1 (A1), SW6501.2, SW6502.2, SW6503.2, SW6504.2
- net PWRON_N: now also D6501.2 (A2), SW6501.1
- net SARADC_VOLUP: now also D6502.2 (A2), SW6502.1
- net VOLDN_N: now also D6503.2 (A2), R6501.2, SW6503.1
- net vcca1v8_pmu: now also R6501.1
Changed lines of the file:
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@@
 (title_block (title "Side buttons") (date "2026-10-25") (rev "A") (company "The OpenDAP Project") (comment 1 "blk.buttons") (comment 2 "Power, Action, Vol+ and Vol-, each with its ESD diode"))
 (symbol (lib_id "Switch:SW_Push") (at 30.48 60.96 270) (unit 1) (body_style 1) (exclude_from_sim no) (in_bom yes) (on_board yes) (dnp no)
-  (property "Reference" "SW5601" (at 36.83 59.69 270) (effects (font (size 1.27 1.27))))
+  (property "Reference" "SW6501" (at 36.83 59.69 270) (effects (font (size 1.27 1.27))))
   (property "Value" "PTS815" (at 36.83 62.23 270) (effects (font (size 1.27 1.27))))
   (property "Footprint" "T1_Main_Board:SW_CK_PTS815" (at 30.48 60.96 0) (effects (font (size 1.27 1.27))) (hide yes))
@@
   (pin "1")
   (pin "2")
-  (instances (project "t1-main-board" (path "/7746052e-d7f9-59ad-ba73-bd2b74439529/afc5e553-cbff-5b60-bd19-e1f58e5228b5" (reference "SW5601") (unit 1))))
+  (instances (project "t1-main-board" (path "/7746052e-d7f9-59ad-ba73-bd2b74439529/afc5e553-cbff-5b60-bd19-e1f58e5228b5" (reference "SW6501") (unit 1))))
 )
 (wire (pts (xy 30.48 55.88) (xy 30.48 53.34)) (stroke (width 0) (type default)))
@@
 )
 (symbol (lib_id "Switch:SW_Push") (at 60.96 60.96 270) (unit 1) (body_style 1) (exclude_from_sim no) (in_bom yes) (on_board yes) (dnp no)
-  (property "Reference" "SW5602" (at 67.31 59.69 270) (effects (font (size 1.27 1.27))))
+  (property "Reference" "SW6502" (at 67.31 59.69 270) (effects (font (size 1.27 1.27))))
   (property "Value" "PTS815" (at 67.31 62.23 270) (effects (font (size 1.27 1.27))))
   (property "Footprint" "T1_Main_Board:SW_CK_PTS815" (at 60.96 60.96 0) (effects (font (size 1.27 1.27))) (hide yes))
@@
   (pin "1")
   (pin "2")
-  (instances (project "t1-main-board" (path "/7746052e-d7f9-59ad-ba73-bd2b74439529/afc5e553-cbff-5b60-bd19-e1f58e5228b5" (reference "SW5602") (unit 1))))
+  (instances (project "t1-main-board" (path "/7746052e-d7f9-59ad-ba73-bd2b74439529/afc5e553-cbff-5b60-bd19-e1f58e5228b5" (reference "SW6502") (unit 1))))
 )
 (wire (pts (xy 60.96 55.88) (xy 60.96 53.34)) (stroke (width 0) (type default)))
@@
 )
 (symbol (lib_id "Switch:SW_Push") (at 91.44 60.96 270) (unit 1) (body_style 1) (exclude_from_sim no) (in_bom yes) (on_board yes) (dnp no)
-  (property "Reference" "SW5603" (at 97.79 59.69 270) (effects (font (size 1.27 1.27))))
+  (property "Reference" "SW6503" (at 97.79 59.69 270) (effects (font (size 1.27 1.27))))
   (property "Value" "PTS815" (at 97.79 62.23 270) (effects (font (size 1.27 1.27))))
   (property "Footprint" "T1_Main_Board:SW_CK_PTS815" (at 91.44 60.96 0) (effects (font (size 1.27 1.27))) (hide yes))
@@
   (pin "1")
   (pin "2")
-  (instances (project "t1-main-board" (path "/7746052e-d7f9-59ad-ba73-bd2b74439529/afc5e553-cbff-5b60-bd19-e1f58e5228b5" (reference "SW5603") (unit 1))))
+  (instances (project "t1-main-board" (path "/7746052e-d7f9-59ad-ba73-bd2b74439529/afc5e553-cbff-5b60-bd19-e1f58e5228b5" (reference "SW6503") (unit 1))))
 )
 (wire (pts (xy 91.44 55.88) (xy 91.44 53.34)) (stroke (width 0) (type default)))
@@
 )
 (symbol (lib_id "Switch:SW_Push") (at 121.92 60.96 270) (unit 1) (body_style 1) (exclude_from_sim no) (in_bom yes) (on_board yes) (dnp no)
-  (property "Reference" "SW5604" (at 128.27 59.69 270) (effects (font (size 1.27 1.27))))
+  (property "Reference" "SW6504" (at 128.27 59.69 270) (effects (font (size 1.27 1.27))))
   (property "Value" "Action (part open)" (at 135.89 62.23 270) (effects (font (size 1.27 1.27))))
   (property "Footprint" "Button_Switch_SMD:SW_Push_1P1T_NO_CK_KMR2" (at 121.92 60.96 0) (effects (font (size 1.27 1.27))) (hide yes))
@@
   (pin "1")
   (pin "2")
-  (instances (project "t1-main-board" (path "/7746052e-d7f9-59ad-ba73-bd2b74439529/afc5e553-cbff-5b60-bd19-e1f58e5228b5" (reference "SW5604") (unit 1))))
+  (instances (project "t1-main-board" (path "/7746052e-d7f9-59ad-ba73-bd2b74439529/afc5e553-cbff-5b60-bd19-e1f58e5228b5" (reference "SW6504") (unit 1))))
 )
 (wire (pts (xy 121.92 55.88) (xy 121.92 53.34)) (stroke (width 0) (type default)))
@@
 (text "Buttons (BOM v1 lines 76, 77)" (exclude_from_sim no) (at 24.13 34.29 0) (effects (font (size 2.54 2.54)) (justify left bottom)))
 (symbol (lib_id "Device:R") (at 176.53 48.26 0) (unit 1) (body_style 1) (exclude_from_sim no) (in_bom yes) (on_board yes) (dnp no)
-  (property "Reference" "R5601" (at 177.8 46.99 0) (effects (font (size 1.27 1.27)) (justify left)))
+  (property "Reference" "R6501" (at 177.8 46.99 0) (effects (font (size 1.27 1.27)) (justify left)))
   (property "Value" "100 kΩ" (at 177.8 49.53 0) (effects (font (size 1.27 1.27)) (justify left)))
   (property "Footprint" "Resistor_SMD:R_0402_1005Metric" (at 176.53 48.26 0) (effects (font (size 1.27 1.27))) (hide yes))
@@
   (pin "1")
   (pin "2")
-  (instances (project "t1-main-board" (path "/7746052e-d7f9-59ad-ba73-bd2b74439529/afc5e553-cbff-5b60-bd19-e1f58e5228b5" (reference "R5601") (unit 1))))
+  (instances (project "t1-main-board" (path "/7746052e-d7f9-59ad-ba73-bd2b74439529/afc5e553-cbff-5b60-bd19-e1f58e5228b5" (reference "R6501") (unit 1))))
 )
 (wire (pts (xy 176.53 44.45) (xy 176.53 41.91)) (stroke (width 0) (type default)))
@@
 (text "Vol- pull-up 100 kΩ (pinout v1 §4)" (exclude_from_sim no) (at 165.1 34.29 0) (effects (font (size 2.54 2.54)) (justify left bottom)))
 (symbol (lib_id "Device:D_TVS") (at 30.48 113.03 90) (unit 1) (body_style 1) (exclude_from_sim no) (in_bom yes) (on_board yes) (dnp no)
-  (property "Reference" "D5601" (at 35.92 111.76 90) (effects (font (size 1.27 1.27))))
+  (property "Reference" "D6501" (at 35.92 111.76 90) (effects (font (size 1.27 1.27))))
   (property "Value" "TPD1E10B06" (at 38.82 114.3 90) (effects (font (size 1.27 1.27))))
   (property "Footprint" "Package_SON:Texas_DPY0002A_0.6x1mm_P0.65mm" (at 30.48 113.03 0) (effects (font (size 1.27 1.27))) (hide yes))
@@
   (pin "1")
   (pin "2")
-  (instances (project "t1-main-board" (path "/7746052e-d7f9-59ad-ba73-bd2b74439529/afc5e553-cbff-5b60-bd19-e1f58e5228b5" (reference "D5601") (unit 1))))
+  (instances (project "t1-main-board" (path "/7746052e-d7f9-59ad-ba73-bd2b74439529/afc5e553-cbff-5b60-bd19-e1f58e5228b5" (reference "D6501") (unit 1))))
 )
 (wire (pts (xy 30.48 109.22) (xy 30.48 106.68)) (stroke (width 0) (type default)))
@@
 )
 (symbol (lib_id "Device:D_TVS") (at 53.34 113.03 90) (unit 1) (body_style 1) (exclude_from_sim no) (in_bom yes) (on_board yes) (dnp no)
-  (property "Reference" "D5602" (at 58.78 111.76 90) (effects (font (size 1.27 1.27))))
+  (property "Reference" "D6502" (at 58.78 111.76 90) (effects (font (size 1.27 1.27))))
   (property "Value" "TPD1E10B06" (at 61.68 114.3 90) (effects (font (size 1.27 1.27))))
   (property "Footprint" "Package_SON:Texas_DPY0002A_0.6x1mm_P0.65mm" (at 53.34 113.03 0) (effects (font (size 1.27 1.27))) (hide yes))
@@
   (pin "1")
   (pin "2")
-  (instances (project "t1-main-board" (path "/7746052e-d7f9-59ad-ba73-bd2b74439529/afc5e553-cbff-5b60-bd19-e1f58e5228b5" (reference "D5602") (unit 1))))
+  (instances (project "t1-main-board" (path "/7746052e-d7f9-59ad-ba73-bd2b74439529/afc5e553-cbff-5b60-bd19-e1f58e5228b5" (reference "D6502") (unit 1))))
 )
 (wire (pts (xy 53.34 109.22) (xy 53.34 106.68)) (stroke (width 0) (type default)))
@@
 )
 (symbol (lib_id "Device:D_TVS") (at 76.2 113.03 90) (unit 1) (body_style 1) (exclude_from_sim no) (in_bom yes) (on_board yes) (dnp no)
-  (property "Reference" "D5603" (at 81.64 111.76 90) (effects (font (size 1.27 1.27))))
+  (property "Reference" "D6503" (at 81.64 111.76 90) (effects (font (size 1.27 1.27))))
   (property "Value" "TPD1E10B06" (at 84.54 114.3 90) (effects (font (size 1.27 1.27))))
   (property "Footprint" "Package_SON:Texas_DPY0002A_0.6x1mm_P0.65mm" (at 76.2 113.03 0) (effects (font (size 1.27 1.27))) (hide yes))
@@
   (pin "1")
   (pin "2")
-  (instances (project "t1-main-board" (path "/7746052e-d7f9-59ad-ba73-bd2b74439529/afc5e553-cbff-5b60-bd19-e1f58e5228b5" (reference "D5603") (unit 1))))
+  (instances (project "t1-main-board" (path "/7746052e-d7f9-59ad-ba73-bd2b74439529/afc5e553-cbff-5b60-bd19-e1f58e5228b5" (reference "D6503") (unit 1))))
 )
 (wire (pts (xy 76.2 109.22) (xy 76.2 106.68)) (stroke (width 0) (type default)))
@@
 )
 (symbol (lib_id "Device:D_TVS") (at 99.06 113.03 90) (unit 1) (body_style 1) (exclude_from_sim no) (in_bom yes) (on_board yes) (dnp no)
-  (property "Reference" "D5604" (at 104.5 111.76 90) (effects (font (size 1.27 1.27))))
+  (property "Reference" "D6504" (at 104.5 111.76 90) (effects (font (size 1.27 1.27))))
   (property "Value" "TPD1E10B06" (at 107.4 114.3 90) (effects (font (size 1.27 1.27))))
   (property "Footprint" "Package_SON:Texas_DPY0002A_0.6x1mm_P0.65mm" (at 99.06 113.03 0) (effects (font (size 1.27 1.27))) (hide yes))
@@
   (pin "1")
   (pin "2")
-  (instances (project "t1-main-board" (path "/7746052e-d7f9-59ad-ba73-bd2b74439529/afc5e553-cbff-5b60-bd19-e1f58e5228b5" (reference "D5604") (unit 1))))
+  (instances (project "t1-main-board" (path "/7746052e-d7f9-59ad-ba73-bd2b74439529/afc5e553-cbff-5b60-bd19-e1f58e5228b5" (reference "D6504") (unit 1))))
 )
 (wire (pts (xy 99.06 109.22) (xy 99.06 106.68)) (stroke (width 0) (type default)))
