File: board/hardware/t1-main-board/buttons.kicad_sch (KiCad schematic)
At the start: 9 parts, among them SW6501 PTS815, SW6502 PTS815, SW6503 PTS815, SW6504 Action (part open)

Commit message: Board: capture blk.debug
Debug UART2 (1.8 V) and I2S/DSD pads with ground pads, reset, PMIC and
power-key pads (PCB-T-09), a pad on every spare SoC GPIO whose pinout v1
row names one (the DEBUG bus, on the SoC's right edge), and a rail pad
for each power-tree rail no other sheet probes (PCB-T-02). Each DAC
sheet carries a pad on its MCLK. The spares pinout v1 leaves without a
pad now carry no-connect flags. On the root, facing sheet pins are
joined directly only where the route meets no other symbol.

Co-Authored-By: Claude Opus 5.5 <noreply@anthropic.com>
Claude-Session: https://claude.ai/code/session_01Ei262h3TpgY9vyfNLMi5Mn
Parts:
- removed D6501, D6502, D6503, D6504: TPD1E10B06, Package_SON:Texas_DPY0002A_0.6x1mm_P0.65mm, symbol Device:D_TVS
- removed R6501: 100 kΩ, Resistor_SMD:R_0402_1005Metric, symbol Device:R
- removed SW6501, SW6502, SW6503: PTS815, T1_Main_Board:SW_CK_PTS815, symbol Switch:SW_Push
- removed SW6504: Action (part open), Button_Switch_SMD:SW_Push_1P1T_NO_CK_KMR2, symbol Switch:SW_Push
- added D6601, D6602, D6603, D6604: TPD1E10B06, Package_SON:Texas_DPY0002A_0.6x1mm_P0.65mm, symbol Device:D_TVS
- added R6601: 100 kΩ, Resistor_SMD:R_0402_1005Metric, symbol Device:R
- added SW6601, SW6602, SW6603: PTS815, T1_Main_Board:SW_CK_PTS815, symbol Switch:SW_Push
- added SW6604: Action (part open), Button_Switch_SMD:SW_Push_1P1T_NO_CK_KMR2, symbol Switch:SW_Push
Connections:
- net ACTION_BTN_N: now also D6604.2 (A2), SW6604.1
- net GND: now also D6601.1 (A1), D6602.1 (A1), D6603.1 (A1), D6604.1 (A1), SW6601.2, SW6602.2, SW6603.2, SW6604.2
- net PWRON_N: now also D6601.2 (A2), SW6601.1
- net SARADC_VOLUP: now also D6602.2 (A2), SW6602.1
- net VOLDN_N: now also D6603.2 (A2), R6601.2, SW6603.1
- net vcca1v8_pmu: now also R6601.1
Changed lines of the file:
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@@
 (title_block (title "Side buttons") (date "2026-10-25") (rev "A") (company "The OpenDAP Project") (comment 1 "blk.buttons") (comment 2 "Power, Action, Vol+ and Vol-, each with its ESD diode"))
 (symbol (lib_id "Switch:SW_Push") (at 30.48 60.96 270) (unit 1) (body_style 1) (exclude_from_sim no) (in_bom yes) (on_board yes) (dnp no)
-  (property "Reference" "SW6501" (at 36.83 59.69 270) (effects (font (size 1.27 1.27))))
+  (property "Reference" "SW6601" (at 36.83 59.69 270) (effects (font (size 1.27 1.27))))
   (property "Value" "PTS815" (at 36.83 62.23 270) (effects (font (size 1.27 1.27))))
   (property "Footprint" "T1_Main_Board:SW_CK_PTS815" (at 30.48 60.96 0) (effects (font (size 1.27 1.27))) (hide yes))
@@
   (pin "1")
   (pin "2")
-  (instances (project "t1-main-board" (path "/7746052e-d7f9-59ad-ba73-bd2b74439529/afc5e553-cbff-5b60-bd19-e1f58e5228b5" (reference "SW6501") (unit 1))))
+  (instances (project "t1-main-board" (path "/7746052e-d7f9-59ad-ba73-bd2b74439529/afc5e553-cbff-5b60-bd19-e1f58e5228b5" (reference "SW6601") (unit 1))))
 )
 (wire (pts (xy 30.48 55.88) (xy 30.48 53.34)) (stroke (width 0) (type default)))
@@
 )
 (symbol (lib_id "Switch:SW_Push") (at 60.96 60.96 270) (unit 1) (body_style 1) (exclude_from_sim no) (in_bom yes) (on_board yes) (dnp no)
-  (property "Reference" "SW6502" (at 67.31 59.69 270) (effects (font (size 1.27 1.27))))
+  (property "Reference" "SW6602" (at 67.31 59.69 270) (effects (font (size 1.27 1.27))))
   (property "Value" "PTS815" (at 67.31 62.23 270) (effects (font (size 1.27 1.27))))
   (property "Footprint" "T1_Main_Board:SW_CK_PTS815" (at 60.96 60.96 0) (effects (font (size 1.27 1.27))) (hide yes))
@@
   (pin "1")
   (pin "2")
-  (instances (project "t1-main-board" (path "/7746052e-d7f9-59ad-ba73-bd2b74439529/afc5e553-cbff-5b60-bd19-e1f58e5228b5" (reference "SW6502") (unit 1))))
+  (instances (project "t1-main-board" (path "/7746052e-d7f9-59ad-ba73-bd2b74439529/afc5e553-cbff-5b60-bd19-e1f58e5228b5" (reference "SW6602") (unit 1))))
 )
 (wire (pts (xy 60.96 55.88) (xy 60.96 53.34)) (stroke (width 0) (type default)))
@@
 )
 (symbol (lib_id "Switch:SW_Push") (at 91.44 60.96 270) (unit 1) (body_style 1) (exclude_from_sim no) (in_bom yes) (on_board yes) (dnp no)
-  (property "Reference" "SW6503" (at 97.79 59.69 270) (effects (font (size 1.27 1.27))))
+  (property "Reference" "SW6603" (at 97.79 59.69 270) (effects (font (size 1.27 1.27))))
   (property "Value" "PTS815" (at 97.79 62.23 270) (effects (font (size 1.27 1.27))))
   (property "Footprint" "T1_Main_Board:SW_CK_PTS815" (at 91.44 60.96 0) (effects (font (size 1.27 1.27))) (hide yes))
@@
   (pin "1")
   (pin "2")
-  (instances (project "t1-main-board" (path "/7746052e-d7f9-59ad-ba73-bd2b74439529/afc5e553-cbff-5b60-bd19-e1f58e5228b5" (reference "SW6503") (unit 1))))
+  (instances (project "t1-main-board" (path "/7746052e-d7f9-59ad-ba73-bd2b74439529/afc5e553-cbff-5b60-bd19-e1f58e5228b5" (reference "SW6603") (unit 1))))
 )
 (wire (pts (xy 91.44 55.88) (xy 91.44 53.34)) (stroke (width 0) (type default)))
@@
 )
 (symbol (lib_id "Switch:SW_Push") (at 121.92 60.96 270) (unit 1) (body_style 1) (exclude_from_sim no) (in_bom yes) (on_board yes) (dnp no)
-  (property "Reference" "SW6504" (at 128.27 59.69 270) (effects (font (size 1.27 1.27))))
+  (property "Reference" "SW6604" (at 128.27 59.69 270) (effects (font (size 1.27 1.27))))
   (property "Value" "Action (part open)" (at 135.89 62.23 270) (effects (font (size 1.27 1.27))))
   (property "Footprint" "Button_Switch_SMD:SW_Push_1P1T_NO_CK_KMR2" (at 121.92 60.96 0) (effects (font (size 1.27 1.27))) (hide yes))
@@
   (pin "1")
   (pin "2")
-  (instances (project "t1-main-board" (path "/7746052e-d7f9-59ad-ba73-bd2b74439529/afc5e553-cbff-5b60-bd19-e1f58e5228b5" (reference "SW6504") (unit 1))))
+  (instances (project "t1-main-board" (path "/7746052e-d7f9-59ad-ba73-bd2b74439529/afc5e553-cbff-5b60-bd19-e1f58e5228b5" (reference "SW6604") (unit 1))))
 )
 (wire (pts (xy 121.92 55.88) (xy 121.92 53.34)) (stroke (width 0) (type default)))
@@
 (text "Buttons (BOM v1 lines 76, 77)" (exclude_from_sim no) (at 24.13 34.29 0) (effects (font (size 2.54 2.54)) (justify left bottom)))
 (symbol (lib_id "Device:R") (at 176.53 48.26 0) (unit 1) (body_style 1) (exclude_from_sim no) (in_bom yes) (on_board yes) (dnp no)
-  (property "Reference" "R6501" (at 177.8 46.99 0) (effects (font (size 1.27 1.27)) (justify left)))
+  (property "Reference" "R6601" (at 177.8 46.99 0) (effects (font (size 1.27 1.27)) (justify left)))
   (property "Value" "100 kΩ" (at 177.8 49.53 0) (effects (font (size 1.27 1.27)) (justify left)))
   (property "Footprint" "Resistor_SMD:R_0402_1005Metric" (at 176.53 48.26 0) (effects (font (size 1.27 1.27))) (hide yes))
@@
   (pin "1")
   (pin "2")
-  (instances (project "t1-main-board" (path "/7746052e-d7f9-59ad-ba73-bd2b74439529/afc5e553-cbff-5b60-bd19-e1f58e5228b5" (reference "R6501") (unit 1))))
+  (instances (project "t1-main-board" (path "/7746052e-d7f9-59ad-ba73-bd2b74439529/afc5e553-cbff-5b60-bd19-e1f58e5228b5" (reference "R6601") (unit 1))))
 )
 (wire (pts (xy 176.53 44.45) (xy 176.53 41.91)) (stroke (width 0) (type default)))
@@
 (text "Vol- pull-up 100 kΩ (pinout v1 §4)" (exclude_from_sim no) (at 165.1 34.29 0) (effects (font (size 2.54 2.54)) (justify left bottom)))
 (symbol (lib_id "Device:D_TVS") (at 30.48 113.03 90) (unit 1) (body_style 1) (exclude_from_sim no) (in_bom yes) (on_board yes) (dnp no)
-  (property "Reference" "D6501" (at 35.92 111.76 90) (effects (font (size 1.27 1.27))))
+  (property "Reference" "D6601" (at 35.92 111.76 90) (effects (font (size 1.27 1.27))))
   (property "Value" "TPD1E10B06" (at 38.82 114.3 90) (effects (font (size 1.27 1.27))))
   (property "Footprint" "Package_SON:Texas_DPY0002A_0.6x1mm_P0.65mm" (at 30.48 113.03 0) (effects (font (size 1.27 1.27))) (hide yes))
@@
   (pin "1")
   (pin "2")
-  (instances (project "t1-main-board" (path "/7746052e-d7f9-59ad-ba73-bd2b74439529/afc5e553-cbff-5b60-bd19-e1f58e5228b5" (reference "D6501") (unit 1))))
+  (instances (project "t1-main-board" (path "/7746052e-d7f9-59ad-ba73-bd2b74439529/afc5e553-cbff-5b60-bd19-e1f58e5228b5" (reference "D6601") (unit 1))))
 )
 (wire (pts (xy 30.48 109.22) (xy 30.48 106.68)) (stroke (width 0) (type default)))
@@
 )
 (symbol (lib_id "Device:D_TVS") (at 53.34 113.03 90) (unit 1) (body_style 1) (exclude_from_sim no) (in_bom yes) (on_board yes) (dnp no)
-  (property "Reference" "D6502" (at 58.78 111.76 90) (effects (font (size 1.27 1.27))))
+  (property "Reference" "D6602" (at 58.78 111.76 90) (effects (font (size 1.27 1.27))))
   (property "Value" "TPD1E10B06" (at 61.68 114.3 90) (effects (font (size 1.27 1.27))))
   (property "Footprint" "Package_SON:Texas_DPY0002A_0.6x1mm_P0.65mm" (at 53.34 113.03 0) (effects (font (size 1.27 1.27))) (hide yes))
@@
   (pin "1")
   (pin "2")
-  (instances (project "t1-main-board" (path "/7746052e-d7f9-59ad-ba73-bd2b74439529/afc5e553-cbff-5b60-bd19-e1f58e5228b5" (reference "D6502") (unit 1))))
+  (instances (project "t1-main-board" (path "/7746052e-d7f9-59ad-ba73-bd2b74439529/afc5e553-cbff-5b60-bd19-e1f58e5228b5" (reference "D6602") (unit 1))))
 )
 (wire (pts (xy 53.34 109.22) (xy 53.34 106.68)) (stroke (width 0) (type default)))
@@
 )
 (symbol (lib_id "Device:D_TVS") (at 76.2 113.03 90) (unit 1) (body_style 1) (exclude_from_sim no) (in_bom yes) (on_board yes) (dnp no)
-  (property "Reference" "D6503" (at 81.64 111.76 90) (effects (font (size 1.27 1.27))))
+  (property "Reference" "D6603" (at 81.64 111.76 90) (effects (font (size 1.27 1.27))))
   (property "Value" "TPD1E10B06" (at 84.54 114.3 90) (effects (font (size 1.27 1.27))))
   (property "Footprint" "Package_SON:Texas_DPY0002A_0.6x1mm_P0.65mm" (at 76.2 113.03 0) (effects (font (size 1.27 1.27))) (hide yes))
@@
   (pin "1")
   (pin "2")
-  (instances (project "t1-main-board" (path "/7746052e-d7f9-59ad-ba73-bd2b74439529/afc5e553-cbff-5b60-bd19-e1f58e5228b5" (reference "D6503") (unit 1))))
+  (instances (project "t1-main-board" (path "/7746052e-d7f9-59ad-ba73-bd2b74439529/afc5e553-cbff-5b60-bd19-e1f58e5228b5" (reference "D6603") (unit 1))))
 )
 (wire (pts (xy 76.2 109.22) (xy 76.2 106.68)) (stroke (width 0) (type default)))
@@
 )
 (symbol (lib_id "Device:D_TVS") (at 99.06 113.03 90) (unit 1) (body_style 1) (exclude_from_sim no) (in_bom yes) (on_board yes) (dnp no)
-  (property "Reference" "D6504" (at 104.5 111.76 90) (effects (font (size 1.27 1.27))))
+  (property "Reference" "D6604" (at 104.5 111.76 90) (effects (font (size 1.27 1.27))))
   (property "Value" "TPD1E10B06" (at 107.4 114.3 90) (effects (font (size 1.27 1.27))))
   (property "Footprint" "Package_SON:Texas_DPY0002A_0.6x1mm_P0.65mm" (at 99.06 113.03 0) (effects (font (size 1.27 1.27))) (hide yes))
@@
   (pin "1")
   (pin "2")
-  (instances (project "t1-main-board" (path "/7746052e-d7f9-59ad-ba73-bd2b74439529/afc5e553-cbff-5b60-bd19-e1f58e5228b5" (reference "D6504") (unit 1))))
+  (instances (project "t1-main-board" (path "/7746052e-d7f9-59ad-ba73-bd2b74439529/afc5e553-cbff-5b60-bd19-e1f58e5228b5" (reference "D6604") (unit 1))))
 )
 (wire (pts (xy 99.06 109.22) (xy 99.06 106.68)) (stroke (width 0) (type default)))

Commit message: Board: capture blk.cover-detect
COVER_DET_N on GPIO0_A6 (AJ38, PMUIO1, wake-capable), recorded in
pinout v1 (closes feature blocks G22): board-edge input and ground pads
for the case's actuator, 100 kΩ to vcc3v3_pmu, TPD1E10B06 at the pad
(BOM v1 line 143, PCB-L-10). The line rides the KEYS bus with the
buttons.

Co-Authored-By: Claude Opus 5.5 <noreply@anthropic.com>
Claude-Session: https://claude.ai/code/session_01Ei262h3TpgY9vyfNLMi5Mn
Parts:
- removed D6601, D6602, D6603, D6604: TPD1E10B06, Package_SON:Texas_DPY0002A_0.6x1mm_P0.65mm, symbol Device:D_TVS
- removed R6601: 100 kΩ, Resistor_SMD:R_0402_1005Metric, symbol Device:R
- removed SW6601, SW6602, SW6603: PTS815, T1_Main_Board:SW_CK_PTS815, symbol Switch:SW_Push
- removed SW6604: Action (part open), Button_Switch_SMD:SW_Push_1P1T_NO_CK_KMR2, symbol Switch:SW_Push
- added D6701, D6702, D6703, D6704: TPD1E10B06, Package_SON:Texas_DPY0002A_0.6x1mm_P0.65mm, symbol Device:D_TVS
- added R6701: 100 kΩ, Resistor_SMD:R_0402_1005Metric, symbol Device:R
- added SW6701, SW6702, SW6703: PTS815, T1_Main_Board:SW_CK_PTS815, symbol Switch:SW_Push
- added SW6704: Action (part open), Button_Switch_SMD:SW_Push_1P1T_NO_CK_KMR2, symbol Switch:SW_Push
Connections:
- net ACTION_BTN_N: now also D6704.2 (A2), SW6704.1
- net GND: now also D6701.1 (A1), D6702.1 (A1), D6703.1 (A1), D6704.1 (A1), SW6701.2, SW6702.2, SW6703.2, SW6704.2
- net PWRON_N: now also D6701.2 (A2), SW6701.1
- net SARADC_VOLUP: now also D6702.2 (A2), SW6702.1
- net VOLDN_N: now also D6703.2 (A2), R6701.2, SW6703.1
- net vcca1v8_pmu: now also R6701.1
Changed lines of the file:
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@@
 (title_block (title "Side buttons") (date "2026-10-25") (rev "A") (company "The OpenDAP Project") (comment 1 "blk.buttons") (comment 2 "Power, Action, Vol+ and Vol-, each with its ESD diode"))
 (symbol (lib_id "Switch:SW_Push") (at 30.48 60.96 270) (unit 1) (body_style 1) (exclude_from_sim no) (in_bom yes) (on_board yes) (dnp no)
-  (property "Reference" "SW6601" (at 36.83 59.69 270) (effects (font (size 1.27 1.27))))
+  (property "Reference" "SW6701" (at 36.83 59.69 270) (effects (font (size 1.27 1.27))))
   (property "Value" "PTS815" (at 36.83 62.23 270) (effects (font (size 1.27 1.27))))
   (property "Footprint" "T1_Main_Board:SW_CK_PTS815" (at 30.48 60.96 0) (effects (font (size 1.27 1.27))) (hide yes))
@@
   (pin "1")
   (pin "2")
-  (instances (project "t1-main-board" (path "/7746052e-d7f9-59ad-ba73-bd2b74439529/afc5e553-cbff-5b60-bd19-e1f58e5228b5" (reference "SW6601") (unit 1))))
+  (instances (project "t1-main-board" (path "/7746052e-d7f9-59ad-ba73-bd2b74439529/afc5e553-cbff-5b60-bd19-e1f58e5228b5" (reference "SW6701") (unit 1))))
 )
 (wire (pts (xy 30.48 55.88) (xy 30.48 53.34)) (stroke (width 0) (type default)))
@@
 )
 (symbol (lib_id "Switch:SW_Push") (at 60.96 60.96 270) (unit 1) (body_style 1) (exclude_from_sim no) (in_bom yes) (on_board yes) (dnp no)
-  (property "Reference" "SW6602" (at 67.31 59.69 270) (effects (font (size 1.27 1.27))))
+  (property "Reference" "SW6702" (at 67.31 59.69 270) (effects (font (size 1.27 1.27))))
   (property "Value" "PTS815" (at 67.31 62.23 270) (effects (font (size 1.27 1.27))))
   (property "Footprint" "T1_Main_Board:SW_CK_PTS815" (at 60.96 60.96 0) (effects (font (size 1.27 1.27))) (hide yes))
@@
   (pin "1")
   (pin "2")
-  (instances (project "t1-main-board" (path "/7746052e-d7f9-59ad-ba73-bd2b74439529/afc5e553-cbff-5b60-bd19-e1f58e5228b5" (reference "SW6602") (unit 1))))
+  (instances (project "t1-main-board" (path "/7746052e-d7f9-59ad-ba73-bd2b74439529/afc5e553-cbff-5b60-bd19-e1f58e5228b5" (reference "SW6702") (unit 1))))
 )
 (wire (pts (xy 60.96 55.88) (xy 60.96 53.34)) (stroke (width 0) (type default)))
@@
 )
 (symbol (lib_id "Switch:SW_Push") (at 91.44 60.96 270) (unit 1) (body_style 1) (exclude_from_sim no) (in_bom yes) (on_board yes) (dnp no)
-  (property "Reference" "SW6603" (at 97.79 59.69 270) (effects (font (size 1.27 1.27))))
+  (property "Reference" "SW6703" (at 97.79 59.69 270) (effects (font (size 1.27 1.27))))
   (property "Value" "PTS815" (at 97.79 62.23 270) (effects (font (size 1.27 1.27))))
   (property "Footprint" "T1_Main_Board:SW_CK_PTS815" (at 91.44 60.96 0) (effects (font (size 1.27 1.27))) (hide yes))
@@
   (pin "1")
   (pin "2")
-  (instances (project "t1-main-board" (path "/7746052e-d7f9-59ad-ba73-bd2b74439529/afc5e553-cbff-5b60-bd19-e1f58e5228b5" (reference "SW6603") (unit 1))))
+  (instances (project "t1-main-board" (path "/7746052e-d7f9-59ad-ba73-bd2b74439529/afc5e553-cbff-5b60-bd19-e1f58e5228b5" (reference "SW6703") (unit 1))))
 )
 (wire (pts (xy 91.44 55.88) (xy 91.44 53.34)) (stroke (width 0) (type default)))
@@
 )
 (symbol (lib_id "Switch:SW_Push") (at 121.92 60.96 270) (unit 1) (body_style 1) (exclude_from_sim no) (in_bom yes) (on_board yes) (dnp no)
-  (property "Reference" "SW6604" (at 128.27 59.69 270) (effects (font (size 1.27 1.27))))
+  (property "Reference" "SW6704" (at 128.27 59.69 270) (effects (font (size 1.27 1.27))))
   (property "Value" "Action (part open)" (at 135.89 62.23 270) (effects (font (size 1.27 1.27))))
   (property "Footprint" "Button_Switch_SMD:SW_Push_1P1T_NO_CK_KMR2" (at 121.92 60.96 0) (effects (font (size 1.27 1.27))) (hide yes))
@@
   (pin "1")
   (pin "2")
-  (instances (project "t1-main-board" (path "/7746052e-d7f9-59ad-ba73-bd2b74439529/afc5e553-cbff-5b60-bd19-e1f58e5228b5" (reference "SW6604") (unit 1))))
+  (instances (project "t1-main-board" (path "/7746052e-d7f9-59ad-ba73-bd2b74439529/afc5e553-cbff-5b60-bd19-e1f58e5228b5" (reference "SW6704") (unit 1))))
 )
 (wire (pts (xy 121.92 55.88) (xy 121.92 53.34)) (stroke (width 0) (type default)))
@@
 (text "Buttons (BOM v1 lines 76, 77)" (exclude_from_sim no) (at 24.13 34.29 0) (effects (font (size 2.54 2.54)) (justify left bottom)))
 (symbol (lib_id "Device:R") (at 176.53 48.26 0) (unit 1) (body_style 1) (exclude_from_sim no) (in_bom yes) (on_board yes) (dnp no)
-  (property "Reference" "R6601" (at 177.8 46.99 0) (effects (font (size 1.27 1.27)) (justify left)))
+  (property "Reference" "R6701" (at 177.8 46.99 0) (effects (font (size 1.27 1.27)) (justify left)))
   (property "Value" "100 kΩ" (at 177.8 49.53 0) (effects (font (size 1.27 1.27)) (justify left)))
   (property "Footprint" "Resistor_SMD:R_0402_1005Metric" (at 176.53 48.26 0) (effects (font (size 1.27 1.27))) (hide yes))
@@
   (pin "1")
   (pin "2")
-  (instances (project "t1-main-board" (path "/7746052e-d7f9-59ad-ba73-bd2b74439529/afc5e553-cbff-5b60-bd19-e1f58e5228b5" (reference "R6601") (unit 1))))
+  (instances (project "t1-main-board" (path "/7746052e-d7f9-59ad-ba73-bd2b74439529/afc5e553-cbff-5b60-bd19-e1f58e5228b5" (reference "R6701") (unit 1))))
 )
 (wire (pts (xy 176.53 44.45) (xy 176.53 41.91)) (stroke (width 0) (type default)))
@@
 (text "Vol- pull-up 100 kΩ (pinout v1 §4)" (exclude_from_sim no) (at 165.1 34.29 0) (effects (font (size 2.54 2.54)) (justify left bottom)))
 (symbol (lib_id "Device:D_TVS") (at 30.48 113.03 90) (unit 1) (body_style 1) (exclude_from_sim no) (in_bom yes) (on_board yes) (dnp no)
-  (property "Reference" "D6601" (at 35.92 111.76 90) (effects (font (size 1.27 1.27))))
+  (property "Reference" "D6701" (at 35.92 111.76 90) (effects (font (size 1.27 1.27))))
   (property "Value" "TPD1E10B06" (at 38.82 114.3 90) (effects (font (size 1.27 1.27))))
   (property "Footprint" "Package_SON:Texas_DPY0002A_0.6x1mm_P0.65mm" (at 30.48 113.03 0) (effects (font (size 1.27 1.27))) (hide yes))
@@
   (pin "1")
   (pin "2")
-  (instances (project "t1-main-board" (path "/7746052e-d7f9-59ad-ba73-bd2b74439529/afc5e553-cbff-5b60-bd19-e1f58e5228b5" (reference "D6601") (unit 1))))
+  (instances (project "t1-main-board" (path "/7746052e-d7f9-59ad-ba73-bd2b74439529/afc5e553-cbff-5b60-bd19-e1f58e5228b5" (reference "D6701") (unit 1))))
 )
 (wire (pts (xy 30.48 109.22) (xy 30.48 106.68)) (stroke (width 0) (type default)))
@@
 )
 (symbol (lib_id "Device:D_TVS") (at 53.34 113.03 90) (unit 1) (body_style 1) (exclude_from_sim no) (in_bom yes) (on_board yes) (dnp no)
-  (property "Reference" "D6602" (at 58.78 111.76 90) (effects (font (size 1.27 1.27))))
+  (property "Reference" "D6702" (at 58.78 111.76 90) (effects (font (size 1.27 1.27))))
   (property "Value" "TPD1E10B06" (at 61.68 114.3 90) (effects (font (size 1.27 1.27))))
   (property "Footprint" "Package_SON:Texas_DPY0002A_0.6x1mm_P0.65mm" (at 53.34 113.03 0) (effects (font (size 1.27 1.27))) (hide yes))
@@
   (pin "1")
   (pin "2")
-  (instances (project "t1-main-board" (path "/7746052e-d7f9-59ad-ba73-bd2b74439529/afc5e553-cbff-5b60-bd19-e1f58e5228b5" (reference "D6602") (unit 1))))
+  (instances (project "t1-main-board" (path "/7746052e-d7f9-59ad-ba73-bd2b74439529/afc5e553-cbff-5b60-bd19-e1f58e5228b5" (reference "D6702") (unit 1))))
 )
 (wire (pts (xy 53.34 109.22) (xy 53.34 106.68)) (stroke (width 0) (type default)))
@@
 )
 (symbol (lib_id "Device:D_TVS") (at 76.2 113.03 90) (unit 1) (body_style 1) (exclude_from_sim no) (in_bom yes) (on_board yes) (dnp no)
-  (property "Reference" "D6603" (at 81.64 111.76 90) (effects (font (size 1.27 1.27))))
+  (property "Reference" "D6703" (at 81.64 111.76 90) (effects (font (size 1.27 1.27))))
   (property "Value" "TPD1E10B06" (at 84.54 114.3 90) (effects (font (size 1.27 1.27))))
   (property "Footprint" "Package_SON:Texas_DPY0002A_0.6x1mm_P0.65mm" (at 76.2 113.03 0) (effects (font (size 1.27 1.27))) (hide yes))
@@
   (pin "1")
   (pin "2")
-  (instances (project "t1-main-board" (path "/7746052e-d7f9-59ad-ba73-bd2b74439529/afc5e553-cbff-5b60-bd19-e1f58e5228b5" (reference "D6603") (unit 1))))
+  (instances (project "t1-main-board" (path "/7746052e-d7f9-59ad-ba73-bd2b74439529/afc5e553-cbff-5b60-bd19-e1f58e5228b5" (reference "D6703") (unit 1))))
 )
 (wire (pts (xy 76.2 109.22) (xy 76.2 106.68)) (stroke (width 0) (type default)))
@@
 )
 (symbol (lib_id "Device:D_TVS") (at 99.06 113.03 90) (unit 1) (body_style 1) (exclude_from_sim no) (in_bom yes) (on_board yes) (dnp no)
-  (property "Reference" "D6604" (at 104.5 111.76 90) (effects (font (size 1.27 1.27))))
+  (property "Reference" "D6704" (at 104.5 111.76 90) (effects (font (size 1.27 1.27))))
   (property "Value" "TPD1E10B06" (at 107.4 114.3 90) (effects (font (size 1.27 1.27))))
   (property "Footprint" "Package_SON:Texas_DPY0002A_0.6x1mm_P0.65mm" (at 99.06 113.03 0) (effects (font (size 1.27 1.27))) (hide yes))
@@
   (pin "1")
   (pin "2")
-  (instances (project "t1-main-board" (path "/7746052e-d7f9-59ad-ba73-bd2b74439529/afc5e553-cbff-5b60-bd19-e1f58e5228b5" (reference "D6604") (unit 1))))
+  (instances (project "t1-main-board" (path "/7746052e-d7f9-59ad-ba73-bd2b74439529/afc5e553-cbff-5b60-bd19-e1f58e5228b5" (reference "D6704") (unit 1))))
 )
 (wire (pts (xy 99.06 109.22) (xy 99.06 106.68)) (stroke (width 0) (type default)))
