File: board/hardware/t1-main-board/buttons.kicad_sch (KiCad schematic)
At the start: 9 parts, among them SW6701 PTS815, SW6702 PTS815, SW6703 PTS815, SW6704 Action (part open)

Commit message: Board: capture blk.mic-ambient and links #34, #35
IM73D122 on PDM CLK1 and SDI1 (BOM v1 line 34, pinout v1 AK2 and 1P2),
LR to ground, 22 Ω clock series, VDD from MIC_1V8 through link #35.
Link #34 on blk.mic-main makes the faceplate branch the rail MIC_1V8_FP
for contact 40 (power tree §4.12, G10). kicad-lib moves to e46bda4 for
the IM73D122, TPS3808G01, SN74LVC1G58 and BAT54 parts.

Co-Authored-By: Claude Opus 5.5 <noreply@anthropic.com>
Claude-Session: https://claude.ai/code/session_01Ei262h3TpgY9vyfNLMi5Mn
Parts:
- removed D6701, D6702, D6703, D6704: TPD1E10B06, Package_SON:Texas_DPY0002A_0.6x1mm_P0.65mm, symbol Device:D_TVS
- removed R6701: 100 kΩ, Resistor_SMD:R_0402_1005Metric, symbol Device:R
- removed SW6701, SW6702, SW6703: PTS815, T1_Main_Board:SW_CK_PTS815, symbol Switch:SW_Push
- removed SW6704: Action (part open), Button_Switch_SMD:SW_Push_1P1T_NO_CK_KMR2, symbol Switch:SW_Push
- added D6801, D6802, D6803, D6804: TPD1E10B06, Package_SON:Texas_DPY0002A_0.6x1mm_P0.65mm, symbol Device:D_TVS
- added R6801: 100 kΩ, Resistor_SMD:R_0402_1005Metric, symbol Device:R
- added SW6801, SW6802, SW6803: PTS815, T1_Main_Board:SW_CK_PTS815, symbol Switch:SW_Push
- added SW6804: Action (part open), Button_Switch_SMD:SW_Push_1P1T_NO_CK_KMR2, symbol Switch:SW_Push
Connections:
- net ACTION_BTN_N: now also D6804.2 (A2), SW6804.1
- net GND: now also D6801.1 (A1), D6802.1 (A1), D6803.1 (A1), D6804.1 (A1), SW6801.2, SW6802.2, SW6803.2, SW6804.2
- net PWRON_N: now also D6801.2 (A2), SW6801.1
- net SARADC_VOLUP: now also D6802.2 (A2), SW6802.1
- net VOLDN_N: now also D6803.2 (A2), R6801.2, SW6803.1
- net vcca1v8_pmu: now also R6801.1

Commit message: Board: capture blk.maskrom
Power + Vol- at a cold power-on pull eMMC D0 low inside the TPS3808G01
boot window (BOM v1 lines 35, 78, 97, 98; sim/maskrom): SENSE 280k/100k,
CT 390 nF, WINDOW_N with its pad, SN74LVC1G57 and SN74LVC1G58 on
vcca1v8_pmu, BAT54 from PWRON_N, DMG1012T through 1 kΩ to EMMC_D0.
Every block in use now has its sheet; the README states the remaining
single-pin nets.

Co-Authored-By: Claude Opus 5.5 <noreply@anthropic.com>
Claude-Session: https://claude.ai/code/session_01Ei262h3TpgY9vyfNLMi5Mn
Parts:
- removed D6801, D6802, D6803, D6804: TPD1E10B06, Package_SON:Texas_DPY0002A_0.6x1mm_P0.65mm, symbol Device:D_TVS
- removed R6801: 100 kΩ, Resistor_SMD:R_0402_1005Metric, symbol Device:R
- removed SW6801, SW6802, SW6803: PTS815, T1_Main_Board:SW_CK_PTS815, symbol Switch:SW_Push
- removed SW6804: Action (part open), Button_Switch_SMD:SW_Push_1P1T_NO_CK_KMR2, symbol Switch:SW_Push
- added D6901, D6902, D6903, D6904: TPD1E10B06, Package_SON:Texas_DPY0002A_0.6x1mm_P0.65mm, symbol Device:D_TVS
- added R6901: 100 kΩ, Resistor_SMD:R_0402_1005Metric, symbol Device:R
- added SW6901, SW6902, SW6903: PTS815, T1_Main_Board:SW_CK_PTS815, symbol Switch:SW_Push
- added SW6904: Action (part open), Button_Switch_SMD:SW_Push_1P1T_NO_CK_KMR2, symbol Switch:SW_Push
Connections:
- net ACTION_BTN_N: now also D6904.2 (A2), SW6904.1
- net GND: now also D6901.1 (A1), D6902.1 (A1), D6903.1 (A1), D6904.1 (A1), SW6901.2, SW6902.2, SW6903.2, SW6904.2
- net PWRON_N: now also D6901.2 (A2), SW6901.1
- net SARADC_VOLUP: now also D6902.2 (A2), SW6902.1
- net VOLDN_N: now also D6903.2 (A2), R6901.2, SW6903.1
- net vcca1v8_pmu: now also R6901.1
Changed lines of the file:
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@@
 (title_block (title "Side buttons") (date "2026-10-25") (rev "A") (company "The OpenDAP Project") (comment 1 "blk.buttons") (comment 2 "Power, Action, Vol+ and Vol-, each with its ESD diode"))
 (symbol (lib_id "Switch:SW_Push") (at 30.48 60.96 270) (unit 1) (body_style 1) (exclude_from_sim no) (in_bom yes) (on_board yes) (dnp no)
-  (property "Reference" "SW6801" (at 36.83 59.69 270) (effects (font (size 1.27 1.27))))
+  (property "Reference" "SW6901" (at 36.83 59.69 270) (effects (font (size 1.27 1.27))))
   (property "Value" "PTS815" (at 36.83 62.23 270) (effects (font (size 1.27 1.27))))
   (property "Footprint" "T1_Main_Board:SW_CK_PTS815" (at 30.48 60.96 0) (effects (font (size 1.27 1.27))) (hide yes))
@@
   (pin "1")
   (pin "2")
-  (instances (project "t1-main-board" (path "/7746052e-d7f9-59ad-ba73-bd2b74439529/afc5e553-cbff-5b60-bd19-e1f58e5228b5" (reference "SW6801") (unit 1))))
+  (instances (project "t1-main-board" (path "/7746052e-d7f9-59ad-ba73-bd2b74439529/afc5e553-cbff-5b60-bd19-e1f58e5228b5" (reference "SW6901") (unit 1))))
 )
 (wire (pts (xy 30.48 55.88) (xy 30.48 53.34)) (stroke (width 0) (type default)))
@@
 )
 (symbol (lib_id "Switch:SW_Push") (at 60.96 60.96 270) (unit 1) (body_style 1) (exclude_from_sim no) (in_bom yes) (on_board yes) (dnp no)
-  (property "Reference" "SW6802" (at 67.31 59.69 270) (effects (font (size 1.27 1.27))))
+  (property "Reference" "SW6902" (at 67.31 59.69 270) (effects (font (size 1.27 1.27))))
   (property "Value" "PTS815" (at 67.31 62.23 270) (effects (font (size 1.27 1.27))))
   (property "Footprint" "T1_Main_Board:SW_CK_PTS815" (at 60.96 60.96 0) (effects (font (size 1.27 1.27))) (hide yes))
@@
   (pin "1")
   (pin "2")
-  (instances (project "t1-main-board" (path "/7746052e-d7f9-59ad-ba73-bd2b74439529/afc5e553-cbff-5b60-bd19-e1f58e5228b5" (reference "SW6802") (unit 1))))
+  (instances (project "t1-main-board" (path "/7746052e-d7f9-59ad-ba73-bd2b74439529/afc5e553-cbff-5b60-bd19-e1f58e5228b5" (reference "SW6902") (unit 1))))
 )
 (wire (pts (xy 60.96 55.88) (xy 60.96 53.34)) (stroke (width 0) (type default)))
@@
 )
 (symbol (lib_id "Switch:SW_Push") (at 91.44 60.96 270) (unit 1) (body_style 1) (exclude_from_sim no) (in_bom yes) (on_board yes) (dnp no)
-  (property "Reference" "SW6803" (at 97.79 59.69 270) (effects (font (size 1.27 1.27))))
+  (property "Reference" "SW6903" (at 97.79 59.69 270) (effects (font (size 1.27 1.27))))
   (property "Value" "PTS815" (at 97.79 62.23 270) (effects (font (size 1.27 1.27))))
   (property "Footprint" "T1_Main_Board:SW_CK_PTS815" (at 91.44 60.96 0) (effects (font (size 1.27 1.27))) (hide yes))
@@
   (pin "1")
   (pin "2")
-  (instances (project "t1-main-board" (path "/7746052e-d7f9-59ad-ba73-bd2b74439529/afc5e553-cbff-5b60-bd19-e1f58e5228b5" (reference "SW6803") (unit 1))))
+  (instances (project "t1-main-board" (path "/7746052e-d7f9-59ad-ba73-bd2b74439529/afc5e553-cbff-5b60-bd19-e1f58e5228b5" (reference "SW6903") (unit 1))))
 )
 (wire (pts (xy 91.44 55.88) (xy 91.44 53.34)) (stroke (width 0) (type default)))
@@
 )
 (symbol (lib_id "Switch:SW_Push") (at 121.92 60.96 270) (unit 1) (body_style 1) (exclude_from_sim no) (in_bom yes) (on_board yes) (dnp no)
-  (property "Reference" "SW6804" (at 128.27 59.69 270) (effects (font (size 1.27 1.27))))
+  (property "Reference" "SW6904" (at 128.27 59.69 270) (effects (font (size 1.27 1.27))))
   (property "Value" "Action (part open)" (at 135.89 62.23 270) (effects (font (size 1.27 1.27))))
   (property "Footprint" "Button_Switch_SMD:SW_Push_1P1T_NO_CK_KMR2" (at 121.92 60.96 0) (effects (font (size 1.27 1.27))) (hide yes))
@@
   (pin "1")
   (pin "2")
-  (instances (project "t1-main-board" (path "/7746052e-d7f9-59ad-ba73-bd2b74439529/afc5e553-cbff-5b60-bd19-e1f58e5228b5" (reference "SW6804") (unit 1))))
+  (instances (project "t1-main-board" (path "/7746052e-d7f9-59ad-ba73-bd2b74439529/afc5e553-cbff-5b60-bd19-e1f58e5228b5" (reference "SW6904") (unit 1))))
 )
 (wire (pts (xy 121.92 55.88) (xy 121.92 53.34)) (stroke (width 0) (type default)))
@@
 (text "Buttons (BOM v1 lines 76, 77)" (exclude_from_sim no) (at 24.13 34.29 0) (effects (font (size 2.54 2.54)) (justify left bottom)))
 (symbol (lib_id "Device:R") (at 176.53 48.26 0) (unit 1) (body_style 1) (exclude_from_sim no) (in_bom yes) (on_board yes) (dnp no)
-  (property "Reference" "R6801" (at 177.8 46.99 0) (effects (font (size 1.27 1.27)) (justify left)))
+  (property "Reference" "R6901" (at 177.8 46.99 0) (effects (font (size 1.27 1.27)) (justify left)))
   (property "Value" "100 kΩ" (at 177.8 49.53 0) (effects (font (size 1.27 1.27)) (justify left)))
   (property "Footprint" "Resistor_SMD:R_0402_1005Metric" (at 176.53 48.26 0) (effects (font (size 1.27 1.27))) (hide yes))
@@
   (pin "1")
   (pin "2")
-  (instances (project "t1-main-board" (path "/7746052e-d7f9-59ad-ba73-bd2b74439529/afc5e553-cbff-5b60-bd19-e1f58e5228b5" (reference "R6801") (unit 1))))
+  (instances (project "t1-main-board" (path "/7746052e-d7f9-59ad-ba73-bd2b74439529/afc5e553-cbff-5b60-bd19-e1f58e5228b5" (reference "R6901") (unit 1))))
 )
 (wire (pts (xy 176.53 44.45) (xy 176.53 41.91)) (stroke (width 0) (type default)))
@@
 (text "Vol- pull-up 100 kΩ (pinout v1 §4)" (exclude_from_sim no) (at 165.1 34.29 0) (effects (font (size 2.54 2.54)) (justify left bottom)))
 (symbol (lib_id "Device:D_TVS") (at 30.48 113.03 90) (unit 1) (body_style 1) (exclude_from_sim no) (in_bom yes) (on_board yes) (dnp no)
-  (property "Reference" "D6801" (at 35.92 111.76 90) (effects (font (size 1.27 1.27))))
+  (property "Reference" "D6901" (at 35.92 111.76 90) (effects (font (size 1.27 1.27))))
   (property "Value" "TPD1E10B06" (at 38.82 114.3 90) (effects (font (size 1.27 1.27))))
   (property "Footprint" "Package_SON:Texas_DPY0002A_0.6x1mm_P0.65mm" (at 30.48 113.03 0) (effects (font (size 1.27 1.27))) (hide yes))
@@
   (pin "1")
   (pin "2")
-  (instances (project "t1-main-board" (path "/7746052e-d7f9-59ad-ba73-bd2b74439529/afc5e553-cbff-5b60-bd19-e1f58e5228b5" (reference "D6801") (unit 1))))
+  (instances (project "t1-main-board" (path "/7746052e-d7f9-59ad-ba73-bd2b74439529/afc5e553-cbff-5b60-bd19-e1f58e5228b5" (reference "D6901") (unit 1))))
 )
 (wire (pts (xy 30.48 109.22) (xy 30.48 106.68)) (stroke (width 0) (type default)))
@@
 )
 (symbol (lib_id "Device:D_TVS") (at 53.34 113.03 90) (unit 1) (body_style 1) (exclude_from_sim no) (in_bom yes) (on_board yes) (dnp no)
-  (property "Reference" "D6802" (at 58.78 111.76 90) (effects (font (size 1.27 1.27))))
+  (property "Reference" "D6902" (at 58.78 111.76 90) (effects (font (size 1.27 1.27))))
   (property "Value" "TPD1E10B06" (at 61.68 114.3 90) (effects (font (size 1.27 1.27))))
   (property "Footprint" "Package_SON:Texas_DPY0002A_0.6x1mm_P0.65mm" (at 53.34 113.03 0) (effects (font (size 1.27 1.27))) (hide yes))
@@
   (pin "1")
   (pin "2")
-  (instances (project "t1-main-board" (path "/7746052e-d7f9-59ad-ba73-bd2b74439529/afc5e553-cbff-5b60-bd19-e1f58e5228b5" (reference "D6802") (unit 1))))
+  (instances (project "t1-main-board" (path "/7746052e-d7f9-59ad-ba73-bd2b74439529/afc5e553-cbff-5b60-bd19-e1f58e5228b5" (reference "D6902") (unit 1))))
 )
 (wire (pts (xy 53.34 109.22) (xy 53.34 106.68)) (stroke (width 0) (type default)))
@@
 )
 (symbol (lib_id "Device:D_TVS") (at 76.2 113.03 90) (unit 1) (body_style 1) (exclude_from_sim no) (in_bom yes) (on_board yes) (dnp no)
-  (property "Reference" "D6803" (at 81.64 111.76 90) (effects (font (size 1.27 1.27))))
+  (property "Reference" "D6903" (at 81.64 111.76 90) (effects (font (size 1.27 1.27))))
   (property "Value" "TPD1E10B06" (at 84.54 114.3 90) (effects (font (size 1.27 1.27))))
   (property "Footprint" "Package_SON:Texas_DPY0002A_0.6x1mm_P0.65mm" (at 76.2 113.03 0) (effects (font (size 1.27 1.27))) (hide yes))
@@
   (pin "1")
   (pin "2")
-  (instances (project "t1-main-board" (path "/7746052e-d7f9-59ad-ba73-bd2b74439529/afc5e553-cbff-5b60-bd19-e1f58e5228b5" (reference "D6803") (unit 1))))
+  (instances (project "t1-main-board" (path "/7746052e-d7f9-59ad-ba73-bd2b74439529/afc5e553-cbff-5b60-bd19-e1f58e5228b5" (reference "D6903") (unit 1))))
 )
 (wire (pts (xy 76.2 109.22) (xy 76.2 106.68)) (stroke (width 0) (type default)))
@@
 )
 (symbol (lib_id "Device:D_TVS") (at 99.06 113.03 90) (unit 1) (body_style 1) (exclude_from_sim no) (in_bom yes) (on_board yes) (dnp no)
-  (property "Reference" "D6804" (at 104.5 111.76 90) (effects (font (size 1.27 1.27))))
+  (property "Reference" "D6904" (at 104.5 111.76 90) (effects (font (size 1.27 1.27))))
   (property "Value" "TPD1E10B06" (at 107.4 114.3 90) (effects (font (size 1.27 1.27))))
   (property "Footprint" "Package_SON:Texas_DPY0002A_0.6x1mm_P0.65mm" (at 99.06 113.03 0) (effects (font (size 1.27 1.27))) (hide yes))
@@
   (pin "1")
   (pin "2")
-  (instances (project "t1-main-board" (path "/7746052e-d7f9-59ad-ba73-bd2b74439529/afc5e553-cbff-5b60-bd19-e1f58e5228b5" (reference "D6804") (unit 1))))
+  (instances (project "t1-main-board" (path "/7746052e-d7f9-59ad-ba73-bd2b74439529/afc5e553-cbff-5b60-bd19-e1f58e5228b5" (reference "D6904") (unit 1))))
 )
 (wire (pts (xy 99.06 109.22) (xy 99.06 106.68)) (stroke (width 0) (type default)))
