File: board/hardware/t1-main-board/charger-input.kicad_sch (KiCad schematic)
At the start: 17 parts, among them U501 TPS2121RUXR

Commit message: Compaction: lower inductors, 0201 decoupling, 0.8 mm signal test pads
A matrix tool (hardware/studies/compaction) checks each candidate against
the design's stresses: same inductance, design peak <= 70 % and the
converter's maximum limit <= 100 % of Isat (30 % drop), height zones,
ratings at least twice the rail, PCB-D-06; sourcing outcome per part.

Applied (placement v1 decision 12, BOM v1.15):
- L601, L4401: XGL4015-102MEC (1.5 mm) for XAL/XGL4020-102MEC (2.1 mm);
- L1001, L5101: XGL4015-471MEC (1.5 mm) for Wurth 744373240047, on the
  stock XxL4020 land (the Wurth land was never drawn);
- L1201 is 1.2 mm (XGL4012, per-MPN heights): it moves next to the SoC;
- 58 x 100 nF decoupling on rails <= 3.3 V in core/IO/radio: 0201;
- 51 test pads on signal nets: 0.8 mm (PCB-D-06 v0.16, JLCPCB guide).
Kept: L901, L2802 (XGL4015 at 103 % of Isat at the limit); no thinner
0805/1206 capacitor passes (obsolete, NRND or unlisted).

Board need 113 % -> 111 % (core band 227 -> 203 %, power band 258 ->
233 %, radio band 19 -> 0 %); only C904 still relies on PCB-Z-04.
ERC 0 errors, craft Q1 met, DRC 0 errors (605 warnings), pcb and study
tests pass, rules test board PASS.

Co-Authored-By: Claude Opus 5.5 <noreply@anthropic.com>
Claude-Session: https://claude.ai/code/session_01Ei262h3TpgY9vyfNLMi5Mn
Parts:
- TP504: footprint TestPoint:TestPoint_Pad_D1.0mm -> T1_Main_Board:TestPoint_Pad_D0.8mm
Changed lines of the file:
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@@
   (property "Reference" "TP504" (at 137.16 144.78 0) (effects (font (size 1.27 1.27)) (justify right)))
   (property "Value" "MUX_ST" (at 137.16 147.32 0) (effects (font (size 1.27 1.27)) (justify right)))
-  (property "Footprint" "TestPoint:TestPoint_Pad_D1.0mm" (at 138.43 149.86 0) (effects (font (size 1.27 1.27))) (hide yes))
+  (property "Footprint" "T1_Main_Board:TestPoint_Pad_D0.8mm" (at 138.43 149.86 0) (effects (font (size 1.27 1.27))) (hide yes))
   (property "Datasheet" "~" (at 138.43 149.86 0) (effects (font (size 1.27 1.27))) (hide yes))
-  (property "Description" "Test pad, 1.0 mm" (at 138.43 149.86 0) (effects (font (size 1.27 1.27))) (hide yes))
+  (property "Description" "Test pad, 0.8 mm, signal net" (at 138.43 149.86 0) (effects (font (size 1.27 1.27))) (hide yes))
   (property "Block" "blk.charger-input" (at 138.43 149.86 0) (effects (font (size 1.27 1.27))) (hide yes))
   (pin "1")

Commit message: Board on libs v0.2.0: lower-case kebab vendor keys (HL-13)
The libs submodule moves to v0.2.0 (5f24483). Every library nickname in
the generator, the placement tool and the floorplan study follows the
key table (Texas_Instruments -> texas-instruments, OpenDAP_Device ->
opendap-generic, Rockchip and Rockchip_PMIC -> rockchip, ...); the
library tables are written from the files. Schematic and board
regenerated.

Checks: ERC 0 errors (warnings unchanged); DRC 0 errors, 605 warnings,
the same counts by type, schematic parity 0; every placement identical;
craft Q1 met; pcb tests pass; STEP export resolves every libs 3D model
(the 27 parts without a model are KiCad stock lands that have none).

Co-Authored-By: Claude Opus 5.5 <noreply@anthropic.com>
Claude-Session: https://claude.ai/code/session_01Ei262h3TpgY9vyfNLMi5Mn
Parts:
- U501: footprint Texas_Instruments:Texas_RUX0012A_VQFN-HR-12_2x2.5mm_P0.5mm -> texas-instruments:Texas_RUX0012A_VQFN-HR-12_2x2.5mm_P0.5mm; symbol Texas_Instruments:TPS2121RUXR -> texas-instruments:TPS2121RUXR
Changed lines of the file:
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@@
 (paper "A3")
 (title_block (title "Charger: input mux") (date "2026-10-25") (rev "A") (company "The OpenDAP Project") (comment 1 "blk.charger-input") (comment 2 "TPS2121 picks USB-C or the HAT port into VBUS_CHG; the OV interlocks"))
-(symbol (lib_id "Texas_Instruments:TPS2121RUXR") (at 49.53 77.47 0) (unit 1) (body_style 1) (exclude_from_sim no) (in_bom yes) (on_board yes) (dnp no)
+(symbol (lib_id "texas-instruments:TPS2121RUXR") (at 49.53 77.47 0) (unit 1) (body_style 1) (exclude_from_sim no) (in_bom yes) (on_board yes) (dnp no)
   (property "Reference" "U501" (at 53.34 55.88 0) (effects (font (size 1.27 1.27)) (justify left)))
   (property "Value" "TPS2121RUXR" (at 53.34 53.34 0) (effects (font (size 1.27 1.27)) (justify left)))
-  (property "Footprint" "Texas_Instruments:Texas_RUX0012A_VQFN-HR-12_2x2.5mm_P0.5mm" (at 49.53 77.47 0) (effects (font (size 1.27 1.27))) (hide yes))
+  (property "Footprint" "texas-instruments:Texas_RUX0012A_VQFN-HR-12_2x2.5mm_P0.5mm" (at 49.53 77.47 0) (effects (font (size 1.27 1.27))) (hide yes))
   (property "Datasheet" "https://www.ti.com/lit/ds/symlink/tps2121.pdf" (at 49.53 77.47 0) (effects (font (size 1.27 1.27))) (hide yes))
   (property "Description" "2.8-22 V dual-input priority power multiplexer with seamless switchover, 4.5 A, adjustable current limit, VQFN-HR-12 (RUX0012A) 2 x 2.5 mm" (at 49.53 77.47 0) (effects (font (size 1.27 1.27))) (hide yes))
