File: board/hardware/t1-main-board/gpio-expander.kicad_sch (KiCad schematic)
At the start: 13 parts, among them U5101 TCA6416ARTWR

Commit message: Board: capture blk.current-monitors
Five INA236 on I2C1 (0x40-0x43, 0x48) with their shunts, per power tree
§4.12 and BOM v1 lines 54 and 136. The measured branches are rails of
their own (VSYS_SRC, VSYS_LV_AUDIO, VSYS_AUDIO, VSYS_LV_BL, VSYS_P5V1),
fed through the shunts on this sheet; the charger, audio, backlight and
5.1 V sheets take them. The root's layout may leave a stack level empty,
so the block sits under the notes; IC bboxes hold turned rail values;
passive rows hold a bottom rail's text.

Co-Authored-By: Claude Opus 5.5 <noreply@anthropic.com>
Claude-Session: https://claude.ai/code/session_01Ei262h3TpgY9vyfNLMi5Mn
Parts:
- removed C5101, C5102: 100 nF, Capacitor_SMD:C_0402_1005Metric, symbol Device:C
- removed R5101, R5106, R5107, R5108, R5109, R5110: 10 kΩ, Resistor_SMD:R_0402_1005Metric, symbol Device:R
- removed R5102, R5103, R5104, R5105: 100 kΩ, Resistor_SMD:R_0402_1005Metric, symbol Device:R
- removed U5101: TCA6416ARTWR, Texas_Instruments:Texas_RTW0024B_WQFN-24-1EP_4x4mm_P0.5mm_EP2.45x2.45mm_ThermalVias, symbol Texas_Instruments:TCA6416ARTWR
- added C5201, C5202: 100 nF, Capacitor_SMD:C_0402_1005Metric, symbol Device:C
- added R5201, R5206, R5207, R5208, R5209, R5210: 10 kΩ, Resistor_SMD:R_0402_1005Metric, symbol Device:R
- added R5202, R5203, R5204, R5205: 100 kΩ, Resistor_SMD:R_0402_1005Metric, symbol Device:R
- added U5201: TCA6416ARTWR, Texas_Instruments:Texas_RTW0024B_WQFN-24-1EP_4x4mm_P0.5mm_EP2.45x2.45mm_ThermalVias, symbol Texas_Instruments:TCA6416ARTWR
Connections:
- net EFUSE_5V_FLT_N: now also R5209.2, U5201.16 (P16)
- net EFUSE_HAT5V_FLT_N: now also R5208.2, U5201.15 (P15)
- net EFUSE_VBUS_FLT_N: now also R5210.2, U5201.17 (P17)
- net EXP_INT_N: now also U5201.22 (INT)
- net EXP_RESET_N: now also R5201.2, U5201.24 (RESET)
- net FP_DET_N: now also U5201.12 (P12)
- net FP_GPIO0: now also U5201.13 (P13)
- net FP_GPIO1: now also U5201.14 (P14)
- net FP_IO_EN: now also U5201.1 (P00)
- net GND: now also C5201.2, C5202.2, R5202.2, R5203.2, R5204.2, R5205.2, U5201.25 (EP), U5201.9 (GND)
- net HAPTIC_EN: now also R5204.1, U5201.5 (P04)
- net HAT5V_EN: now also R5202.1, U5201.3 (P02)
- net HAT_VBUS_DISCH: now also U5201.2 (P01)
- net HP_DET_BAL: now also R5207.2, U5201.11 (P11)
- net HP_DET_SE: now also R5206.2, U5201.10 (P10)
- net I2C2_SCL: now also U5201.19 (SCL)
- net I2C2_SDA: now also U5201.20 (SDA)
- net NFC_PWR_EN: now also R5205.1, U5201.6 (P05)
- net USB_SRC_ON: now also R5203.1, U5201.4 (P03)
- net WL_PD_HOLD_N: now also U5201.8 (P07)
- net WL_PWR_EN: now also U5201.7 (P06)
- net vcc3v3_sys: now also C5202.1, R5206.1, R5207.1, R5208.1, R5209.1, R5210.1, U5201.18 (ADDR), U5201.21 (VCCP)
- net vcca1v8_pmu: now also C5201.1, R5201.1, U5201.23 (VCCI)

Commit message: Board: capture blk.status-led
LP5521 at 0x32 on I2C2 (BOM v1 line 105) with its charge-pump
capacitors, EN on vcca1v8_pmu, VDD from VSYS_LV through link #22;
LED_R/G/B reach the faceplate connector as the LED bus alias. The
faceplate row of the root is re-packed so five full columns sit left of
the title block.

Co-Authored-By: Claude Opus 5.5 <noreply@anthropic.com>
Claude-Session: https://claude.ai/code/session_01Ei262h3TpgY9vyfNLMi5Mn
Parts:
- removed C5201, C5202: 100 nF, Capacitor_SMD:C_0402_1005Metric, symbol Device:C
- removed R5201, R5206, R5207, R5208, R5209, R5210: 10 kΩ, Resistor_SMD:R_0402_1005Metric, symbol Device:R
- removed R5202, R5203, R5204, R5205: 100 kΩ, Resistor_SMD:R_0402_1005Metric, symbol Device:R
- removed U5201: TCA6416ARTWR, Texas_Instruments:Texas_RTW0024B_WQFN-24-1EP_4x4mm_P0.5mm_EP2.45x2.45mm_ThermalVias, symbol Texas_Instruments:TCA6416ARTWR
- added C6301, C6302: 100 nF, Capacitor_SMD:C_0402_1005Metric, symbol Device:C
- added R6301, R6306, R6307, R6308, R6309, R6310: 10 kΩ, Resistor_SMD:R_0402_1005Metric, symbol Device:R
- added R6302, R6303, R6304, R6305: 100 kΩ, Resistor_SMD:R_0402_1005Metric, symbol Device:R
- added U6301: TCA6416ARTWR, Texas_Instruments:Texas_RTW0024B_WQFN-24-1EP_4x4mm_P0.5mm_EP2.45x2.45mm_ThermalVias, symbol Texas_Instruments:TCA6416ARTWR
Connections:
- net EFUSE_5V_FLT_N: now also R6309.2, U6301.16 (P16)
- net EFUSE_HAT5V_FLT_N: now also R6308.2, U6301.15 (P15)
- net EFUSE_VBUS_FLT_N: now also R6310.2, U6301.17 (P17)
- net EXP_INT_N: now also U6301.22 (INT)
- net EXP_RESET_N: now also R6301.2, U6301.24 (RESET)
- net FP_DET_N: now also U6301.12 (P12)
- net FP_GPIO0: now also U6301.13 (P13)
- net FP_GPIO1: now also U6301.14 (P14)
- net FP_IO_EN: now also U6301.1 (P00)
- net GND: now also C6301.2, C6302.2, R6302.2, R6303.2, R6304.2, R6305.2, U6301.25 (EP), U6301.9 (GND)
- net HAPTIC_EN: now also R6304.1, U6301.5 (P04)
- net HAT5V_EN: now also R6302.1, U6301.3 (P02)
- net HAT_VBUS_DISCH: now also U6301.2 (P01)
- net HP_DET_BAL: now also R6307.2, U6301.11 (P11)
- net HP_DET_SE: now also R6306.2, U6301.10 (P10)
- net I2C2_SCL: now also U6301.19 (SCL)
- net I2C2_SDA: now also U6301.20 (SDA)
- net NFC_PWR_EN: now also R6305.1, U6301.6 (P05)
- net USB_SRC_ON: now also R6303.1, U6301.4 (P03)
- net WL_PD_HOLD_N: now also U6301.8 (P07)
- net WL_PWR_EN: now also U6301.7 (P06)
- net vcc3v3_sys: now also C6302.1, R6306.1, R6307.1, R6308.1, R6309.1, R6310.1, U6301.18 (ADDR), U6301.21 (VCCP)
- net vcca1v8_pmu: now also C6301.1, R6301.1, U6301.23 (VCCI)

Commit message: Board: capture blk.debug
Debug UART2 (1.8 V) and I2S/DSD pads with ground pads, reset, PMIC and
power-key pads (PCB-T-09), a pad on every spare SoC GPIO whose pinout v1
row names one (the DEBUG bus, on the SoC's right edge), and a rail pad
for each power-tree rail no other sheet probes (PCB-T-02). Each DAC
sheet carries a pad on its MCLK. The spares pinout v1 leaves without a
pad now carry no-connect flags. On the root, facing sheet pins are
joined directly only where the route meets no other symbol.

Co-Authored-By: Claude Opus 5.5 <noreply@anthropic.com>
Claude-Session: https://claude.ai/code/session_01Ei262h3TpgY9vyfNLMi5Mn
Parts:
- removed C6301, C6302: 100 nF, Capacitor_SMD:C_0402_1005Metric, symbol Device:C
- removed R6301, R6306, R6307, R6308, R6309, R6310: 10 kΩ, Resistor_SMD:R_0402_1005Metric, symbol Device:R
- removed R6302, R6303, R6304, R6305: 100 kΩ, Resistor_SMD:R_0402_1005Metric, symbol Device:R
- removed U6301: TCA6416ARTWR, Texas_Instruments:Texas_RTW0024B_WQFN-24-1EP_4x4mm_P0.5mm_EP2.45x2.45mm_ThermalVias, symbol Texas_Instruments:TCA6416ARTWR
- added C6401, C6402: 100 nF, Capacitor_SMD:C_0402_1005Metric, symbol Device:C
- added R6401, R6406, R6407, R6408, R6409, R6410: 10 kΩ, Resistor_SMD:R_0402_1005Metric, symbol Device:R
- added R6402, R6403, R6404, R6405: 100 kΩ, Resistor_SMD:R_0402_1005Metric, symbol Device:R
- added U6401: TCA6416ARTWR, Texas_Instruments:Texas_RTW0024B_WQFN-24-1EP_4x4mm_P0.5mm_EP2.45x2.45mm_ThermalVias, symbol Texas_Instruments:TCA6416ARTWR
Connections:
- net EFUSE_5V_FLT_N: now also R6409.2, U6401.16 (P16)
- net EFUSE_HAT5V_FLT_N: now also R6408.2, U6401.15 (P15)
- net EFUSE_VBUS_FLT_N: now also R6410.2, U6401.17 (P17)
- net EXP_INT_N: now also U6401.22 (INT)
- net EXP_RESET_N: now also R6401.2, U6401.24 (RESET)
- net FP_DET_N: now also U6401.12 (P12)
- net FP_GPIO0: now also U6401.13 (P13)
- net FP_GPIO1: now also U6401.14 (P14)
- net FP_IO_EN: now also U6401.1 (P00)
- net GND: now also C6401.2, C6402.2, R6402.2, R6403.2, R6404.2, R6405.2, U6401.25 (EP), U6401.9 (GND)
- net HAPTIC_EN: now also R6404.1, U6401.5 (P04)
- net HAT5V_EN: now also R6402.1, U6401.3 (P02)
- net HAT_VBUS_DISCH: now also U6401.2 (P01)
- net HP_DET_BAL: now also R6407.2, U6401.11 (P11)
- net HP_DET_SE: now also R6406.2, U6401.10 (P10)
- net I2C2_SCL: now also U6401.19 (SCL)
- net I2C2_SDA: now also U6401.20 (SDA)
- net NFC_PWR_EN: now also R6405.1, U6401.6 (P05)
- net USB_SRC_ON: now also R6403.1, U6401.4 (P03)
- net WL_PD_HOLD_N: now also U6401.8 (P07)
- net WL_PWR_EN: now also U6401.7 (P06)
- net vcc3v3_sys: now also C6402.1, R6406.1, R6407.1, R6408.1, R6409.1, R6410.1, U6401.18 (ADDR), U6401.21 (VCCP)
- net vcca1v8_pmu: now also C6401.1, R6401.1, U6401.23 (VCCI)

Commit message: Board: capture blk.cover-detect
COVER_DET_N on GPIO0_A6 (AJ38, PMUIO1, wake-capable), recorded in
pinout v1 (closes feature blocks G22): board-edge input and ground pads
for the case's actuator, 100 kΩ to vcc3v3_pmu, TPD1E10B06 at the pad
(BOM v1 line 143, PCB-L-10). The line rides the KEYS bus with the
buttons.

Co-Authored-By: Claude Opus 5.5 <noreply@anthropic.com>
Claude-Session: https://claude.ai/code/session_01Ei262h3TpgY9vyfNLMi5Mn
Parts:
- removed C6401, C6402: 100 nF, Capacitor_SMD:C_0402_1005Metric, symbol Device:C
- removed R6401, R6406, R6407, R6408, R6409, R6410: 10 kΩ, Resistor_SMD:R_0402_1005Metric, symbol Device:R
- removed R6402, R6403, R6404, R6405: 100 kΩ, Resistor_SMD:R_0402_1005Metric, symbol Device:R
- removed U6401: TCA6416ARTWR, Texas_Instruments:Texas_RTW0024B_WQFN-24-1EP_4x4mm_P0.5mm_EP2.45x2.45mm_ThermalVias, symbol Texas_Instruments:TCA6416ARTWR
- added C6501, C6502: 100 nF, Capacitor_SMD:C_0402_1005Metric, symbol Device:C
- added R6501, R6506, R6507, R6508, R6509, R6510: 10 kΩ, Resistor_SMD:R_0402_1005Metric, symbol Device:R
- added R6502, R6503, R6504, R6505: 100 kΩ, Resistor_SMD:R_0402_1005Metric, symbol Device:R
- added U6501: TCA6416ARTWR, Texas_Instruments:Texas_RTW0024B_WQFN-24-1EP_4x4mm_P0.5mm_EP2.45x2.45mm_ThermalVias, symbol Texas_Instruments:TCA6416ARTWR
Connections:
- net EFUSE_5V_FLT_N: now also R6509.2, U6501.16 (P16)
- net EFUSE_HAT5V_FLT_N: now also R6508.2, U6501.15 (P15)
- net EFUSE_VBUS_FLT_N: now also R6510.2, U6501.17 (P17)
- net EXP_INT_N: now also U6501.22 (INT)
- net EXP_RESET_N: now also R6501.2, U6501.24 (RESET)
- net FP_DET_N: now also U6501.12 (P12)
- net FP_GPIO0: now also U6501.13 (P13)
- net FP_GPIO1: now also U6501.14 (P14)
- net FP_IO_EN: now also U6501.1 (P00)
- net GND: now also C6501.2, C6502.2, R6502.2, R6503.2, R6504.2, R6505.2, U6501.25 (EP), U6501.9 (GND)
- net HAPTIC_EN: now also R6504.1, U6501.5 (P04)
- net HAT5V_EN: now also R6502.1, U6501.3 (P02)
- net HAT_VBUS_DISCH: now also U6501.2 (P01)
- net HP_DET_BAL: now also R6507.2, U6501.11 (P11)
- net HP_DET_SE: now also R6506.2, U6501.10 (P10)
- net I2C2_SCL: now also U6501.19 (SCL)
- net I2C2_SDA: now also U6501.20 (SDA)
- net NFC_PWR_EN: now also R6505.1, U6501.6 (P05)
- net USB_SRC_ON: now also R6503.1, U6501.4 (P03)
- net WL_PD_HOLD_N: now also U6501.8 (P07)
- net WL_PWR_EN: now also U6501.7 (P06)
- net vcc3v3_sys: now also C6502.1, R6506.1, R6507.1, R6508.1, R6509.1, R6510.1, U6501.18 (ADDR), U6501.21 (VCCP)
- net vcca1v8_pmu: now also C6501.1, R6501.1, U6501.23 (VCCI)

Commit message: Board: capture blk.mic-ambient and links #34, #35
IM73D122 on PDM CLK1 and SDI1 (BOM v1 line 34, pinout v1 AK2 and 1P2),
LR to ground, 22 Ω clock series, VDD from MIC_1V8 through link #35.
Link #34 on blk.mic-main makes the faceplate branch the rail MIC_1V8_FP
for contact 40 (power tree §4.12, G10). kicad-lib moves to e46bda4 for
the IM73D122, TPS3808G01, SN74LVC1G58 and BAT54 parts.

Co-Authored-By: Claude Opus 5.5 <noreply@anthropic.com>
Claude-Session: https://claude.ai/code/session_01Ei262h3TpgY9vyfNLMi5Mn
Parts:
- removed C6501, C6502: 100 nF, Capacitor_SMD:C_0402_1005Metric, symbol Device:C
- removed R6501, R6506, R6507, R6508, R6509, R6510: 10 kΩ, Resistor_SMD:R_0402_1005Metric, symbol Device:R
- removed R6502, R6503, R6504, R6505: 100 kΩ, Resistor_SMD:R_0402_1005Metric, symbol Device:R
- removed U6501: TCA6416ARTWR, Texas_Instruments:Texas_RTW0024B_WQFN-24-1EP_4x4mm_P0.5mm_EP2.45x2.45mm_ThermalVias, symbol Texas_Instruments:TCA6416ARTWR
- added C6601, C6602: 100 nF, Capacitor_SMD:C_0402_1005Metric, symbol Device:C
- added R6601, R6606, R6607, R6608, R6609, R6610: 10 kΩ, Resistor_SMD:R_0402_1005Metric, symbol Device:R
- added R6602, R6603, R6604, R6605: 100 kΩ, Resistor_SMD:R_0402_1005Metric, symbol Device:R
- added U6601: TCA6416ARTWR, Texas_Instruments:Texas_RTW0024B_WQFN-24-1EP_4x4mm_P0.5mm_EP2.45x2.45mm_ThermalVias, symbol Texas_Instruments:TCA6416ARTWR
Connections:
- net EFUSE_5V_FLT_N: now also R6609.2, U6601.16 (P16)
- net EFUSE_HAT5V_FLT_N: now also R6608.2, U6601.15 (P15)
- net EFUSE_VBUS_FLT_N: now also R6610.2, U6601.17 (P17)
- net EXP_INT_N: now also U6601.22 (INT)
- net EXP_RESET_N: now also R6601.2, U6601.24 (RESET)
- net FP_DET_N: now also U6601.12 (P12)
- net FP_GPIO0: now also U6601.13 (P13)
- net FP_GPIO1: now also U6601.14 (P14)
- net FP_IO_EN: now also U6601.1 (P00)
- net GND: now also C6601.2, C6602.2, R6602.2, R6603.2, R6604.2, R6605.2, U6601.25 (EP), U6601.9 (GND)
- net HAPTIC_EN: now also R6604.1, U6601.5 (P04)
- net HAT5V_EN: now also R6602.1, U6601.3 (P02)
- net HAT_VBUS_DISCH: now also U6601.2 (P01)
- net HP_DET_BAL: now also R6607.2, U6601.11 (P11)
- net HP_DET_SE: now also R6606.2, U6601.10 (P10)
- net I2C2_SCL: now also U6601.19 (SCL)
- net I2C2_SDA: now also U6601.20 (SDA)
- net NFC_PWR_EN: now also R6605.1, U6601.6 (P05)
- net USB_SRC_ON: now also R6603.1, U6601.4 (P03)
- net WL_PD_HOLD_N: now also U6601.8 (P07)
- net WL_PWR_EN: now also U6601.7 (P06)
- net vcc3v3_sys: now also C6602.1, R6606.1, R6607.1, R6608.1, R6609.1, R6610.1, U6601.18 (ADDR), U6601.21 (VCCP)
- net vcca1v8_pmu: now also C6601.1, R6601.1, U6601.23 (VCCI)

Commit message: Board: capture blk.maskrom
Power + Vol- at a cold power-on pull eMMC D0 low inside the TPS3808G01
boot window (BOM v1 lines 35, 78, 97, 98; sim/maskrom): SENSE 280k/100k,
CT 390 nF, WINDOW_N with its pad, SN74LVC1G57 and SN74LVC1G58 on
vcca1v8_pmu, BAT54 from PWRON_N, DMG1012T through 1 kΩ to EMMC_D0.
Every block in use now has its sheet; the README states the remaining
single-pin nets.

Co-Authored-By: Claude Opus 5.5 <noreply@anthropic.com>
Claude-Session: https://claude.ai/code/session_01Ei262h3TpgY9vyfNLMi5Mn
Parts:
- removed C6601, C6602: 100 nF, Capacitor_SMD:C_0402_1005Metric, symbol Device:C
- removed R6601, R6606, R6607, R6608, R6609, R6610: 10 kΩ, Resistor_SMD:R_0402_1005Metric, symbol Device:R
- removed R6602, R6603, R6604, R6605: 100 kΩ, Resistor_SMD:R_0402_1005Metric, symbol Device:R
- removed U6601: TCA6416ARTWR, Texas_Instruments:Texas_RTW0024B_WQFN-24-1EP_4x4mm_P0.5mm_EP2.45x2.45mm_ThermalVias, symbol Texas_Instruments:TCA6416ARTWR
- added C6701, C6702: 100 nF, Capacitor_SMD:C_0402_1005Metric, symbol Device:C
- added R6701, R6706, R6707, R6708, R6709, R6710: 10 kΩ, Resistor_SMD:R_0402_1005Metric, symbol Device:R
- added R6702, R6703, R6704, R6705: 100 kΩ, Resistor_SMD:R_0402_1005Metric, symbol Device:R
- added U6701: TCA6416ARTWR, Texas_Instruments:Texas_RTW0024B_WQFN-24-1EP_4x4mm_P0.5mm_EP2.45x2.45mm_ThermalVias, symbol Texas_Instruments:TCA6416ARTWR
Connections:
- net EFUSE_5V_FLT_N: now also R6709.2, U6701.16 (P16)
- net EFUSE_HAT5V_FLT_N: now also R6708.2, U6701.15 (P15)
- net EFUSE_VBUS_FLT_N: now also R6710.2, U6701.17 (P17)
- net EXP_INT_N: now also U6701.22 (INT)
- net EXP_RESET_N: now also R6701.2, U6701.24 (RESET)
- net FP_DET_N: now also U6701.12 (P12)
- net FP_GPIO0: now also U6701.13 (P13)
- net FP_GPIO1: now also U6701.14 (P14)
- net FP_IO_EN: now also U6701.1 (P00)
- net GND: now also C6701.2, C6702.2, R6702.2, R6703.2, R6704.2, R6705.2, U6701.25 (EP), U6701.9 (GND)
- net HAPTIC_EN: now also R6704.1, U6701.5 (P04)
- net HAT5V_EN: now also R6702.1, U6701.3 (P02)
- net HAT_VBUS_DISCH: now also U6701.2 (P01)
- net HP_DET_BAL: now also R6707.2, U6701.11 (P11)
- net HP_DET_SE: now also R6706.2, U6701.10 (P10)
- net I2C2_SCL: now also U6701.19 (SCL)
- net I2C2_SDA: now also U6701.20 (SDA)
- net NFC_PWR_EN: now also R6705.1, U6701.6 (P05)
- net USB_SRC_ON: now also R6703.1, U6701.4 (P03)
- net WL_PD_HOLD_N: now also U6701.8 (P07)
- net WL_PWR_EN: now also U6701.7 (P06)
- net vcc3v3_sys: now also C6702.1, R6706.1, R6707.1, R6708.1, R6709.1, R6710.1, U6701.18 (ADDR), U6701.21 (VCCP)
- net vcca1v8_pmu: now also C6701.1, R6701.1, U6701.23 (VCCI)

Commit message: Compaction: lower inductors, 0201 decoupling, 0.8 mm signal test pads
A matrix tool (hardware/studies/compaction) checks each candidate against
the design's stresses: same inductance, design peak <= 70 % and the
converter's maximum limit <= 100 % of Isat (30 % drop), height zones,
ratings at least twice the rail, PCB-D-06; sourcing outcome per part.

Applied (placement v1 decision 12, BOM v1.15):
- L601, L4401: XGL4015-102MEC (1.5 mm) for XAL/XGL4020-102MEC (2.1 mm);
- L1001, L5101: XGL4015-471MEC (1.5 mm) for Wurth 744373240047, on the
  stock XxL4020 land (the Wurth land was never drawn);
- L1201 is 1.2 mm (XGL4012, per-MPN heights): it moves next to the SoC;
- 58 x 100 nF decoupling on rails <= 3.3 V in core/IO/radio: 0201;
- 51 test pads on signal nets: 0.8 mm (PCB-D-06 v0.16, JLCPCB guide).
Kept: L901, L2802 (XGL4015 at 103 % of Isat at the limit); no thinner
0805/1206 capacitor passes (obsolete, NRND or unlisted).

Board need 113 % -> 111 % (core band 227 -> 203 %, power band 258 ->
233 %, radio band 19 -> 0 %); only C904 still relies on PCB-Z-04.
ERC 0 errors, craft Q1 met, DRC 0 errors (605 warnings), pcb and study
tests pass, rules test board PASS.

Co-Authored-By: Claude Opus 5.5 <noreply@anthropic.com>
Claude-Session: https://claude.ai/code/session_01Ei262h3TpgY9vyfNLMi5Mn
Parts:
- C6701, C6702: footprint Capacitor_SMD:C_0402_1005Metric -> Capacitor_SMD:C_0201_0603Metric; MPN GRM155R71C104KA88D -> GRM033R61A104KE15D
Changed lines of the file:
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@@
   (property "Reference" "C6701" (at 124.46 46.99 0) (effects (font (size 1.27 1.27)) (justify left)))
   (property "Value" "100 nF" (at 124.46 49.53 0) (effects (font (size 1.27 1.27)) (justify left)))
-  (property "Footprint" "Capacitor_SMD:C_0402_1005Metric" (at 121.92 48.26 0) (effects (font (size 1.27 1.27))) (hide yes))
-  (property "Datasheet" "https://www.murata.com/en-us/products/productdetail?partno=GRM155R71C104KA88D" (at 121.92 48.26 0) (effects (font (size 1.27 1.27))) (hide yes))
-  (property "Description" "Capacitor, 100 nF, 16 V, X7R, 0402" (at 121.92 48.26 0) (effects (font (size 1.27 1.27))) (hide yes))
+  (property "Footprint" "Capacitor_SMD:C_0201_0603Metric" (at 121.92 48.26 0) (effects (font (size 1.27 1.27))) (hide yes))
+  (property "Datasheet" "https://www.murata.com/en-us/products/productdetail?partno=GRM033R61A104KE15D" (at 121.92 48.26 0) (effects (font (size 1.27 1.27))) (hide yes))
+  (property "Description" "Capacitor, 100 nF, 10 V, X5R, 0201" (at 121.92 48.26 0) (effects (font (size 1.27 1.27))) (hide yes))
   (property "Manufacturer" "Murata" (at 121.92 48.26 0) (effects (font (size 1.27 1.27))) (hide yes))
-  (property "MPN" "GRM155R71C104KA88D" (at 121.92 48.26 0) (effects (font (size 1.27 1.27))) (hide yes))
+  (property "MPN" "GRM033R61A104KE15D" (at 121.92 48.26 0) (effects (font (size 1.27 1.27))) (hide yes))
   (property "Block" "blk.gpio-expander" (at 121.92 48.26 0) (effects (font (size 1.27 1.27))) (hide yes))
   (pin "1")
@@
   (property "Reference" "C6702" (at 143.51 46.99 0) (effects (font (size 1.27 1.27)) (justify left)))
   (property "Value" "100 nF" (at 143.51 49.53 0) (effects (font (size 1.27 1.27)) (justify left)))
-  (property "Footprint" "Capacitor_SMD:C_0402_1005Metric" (at 140.97 48.26 0) (effects (font (size 1.27 1.27))) (hide yes))
-  (property "Datasheet" "https://www.murata.com/en-us/products/productdetail?partno=GRM155R71C104KA88D" (at 140.97 48.26 0) (effects (font (size 1.27 1.27))) (hide yes))
-  (property "Description" "Capacitor, 100 nF, 16 V, X7R, 0402" (at 140.97 48.26 0) (effects (font (size 1.27 1.27))) (hide yes))
+  (property "Footprint" "Capacitor_SMD:C_0201_0603Metric" (at 140.97 48.26 0) (effects (font (size 1.27 1.27))) (hide yes))
+  (property "Datasheet" "https://www.murata.com/en-us/products/productdetail?partno=GRM033R61A104KE15D" (at 140.97 48.26 0) (effects (font (size 1.27 1.27))) (hide yes))
+  (property "Description" "Capacitor, 100 nF, 10 V, X5R, 0201" (at 140.97 48.26 0) (effects (font (size 1.27 1.27))) (hide yes))
   (property "Manufacturer" "Murata" (at 140.97 48.26 0) (effects (font (size 1.27 1.27))) (hide yes))
-  (property "MPN" "GRM155R71C104KA88D" (at 140.97 48.26 0) (effects (font (size 1.27 1.27))) (hide yes))
+  (property "MPN" "GRM033R61A104KE15D" (at 140.97 48.26 0) (effects (font (size 1.27 1.27))) (hide yes))
   (property "Block" "blk.gpio-expander" (at 140.97 48.26 0) (effects (font (size 1.27 1.27))) (hide yes))
   (pin "1")

Commit message: Board on libs v0.2.0: lower-case kebab vendor keys (HL-13)
The libs submodule moves to v0.2.0 (5f24483). Every library nickname in
the generator, the placement tool and the floorplan study follows the
key table (Texas_Instruments -> texas-instruments, OpenDAP_Device ->
opendap-generic, Rockchip and Rockchip_PMIC -> rockchip, ...); the
library tables are written from the files. Schematic and board
regenerated.

Checks: ERC 0 errors (warnings unchanged); DRC 0 errors, 605 warnings,
the same counts by type, schematic parity 0; every placement identical;
craft Q1 met; pcb tests pass; STEP export resolves every libs 3D model
(the 27 parts without a model are KiCad stock lands that have none).

Co-Authored-By: Claude Opus 5.5 <noreply@anthropic.com>
Claude-Session: https://claude.ai/code/session_01Ei262h3TpgY9vyfNLMi5Mn
Parts:
- U6701: footprint Texas_Instruments:Texas_RTW0024B_WQFN-24-1EP_4x4mm_P0.5mm_EP2.45x2.45mm_ThermalVias -> texas-instruments:Texas_RTW0024B_WQFN-24-1EP_4x4mm_P0.5mm_EP2.45x2.45mm_ThermalVias; symbol Texas_Instruments:TCA6416ARTWR -> texas-instruments:TCA6416ARTWR
Changed lines of the file:
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@@
 (paper "A3")
 (title_block (title "GPIO expander") (date "2026-10-25") (rev "A") (company "The OpenDAP Project") (comment 1 "blk.gpio-expander") (comment 2 "TCA6416A on I2C2: slow enables with their off-state pulls, detects and fault inputs"))
-(symbol (lib_id "Texas_Instruments:TCA6416ARTWR") (at 80.01 95.25 0) (unit 1) (body_style 1) (exclude_from_sim no) (in_bom yes) (on_board yes) (dnp no)
+(symbol (lib_id "texas-instruments:TCA6416ARTWR") (at 80.01 95.25 0) (unit 1) (body_style 1) (exclude_from_sim no) (in_bom yes) (on_board yes) (dnp no)
   (property "Reference" "U6701" (at 83.82 58.42 0) (effects (font (size 1.27 1.27)) (justify left)))
   (property "Value" "TCA6416ARTWR" (at 83.82 55.88 0) (effects (font (size 1.27 1.27)) (justify left)))
-  (property "Footprint" "Texas_Instruments:Texas_RTW0024B_WQFN-24-1EP_4x4mm_P0.5mm_EP2.45x2.45mm_ThermalVias" (at 80.01 95.25 0) (effects (font (size 1.27 1.27))) (hide yes))
+  (property "Footprint" "texas-instruments:Texas_RTW0024B_WQFN-24-1EP_4x4mm_P0.5mm_EP2.45x2.45mm_ThermalVias" (at 80.01 95.25 0) (effects (font (size 1.27 1.27))) (hide yes))
   (property "Datasheet" "https://www.ti.com/lit/ds/symlink/tca6416a.pdf" (at 80.01 95.25 0) (effects (font (size 1.27 1.27))) (hide yes))
   (property "Description" "16-bit I2C and SMBus I/O expander, separate 1.65-5.5 V I2C-side (VCCI) and port-side (VCCP) supplies, interrupt output, reset input, WQFN-24 (RTW0024B) 4 x 4 mm with exposed pad" (at 80.01 95.25 0) (effects (font (size 1.27 1.27))) (hide yes))
