File: board/hardware/t1-main-board/imu.kicad_sch (KiCad schematic)
At the start: 6 parts, among them U5201 LSM6DSV16XTR

Commit message: Board: capture blk.current-monitors
Five INA236 on I2C1 (0x40-0x43, 0x48) with their shunts, per power tree
§4.12 and BOM v1 lines 54 and 136. The measured branches are rails of
their own (VSYS_SRC, VSYS_LV_AUDIO, VSYS_AUDIO, VSYS_LV_BL, VSYS_P5V1),
fed through the shunts on this sheet; the charger, audio, backlight and
5.1 V sheets take them. The root's layout may leave a stack level empty,
so the block sits under the notes; IC bboxes hold turned rail values;
passive rows hold a bottom rail's text.

Co-Authored-By: Claude Opus 5.5 <noreply@anthropic.com>
Claude-Session: https://claude.ai/code/session_01Ei262h3TpgY9vyfNLMi5Mn
Parts:
- removed C5201, C5202: 100 nF, Capacitor_SMD:C_0402_1005Metric, symbol Device:C
- removed R5201: 10 Ω, Resistor_SMD:R_0603_1608Metric, symbol Device:R
- removed TP5201: vcca1v8_pmu, TestPoint:TestPoint_Pad_D1.0mm, symbol Connector:TestPoint
- removed TP5202: IMU_VDD, TestPoint:TestPoint_Pad_D1.0mm, symbol Connector:TestPoint
- removed U5201: LSM6DSV16XTR, STMicroelectronics:ST_LGA-14L_2.5x3mm_P0.5mm, symbol STMicroelectronics:LSM6DSV16XTR
- added C5301, C5302: 100 nF, Capacitor_SMD:C_0402_1005Metric, symbol Device:C
- added R5301: 10 Ω, Resistor_SMD:R_0603_1608Metric, symbol Device:R
- added TP5301: vcca1v8_pmu, TestPoint:TestPoint_Pad_D1.0mm, symbol Connector:TestPoint
- added TP5302: IMU_VDD, TestPoint:TestPoint_Pad_D1.0mm, symbol Connector:TestPoint
- added U5301: LSM6DSV16XTR, STMicroelectronics:ST_LGA-14L_2.5x3mm_P0.5mm, symbol STMicroelectronics:LSM6DSV16XTR
Connections:
- net GND: now also C5301.2, C5302.2, U5301.1 (SDO/SA0), U5301.2 (SDx/AH1/Qvar1), U5301.3 (SCx/AH2/Qvar2), U5301.6 (GND), U5301.7 (GND)
- net I2C2_SCL: now also U5301.13 (SCL)
- net I2C2_SDA: now also U5301.14 (SDA)
- net IMU_INT1: now also U5301.4 (INT1)
- net IMU_VDD: now also C5301.1, C5302.1, R5301.2, TP5302.1, U5301.12 (CS), U5301.5 (Vdd_IO), U5301.8 (Vdd)
- net vcca1v8_pmu: now also R5301.1, TP5301.1
Changed lines of the file:
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@@
 (title_block (title "Motion sensor") (date "2026-10-25") (rev "A") (company "The OpenDAP Project") (comment 1 "blk.imu") (comment 2 "LSM6DSV16X on I2C2 at 0x6A, INT1 wake on motion, always on"))
 (symbol (lib_id "STMicroelectronics:LSM6DSV16XTR") (at 55.88 77.47 0) (unit 1) (body_style 1) (exclude_from_sim no) (in_bom yes) (on_board yes) (dnp no)
-  (property "Reference" "U5201" (at 59.69 50.8 0) (effects (font (size 1.27 1.27)) (justify left)))
+  (property "Reference" "U5301" (at 59.69 50.8 0) (effects (font (size 1.27 1.27)) (justify left)))
   (property "Value" "LSM6DSV16XTR" (at 59.69 48.26 0) (effects (font (size 1.27 1.27)) (justify left)))
   (property "Footprint" "STMicroelectronics:ST_LGA-14L_2.5x3mm_P0.5mm" (at 55.88 77.47 0) (effects (font (size 1.27 1.27))) (hide yes))
@@
   (pin "6")
   (pin "7")
-  (instances (project "t1-main-board" (path "/7746052e-d7f9-59ad-ba73-bd2b74439529/cab3b4fb-5ec0-5c66-a197-75b8941e1631" (reference "U5201") (unit 1))))
+  (instances (project "t1-main-board" (path "/7746052e-d7f9-59ad-ba73-bd2b74439529/cab3b4fb-5ec0-5c66-a197-75b8941e1631" (reference "U5301") (unit 1))))
 )
 (wire (pts (xy 53.34 49.53) (xy 53.34 46.99)) (stroke (width 0) (type default)))
@@
 (no_connect (at 73.66 69.85))
 (symbol (lib_id "Device:C") (at 91.44 53.34 0) (unit 1) (body_style 1) (exclude_from_sim no) (in_bom yes) (on_board yes) (dnp no)
-  (property "Reference" "C5201" (at 93.98 52.07 0) (effects (font (size 1.27 1.27)) (justify left)))
+  (property "Reference" "C5301" (at 93.98 52.07 0) (effects (font (size 1.27 1.27)) (justify left)))
   (property "Value" "100 nF" (at 93.98 54.61 0) (effects (font (size 1.27 1.27)) (justify left)))
   (property "Footprint" "Capacitor_SMD:C_0402_1005Metric" (at 91.44 53.34 0) (effects (font (size 1.27 1.27))) (hide yes))
@@
   (pin "1")
   (pin "2")
-  (instances (project "t1-main-board" (path "/7746052e-d7f9-59ad-ba73-bd2b74439529/cab3b4fb-5ec0-5c66-a197-75b8941e1631" (reference "C5201") (unit 1))))
+  (instances (project "t1-main-board" (path "/7746052e-d7f9-59ad-ba73-bd2b74439529/cab3b4fb-5ec0-5c66-a197-75b8941e1631" (reference "C5301") (unit 1))))
 )
 (wire (pts (xy 91.44 49.53) (xy 91.44 46.99)) (stroke (width 0) (type default)))
@@
 )
 (symbol (lib_id "Device:C") (at 105.41 53.34 0) (unit 1) (body_style 1) (exclude_from_sim no) (in_bom yes) (on_board yes) (dnp no)
-  (property "Reference" "C5202" (at 107.95 52.07 0) (effects (font (size 1.27 1.27)) (justify left)))
+  (property "Reference" "C5302" (at 107.95 52.07 0) (effects (font (size 1.27 1.27)) (justify left)))
   (property "Value" "100 nF" (at 107.95 54.61 0) (effects (font (size 1.27 1.27)) (justify left)))
   (property "Footprint" "Capacitor_SMD:C_0402_1005Metric" (at 105.41 53.34 0) (effects (font (size 1.27 1.27))) (hide yes))
@@
   (pin "1")
   (pin "2")
-  (instances (project "t1-main-board" (path "/7746052e-d7f9-59ad-ba73-bd2b74439529/cab3b4fb-5ec0-5c66-a197-75b8941e1631" (reference "C5202") (unit 1))))
+  (instances (project "t1-main-board" (path "/7746052e-d7f9-59ad-ba73-bd2b74439529/cab3b4fb-5ec0-5c66-a197-75b8941e1631" (reference "C5302") (unit 1))))
 )
 (wire (pts (xy 105.41 49.53) (xy 105.41 46.99)) (stroke (width 0) (type default)))
@@
 (text "LSM6DSV16X at I2C2 0x6A (BOM v1 line 59)" (exclude_from_sim no) (at 24.13 34.29 0) (effects (font (size 2.54 2.54)) (justify left bottom)))
 (symbol (lib_id "Device:R") (at 163.83 50.8 90) (unit 1) (body_style 1) (exclude_from_sim no) (in_bom yes) (on_board yes) (dnp no)
-  (property "Reference" "R5201" (at 161.29 46.99 90) (effects (font (size 1.27 1.27))))
+  (property "Reference" "R5301" (at 161.29 46.99 90) (effects (font (size 1.27 1.27))))
   (property "Value" "10 Ω" (at 161.29 53.34 90) (effects (font (size 1.27 1.27))))
   (property "Spec" "0603" (at 161.29 55.88 90) (effects (font (size 1.27 1.27))))
@@
   (pin "1")
   (pin "2")
-  (instances (project "t1-main-board" (path "/7746052e-d7f9-59ad-ba73-bd2b74439529/cab3b4fb-5ec0-5c66-a197-75b8941e1631" (reference "R5201") (unit 1) (variant (name "production") (field (name "Value") (value "0 Ω")) (field (name "MPN") (value "RC0603JR-070RL")) (field (name "Manufacturer") (value "YAGEO"))))))
+  (instances (project "t1-main-board" (path "/7746052e-d7f9-59ad-ba73-bd2b74439529/cab3b4fb-5ec0-5c66-a197-75b8941e1631" (reference "R5301") (unit 1) (variant (name "production") (field (name "Value") (value "0 Ω")) (field (name "MPN") (value "RC0603JR-070RL")) (field (name "Manufacturer") (value "YAGEO"))))))
 )
 (rectangle (start 140.97 38.1) (end 181.61 58.42) (stroke (width 0) (type dash)) (fill (type none)))
@@
 (wire (pts (xy 157.48 50.8) (xy 157.48 48.26)) (stroke (width 0) (type default)))
 (symbol (lib_id "Connector:TestPoint") (at 157.48 48.26 0) (unit 1) (body_style 1) (exclude_from_sim no) (in_bom no) (on_board yes) (dnp no)
-  (property "Reference" "TP5201" (at 156.21 43.18 0) (effects (font (size 1.27 1.27)) (justify right)))
+  (property "Reference" "TP5301" (at 156.21 43.18 0) (effects (font (size 1.27 1.27)) (justify right)))
   (property "Value" "vcca1v8_pmu" (at 156.21 45.72 0) (effects (font (size 1.27 1.27)) (justify right)))
   (property "Footprint" "TestPoint:TestPoint_Pad_D1.0mm" (at 157.48 48.26 0) (effects (font (size 1.27 1.27))) (hide yes))
@@
   (property "Block" "blk.imu" (at 157.48 48.26 0) (effects (font (size 1.27 1.27))) (hide yes))
   (pin "1")
-  (instances (project "t1-main-board" (path "/7746052e-d7f9-59ad-ba73-bd2b74439529/cab3b4fb-5ec0-5c66-a197-75b8941e1631" (reference "TP5201") (unit 1))))
+  (instances (project "t1-main-board" (path "/7746052e-d7f9-59ad-ba73-bd2b74439529/cab3b4fb-5ec0-5c66-a197-75b8941e1631" (reference "TP5301") (unit 1))))
 )
 (symbol (lib_id "power:VCC") (at 138.43 50.8 90) (unit 1) (body_style 1) (exclude_from_sim no) (in_bom yes) (on_board yes) (dnp no)
@@
 (wire (pts (xy 170.18 50.8) (xy 170.18 48.26)) (stroke (width 0) (type default)))
 (symbol (lib_id "Connector:TestPoint") (at 170.18 48.26 0) (unit 1) (body_style 1) (exclude_from_sim no) (in_bom no) (on_board yes) (dnp no)
-  (property "Reference" "TP5202" (at 171.45 43.18 0) (effects (font (size 1.27 1.27)) (justify left)))
+  (property "Reference" "TP5302" (at 171.45 43.18 0) (effects (font (size 1.27 1.27)) (justify left)))
   (property "Value" "IMU_VDD" (at 171.45 45.72 0) (effects (font (size 1.27 1.27)) (justify left)))
   (property "Footprint" "TestPoint:TestPoint_Pad_D1.0mm" (at 170.18 48.26 0) (effects (font (size 1.27 1.27))) (hide yes))
@@
   (property "Block" "blk.imu" (at 170.18 48.26 0) (effects (font (size 1.27 1.27))) (hide yes))
   (pin "1")
-  (instances (project "t1-main-board" (path "/7746052e-d7f9-59ad-ba73-bd2b74439529/cab3b4fb-5ec0-5c66-a197-75b8941e1631" (reference "TP5202") (unit 1))))
+  (instances (project "t1-main-board" (path "/7746052e-d7f9-59ad-ba73-bd2b74439529/cab3b4fb-5ec0-5c66-a197-75b8941e1631" (reference "TP5302") (unit 1))))
 )
 (junction (at 189.23 50.8) (diameter 0) (color 0 0 0 0))

Commit message: Board: capture blk.status-led
LP5521 at 0x32 on I2C2 (BOM v1 line 105) with its charge-pump
capacitors, EN on vcca1v8_pmu, VDD from VSYS_LV through link #22;
LED_R/G/B reach the faceplate connector as the LED bus alias. The
faceplate row of the root is re-packed so five full columns sit left of
the title block.

Co-Authored-By: Claude Opus 5.5 <noreply@anthropic.com>
Claude-Session: https://claude.ai/code/session_01Ei262h3TpgY9vyfNLMi5Mn
Parts:
- removed C5301, C5302: 100 nF, Capacitor_SMD:C_0402_1005Metric, symbol Device:C
- removed R5301: 10 Ω, Resistor_SMD:R_0603_1608Metric, symbol Device:R
- removed TP5301: vcca1v8_pmu, TestPoint:TestPoint_Pad_D1.0mm, symbol Connector:TestPoint
- removed TP5302: IMU_VDD, TestPoint:TestPoint_Pad_D1.0mm, symbol Connector:TestPoint
- removed U5301: LSM6DSV16XTR, STMicroelectronics:ST_LGA-14L_2.5x3mm_P0.5mm, symbol STMicroelectronics:LSM6DSV16XTR
- added C5901, C5902: 100 nF, Capacitor_SMD:C_0402_1005Metric, symbol Device:C
- added R5901: 10 Ω, Resistor_SMD:R_0603_1608Metric, symbol Device:R
- added TP5901: vcca1v8_pmu, TestPoint:TestPoint_Pad_D1.0mm, symbol Connector:TestPoint
- added TP5902: IMU_VDD, TestPoint:TestPoint_Pad_D1.0mm, symbol Connector:TestPoint
- added U5901: LSM6DSV16XTR, STMicroelectronics:ST_LGA-14L_2.5x3mm_P0.5mm, symbol STMicroelectronics:LSM6DSV16XTR
Connections:
- net GND: now also C5901.2, C5902.2, U5901.1 (SDO/SA0), U5901.2 (SDx/AH1/Qvar1), U5901.3 (SCx/AH2/Qvar2), U5901.6 (GND), U5901.7 (GND)
- net I2C2_SCL: now also U5901.13 (SCL)
- net I2C2_SDA: now also U5901.14 (SDA)
- net IMU_INT1: now also U5901.4 (INT1)
- net IMU_VDD: now also C5901.1, C5902.1, R5901.2, TP5902.1, U5901.12 (CS), U5901.5 (Vdd_IO), U5901.8 (Vdd)
- net vcca1v8_pmu: now also R5901.1, TP5901.1
Changed lines of the file:
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@@
 (title_block (title "Motion sensor") (date "2026-10-25") (rev "A") (company "The OpenDAP Project") (comment 1 "blk.imu") (comment 2 "LSM6DSV16X on I2C2 at 0x6A, INT1 wake on motion, always on"))
 (symbol (lib_id "STMicroelectronics:LSM6DSV16XTR") (at 55.88 77.47 0) (unit 1) (body_style 1) (exclude_from_sim no) (in_bom yes) (on_board yes) (dnp no)
-  (property "Reference" "U5301" (at 59.69 50.8 0) (effects (font (size 1.27 1.27)) (justify left)))
+  (property "Reference" "U5901" (at 59.69 50.8 0) (effects (font (size 1.27 1.27)) (justify left)))
   (property "Value" "LSM6DSV16XTR" (at 59.69 48.26 0) (effects (font (size 1.27 1.27)) (justify left)))
   (property "Footprint" "STMicroelectronics:ST_LGA-14L_2.5x3mm_P0.5mm" (at 55.88 77.47 0) (effects (font (size 1.27 1.27))) (hide yes))
@@
   (pin "6")
   (pin "7")
-  (instances (project "t1-main-board" (path "/7746052e-d7f9-59ad-ba73-bd2b74439529/cab3b4fb-5ec0-5c66-a197-75b8941e1631" (reference "U5301") (unit 1))))
+  (instances (project "t1-main-board" (path "/7746052e-d7f9-59ad-ba73-bd2b74439529/cab3b4fb-5ec0-5c66-a197-75b8941e1631" (reference "U5901") (unit 1))))
 )
 (wire (pts (xy 53.34 49.53) (xy 53.34 46.99)) (stroke (width 0) (type default)))
@@
 (no_connect (at 73.66 69.85))
 (symbol (lib_id "Device:C") (at 91.44 53.34 0) (unit 1) (body_style 1) (exclude_from_sim no) (in_bom yes) (on_board yes) (dnp no)
-  (property "Reference" "C5301" (at 93.98 52.07 0) (effects (font (size 1.27 1.27)) (justify left)))
+  (property "Reference" "C5901" (at 93.98 52.07 0) (effects (font (size 1.27 1.27)) (justify left)))
   (property "Value" "100 nF" (at 93.98 54.61 0) (effects (font (size 1.27 1.27)) (justify left)))
   (property "Footprint" "Capacitor_SMD:C_0402_1005Metric" (at 91.44 53.34 0) (effects (font (size 1.27 1.27))) (hide yes))
@@
   (pin "1")
   (pin "2")
-  (instances (project "t1-main-board" (path "/7746052e-d7f9-59ad-ba73-bd2b74439529/cab3b4fb-5ec0-5c66-a197-75b8941e1631" (reference "C5301") (unit 1))))
+  (instances (project "t1-main-board" (path "/7746052e-d7f9-59ad-ba73-bd2b74439529/cab3b4fb-5ec0-5c66-a197-75b8941e1631" (reference "C5901") (unit 1))))
 )
 (wire (pts (xy 91.44 49.53) (xy 91.44 46.99)) (stroke (width 0) (type default)))
@@
 )
 (symbol (lib_id "Device:C") (at 105.41 53.34 0) (unit 1) (body_style 1) (exclude_from_sim no) (in_bom yes) (on_board yes) (dnp no)
-  (property "Reference" "C5302" (at 107.95 52.07 0) (effects (font (size 1.27 1.27)) (justify left)))
+  (property "Reference" "C5902" (at 107.95 52.07 0) (effects (font (size 1.27 1.27)) (justify left)))
   (property "Value" "100 nF" (at 107.95 54.61 0) (effects (font (size 1.27 1.27)) (justify left)))
   (property "Footprint" "Capacitor_SMD:C_0402_1005Metric" (at 105.41 53.34 0) (effects (font (size 1.27 1.27))) (hide yes))
@@
   (pin "1")
   (pin "2")
-  (instances (project "t1-main-board" (path "/7746052e-d7f9-59ad-ba73-bd2b74439529/cab3b4fb-5ec0-5c66-a197-75b8941e1631" (reference "C5302") (unit 1))))
+  (instances (project "t1-main-board" (path "/7746052e-d7f9-59ad-ba73-bd2b74439529/cab3b4fb-5ec0-5c66-a197-75b8941e1631" (reference "C5902") (unit 1))))
 )
 (wire (pts (xy 105.41 49.53) (xy 105.41 46.99)) (stroke (width 0) (type default)))
@@
 (text "LSM6DSV16X at I2C2 0x6A (BOM v1 line 59)" (exclude_from_sim no) (at 24.13 34.29 0) (effects (font (size 2.54 2.54)) (justify left bottom)))
 (symbol (lib_id "Device:R") (at 163.83 50.8 90) (unit 1) (body_style 1) (exclude_from_sim no) (in_bom yes) (on_board yes) (dnp no)
-  (property "Reference" "R5301" (at 161.29 46.99 90) (effects (font (size 1.27 1.27))))
+  (property "Reference" "R5901" (at 161.29 46.99 90) (effects (font (size 1.27 1.27))))
   (property "Value" "10 Ω" (at 161.29 53.34 90) (effects (font (size 1.27 1.27))))
   (property "Spec" "0603" (at 161.29 55.88 90) (effects (font (size 1.27 1.27))))
@@
   (pin "1")
   (pin "2")
-  (instances (project "t1-main-board" (path "/7746052e-d7f9-59ad-ba73-bd2b74439529/cab3b4fb-5ec0-5c66-a197-75b8941e1631" (reference "R5301") (unit 1) (variant (name "production") (field (name "Value") (value "0 Ω")) (field (name "MPN") (value "RC0603JR-070RL")) (field (name "Manufacturer") (value "YAGEO"))))))
+  (instances (project "t1-main-board" (path "/7746052e-d7f9-59ad-ba73-bd2b74439529/cab3b4fb-5ec0-5c66-a197-75b8941e1631" (reference "R5901") (unit 1) (variant (name "production") (field (name "Value") (value "0 Ω")) (field (name "MPN") (value "RC0603JR-070RL")) (field (name "Manufacturer") (value "YAGEO"))))))
 )
 (rectangle (start 140.97 38.1) (end 181.61 58.42) (stroke (width 0) (type dash)) (fill (type none)))
@@
 (wire (pts (xy 157.48 50.8) (xy 157.48 48.26)) (stroke (width 0) (type default)))
 (symbol (lib_id "Connector:TestPoint") (at 157.48 48.26 0) (unit 1) (body_style 1) (exclude_from_sim no) (in_bom no) (on_board yes) (dnp no)
-  (property "Reference" "TP5301" (at 156.21 43.18 0) (effects (font (size 1.27 1.27)) (justify right)))
+  (property "Reference" "TP5901" (at 156.21 43.18 0) (effects (font (size 1.27 1.27)) (justify right)))
   (property "Value" "vcca1v8_pmu" (at 156.21 45.72 0) (effects (font (size 1.27 1.27)) (justify right)))
   (property "Footprint" "TestPoint:TestPoint_Pad_D1.0mm" (at 157.48 48.26 0) (effects (font (size 1.27 1.27))) (hide yes))
@@
   (property "Block" "blk.imu" (at 157.48 48.26 0) (effects (font (size 1.27 1.27))) (hide yes))
   (pin "1")
-  (instances (project "t1-main-board" (path "/7746052e-d7f9-59ad-ba73-bd2b74439529/cab3b4fb-5ec0-5c66-a197-75b8941e1631" (reference "TP5301") (unit 1))))
+  (instances (project "t1-main-board" (path "/7746052e-d7f9-59ad-ba73-bd2b74439529/cab3b4fb-5ec0-5c66-a197-75b8941e1631" (reference "TP5901") (unit 1))))
 )
 (symbol (lib_id "power:VCC") (at 138.43 50.8 90) (unit 1) (body_style 1) (exclude_from_sim no) (in_bom yes) (on_board yes) (dnp no)
@@
 (wire (pts (xy 170.18 50.8) (xy 170.18 48.26)) (stroke (width 0) (type default)))
 (symbol (lib_id "Connector:TestPoint") (at 170.18 48.26 0) (unit 1) (body_style 1) (exclude_from_sim no) (in_bom no) (on_board yes) (dnp no)
-  (property "Reference" "TP5302" (at 171.45 43.18 0) (effects (font (size 1.27 1.27)) (justify left)))
+  (property "Reference" "TP5902" (at 171.45 43.18 0) (effects (font (size 1.27 1.27)) (justify left)))
   (property "Value" "IMU_VDD" (at 171.45 45.72 0) (effects (font (size 1.27 1.27)) (justify left)))
   (property "Footprint" "TestPoint:TestPoint_Pad_D1.0mm" (at 170.18 48.26 0) (effects (font (size 1.27 1.27))) (hide yes))
@@
   (property "Block" "blk.imu" (at 170.18 48.26 0) (effects (font (size 1.27 1.27))) (hide yes))
   (pin "1")
-  (instances (project "t1-main-board" (path "/7746052e-d7f9-59ad-ba73-bd2b74439529/cab3b4fb-5ec0-5c66-a197-75b8941e1631" (reference "TP5302") (unit 1))))
+  (instances (project "t1-main-board" (path "/7746052e-d7f9-59ad-ba73-bd2b74439529/cab3b4fb-5ec0-5c66-a197-75b8941e1631" (reference "TP5902") (unit 1))))
 )
 (junction (at 189.23 50.8) (diameter 0) (color 0 0 0 0))
