File: board/hardware/t1-main-board/imu.kicad_sch (KiCad schematic)
At the start: 6 parts, among them U5901 LSM6DSV16XTR

Commit message: Board: capture blk.debug
Debug UART2 (1.8 V) and I2S/DSD pads with ground pads, reset, PMIC and
power-key pads (PCB-T-09), a pad on every spare SoC GPIO whose pinout v1
row names one (the DEBUG bus, on the SoC's right edge), and a rail pad
for each power-tree rail no other sheet probes (PCB-T-02). Each DAC
sheet carries a pad on its MCLK. The spares pinout v1 leaves without a
pad now carry no-connect flags. On the root, facing sheet pins are
joined directly only where the route meets no other symbol.

Co-Authored-By: Claude Opus 5.5 <noreply@anthropic.com>
Claude-Session: https://claude.ai/code/session_01Ei262h3TpgY9vyfNLMi5Mn
Parts:
- removed C5901, C5902: 100 nF, Capacitor_SMD:C_0402_1005Metric, symbol Device:C
- removed R5901: 10 Ω, Resistor_SMD:R_0603_1608Metric, symbol Device:R
- removed TP5901: vcca1v8_pmu, TestPoint:TestPoint_Pad_D1.0mm, symbol Connector:TestPoint
- removed TP5902: IMU_VDD, TestPoint:TestPoint_Pad_D1.0mm, symbol Connector:TestPoint
- removed U5901: LSM6DSV16XTR, STMicroelectronics:ST_LGA-14L_2.5x3mm_P0.5mm, symbol STMicroelectronics:LSM6DSV16XTR
- added C6001, C6002: 100 nF, Capacitor_SMD:C_0402_1005Metric, symbol Device:C
- added R6001: 10 Ω, Resistor_SMD:R_0603_1608Metric, symbol Device:R
- added TP6001: vcca1v8_pmu, TestPoint:TestPoint_Pad_D1.0mm, symbol Connector:TestPoint
- added TP6002: IMU_VDD, TestPoint:TestPoint_Pad_D1.0mm, symbol Connector:TestPoint
- added U6001: LSM6DSV16XTR, STMicroelectronics:ST_LGA-14L_2.5x3mm_P0.5mm, symbol STMicroelectronics:LSM6DSV16XTR
Connections:
- net GND: now also C6001.2, C6002.2, U6001.1 (SDO/SA0), U6001.2 (SDx/AH1/Qvar1), U6001.3 (SCx/AH2/Qvar2), U6001.6 (GND), U6001.7 (GND)
- net I2C2_SCL: now also U6001.13 (SCL)
- net I2C2_SDA: now also U6001.14 (SDA)
- net IMU_INT1: now also U6001.4 (INT1)
- net IMU_VDD: now also C6001.1, C6002.1, R6001.2, TP6002.1, U6001.12 (CS), U6001.5 (Vdd_IO), U6001.8 (Vdd)
- net vcca1v8_pmu: now also R6001.1, TP6001.1
Changed lines of the file:
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@@
 (title_block (title "Motion sensor") (date "2026-10-25") (rev "A") (company "The OpenDAP Project") (comment 1 "blk.imu") (comment 2 "LSM6DSV16X on I2C2 at 0x6A, INT1 wake on motion, always on"))
 (symbol (lib_id "STMicroelectronics:LSM6DSV16XTR") (at 55.88 77.47 0) (unit 1) (body_style 1) (exclude_from_sim no) (in_bom yes) (on_board yes) (dnp no)
-  (property "Reference" "U5901" (at 59.69 50.8 0) (effects (font (size 1.27 1.27)) (justify left)))
+  (property "Reference" "U6001" (at 59.69 50.8 0) (effects (font (size 1.27 1.27)) (justify left)))
   (property "Value" "LSM6DSV16XTR" (at 59.69 48.26 0) (effects (font (size 1.27 1.27)) (justify left)))
   (property "Footprint" "STMicroelectronics:ST_LGA-14L_2.5x3mm_P0.5mm" (at 55.88 77.47 0) (effects (font (size 1.27 1.27))) (hide yes))
@@
   (pin "6")
   (pin "7")
-  (instances (project "t1-main-board" (path "/7746052e-d7f9-59ad-ba73-bd2b74439529/cab3b4fb-5ec0-5c66-a197-75b8941e1631" (reference "U5901") (unit 1))))
+  (instances (project "t1-main-board" (path "/7746052e-d7f9-59ad-ba73-bd2b74439529/cab3b4fb-5ec0-5c66-a197-75b8941e1631" (reference "U6001") (unit 1))))
 )
 (wire (pts (xy 53.34 49.53) (xy 53.34 46.99)) (stroke (width 0) (type default)))
@@
 (no_connect (at 73.66 69.85))
 (symbol (lib_id "Device:C") (at 91.44 53.34 0) (unit 1) (body_style 1) (exclude_from_sim no) (in_bom yes) (on_board yes) (dnp no)
-  (property "Reference" "C5901" (at 93.98 52.07 0) (effects (font (size 1.27 1.27)) (justify left)))
+  (property "Reference" "C6001" (at 93.98 52.07 0) (effects (font (size 1.27 1.27)) (justify left)))
   (property "Value" "100 nF" (at 93.98 54.61 0) (effects (font (size 1.27 1.27)) (justify left)))
   (property "Footprint" "Capacitor_SMD:C_0402_1005Metric" (at 91.44 53.34 0) (effects (font (size 1.27 1.27))) (hide yes))
@@
   (pin "1")
   (pin "2")
-  (instances (project "t1-main-board" (path "/7746052e-d7f9-59ad-ba73-bd2b74439529/cab3b4fb-5ec0-5c66-a197-75b8941e1631" (reference "C5901") (unit 1))))
+  (instances (project "t1-main-board" (path "/7746052e-d7f9-59ad-ba73-bd2b74439529/cab3b4fb-5ec0-5c66-a197-75b8941e1631" (reference "C6001") (unit 1))))
 )
 (wire (pts (xy 91.44 49.53) (xy 91.44 46.99)) (stroke (width 0) (type default)))
@@
 )
 (symbol (lib_id "Device:C") (at 105.41 53.34 0) (unit 1) (body_style 1) (exclude_from_sim no) (in_bom yes) (on_board yes) (dnp no)
-  (property "Reference" "C5902" (at 107.95 52.07 0) (effects (font (size 1.27 1.27)) (justify left)))
+  (property "Reference" "C6002" (at 107.95 52.07 0) (effects (font (size 1.27 1.27)) (justify left)))
   (property "Value" "100 nF" (at 107.95 54.61 0) (effects (font (size 1.27 1.27)) (justify left)))
   (property "Footprint" "Capacitor_SMD:C_0402_1005Metric" (at 105.41 53.34 0) (effects (font (size 1.27 1.27))) (hide yes))
@@
   (pin "1")
   (pin "2")
-  (instances (project "t1-main-board" (path "/7746052e-d7f9-59ad-ba73-bd2b74439529/cab3b4fb-5ec0-5c66-a197-75b8941e1631" (reference "C5902") (unit 1))))
+  (instances (project "t1-main-board" (path "/7746052e-d7f9-59ad-ba73-bd2b74439529/cab3b4fb-5ec0-5c66-a197-75b8941e1631" (reference "C6002") (unit 1))))
 )
 (wire (pts (xy 105.41 49.53) (xy 105.41 46.99)) (stroke (width 0) (type default)))
@@
 (text "LSM6DSV16X at I2C2 0x6A (BOM v1 line 59)" (exclude_from_sim no) (at 24.13 34.29 0) (effects (font (size 2.54 2.54)) (justify left bottom)))
 (symbol (lib_id "Device:R") (at 163.83 50.8 90) (unit 1) (body_style 1) (exclude_from_sim no) (in_bom yes) (on_board yes) (dnp no)
-  (property "Reference" "R5901" (at 161.29 46.99 90) (effects (font (size 1.27 1.27))))
+  (property "Reference" "R6001" (at 161.29 46.99 90) (effects (font (size 1.27 1.27))))
   (property "Value" "10 Ω" (at 161.29 53.34 90) (effects (font (size 1.27 1.27))))
   (property "Spec" "0603" (at 161.29 55.88 90) (effects (font (size 1.27 1.27))))
@@
   (pin "1")
   (pin "2")
-  (instances (project "t1-main-board" (path "/7746052e-d7f9-59ad-ba73-bd2b74439529/cab3b4fb-5ec0-5c66-a197-75b8941e1631" (reference "R5901") (unit 1) (variant (name "production") (field (name "Value") (value "0 Ω")) (field (name "MPN") (value "RC0603JR-070RL")) (field (name "Manufacturer") (value "YAGEO"))))))
+  (instances (project "t1-main-board" (path "/7746052e-d7f9-59ad-ba73-bd2b74439529/cab3b4fb-5ec0-5c66-a197-75b8941e1631" (reference "R6001") (unit 1) (variant (name "production") (field (name "Value") (value "0 Ω")) (field (name "MPN") (value "RC0603JR-070RL")) (field (name "Manufacturer") (value "YAGEO"))))))
 )
 (rectangle (start 140.97 38.1) (end 181.61 58.42) (stroke (width 0) (type dash)) (fill (type none)))
@@
 (wire (pts (xy 157.48 50.8) (xy 157.48 48.26)) (stroke (width 0) (type default)))
 (symbol (lib_id "Connector:TestPoint") (at 157.48 48.26 0) (unit 1) (body_style 1) (exclude_from_sim no) (in_bom no) (on_board yes) (dnp no)
-  (property "Reference" "TP5901" (at 156.21 43.18 0) (effects (font (size 1.27 1.27)) (justify right)))
+  (property "Reference" "TP6001" (at 156.21 43.18 0) (effects (font (size 1.27 1.27)) (justify right)))
   (property "Value" "vcca1v8_pmu" (at 156.21 45.72 0) (effects (font (size 1.27 1.27)) (justify right)))
   (property "Footprint" "TestPoint:TestPoint_Pad_D1.0mm" (at 157.48 48.26 0) (effects (font (size 1.27 1.27))) (hide yes))
@@
   (property "Block" "blk.imu" (at 157.48 48.26 0) (effects (font (size 1.27 1.27))) (hide yes))
   (pin "1")
-  (instances (project "t1-main-board" (path "/7746052e-d7f9-59ad-ba73-bd2b74439529/cab3b4fb-5ec0-5c66-a197-75b8941e1631" (reference "TP5901") (unit 1))))
+  (instances (project "t1-main-board" (path "/7746052e-d7f9-59ad-ba73-bd2b74439529/cab3b4fb-5ec0-5c66-a197-75b8941e1631" (reference "TP6001") (unit 1))))
 )
 (symbol (lib_id "power:VCC") (at 138.43 50.8 90) (unit 1) (body_style 1) (exclude_from_sim no) (in_bom yes) (on_board yes) (dnp no)
@@
 (wire (pts (xy 170.18 50.8) (xy 170.18 48.26)) (stroke (width 0) (type default)))
 (symbol (lib_id "Connector:TestPoint") (at 170.18 48.26 0) (unit 1) (body_style 1) (exclude_from_sim no) (in_bom no) (on_board yes) (dnp no)
-  (property "Reference" "TP5902" (at 171.45 43.18 0) (effects (font (size 1.27 1.27)) (justify left)))
+  (property "Reference" "TP6002" (at 171.45 43.18 0) (effects (font (size 1.27 1.27)) (justify left)))
   (property "Value" "IMU_VDD" (at 171.45 45.72 0) (effects (font (size 1.27 1.27)) (justify left)))
   (property "Footprint" "TestPoint:TestPoint_Pad_D1.0mm" (at 170.18 48.26 0) (effects (font (size 1.27 1.27))) (hide yes))
@@
   (property "Block" "blk.imu" (at 170.18 48.26 0) (effects (font (size 1.27 1.27))) (hide yes))
   (pin "1")
-  (instances (project "t1-main-board" (path "/7746052e-d7f9-59ad-ba73-bd2b74439529/cab3b4fb-5ec0-5c66-a197-75b8941e1631" (reference "TP5902") (unit 1))))
+  (instances (project "t1-main-board" (path "/7746052e-d7f9-59ad-ba73-bd2b74439529/cab3b4fb-5ec0-5c66-a197-75b8941e1631" (reference "TP6002") (unit 1))))
 )
 (junction (at 189.23 50.8) (diameter 0) (color 0 0 0 0))

Commit message: Board: capture blk.cover-detect
COVER_DET_N on GPIO0_A6 (AJ38, PMUIO1, wake-capable), recorded in
pinout v1 (closes feature blocks G22): board-edge input and ground pads
for the case's actuator, 100 kΩ to vcc3v3_pmu, TPD1E10B06 at the pad
(BOM v1 line 143, PCB-L-10). The line rides the KEYS bus with the
buttons.

Co-Authored-By: Claude Opus 5.5 <noreply@anthropic.com>
Claude-Session: https://claude.ai/code/session_01Ei262h3TpgY9vyfNLMi5Mn
Parts:
- removed C6001, C6002: 100 nF, Capacitor_SMD:C_0402_1005Metric, symbol Device:C
- removed R6001: 10 Ω, Resistor_SMD:R_0603_1608Metric, symbol Device:R
- removed TP6001: vcca1v8_pmu, TestPoint:TestPoint_Pad_D1.0mm, symbol Connector:TestPoint
- removed TP6002: IMU_VDD, TestPoint:TestPoint_Pad_D1.0mm, symbol Connector:TestPoint
- removed U6001: LSM6DSV16XTR, STMicroelectronics:ST_LGA-14L_2.5x3mm_P0.5mm, symbol STMicroelectronics:LSM6DSV16XTR
- added C6101, C6102: 100 nF, Capacitor_SMD:C_0402_1005Metric, symbol Device:C
- added R6101: 10 Ω, Resistor_SMD:R_0603_1608Metric, symbol Device:R
- added TP6101: vcca1v8_pmu, TestPoint:TestPoint_Pad_D1.0mm, symbol Connector:TestPoint
- added TP6102: IMU_VDD, TestPoint:TestPoint_Pad_D1.0mm, symbol Connector:TestPoint
- added U6101: LSM6DSV16XTR, STMicroelectronics:ST_LGA-14L_2.5x3mm_P0.5mm, symbol STMicroelectronics:LSM6DSV16XTR
Connections:
- net GND: now also C6101.2, C6102.2, U6101.1 (SDO/SA0), U6101.2 (SDx/AH1/Qvar1), U6101.3 (SCx/AH2/Qvar2), U6101.6 (GND), U6101.7 (GND)
- net I2C2_SCL: now also U6101.13 (SCL)
- net I2C2_SDA: now also U6101.14 (SDA)
- net IMU_INT1: now also U6101.4 (INT1)
- net IMU_VDD: now also C6101.1, C6102.1, R6101.2, TP6102.1, U6101.12 (CS), U6101.5 (Vdd_IO), U6101.8 (Vdd)
- net vcca1v8_pmu: now also R6101.1, TP6101.1
Changed lines of the file:
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@@
 (title_block (title "Motion sensor") (date "2026-10-25") (rev "A") (company "The OpenDAP Project") (comment 1 "blk.imu") (comment 2 "LSM6DSV16X on I2C2 at 0x6A, INT1 wake on motion, always on"))
 (symbol (lib_id "STMicroelectronics:LSM6DSV16XTR") (at 55.88 77.47 0) (unit 1) (body_style 1) (exclude_from_sim no) (in_bom yes) (on_board yes) (dnp no)
-  (property "Reference" "U6001" (at 59.69 50.8 0) (effects (font (size 1.27 1.27)) (justify left)))
+  (property "Reference" "U6101" (at 59.69 50.8 0) (effects (font (size 1.27 1.27)) (justify left)))
   (property "Value" "LSM6DSV16XTR" (at 59.69 48.26 0) (effects (font (size 1.27 1.27)) (justify left)))
   (property "Footprint" "STMicroelectronics:ST_LGA-14L_2.5x3mm_P0.5mm" (at 55.88 77.47 0) (effects (font (size 1.27 1.27))) (hide yes))
@@
   (pin "6")
   (pin "7")
-  (instances (project "t1-main-board" (path "/7746052e-d7f9-59ad-ba73-bd2b74439529/cab3b4fb-5ec0-5c66-a197-75b8941e1631" (reference "U6001") (unit 1))))
+  (instances (project "t1-main-board" (path "/7746052e-d7f9-59ad-ba73-bd2b74439529/cab3b4fb-5ec0-5c66-a197-75b8941e1631" (reference "U6101") (unit 1))))
 )
 (wire (pts (xy 53.34 49.53) (xy 53.34 46.99)) (stroke (width 0) (type default)))
@@
 (no_connect (at 73.66 69.85))
 (symbol (lib_id "Device:C") (at 91.44 53.34 0) (unit 1) (body_style 1) (exclude_from_sim no) (in_bom yes) (on_board yes) (dnp no)
-  (property "Reference" "C6001" (at 93.98 52.07 0) (effects (font (size 1.27 1.27)) (justify left)))
+  (property "Reference" "C6101" (at 93.98 52.07 0) (effects (font (size 1.27 1.27)) (justify left)))
   (property "Value" "100 nF" (at 93.98 54.61 0) (effects (font (size 1.27 1.27)) (justify left)))
   (property "Footprint" "Capacitor_SMD:C_0402_1005Metric" (at 91.44 53.34 0) (effects (font (size 1.27 1.27))) (hide yes))
@@
   (pin "1")
   (pin "2")
-  (instances (project "t1-main-board" (path "/7746052e-d7f9-59ad-ba73-bd2b74439529/cab3b4fb-5ec0-5c66-a197-75b8941e1631" (reference "C6001") (unit 1))))
+  (instances (project "t1-main-board" (path "/7746052e-d7f9-59ad-ba73-bd2b74439529/cab3b4fb-5ec0-5c66-a197-75b8941e1631" (reference "C6101") (unit 1))))
 )
 (wire (pts (xy 91.44 49.53) (xy 91.44 46.99)) (stroke (width 0) (type default)))
@@
 )
 (symbol (lib_id "Device:C") (at 105.41 53.34 0) (unit 1) (body_style 1) (exclude_from_sim no) (in_bom yes) (on_board yes) (dnp no)
-  (property "Reference" "C6002" (at 107.95 52.07 0) (effects (font (size 1.27 1.27)) (justify left)))
+  (property "Reference" "C6102" (at 107.95 52.07 0) (effects (font (size 1.27 1.27)) (justify left)))
   (property "Value" "100 nF" (at 107.95 54.61 0) (effects (font (size 1.27 1.27)) (justify left)))
   (property "Footprint" "Capacitor_SMD:C_0402_1005Metric" (at 105.41 53.34 0) (effects (font (size 1.27 1.27))) (hide yes))
@@
   (pin "1")
   (pin "2")
-  (instances (project "t1-main-board" (path "/7746052e-d7f9-59ad-ba73-bd2b74439529/cab3b4fb-5ec0-5c66-a197-75b8941e1631" (reference "C6002") (unit 1))))
+  (instances (project "t1-main-board" (path "/7746052e-d7f9-59ad-ba73-bd2b74439529/cab3b4fb-5ec0-5c66-a197-75b8941e1631" (reference "C6102") (unit 1))))
 )
 (wire (pts (xy 105.41 49.53) (xy 105.41 46.99)) (stroke (width 0) (type default)))
@@
 (text "LSM6DSV16X at I2C2 0x6A (BOM v1 line 59)" (exclude_from_sim no) (at 24.13 34.29 0) (effects (font (size 2.54 2.54)) (justify left bottom)))
 (symbol (lib_id "Device:R") (at 163.83 50.8 90) (unit 1) (body_style 1) (exclude_from_sim no) (in_bom yes) (on_board yes) (dnp no)
-  (property "Reference" "R6001" (at 161.29 46.99 90) (effects (font (size 1.27 1.27))))
+  (property "Reference" "R6101" (at 161.29 46.99 90) (effects (font (size 1.27 1.27))))
   (property "Value" "10 Ω" (at 161.29 53.34 90) (effects (font (size 1.27 1.27))))
   (property "Spec" "0603" (at 161.29 55.88 90) (effects (font (size 1.27 1.27))))
@@
   (pin "1")
   (pin "2")
-  (instances (project "t1-main-board" (path "/7746052e-d7f9-59ad-ba73-bd2b74439529/cab3b4fb-5ec0-5c66-a197-75b8941e1631" (reference "R6001") (unit 1) (variant (name "production") (field (name "Value") (value "0 Ω")) (field (name "MPN") (value "RC0603JR-070RL")) (field (name "Manufacturer") (value "YAGEO"))))))
+  (instances (project "t1-main-board" (path "/7746052e-d7f9-59ad-ba73-bd2b74439529/cab3b4fb-5ec0-5c66-a197-75b8941e1631" (reference "R6101") (unit 1) (variant (name "production") (field (name "Value") (value "0 Ω")) (field (name "MPN") (value "RC0603JR-070RL")) (field (name "Manufacturer") (value "YAGEO"))))))
 )
 (rectangle (start 140.97 38.1) (end 181.61 58.42) (stroke (width 0) (type dash)) (fill (type none)))
@@
 (wire (pts (xy 157.48 50.8) (xy 157.48 48.26)) (stroke (width 0) (type default)))
 (symbol (lib_id "Connector:TestPoint") (at 157.48 48.26 0) (unit 1) (body_style 1) (exclude_from_sim no) (in_bom no) (on_board yes) (dnp no)
-  (property "Reference" "TP6001" (at 156.21 43.18 0) (effects (font (size 1.27 1.27)) (justify right)))
+  (property "Reference" "TP6101" (at 156.21 43.18 0) (effects (font (size 1.27 1.27)) (justify right)))
   (property "Value" "vcca1v8_pmu" (at 156.21 45.72 0) (effects (font (size 1.27 1.27)) (justify right)))
   (property "Footprint" "TestPoint:TestPoint_Pad_D1.0mm" (at 157.48 48.26 0) (effects (font (size 1.27 1.27))) (hide yes))
@@
   (property "Block" "blk.imu" (at 157.48 48.26 0) (effects (font (size 1.27 1.27))) (hide yes))
   (pin "1")
-  (instances (project "t1-main-board" (path "/7746052e-d7f9-59ad-ba73-bd2b74439529/cab3b4fb-5ec0-5c66-a197-75b8941e1631" (reference "TP6001") (unit 1))))
+  (instances (project "t1-main-board" (path "/7746052e-d7f9-59ad-ba73-bd2b74439529/cab3b4fb-5ec0-5c66-a197-75b8941e1631" (reference "TP6101") (unit 1))))
 )
 (symbol (lib_id "power:VCC") (at 138.43 50.8 90) (unit 1) (body_style 1) (exclude_from_sim no) (in_bom yes) (on_board yes) (dnp no)
@@
 (wire (pts (xy 170.18 50.8) (xy 170.18 48.26)) (stroke (width 0) (type default)))
 (symbol (lib_id "Connector:TestPoint") (at 170.18 48.26 0) (unit 1) (body_style 1) (exclude_from_sim no) (in_bom no) (on_board yes) (dnp no)
-  (property "Reference" "TP6002" (at 171.45 43.18 0) (effects (font (size 1.27 1.27)) (justify left)))
+  (property "Reference" "TP6102" (at 171.45 43.18 0) (effects (font (size 1.27 1.27)) (justify left)))
   (property "Value" "IMU_VDD" (at 171.45 45.72 0) (effects (font (size 1.27 1.27)) (justify left)))
   (property "Footprint" "TestPoint:TestPoint_Pad_D1.0mm" (at 170.18 48.26 0) (effects (font (size 1.27 1.27))) (hide yes))
@@
   (property "Block" "blk.imu" (at 170.18 48.26 0) (effects (font (size 1.27 1.27))) (hide yes))
   (pin "1")
-  (instances (project "t1-main-board" (path "/7746052e-d7f9-59ad-ba73-bd2b74439529/cab3b4fb-5ec0-5c66-a197-75b8941e1631" (reference "TP6002") (unit 1))))
+  (instances (project "t1-main-board" (path "/7746052e-d7f9-59ad-ba73-bd2b74439529/cab3b4fb-5ec0-5c66-a197-75b8941e1631" (reference "TP6102") (unit 1))))
 )
 (junction (at 189.23 50.8) (diameter 0) (color 0 0 0 0))

Commit message: Board: capture blk.mic-ambient and links #34, #35
IM73D122 on PDM CLK1 and SDI1 (BOM v1 line 34, pinout v1 AK2 and 1P2),
LR to ground, 22 Ω clock series, VDD from MIC_1V8 through link #35.
Link #34 on blk.mic-main makes the faceplate branch the rail MIC_1V8_FP
for contact 40 (power tree §4.12, G10). kicad-lib moves to e46bda4 for
the IM73D122, TPS3808G01, SN74LVC1G58 and BAT54 parts.

Co-Authored-By: Claude Opus 5.5 <noreply@anthropic.com>
Claude-Session: https://claude.ai/code/session_01Ei262h3TpgY9vyfNLMi5Mn
Parts:
- removed C6101, C6102: 100 nF, Capacitor_SMD:C_0402_1005Metric, symbol Device:C
- removed R6101: 10 Ω, Resistor_SMD:R_0603_1608Metric, symbol Device:R
- removed TP6101: vcca1v8_pmu, TestPoint:TestPoint_Pad_D1.0mm, symbol Connector:TestPoint
- removed TP6102: IMU_VDD, TestPoint:TestPoint_Pad_D1.0mm, symbol Connector:TestPoint
- removed U6101: LSM6DSV16XTR, STMicroelectronics:ST_LGA-14L_2.5x3mm_P0.5mm, symbol STMicroelectronics:LSM6DSV16XTR
- added C6201, C6202: 100 nF, Capacitor_SMD:C_0402_1005Metric, symbol Device:C
- added R6201: 10 Ω, Resistor_SMD:R_0603_1608Metric, symbol Device:R
- added TP6201: vcca1v8_pmu, TestPoint:TestPoint_Pad_D1.0mm, symbol Connector:TestPoint
- added TP6202: IMU_VDD, TestPoint:TestPoint_Pad_D1.0mm, symbol Connector:TestPoint
- added U6201: LSM6DSV16XTR, STMicroelectronics:ST_LGA-14L_2.5x3mm_P0.5mm, symbol STMicroelectronics:LSM6DSV16XTR
Connections:
- net GND: now also C6201.2, C6202.2, U6201.1 (SDO/SA0), U6201.2 (SDx/AH1/Qvar1), U6201.3 (SCx/AH2/Qvar2), U6201.6 (GND), U6201.7 (GND)
- net I2C2_SCL: now also U6201.13 (SCL)
- net I2C2_SDA: now also U6201.14 (SDA)
- net IMU_INT1: now also U6201.4 (INT1)
- net IMU_VDD: now also C6201.1, C6202.1, R6201.2, TP6202.1, U6201.12 (CS), U6201.5 (Vdd_IO), U6201.8 (Vdd)
- net vcca1v8_pmu: now also R6201.1, TP6201.1
