File: board/hardware/t1-main-board/imu.kicad_sch (KiCad schematic)
At the start: 6 parts, among them U6201 LSM6DSV16XTR

Commit message: Board: capture blk.maskrom
Power + Vol- at a cold power-on pull eMMC D0 low inside the TPS3808G01
boot window (BOM v1 lines 35, 78, 97, 98; sim/maskrom): SENSE 280k/100k,
CT 390 nF, WINDOW_N with its pad, SN74LVC1G57 and SN74LVC1G58 on
vcca1v8_pmu, BAT54 from PWRON_N, DMG1012T through 1 kΩ to EMMC_D0.
Every block in use now has its sheet; the README states the remaining
single-pin nets.

Co-Authored-By: Claude Opus 5.5 <noreply@anthropic.com>
Claude-Session: https://claude.ai/code/session_01Ei262h3TpgY9vyfNLMi5Mn
Parts:
- removed C6201, C6202: 100 nF, Capacitor_SMD:C_0402_1005Metric, symbol Device:C
- removed R6201: 10 Ω, Resistor_SMD:R_0603_1608Metric, symbol Device:R
- removed TP6201: vcca1v8_pmu, TestPoint:TestPoint_Pad_D1.0mm, symbol Connector:TestPoint
- removed TP6202: IMU_VDD, TestPoint:TestPoint_Pad_D1.0mm, symbol Connector:TestPoint
- removed U6201: LSM6DSV16XTR, STMicroelectronics:ST_LGA-14L_2.5x3mm_P0.5mm, symbol STMicroelectronics:LSM6DSV16XTR
- added C6301, C6302: 100 nF, Capacitor_SMD:C_0402_1005Metric, symbol Device:C
- added R6301: 10 Ω, Resistor_SMD:R_0603_1608Metric, symbol Device:R
- added TP6301: vcca1v8_pmu, TestPoint:TestPoint_Pad_D1.0mm, symbol Connector:TestPoint
- added TP6302: IMU_VDD, TestPoint:TestPoint_Pad_D1.0mm, symbol Connector:TestPoint
- added U6301: LSM6DSV16XTR, STMicroelectronics:ST_LGA-14L_2.5x3mm_P0.5mm, symbol STMicroelectronics:LSM6DSV16XTR
Connections:
- net GND: now also C6301.2, C6302.2, U6301.1 (SDO/SA0), U6301.2 (SDx/AH1/Qvar1), U6301.3 (SCx/AH2/Qvar2), U6301.6 (GND), U6301.7 (GND)
- net I2C2_SCL: now also U6301.13 (SCL)
- net I2C2_SDA: now also U6301.14 (SDA)
- net IMU_INT1: now also U6301.4 (INT1)
- net IMU_VDD: now also C6301.1, C6302.1, R6301.2, TP6302.1, U6301.12 (CS), U6301.5 (Vdd_IO), U6301.8 (Vdd)
- net vcca1v8_pmu: now also R6301.1, TP6301.1
Changed lines of the file:
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@@
 (title_block (title "Motion sensor") (date "2026-10-25") (rev "A") (company "The OpenDAP Project") (comment 1 "blk.imu") (comment 2 "LSM6DSV16X on I2C2 at 0x6A, INT1 wake on motion, always on"))
 (symbol (lib_id "STMicroelectronics:LSM6DSV16XTR") (at 55.88 77.47 0) (unit 1) (body_style 1) (exclude_from_sim no) (in_bom yes) (on_board yes) (dnp no)
-  (property "Reference" "U6201" (at 59.69 50.8 0) (effects (font (size 1.27 1.27)) (justify left)))
+  (property "Reference" "U6301" (at 59.69 50.8 0) (effects (font (size 1.27 1.27)) (justify left)))
   (property "Value" "LSM6DSV16XTR" (at 59.69 48.26 0) (effects (font (size 1.27 1.27)) (justify left)))
   (property "Footprint" "STMicroelectronics:ST_LGA-14L_2.5x3mm_P0.5mm" (at 55.88 77.47 0) (effects (font (size 1.27 1.27))) (hide yes))
@@
   (pin "6")
   (pin "7")
-  (instances (project "t1-main-board" (path "/7746052e-d7f9-59ad-ba73-bd2b74439529/cab3b4fb-5ec0-5c66-a197-75b8941e1631" (reference "U6201") (unit 1))))
+  (instances (project "t1-main-board" (path "/7746052e-d7f9-59ad-ba73-bd2b74439529/cab3b4fb-5ec0-5c66-a197-75b8941e1631" (reference "U6301") (unit 1))))
 )
 (wire (pts (xy 53.34 49.53) (xy 53.34 46.99)) (stroke (width 0) (type default)))
@@
 (no_connect (at 73.66 69.85))
 (symbol (lib_id "Device:C") (at 91.44 53.34 0) (unit 1) (body_style 1) (exclude_from_sim no) (in_bom yes) (on_board yes) (dnp no)
-  (property "Reference" "C6201" (at 93.98 52.07 0) (effects (font (size 1.27 1.27)) (justify left)))
+  (property "Reference" "C6301" (at 93.98 52.07 0) (effects (font (size 1.27 1.27)) (justify left)))
   (property "Value" "100 nF" (at 93.98 54.61 0) (effects (font (size 1.27 1.27)) (justify left)))
   (property "Footprint" "Capacitor_SMD:C_0402_1005Metric" (at 91.44 53.34 0) (effects (font (size 1.27 1.27))) (hide yes))
@@
   (pin "1")
   (pin "2")
-  (instances (project "t1-main-board" (path "/7746052e-d7f9-59ad-ba73-bd2b74439529/cab3b4fb-5ec0-5c66-a197-75b8941e1631" (reference "C6201") (unit 1))))
+  (instances (project "t1-main-board" (path "/7746052e-d7f9-59ad-ba73-bd2b74439529/cab3b4fb-5ec0-5c66-a197-75b8941e1631" (reference "C6301") (unit 1))))
 )
 (wire (pts (xy 91.44 49.53) (xy 91.44 46.99)) (stroke (width 0) (type default)))
@@
 )
 (symbol (lib_id "Device:C") (at 105.41 53.34 0) (unit 1) (body_style 1) (exclude_from_sim no) (in_bom yes) (on_board yes) (dnp no)
-  (property "Reference" "C6202" (at 107.95 52.07 0) (effects (font (size 1.27 1.27)) (justify left)))
+  (property "Reference" "C6302" (at 107.95 52.07 0) (effects (font (size 1.27 1.27)) (justify left)))
   (property "Value" "100 nF" (at 107.95 54.61 0) (effects (font (size 1.27 1.27)) (justify left)))
   (property "Footprint" "Capacitor_SMD:C_0402_1005Metric" (at 105.41 53.34 0) (effects (font (size 1.27 1.27))) (hide yes))
@@
   (pin "1")
   (pin "2")
-  (instances (project "t1-main-board" (path "/7746052e-d7f9-59ad-ba73-bd2b74439529/cab3b4fb-5ec0-5c66-a197-75b8941e1631" (reference "C6202") (unit 1))))
+  (instances (project "t1-main-board" (path "/7746052e-d7f9-59ad-ba73-bd2b74439529/cab3b4fb-5ec0-5c66-a197-75b8941e1631" (reference "C6302") (unit 1))))
 )
 (wire (pts (xy 105.41 49.53) (xy 105.41 46.99)) (stroke (width 0) (type default)))
@@
 (text "LSM6DSV16X at I2C2 0x6A (BOM v1 line 59)" (exclude_from_sim no) (at 24.13 34.29 0) (effects (font (size 2.54 2.54)) (justify left bottom)))
 (symbol (lib_id "Device:R") (at 163.83 50.8 90) (unit 1) (body_style 1) (exclude_from_sim no) (in_bom yes) (on_board yes) (dnp no)
-  (property "Reference" "R6201" (at 161.29 46.99 90) (effects (font (size 1.27 1.27))))
+  (property "Reference" "R6301" (at 161.29 46.99 90) (effects (font (size 1.27 1.27))))
   (property "Value" "10 Ω" (at 161.29 53.34 90) (effects (font (size 1.27 1.27))))
   (property "Spec" "0603" (at 161.29 55.88 90) (effects (font (size 1.27 1.27))))
@@
   (pin "1")
   (pin "2")
-  (instances (project "t1-main-board" (path "/7746052e-d7f9-59ad-ba73-bd2b74439529/cab3b4fb-5ec0-5c66-a197-75b8941e1631" (reference "R6201") (unit 1) (variant (name "production") (field (name "Value") (value "0 Ω")) (field (name "MPN") (value "RC0603JR-070RL")) (field (name "Manufacturer") (value "YAGEO"))))))
+  (instances (project "t1-main-board" (path "/7746052e-d7f9-59ad-ba73-bd2b74439529/cab3b4fb-5ec0-5c66-a197-75b8941e1631" (reference "R6301") (unit 1) (variant (name "production") (field (name "Value") (value "0 Ω")) (field (name "MPN") (value "RC0603JR-070RL")) (field (name "Manufacturer") (value "YAGEO"))))))
 )
 (rectangle (start 140.97 38.1) (end 181.61 58.42) (stroke (width 0) (type dash)) (fill (type none)))
@@
 (wire (pts (xy 157.48 50.8) (xy 157.48 48.26)) (stroke (width 0) (type default)))
 (symbol (lib_id "Connector:TestPoint") (at 157.48 48.26 0) (unit 1) (body_style 1) (exclude_from_sim no) (in_bom no) (on_board yes) (dnp no)
-  (property "Reference" "TP6201" (at 156.21 43.18 0) (effects (font (size 1.27 1.27)) (justify right)))
+  (property "Reference" "TP6301" (at 156.21 43.18 0) (effects (font (size 1.27 1.27)) (justify right)))
   (property "Value" "vcca1v8_pmu" (at 156.21 45.72 0) (effects (font (size 1.27 1.27)) (justify right)))
   (property "Footprint" "TestPoint:TestPoint_Pad_D1.0mm" (at 157.48 48.26 0) (effects (font (size 1.27 1.27))) (hide yes))
@@
   (property "Block" "blk.imu" (at 157.48 48.26 0) (effects (font (size 1.27 1.27))) (hide yes))
   (pin "1")
-  (instances (project "t1-main-board" (path "/7746052e-d7f9-59ad-ba73-bd2b74439529/cab3b4fb-5ec0-5c66-a197-75b8941e1631" (reference "TP6201") (unit 1))))
+  (instances (project "t1-main-board" (path "/7746052e-d7f9-59ad-ba73-bd2b74439529/cab3b4fb-5ec0-5c66-a197-75b8941e1631" (reference "TP6301") (unit 1))))
 )
 (symbol (lib_id "power:VCC") (at 138.43 50.8 90) (unit 1) (body_style 1) (exclude_from_sim no) (in_bom yes) (on_board yes) (dnp no)
@@
 (wire (pts (xy 170.18 50.8) (xy 170.18 48.26)) (stroke (width 0) (type default)))
 (symbol (lib_id "Connector:TestPoint") (at 170.18 48.26 0) (unit 1) (body_style 1) (exclude_from_sim no) (in_bom no) (on_board yes) (dnp no)
-  (property "Reference" "TP6202" (at 171.45 43.18 0) (effects (font (size 1.27 1.27)) (justify left)))
+  (property "Reference" "TP6302" (at 171.45 43.18 0) (effects (font (size 1.27 1.27)) (justify left)))
   (property "Value" "IMU_VDD" (at 171.45 45.72 0) (effects (font (size 1.27 1.27)) (justify left)))
   (property "Footprint" "TestPoint:TestPoint_Pad_D1.0mm" (at 170.18 48.26 0) (effects (font (size 1.27 1.27))) (hide yes))
@@
   (property "Block" "blk.imu" (at 170.18 48.26 0) (effects (font (size 1.27 1.27))) (hide yes))
   (pin "1")
-  (instances (project "t1-main-board" (path "/7746052e-d7f9-59ad-ba73-bd2b74439529/cab3b4fb-5ec0-5c66-a197-75b8941e1631" (reference "TP6202") (unit 1))))
+  (instances (project "t1-main-board" (path "/7746052e-d7f9-59ad-ba73-bd2b74439529/cab3b4fb-5ec0-5c66-a197-75b8941e1631" (reference "TP6302") (unit 1))))
 )
 (junction (at 189.23 50.8) (diameter 0) (color 0 0 0 0))

Commit message: Compaction: lower inductors, 0201 decoupling, 0.8 mm signal test pads
A matrix tool (hardware/studies/compaction) checks each candidate against
the design's stresses: same inductance, design peak <= 70 % and the
converter's maximum limit <= 100 % of Isat (30 % drop), height zones,
ratings at least twice the rail, PCB-D-06; sourcing outcome per part.

Applied (placement v1 decision 12, BOM v1.15):
- L601, L4401: XGL4015-102MEC (1.5 mm) for XAL/XGL4020-102MEC (2.1 mm);
- L1001, L5101: XGL4015-471MEC (1.5 mm) for Wurth 744373240047, on the
  stock XxL4020 land (the Wurth land was never drawn);
- L1201 is 1.2 mm (XGL4012, per-MPN heights): it moves next to the SoC;
- 58 x 100 nF decoupling on rails <= 3.3 V in core/IO/radio: 0201;
- 51 test pads on signal nets: 0.8 mm (PCB-D-06 v0.16, JLCPCB guide).
Kept: L901, L2802 (XGL4015 at 103 % of Isat at the limit); no thinner
0805/1206 capacitor passes (obsolete, NRND or unlisted).

Board need 113 % -> 111 % (core band 227 -> 203 %, power band 258 ->
233 %, radio band 19 -> 0 %); only C904 still relies on PCB-Z-04.
ERC 0 errors, craft Q1 met, DRC 0 errors (605 warnings), pcb and study
tests pass, rules test board PASS.

Co-Authored-By: Claude Opus 5.5 <noreply@anthropic.com>
Claude-Session: https://claude.ai/code/session_01Ei262h3TpgY9vyfNLMi5Mn
Parts:
- C6301, C6302: footprint Capacitor_SMD:C_0402_1005Metric -> Capacitor_SMD:C_0201_0603Metric; MPN GRM155R71C104KA88D -> GRM033R61A104KE15D
Changed lines of the file:
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@@
   (property "Reference" "C6301" (at 93.98 52.07 0) (effects (font (size 1.27 1.27)) (justify left)))
   (property "Value" "100 nF" (at 93.98 54.61 0) (effects (font (size 1.27 1.27)) (justify left)))
-  (property "Footprint" "Capacitor_SMD:C_0402_1005Metric" (at 91.44 53.34 0) (effects (font (size 1.27 1.27))) (hide yes))
-  (property "Datasheet" "https://www.murata.com/en-us/products/productdetail?partno=GRM155R71C104KA88D" (at 91.44 53.34 0) (effects (font (size 1.27 1.27))) (hide yes))
-  (property "Description" "Capacitor, 100 nF, 16 V, X7R, 0402" (at 91.44 53.34 0) (effects (font (size 1.27 1.27))) (hide yes))
+  (property "Footprint" "Capacitor_SMD:C_0201_0603Metric" (at 91.44 53.34 0) (effects (font (size 1.27 1.27))) (hide yes))
+  (property "Datasheet" "https://www.murata.com/en-us/products/productdetail?partno=GRM033R61A104KE15D" (at 91.44 53.34 0) (effects (font (size 1.27 1.27))) (hide yes))
+  (property "Description" "Capacitor, 100 nF, 10 V, X5R, 0201" (at 91.44 53.34 0) (effects (font (size 1.27 1.27))) (hide yes))
   (property "Manufacturer" "Murata" (at 91.44 53.34 0) (effects (font (size 1.27 1.27))) (hide yes))
-  (property "MPN" "GRM155R71C104KA88D" (at 91.44 53.34 0) (effects (font (size 1.27 1.27))) (hide yes))
+  (property "MPN" "GRM033R61A104KE15D" (at 91.44 53.34 0) (effects (font (size 1.27 1.27))) (hide yes))
   (property "Block" "blk.imu" (at 91.44 53.34 0) (effects (font (size 1.27 1.27))) (hide yes))
   (pin "1")
@@
   (property "Reference" "C6302" (at 107.95 52.07 0) (effects (font (size 1.27 1.27)) (justify left)))
   (property "Value" "100 nF" (at 107.95 54.61 0) (effects (font (size 1.27 1.27)) (justify left)))
-  (property "Footprint" "Capacitor_SMD:C_0402_1005Metric" (at 105.41 53.34 0) (effects (font (size 1.27 1.27))) (hide yes))
-  (property "Datasheet" "https://www.murata.com/en-us/products/productdetail?partno=GRM155R71C104KA88D" (at 105.41 53.34 0) (effects (font (size 1.27 1.27))) (hide yes))
-  (property "Description" "Capacitor, 100 nF, 16 V, X7R, 0402" (at 105.41 53.34 0) (effects (font (size 1.27 1.27))) (hide yes))
+  (property "Footprint" "Capacitor_SMD:C_0201_0603Metric" (at 105.41 53.34 0) (effects (font (size 1.27 1.27))) (hide yes))
+  (property "Datasheet" "https://www.murata.com/en-us/products/productdetail?partno=GRM033R61A104KE15D" (at 105.41 53.34 0) (effects (font (size 1.27 1.27))) (hide yes))
+  (property "Description" "Capacitor, 100 nF, 10 V, X5R, 0201" (at 105.41 53.34 0) (effects (font (size 1.27 1.27))) (hide yes))
   (property "Manufacturer" "Murata" (at 105.41 53.34 0) (effects (font (size 1.27 1.27))) (hide yes))
-  (property "MPN" "GRM155R71C104KA88D" (at 105.41 53.34 0) (effects (font (size 1.27 1.27))) (hide yes))
+  (property "MPN" "GRM033R61A104KE15D" (at 105.41 53.34 0) (effects (font (size 1.27 1.27))) (hide yes))
   (property "Block" "blk.imu" (at 105.41 53.34 0) (effects (font (size 1.27 1.27))) (hide yes))
   (pin "1")

Commit message: Board on libs v0.2.0: lower-case kebab vendor keys (HL-13)
The libs submodule moves to v0.2.0 (5f24483). Every library nickname in
the generator, the placement tool and the floorplan study follows the
key table (Texas_Instruments -> texas-instruments, OpenDAP_Device ->
opendap-generic, Rockchip and Rockchip_PMIC -> rockchip, ...); the
library tables are written from the files. Schematic and board
regenerated.

Checks: ERC 0 errors (warnings unchanged); DRC 0 errors, 605 warnings,
the same counts by type, schematic parity 0; every placement identical;
craft Q1 met; pcb tests pass; STEP export resolves every libs 3D model
(the 27 parts without a model are KiCad stock lands that have none).

Co-Authored-By: Claude Opus 5.5 <noreply@anthropic.com>
Claude-Session: https://claude.ai/code/session_01Ei262h3TpgY9vyfNLMi5Mn
Parts:
- U6301: footprint STMicroelectronics:ST_LGA-14L_2.5x3mm_P0.5mm -> stmicroelectronics:ST_LGA-14L_2.5x3mm_P0.5mm; symbol STMicroelectronics:LSM6DSV16XTR -> stmicroelectronics:LSM6DSV16XTR
Changed lines of the file:
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@@
 (paper "A4")
 (title_block (title "Motion sensor") (date "2026-10-25") (rev "A") (company "The OpenDAP Project") (comment 1 "blk.imu") (comment 2 "LSM6DSV16X on I2C2 at 0x6A, INT1 wake on motion, always on"))
-(symbol (lib_id "STMicroelectronics:LSM6DSV16XTR") (at 55.88 77.47 0) (unit 1) (body_style 1) (exclude_from_sim no) (in_bom yes) (on_board yes) (dnp no)
+(symbol (lib_id "stmicroelectronics:LSM6DSV16XTR") (at 55.88 77.47 0) (unit 1) (body_style 1) (exclude_from_sim no) (in_bom yes) (on_board yes) (dnp no)
   (property "Reference" "U6301" (at 59.69 50.8 0) (effects (font (size 1.27 1.27)) (justify left)))
   (property "Value" "LSM6DSV16XTR" (at 59.69 48.26 0) (effects (font (size 1.27 1.27)) (justify left)))
-  (property "Footprint" "STMicroelectronics:ST_LGA-14L_2.5x3mm_P0.5mm" (at 55.88 77.47 0) (effects (font (size 1.27 1.27))) (hide yes))
+  (property "Footprint" "stmicroelectronics:ST_LGA-14L_2.5x3mm_P0.5mm" (at 55.88 77.47 0) (effects (font (size 1.27 1.27))) (hide yes))
   (property "Datasheet" "https://www.st.com/resource/en/datasheet/lsm6dsv16x.pdf" (at 55.88 77.47 0) (effects (font (size 1.27 1.27))) (hide yes))
   (property "Description" "6-axis IMU, 3-axis accelerometer and 3-axis gyroscope, sensor fusion, finite state machine, machine learning core, Qvar, I2C / MIPI I3C / SPI, two interrupts, LGA-14L 2.5 x 3.0 mm" (at 55.88 77.47 0) (effects (font (size 1.27 1.27))) (hide yes))
