File: board/hardware/t1-main-board/microsd.kicad_sch (KiCad schematic)
At the start: 15 parts, among them J6201 DM3AT-SF-PEJM5, U6201 TPD4E05U06DQAR, U6202 TPD4E05U06DQAR

Commit message: Board: capture blk.current-monitors
Five INA236 on I2C1 (0x40-0x43, 0x48) with their shunts, per power tree
§4.12 and BOM v1 lines 54 and 136. The measured branches are rails of
their own (VSYS_SRC, VSYS_LV_AUDIO, VSYS_AUDIO, VSYS_LV_BL, VSYS_P5V1),
fed through the shunts on this sheet; the charger, audio, backlight and
5.1 V sheets take them. The root's layout may leave a stack level empty,
so the block sits under the notes; IC bboxes hold turned rail values;
passive rows hold a bottom rail's text.

Co-Authored-By: Claude Opus 5.5 <noreply@anthropic.com>
Claude-Session: https://claude.ai/code/session_01Ei262h3TpgY9vyfNLMi5Mn
Parts:
- removed C6201: 10 µF, Capacitor_SMD:C_0603_1608Metric, symbol Device:C
- removed C6202: 100 nF, Capacitor_SMD:C_0402_1005Metric, symbol Device:C
- removed J6201: DM3AT-SF-PEJM5, Hirose:Hirose_DM3AT-SF-PEJM5_microSD_PushPush_Top, symbol Hirose:DM3AT-SF-PEJM5
- removed R6201, R6202, R6203, R6204, R6205, R6206: 22 Ω, Resistor_SMD:R_0402_1005Metric, symbol Device:R
- removed R6207: 100 Ω, Resistor_SMD:R_0402_1005Metric, symbol Device:R
- removed R6208: 100 mΩ, Resistor_SMD:R_0603_1608Metric, symbol Device:R
- removed TP6201: vcc3v3_sd, TestPoint:TestPoint_Pad_D1.0mm, symbol Connector:TestPoint
- removed TP6202: SD_VDD, TestPoint:TestPoint_Pad_D1.0mm, symbol Connector:TestPoint
- removed U6201, U6202: TPD4E05U06DQAR, Texas_Instruments:Texas_DQA0010A_USON-10_1x2.5mm_P0.5mm, symbol Texas_Instruments:TPD4E05U06DQAR
- added C6301: 10 µF, Capacitor_SMD:C_0603_1608Metric, symbol Device:C
- added C6302: 100 nF, Capacitor_SMD:C_0402_1005Metric, symbol Device:C
- added J6301: DM3AT-SF-PEJM5, Hirose:Hirose_DM3AT-SF-PEJM5_microSD_PushPush_Top, symbol Hirose:DM3AT-SF-PEJM5
- added R6301, R6302, R6303, R6304, R6305, R6306: 22 Ω, Resistor_SMD:R_0402_1005Metric, symbol Device:R
- added R6307: 100 Ω, Resistor_SMD:R_0402_1005Metric, symbol Device:R
- added R6308: 100 mΩ, Resistor_SMD:R_0603_1608Metric, symbol Device:R
- added TP6301: vcc3v3_sd, TestPoint:TestPoint_Pad_D1.0mm, symbol Connector:TestPoint
- added TP6302: SD_VDD, TestPoint:TestPoint_Pad_D1.0mm, symbol Connector:TestPoint
- added U6301, U6302: TPD4E05U06DQAR, Texas_Instruments:Texas_DQA0010A_USON-10_1x2.5mm_P0.5mm, symbol Texas_Instruments:TPD4E05U06DQAR
Connections:
- net GND: now also C6301.2, C6302.2, J6301.6 (VSS), J6301.B (DET_B), J6301.S1 (SHIELD), U6301.3 (GND), U6301.8 (GND), U6302.3 (GND), U6302.8 (GND)
- net SD_CLK: now also R6301.1
- net SD_CLK_C: now also J6301.5 (CLK), R6301.2, U6301.1 (D1+)
- net SD_CMD: now also R6302.1
- net SD_CMD_C: now also J6301.3 (CMD), R6302.2, U6301.2 (D1-)
- net SD_D0: now also R6303.1
- net SD_D0_C: now also J6301.7 (DAT0), R6303.2, U6301.4 (D2+)
- net SD_D1: now also R6304.1
- net SD_D1_C: now also J6301.8 (DAT1), R6304.2, U6301.5 (D2-)
- net SD_D2: now also R6305.1
- net SD_D2_C: now also J6301.1 (DAT2), R6305.2, U6302.1 (D1+)
- net SD_D3: now also R6306.1
- net SD_D3_C: now also J6301.2 (CD/DAT3), R6306.2, U6302.2 (D1-)
- net SD_DET_C: now also J6301.A (DET_A), R6307.2
- net SD_DET_N: now also R6307.1
- net SD_VDD: now also C6301.1, C6302.1, J6301.4 (VDD), R6308.2, TP6302.1
- net vcc3v3_sd: now also R6308.1, TP6301.1

Commit message: Board: capture blk.status-led
LP5521 at 0x32 on I2C2 (BOM v1 line 105) with its charge-pump
capacitors, EN on vcca1v8_pmu, VDD from VSYS_LV through link #22;
LED_R/G/B reach the faceplate connector as the LED bus alias. The
faceplate row of the root is re-packed so five full columns sit left of
the title block.

Co-Authored-By: Claude Opus 5.5 <noreply@anthropic.com>
Claude-Session: https://claude.ai/code/session_01Ei262h3TpgY9vyfNLMi5Mn
Parts:
- removed C6301: 10 µF, Capacitor_SMD:C_0603_1608Metric, symbol Device:C
- removed C6302: 100 nF, Capacitor_SMD:C_0402_1005Metric, symbol Device:C
- removed J6301: DM3AT-SF-PEJM5, Hirose:Hirose_DM3AT-SF-PEJM5_microSD_PushPush_Top, symbol Hirose:DM3AT-SF-PEJM5
- removed R6301, R6302, R6303, R6304, R6305, R6306: 22 Ω, Resistor_SMD:R_0402_1005Metric, symbol Device:R
- removed R6307: 100 Ω, Resistor_SMD:R_0402_1005Metric, symbol Device:R
- removed R6308: 100 mΩ, Resistor_SMD:R_0603_1608Metric, symbol Device:R
- removed TP6301: vcc3v3_sd, TestPoint:TestPoint_Pad_D1.0mm, symbol Connector:TestPoint
- removed TP6302: SD_VDD, TestPoint:TestPoint_Pad_D1.0mm, symbol Connector:TestPoint
- removed U6301, U6302: TPD4E05U06DQAR, Texas_Instruments:Texas_DQA0010A_USON-10_1x2.5mm_P0.5mm, symbol Texas_Instruments:TPD4E05U06DQAR
- added C5801: 10 µF, Capacitor_SMD:C_0603_1608Metric, symbol Device:C
- added C5802: 100 nF, Capacitor_SMD:C_0402_1005Metric, symbol Device:C
- added J5801: DM3AT-SF-PEJM5, Hirose:Hirose_DM3AT-SF-PEJM5_microSD_PushPush_Top, symbol Hirose:DM3AT-SF-PEJM5
- added R5801, R5802, R5803, R5804, R5805, R5806: 22 Ω, Resistor_SMD:R_0402_1005Metric, symbol Device:R
- added R5807: 100 Ω, Resistor_SMD:R_0402_1005Metric, symbol Device:R
- added R5808: 100 mΩ, Resistor_SMD:R_0603_1608Metric, symbol Device:R
- added TP5801: vcc3v3_sd, TestPoint:TestPoint_Pad_D1.0mm, symbol Connector:TestPoint
- added TP5802: SD_VDD, TestPoint:TestPoint_Pad_D1.0mm, symbol Connector:TestPoint
- added U5801, U5802: TPD4E05U06DQAR, Texas_Instruments:Texas_DQA0010A_USON-10_1x2.5mm_P0.5mm, symbol Texas_Instruments:TPD4E05U06DQAR
Connections:
- net GND: now also C5801.2, C5802.2, J5801.6 (VSS), J5801.B (DET_B), J5801.S1 (SHIELD), U5801.3 (GND), U5801.8 (GND), U5802.3 (GND), U5802.8 (GND)
- net SD_CLK: now also R5801.1
- net SD_CLK_C: now also J5801.5 (CLK), R5801.2, U5801.1 (D1+)
- net SD_CMD: now also R5802.1
- net SD_CMD_C: now also J5801.3 (CMD), R5802.2, U5801.2 (D1-)
- net SD_D0: now also R5803.1
- net SD_D0_C: now also J5801.7 (DAT0), R5803.2, U5801.4 (D2+)
- net SD_D1: now also R5804.1
- net SD_D1_C: now also J5801.8 (DAT1), R5804.2, U5801.5 (D2-)
- net SD_D2: now also R5805.1
- net SD_D2_C: now also J5801.1 (DAT2), R5805.2, U5802.1 (D1+)
- net SD_D3: now also R5806.1
- net SD_D3_C: now also J5801.2 (CD/DAT3), R5806.2, U5802.2 (D1-)
- net SD_DET_C: now also J5801.A (DET_A), R5807.2
- net SD_DET_N: now also R5807.1
- net SD_VDD: now also C5801.1, C5802.1, J5801.4 (VDD), R5808.2, TP5802.1
- net vcc3v3_sd: now also R5808.1, TP5801.1

Commit message: Board: capture blk.debug
Debug UART2 (1.8 V) and I2S/DSD pads with ground pads, reset, PMIC and
power-key pads (PCB-T-09), a pad on every spare SoC GPIO whose pinout v1
row names one (the DEBUG bus, on the SoC's right edge), and a rail pad
for each power-tree rail no other sheet probes (PCB-T-02). Each DAC
sheet carries a pad on its MCLK. The spares pinout v1 leaves without a
pad now carry no-connect flags. On the root, facing sheet pins are
joined directly only where the route meets no other symbol.

Co-Authored-By: Claude Opus 5.5 <noreply@anthropic.com>
Claude-Session: https://claude.ai/code/session_01Ei262h3TpgY9vyfNLMi5Mn
Parts:
- removed C5801: 10 µF, Capacitor_SMD:C_0603_1608Metric, symbol Device:C
- removed C5802: 100 nF, Capacitor_SMD:C_0402_1005Metric, symbol Device:C
- removed J5801: DM3AT-SF-PEJM5, Hirose:Hirose_DM3AT-SF-PEJM5_microSD_PushPush_Top, symbol Hirose:DM3AT-SF-PEJM5
- removed R5801, R5802, R5803, R5804, R5805, R5806: 22 Ω, Resistor_SMD:R_0402_1005Metric, symbol Device:R
- removed R5807: 100 Ω, Resistor_SMD:R_0402_1005Metric, symbol Device:R
- removed R5808: 100 mΩ, Resistor_SMD:R_0603_1608Metric, symbol Device:R
- removed TP5801: vcc3v3_sd, TestPoint:TestPoint_Pad_D1.0mm, symbol Connector:TestPoint
- removed TP5802: SD_VDD, TestPoint:TestPoint_Pad_D1.0mm, symbol Connector:TestPoint
- removed U5801, U5802: TPD4E05U06DQAR, Texas_Instruments:Texas_DQA0010A_USON-10_1x2.5mm_P0.5mm, symbol Texas_Instruments:TPD4E05U06DQAR
- added C5901: 10 µF, Capacitor_SMD:C_0603_1608Metric, symbol Device:C
- added C5902: 100 nF, Capacitor_SMD:C_0402_1005Metric, symbol Device:C
- added J5901: DM3AT-SF-PEJM5, Hirose:Hirose_DM3AT-SF-PEJM5_microSD_PushPush_Top, symbol Hirose:DM3AT-SF-PEJM5
- added R5901, R5902, R5903, R5904, R5905, R5906: 22 Ω, Resistor_SMD:R_0402_1005Metric, symbol Device:R
- added R5907: 100 Ω, Resistor_SMD:R_0402_1005Metric, symbol Device:R
- added R5908: 100 mΩ, Resistor_SMD:R_0603_1608Metric, symbol Device:R
- added TP5901: vcc3v3_sd, TestPoint:TestPoint_Pad_D1.0mm, symbol Connector:TestPoint
- added TP5902: SD_VDD, TestPoint:TestPoint_Pad_D1.0mm, symbol Connector:TestPoint
- added U5901, U5902: TPD4E05U06DQAR, Texas_Instruments:Texas_DQA0010A_USON-10_1x2.5mm_P0.5mm, symbol Texas_Instruments:TPD4E05U06DQAR
Connections:
- net GND: now also C5901.2, C5902.2, J5901.6 (VSS), J5901.B (DET_B), J5901.S1 (SHIELD), U5901.3 (GND), U5901.8 (GND), U5902.3 (GND), U5902.8 (GND)
- net SD_CLK: now also R5901.1
- net SD_CLK_C: now also J5901.5 (CLK), R5901.2, U5901.1 (D1+)
- net SD_CMD: now also R5902.1
- net SD_CMD_C: now also J5901.3 (CMD), R5902.2, U5901.2 (D1-)
- net SD_D0: now also R5903.1
- net SD_D0_C: now also J5901.7 (DAT0), R5903.2, U5901.4 (D2+)
- net SD_D1: now also R5904.1
- net SD_D1_C: now also J5901.8 (DAT1), R5904.2, U5901.5 (D2-)
- net SD_D2: now also R5905.1
- net SD_D2_C: now also J5901.1 (DAT2), R5905.2, U5902.1 (D1+)
- net SD_D3: now also R5906.1
- net SD_D3_C: now also J5901.2 (CD/DAT3), R5906.2, U5902.2 (D1-)
- net SD_DET_C: now also J5901.A (DET_A), R5907.2
- net SD_DET_N: now also R5907.1
- net SD_VDD: now also C5901.1, C5902.1, J5901.4 (VDD), R5908.2, TP5902.1
- net vcc3v3_sd: now also R5908.1, TP5901.1

Commit message: Board: capture blk.cover-detect
COVER_DET_N on GPIO0_A6 (AJ38, PMUIO1, wake-capable), recorded in
pinout v1 (closes feature blocks G22): board-edge input and ground pads
for the case's actuator, 100 kΩ to vcc3v3_pmu, TPD1E10B06 at the pad
(BOM v1 line 143, PCB-L-10). The line rides the KEYS bus with the
buttons.

Co-Authored-By: Claude Opus 5.5 <noreply@anthropic.com>
Claude-Session: https://claude.ai/code/session_01Ei262h3TpgY9vyfNLMi5Mn
Parts:
- removed C5901: 10 µF, Capacitor_SMD:C_0603_1608Metric, symbol Device:C
- removed C5902: 100 nF, Capacitor_SMD:C_0402_1005Metric, symbol Device:C
- removed J5901: DM3AT-SF-PEJM5, Hirose:Hirose_DM3AT-SF-PEJM5_microSD_PushPush_Top, symbol Hirose:DM3AT-SF-PEJM5
- removed R5901, R5902, R5903, R5904, R5905, R5906: 22 Ω, Resistor_SMD:R_0402_1005Metric, symbol Device:R
- removed R5907: 100 Ω, Resistor_SMD:R_0402_1005Metric, symbol Device:R
- removed R5908: 100 mΩ, Resistor_SMD:R_0603_1608Metric, symbol Device:R
- removed TP5901: vcc3v3_sd, TestPoint:TestPoint_Pad_D1.0mm, symbol Connector:TestPoint
- removed TP5902: SD_VDD, TestPoint:TestPoint_Pad_D1.0mm, symbol Connector:TestPoint
- removed U5901, U5902: TPD4E05U06DQAR, Texas_Instruments:Texas_DQA0010A_USON-10_1x2.5mm_P0.5mm, symbol Texas_Instruments:TPD4E05U06DQAR
- added C6001: 10 µF, Capacitor_SMD:C_0603_1608Metric, symbol Device:C
- added C6002: 100 nF, Capacitor_SMD:C_0402_1005Metric, symbol Device:C
- added J6001: DM3AT-SF-PEJM5, Hirose:Hirose_DM3AT-SF-PEJM5_microSD_PushPush_Top, symbol Hirose:DM3AT-SF-PEJM5
- added R6001, R6002, R6003, R6004, R6005, R6006: 22 Ω, Resistor_SMD:R_0402_1005Metric, symbol Device:R
- added R6007: 100 Ω, Resistor_SMD:R_0402_1005Metric, symbol Device:R
- added R6008: 100 mΩ, Resistor_SMD:R_0603_1608Metric, symbol Device:R
- added TP6001: vcc3v3_sd, TestPoint:TestPoint_Pad_D1.0mm, symbol Connector:TestPoint
- added TP6002: SD_VDD, TestPoint:TestPoint_Pad_D1.0mm, symbol Connector:TestPoint
- added U6001, U6002: TPD4E05U06DQAR, Texas_Instruments:Texas_DQA0010A_USON-10_1x2.5mm_P0.5mm, symbol Texas_Instruments:TPD4E05U06DQAR
Connections:
- net GND: now also C6001.2, C6002.2, J6001.6 (VSS), J6001.B (DET_B), J6001.S1 (SHIELD), U6001.3 (GND), U6001.8 (GND), U6002.3 (GND), U6002.8 (GND)
- net SD_CLK: now also R6001.1
- net SD_CLK_C: now also J6001.5 (CLK), R6001.2, U6001.1 (D1+)
- net SD_CMD: now also R6002.1
- net SD_CMD_C: now also J6001.3 (CMD), R6002.2, U6001.2 (D1-)
- net SD_D0: now also R6003.1
- net SD_D0_C: now also J6001.7 (DAT0), R6003.2, U6001.4 (D2+)
- net SD_D1: now also R6004.1
- net SD_D1_C: now also J6001.8 (DAT1), R6004.2, U6001.5 (D2-)
- net SD_D2: now also R6005.1
- net SD_D2_C: now also J6001.1 (DAT2), R6005.2, U6002.1 (D1+)
- net SD_D3: now also R6006.1
- net SD_D3_C: now also J6001.2 (CD/DAT3), R6006.2, U6002.2 (D1-)
- net SD_DET_C: now also J6001.A (DET_A), R6007.2
- net SD_DET_N: now also R6007.1
- net SD_VDD: now also C6001.1, C6002.1, J6001.4 (VDD), R6008.2, TP6002.1
- net vcc3v3_sd: now also R6008.1, TP6001.1

Commit message: Board: capture blk.mic-ambient and links #34, #35
IM73D122 on PDM CLK1 and SDI1 (BOM v1 line 34, pinout v1 AK2 and 1P2),
LR to ground, 22 Ω clock series, VDD from MIC_1V8 through link #35.
Link #34 on blk.mic-main makes the faceplate branch the rail MIC_1V8_FP
for contact 40 (power tree §4.12, G10). kicad-lib moves to e46bda4 for
the IM73D122, TPS3808G01, SN74LVC1G58 and BAT54 parts.

Co-Authored-By: Claude Opus 5.5 <noreply@anthropic.com>
Claude-Session: https://claude.ai/code/session_01Ei262h3TpgY9vyfNLMi5Mn
Parts:
- removed C6001: 10 µF, Capacitor_SMD:C_0603_1608Metric, symbol Device:C
- removed C6002: 100 nF, Capacitor_SMD:C_0402_1005Metric, symbol Device:C
- removed J6001: DM3AT-SF-PEJM5, Hirose:Hirose_DM3AT-SF-PEJM5_microSD_PushPush_Top, symbol Hirose:DM3AT-SF-PEJM5
- removed R6001, R6002, R6003, R6004, R6005, R6006: 22 Ω, Resistor_SMD:R_0402_1005Metric, symbol Device:R
- removed R6007: 100 Ω, Resistor_SMD:R_0402_1005Metric, symbol Device:R
- removed R6008: 100 mΩ, Resistor_SMD:R_0603_1608Metric, symbol Device:R
- removed TP6001: vcc3v3_sd, TestPoint:TestPoint_Pad_D1.0mm, symbol Connector:TestPoint
- removed TP6002: SD_VDD, TestPoint:TestPoint_Pad_D1.0mm, symbol Connector:TestPoint
- removed U6001, U6002: TPD4E05U06DQAR, Texas_Instruments:Texas_DQA0010A_USON-10_1x2.5mm_P0.5mm, symbol Texas_Instruments:TPD4E05U06DQAR
- added C6101: 10 µF, Capacitor_SMD:C_0603_1608Metric, symbol Device:C
- added C6102: 100 nF, Capacitor_SMD:C_0402_1005Metric, symbol Device:C
- added J6101: DM3AT-SF-PEJM5, Hirose:Hirose_DM3AT-SF-PEJM5_microSD_PushPush_Top, symbol Hirose:DM3AT-SF-PEJM5
- added R6101, R6102, R6103, R6104, R6105, R6106: 22 Ω, Resistor_SMD:R_0402_1005Metric, symbol Device:R
- added R6107: 100 Ω, Resistor_SMD:R_0402_1005Metric, symbol Device:R
- added R6108: 100 mΩ, Resistor_SMD:R_0603_1608Metric, symbol Device:R
- added TP6101: vcc3v3_sd, TestPoint:TestPoint_Pad_D1.0mm, symbol Connector:TestPoint
- added TP6102: SD_VDD, TestPoint:TestPoint_Pad_D1.0mm, symbol Connector:TestPoint
- added U6101, U6102: TPD4E05U06DQAR, Texas_Instruments:Texas_DQA0010A_USON-10_1x2.5mm_P0.5mm, symbol Texas_Instruments:TPD4E05U06DQAR
Connections:
- net GND: now also C6101.2, C6102.2, J6101.6 (VSS), J6101.B (DET_B), J6101.S1 (SHIELD), U6101.3 (GND), U6101.8 (GND), U6102.3 (GND), U6102.8 (GND)
- net SD_CLK: now also R6101.1
- net SD_CLK_C: now also J6101.5 (CLK), R6101.2, U6101.1 (D1+)
- net SD_CMD: now also R6102.1
- net SD_CMD_C: now also J6101.3 (CMD), R6102.2, U6101.2 (D1-)
- net SD_D0: now also R6103.1
- net SD_D0_C: now also J6101.7 (DAT0), R6103.2, U6101.4 (D2+)
- net SD_D1: now also R6104.1
- net SD_D1_C: now also J6101.8 (DAT1), R6104.2, U6101.5 (D2-)
- net SD_D2: now also R6105.1
- net SD_D2_C: now also J6101.1 (DAT2), R6105.2, U6102.1 (D1+)
- net SD_D3: now also R6106.1
- net SD_D3_C: now also J6101.2 (CD/DAT3), R6106.2, U6102.2 (D1-)
- net SD_DET_C: now also J6101.A (DET_A), R6107.2
- net SD_DET_N: now also R6107.1
- net SD_VDD: now also C6101.1, C6102.1, J6101.4 (VDD), R6108.2, TP6102.1
- net vcc3v3_sd: now also R6108.1, TP6101.1

Commit message: Board: capture blk.maskrom
Power + Vol- at a cold power-on pull eMMC D0 low inside the TPS3808G01
boot window (BOM v1 lines 35, 78, 97, 98; sim/maskrom): SENSE 280k/100k,
CT 390 nF, WINDOW_N with its pad, SN74LVC1G57 and SN74LVC1G58 on
vcca1v8_pmu, BAT54 from PWRON_N, DMG1012T through 1 kΩ to EMMC_D0.
Every block in use now has its sheet; the README states the remaining
single-pin nets.

Co-Authored-By: Claude Opus 5.5 <noreply@anthropic.com>
Claude-Session: https://claude.ai/code/session_01Ei262h3TpgY9vyfNLMi5Mn
Parts:
- removed C6101: 10 µF, Capacitor_SMD:C_0603_1608Metric, symbol Device:C
- removed C6102: 100 nF, Capacitor_SMD:C_0402_1005Metric, symbol Device:C
- removed J6101: DM3AT-SF-PEJM5, Hirose:Hirose_DM3AT-SF-PEJM5_microSD_PushPush_Top, symbol Hirose:DM3AT-SF-PEJM5
- removed R6101, R6102, R6103, R6104, R6105, R6106: 22 Ω, Resistor_SMD:R_0402_1005Metric, symbol Device:R
- removed R6107: 100 Ω, Resistor_SMD:R_0402_1005Metric, symbol Device:R
- removed R6108: 100 mΩ, Resistor_SMD:R_0603_1608Metric, symbol Device:R
- removed TP6101: vcc3v3_sd, TestPoint:TestPoint_Pad_D1.0mm, symbol Connector:TestPoint
- removed TP6102: SD_VDD, TestPoint:TestPoint_Pad_D1.0mm, symbol Connector:TestPoint
- removed U6101, U6102: TPD4E05U06DQAR, Texas_Instruments:Texas_DQA0010A_USON-10_1x2.5mm_P0.5mm, symbol Texas_Instruments:TPD4E05U06DQAR
- added C6201: 10 µF, Capacitor_SMD:C_0603_1608Metric, symbol Device:C
- added C6202: 100 nF, Capacitor_SMD:C_0402_1005Metric, symbol Device:C
- added J6201: DM3AT-SF-PEJM5, Hirose:Hirose_DM3AT-SF-PEJM5_microSD_PushPush_Top, symbol Hirose:DM3AT-SF-PEJM5
- added R6201, R6202, R6203, R6204, R6205, R6206: 22 Ω, Resistor_SMD:R_0402_1005Metric, symbol Device:R
- added R6207: 100 Ω, Resistor_SMD:R_0402_1005Metric, symbol Device:R
- added R6208: 100 mΩ, Resistor_SMD:R_0603_1608Metric, symbol Device:R
- added TP6201: vcc3v3_sd, TestPoint:TestPoint_Pad_D1.0mm, symbol Connector:TestPoint
- added TP6202: SD_VDD, TestPoint:TestPoint_Pad_D1.0mm, symbol Connector:TestPoint
- added U6201, U6202: TPD4E05U06DQAR, Texas_Instruments:Texas_DQA0010A_USON-10_1x2.5mm_P0.5mm, symbol Texas_Instruments:TPD4E05U06DQAR
Connections:
- net GND: now also C6201.2, C6202.2, J6201.6 (VSS), J6201.B (DET_B), J6201.S1 (SHIELD), U6201.3 (GND), U6201.8 (GND), U6202.3 (GND), U6202.8 (GND)
- net SD_CLK: now also R6201.1
- net SD_CLK_C: now also J6201.5 (CLK), R6201.2, U6201.1 (D1+)
- net SD_CMD: now also R6202.1
- net SD_CMD_C: now also J6201.3 (CMD), R6202.2, U6201.2 (D1-)
- net SD_D0: now also R6203.1
- net SD_D0_C: now also J6201.7 (DAT0), R6203.2, U6201.4 (D2+)
- net SD_D1: now also R6204.1
- net SD_D1_C: now also J6201.8 (DAT1), R6204.2, U6201.5 (D2-)
- net SD_D2: now also R6205.1
- net SD_D2_C: now also J6201.1 (DAT2), R6205.2, U6202.1 (D1+)
- net SD_D3: now also R6206.1
- net SD_D3_C: now also J6201.2 (CD/DAT3), R6206.2, U6202.2 (D1-)
- net SD_DET_C: now also J6201.A (DET_A), R6207.2
- net SD_DET_N: now also R6207.1
- net SD_VDD: now also C6201.1, C6202.1, J6201.4 (VDD), R6208.2, TP6202.1
- net vcc3v3_sd: now also R6208.1, TP6201.1

Commit message: Compaction: lower inductors, 0201 decoupling, 0.8 mm signal test pads
A matrix tool (hardware/studies/compaction) checks each candidate against
the design's stresses: same inductance, design peak <= 70 % and the
converter's maximum limit <= 100 % of Isat (30 % drop), height zones,
ratings at least twice the rail, PCB-D-06; sourcing outcome per part.

Applied (placement v1 decision 12, BOM v1.15):
- L601, L4401: XGL4015-102MEC (1.5 mm) for XAL/XGL4020-102MEC (2.1 mm);
- L1001, L5101: XGL4015-471MEC (1.5 mm) for Wurth 744373240047, on the
  stock XxL4020 land (the Wurth land was never drawn);
- L1201 is 1.2 mm (XGL4012, per-MPN heights): it moves next to the SoC;
- 58 x 100 nF decoupling on rails <= 3.3 V in core/IO/radio: 0201;
- 51 test pads on signal nets: 0.8 mm (PCB-D-06 v0.16, JLCPCB guide).
Kept: L901, L2802 (XGL4015 at 103 % of Isat at the limit); no thinner
0805/1206 capacitor passes (obsolete, NRND or unlisted).

Board need 113 % -> 111 % (core band 227 -> 203 %, power band 258 ->
233 %, radio band 19 -> 0 %); only C904 still relies on PCB-Z-04.
ERC 0 errors, craft Q1 met, DRC 0 errors (605 warnings), pcb and study
tests pass, rules test board PASS.

Co-Authored-By: Claude Opus 5.5 <noreply@anthropic.com>
Claude-Session: https://claude.ai/code/session_01Ei262h3TpgY9vyfNLMi5Mn
Parts:
- C6202: footprint Capacitor_SMD:C_0402_1005Metric -> Capacitor_SMD:C_0201_0603Metric; MPN GRM155R71C104KA88D -> GRM033R61A104KE15D
Changed lines of the file:
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@@
   (property "Reference" "C6202" (at 104.14 50.8 0) (effects (font (size 1.27 1.27)) (justify left)))
   (property "Value" "100 nF" (at 104.14 53.34 0) (effects (font (size 1.27 1.27)) (justify left)))
-  (property "Footprint" "Capacitor_SMD:C_0402_1005Metric" (at 101.6 52.07 0) (effects (font (size 1.27 1.27))) (hide yes))
-  (property "Datasheet" "https://www.murata.com/en-us/products/productdetail?partno=GRM155R71C104KA88D" (at 101.6 52.07 0) (effects (font (size 1.27 1.27))) (hide yes))
-  (property "Description" "Capacitor, 100 nF, 16 V, X7R, 0402" (at 101.6 52.07 0) (effects (font (size 1.27 1.27))) (hide yes))
+  (property "Footprint" "Capacitor_SMD:C_0201_0603Metric" (at 101.6 52.07 0) (effects (font (size 1.27 1.27))) (hide yes))
+  (property "Datasheet" "https://www.murata.com/en-us/products/productdetail?partno=GRM033R61A104KE15D" (at 101.6 52.07 0) (effects (font (size 1.27 1.27))) (hide yes))
+  (property "Description" "Capacitor, 100 nF, 10 V, X5R, 0201" (at 101.6 52.07 0) (effects (font (size 1.27 1.27))) (hide yes))
   (property "Manufacturer" "Murata" (at 101.6 52.07 0) (effects (font (size 1.27 1.27))) (hide yes))
-  (property "MPN" "GRM155R71C104KA88D" (at 101.6 52.07 0) (effects (font (size 1.27 1.27))) (hide yes))
+  (property "MPN" "GRM033R61A104KE15D" (at 101.6 52.07 0) (effects (font (size 1.27 1.27))) (hide yes))
   (property "Block" "blk.microsd" (at 101.6 52.07 0) (effects (font (size 1.27 1.27))) (hide yes))
   (pin "1")
