File: board/hardware/t1-main-board/microsd.kicad_sch (KiCad schematic)
At the start: 15 parts, among them J6201 DM3AT-SF-PEJM5, U6201 TPD4E05U06DQAR, U6202 TPD4E05U06DQAR

Commit message: Board on libs v0.2.0: lower-case kebab vendor keys (HL-13)
The libs submodule moves to v0.2.0 (5f24483). Every library nickname in
the generator, the placement tool and the floorplan study follows the
key table (Texas_Instruments -> texas-instruments, OpenDAP_Device ->
opendap-generic, Rockchip and Rockchip_PMIC -> rockchip, ...); the
library tables are written from the files. Schematic and board
regenerated.

Checks: ERC 0 errors (warnings unchanged); DRC 0 errors, 605 warnings,
the same counts by type, schematic parity 0; every placement identical;
craft Q1 met; pcb tests pass; STEP export resolves every libs 3D model
(the 27 parts without a model are KiCad stock lands that have none).

Co-Authored-By: Claude Opus 5.5 <noreply@anthropic.com>
Claude-Session: https://claude.ai/code/session_01Ei262h3TpgY9vyfNLMi5Mn
Parts:
- J6201: footprint Hirose:Hirose_DM3AT-SF-PEJM5_microSD_PushPush_Top -> hirose:Hirose_DM3AT-SF-PEJM5_microSD_PushPush_Top; symbol Hirose:DM3AT-SF-PEJM5 -> hirose:DM3AT-SF-PEJM5
- U6201, U6202: footprint Texas_Instruments:Texas_DQA0010A_USON-10_1x2.5mm_P0.5mm -> texas-instruments:Texas_DQA0010A_USON-10_1x2.5mm_P0.5mm; symbol Texas_Instruments:TPD4E05U06DQAR -> texas-instruments:TPD4E05U06DQAR
Changed lines of the file:
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@@
 (paper "A4")
 (title_block (title "microSD socket") (date "2026-10-25") (rev "A") (company "The OpenDAP Project") (comment 1 "blk.microsd") (comment 2 "DM3AT socket, SDMMC0 series resistors, card detect and ESD"))
-(symbol (lib_id "Hirose:DM3AT-SF-PEJM5") (at 53.34 73.66 0) (unit 1) (body_style 1) (exclude_from_sim no) (in_bom yes) (on_board yes) (dnp no)
+(symbol (lib_id "hirose:DM3AT-SF-PEJM5") (at 53.34 73.66 0) (unit 1) (body_style 1) (exclude_from_sim no) (in_bom yes) (on_board yes) (dnp no)
   (property "Reference" "J6201" (at 54.61 49.53 0) (effects (font (size 1.27 1.27)) (justify left)))
   (property "Value" "DM3AT-SF-PEJM5" (at 54.61 46.99 0) (effects (font (size 1.27 1.27)) (justify left)))
-  (property "Footprint" "Hirose:Hirose_DM3AT-SF-PEJM5_microSD_PushPush_Top" (at 53.34 73.66 0) (effects (font (size 1.27 1.27))) (hide yes))
+  (property "Footprint" "hirose:Hirose_DM3AT-SF-PEJM5_microSD_PushPush_Top" (at 53.34 73.66 0) (effects (font (size 1.27 1.27))) (hide yes))
   (property "Datasheet" "https://www.hirose.com/en/product/series/DM3" (at 53.34 73.66 0) (effects (font (size 1.27 1.27))) (hide yes))
   (property "Description" "microSD card connector, push-push, top board mounting, SMT, normally-open card-detection switch" (at 53.34 73.66 0) (effects (font (size 1.27 1.27))) (hide yes))
@@
 (rectangle (start 120.65 35.56) (end 187.96 114.3) (stroke (width 0) (type dash)) (fill (type none)))
 (text "Series resistors (HDG p. 52)" (exclude_from_sim no) (at 121.92 34.29 0) (effects (font (size 2.54 2.54)) (justify left bottom)))
-(symbol (lib_id "Texas_Instruments:TPD4E05U06DQAR") (at 218.44 59.69 0) (unit 1) (body_style 1) (exclude_from_sim no) (in_bom yes) (on_board yes) (dnp no)
+(symbol (lib_id "texas-instruments:TPD4E05U06DQAR") (at 218.44 59.69 0) (unit 1) (body_style 1) (exclude_from_sim no) (in_bom yes) (on_board yes) (dnp no)
   (property "Reference" "U6201" (at 212.09 43.18 0) (effects (font (size 1.27 1.27)) (justify left)))
   (property "Value" "TPD4E05U06DQAR" (at 212.09 40.64 0) (effects (font (size 1.27 1.27)) (justify left)))
-  (property "Footprint" "Texas_Instruments:Texas_DQA0010A_USON-10_1x2.5mm_P0.5mm" (at 218.44 59.69 0) (effects (font (size 1.27 1.27))) (hide yes))
+  (property "Footprint" "texas-instruments:Texas_DQA0010A_USON-10_1x2.5mm_P0.5mm" (at 218.44 59.69 0) (effects (font (size 1.27 1.27))) (hide yes))
   (property "Datasheet" "https://www.ti.com/lit/ds/symlink/tpd4e05u06.pdf" (at 218.44 59.69 0) (effects (font (size 1.27 1.27))) (hide yes))
   (property "Description" "4-channel ESD protection, 0.5 pF, 5.5 V stand-off, IEC 61000-4-2 level 4, flow-through routing, USON-10 (DQA0010A) 1 x 2.5 mm" (at 218.44 59.69 0) (effects (font (size 1.27 1.27))) (hide yes))
@@
 (no_connect (at 228.6 59.69))
 (no_connect (at 228.6 62.23))
-(symbol (lib_id "Texas_Instruments:TPD4E05U06DQAR") (at 260.35 59.69 0) (unit 1) (body_style 1) (exclude_from_sim no) (in_bom yes) (on_board yes) (dnp no)
+(symbol (lib_id "texas-instruments:TPD4E05U06DQAR") (at 260.35 59.69 0) (unit 1) (body_style 1) (exclude_from_sim no) (in_bom yes) (on_board yes) (dnp no)
   (property "Reference" "U6202" (at 254 43.18 0) (effects (font (size 1.27 1.27)) (justify left)))
   (property "Value" "TPD4E05U06DQAR" (at 254 40.64 0) (effects (font (size 1.27 1.27)) (justify left)))
-  (property "Footprint" "Texas_Instruments:Texas_DQA0010A_USON-10_1x2.5mm_P0.5mm" (at 260.35 59.69 0) (effects (font (size 1.27 1.27))) (hide yes))
+  (property "Footprint" "texas-instruments:Texas_DQA0010A_USON-10_1x2.5mm_P0.5mm" (at 260.35 59.69 0) (effects (font (size 1.27 1.27))) (hide yes))
   (property "Datasheet" "https://www.ti.com/lit/ds/symlink/tpd4e05u06.pdf" (at 260.35 59.69 0) (effects (font (size 1.27 1.27))) (hide yes))
   (property "Description" "4-channel ESD protection, 0.5 pF, 5.5 V stand-off, IEC 61000-4-2 level 4, flow-through routing, USON-10 (DQA0010A) 1 x 2.5 mm" (at 260.35 59.69 0) (effects (font (size 1.27 1.27))) (hide yes))
