File: board/hardware/t1-main-board/nfc-tag.kicad_sch (KiCad schematic)
At the start: 7 parts, among them U5301 NT3H2111W0FHKH

Commit message: Board: capture blk.current-monitors
Five INA236 on I2C1 (0x40-0x43, 0x48) with their shunts, per power tree
§4.12 and BOM v1 lines 54 and 136. The measured branches are rails of
their own (VSYS_SRC, VSYS_LV_AUDIO, VSYS_AUDIO, VSYS_LV_BL, VSYS_P5V1),
fed through the shunts on this sheet; the charger, audio, backlight and
5.1 V sheets take them. The root's layout may leave a stack level empty,
so the block sits under the notes; IC bboxes hold turned rail values;
passive rows hold a bottom rail's text.

Co-Authored-By: Claude Opus 5.5 <noreply@anthropic.com>
Claude-Session: https://claude.ai/code/session_01Ei262h3TpgY9vyfNLMi5Mn
Parts:
- removed C5301: 100 nF, Capacitor_SMD:C_0402_1005Metric, symbol Device:C
- removed R5301: 10 Ω, Resistor_SMD:R_0603_1608Metric, symbol Device:R
- removed TP5301: vcca1v8_pmu, TestPoint:TestPoint_Pad_D1.0mm, symbol Connector:TestPoint
- removed TP5302: NFC_TAG_VCC, TestPoint:TestPoint_Pad_D1.0mm, symbol Connector:TestPoint
- removed TP5303: NFC_TAG_LA, TestPoint:TestPoint_Pad_D1.0mm, symbol Connector:TestPoint
- removed TP5304: NFC_TAG_LB, TestPoint:TestPoint_Pad_D1.0mm, symbol Connector:TestPoint
- removed U5301: NT3H2111W0FHKH, NXP:NXP_SOT902-3_XQFN-8_1.6x1.6mm_P0.5mm, symbol NXP:NT3H2111W0FHKH
- added C5401: 100 nF, Capacitor_SMD:C_0402_1005Metric, symbol Device:C
- added R5401: 10 Ω, Resistor_SMD:R_0603_1608Metric, symbol Device:R
- added TP5401: vcca1v8_pmu, TestPoint:TestPoint_Pad_D1.0mm, symbol Connector:TestPoint
- added TP5402: NFC_TAG_VCC, TestPoint:TestPoint_Pad_D1.0mm, symbol Connector:TestPoint
- added TP5403: NFC_TAG_LA, TestPoint:TestPoint_Pad_D1.0mm, symbol Connector:TestPoint
- added TP5404: NFC_TAG_LB, TestPoint:TestPoint_Pad_D1.0mm, symbol Connector:TestPoint
- added U5401: NT3H2111W0FHKH, NXP:NXP_SOT902-3_XQFN-8_1.6x1.6mm_P0.5mm, symbol NXP:NT3H2111W0FHKH
Connections:
- net GND: now also C5401.2, U5401.2 (VSS)
- net I2C2_SCL: now also U5401.3 (SCL)
- net I2C2_SDA: now also U5401.5 (SDA)
- net NFC_FD_N: now also U5401.4 (FD)
- net NFC_TAG_LA: now also TP5403.1, U5401.1 (LA)
- net NFC_TAG_LB: now also TP5404.1, U5401.8 (LB)
- net NFC_TAG_VCC: now also C5401.1, R5401.2, TP5402.1, U5401.6 (VCC)
- net vcca1v8_pmu: now also R5401.1, TP5401.1
Changed lines of the file:
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@@
 (title_block (title "NFC tag") (date "2026-10-25") (rev "A") (company "The OpenDAP Project") (comment 1 "blk.nfc-tag") (comment 2 "NTAG I2C plus on I2C2 at 0x55, field detect and the loop antenna contacts"))
 (symbol (lib_id "NXP:NT3H2111W0FHKH") (at 50.8 72.39 0) (unit 1) (body_style 1) (exclude_from_sim no) (in_bom yes) (on_board yes) (dnp no)
-  (property "Reference" "U5301" (at 52.07 54.61 0) (effects (font (size 1.27 1.27)) (justify left)))
+  (property "Reference" "U5401" (at 52.07 54.61 0) (effects (font (size 1.27 1.27)) (justify left)))
   (property "Value" "NT3H2111W0FHKH" (at 52.07 52.07 0) (effects (font (size 1.27 1.27)) (justify left)))
   (property "Footprint" "NXP:NXP_SOT902-3_XQFN-8_1.6x1.6mm_P0.5mm" (at 50.8 72.39 0) (effects (font (size 1.27 1.27))) (hide yes))
@@
   (pin "6")
   (pin "2")
-  (instances (project "t1-main-board" (path "/7746052e-d7f9-59ad-ba73-bd2b74439529/338b6b86-006f-5bfa-ad71-6e8aca3fbcdb" (reference "U5301") (unit 1))))
+  (instances (project "t1-main-board" (path "/7746052e-d7f9-59ad-ba73-bd2b74439529/338b6b86-006f-5bfa-ad71-6e8aca3fbcdb" (reference "U5401") (unit 1))))
 )
 (wire (pts (xy 40.64 67.31) (xy 38.1 67.31)) (stroke (width 0) (type default)))
@@
 )
 (symbol (lib_id "Device:C") (at 78.74 58.42 0) (unit 1) (body_style 1) (exclude_from_sim no) (in_bom yes) (on_board yes) (dnp no)
-  (property "Reference" "C5301" (at 81.28 57.15 0) (effects (font (size 1.27 1.27)) (justify left)))
+  (property "Reference" "C5401" (at 81.28 57.15 0) (effects (font (size 1.27 1.27)) (justify left)))
   (property "Value" "100 nF" (at 81.28 59.69 0) (effects (font (size 1.27 1.27)) (justify left)))
   (property "Footprint" "Capacitor_SMD:C_0402_1005Metric" (at 78.74 58.42 0) (effects (font (size 1.27 1.27))) (hide yes))
@@
   (pin "1")
   (pin "2")
-  (instances (project "t1-main-board" (path "/7746052e-d7f9-59ad-ba73-bd2b74439529/338b6b86-006f-5bfa-ad71-6e8aca3fbcdb" (reference "C5301") (unit 1))))
+  (instances (project "t1-main-board" (path "/7746052e-d7f9-59ad-ba73-bd2b74439529/338b6b86-006f-5bfa-ad71-6e8aca3fbcdb" (reference "C5401") (unit 1))))
 )
 (wire (pts (xy 78.74 54.61) (xy 78.74 52.07)) (stroke (width 0) (type default)))
@@
 (text "NT3H2111 NTAG I2C plus at I2C2 0x55 (BOM v1 line 125)" (exclude_from_sim no) (at 24.13 34.29 0) (effects (font (size 2.54 2.54)) (justify left bottom)))
 (symbol (lib_id "Device:R") (at 191.77 50.8 90) (unit 1) (body_style 1) (exclude_from_sim no) (in_bom yes) (on_board yes) (dnp no)
-  (property "Reference" "R5301" (at 189.23 46.99 90) (effects (font (size 1.27 1.27))))
+  (property "Reference" "R5401" (at 189.23 46.99 90) (effects (font (size 1.27 1.27))))
   (property "Value" "10 Ω" (at 189.23 53.34 90) (effects (font (size 1.27 1.27))))
   (property "Spec" "0603" (at 189.23 55.88 90) (effects (font (size 1.27 1.27))))
@@
   (pin "1")
   (pin "2")
-  (instances (project "t1-main-board" (path "/7746052e-d7f9-59ad-ba73-bd2b74439529/338b6b86-006f-5bfa-ad71-6e8aca3fbcdb" (reference "R5301") (unit 1) (variant (name "production") (field (name "Value") (value "0 Ω")) (field (name "MPN") (value "RC0603JR-070RL")) (field (name "Manufacturer") (value "YAGEO"))))))
+  (instances (project "t1-main-board" (path "/7746052e-d7f9-59ad-ba73-bd2b74439529/338b6b86-006f-5bfa-ad71-6e8aca3fbcdb" (reference "R5401") (unit 1) (variant (name "production") (field (name "Value") (value "0 Ω")) (field (name "MPN") (value "RC0603JR-070RL")) (field (name "Manufacturer") (value "YAGEO"))))))
 )
 (rectangle (start 168.91 38.1) (end 214.63 58.42) (stroke (width 0) (type dash)) (fill (type none)))
@@
 (wire (pts (xy 185.42 50.8) (xy 185.42 48.26)) (stroke (width 0) (type default)))
 (symbol (lib_id "Connector:TestPoint") (at 185.42 48.26 0) (unit 1) (body_style 1) (exclude_from_sim no) (in_bom no) (on_board yes) (dnp no)
-  (property "Reference" "TP5301" (at 184.15 43.18 0) (effects (font (size 1.27 1.27)) (justify right)))
+  (property "Reference" "TP5401" (at 184.15 43.18 0) (effects (font (size 1.27 1.27)) (justify right)))
   (property "Value" "vcca1v8_pmu" (at 184.15 45.72 0) (effects (font (size 1.27 1.27)) (justify right)))
   (property "Footprint" "TestPoint:TestPoint_Pad_D1.0mm" (at 185.42 48.26 0) (effects (font (size 1.27 1.27))) (hide yes))
@@
   (property "Block" "blk.nfc-tag" (at 185.42 48.26 0) (effects (font (size 1.27 1.27))) (hide yes))
   (pin "1")
-  (instances (project "t1-main-board" (path "/7746052e-d7f9-59ad-ba73-bd2b74439529/338b6b86-006f-5bfa-ad71-6e8aca3fbcdb" (reference "TP5301") (unit 1))))
+  (instances (project "t1-main-board" (path "/7746052e-d7f9-59ad-ba73-bd2b74439529/338b6b86-006f-5bfa-ad71-6e8aca3fbcdb" (reference "TP5401") (unit 1))))
 )
 (symbol (lib_id "power:VCC") (at 166.37 50.8 90) (unit 1) (body_style 1) (exclude_from_sim no) (in_bom yes) (on_board yes) (dnp no)
@@
 (wire (pts (xy 198.12 50.8) (xy 198.12 48.26)) (stroke (width 0) (type default)))
 (symbol (lib_id "Connector:TestPoint") (at 198.12 48.26 0) (unit 1) (body_style 1) (exclude_from_sim no) (in_bom no) (on_board yes) (dnp no)
-  (property "Reference" "TP5302" (at 199.39 43.18 0) (effects (font (size 1.27 1.27)) (justify left)))
+  (property "Reference" "TP5402" (at 199.39 43.18 0) (effects (font (size 1.27 1.27)) (justify left)))
   (property "Value" "NFC_TAG_VCC" (at 199.39 45.72 0) (effects (font (size 1.27 1.27)) (justify left)))
   (property "Footprint" "TestPoint:TestPoint_Pad_D1.0mm" (at 198.12 48.26 0) (effects (font (size 1.27 1.27))) (hide yes))
@@
   (property "Block" "blk.nfc-tag" (at 198.12 48.26 0) (effects (font (size 1.27 1.27))) (hide yes))
   (pin "1")
-  (instances (project "t1-main-board" (path "/7746052e-d7f9-59ad-ba73-bd2b74439529/338b6b86-006f-5bfa-ad71-6e8aca3fbcdb" (reference "TP5302") (unit 1))))
+  (instances (project "t1-main-board" (path "/7746052e-d7f9-59ad-ba73-bd2b74439529/338b6b86-006f-5bfa-ad71-6e8aca3fbcdb" (reference "TP5402") (unit 1))))
 )
 (junction (at 222.25 50.8) (diameter 0) (color 0 0 0 0))
@@
 )
 (symbol (lib_id "Connector:TestPoint") (at 168.91 81.28 0) (unit 1) (body_style 1) (exclude_from_sim no) (in_bom no) (on_board yes) (dnp no)
-  (property "Reference" "TP5303" (at 167.64 76.2 0) (effects (font (size 1.27 1.27)) (justify right)))
+  (property "Reference" "TP5403" (at 167.64 76.2 0) (effects (font (size 1.27 1.27)) (justify right)))
   (property "Value" "NFC_TAG_LA" (at 167.64 78.74 0) (effects (font (size 1.27 1.27)) (justify right)))
   (property "Footprint" "TestPoint:TestPoint_Pad_D1.0mm" (at 168.91 81.28 0) (effects (font (size 1.27 1.27))) (hide yes))
@@
   (property "Block" "blk.nfc-tag" (at 168.91 81.28 0) (effects (font (size 1.27 1.27))) (hide yes))
   (pin "1")
-  (instances (project "t1-main-board" (path "/7746052e-d7f9-59ad-ba73-bd2b74439529/338b6b86-006f-5bfa-ad71-6e8aca3fbcdb" (reference "TP5303") (unit 1))))
+  (instances (project "t1-main-board" (path "/7746052e-d7f9-59ad-ba73-bd2b74439529/338b6b86-006f-5bfa-ad71-6e8aca3fbcdb" (reference "TP5403") (unit 1))))
 )
 (symbol (lib_id "Connector:TestPoint") (at 186.69 81.28 0) (unit 1) (body_style 1) (exclude_from_sim no) (in_bom no) (on_board yes) (dnp no)
-  (property "Reference" "TP5304" (at 185.42 76.2 0) (effects (font (size 1.27 1.27)) (justify right)))
+  (property "Reference" "TP5404" (at 185.42 76.2 0) (effects (font (size 1.27 1.27)) (justify right)))
   (property "Value" "NFC_TAG_LB" (at 185.42 78.74 0) (effects (font (size 1.27 1.27)) (justify right)))
   (property "Footprint" "TestPoint:TestPoint_Pad_D1.0mm" (at 186.69 81.28 0) (effects (font (size 1.27 1.27))) (hide yes))
@@
   (property "Block" "blk.nfc-tag" (at 186.69 81.28 0) (effects (font (size 1.27 1.27))) (hide yes))
   (pin "1")
-  (instances (project "t1-main-board" (path "/7746052e-d7f9-59ad-ba73-bd2b74439529/338b6b86-006f-5bfa-ad71-6e8aca3fbcdb" (reference "TP5304") (unit 1))))
+  (instances (project "t1-main-board" (path "/7746052e-d7f9-59ad-ba73-bd2b74439529/338b6b86-006f-5bfa-ad71-6e8aca3fbcdb" (reference "TP5404") (unit 1))))
 )
 (rectangle (start 152.4 71.12) (end 245.11 97.79) (stroke (width 0) (type dash)) (fill (type none)))

Commit message: Board: capture blk.status-led
LP5521 at 0x32 on I2C2 (BOM v1 line 105) with its charge-pump
capacitors, EN on vcca1v8_pmu, VDD from VSYS_LV through link #22;
LED_R/G/B reach the faceplate connector as the LED bus alias. The
faceplate row of the root is re-packed so five full columns sit left of
the title block.

Co-Authored-By: Claude Opus 5.5 <noreply@anthropic.com>
Claude-Session: https://claude.ai/code/session_01Ei262h3TpgY9vyfNLMi5Mn
Parts:
- removed C5401: 100 nF, Capacitor_SMD:C_0402_1005Metric, symbol Device:C
- removed R5401: 10 Ω, Resistor_SMD:R_0603_1608Metric, symbol Device:R
- removed TP5401: vcca1v8_pmu, TestPoint:TestPoint_Pad_D1.0mm, symbol Connector:TestPoint
- removed TP5402: NFC_TAG_VCC, TestPoint:TestPoint_Pad_D1.0mm, symbol Connector:TestPoint
- removed TP5403: NFC_TAG_LA, TestPoint:TestPoint_Pad_D1.0mm, symbol Connector:TestPoint
- removed TP5404: NFC_TAG_LB, TestPoint:TestPoint_Pad_D1.0mm, symbol Connector:TestPoint
- removed U5401: NT3H2111W0FHKH, NXP:NXP_SOT902-3_XQFN-8_1.6x1.6mm_P0.5mm, symbol NXP:NT3H2111W0FHKH
- added C6001: 100 nF, Capacitor_SMD:C_0402_1005Metric, symbol Device:C
- added R6001: 10 Ω, Resistor_SMD:R_0603_1608Metric, symbol Device:R
- added TP6001: vcca1v8_pmu, TestPoint:TestPoint_Pad_D1.0mm, symbol Connector:TestPoint
- added TP6002: NFC_TAG_VCC, TestPoint:TestPoint_Pad_D1.0mm, symbol Connector:TestPoint
- added TP6003: NFC_TAG_LA, TestPoint:TestPoint_Pad_D1.0mm, symbol Connector:TestPoint
- added TP6004: NFC_TAG_LB, TestPoint:TestPoint_Pad_D1.0mm, symbol Connector:TestPoint
- added U6001: NT3H2111W0FHKH, NXP:NXP_SOT902-3_XQFN-8_1.6x1.6mm_P0.5mm, symbol NXP:NT3H2111W0FHKH
Connections:
- net GND: now also C6001.2, U6001.2 (VSS)
- net I2C2_SCL: now also U6001.3 (SCL)
- net I2C2_SDA: now also U6001.5 (SDA)
- net NFC_FD_N: now also U6001.4 (FD)
- net NFC_TAG_LA: now also TP6003.1, U6001.1 (LA)
- net NFC_TAG_LB: now also TP6004.1, U6001.8 (LB)
- net NFC_TAG_VCC: now also C6001.1, R6001.2, TP6002.1, U6001.6 (VCC)
- net vcca1v8_pmu: now also R6001.1, TP6001.1
Changed lines of the file:
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@@
 (title_block (title "NFC tag") (date "2026-10-25") (rev "A") (company "The OpenDAP Project") (comment 1 "blk.nfc-tag") (comment 2 "NTAG I2C plus on I2C2 at 0x55, field detect and the loop antenna contacts"))
 (symbol (lib_id "NXP:NT3H2111W0FHKH") (at 50.8 72.39 0) (unit 1) (body_style 1) (exclude_from_sim no) (in_bom yes) (on_board yes) (dnp no)
-  (property "Reference" "U5401" (at 52.07 54.61 0) (effects (font (size 1.27 1.27)) (justify left)))
+  (property "Reference" "U6001" (at 52.07 54.61 0) (effects (font (size 1.27 1.27)) (justify left)))
   (property "Value" "NT3H2111W0FHKH" (at 52.07 52.07 0) (effects (font (size 1.27 1.27)) (justify left)))
   (property "Footprint" "NXP:NXP_SOT902-3_XQFN-8_1.6x1.6mm_P0.5mm" (at 50.8 72.39 0) (effects (font (size 1.27 1.27))) (hide yes))
@@
   (pin "6")
   (pin "2")
-  (instances (project "t1-main-board" (path "/7746052e-d7f9-59ad-ba73-bd2b74439529/338b6b86-006f-5bfa-ad71-6e8aca3fbcdb" (reference "U5401") (unit 1))))
+  (instances (project "t1-main-board" (path "/7746052e-d7f9-59ad-ba73-bd2b74439529/338b6b86-006f-5bfa-ad71-6e8aca3fbcdb" (reference "U6001") (unit 1))))
 )
 (wire (pts (xy 40.64 67.31) (xy 38.1 67.31)) (stroke (width 0) (type default)))
@@
 )
 (symbol (lib_id "Device:C") (at 78.74 58.42 0) (unit 1) (body_style 1) (exclude_from_sim no) (in_bom yes) (on_board yes) (dnp no)
-  (property "Reference" "C5401" (at 81.28 57.15 0) (effects (font (size 1.27 1.27)) (justify left)))
+  (property "Reference" "C6001" (at 81.28 57.15 0) (effects (font (size 1.27 1.27)) (justify left)))
   (property "Value" "100 nF" (at 81.28 59.69 0) (effects (font (size 1.27 1.27)) (justify left)))
   (property "Footprint" "Capacitor_SMD:C_0402_1005Metric" (at 78.74 58.42 0) (effects (font (size 1.27 1.27))) (hide yes))
@@
   (pin "1")
   (pin "2")
-  (instances (project "t1-main-board" (path "/7746052e-d7f9-59ad-ba73-bd2b74439529/338b6b86-006f-5bfa-ad71-6e8aca3fbcdb" (reference "C5401") (unit 1))))
+  (instances (project "t1-main-board" (path "/7746052e-d7f9-59ad-ba73-bd2b74439529/338b6b86-006f-5bfa-ad71-6e8aca3fbcdb" (reference "C6001") (unit 1))))
 )
 (wire (pts (xy 78.74 54.61) (xy 78.74 52.07)) (stroke (width 0) (type default)))
@@
 (text "NT3H2111 NTAG I2C plus at I2C2 0x55 (BOM v1 line 125)" (exclude_from_sim no) (at 24.13 34.29 0) (effects (font (size 2.54 2.54)) (justify left bottom)))
 (symbol (lib_id "Device:R") (at 191.77 50.8 90) (unit 1) (body_style 1) (exclude_from_sim no) (in_bom yes) (on_board yes) (dnp no)
-  (property "Reference" "R5401" (at 189.23 46.99 90) (effects (font (size 1.27 1.27))))
+  (property "Reference" "R6001" (at 189.23 46.99 90) (effects (font (size 1.27 1.27))))
   (property "Value" "10 Ω" (at 189.23 53.34 90) (effects (font (size 1.27 1.27))))
   (property "Spec" "0603" (at 189.23 55.88 90) (effects (font (size 1.27 1.27))))
@@
   (pin "1")
   (pin "2")
-  (instances (project "t1-main-board" (path "/7746052e-d7f9-59ad-ba73-bd2b74439529/338b6b86-006f-5bfa-ad71-6e8aca3fbcdb" (reference "R5401") (unit 1) (variant (name "production") (field (name "Value") (value "0 Ω")) (field (name "MPN") (value "RC0603JR-070RL")) (field (name "Manufacturer") (value "YAGEO"))))))
+  (instances (project "t1-main-board" (path "/7746052e-d7f9-59ad-ba73-bd2b74439529/338b6b86-006f-5bfa-ad71-6e8aca3fbcdb" (reference "R6001") (unit 1) (variant (name "production") (field (name "Value") (value "0 Ω")) (field (name "MPN") (value "RC0603JR-070RL")) (field (name "Manufacturer") (value "YAGEO"))))))
 )
 (rectangle (start 168.91 38.1) (end 214.63 58.42) (stroke (width 0) (type dash)) (fill (type none)))
@@
 (wire (pts (xy 185.42 50.8) (xy 185.42 48.26)) (stroke (width 0) (type default)))
 (symbol (lib_id "Connector:TestPoint") (at 185.42 48.26 0) (unit 1) (body_style 1) (exclude_from_sim no) (in_bom no) (on_board yes) (dnp no)
-  (property "Reference" "TP5401" (at 184.15 43.18 0) (effects (font (size 1.27 1.27)) (justify right)))
+  (property "Reference" "TP6001" (at 184.15 43.18 0) (effects (font (size 1.27 1.27)) (justify right)))
   (property "Value" "vcca1v8_pmu" (at 184.15 45.72 0) (effects (font (size 1.27 1.27)) (justify right)))
   (property "Footprint" "TestPoint:TestPoint_Pad_D1.0mm" (at 185.42 48.26 0) (effects (font (size 1.27 1.27))) (hide yes))
@@
   (property "Block" "blk.nfc-tag" (at 185.42 48.26 0) (effects (font (size 1.27 1.27))) (hide yes))
   (pin "1")
-  (instances (project "t1-main-board" (path "/7746052e-d7f9-59ad-ba73-bd2b74439529/338b6b86-006f-5bfa-ad71-6e8aca3fbcdb" (reference "TP5401") (unit 1))))
+  (instances (project "t1-main-board" (path "/7746052e-d7f9-59ad-ba73-bd2b74439529/338b6b86-006f-5bfa-ad71-6e8aca3fbcdb" (reference "TP6001") (unit 1))))
 )
 (symbol (lib_id "power:VCC") (at 166.37 50.8 90) (unit 1) (body_style 1) (exclude_from_sim no) (in_bom yes) (on_board yes) (dnp no)
@@
 (wire (pts (xy 198.12 50.8) (xy 198.12 48.26)) (stroke (width 0) (type default)))
 (symbol (lib_id "Connector:TestPoint") (at 198.12 48.26 0) (unit 1) (body_style 1) (exclude_from_sim no) (in_bom no) (on_board yes) (dnp no)
-  (property "Reference" "TP5402" (at 199.39 43.18 0) (effects (font (size 1.27 1.27)) (justify left)))
+  (property "Reference" "TP6002" (at 199.39 43.18 0) (effects (font (size 1.27 1.27)) (justify left)))
   (property "Value" "NFC_TAG_VCC" (at 199.39 45.72 0) (effects (font (size 1.27 1.27)) (justify left)))
   (property "Footprint" "TestPoint:TestPoint_Pad_D1.0mm" (at 198.12 48.26 0) (effects (font (size 1.27 1.27))) (hide yes))
@@
   (property "Block" "blk.nfc-tag" (at 198.12 48.26 0) (effects (font (size 1.27 1.27))) (hide yes))
   (pin "1")
-  (instances (project "t1-main-board" (path "/7746052e-d7f9-59ad-ba73-bd2b74439529/338b6b86-006f-5bfa-ad71-6e8aca3fbcdb" (reference "TP5402") (unit 1))))
+  (instances (project "t1-main-board" (path "/7746052e-d7f9-59ad-ba73-bd2b74439529/338b6b86-006f-5bfa-ad71-6e8aca3fbcdb" (reference "TP6002") (unit 1))))
 )
 (junction (at 222.25 50.8) (diameter 0) (color 0 0 0 0))
@@
 )
 (symbol (lib_id "Connector:TestPoint") (at 168.91 81.28 0) (unit 1) (body_style 1) (exclude_from_sim no) (in_bom no) (on_board yes) (dnp no)
-  (property "Reference" "TP5403" (at 167.64 76.2 0) (effects (font (size 1.27 1.27)) (justify right)))
+  (property "Reference" "TP6003" (at 167.64 76.2 0) (effects (font (size 1.27 1.27)) (justify right)))
   (property "Value" "NFC_TAG_LA" (at 167.64 78.74 0) (effects (font (size 1.27 1.27)) (justify right)))
   (property "Footprint" "TestPoint:TestPoint_Pad_D1.0mm" (at 168.91 81.28 0) (effects (font (size 1.27 1.27))) (hide yes))
@@
   (property "Block" "blk.nfc-tag" (at 168.91 81.28 0) (effects (font (size 1.27 1.27))) (hide yes))
   (pin "1")
-  (instances (project "t1-main-board" (path "/7746052e-d7f9-59ad-ba73-bd2b74439529/338b6b86-006f-5bfa-ad71-6e8aca3fbcdb" (reference "TP5403") (unit 1))))
+  (instances (project "t1-main-board" (path "/7746052e-d7f9-59ad-ba73-bd2b74439529/338b6b86-006f-5bfa-ad71-6e8aca3fbcdb" (reference "TP6003") (unit 1))))
 )
 (symbol (lib_id "Connector:TestPoint") (at 186.69 81.28 0) (unit 1) (body_style 1) (exclude_from_sim no) (in_bom no) (on_board yes) (dnp no)
-  (property "Reference" "TP5404" (at 185.42 76.2 0) (effects (font (size 1.27 1.27)) (justify right)))
+  (property "Reference" "TP6004" (at 185.42 76.2 0) (effects (font (size 1.27 1.27)) (justify right)))
   (property "Value" "NFC_TAG_LB" (at 185.42 78.74 0) (effects (font (size 1.27 1.27)) (justify right)))
   (property "Footprint" "TestPoint:TestPoint_Pad_D1.0mm" (at 186.69 81.28 0) (effects (font (size 1.27 1.27))) (hide yes))
@@
   (property "Block" "blk.nfc-tag" (at 186.69 81.28 0) (effects (font (size 1.27 1.27))) (hide yes))
   (pin "1")
-  (instances (project "t1-main-board" (path "/7746052e-d7f9-59ad-ba73-bd2b74439529/338b6b86-006f-5bfa-ad71-6e8aca3fbcdb" (reference "TP5404") (unit 1))))
+  (instances (project "t1-main-board" (path "/7746052e-d7f9-59ad-ba73-bd2b74439529/338b6b86-006f-5bfa-ad71-6e8aca3fbcdb" (reference "TP6004") (unit 1))))
 )
 (rectangle (start 152.4 71.12) (end 245.11 97.79) (stroke (width 0) (type dash)) (fill (type none)))
