File: board/hardware/t1-main-board/nfc-tag.kicad_sch (KiCad schematic)
At the start: 7 parts, among them U6001 NT3H2111W0FHKH

Commit message: Board: capture blk.debug
Debug UART2 (1.8 V) and I2S/DSD pads with ground pads, reset, PMIC and
power-key pads (PCB-T-09), a pad on every spare SoC GPIO whose pinout v1
row names one (the DEBUG bus, on the SoC's right edge), and a rail pad
for each power-tree rail no other sheet probes (PCB-T-02). Each DAC
sheet carries a pad on its MCLK. The spares pinout v1 leaves without a
pad now carry no-connect flags. On the root, facing sheet pins are
joined directly only where the route meets no other symbol.

Co-Authored-By: Claude Opus 5.5 <noreply@anthropic.com>
Claude-Session: https://claude.ai/code/session_01Ei262h3TpgY9vyfNLMi5Mn
Parts:
- removed C6001: 100 nF, Capacitor_SMD:C_0402_1005Metric, symbol Device:C
- removed R6001: 10 Ω, Resistor_SMD:R_0603_1608Metric, symbol Device:R
- removed TP6001: vcca1v8_pmu, TestPoint:TestPoint_Pad_D1.0mm, symbol Connector:TestPoint
- removed TP6002: NFC_TAG_VCC, TestPoint:TestPoint_Pad_D1.0mm, symbol Connector:TestPoint
- removed TP6003: NFC_TAG_LA, TestPoint:TestPoint_Pad_D1.0mm, symbol Connector:TestPoint
- removed TP6004: NFC_TAG_LB, TestPoint:TestPoint_Pad_D1.0mm, symbol Connector:TestPoint
- removed U6001: NT3H2111W0FHKH, NXP:NXP_SOT902-3_XQFN-8_1.6x1.6mm_P0.5mm, symbol NXP:NT3H2111W0FHKH
- added C6101: 100 nF, Capacitor_SMD:C_0402_1005Metric, symbol Device:C
- added R6101: 10 Ω, Resistor_SMD:R_0603_1608Metric, symbol Device:R
- added TP6101: vcca1v8_pmu, TestPoint:TestPoint_Pad_D1.0mm, symbol Connector:TestPoint
- added TP6102: NFC_TAG_VCC, TestPoint:TestPoint_Pad_D1.0mm, symbol Connector:TestPoint
- added TP6103: NFC_TAG_LA, TestPoint:TestPoint_Pad_D1.0mm, symbol Connector:TestPoint
- added TP6104: NFC_TAG_LB, TestPoint:TestPoint_Pad_D1.0mm, symbol Connector:TestPoint
- added U6101: NT3H2111W0FHKH, NXP:NXP_SOT902-3_XQFN-8_1.6x1.6mm_P0.5mm, symbol NXP:NT3H2111W0FHKH
Connections:
- net GND: now also C6101.2, U6101.2 (VSS)
- net I2C2_SCL: now also U6101.3 (SCL)
- net I2C2_SDA: now also U6101.5 (SDA)
- net NFC_FD_N: now also U6101.4 (FD)
- net NFC_TAG_LA: now also TP6103.1, U6101.1 (LA)
- net NFC_TAG_LB: now also TP6104.1, U6101.8 (LB)
- net NFC_TAG_VCC: now also C6101.1, R6101.2, TP6102.1, U6101.6 (VCC)
- net vcca1v8_pmu: now also R6101.1, TP6101.1
Changed lines of the file:
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@@
 (title_block (title "NFC tag") (date "2026-10-25") (rev "A") (company "The OpenDAP Project") (comment 1 "blk.nfc-tag") (comment 2 "NTAG I2C plus on I2C2 at 0x55, field detect and the loop antenna contacts"))
 (symbol (lib_id "NXP:NT3H2111W0FHKH") (at 50.8 72.39 0) (unit 1) (body_style 1) (exclude_from_sim no) (in_bom yes) (on_board yes) (dnp no)
-  (property "Reference" "U6001" (at 52.07 54.61 0) (effects (font (size 1.27 1.27)) (justify left)))
+  (property "Reference" "U6101" (at 52.07 54.61 0) (effects (font (size 1.27 1.27)) (justify left)))
   (property "Value" "NT3H2111W0FHKH" (at 52.07 52.07 0) (effects (font (size 1.27 1.27)) (justify left)))
   (property "Footprint" "NXP:NXP_SOT902-3_XQFN-8_1.6x1.6mm_P0.5mm" (at 50.8 72.39 0) (effects (font (size 1.27 1.27))) (hide yes))
@@
   (pin "6")
   (pin "2")
-  (instances (project "t1-main-board" (path "/7746052e-d7f9-59ad-ba73-bd2b74439529/338b6b86-006f-5bfa-ad71-6e8aca3fbcdb" (reference "U6001") (unit 1))))
+  (instances (project "t1-main-board" (path "/7746052e-d7f9-59ad-ba73-bd2b74439529/338b6b86-006f-5bfa-ad71-6e8aca3fbcdb" (reference "U6101") (unit 1))))
 )
 (wire (pts (xy 40.64 67.31) (xy 38.1 67.31)) (stroke (width 0) (type default)))
@@
 )
 (symbol (lib_id "Device:C") (at 78.74 58.42 0) (unit 1) (body_style 1) (exclude_from_sim no) (in_bom yes) (on_board yes) (dnp no)
-  (property "Reference" "C6001" (at 81.28 57.15 0) (effects (font (size 1.27 1.27)) (justify left)))
+  (property "Reference" "C6101" (at 81.28 57.15 0) (effects (font (size 1.27 1.27)) (justify left)))
   (property "Value" "100 nF" (at 81.28 59.69 0) (effects (font (size 1.27 1.27)) (justify left)))
   (property "Footprint" "Capacitor_SMD:C_0402_1005Metric" (at 78.74 58.42 0) (effects (font (size 1.27 1.27))) (hide yes))
@@
   (pin "1")
   (pin "2")
-  (instances (project "t1-main-board" (path "/7746052e-d7f9-59ad-ba73-bd2b74439529/338b6b86-006f-5bfa-ad71-6e8aca3fbcdb" (reference "C6001") (unit 1))))
+  (instances (project "t1-main-board" (path "/7746052e-d7f9-59ad-ba73-bd2b74439529/338b6b86-006f-5bfa-ad71-6e8aca3fbcdb" (reference "C6101") (unit 1))))
 )
 (wire (pts (xy 78.74 54.61) (xy 78.74 52.07)) (stroke (width 0) (type default)))
@@
 (text "NT3H2111 NTAG I2C plus at I2C2 0x55 (BOM v1 line 125)" (exclude_from_sim no) (at 24.13 34.29 0) (effects (font (size 2.54 2.54)) (justify left bottom)))
 (symbol (lib_id "Device:R") (at 191.77 50.8 90) (unit 1) (body_style 1) (exclude_from_sim no) (in_bom yes) (on_board yes) (dnp no)
-  (property "Reference" "R6001" (at 189.23 46.99 90) (effects (font (size 1.27 1.27))))
+  (property "Reference" "R6101" (at 189.23 46.99 90) (effects (font (size 1.27 1.27))))
   (property "Value" "10 Ω" (at 189.23 53.34 90) (effects (font (size 1.27 1.27))))
   (property "Spec" "0603" (at 189.23 55.88 90) (effects (font (size 1.27 1.27))))
@@
   (pin "1")
   (pin "2")
-  (instances (project "t1-main-board" (path "/7746052e-d7f9-59ad-ba73-bd2b74439529/338b6b86-006f-5bfa-ad71-6e8aca3fbcdb" (reference "R6001") (unit 1) (variant (name "production") (field (name "Value") (value "0 Ω")) (field (name "MPN") (value "RC0603JR-070RL")) (field (name "Manufacturer") (value "YAGEO"))))))
+  (instances (project "t1-main-board" (path "/7746052e-d7f9-59ad-ba73-bd2b74439529/338b6b86-006f-5bfa-ad71-6e8aca3fbcdb" (reference "R6101") (unit 1) (variant (name "production") (field (name "Value") (value "0 Ω")) (field (name "MPN") (value "RC0603JR-070RL")) (field (name "Manufacturer") (value "YAGEO"))))))
 )
 (rectangle (start 168.91 38.1) (end 214.63 58.42) (stroke (width 0) (type dash)) (fill (type none)))
@@
 (wire (pts (xy 185.42 50.8) (xy 185.42 48.26)) (stroke (width 0) (type default)))
 (symbol (lib_id "Connector:TestPoint") (at 185.42 48.26 0) (unit 1) (body_style 1) (exclude_from_sim no) (in_bom no) (on_board yes) (dnp no)
-  (property "Reference" "TP6001" (at 184.15 43.18 0) (effects (font (size 1.27 1.27)) (justify right)))
+  (property "Reference" "TP6101" (at 184.15 43.18 0) (effects (font (size 1.27 1.27)) (justify right)))
   (property "Value" "vcca1v8_pmu" (at 184.15 45.72 0) (effects (font (size 1.27 1.27)) (justify right)))
   (property "Footprint" "TestPoint:TestPoint_Pad_D1.0mm" (at 185.42 48.26 0) (effects (font (size 1.27 1.27))) (hide yes))
@@
   (property "Block" "blk.nfc-tag" (at 185.42 48.26 0) (effects (font (size 1.27 1.27))) (hide yes))
   (pin "1")
-  (instances (project "t1-main-board" (path "/7746052e-d7f9-59ad-ba73-bd2b74439529/338b6b86-006f-5bfa-ad71-6e8aca3fbcdb" (reference "TP6001") (unit 1))))
+  (instances (project "t1-main-board" (path "/7746052e-d7f9-59ad-ba73-bd2b74439529/338b6b86-006f-5bfa-ad71-6e8aca3fbcdb" (reference "TP6101") (unit 1))))
 )
 (symbol (lib_id "power:VCC") (at 166.37 50.8 90) (unit 1) (body_style 1) (exclude_from_sim no) (in_bom yes) (on_board yes) (dnp no)
@@
 (wire (pts (xy 198.12 50.8) (xy 198.12 48.26)) (stroke (width 0) (type default)))
 (symbol (lib_id "Connector:TestPoint") (at 198.12 48.26 0) (unit 1) (body_style 1) (exclude_from_sim no) (in_bom no) (on_board yes) (dnp no)
-  (property "Reference" "TP6002" (at 199.39 43.18 0) (effects (font (size 1.27 1.27)) (justify left)))
+  (property "Reference" "TP6102" (at 199.39 43.18 0) (effects (font (size 1.27 1.27)) (justify left)))
   (property "Value" "NFC_TAG_VCC" (at 199.39 45.72 0) (effects (font (size 1.27 1.27)) (justify left)))
   (property "Footprint" "TestPoint:TestPoint_Pad_D1.0mm" (at 198.12 48.26 0) (effects (font (size 1.27 1.27))) (hide yes))
@@
   (property "Block" "blk.nfc-tag" (at 198.12 48.26 0) (effects (font (size 1.27 1.27))) (hide yes))
   (pin "1")
-  (instances (project "t1-main-board" (path "/7746052e-d7f9-59ad-ba73-bd2b74439529/338b6b86-006f-5bfa-ad71-6e8aca3fbcdb" (reference "TP6002") (unit 1))))
+  (instances (project "t1-main-board" (path "/7746052e-d7f9-59ad-ba73-bd2b74439529/338b6b86-006f-5bfa-ad71-6e8aca3fbcdb" (reference "TP6102") (unit 1))))
 )
 (junction (at 222.25 50.8) (diameter 0) (color 0 0 0 0))
@@
 )
 (symbol (lib_id "Connector:TestPoint") (at 168.91 81.28 0) (unit 1) (body_style 1) (exclude_from_sim no) (in_bom no) (on_board yes) (dnp no)
-  (property "Reference" "TP6003" (at 167.64 76.2 0) (effects (font (size 1.27 1.27)) (justify right)))
+  (property "Reference" "TP6103" (at 167.64 76.2 0) (effects (font (size 1.27 1.27)) (justify right)))
   (property "Value" "NFC_TAG_LA" (at 167.64 78.74 0) (effects (font (size 1.27 1.27)) (justify right)))
   (property "Footprint" "TestPoint:TestPoint_Pad_D1.0mm" (at 168.91 81.28 0) (effects (font (size 1.27 1.27))) (hide yes))
@@
   (property "Block" "blk.nfc-tag" (at 168.91 81.28 0) (effects (font (size 1.27 1.27))) (hide yes))
   (pin "1")
-  (instances (project "t1-main-board" (path "/7746052e-d7f9-59ad-ba73-bd2b74439529/338b6b86-006f-5bfa-ad71-6e8aca3fbcdb" (reference "TP6003") (unit 1))))
+  (instances (project "t1-main-board" (path "/7746052e-d7f9-59ad-ba73-bd2b74439529/338b6b86-006f-5bfa-ad71-6e8aca3fbcdb" (reference "TP6103") (unit 1))))
 )
 (symbol (lib_id "Connector:TestPoint") (at 186.69 81.28 0) (unit 1) (body_style 1) (exclude_from_sim no) (in_bom no) (on_board yes) (dnp no)
-  (property "Reference" "TP6004" (at 185.42 76.2 0) (effects (font (size 1.27 1.27)) (justify right)))
+  (property "Reference" "TP6104" (at 185.42 76.2 0) (effects (font (size 1.27 1.27)) (justify right)))
   (property "Value" "NFC_TAG_LB" (at 185.42 78.74 0) (effects (font (size 1.27 1.27)) (justify right)))
   (property "Footprint" "TestPoint:TestPoint_Pad_D1.0mm" (at 186.69 81.28 0) (effects (font (size 1.27 1.27))) (hide yes))
@@
   (property "Block" "blk.nfc-tag" (at 186.69 81.28 0) (effects (font (size 1.27 1.27))) (hide yes))
   (pin "1")
-  (instances (project "t1-main-board" (path "/7746052e-d7f9-59ad-ba73-bd2b74439529/338b6b86-006f-5bfa-ad71-6e8aca3fbcdb" (reference "TP6004") (unit 1))))
+  (instances (project "t1-main-board" (path "/7746052e-d7f9-59ad-ba73-bd2b74439529/338b6b86-006f-5bfa-ad71-6e8aca3fbcdb" (reference "TP6104") (unit 1))))
 )
 (rectangle (start 152.4 71.12) (end 245.11 97.79) (stroke (width 0) (type dash)) (fill (type none)))

Commit message: Board: capture blk.cover-detect
COVER_DET_N on GPIO0_A6 (AJ38, PMUIO1, wake-capable), recorded in
pinout v1 (closes feature blocks G22): board-edge input and ground pads
for the case's actuator, 100 kΩ to vcc3v3_pmu, TPD1E10B06 at the pad
(BOM v1 line 143, PCB-L-10). The line rides the KEYS bus with the
buttons.

Co-Authored-By: Claude Opus 5.5 <noreply@anthropic.com>
Claude-Session: https://claude.ai/code/session_01Ei262h3TpgY9vyfNLMi5Mn
Parts:
- removed C6101: 100 nF, Capacitor_SMD:C_0402_1005Metric, symbol Device:C
- removed R6101: 10 Ω, Resistor_SMD:R_0603_1608Metric, symbol Device:R
- removed TP6101: vcca1v8_pmu, TestPoint:TestPoint_Pad_D1.0mm, symbol Connector:TestPoint
- removed TP6102: NFC_TAG_VCC, TestPoint:TestPoint_Pad_D1.0mm, symbol Connector:TestPoint
- removed TP6103: NFC_TAG_LA, TestPoint:TestPoint_Pad_D1.0mm, symbol Connector:TestPoint
- removed TP6104: NFC_TAG_LB, TestPoint:TestPoint_Pad_D1.0mm, symbol Connector:TestPoint
- removed U6101: NT3H2111W0FHKH, NXP:NXP_SOT902-3_XQFN-8_1.6x1.6mm_P0.5mm, symbol NXP:NT3H2111W0FHKH
- added C6201: 100 nF, Capacitor_SMD:C_0402_1005Metric, symbol Device:C
- added R6201: 10 Ω, Resistor_SMD:R_0603_1608Metric, symbol Device:R
- added TP6201: vcca1v8_pmu, TestPoint:TestPoint_Pad_D1.0mm, symbol Connector:TestPoint
- added TP6202: NFC_TAG_VCC, TestPoint:TestPoint_Pad_D1.0mm, symbol Connector:TestPoint
- added TP6203: NFC_TAG_LA, TestPoint:TestPoint_Pad_D1.0mm, symbol Connector:TestPoint
- added TP6204: NFC_TAG_LB, TestPoint:TestPoint_Pad_D1.0mm, symbol Connector:TestPoint
- added U6201: NT3H2111W0FHKH, NXP:NXP_SOT902-3_XQFN-8_1.6x1.6mm_P0.5mm, symbol NXP:NT3H2111W0FHKH
Connections:
- net GND: now also C6201.2, U6201.2 (VSS)
- net I2C2_SCL: now also U6201.3 (SCL)
- net I2C2_SDA: now also U6201.5 (SDA)
- net NFC_FD_N: now also U6201.4 (FD)
- net NFC_TAG_LA: now also TP6203.1, U6201.1 (LA)
- net NFC_TAG_LB: now also TP6204.1, U6201.8 (LB)
- net NFC_TAG_VCC: now also C6201.1, R6201.2, TP6202.1, U6201.6 (VCC)
- net vcca1v8_pmu: now also R6201.1, TP6201.1
Changed lines of the file:
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@@
 (title_block (title "NFC tag") (date "2026-10-25") (rev "A") (company "The OpenDAP Project") (comment 1 "blk.nfc-tag") (comment 2 "NTAG I2C plus on I2C2 at 0x55, field detect and the loop antenna contacts"))
 (symbol (lib_id "NXP:NT3H2111W0FHKH") (at 50.8 72.39 0) (unit 1) (body_style 1) (exclude_from_sim no) (in_bom yes) (on_board yes) (dnp no)
-  (property "Reference" "U6101" (at 52.07 54.61 0) (effects (font (size 1.27 1.27)) (justify left)))
+  (property "Reference" "U6201" (at 52.07 54.61 0) (effects (font (size 1.27 1.27)) (justify left)))
   (property "Value" "NT3H2111W0FHKH" (at 52.07 52.07 0) (effects (font (size 1.27 1.27)) (justify left)))
   (property "Footprint" "NXP:NXP_SOT902-3_XQFN-8_1.6x1.6mm_P0.5mm" (at 50.8 72.39 0) (effects (font (size 1.27 1.27))) (hide yes))
@@
   (pin "6")
   (pin "2")
-  (instances (project "t1-main-board" (path "/7746052e-d7f9-59ad-ba73-bd2b74439529/338b6b86-006f-5bfa-ad71-6e8aca3fbcdb" (reference "U6101") (unit 1))))
+  (instances (project "t1-main-board" (path "/7746052e-d7f9-59ad-ba73-bd2b74439529/338b6b86-006f-5bfa-ad71-6e8aca3fbcdb" (reference "U6201") (unit 1))))
 )
 (wire (pts (xy 40.64 67.31) (xy 38.1 67.31)) (stroke (width 0) (type default)))
@@
 )
 (symbol (lib_id "Device:C") (at 78.74 58.42 0) (unit 1) (body_style 1) (exclude_from_sim no) (in_bom yes) (on_board yes) (dnp no)
-  (property "Reference" "C6101" (at 81.28 57.15 0) (effects (font (size 1.27 1.27)) (justify left)))
+  (property "Reference" "C6201" (at 81.28 57.15 0) (effects (font (size 1.27 1.27)) (justify left)))
   (property "Value" "100 nF" (at 81.28 59.69 0) (effects (font (size 1.27 1.27)) (justify left)))
   (property "Footprint" "Capacitor_SMD:C_0402_1005Metric" (at 78.74 58.42 0) (effects (font (size 1.27 1.27))) (hide yes))
@@
   (pin "1")
   (pin "2")
-  (instances (project "t1-main-board" (path "/7746052e-d7f9-59ad-ba73-bd2b74439529/338b6b86-006f-5bfa-ad71-6e8aca3fbcdb" (reference "C6101") (unit 1))))
+  (instances (project "t1-main-board" (path "/7746052e-d7f9-59ad-ba73-bd2b74439529/338b6b86-006f-5bfa-ad71-6e8aca3fbcdb" (reference "C6201") (unit 1))))
 )
 (wire (pts (xy 78.74 54.61) (xy 78.74 52.07)) (stroke (width 0) (type default)))
@@
 (text "NT3H2111 NTAG I2C plus at I2C2 0x55 (BOM v1 line 125)" (exclude_from_sim no) (at 24.13 34.29 0) (effects (font (size 2.54 2.54)) (justify left bottom)))
 (symbol (lib_id "Device:R") (at 191.77 50.8 90) (unit 1) (body_style 1) (exclude_from_sim no) (in_bom yes) (on_board yes) (dnp no)
-  (property "Reference" "R6101" (at 189.23 46.99 90) (effects (font (size 1.27 1.27))))
+  (property "Reference" "R6201" (at 189.23 46.99 90) (effects (font (size 1.27 1.27))))
   (property "Value" "10 Ω" (at 189.23 53.34 90) (effects (font (size 1.27 1.27))))
   (property "Spec" "0603" (at 189.23 55.88 90) (effects (font (size 1.27 1.27))))
@@
   (pin "1")
   (pin "2")
-  (instances (project "t1-main-board" (path "/7746052e-d7f9-59ad-ba73-bd2b74439529/338b6b86-006f-5bfa-ad71-6e8aca3fbcdb" (reference "R6101") (unit 1) (variant (name "production") (field (name "Value") (value "0 Ω")) (field (name "MPN") (value "RC0603JR-070RL")) (field (name "Manufacturer") (value "YAGEO"))))))
+  (instances (project "t1-main-board" (path "/7746052e-d7f9-59ad-ba73-bd2b74439529/338b6b86-006f-5bfa-ad71-6e8aca3fbcdb" (reference "R6201") (unit 1) (variant (name "production") (field (name "Value") (value "0 Ω")) (field (name "MPN") (value "RC0603JR-070RL")) (field (name "Manufacturer") (value "YAGEO"))))))
 )
 (rectangle (start 168.91 38.1) (end 214.63 58.42) (stroke (width 0) (type dash)) (fill (type none)))
@@
 (wire (pts (xy 185.42 50.8) (xy 185.42 48.26)) (stroke (width 0) (type default)))
 (symbol (lib_id "Connector:TestPoint") (at 185.42 48.26 0) (unit 1) (body_style 1) (exclude_from_sim no) (in_bom no) (on_board yes) (dnp no)
-  (property "Reference" "TP6101" (at 184.15 43.18 0) (effects (font (size 1.27 1.27)) (justify right)))
+  (property "Reference" "TP6201" (at 184.15 43.18 0) (effects (font (size 1.27 1.27)) (justify right)))
   (property "Value" "vcca1v8_pmu" (at 184.15 45.72 0) (effects (font (size 1.27 1.27)) (justify right)))
   (property "Footprint" "TestPoint:TestPoint_Pad_D1.0mm" (at 185.42 48.26 0) (effects (font (size 1.27 1.27))) (hide yes))
@@
   (property "Block" "blk.nfc-tag" (at 185.42 48.26 0) (effects (font (size 1.27 1.27))) (hide yes))
   (pin "1")
-  (instances (project "t1-main-board" (path "/7746052e-d7f9-59ad-ba73-bd2b74439529/338b6b86-006f-5bfa-ad71-6e8aca3fbcdb" (reference "TP6101") (unit 1))))
+  (instances (project "t1-main-board" (path "/7746052e-d7f9-59ad-ba73-bd2b74439529/338b6b86-006f-5bfa-ad71-6e8aca3fbcdb" (reference "TP6201") (unit 1))))
 )
 (symbol (lib_id "power:VCC") (at 166.37 50.8 90) (unit 1) (body_style 1) (exclude_from_sim no) (in_bom yes) (on_board yes) (dnp no)
@@
 (wire (pts (xy 198.12 50.8) (xy 198.12 48.26)) (stroke (width 0) (type default)))
 (symbol (lib_id "Connector:TestPoint") (at 198.12 48.26 0) (unit 1) (body_style 1) (exclude_from_sim no) (in_bom no) (on_board yes) (dnp no)
-  (property "Reference" "TP6102" (at 199.39 43.18 0) (effects (font (size 1.27 1.27)) (justify left)))
+  (property "Reference" "TP6202" (at 199.39 43.18 0) (effects (font (size 1.27 1.27)) (justify left)))
   (property "Value" "NFC_TAG_VCC" (at 199.39 45.72 0) (effects (font (size 1.27 1.27)) (justify left)))
   (property "Footprint" "TestPoint:TestPoint_Pad_D1.0mm" (at 198.12 48.26 0) (effects (font (size 1.27 1.27))) (hide yes))
@@
   (property "Block" "blk.nfc-tag" (at 198.12 48.26 0) (effects (font (size 1.27 1.27))) (hide yes))
   (pin "1")
-  (instances (project "t1-main-board" (path "/7746052e-d7f9-59ad-ba73-bd2b74439529/338b6b86-006f-5bfa-ad71-6e8aca3fbcdb" (reference "TP6102") (unit 1))))
+  (instances (project "t1-main-board" (path "/7746052e-d7f9-59ad-ba73-bd2b74439529/338b6b86-006f-5bfa-ad71-6e8aca3fbcdb" (reference "TP6202") (unit 1))))
 )
 (junction (at 222.25 50.8) (diameter 0) (color 0 0 0 0))
@@
 )
 (symbol (lib_id "Connector:TestPoint") (at 168.91 81.28 0) (unit 1) (body_style 1) (exclude_from_sim no) (in_bom no) (on_board yes) (dnp no)
-  (property "Reference" "TP6103" (at 167.64 76.2 0) (effects (font (size 1.27 1.27)) (justify right)))
+  (property "Reference" "TP6203" (at 167.64 76.2 0) (effects (font (size 1.27 1.27)) (justify right)))
   (property "Value" "NFC_TAG_LA" (at 167.64 78.74 0) (effects (font (size 1.27 1.27)) (justify right)))
   (property "Footprint" "TestPoint:TestPoint_Pad_D1.0mm" (at 168.91 81.28 0) (effects (font (size 1.27 1.27))) (hide yes))
@@
   (property "Block" "blk.nfc-tag" (at 168.91 81.28 0) (effects (font (size 1.27 1.27))) (hide yes))
   (pin "1")
-  (instances (project "t1-main-board" (path "/7746052e-d7f9-59ad-ba73-bd2b74439529/338b6b86-006f-5bfa-ad71-6e8aca3fbcdb" (reference "TP6103") (unit 1))))
+  (instances (project "t1-main-board" (path "/7746052e-d7f9-59ad-ba73-bd2b74439529/338b6b86-006f-5bfa-ad71-6e8aca3fbcdb" (reference "TP6203") (unit 1))))
 )
 (symbol (lib_id "Connector:TestPoint") (at 186.69 81.28 0) (unit 1) (body_style 1) (exclude_from_sim no) (in_bom no) (on_board yes) (dnp no)
-  (property "Reference" "TP6104" (at 185.42 76.2 0) (effects (font (size 1.27 1.27)) (justify right)))
+  (property "Reference" "TP6204" (at 185.42 76.2 0) (effects (font (size 1.27 1.27)) (justify right)))
   (property "Value" "NFC_TAG_LB" (at 185.42 78.74 0) (effects (font (size 1.27 1.27)) (justify right)))
   (property "Footprint" "TestPoint:TestPoint_Pad_D1.0mm" (at 186.69 81.28 0) (effects (font (size 1.27 1.27))) (hide yes))
@@
   (property "Block" "blk.nfc-tag" (at 186.69 81.28 0) (effects (font (size 1.27 1.27))) (hide yes))
   (pin "1")
-  (instances (project "t1-main-board" (path "/7746052e-d7f9-59ad-ba73-bd2b74439529/338b6b86-006f-5bfa-ad71-6e8aca3fbcdb" (reference "TP6104") (unit 1))))
+  (instances (project "t1-main-board" (path "/7746052e-d7f9-59ad-ba73-bd2b74439529/338b6b86-006f-5bfa-ad71-6e8aca3fbcdb" (reference "TP6204") (unit 1))))
 )
 (rectangle (start 152.4 71.12) (end 245.11 97.79) (stroke (width 0) (type dash)) (fill (type none)))

Commit message: Board: capture blk.mic-ambient and links #34, #35
IM73D122 on PDM CLK1 and SDI1 (BOM v1 line 34, pinout v1 AK2 and 1P2),
LR to ground, 22 Ω clock series, VDD from MIC_1V8 through link #35.
Link #34 on blk.mic-main makes the faceplate branch the rail MIC_1V8_FP
for contact 40 (power tree §4.12, G10). kicad-lib moves to e46bda4 for
the IM73D122, TPS3808G01, SN74LVC1G58 and BAT54 parts.

Co-Authored-By: Claude Opus 5.5 <noreply@anthropic.com>
Claude-Session: https://claude.ai/code/session_01Ei262h3TpgY9vyfNLMi5Mn
Parts:
- removed C6201: 100 nF, Capacitor_SMD:C_0402_1005Metric, symbol Device:C
- removed R6201: 10 Ω, Resistor_SMD:R_0603_1608Metric, symbol Device:R
- removed TP6201: vcca1v8_pmu, TestPoint:TestPoint_Pad_D1.0mm, symbol Connector:TestPoint
- removed TP6202: NFC_TAG_VCC, TestPoint:TestPoint_Pad_D1.0mm, symbol Connector:TestPoint
- removed TP6203: NFC_TAG_LA, TestPoint:TestPoint_Pad_D1.0mm, symbol Connector:TestPoint
- removed TP6204: NFC_TAG_LB, TestPoint:TestPoint_Pad_D1.0mm, symbol Connector:TestPoint
- removed U6201: NT3H2111W0FHKH, NXP:NXP_SOT902-3_XQFN-8_1.6x1.6mm_P0.5mm, symbol NXP:NT3H2111W0FHKH
- added C6301: 100 nF, Capacitor_SMD:C_0402_1005Metric, symbol Device:C
- added R6301: 10 Ω, Resistor_SMD:R_0603_1608Metric, symbol Device:R
- added TP6301: vcca1v8_pmu, TestPoint:TestPoint_Pad_D1.0mm, symbol Connector:TestPoint
- added TP6302: NFC_TAG_VCC, TestPoint:TestPoint_Pad_D1.0mm, symbol Connector:TestPoint
- added TP6303: NFC_TAG_LA, TestPoint:TestPoint_Pad_D1.0mm, symbol Connector:TestPoint
- added TP6304: NFC_TAG_LB, TestPoint:TestPoint_Pad_D1.0mm, symbol Connector:TestPoint
- added U6301: NT3H2111W0FHKH, NXP:NXP_SOT902-3_XQFN-8_1.6x1.6mm_P0.5mm, symbol NXP:NT3H2111W0FHKH
Connections:
- net GND: now also C6301.2, U6301.2 (VSS)
- net I2C2_SCL: now also U6301.3 (SCL)
- net I2C2_SDA: now also U6301.5 (SDA)
- net NFC_FD_N: now also U6301.4 (FD)
- net NFC_TAG_LA: now also TP6303.1, U6301.1 (LA)
- net NFC_TAG_LB: now also TP6304.1, U6301.8 (LB)
- net NFC_TAG_VCC: now also C6301.1, R6301.2, TP6302.1, U6301.6 (VCC)
- net vcca1v8_pmu: now also R6301.1, TP6301.1
