File: board/hardware/t1-main-board/nfc-tag.kicad_sch (KiCad schematic)
At the start: 7 parts, among them U6301 NT3H2111W0FHKH

Commit message: Board: capture blk.maskrom
Power + Vol- at a cold power-on pull eMMC D0 low inside the TPS3808G01
boot window (BOM v1 lines 35, 78, 97, 98; sim/maskrom): SENSE 280k/100k,
CT 390 nF, WINDOW_N with its pad, SN74LVC1G57 and SN74LVC1G58 on
vcca1v8_pmu, BAT54 from PWRON_N, DMG1012T through 1 kΩ to EMMC_D0.
Every block in use now has its sheet; the README states the remaining
single-pin nets.

Co-Authored-By: Claude Opus 5.5 <noreply@anthropic.com>
Claude-Session: https://claude.ai/code/session_01Ei262h3TpgY9vyfNLMi5Mn
Parts:
- removed C6301: 100 nF, Capacitor_SMD:C_0402_1005Metric, symbol Device:C
- removed R6301: 10 Ω, Resistor_SMD:R_0603_1608Metric, symbol Device:R
- removed TP6301: vcca1v8_pmu, TestPoint:TestPoint_Pad_D1.0mm, symbol Connector:TestPoint
- removed TP6302: NFC_TAG_VCC, TestPoint:TestPoint_Pad_D1.0mm, symbol Connector:TestPoint
- removed TP6303: NFC_TAG_LA, TestPoint:TestPoint_Pad_D1.0mm, symbol Connector:TestPoint
- removed TP6304: NFC_TAG_LB, TestPoint:TestPoint_Pad_D1.0mm, symbol Connector:TestPoint
- removed U6301: NT3H2111W0FHKH, NXP:NXP_SOT902-3_XQFN-8_1.6x1.6mm_P0.5mm, symbol NXP:NT3H2111W0FHKH
- added C6401: 100 nF, Capacitor_SMD:C_0402_1005Metric, symbol Device:C
- added R6401: 10 Ω, Resistor_SMD:R_0603_1608Metric, symbol Device:R
- added TP6401: vcca1v8_pmu, TestPoint:TestPoint_Pad_D1.0mm, symbol Connector:TestPoint
- added TP6402: NFC_TAG_VCC, TestPoint:TestPoint_Pad_D1.0mm, symbol Connector:TestPoint
- added TP6403: NFC_TAG_LA, TestPoint:TestPoint_Pad_D1.0mm, symbol Connector:TestPoint
- added TP6404: NFC_TAG_LB, TestPoint:TestPoint_Pad_D1.0mm, symbol Connector:TestPoint
- added U6401: NT3H2111W0FHKH, NXP:NXP_SOT902-3_XQFN-8_1.6x1.6mm_P0.5mm, symbol NXP:NT3H2111W0FHKH
Connections:
- net GND: now also C6401.2, U6401.2 (VSS)
- net I2C2_SCL: now also U6401.3 (SCL)
- net I2C2_SDA: now also U6401.5 (SDA)
- net NFC_FD_N: now also U6401.4 (FD)
- net NFC_TAG_LA: now also TP6403.1, U6401.1 (LA)
- net NFC_TAG_LB: now also TP6404.1, U6401.8 (LB)
- net NFC_TAG_VCC: now also C6401.1, R6401.2, TP6402.1, U6401.6 (VCC)
- net vcca1v8_pmu: now also R6401.1, TP6401.1
Changed lines of the file:
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@@
 (title_block (title "NFC tag") (date "2026-10-25") (rev "A") (company "The OpenDAP Project") (comment 1 "blk.nfc-tag") (comment 2 "NTAG I2C plus on I2C2 at 0x55, field detect and the loop antenna contacts"))
 (symbol (lib_id "NXP:NT3H2111W0FHKH") (at 50.8 72.39 0) (unit 1) (body_style 1) (exclude_from_sim no) (in_bom yes) (on_board yes) (dnp no)
-  (property "Reference" "U6301" (at 52.07 54.61 0) (effects (font (size 1.27 1.27)) (justify left)))
+  (property "Reference" "U6401" (at 52.07 54.61 0) (effects (font (size 1.27 1.27)) (justify left)))
   (property "Value" "NT3H2111W0FHKH" (at 52.07 52.07 0) (effects (font (size 1.27 1.27)) (justify left)))
   (property "Footprint" "NXP:NXP_SOT902-3_XQFN-8_1.6x1.6mm_P0.5mm" (at 50.8 72.39 0) (effects (font (size 1.27 1.27))) (hide yes))
@@
   (pin "6")
   (pin "2")
-  (instances (project "t1-main-board" (path "/7746052e-d7f9-59ad-ba73-bd2b74439529/338b6b86-006f-5bfa-ad71-6e8aca3fbcdb" (reference "U6301") (unit 1))))
+  (instances (project "t1-main-board" (path "/7746052e-d7f9-59ad-ba73-bd2b74439529/338b6b86-006f-5bfa-ad71-6e8aca3fbcdb" (reference "U6401") (unit 1))))
 )
 (wire (pts (xy 40.64 67.31) (xy 38.1 67.31)) (stroke (width 0) (type default)))
@@
 )
 (symbol (lib_id "Device:C") (at 78.74 58.42 0) (unit 1) (body_style 1) (exclude_from_sim no) (in_bom yes) (on_board yes) (dnp no)
-  (property "Reference" "C6301" (at 81.28 57.15 0) (effects (font (size 1.27 1.27)) (justify left)))
+  (property "Reference" "C6401" (at 81.28 57.15 0) (effects (font (size 1.27 1.27)) (justify left)))
   (property "Value" "100 nF" (at 81.28 59.69 0) (effects (font (size 1.27 1.27)) (justify left)))
   (property "Footprint" "Capacitor_SMD:C_0402_1005Metric" (at 78.74 58.42 0) (effects (font (size 1.27 1.27))) (hide yes))
@@
   (pin "1")
   (pin "2")
-  (instances (project "t1-main-board" (path "/7746052e-d7f9-59ad-ba73-bd2b74439529/338b6b86-006f-5bfa-ad71-6e8aca3fbcdb" (reference "C6301") (unit 1))))
+  (instances (project "t1-main-board" (path "/7746052e-d7f9-59ad-ba73-bd2b74439529/338b6b86-006f-5bfa-ad71-6e8aca3fbcdb" (reference "C6401") (unit 1))))
 )
 (wire (pts (xy 78.74 54.61) (xy 78.74 52.07)) (stroke (width 0) (type default)))
@@
 (text "NT3H2111 NTAG I2C plus at I2C2 0x55 (BOM v1 line 125)" (exclude_from_sim no) (at 24.13 34.29 0) (effects (font (size 2.54 2.54)) (justify left bottom)))
 (symbol (lib_id "Device:R") (at 191.77 50.8 90) (unit 1) (body_style 1) (exclude_from_sim no) (in_bom yes) (on_board yes) (dnp no)
-  (property "Reference" "R6301" (at 189.23 46.99 90) (effects (font (size 1.27 1.27))))
+  (property "Reference" "R6401" (at 189.23 46.99 90) (effects (font (size 1.27 1.27))))
   (property "Value" "10 Ω" (at 189.23 53.34 90) (effects (font (size 1.27 1.27))))
   (property "Spec" "0603" (at 189.23 55.88 90) (effects (font (size 1.27 1.27))))
@@
   (pin "1")
   (pin "2")
-  (instances (project "t1-main-board" (path "/7746052e-d7f9-59ad-ba73-bd2b74439529/338b6b86-006f-5bfa-ad71-6e8aca3fbcdb" (reference "R6301") (unit 1) (variant (name "production") (field (name "Value") (value "0 Ω")) (field (name "MPN") (value "RC0603JR-070RL")) (field (name "Manufacturer") (value "YAGEO"))))))
+  (instances (project "t1-main-board" (path "/7746052e-d7f9-59ad-ba73-bd2b74439529/338b6b86-006f-5bfa-ad71-6e8aca3fbcdb" (reference "R6401") (unit 1) (variant (name "production") (field (name "Value") (value "0 Ω")) (field (name "MPN") (value "RC0603JR-070RL")) (field (name "Manufacturer") (value "YAGEO"))))))
 )
 (rectangle (start 168.91 38.1) (end 214.63 58.42) (stroke (width 0) (type dash)) (fill (type none)))
@@
 (wire (pts (xy 185.42 50.8) (xy 185.42 48.26)) (stroke (width 0) (type default)))
 (symbol (lib_id "Connector:TestPoint") (at 185.42 48.26 0) (unit 1) (body_style 1) (exclude_from_sim no) (in_bom no) (on_board yes) (dnp no)
-  (property "Reference" "TP6301" (at 184.15 43.18 0) (effects (font (size 1.27 1.27)) (justify right)))
+  (property "Reference" "TP6401" (at 184.15 43.18 0) (effects (font (size 1.27 1.27)) (justify right)))
   (property "Value" "vcca1v8_pmu" (at 184.15 45.72 0) (effects (font (size 1.27 1.27)) (justify right)))
   (property "Footprint" "TestPoint:TestPoint_Pad_D1.0mm" (at 185.42 48.26 0) (effects (font (size 1.27 1.27))) (hide yes))
@@
   (property "Block" "blk.nfc-tag" (at 185.42 48.26 0) (effects (font (size 1.27 1.27))) (hide yes))
   (pin "1")
-  (instances (project "t1-main-board" (path "/7746052e-d7f9-59ad-ba73-bd2b74439529/338b6b86-006f-5bfa-ad71-6e8aca3fbcdb" (reference "TP6301") (unit 1))))
+  (instances (project "t1-main-board" (path "/7746052e-d7f9-59ad-ba73-bd2b74439529/338b6b86-006f-5bfa-ad71-6e8aca3fbcdb" (reference "TP6401") (unit 1))))
 )
 (symbol (lib_id "power:VCC") (at 166.37 50.8 90) (unit 1) (body_style 1) (exclude_from_sim no) (in_bom yes) (on_board yes) (dnp no)
@@
 (wire (pts (xy 198.12 50.8) (xy 198.12 48.26)) (stroke (width 0) (type default)))
 (symbol (lib_id "Connector:TestPoint") (at 198.12 48.26 0) (unit 1) (body_style 1) (exclude_from_sim no) (in_bom no) (on_board yes) (dnp no)
-  (property "Reference" "TP6302" (at 199.39 43.18 0) (effects (font (size 1.27 1.27)) (justify left)))
+  (property "Reference" "TP6402" (at 199.39 43.18 0) (effects (font (size 1.27 1.27)) (justify left)))
   (property "Value" "NFC_TAG_VCC" (at 199.39 45.72 0) (effects (font (size 1.27 1.27)) (justify left)))
   (property "Footprint" "TestPoint:TestPoint_Pad_D1.0mm" (at 198.12 48.26 0) (effects (font (size 1.27 1.27))) (hide yes))
@@
   (property "Block" "blk.nfc-tag" (at 198.12 48.26 0) (effects (font (size 1.27 1.27))) (hide yes))
   (pin "1")
-  (instances (project "t1-main-board" (path "/7746052e-d7f9-59ad-ba73-bd2b74439529/338b6b86-006f-5bfa-ad71-6e8aca3fbcdb" (reference "TP6302") (unit 1))))
+  (instances (project "t1-main-board" (path "/7746052e-d7f9-59ad-ba73-bd2b74439529/338b6b86-006f-5bfa-ad71-6e8aca3fbcdb" (reference "TP6402") (unit 1))))
 )
 (junction (at 222.25 50.8) (diameter 0) (color 0 0 0 0))
@@
 )
 (symbol (lib_id "Connector:TestPoint") (at 168.91 81.28 0) (unit 1) (body_style 1) (exclude_from_sim no) (in_bom no) (on_board yes) (dnp no)
-  (property "Reference" "TP6303" (at 167.64 76.2 0) (effects (font (size 1.27 1.27)) (justify right)))
+  (property "Reference" "TP6403" (at 167.64 76.2 0) (effects (font (size 1.27 1.27)) (justify right)))
   (property "Value" "NFC_TAG_LA" (at 167.64 78.74 0) (effects (font (size 1.27 1.27)) (justify right)))
   (property "Footprint" "TestPoint:TestPoint_Pad_D1.0mm" (at 168.91 81.28 0) (effects (font (size 1.27 1.27))) (hide yes))
@@
   (property "Block" "blk.nfc-tag" (at 168.91 81.28 0) (effects (font (size 1.27 1.27))) (hide yes))
   (pin "1")
-  (instances (project "t1-main-board" (path "/7746052e-d7f9-59ad-ba73-bd2b74439529/338b6b86-006f-5bfa-ad71-6e8aca3fbcdb" (reference "TP6303") (unit 1))))
+  (instances (project "t1-main-board" (path "/7746052e-d7f9-59ad-ba73-bd2b74439529/338b6b86-006f-5bfa-ad71-6e8aca3fbcdb" (reference "TP6403") (unit 1))))
 )
 (symbol (lib_id "Connector:TestPoint") (at 186.69 81.28 0) (unit 1) (body_style 1) (exclude_from_sim no) (in_bom no) (on_board yes) (dnp no)
-  (property "Reference" "TP6304" (at 185.42 76.2 0) (effects (font (size 1.27 1.27)) (justify right)))
+  (property "Reference" "TP6404" (at 185.42 76.2 0) (effects (font (size 1.27 1.27)) (justify right)))
   (property "Value" "NFC_TAG_LB" (at 185.42 78.74 0) (effects (font (size 1.27 1.27)) (justify right)))
   (property "Footprint" "TestPoint:TestPoint_Pad_D1.0mm" (at 186.69 81.28 0) (effects (font (size 1.27 1.27))) (hide yes))
@@
   (property "Block" "blk.nfc-tag" (at 186.69 81.28 0) (effects (font (size 1.27 1.27))) (hide yes))
   (pin "1")
-  (instances (project "t1-main-board" (path "/7746052e-d7f9-59ad-ba73-bd2b74439529/338b6b86-006f-5bfa-ad71-6e8aca3fbcdb" (reference "TP6304") (unit 1))))
+  (instances (project "t1-main-board" (path "/7746052e-d7f9-59ad-ba73-bd2b74439529/338b6b86-006f-5bfa-ad71-6e8aca3fbcdb" (reference "TP6404") (unit 1))))
 )
 (rectangle (start 152.4 71.12) (end 245.11 97.79) (stroke (width 0) (type dash)) (fill (type none)))

Commit message: Compaction: lower inductors, 0201 decoupling, 0.8 mm signal test pads
A matrix tool (hardware/studies/compaction) checks each candidate against
the design's stresses: same inductance, design peak <= 70 % and the
converter's maximum limit <= 100 % of Isat (30 % drop), height zones,
ratings at least twice the rail, PCB-D-06; sourcing outcome per part.

Applied (placement v1 decision 12, BOM v1.15):
- L601, L4401: XGL4015-102MEC (1.5 mm) for XAL/XGL4020-102MEC (2.1 mm);
- L1001, L5101: XGL4015-471MEC (1.5 mm) for Wurth 744373240047, on the
  stock XxL4020 land (the Wurth land was never drawn);
- L1201 is 1.2 mm (XGL4012, per-MPN heights): it moves next to the SoC;
- 58 x 100 nF decoupling on rails <= 3.3 V in core/IO/radio: 0201;
- 51 test pads on signal nets: 0.8 mm (PCB-D-06 v0.16, JLCPCB guide).
Kept: L901, L2802 (XGL4015 at 103 % of Isat at the limit); no thinner
0805/1206 capacitor passes (obsolete, NRND or unlisted).

Board need 113 % -> 111 % (core band 227 -> 203 %, power band 258 ->
233 %, radio band 19 -> 0 %); only C904 still relies on PCB-Z-04.
ERC 0 errors, craft Q1 met, DRC 0 errors (605 warnings), pcb and study
tests pass, rules test board PASS.

Co-Authored-By: Claude Opus 5.5 <noreply@anthropic.com>
Claude-Session: https://claude.ai/code/session_01Ei262h3TpgY9vyfNLMi5Mn
Parts:
- C6401: footprint Capacitor_SMD:C_0402_1005Metric -> Capacitor_SMD:C_0201_0603Metric; MPN GRM155R71C104KA88D -> GRM033R61A104KE15D
Changed lines of the file:
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@@
   (property "Reference" "C6401" (at 81.28 57.15 0) (effects (font (size 1.27 1.27)) (justify left)))
   (property "Value" "100 nF" (at 81.28 59.69 0) (effects (font (size 1.27 1.27)) (justify left)))
-  (property "Footprint" "Capacitor_SMD:C_0402_1005Metric" (at 78.74 58.42 0) (effects (font (size 1.27 1.27))) (hide yes))
-  (property "Datasheet" "https://www.murata.com/en-us/products/productdetail?partno=GRM155R71C104KA88D" (at 78.74 58.42 0) (effects (font (size 1.27 1.27))) (hide yes))
-  (property "Description" "Capacitor, 100 nF, 16 V, X7R, 0402" (at 78.74 58.42 0) (effects (font (size 1.27 1.27))) (hide yes))
+  (property "Footprint" "Capacitor_SMD:C_0201_0603Metric" (at 78.74 58.42 0) (effects (font (size 1.27 1.27))) (hide yes))
+  (property "Datasheet" "https://www.murata.com/en-us/products/productdetail?partno=GRM033R61A104KE15D" (at 78.74 58.42 0) (effects (font (size 1.27 1.27))) (hide yes))
+  (property "Description" "Capacitor, 100 nF, 10 V, X5R, 0201" (at 78.74 58.42 0) (effects (font (size 1.27 1.27))) (hide yes))
   (property "Manufacturer" "Murata" (at 78.74 58.42 0) (effects (font (size 1.27 1.27))) (hide yes))
-  (property "MPN" "GRM155R71C104KA88D" (at 78.74 58.42 0) (effects (font (size 1.27 1.27))) (hide yes))
+  (property "MPN" "GRM033R61A104KE15D" (at 78.74 58.42 0) (effects (font (size 1.27 1.27))) (hide yes))
   (property "Block" "blk.nfc-tag" (at 78.74 58.42 0) (effects (font (size 1.27 1.27))) (hide yes))
   (pin "1")

Commit message: Board on libs v0.2.0: lower-case kebab vendor keys (HL-13)
The libs submodule moves to v0.2.0 (5f24483). Every library nickname in
the generator, the placement tool and the floorplan study follows the
key table (Texas_Instruments -> texas-instruments, OpenDAP_Device ->
opendap-generic, Rockchip and Rockchip_PMIC -> rockchip, ...); the
library tables are written from the files. Schematic and board
regenerated.

Checks: ERC 0 errors (warnings unchanged); DRC 0 errors, 605 warnings,
the same counts by type, schematic parity 0; every placement identical;
craft Q1 met; pcb tests pass; STEP export resolves every libs 3D model
(the 27 parts without a model are KiCad stock lands that have none).

Co-Authored-By: Claude Opus 5.5 <noreply@anthropic.com>
Claude-Session: https://claude.ai/code/session_01Ei262h3TpgY9vyfNLMi5Mn
Parts:
- U6401: footprint NXP:NXP_SOT902-3_XQFN-8_1.6x1.6mm_P0.5mm -> nxp:NXP_SOT902-3_XQFN-8_1.6x1.6mm_P0.5mm; symbol NXP:NT3H2111W0FHKH -> nxp:NT3H2111W0FHKH
Changed lines of the file:
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@@
 (paper "A4")
 (title_block (title "NFC tag") (date "2026-10-25") (rev "A") (company "The OpenDAP Project") (comment 1 "blk.nfc-tag") (comment 2 "NTAG I2C plus on I2C2 at 0x55, field detect and the loop antenna contacts"))
-(symbol (lib_id "NXP:NT3H2111W0FHKH") (at 50.8 72.39 0) (unit 1) (body_style 1) (exclude_from_sim no) (in_bom yes) (on_board yes) (dnp no)
+(symbol (lib_id "nxp:NT3H2111W0FHKH") (at 50.8 72.39 0) (unit 1) (body_style 1) (exclude_from_sim no) (in_bom yes) (on_board yes) (dnp no)
   (property "Reference" "U6401" (at 52.07 54.61 0) (effects (font (size 1.27 1.27)) (justify left)))
   (property "Value" "NT3H2111W0FHKH" (at 52.07 52.07 0) (effects (font (size 1.27 1.27)) (justify left)))
-  (property "Footprint" "NXP:NXP_SOT902-3_XQFN-8_1.6x1.6mm_P0.5mm" (at 50.8 72.39 0) (effects (font (size 1.27 1.27))) (hide yes))
+  (property "Footprint" "nxp:NXP_SOT902-3_XQFN-8_1.6x1.6mm_P0.5mm" (at 50.8 72.39 0) (effects (font (size 1.27 1.27))) (hide yes))
   (property "Datasheet" "https://www.nxp.com/docs/en/data-sheet/NT3H2111_2211.pdf" (at 50.8 72.39 0) (effects (font (size 1.27 1.27))) (hide yes))
   (property "Description" "NTAG I2C plus 1k: NFC Forum Type 2 Tag with I2C interface, field detection, energy harvesting, 1.67-3.6 V, XQFN8 (SOT902-3) 1.6 x 1.6 mm" (at 50.8 72.39 0) (effects (font (size 1.27 1.27))) (hide yes))
