File: board/hardware/t1-main-board/charger-battery.kicad_sch (KiCad schematic)
At the start: 14 parts, among them J701 70-9258-001-120-006, J702 70-9258-001-120-006, J703 70-9258-001-120-006, J704 70-9258-001-120-006, J705 70-9258-001-120-006, J706 70-9258-001-120-006, Q701 CSD17575Q3

Commit message: Board on libs v0.2.0: lower-case kebab vendor keys (HL-13)
The libs submodule moves to v0.2.0 (5f24483). Every library nickname in
the generator, the placement tool and the floorplan study follows the
key table (Texas_Instruments -> texas-instruments, OpenDAP_Device ->
opendap-generic, Rockchip and Rockchip_PMIC -> rockchip, ...); the
library tables are written from the files. Schematic and board
regenerated.

Checks: ERC 0 errors (warnings unchanged); DRC 0 errors, 605 warnings,
the same counts by type, schematic parity 0; every placement identical;
craft Q1 met; pcb tests pass; STEP export resolves every libs 3D model
(the 27 parts without a model are KiCad stock lands that have none).

Co-Authored-By: Claude Opus 5.5 <noreply@anthropic.com>
Claude-Session: https://claude.ai/code/session_01Ei262h3TpgY9vyfNLMi5Mn
Parts:
- J701, J702, J703, J704, J705, J706: footprint KYOCERA_AVX:KYOCERA_AVX_9258-100_70-9258-001-120-006_SpringFinger_Pad7.0x2.7mm -> kyocera-avx:KYOCERA_AVX_9258-100_70-9258-001-120-006_SpringFinger_Pad7.0x2.7mm; symbol KYOCERA_AVX:70-9258-001-120-006 -> kyocera-avx:70-9258-001-120-006
- Q701: footprint Texas_Instruments:Texas_Q3_SON-8_3.3x3.3mm_P0.65mm -> texas-instruments:Texas_Q3_SON-8_3.3x3.3mm_P0.65mm; symbol Texas_Instruments:CSD17575Q3 -> texas-instruments:CSD17575Q3
Changed lines of the file:
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@@
 (paper "A3")
 (title_block (title "Charger: battery path") (date "2026-10-25") (rev "A") (company "The OpenDAP Project") (comment 1 "blk.charger-battery") (comment 2 "Ship FET, 5 A fuse, BATP and the six battery contacts with their ESD"))
-(symbol (lib_id "Texas_Instruments:CSD17575Q3") (at 48.26 58.42 0) (unit 1) (body_style 1) (exclude_from_sim no) (in_bom yes) (on_board yes) (dnp no)
+(symbol (lib_id "texas-instruments:CSD17575Q3") (at 48.26 58.42 0) (unit 1) (body_style 1) (exclude_from_sim no) (in_bom yes) (on_board yes) (dnp no)
   (property "Reference" "Q701" (at 57.15 53.34 0) (effects (font (size 1.27 1.27)) (justify left)))
   (property "Value" "CSD17575Q3" (at 57.15 50.8 0) (effects (font (size 1.27 1.27)) (justify left)))
-  (property "Footprint" "Texas_Instruments:Texas_Q3_SON-8_3.3x3.3mm_P0.65mm" (at 48.26 58.42 0) (effects (font (size 1.27 1.27))) (hide yes))
+  (property "Footprint" "texas-instruments:Texas_Q3_SON-8_3.3x3.3mm_P0.65mm" (at 48.26 58.42 0) (effects (font (size 1.27 1.27))) (hide yes))
   (property "Datasheet" "https://www.ti.com/lit/ds/symlink/csd17575q3.pdf" (at 48.26 58.42 0) (effects (font (size 1.27 1.27))) (hide yes))
   (property "Description" "N-channel NexFET power MOSFET, 30 V, 1.9 / 2.6 mOhm at VGS 10 / 4.5 V, SON 3.3 x 3.3 mm (Q3)" (at 48.26 58.42 0) (effects (font (size 1.27 1.27))) (hide yes))
@@
 (rectangle (start 22.86 35.56) (end 215.9 81.28) (stroke (width 0) (type dash)) (fill (type none)))
 (text "Battery path: ship FET, 5 A fuse, BATP (ADR 0014 item 6, ADR 0017, ADR 0020 item 6)" (exclude_from_sim no) (at 24.13 34.29 0) (effects (font (size 2.54 2.54)) (justify left bottom)))
-(symbol (lib_id "KYOCERA_AVX:70-9258-001-120-006") (at 46.99 106.68 0) (unit 1) (body_style 1) (exclude_from_sim no) (in_bom yes) (on_board yes) (dnp no)
+(symbol (lib_id "kyocera-avx:70-9258-001-120-006") (at 46.99 106.68 0) (unit 1) (body_style 1) (exclude_from_sim no) (in_bom yes) (on_board yes) (dnp no)
   (property "Reference" "J701" (at 39.37 99.06 0) (effects (font (size 1.27 1.27)) (justify left)))
   (property "Value" "70-9258-001-120-006" (at 39.37 96.52 0) (effects (font (size 1.27 1.27)) (justify left)))
-  (property "Footprint" "KYOCERA_AVX:KYOCERA_AVX_9258-100_70-9258-001-120-006_SpringFinger_Pad7.0x2.7mm" (at 46.99 106.68 0) (effects (font (size 1.27 1.27))) (hide yes))
+  (property "Footprint" "kyocera-avx:KYOCERA_AVX_9258-100_70-9258-001-120-006_SpringFinger_Pad7.0x2.7mm" (at 46.99 106.68 0) (effects (font (size 1.27 1.27))) (hide yes))
   (property "Datasheet" "https://datasheets.kyocera-avx.com/9258-100.pdf" (at 46.99 106.68 0) (effects (font (size 1.27 1.27))) (hide yes))
   (property "Description" "Single-way SMT spring-finger compression contact, 6 A, 0.4 um gold, deflected height 1.6-2.8 mm (9258-100 type 120)" (at 46.99 106.68 0) (effects (font (size 1.27 1.27))) (hide yes))
@@
 )
 (wire (pts (xy 36.83 106.68) (xy 34.29 106.68)) (stroke (width 0) (type default)))
-(symbol (lib_id "KYOCERA_AVX:70-9258-001-120-006") (at 92.71 106.68 0) (unit 1) (body_style 1) (exclude_from_sim no) (in_bom yes) (on_board yes) (dnp no)
+(symbol (lib_id "kyocera-avx:70-9258-001-120-006") (at 92.71 106.68 0) (unit 1) (body_style 1) (exclude_from_sim no) (in_bom yes) (on_board yes) (dnp no)
   (property "Reference" "J702" (at 85.09 99.06 0) (effects (font (size 1.27 1.27)) (justify left)))
   (property "Value" "70-9258-001-120-006" (at 85.09 96.52 0) (effects (font (size 1.27 1.27)) (justify left)))
-  (property "Footprint" "KYOCERA_AVX:KYOCERA_AVX_9258-100_70-9258-001-120-006_SpringFinger_Pad7.0x2.7mm" (at 92.71 106.68 0) (effects (font (size 1.27 1.27))) (hide yes))
+  (property "Footprint" "kyocera-avx:KYOCERA_AVX_9258-100_70-9258-001-120-006_SpringFinger_Pad7.0x2.7mm" (at 92.71 106.68 0) (effects (font (size 1.27 1.27))) (hide yes))
   (property "Datasheet" "https://datasheets.kyocera-avx.com/9258-100.pdf" (at 92.71 106.68 0) (effects (font (size 1.27 1.27))) (hide yes))
   (property "Description" "Single-way SMT spring-finger compression contact, 6 A, 0.4 um gold, deflected height 1.6-2.8 mm (9258-100 type 120)" (at 92.71 106.68 0) (effects (font (size 1.27 1.27))) (hide yes))
@@
 )
 (wire (pts (xy 82.55 106.68) (xy 80.01 106.68)) (stroke (width 0) (type default)))
-(symbol (lib_id "KYOCERA_AVX:70-9258-001-120-006") (at 138.43 106.68 0) (unit 1) (body_style 1) (exclude_from_sim no) (in_bom yes) (on_board yes) (dnp no)
+(symbol (lib_id "kyocera-avx:70-9258-001-120-006") (at 138.43 106.68 0) (unit 1) (body_style 1) (exclude_from_sim no) (in_bom yes) (on_board yes) (dnp no)
   (property "Reference" "J703" (at 130.81 99.06 0) (effects (font (size 1.27 1.27)) (justify left)))
   (property "Value" "70-9258-001-120-006" (at 130.81 96.52 0) (effects (font (size 1.27 1.27)) (justify left)))
-  (property "Footprint" "KYOCERA_AVX:KYOCERA_AVX_9258-100_70-9258-001-120-006_SpringFinger_Pad7.0x2.7mm" (at 138.43 106.68 0) (effects (font (size 1.27 1.27))) (hide yes))
+  (property "Footprint" "kyocera-avx:KYOCERA_AVX_9258-100_70-9258-001-120-006_SpringFinger_Pad7.0x2.7mm" (at 138.43 106.68 0) (effects (font (size 1.27 1.27))) (hide yes))
   (property "Datasheet" "https://datasheets.kyocera-avx.com/9258-100.pdf" (at 138.43 106.68 0) (effects (font (size 1.27 1.27))) (hide yes))
   (property "Description" "Single-way SMT spring-finger compression contact, 6 A, 0.4 um gold, deflected height 1.6-2.8 mm (9258-100 type 120)" (at 138.43 106.68 0) (effects (font (size 1.27 1.27))) (hide yes))
@@
 )
 (wire (pts (xy 128.27 106.68) (xy 125.73 106.68)) (stroke (width 0) (type default)))
-(symbol (lib_id "KYOCERA_AVX:70-9258-001-120-006") (at 46.99 127 0) (unit 1) (body_style 1) (exclude_from_sim no) (in_bom yes) (on_board yes) (dnp no)
+(symbol (lib_id "kyocera-avx:70-9258-001-120-006") (at 46.99 127 0) (unit 1) (body_style 1) (exclude_from_sim no) (in_bom yes) (on_board yes) (dnp no)
   (property "Reference" "J704" (at 39.37 119.38 0) (effects (font (size 1.27 1.27)) (justify left)))
   (property "Value" "70-9258-001-120-006" (at 39.37 116.84 0) (effects (font (size 1.27 1.27)) (justify left)))
-  (property "Footprint" "KYOCERA_AVX:KYOCERA_AVX_9258-100_70-9258-001-120-006_SpringFinger_Pad7.0x2.7mm" (at 46.99 127 0) (effects (font (size 1.27 1.27))) (hide yes))
+  (property "Footprint" "kyocera-avx:KYOCERA_AVX_9258-100_70-9258-001-120-006_SpringFinger_Pad7.0x2.7mm" (at 46.99 127 0) (effects (font (size 1.27 1.27))) (hide yes))
   (property "Datasheet" "https://datasheets.kyocera-avx.com/9258-100.pdf" (at 46.99 127 0) (effects (font (size 1.27 1.27))) (hide yes))
   (property "Description" "Single-way SMT spring-finger compression contact, 6 A, 0.4 um gold, deflected height 1.6-2.8 mm (9258-100 type 120)" (at 46.99 127 0) (effects (font (size 1.27 1.27))) (hide yes))
@@
 )
 (wire (pts (xy 36.83 127) (xy 34.29 127)) (stroke (width 0) (type default)))
-(symbol (lib_id "KYOCERA_AVX:70-9258-001-120-006") (at 92.71 127 0) (unit 1) (body_style 1) (exclude_from_sim no) (in_bom yes) (on_board yes) (dnp no)
+(symbol (lib_id "kyocera-avx:70-9258-001-120-006") (at 92.71 127 0) (unit 1) (body_style 1) (exclude_from_sim no) (in_bom yes) (on_board yes) (dnp no)
   (property "Reference" "J705" (at 85.09 119.38 0) (effects (font (size 1.27 1.27)) (justify left)))
   (property "Value" "70-9258-001-120-006" (at 85.09 116.84 0) (effects (font (size 1.27 1.27)) (justify left)))
-  (property "Footprint" "KYOCERA_AVX:KYOCERA_AVX_9258-100_70-9258-001-120-006_SpringFinger_Pad7.0x2.7mm" (at 92.71 127 0) (effects (font (size 1.27 1.27))) (hide yes))
+  (property "Footprint" "kyocera-avx:KYOCERA_AVX_9258-100_70-9258-001-120-006_SpringFinger_Pad7.0x2.7mm" (at 92.71 127 0) (effects (font (size 1.27 1.27))) (hide yes))
   (property "Datasheet" "https://datasheets.kyocera-avx.com/9258-100.pdf" (at 92.71 127 0) (effects (font (size 1.27 1.27))) (hide yes))
   (property "Description" "Single-way SMT spring-finger compression contact, 6 A, 0.4 um gold, deflected height 1.6-2.8 mm (9258-100 type 120)" (at 92.71 127 0) (effects (font (size 1.27 1.27))) (hide yes))
@@
   (instances (project "t1-main-board" (path "/7746052e-d7f9-59ad-ba73-bd2b74439529/4dc73b6d-736f-5398-a907-27e20ed1a3e6/ca568731-87ea-5ff9-adf5-a3b161dd236c" (reference "#PWR0054") (unit 1))))
 )
-(symbol (lib_id "KYOCERA_AVX:70-9258-001-120-006") (at 138.43 127 0) (unit 1) (body_style 1) (exclude_from_sim no) (in_bom yes) (on_board yes) (dnp no)
+(symbol (lib_id "kyocera-avx:70-9258-001-120-006") (at 138.43 127 0) (unit 1) (body_style 1) (exclude_from_sim no) (in_bom yes) (on_board yes) (dnp no)
   (property "Reference" "J706" (at 130.81 119.38 0) (effects (font (size 1.27 1.27)) (justify left)))
   (property "Value" "70-9258-001-120-006" (at 130.81 116.84 0) (effects (font (size 1.27 1.27)) (justify left)))
-  (property "Footprint" "KYOCERA_AVX:KYOCERA_AVX_9258-100_70-9258-001-120-006_SpringFinger_Pad7.0x2.7mm" (at 138.43 127 0) (effects (font (size 1.27 1.27))) (hide yes))
+  (property "Footprint" "kyocera-avx:KYOCERA_AVX_9258-100_70-9258-001-120-006_SpringFinger_Pad7.0x2.7mm" (at 138.43 127 0) (effects (font (size 1.27 1.27))) (hide yes))
   (property "Datasheet" "https://datasheets.kyocera-avx.com/9258-100.pdf" (at 138.43 127 0) (effects (font (size 1.27 1.27))) (hide yes))
   (property "Description" "Single-way SMT spring-finger compression contact, 6 A, 0.4 um gold, deflected height 1.6-2.8 mm (9258-100 type 120)" (at 138.43 127 0) (effects (font (size 1.27 1.27))) (hide yes))

Commit message: Board in the 62.5 x 95.0 mm body: ADR 0025, outline 59.1 x 91.6, 0201 swaps
ADR 0025 supersedes ADR 0016 for t1 ADR 0006's body: board outline from
the body, 1.2 mm walls and 0.5 mm clearance; height zones and stack
restated unchanged; the speaker on a case shelf (PCB-Z-09); pocket
reliefs at the 4.4 mm jack, the microSD (DM3AT push-push kept) and the
side buttons; the audio 0603 -> 0402 swap gated by t1 V2-A08; reserve
(NFC reader, then TPM) recorded, not applied.

- pcb/geometry.py derives the outline from BODY, WALL and CLEARANCE;
  the pocket, display and fixed parts keep their device-frame positions;
  holes keep their edge distance; the speaker shadow becomes a 1.5 mm
  shelf height area (placement, checks, occupancy).
- build.py reports pocket reliefs and routing room; C904 unfixed (it
  now finds back room, so PCB-Z-04 carries no part).
- Generator: parts.area_swap puts 121 generic 0402 resistors (outside
  audio and VBUS paths, >= 10 ohm) and five 100 nF signal capacitors in
  0201 (BOM v1.16); schematic and board regenerated.
- Result: 1,012/1,012 placed, 98.8 % by the floorplan method (was 111 %),
  factor left 1.68 (was 1.49); DRC 0 errors, ERC 0 errors, 0 check
  findings, pcb tests 20/20, schematic craft Q1 met.
- Specs: PCB constraints v0.17 (M-01, M-02, M-08, Z-02, Z-06 to Z-09,
  R-07), placement v1.1 (section 3, decisions 4 and 13, checks, open
  items with the gated swaps and the reserve), floorplan v1 section 1,
  BOM v1.16.

Co-Authored-By: Claude Opus 5.5 <noreply@anthropic.com>
Claude-Session: https://claude.ai/code/session_01Ei262h3TpgY9vyfNLMi5Mn
Parts:
- R701: footprint Resistor_SMD:R_0402_1005Metric -> Resistor_SMD:R_0201_0603Metric; MPN RC0402FR-07100RL -> RC0201FR-07100RL
Changed lines of the file:
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@@
   (property "Reference" "R701" (at 97.79 71.12 90) (effects (font (size 1.27 1.27))))
   (property "Value" "100 Ω" (at 97.79 76.2 90) (effects (font (size 1.27 1.27))))
-  (property "Footprint" "Resistor_SMD:R_0402_1005Metric" (at 97.79 73.66 0) (effects (font (size 1.27 1.27))) (hide yes))
-  (property "Datasheet" "https://yageogroup.com/en/ProductSearch/PartNumberSearch?part=RC0402FR-07100RL" (at 97.79 73.66 0) (effects (font (size 1.27 1.27))) (hide yes))
-  (property "Description" "Resistor, 100 Ω, 1 %, 1/16 W, 0402" (at 97.79 73.66 0) (effects (font (size 1.27 1.27))) (hide yes))
+  (property "Footprint" "Resistor_SMD:R_0201_0603Metric" (at 97.79 73.66 0) (effects (font (size 1.27 1.27))) (hide yes))
+  (property "Datasheet" "https://yageogroup.com/en/ProductSearch/PartNumberSearch?part=RC0201FR-07100RL" (at 97.79 73.66 0) (effects (font (size 1.27 1.27))) (hide yes))
+  (property "Description" "Resistor, 100 Ω, 1 %, 1/20 W, 0201" (at 97.79 73.66 0) (effects (font (size 1.27 1.27))) (hide yes))
   (property "Manufacturer" "YAGEO" (at 97.79 73.66 0) (effects (font (size 1.27 1.27))) (hide yes))
-  (property "MPN" "RC0402FR-07100RL" (at 97.79 73.66 0) (effects (font (size 1.27 1.27))) (hide yes))
+  (property "MPN" "RC0201FR-07100RL" (at 97.79 73.66 0) (effects (font (size 1.27 1.27))) (hide yes))
   (property "Block" "blk.charger-battery" (at 97.79 73.66 0) (effects (font (size 1.27 1.27))) (hide yes))
   (pin "1")
