File: board/hardware/t1-main-board/tpm.kicad_sch (KiCad schematic)
At the start: 9 parts, among them U6301 SLB9673XU20FW2613XTMA1

Commit message: Board: capture blk.current-monitors
Five INA236 on I2C1 (0x40-0x43, 0x48) with their shunts, per power tree
§4.12 and BOM v1 lines 54 and 136. The measured branches are rails of
their own (VSYS_SRC, VSYS_LV_AUDIO, VSYS_AUDIO, VSYS_LV_BL, VSYS_P5V1),
fed through the shunts on this sheet; the charger, audio, backlight and
5.1 V sheets take them. The root's layout may leave a stack level empty,
so the block sits under the notes; IC bboxes hold turned rail values;
passive rows hold a bottom rail's text.

Co-Authored-By: Claude Opus 5.5 <noreply@anthropic.com>
Claude-Session: https://claude.ai/code/session_01Ei262h3TpgY9vyfNLMi5Mn
Parts:
- removed C6301: 1 µF, Capacitor_SMD:C_0402_1005Metric, symbol Device:C
- removed C6302, C6303, C6304: 100 nF, Capacitor_SMD:C_0402_1005Metric, symbol Device:C
- removed R6301: 2.2 kΩ, Resistor_SMD:R_0402_1005Metric, symbol Device:R
- removed R6302: 100 mΩ, Resistor_SMD:R_0603_1608Metric, symbol Device:R
- removed TP6301: vcca1v8_pmu, TestPoint:TestPoint_Pad_D1.0mm, symbol Connector:TestPoint
- removed TP6302: TPM_VDD, TestPoint:TestPoint_Pad_D1.0mm, symbol Connector:TestPoint
- removed U6301: SLB9673XU20FW2613XTMA1, Infineon:Infineon_PG-UQFN-32-1_5x5mm_P0.5mm_EP3.6x3.6mm, symbol Infineon:SLB9673XU20FW2613XTMA1
- added C6401: 1 µF, Capacitor_SMD:C_0402_1005Metric, symbol Device:C
- added C6402, C6403, C6404: 100 nF, Capacitor_SMD:C_0402_1005Metric, symbol Device:C
- added R6401: 2.2 kΩ, Resistor_SMD:R_0402_1005Metric, symbol Device:R
- added R6402: 100 mΩ, Resistor_SMD:R_0603_1608Metric, symbol Device:R
- added TP6401: vcca1v8_pmu, TestPoint:TestPoint_Pad_D1.0mm, symbol Connector:TestPoint
- added TP6402: TPM_VDD, TestPoint:TestPoint_Pad_D1.0mm, symbol Connector:TestPoint
- added U6401: SLB9673XU20FW2613XTMA1, Infineon:Infineon_PG-UQFN-32-1_5x5mm_P0.5mm_EP3.6x3.6mm, symbol Infineon:SLB9673XU20FW2613XTMA1
Connections:
- net GND: now also C6401.2, C6402.2, C6403.2, C6404.2, U6401.16 (NCI/GND), U6401.2 (GND), U6401.23 (GND), U6401.32 (GND), U6401.9 (GND), U6401.EP
- net I2C2_SCL: now also U6401.30 (SCL)
- net I2C2_SDA: now also U6401.29 (SDA)
- net TPM_PIRQ_N: now also U6401.18 (I2C_PIRQ#)
- net TPM_RST_N: now also R6401.2, U6401.17 (RST#)
- net TPM_VDD: now also C6401.1, C6402.1, C6403.1, C6404.1, R6401.1, R6402.2, TP6402.1, U6401.1 (VDD), U6401.14 (VDD), U6401.20 (TEST#), U6401.22 (VDD), U6401.8 (NCI/VDD)
- net vcca1v8_pmu: now also R6402.1, TP6401.1
Changed lines of the file:
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@@
 (title_block (title "Hardware key holder") (date "2026-10-25") (rev "A") (company "The OpenDAP Project") (comment 1 "blk.tpm") (comment 2 "SLB9673 TPM 2.0 on I2C2 at 0x2E, always on"))
 (symbol (lib_id "Infineon:SLB9673XU20FW2613XTMA1") (at 69.85 87.63 0) (unit 1) (body_style 1) (exclude_from_sim no) (in_bom yes) (on_board yes) (dnp no)
-  (property "Reference" "U6301" (at 76.2 50.8 0) (effects (font (size 1.27 1.27)) (justify left)))
+  (property "Reference" "U6401" (at 76.2 50.8 0) (effects (font (size 1.27 1.27)) (justify left)))
   (property "Value" "SLB9673XU20FW2613XTMA1" (at 76.2 48.26 0) (effects (font (size 1.27 1.27)) (justify left)))
   (property "Footprint" "Infineon:Infineon_PG-UQFN-32-1_5x5mm_P0.5mm_EP3.6x3.6mm" (at 69.85 87.63 0) (effects (font (size 1.27 1.27))) (hide yes))
@@
   (pin "16")
   (pin "EP")
-  (instances (project "t1-main-board" (path "/7746052e-d7f9-59ad-ba73-bd2b74439529/53ee74be-bcd0-540e-90f4-0921f22107a2" (reference "U6301") (unit 1))))
+  (instances (project "t1-main-board" (path "/7746052e-d7f9-59ad-ba73-bd2b74439529/53ee74be-bcd0-540e-90f4-0921f22107a2" (reference "U6401") (unit 1))))
 )
 (wire (pts (xy 64.77 49.53) (xy 64.77 46.99)) (stroke (width 0) (type default)))
@@
 (no_connect (at 85.09 100.33))
 (symbol (lib_id "Device:C") (at 114.3 53.34 0) (unit 1) (body_style 1) (exclude_from_sim no) (in_bom yes) (on_board yes) (dnp no)
-  (property "Reference" "C6301" (at 116.84 52.07 0) (effects (font (size 1.27 1.27)) (justify left)))
+  (property "Reference" "C6401" (at 116.84 52.07 0) (effects (font (size 1.27 1.27)) (justify left)))
   (property "Value" "1 µF" (at 116.84 54.61 0) (effects (font (size 1.27 1.27)) (justify left)))
   (property "Footprint" "Capacitor_SMD:C_0402_1005Metric" (at 114.3 53.34 0) (effects (font (size 1.27 1.27))) (hide yes))
@@
   (pin "1")
   (pin "2")
-  (instances (project "t1-main-board" (path "/7746052e-d7f9-59ad-ba73-bd2b74439529/53ee74be-bcd0-540e-90f4-0921f22107a2" (reference "C6301") (unit 1))))
+  (instances (project "t1-main-board" (path "/7746052e-d7f9-59ad-ba73-bd2b74439529/53ee74be-bcd0-540e-90f4-0921f22107a2" (reference "C6401") (unit 1))))
 )
 (wire (pts (xy 114.3 49.53) (xy 114.3 46.99)) (stroke (width 0) (type default)))
@@
 )
 (symbol (lib_id "Device:C") (at 127 53.34 0) (unit 1) (body_style 1) (exclude_from_sim no) (in_bom yes) (on_board yes) (dnp no)
-  (property "Reference" "C6302" (at 129.54 52.07 0) (effects (font (size 1.27 1.27)) (justify left)))
+  (property "Reference" "C6402" (at 129.54 52.07 0) (effects (font (size 1.27 1.27)) (justify left)))
   (property "Value" "100 nF" (at 129.54 54.61 0) (effects (font (size 1.27 1.27)) (justify left)))
   (property "Footprint" "Capacitor_SMD:C_0402_1005Metric" (at 127 53.34 0) (effects (font (size 1.27 1.27))) (hide yes))
@@
   (pin "1")
   (pin "2")
-  (instances (project "t1-main-board" (path "/7746052e-d7f9-59ad-ba73-bd2b74439529/53ee74be-bcd0-540e-90f4-0921f22107a2" (reference "C6302") (unit 1))))
+  (instances (project "t1-main-board" (path "/7746052e-d7f9-59ad-ba73-bd2b74439529/53ee74be-bcd0-540e-90f4-0921f22107a2" (reference "C6402") (unit 1))))
 )
 (wire (pts (xy 127 49.53) (xy 127 46.99)) (stroke (width 0) (type default)))
@@
 )
 (symbol (lib_id "Device:C") (at 140.97 53.34 0) (unit 1) (body_style 1) (exclude_from_sim no) (in_bom yes) (on_board yes) (dnp no)
-  (property "Reference" "C6303" (at 143.51 52.07 0) (effects (font (size 1.27 1.27)) (justify left)))
+  (property "Reference" "C6403" (at 143.51 52.07 0) (effects (font (size 1.27 1.27)) (justify left)))
   (property "Value" "100 nF" (at 143.51 54.61 0) (effects (font (size 1.27 1.27)) (justify left)))
   (property "Footprint" "Capacitor_SMD:C_0402_1005Metric" (at 140.97 53.34 0) (effects (font (size 1.27 1.27))) (hide yes))
@@
   (pin "1")
   (pin "2")
-  (instances (project "t1-main-board" (path "/7746052e-d7f9-59ad-ba73-bd2b74439529/53ee74be-bcd0-540e-90f4-0921f22107a2" (reference "C6303") (unit 1))))
+  (instances (project "t1-main-board" (path "/7746052e-d7f9-59ad-ba73-bd2b74439529/53ee74be-bcd0-540e-90f4-0921f22107a2" (reference "C6403") (unit 1))))
 )
 (wire (pts (xy 140.97 49.53) (xy 140.97 46.99)) (stroke (width 0) (type default)))
@@
 )
 (symbol (lib_id "Device:C") (at 154.94 53.34 0) (unit 1) (body_style 1) (exclude_from_sim no) (in_bom yes) (on_board yes) (dnp no)
-  (property "Reference" "C6304" (at 157.48 52.07 0) (effects (font (size 1.27 1.27)) (justify left)))
+  (property "Reference" "C6404" (at 157.48 52.07 0) (effects (font (size 1.27 1.27)) (justify left)))
   (property "Value" "100 nF" (at 157.48 54.61 0) (effects (font (size 1.27 1.27)) (justify left)))
   (property "Footprint" "Capacitor_SMD:C_0402_1005Metric" (at 154.94 53.34 0) (effects (font (size 1.27 1.27))) (hide yes))
@@
   (pin "1")
   (pin "2")
-  (instances (project "t1-main-board" (path "/7746052e-d7f9-59ad-ba73-bd2b74439529/53ee74be-bcd0-540e-90f4-0921f22107a2" (reference "C6304") (unit 1))))
+  (instances (project "t1-main-board" (path "/7746052e-d7f9-59ad-ba73-bd2b74439529/53ee74be-bcd0-540e-90f4-0921f22107a2" (reference "C6404") (unit 1))))
 )
 (wire (pts (xy 154.94 49.53) (xy 154.94 46.99)) (stroke (width 0) (type default)))
@@
 )
 (symbol (lib_id "Device:R") (at 114.3 83.82 0) (unit 1) (body_style 1) (exclude_from_sim no) (in_bom yes) (on_board yes) (dnp no)
-  (property "Reference" "R6301" (at 115.57 82.55 0) (effects (font (size 1.27 1.27)) (justify left)))
+  (property "Reference" "R6401" (at 115.57 82.55 0) (effects (font (size 1.27 1.27)) (justify left)))
   (property "Value" "2.2 kΩ" (at 115.57 85.09 0) (effects (font (size 1.27 1.27)) (justify left)))
   (property "Footprint" "Resistor_SMD:R_0402_1005Metric" (at 114.3 83.82 0) (effects (font (size 1.27 1.27))) (hide yes))
@@
   (pin "1")
   (pin "2")
-  (instances (project "t1-main-board" (path "/7746052e-d7f9-59ad-ba73-bd2b74439529/53ee74be-bcd0-540e-90f4-0921f22107a2" (reference "R6301") (unit 1))))
+  (instances (project "t1-main-board" (path "/7746052e-d7f9-59ad-ba73-bd2b74439529/53ee74be-bcd0-540e-90f4-0921f22107a2" (reference "R6401") (unit 1))))
 )
 (wire (pts (xy 114.3 80.01) (xy 114.3 77.47)) (stroke (width 0) (type default)))
@@
 (text "SLB9673 TPM 2.0 at I2C2 0x2E (BOM v1 line 122)" (exclude_from_sim no) (at 24.13 34.29 0) (effects (font (size 2.54 2.54)) (justify left bottom)))
 (symbol (lib_id "Device:R") (at 213.36 50.8 90) (unit 1) (body_style 1) (exclude_from_sim no) (in_bom yes) (on_board yes) (dnp no)
-  (property "Reference" "R6302" (at 210.82 46.99 90) (effects (font (size 1.27 1.27))))
+  (property "Reference" "R6402" (at 210.82 46.99 90) (effects (font (size 1.27 1.27))))
   (property "Value" "100 mΩ" (at 210.82 53.34 90) (effects (font (size 1.27 1.27))))
   (property "Spec" "0603" (at 210.82 55.88 90) (effects (font (size 1.27 1.27))))
@@
   (pin "1")
   (pin "2")
-  (instances (project "t1-main-board" (path "/7746052e-d7f9-59ad-ba73-bd2b74439529/53ee74be-bcd0-540e-90f4-0921f22107a2" (reference "R6302") (unit 1) (variant (name "production") (field (name "Value") (value "0 Ω")) (field (name "MPN") (value "RC0603JR-070RL")) (field (name "Manufacturer") (value "YAGEO"))))))
+  (instances (project "t1-main-board" (path "/7746052e-d7f9-59ad-ba73-bd2b74439529/53ee74be-bcd0-540e-90f4-0921f22107a2" (reference "R6402") (unit 1) (variant (name "production") (field (name "Value") (value "0 Ω")) (field (name "MPN") (value "RC0603JR-070RL")) (field (name "Manufacturer") (value "YAGEO"))))))
 )
 (rectangle (start 190.5 38.1) (end 231.14 58.42) (stroke (width 0) (type dash)) (fill (type none)))
@@
 (wire (pts (xy 207.01 50.8) (xy 207.01 48.26)) (stroke (width 0) (type default)))
 (symbol (lib_id "Connector:TestPoint") (at 207.01 48.26 0) (unit 1) (body_style 1) (exclude_from_sim no) (in_bom no) (on_board yes) (dnp no)
-  (property "Reference" "TP6301" (at 205.74 43.18 0) (effects (font (size 1.27 1.27)) (justify right)))
+  (property "Reference" "TP6401" (at 205.74 43.18 0) (effects (font (size 1.27 1.27)) (justify right)))
   (property "Value" "vcca1v8_pmu" (at 205.74 45.72 0) (effects (font (size 1.27 1.27)) (justify right)))
   (property "Footprint" "TestPoint:TestPoint_Pad_D1.0mm" (at 207.01 48.26 0) (effects (font (size 1.27 1.27))) (hide yes))
@@
   (property "Block" "blk.tpm" (at 207.01 48.26 0) (effects (font (size 1.27 1.27))) (hide yes))
   (pin "1")
-  (instances (project "t1-main-board" (path "/7746052e-d7f9-59ad-ba73-bd2b74439529/53ee74be-bcd0-540e-90f4-0921f22107a2" (reference "TP6301") (unit 1))))
+  (instances (project "t1-main-board" (path "/7746052e-d7f9-59ad-ba73-bd2b74439529/53ee74be-bcd0-540e-90f4-0921f22107a2" (reference "TP6401") (unit 1))))
 )
 (symbol (lib_id "power:VCC") (at 187.96 50.8 90) (unit 1) (body_style 1) (exclude_from_sim no) (in_bom yes) (on_board yes) (dnp no)
@@
 (wire (pts (xy 219.71 50.8) (xy 219.71 48.26)) (stroke (width 0) (type default)))
 (symbol (lib_id "Connector:TestPoint") (at 219.71 48.26 0) (unit 1) (body_style 1) (exclude_from_sim no) (in_bom no) (on_board yes) (dnp no)
-  (property "Reference" "TP6302" (at 220.98 43.18 0) (effects (font (size 1.27 1.27)) (justify left)))
+  (property "Reference" "TP6402" (at 220.98 43.18 0) (effects (font (size 1.27 1.27)) (justify left)))
   (property "Value" "TPM_VDD" (at 220.98 45.72 0) (effects (font (size 1.27 1.27)) (justify left)))
   (property "Footprint" "TestPoint:TestPoint_Pad_D1.0mm" (at 219.71 48.26 0) (effects (font (size 1.27 1.27))) (hide yes))
@@
   (property "Block" "blk.tpm" (at 219.71 48.26 0) (effects (font (size 1.27 1.27))) (hide yes))
   (pin "1")
-  (instances (project "t1-main-board" (path "/7746052e-d7f9-59ad-ba73-bd2b74439529/53ee74be-bcd0-540e-90f4-0921f22107a2" (reference "TP6302") (unit 1))))
+  (instances (project "t1-main-board" (path "/7746052e-d7f9-59ad-ba73-bd2b74439529/53ee74be-bcd0-540e-90f4-0921f22107a2" (reference "TP6402") (unit 1))))
 )
 (junction (at 238.76 50.8) (diameter 0) (color 0 0 0 0))
