File: board/hardware/t1-main-board/tpm.kicad_sch (KiCad schematic)
At the start: 9 parts, among them U5401 SLB9673XU20FW2613XTMA1

Commit message: Board: capture blk.debug
Debug UART2 (1.8 V) and I2S/DSD pads with ground pads, reset, PMIC and
power-key pads (PCB-T-09), a pad on every spare SoC GPIO whose pinout v1
row names one (the DEBUG bus, on the SoC's right edge), and a rail pad
for each power-tree rail no other sheet probes (PCB-T-02). Each DAC
sheet carries a pad on its MCLK. The spares pinout v1 leaves without a
pad now carry no-connect flags. On the root, facing sheet pins are
joined directly only where the route meets no other symbol.

Co-Authored-By: Claude Opus 5.5 <noreply@anthropic.com>
Claude-Session: https://claude.ai/code/session_01Ei262h3TpgY9vyfNLMi5Mn
Parts:
- removed C5401: 1 µF, Capacitor_SMD:C_0402_1005Metric, symbol Device:C
- removed C5402, C5403, C5404: 100 nF, Capacitor_SMD:C_0402_1005Metric, symbol Device:C
- removed R5401: 2.2 kΩ, Resistor_SMD:R_0402_1005Metric, symbol Device:R
- removed R5402: 100 mΩ, Resistor_SMD:R_0603_1608Metric, symbol Device:R
- removed TP5401: vcca1v8_pmu, TestPoint:TestPoint_Pad_D1.0mm, symbol Connector:TestPoint
- removed TP5402: TPM_VDD, TestPoint:TestPoint_Pad_D1.0mm, symbol Connector:TestPoint
- removed U5401: SLB9673XU20FW2613XTMA1, Infineon:Infineon_PG-UQFN-32-1_5x5mm_P0.5mm_EP3.6x3.6mm, symbol Infineon:SLB9673XU20FW2613XTMA1
- added C5501: 1 µF, Capacitor_SMD:C_0402_1005Metric, symbol Device:C
- added C5502, C5503, C5504: 100 nF, Capacitor_SMD:C_0402_1005Metric, symbol Device:C
- added R5501: 2.2 kΩ, Resistor_SMD:R_0402_1005Metric, symbol Device:R
- added R5502: 100 mΩ, Resistor_SMD:R_0603_1608Metric, symbol Device:R
- added TP5501: vcca1v8_pmu, TestPoint:TestPoint_Pad_D1.0mm, symbol Connector:TestPoint
- added TP5502: TPM_VDD, TestPoint:TestPoint_Pad_D1.0mm, symbol Connector:TestPoint
- added U5501: SLB9673XU20FW2613XTMA1, Infineon:Infineon_PG-UQFN-32-1_5x5mm_P0.5mm_EP3.6x3.6mm, symbol Infineon:SLB9673XU20FW2613XTMA1
Connections:
- net GND: now also C5501.2, C5502.2, C5503.2, C5504.2, U5501.16 (NCI/GND), U5501.2 (GND), U5501.23 (GND), U5501.32 (GND), U5501.9 (GND), U5501.EP
- net I2C2_SCL: now also U5501.30 (SCL)
- net I2C2_SDA: now also U5501.29 (SDA)
- net TPM_PIRQ_N: now also U5501.18 (I2C_PIRQ#)
- net TPM_RST_N: now also R5501.2, U5501.17 (RST#)
- net TPM_VDD: now also C5501.1, C5502.1, C5503.1, C5504.1, R5501.1, R5502.2, TP5502.1, U5501.1 (VDD), U5501.14 (VDD), U5501.20 (TEST#), U5501.22 (VDD), U5501.8 (NCI/VDD)
- net vcca1v8_pmu: now also R5502.1, TP5501.1
Changed lines of the file:
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@@
 (title_block (title "Hardware key holder") (date "2026-10-25") (rev "A") (company "The OpenDAP Project") (comment 1 "blk.tpm") (comment 2 "SLB9673 TPM 2.0 on I2C2 at 0x2E, always on"))
 (symbol (lib_id "Infineon:SLB9673XU20FW2613XTMA1") (at 69.85 87.63 0) (unit 1) (body_style 1) (exclude_from_sim no) (in_bom yes) (on_board yes) (dnp no)
-  (property "Reference" "U5401" (at 76.2 50.8 0) (effects (font (size 1.27 1.27)) (justify left)))
+  (property "Reference" "U5501" (at 76.2 50.8 0) (effects (font (size 1.27 1.27)) (justify left)))
   (property "Value" "SLB9673XU20FW2613XTMA1" (at 76.2 48.26 0) (effects (font (size 1.27 1.27)) (justify left)))
   (property "Footprint" "Infineon:Infineon_PG-UQFN-32-1_5x5mm_P0.5mm_EP3.6x3.6mm" (at 69.85 87.63 0) (effects (font (size 1.27 1.27))) (hide yes))
@@
   (pin "16")
   (pin "EP")
-  (instances (project "t1-main-board" (path "/7746052e-d7f9-59ad-ba73-bd2b74439529/53ee74be-bcd0-540e-90f4-0921f22107a2" (reference "U5401") (unit 1))))
+  (instances (project "t1-main-board" (path "/7746052e-d7f9-59ad-ba73-bd2b74439529/53ee74be-bcd0-540e-90f4-0921f22107a2" (reference "U5501") (unit 1))))
 )
 (wire (pts (xy 64.77 49.53) (xy 64.77 46.99)) (stroke (width 0) (type default)))
@@
 (no_connect (at 85.09 100.33))
 (symbol (lib_id "Device:C") (at 114.3 53.34 0) (unit 1) (body_style 1) (exclude_from_sim no) (in_bom yes) (on_board yes) (dnp no)
-  (property "Reference" "C5401" (at 116.84 52.07 0) (effects (font (size 1.27 1.27)) (justify left)))
+  (property "Reference" "C5501" (at 116.84 52.07 0) (effects (font (size 1.27 1.27)) (justify left)))
   (property "Value" "1 µF" (at 116.84 54.61 0) (effects (font (size 1.27 1.27)) (justify left)))
   (property "Footprint" "Capacitor_SMD:C_0402_1005Metric" (at 114.3 53.34 0) (effects (font (size 1.27 1.27))) (hide yes))
@@
   (pin "1")
   (pin "2")
-  (instances (project "t1-main-board" (path "/7746052e-d7f9-59ad-ba73-bd2b74439529/53ee74be-bcd0-540e-90f4-0921f22107a2" (reference "C5401") (unit 1))))
+  (instances (project "t1-main-board" (path "/7746052e-d7f9-59ad-ba73-bd2b74439529/53ee74be-bcd0-540e-90f4-0921f22107a2" (reference "C5501") (unit 1))))
 )
 (wire (pts (xy 114.3 49.53) (xy 114.3 46.99)) (stroke (width 0) (type default)))
@@
 )
 (symbol (lib_id "Device:C") (at 127 53.34 0) (unit 1) (body_style 1) (exclude_from_sim no) (in_bom yes) (on_board yes) (dnp no)
-  (property "Reference" "C5402" (at 129.54 52.07 0) (effects (font (size 1.27 1.27)) (justify left)))
+  (property "Reference" "C5502" (at 129.54 52.07 0) (effects (font (size 1.27 1.27)) (justify left)))
   (property "Value" "100 nF" (at 129.54 54.61 0) (effects (font (size 1.27 1.27)) (justify left)))
   (property "Footprint" "Capacitor_SMD:C_0402_1005Metric" (at 127 53.34 0) (effects (font (size 1.27 1.27))) (hide yes))
@@
   (pin "1")
   (pin "2")
-  (instances (project "t1-main-board" (path "/7746052e-d7f9-59ad-ba73-bd2b74439529/53ee74be-bcd0-540e-90f4-0921f22107a2" (reference "C5402") (unit 1))))
+  (instances (project "t1-main-board" (path "/7746052e-d7f9-59ad-ba73-bd2b74439529/53ee74be-bcd0-540e-90f4-0921f22107a2" (reference "C5502") (unit 1))))
 )
 (wire (pts (xy 127 49.53) (xy 127 46.99)) (stroke (width 0) (type default)))
@@
 )
 (symbol (lib_id "Device:C") (at 140.97 53.34 0) (unit 1) (body_style 1) (exclude_from_sim no) (in_bom yes) (on_board yes) (dnp no)
-  (property "Reference" "C5403" (at 143.51 52.07 0) (effects (font (size 1.27 1.27)) (justify left)))
+  (property "Reference" "C5503" (at 143.51 52.07 0) (effects (font (size 1.27 1.27)) (justify left)))
   (property "Value" "100 nF" (at 143.51 54.61 0) (effects (font (size 1.27 1.27)) (justify left)))
   (property "Footprint" "Capacitor_SMD:C_0402_1005Metric" (at 140.97 53.34 0) (effects (font (size 1.27 1.27))) (hide yes))
@@
   (pin "1")
   (pin "2")
-  (instances (project "t1-main-board" (path "/7746052e-d7f9-59ad-ba73-bd2b74439529/53ee74be-bcd0-540e-90f4-0921f22107a2" (reference "C5403") (unit 1))))
+  (instances (project "t1-main-board" (path "/7746052e-d7f9-59ad-ba73-bd2b74439529/53ee74be-bcd0-540e-90f4-0921f22107a2" (reference "C5503") (unit 1))))
 )
 (wire (pts (xy 140.97 49.53) (xy 140.97 46.99)) (stroke (width 0) (type default)))
@@
 )
 (symbol (lib_id "Device:C") (at 154.94 53.34 0) (unit 1) (body_style 1) (exclude_from_sim no) (in_bom yes) (on_board yes) (dnp no)
-  (property "Reference" "C5404" (at 157.48 52.07 0) (effects (font (size 1.27 1.27)) (justify left)))
+  (property "Reference" "C5504" (at 157.48 52.07 0) (effects (font (size 1.27 1.27)) (justify left)))
   (property "Value" "100 nF" (at 157.48 54.61 0) (effects (font (size 1.27 1.27)) (justify left)))
   (property "Footprint" "Capacitor_SMD:C_0402_1005Metric" (at 154.94 53.34 0) (effects (font (size 1.27 1.27))) (hide yes))
@@
   (pin "1")
   (pin "2")
-  (instances (project "t1-main-board" (path "/7746052e-d7f9-59ad-ba73-bd2b74439529/53ee74be-bcd0-540e-90f4-0921f22107a2" (reference "C5404") (unit 1))))
+  (instances (project "t1-main-board" (path "/7746052e-d7f9-59ad-ba73-bd2b74439529/53ee74be-bcd0-540e-90f4-0921f22107a2" (reference "C5504") (unit 1))))
 )
 (wire (pts (xy 154.94 49.53) (xy 154.94 46.99)) (stroke (width 0) (type default)))
@@
 )
 (symbol (lib_id "Device:R") (at 114.3 83.82 0) (unit 1) (body_style 1) (exclude_from_sim no) (in_bom yes) (on_board yes) (dnp no)
-  (property "Reference" "R5401" (at 115.57 82.55 0) (effects (font (size 1.27 1.27)) (justify left)))
+  (property "Reference" "R5501" (at 115.57 82.55 0) (effects (font (size 1.27 1.27)) (justify left)))
   (property "Value" "2.2 kΩ" (at 115.57 85.09 0) (effects (font (size 1.27 1.27)) (justify left)))
   (property "Footprint" "Resistor_SMD:R_0402_1005Metric" (at 114.3 83.82 0) (effects (font (size 1.27 1.27))) (hide yes))
@@
   (pin "1")
   (pin "2")
-  (instances (project "t1-main-board" (path "/7746052e-d7f9-59ad-ba73-bd2b74439529/53ee74be-bcd0-540e-90f4-0921f22107a2" (reference "R5401") (unit 1))))
+  (instances (project "t1-main-board" (path "/7746052e-d7f9-59ad-ba73-bd2b74439529/53ee74be-bcd0-540e-90f4-0921f22107a2" (reference "R5501") (unit 1))))
 )
 (wire (pts (xy 114.3 80.01) (xy 114.3 77.47)) (stroke (width 0) (type default)))
@@
 (text "SLB9673 TPM 2.0 at I2C2 0x2E (BOM v1 line 122)" (exclude_from_sim no) (at 24.13 34.29 0) (effects (font (size 2.54 2.54)) (justify left bottom)))
 (symbol (lib_id "Device:R") (at 213.36 50.8 90) (unit 1) (body_style 1) (exclude_from_sim no) (in_bom yes) (on_board yes) (dnp no)
-  (property "Reference" "R5402" (at 210.82 46.99 90) (effects (font (size 1.27 1.27))))
+  (property "Reference" "R5502" (at 210.82 46.99 90) (effects (font (size 1.27 1.27))))
   (property "Value" "100 mΩ" (at 210.82 53.34 90) (effects (font (size 1.27 1.27))))
   (property "Spec" "0603" (at 210.82 55.88 90) (effects (font (size 1.27 1.27))))
@@
   (pin "1")
   (pin "2")
-  (instances (project "t1-main-board" (path "/7746052e-d7f9-59ad-ba73-bd2b74439529/53ee74be-bcd0-540e-90f4-0921f22107a2" (reference "R5402") (unit 1) (variant (name "production") (field (name "Value") (value "0 Ω")) (field (name "MPN") (value "RC0603JR-070RL")) (field (name "Manufacturer") (value "YAGEO"))))))
+  (instances (project "t1-main-board" (path "/7746052e-d7f9-59ad-ba73-bd2b74439529/53ee74be-bcd0-540e-90f4-0921f22107a2" (reference "R5502") (unit 1) (variant (name "production") (field (name "Value") (value "0 Ω")) (field (name "MPN") (value "RC0603JR-070RL")) (field (name "Manufacturer") (value "YAGEO"))))))
 )
 (rectangle (start 190.5 38.1) (end 231.14 58.42) (stroke (width 0) (type dash)) (fill (type none)))
@@
 (wire (pts (xy 207.01 50.8) (xy 207.01 48.26)) (stroke (width 0) (type default)))
 (symbol (lib_id "Connector:TestPoint") (at 207.01 48.26 0) (unit 1) (body_style 1) (exclude_from_sim no) (in_bom no) (on_board yes) (dnp no)
-  (property "Reference" "TP5401" (at 205.74 43.18 0) (effects (font (size 1.27 1.27)) (justify right)))
+  (property "Reference" "TP5501" (at 205.74 43.18 0) (effects (font (size 1.27 1.27)) (justify right)))
   (property "Value" "vcca1v8_pmu" (at 205.74 45.72 0) (effects (font (size 1.27 1.27)) (justify right)))
   (property "Footprint" "TestPoint:TestPoint_Pad_D1.0mm" (at 207.01 48.26 0) (effects (font (size 1.27 1.27))) (hide yes))
@@
   (property "Block" "blk.tpm" (at 207.01 48.26 0) (effects (font (size 1.27 1.27))) (hide yes))
   (pin "1")
-  (instances (project "t1-main-board" (path "/7746052e-d7f9-59ad-ba73-bd2b74439529/53ee74be-bcd0-540e-90f4-0921f22107a2" (reference "TP5401") (unit 1))))
+  (instances (project "t1-main-board" (path "/7746052e-d7f9-59ad-ba73-bd2b74439529/53ee74be-bcd0-540e-90f4-0921f22107a2" (reference "TP5501") (unit 1))))
 )
 (symbol (lib_id "power:VCC") (at 187.96 50.8 90) (unit 1) (body_style 1) (exclude_from_sim no) (in_bom yes) (on_board yes) (dnp no)
@@
 (wire (pts (xy 219.71 50.8) (xy 219.71 48.26)) (stroke (width 0) (type default)))
 (symbol (lib_id "Connector:TestPoint") (at 219.71 48.26 0) (unit 1) (body_style 1) (exclude_from_sim no) (in_bom no) (on_board yes) (dnp no)
-  (property "Reference" "TP5402" (at 220.98 43.18 0) (effects (font (size 1.27 1.27)) (justify left)))
+  (property "Reference" "TP5502" (at 220.98 43.18 0) (effects (font (size 1.27 1.27)) (justify left)))
   (property "Value" "TPM_VDD" (at 220.98 45.72 0) (effects (font (size 1.27 1.27)) (justify left)))
   (property "Footprint" "TestPoint:TestPoint_Pad_D1.0mm" (at 219.71 48.26 0) (effects (font (size 1.27 1.27))) (hide yes))
@@
   (property "Block" "blk.tpm" (at 219.71 48.26 0) (effects (font (size 1.27 1.27))) (hide yes))
   (pin "1")
-  (instances (project "t1-main-board" (path "/7746052e-d7f9-59ad-ba73-bd2b74439529/53ee74be-bcd0-540e-90f4-0921f22107a2" (reference "TP5402") (unit 1))))
+  (instances (project "t1-main-board" (path "/7746052e-d7f9-59ad-ba73-bd2b74439529/53ee74be-bcd0-540e-90f4-0921f22107a2" (reference "TP5502") (unit 1))))
 )
 (junction (at 238.76 50.8) (diameter 0) (color 0 0 0 0))

Commit message: Board: capture blk.mic-ambient and links #34, #35
IM73D122 on PDM CLK1 and SDI1 (BOM v1 line 34, pinout v1 AK2 and 1P2),
LR to ground, 22 Ω clock series, VDD from MIC_1V8 through link #35.
Link #34 on blk.mic-main makes the faceplate branch the rail MIC_1V8_FP
for contact 40 (power tree §4.12, G10). kicad-lib moves to e46bda4 for
the IM73D122, TPS3808G01, SN74LVC1G58 and BAT54 parts.

Co-Authored-By: Claude Opus 5.5 <noreply@anthropic.com>
Claude-Session: https://claude.ai/code/session_01Ei262h3TpgY9vyfNLMi5Mn
Parts:
- removed C5501: 1 µF, Capacitor_SMD:C_0402_1005Metric, symbol Device:C
- removed C5502, C5503, C5504: 100 nF, Capacitor_SMD:C_0402_1005Metric, symbol Device:C
- removed R5501: 2.2 kΩ, Resistor_SMD:R_0402_1005Metric, symbol Device:R
- removed R5502: 100 mΩ, Resistor_SMD:R_0603_1608Metric, symbol Device:R
- removed TP5501: vcca1v8_pmu, TestPoint:TestPoint_Pad_D1.0mm, symbol Connector:TestPoint
- removed TP5502: TPM_VDD, TestPoint:TestPoint_Pad_D1.0mm, symbol Connector:TestPoint
- removed U5501: SLB9673XU20FW2613XTMA1, Infineon:Infineon_PG-UQFN-32-1_5x5mm_P0.5mm_EP3.6x3.6mm, symbol Infineon:SLB9673XU20FW2613XTMA1
- added C5601: 1 µF, Capacitor_SMD:C_0402_1005Metric, symbol Device:C
- added C5602, C5603, C5604: 100 nF, Capacitor_SMD:C_0402_1005Metric, symbol Device:C
- added R5601: 2.2 kΩ, Resistor_SMD:R_0402_1005Metric, symbol Device:R
- added R5602: 100 mΩ, Resistor_SMD:R_0603_1608Metric, symbol Device:R
- added TP5601: vcca1v8_pmu, TestPoint:TestPoint_Pad_D1.0mm, symbol Connector:TestPoint
- added TP5602: TPM_VDD, TestPoint:TestPoint_Pad_D1.0mm, symbol Connector:TestPoint
- added U5601: SLB9673XU20FW2613XTMA1, Infineon:Infineon_PG-UQFN-32-1_5x5mm_P0.5mm_EP3.6x3.6mm, symbol Infineon:SLB9673XU20FW2613XTMA1
Connections:
- net GND: now also C5601.2, C5602.2, C5603.2, C5604.2, U5601.16 (NCI/GND), U5601.2 (GND), U5601.23 (GND), U5601.32 (GND), U5601.9 (GND), U5601.EP
- net I2C2_SCL: now also U5601.30 (SCL)
- net I2C2_SDA: now also U5601.29 (SDA)
- net TPM_PIRQ_N: now also U5601.18 (I2C_PIRQ#)
- net TPM_RST_N: now also R5601.2, U5601.17 (RST#)
- net TPM_VDD: now also C5601.1, C5602.1, C5603.1, C5604.1, R5601.1, R5602.2, TP5602.1, U5601.1 (VDD), U5601.14 (VDD), U5601.20 (TEST#), U5601.22 (VDD), U5601.8 (NCI/VDD)
- net vcca1v8_pmu: now also R5602.1, TP5601.1
