File: board/hardware/t1-main-board/tpm.kicad_sch (KiCad schematic)
At the start: 9 parts, among them U5601 SLB9673XU20FW2613XTMA1

Commit message: Board: capture blk.maskrom
Power + Vol- at a cold power-on pull eMMC D0 low inside the TPS3808G01
boot window (BOM v1 lines 35, 78, 97, 98; sim/maskrom): SENSE 280k/100k,
CT 390 nF, WINDOW_N with its pad, SN74LVC1G57 and SN74LVC1G58 on
vcca1v8_pmu, BAT54 from PWRON_N, DMG1012T through 1 kΩ to EMMC_D0.
Every block in use now has its sheet; the README states the remaining
single-pin nets.

Co-Authored-By: Claude Opus 5.5 <noreply@anthropic.com>
Claude-Session: https://claude.ai/code/session_01Ei262h3TpgY9vyfNLMi5Mn
Parts:
- removed C5601: 1 µF, Capacitor_SMD:C_0402_1005Metric, symbol Device:C
- removed C5602, C5603, C5604: 100 nF, Capacitor_SMD:C_0402_1005Metric, symbol Device:C
- removed R5601: 2.2 kΩ, Resistor_SMD:R_0402_1005Metric, symbol Device:R
- removed R5602: 100 mΩ, Resistor_SMD:R_0603_1608Metric, symbol Device:R
- removed TP5601: vcca1v8_pmu, TestPoint:TestPoint_Pad_D1.0mm, symbol Connector:TestPoint
- removed TP5602: TPM_VDD, TestPoint:TestPoint_Pad_D1.0mm, symbol Connector:TestPoint
- removed U5601: SLB9673XU20FW2613XTMA1, Infineon:Infineon_PG-UQFN-32-1_5x5mm_P0.5mm_EP3.6x3.6mm, symbol Infineon:SLB9673XU20FW2613XTMA1
- added C5701: 1 µF, Capacitor_SMD:C_0402_1005Metric, symbol Device:C
- added C5702, C5703, C5704: 100 nF, Capacitor_SMD:C_0402_1005Metric, symbol Device:C
- added R5701: 2.2 kΩ, Resistor_SMD:R_0402_1005Metric, symbol Device:R
- added R5702: 100 mΩ, Resistor_SMD:R_0603_1608Metric, symbol Device:R
- added TP5701: vcca1v8_pmu, TestPoint:TestPoint_Pad_D1.0mm, symbol Connector:TestPoint
- added TP5702: TPM_VDD, TestPoint:TestPoint_Pad_D1.0mm, symbol Connector:TestPoint
- added U5701: SLB9673XU20FW2613XTMA1, Infineon:Infineon_PG-UQFN-32-1_5x5mm_P0.5mm_EP3.6x3.6mm, symbol Infineon:SLB9673XU20FW2613XTMA1
Connections:
- net GND: now also C5701.2, C5702.2, C5703.2, C5704.2, U5701.16 (NCI/GND), U5701.2 (GND), U5701.23 (GND), U5701.32 (GND), U5701.9 (GND), U5701.EP
- net I2C2_SCL: now also U5701.30 (SCL)
- net I2C2_SDA: now also U5701.29 (SDA)
- net TPM_PIRQ_N: now also U5701.18 (I2C_PIRQ#)
- net TPM_RST_N: now also R5701.2, U5701.17 (RST#)
- net TPM_VDD: now also C5701.1, C5702.1, C5703.1, C5704.1, R5701.1, R5702.2, TP5702.1, U5701.1 (VDD), U5701.14 (VDD), U5701.20 (TEST#), U5701.22 (VDD), U5701.8 (NCI/VDD)
- net vcca1v8_pmu: now also R5702.1, TP5701.1
Changed lines of the file:
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@@
 (title_block (title "Hardware key holder") (date "2026-10-25") (rev "A") (company "The OpenDAP Project") (comment 1 "blk.tpm") (comment 2 "SLB9673 TPM 2.0 on I2C2 at 0x2E, always on"))
 (symbol (lib_id "Infineon:SLB9673XU20FW2613XTMA1") (at 69.85 87.63 0) (unit 1) (body_style 1) (exclude_from_sim no) (in_bom yes) (on_board yes) (dnp no)
-  (property "Reference" "U5601" (at 76.2 50.8 0) (effects (font (size 1.27 1.27)) (justify left)))
+  (property "Reference" "U5701" (at 76.2 50.8 0) (effects (font (size 1.27 1.27)) (justify left)))
   (property "Value" "SLB9673XU20FW2613XTMA1" (at 76.2 48.26 0) (effects (font (size 1.27 1.27)) (justify left)))
   (property "Footprint" "Infineon:Infineon_PG-UQFN-32-1_5x5mm_P0.5mm_EP3.6x3.6mm" (at 69.85 87.63 0) (effects (font (size 1.27 1.27))) (hide yes))
@@
   (pin "16")
   (pin "EP")
-  (instances (project "t1-main-board" (path "/7746052e-d7f9-59ad-ba73-bd2b74439529/53ee74be-bcd0-540e-90f4-0921f22107a2" (reference "U5601") (unit 1))))
+  (instances (project "t1-main-board" (path "/7746052e-d7f9-59ad-ba73-bd2b74439529/53ee74be-bcd0-540e-90f4-0921f22107a2" (reference "U5701") (unit 1))))
 )
 (wire (pts (xy 64.77 49.53) (xy 64.77 46.99)) (stroke (width 0) (type default)))
@@
 (no_connect (at 85.09 100.33))
 (symbol (lib_id "Device:C") (at 114.3 53.34 0) (unit 1) (body_style 1) (exclude_from_sim no) (in_bom yes) (on_board yes) (dnp no)
-  (property "Reference" "C5601" (at 116.84 52.07 0) (effects (font (size 1.27 1.27)) (justify left)))
+  (property "Reference" "C5701" (at 116.84 52.07 0) (effects (font (size 1.27 1.27)) (justify left)))
   (property "Value" "1 µF" (at 116.84 54.61 0) (effects (font (size 1.27 1.27)) (justify left)))
   (property "Footprint" "Capacitor_SMD:C_0402_1005Metric" (at 114.3 53.34 0) (effects (font (size 1.27 1.27))) (hide yes))
@@
   (pin "1")
   (pin "2")
-  (instances (project "t1-main-board" (path "/7746052e-d7f9-59ad-ba73-bd2b74439529/53ee74be-bcd0-540e-90f4-0921f22107a2" (reference "C5601") (unit 1))))
+  (instances (project "t1-main-board" (path "/7746052e-d7f9-59ad-ba73-bd2b74439529/53ee74be-bcd0-540e-90f4-0921f22107a2" (reference "C5701") (unit 1))))
 )
 (wire (pts (xy 114.3 49.53) (xy 114.3 46.99)) (stroke (width 0) (type default)))
@@
 )
 (symbol (lib_id "Device:C") (at 127 53.34 0) (unit 1) (body_style 1) (exclude_from_sim no) (in_bom yes) (on_board yes) (dnp no)
-  (property "Reference" "C5602" (at 129.54 52.07 0) (effects (font (size 1.27 1.27)) (justify left)))
+  (property "Reference" "C5702" (at 129.54 52.07 0) (effects (font (size 1.27 1.27)) (justify left)))
   (property "Value" "100 nF" (at 129.54 54.61 0) (effects (font (size 1.27 1.27)) (justify left)))
   (property "Footprint" "Capacitor_SMD:C_0402_1005Metric" (at 127 53.34 0) (effects (font (size 1.27 1.27))) (hide yes))
@@
   (pin "1")
   (pin "2")
-  (instances (project "t1-main-board" (path "/7746052e-d7f9-59ad-ba73-bd2b74439529/53ee74be-bcd0-540e-90f4-0921f22107a2" (reference "C5602") (unit 1))))
+  (instances (project "t1-main-board" (path "/7746052e-d7f9-59ad-ba73-bd2b74439529/53ee74be-bcd0-540e-90f4-0921f22107a2" (reference "C5702") (unit 1))))
 )
 (wire (pts (xy 127 49.53) (xy 127 46.99)) (stroke (width 0) (type default)))
@@
 )
 (symbol (lib_id "Device:C") (at 140.97 53.34 0) (unit 1) (body_style 1) (exclude_from_sim no) (in_bom yes) (on_board yes) (dnp no)
-  (property "Reference" "C5603" (at 143.51 52.07 0) (effects (font (size 1.27 1.27)) (justify left)))
+  (property "Reference" "C5703" (at 143.51 52.07 0) (effects (font (size 1.27 1.27)) (justify left)))
   (property "Value" "100 nF" (at 143.51 54.61 0) (effects (font (size 1.27 1.27)) (justify left)))
   (property "Footprint" "Capacitor_SMD:C_0402_1005Metric" (at 140.97 53.34 0) (effects (font (size 1.27 1.27))) (hide yes))
@@
   (pin "1")
   (pin "2")
-  (instances (project "t1-main-board" (path "/7746052e-d7f9-59ad-ba73-bd2b74439529/53ee74be-bcd0-540e-90f4-0921f22107a2" (reference "C5603") (unit 1))))
+  (instances (project "t1-main-board" (path "/7746052e-d7f9-59ad-ba73-bd2b74439529/53ee74be-bcd0-540e-90f4-0921f22107a2" (reference "C5703") (unit 1))))
 )
 (wire (pts (xy 140.97 49.53) (xy 140.97 46.99)) (stroke (width 0) (type default)))
@@
 )
 (symbol (lib_id "Device:C") (at 154.94 53.34 0) (unit 1) (body_style 1) (exclude_from_sim no) (in_bom yes) (on_board yes) (dnp no)
-  (property "Reference" "C5604" (at 157.48 52.07 0) (effects (font (size 1.27 1.27)) (justify left)))
+  (property "Reference" "C5704" (at 157.48 52.07 0) (effects (font (size 1.27 1.27)) (justify left)))
   (property "Value" "100 nF" (at 157.48 54.61 0) (effects (font (size 1.27 1.27)) (justify left)))
   (property "Footprint" "Capacitor_SMD:C_0402_1005Metric" (at 154.94 53.34 0) (effects (font (size 1.27 1.27))) (hide yes))
@@
   (pin "1")
   (pin "2")
-  (instances (project "t1-main-board" (path "/7746052e-d7f9-59ad-ba73-bd2b74439529/53ee74be-bcd0-540e-90f4-0921f22107a2" (reference "C5604") (unit 1))))
+  (instances (project "t1-main-board" (path "/7746052e-d7f9-59ad-ba73-bd2b74439529/53ee74be-bcd0-540e-90f4-0921f22107a2" (reference "C5704") (unit 1))))
 )
 (wire (pts (xy 154.94 49.53) (xy 154.94 46.99)) (stroke (width 0) (type default)))
@@
 )
 (symbol (lib_id "Device:R") (at 114.3 83.82 0) (unit 1) (body_style 1) (exclude_from_sim no) (in_bom yes) (on_board yes) (dnp no)
-  (property "Reference" "R5601" (at 115.57 82.55 0) (effects (font (size 1.27 1.27)) (justify left)))
+  (property "Reference" "R5701" (at 115.57 82.55 0) (effects (font (size 1.27 1.27)) (justify left)))
   (property "Value" "2.2 kΩ" (at 115.57 85.09 0) (effects (font (size 1.27 1.27)) (justify left)))
   (property "Footprint" "Resistor_SMD:R_0402_1005Metric" (at 114.3 83.82 0) (effects (font (size 1.27 1.27))) (hide yes))
@@
   (pin "1")
   (pin "2")
-  (instances (project "t1-main-board" (path "/7746052e-d7f9-59ad-ba73-bd2b74439529/53ee74be-bcd0-540e-90f4-0921f22107a2" (reference "R5601") (unit 1))))
+  (instances (project "t1-main-board" (path "/7746052e-d7f9-59ad-ba73-bd2b74439529/53ee74be-bcd0-540e-90f4-0921f22107a2" (reference "R5701") (unit 1))))
 )
 (wire (pts (xy 114.3 80.01) (xy 114.3 77.47)) (stroke (width 0) (type default)))
@@
 (text "SLB9673 TPM 2.0 at I2C2 0x2E (BOM v1 line 122)" (exclude_from_sim no) (at 24.13 34.29 0) (effects (font (size 2.54 2.54)) (justify left bottom)))
 (symbol (lib_id "Device:R") (at 213.36 50.8 90) (unit 1) (body_style 1) (exclude_from_sim no) (in_bom yes) (on_board yes) (dnp no)
-  (property "Reference" "R5602" (at 210.82 46.99 90) (effects (font (size 1.27 1.27))))
+  (property "Reference" "R5702" (at 210.82 46.99 90) (effects (font (size 1.27 1.27))))
   (property "Value" "100 mΩ" (at 210.82 53.34 90) (effects (font (size 1.27 1.27))))
   (property "Spec" "0603" (at 210.82 55.88 90) (effects (font (size 1.27 1.27))))
@@
   (pin "1")
   (pin "2")
-  (instances (project "t1-main-board" (path "/7746052e-d7f9-59ad-ba73-bd2b74439529/53ee74be-bcd0-540e-90f4-0921f22107a2" (reference "R5602") (unit 1) (variant (name "production") (field (name "Value") (value "0 Ω")) (field (name "MPN") (value "RC0603JR-070RL")) (field (name "Manufacturer") (value "YAGEO"))))))
+  (instances (project "t1-main-board" (path "/7746052e-d7f9-59ad-ba73-bd2b74439529/53ee74be-bcd0-540e-90f4-0921f22107a2" (reference "R5702") (unit 1) (variant (name "production") (field (name "Value") (value "0 Ω")) (field (name "MPN") (value "RC0603JR-070RL")) (field (name "Manufacturer") (value "YAGEO"))))))
 )
 (rectangle (start 190.5 38.1) (end 231.14 58.42) (stroke (width 0) (type dash)) (fill (type none)))
@@
 (wire (pts (xy 207.01 50.8) (xy 207.01 48.26)) (stroke (width 0) (type default)))
 (symbol (lib_id "Connector:TestPoint") (at 207.01 48.26 0) (unit 1) (body_style 1) (exclude_from_sim no) (in_bom no) (on_board yes) (dnp no)
-  (property "Reference" "TP5601" (at 205.74 43.18 0) (effects (font (size 1.27 1.27)) (justify right)))
+  (property "Reference" "TP5701" (at 205.74 43.18 0) (effects (font (size 1.27 1.27)) (justify right)))
   (property "Value" "vcca1v8_pmu" (at 205.74 45.72 0) (effects (font (size 1.27 1.27)) (justify right)))
   (property "Footprint" "TestPoint:TestPoint_Pad_D1.0mm" (at 207.01 48.26 0) (effects (font (size 1.27 1.27))) (hide yes))
@@
   (property "Block" "blk.tpm" (at 207.01 48.26 0) (effects (font (size 1.27 1.27))) (hide yes))
   (pin "1")
-  (instances (project "t1-main-board" (path "/7746052e-d7f9-59ad-ba73-bd2b74439529/53ee74be-bcd0-540e-90f4-0921f22107a2" (reference "TP5601") (unit 1))))
+  (instances (project "t1-main-board" (path "/7746052e-d7f9-59ad-ba73-bd2b74439529/53ee74be-bcd0-540e-90f4-0921f22107a2" (reference "TP5701") (unit 1))))
 )
 (symbol (lib_id "power:VCC") (at 187.96 50.8 90) (unit 1) (body_style 1) (exclude_from_sim no) (in_bom yes) (on_board yes) (dnp no)
@@
 (wire (pts (xy 219.71 50.8) (xy 219.71 48.26)) (stroke (width 0) (type default)))
 (symbol (lib_id "Connector:TestPoint") (at 219.71 48.26 0) (unit 1) (body_style 1) (exclude_from_sim no) (in_bom no) (on_board yes) (dnp no)
-  (property "Reference" "TP5602" (at 220.98 43.18 0) (effects (font (size 1.27 1.27)) (justify left)))
+  (property "Reference" "TP5702" (at 220.98 43.18 0) (effects (font (size 1.27 1.27)) (justify left)))
   (property "Value" "TPM_VDD" (at 220.98 45.72 0) (effects (font (size 1.27 1.27)) (justify left)))
   (property "Footprint" "TestPoint:TestPoint_Pad_D1.0mm" (at 219.71 48.26 0) (effects (font (size 1.27 1.27))) (hide yes))
@@
   (property "Block" "blk.tpm" (at 219.71 48.26 0) (effects (font (size 1.27 1.27))) (hide yes))
   (pin "1")
-  (instances (project "t1-main-board" (path "/7746052e-d7f9-59ad-ba73-bd2b74439529/53ee74be-bcd0-540e-90f4-0921f22107a2" (reference "TP5602") (unit 1))))
+  (instances (project "t1-main-board" (path "/7746052e-d7f9-59ad-ba73-bd2b74439529/53ee74be-bcd0-540e-90f4-0921f22107a2" (reference "TP5702") (unit 1))))
 )
 (junction (at 238.76 50.8) (diameter 0) (color 0 0 0 0))

Commit message: Compaction: lower inductors, 0201 decoupling, 0.8 mm signal test pads
A matrix tool (hardware/studies/compaction) checks each candidate against
the design's stresses: same inductance, design peak <= 70 % and the
converter's maximum limit <= 100 % of Isat (30 % drop), height zones,
ratings at least twice the rail, PCB-D-06; sourcing outcome per part.

Applied (placement v1 decision 12, BOM v1.15):
- L601, L4401: XGL4015-102MEC (1.5 mm) for XAL/XGL4020-102MEC (2.1 mm);
- L1001, L5101: XGL4015-471MEC (1.5 mm) for Wurth 744373240047, on the
  stock XxL4020 land (the Wurth land was never drawn);
- L1201 is 1.2 mm (XGL4012, per-MPN heights): it moves next to the SoC;
- 58 x 100 nF decoupling on rails <= 3.3 V in core/IO/radio: 0201;
- 51 test pads on signal nets: 0.8 mm (PCB-D-06 v0.16, JLCPCB guide).
Kept: L901, L2802 (XGL4015 at 103 % of Isat at the limit); no thinner
0805/1206 capacitor passes (obsolete, NRND or unlisted).

Board need 113 % -> 111 % (core band 227 -> 203 %, power band 258 ->
233 %, radio band 19 -> 0 %); only C904 still relies on PCB-Z-04.
ERC 0 errors, craft Q1 met, DRC 0 errors (605 warnings), pcb and study
tests pass, rules test board PASS.

Co-Authored-By: Claude Opus 5.5 <noreply@anthropic.com>
Claude-Session: https://claude.ai/code/session_01Ei262h3TpgY9vyfNLMi5Mn
Parts:
- C5702, C5703, C5704: footprint Capacitor_SMD:C_0402_1005Metric -> Capacitor_SMD:C_0201_0603Metric; MPN GRM155R71C104KA88D -> GRM033R61A104KE15D
Changed lines of the file:
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@@
   (property "Reference" "C5702" (at 129.54 52.07 0) (effects (font (size 1.27 1.27)) (justify left)))
   (property "Value" "100 nF" (at 129.54 54.61 0) (effects (font (size 1.27 1.27)) (justify left)))
-  (property "Footprint" "Capacitor_SMD:C_0402_1005Metric" (at 127 53.34 0) (effects (font (size 1.27 1.27))) (hide yes))
-  (property "Datasheet" "https://www.murata.com/en-us/products/productdetail?partno=GRM155R71C104KA88D" (at 127 53.34 0) (effects (font (size 1.27 1.27))) (hide yes))
-  (property "Description" "Capacitor, 100 nF, 16 V, X7R, 0402" (at 127 53.34 0) (effects (font (size 1.27 1.27))) (hide yes))
+  (property "Footprint" "Capacitor_SMD:C_0201_0603Metric" (at 127 53.34 0) (effects (font (size 1.27 1.27))) (hide yes))
+  (property "Datasheet" "https://www.murata.com/en-us/products/productdetail?partno=GRM033R61A104KE15D" (at 127 53.34 0) (effects (font (size 1.27 1.27))) (hide yes))
+  (property "Description" "Capacitor, 100 nF, 10 V, X5R, 0201" (at 127 53.34 0) (effects (font (size 1.27 1.27))) (hide yes))
   (property "Manufacturer" "Murata" (at 127 53.34 0) (effects (font (size 1.27 1.27))) (hide yes))
-  (property "MPN" "GRM155R71C104KA88D" (at 127 53.34 0) (effects (font (size 1.27 1.27))) (hide yes))
+  (property "MPN" "GRM033R61A104KE15D" (at 127 53.34 0) (effects (font (size 1.27 1.27))) (hide yes))
   (property "Block" "blk.tpm" (at 127 53.34 0) (effects (font (size 1.27 1.27))) (hide yes))
   (pin "1")
@@
   (property "Reference" "C5703" (at 143.51 52.07 0) (effects (font (size 1.27 1.27)) (justify left)))
   (property "Value" "100 nF" (at 143.51 54.61 0) (effects (font (size 1.27 1.27)) (justify left)))
-  (property "Footprint" "Capacitor_SMD:C_0402_1005Metric" (at 140.97 53.34 0) (effects (font (size 1.27 1.27))) (hide yes))
-  (property "Datasheet" "https://www.murata.com/en-us/products/productdetail?partno=GRM155R71C104KA88D" (at 140.97 53.34 0) (effects (font (size 1.27 1.27))) (hide yes))
-  (property "Description" "Capacitor, 100 nF, 16 V, X7R, 0402" (at 140.97 53.34 0) (effects (font (size 1.27 1.27))) (hide yes))
+  (property "Footprint" "Capacitor_SMD:C_0201_0603Metric" (at 140.97 53.34 0) (effects (font (size 1.27 1.27))) (hide yes))
+  (property "Datasheet" "https://www.murata.com/en-us/products/productdetail?partno=GRM033R61A104KE15D" (at 140.97 53.34 0) (effects (font (size 1.27 1.27))) (hide yes))
+  (property "Description" "Capacitor, 100 nF, 10 V, X5R, 0201" (at 140.97 53.34 0) (effects (font (size 1.27 1.27))) (hide yes))
   (property "Manufacturer" "Murata" (at 140.97 53.34 0) (effects (font (size 1.27 1.27))) (hide yes))
-  (property "MPN" "GRM155R71C104KA88D" (at 140.97 53.34 0) (effects (font (size 1.27 1.27))) (hide yes))
+  (property "MPN" "GRM033R61A104KE15D" (at 140.97 53.34 0) (effects (font (size 1.27 1.27))) (hide yes))
   (property "Block" "blk.tpm" (at 140.97 53.34 0) (effects (font (size 1.27 1.27))) (hide yes))
   (pin "1")
@@
   (property "Reference" "C5704" (at 157.48 52.07 0) (effects (font (size 1.27 1.27)) (justify left)))
   (property "Value" "100 nF" (at 157.48 54.61 0) (effects (font (size 1.27 1.27)) (justify left)))
-  (property "Footprint" "Capacitor_SMD:C_0402_1005Metric" (at 154.94 53.34 0) (effects (font (size 1.27 1.27))) (hide yes))
-  (property "Datasheet" "https://www.murata.com/en-us/products/productdetail?partno=GRM155R71C104KA88D" (at 154.94 53.34 0) (effects (font (size 1.27 1.27))) (hide yes))
-  (property "Description" "Capacitor, 100 nF, 16 V, X7R, 0402" (at 154.94 53.34 0) (effects (font (size 1.27 1.27))) (hide yes))
+  (property "Footprint" "Capacitor_SMD:C_0201_0603Metric" (at 154.94 53.34 0) (effects (font (size 1.27 1.27))) (hide yes))
+  (property "Datasheet" "https://www.murata.com/en-us/products/productdetail?partno=GRM033R61A104KE15D" (at 154.94 53.34 0) (effects (font (size 1.27 1.27))) (hide yes))
+  (property "Description" "Capacitor, 100 nF, 10 V, X5R, 0201" (at 154.94 53.34 0) (effects (font (size 1.27 1.27))) (hide yes))
   (property "Manufacturer" "Murata" (at 154.94 53.34 0) (effects (font (size 1.27 1.27))) (hide yes))
-  (property "MPN" "GRM155R71C104KA88D" (at 154.94 53.34 0) (effects (font (size 1.27 1.27))) (hide yes))
+  (property "MPN" "GRM033R61A104KE15D" (at 154.94 53.34 0) (effects (font (size 1.27 1.27))) (hide yes))
   (property "Block" "blk.tpm" (at 154.94 53.34 0) (effects (font (size 1.27 1.27))) (hide yes))
   (pin "1")

Commit message: Board on libs v0.2.0: lower-case kebab vendor keys (HL-13)
The libs submodule moves to v0.2.0 (5f24483). Every library nickname in
the generator, the placement tool and the floorplan study follows the
key table (Texas_Instruments -> texas-instruments, OpenDAP_Device ->
opendap-generic, Rockchip and Rockchip_PMIC -> rockchip, ...); the
library tables are written from the files. Schematic and board
regenerated.

Checks: ERC 0 errors (warnings unchanged); DRC 0 errors, 605 warnings,
the same counts by type, schematic parity 0; every placement identical;
craft Q1 met; pcb tests pass; STEP export resolves every libs 3D model
(the 27 parts without a model are KiCad stock lands that have none).

Co-Authored-By: Claude Opus 5.5 <noreply@anthropic.com>
Claude-Session: https://claude.ai/code/session_01Ei262h3TpgY9vyfNLMi5Mn
Parts:
- U5701: footprint Infineon:Infineon_PG-UQFN-32-1_5x5mm_P0.5mm_EP3.6x3.6mm -> infineon:Infineon_PG-UQFN-32-1_5x5mm_P0.5mm_EP3.6x3.6mm; symbol Infineon:SLB9673XU20FW2613XTMA1 -> infineon:SLB9673XU20FW2613XTMA1
Changed lines of the file:
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@@
 (paper "A4")
 (title_block (title "Hardware key holder") (date "2026-10-25") (rev "A") (company "The OpenDAP Project") (comment 1 "blk.tpm") (comment 2 "SLB9673 TPM 2.0 on I2C2 at 0x2E, always on"))
-(symbol (lib_id "Infineon:SLB9673XU20FW2613XTMA1") (at 69.85 87.63 0) (unit 1) (body_style 1) (exclude_from_sim no) (in_bom yes) (on_board yes) (dnp no)
+(symbol (lib_id "infineon:SLB9673XU20FW2613XTMA1") (at 69.85 87.63 0) (unit 1) (body_style 1) (exclude_from_sim no) (in_bom yes) (on_board yes) (dnp no)
   (property "Reference" "U5701" (at 76.2 50.8 0) (effects (font (size 1.27 1.27)) (justify left)))
   (property "Value" "SLB9673XU20FW2613XTMA1" (at 76.2 48.26 0) (effects (font (size 1.27 1.27)) (justify left)))
-  (property "Footprint" "Infineon:Infineon_PG-UQFN-32-1_5x5mm_P0.5mm_EP3.6x3.6mm" (at 69.85 87.63 0) (effects (font (size 1.27 1.27))) (hide yes))
+  (property "Footprint" "infineon:Infineon_PG-UQFN-32-1_5x5mm_P0.5mm_EP3.6x3.6mm" (at 69.85 87.63 0) (effects (font (size 1.27 1.27))) (hide yes))
   (property "Datasheet" "https://www.farnell.com/datasheets/4146092.pdf" (at 69.85 87.63 0) (effects (font (size 1.27 1.27))) (hide yes))
   (property "Description" "OPTIGA TPM SLB 9673 TPM 2.0, I2C up to 1 MHz, 1.8 V or 3.3 V, -40 to 85 C, PG-UQFN-32 5 x 5 mm, 0.5 mm pitch, exposed pad" (at 69.85 87.63 0) (effects (font (size 1.27 1.27))) (hide yes))
