File: board/hardware/t1-main-board/tpm.kicad_sch (KiCad schematic)
At the start: 9 parts, among them U5701 SLB9673XU20FW2613XTMA1

Commit message: Board in the 62.5 x 95.0 mm body: ADR 0025, outline 59.1 x 91.6, 0201 swaps
ADR 0025 supersedes ADR 0016 for t1 ADR 0006's body: board outline from
the body, 1.2 mm walls and 0.5 mm clearance; height zones and stack
restated unchanged; the speaker on a case shelf (PCB-Z-09); pocket
reliefs at the 4.4 mm jack, the microSD (DM3AT push-push kept) and the
side buttons; the audio 0603 -> 0402 swap gated by t1 V2-A08; reserve
(NFC reader, then TPM) recorded, not applied.

- pcb/geometry.py derives the outline from BODY, WALL and CLEARANCE;
  the pocket, display and fixed parts keep their device-frame positions;
  holes keep their edge distance; the speaker shadow becomes a 1.5 mm
  shelf height area (placement, checks, occupancy).
- build.py reports pocket reliefs and routing room; C904 unfixed (it
  now finds back room, so PCB-Z-04 carries no part).
- Generator: parts.area_swap puts 121 generic 0402 resistors (outside
  audio and VBUS paths, >= 10 ohm) and five 100 nF signal capacitors in
  0201 (BOM v1.16); schematic and board regenerated.
- Result: 1,012/1,012 placed, 98.8 % by the floorplan method (was 111 %),
  factor left 1.68 (was 1.49); DRC 0 errors, ERC 0 errors, 0 check
  findings, pcb tests 20/20, schematic craft Q1 met.
- Specs: PCB constraints v0.17 (M-01, M-02, M-08, Z-02, Z-06 to Z-09,
  R-07), placement v1.1 (section 3, decisions 4 and 13, checks, open
  items with the gated swaps and the reserve), floorplan v1 section 1,
  BOM v1.16.

Co-Authored-By: Claude Opus 5.5 <noreply@anthropic.com>
Claude-Session: https://claude.ai/code/session_01Ei262h3TpgY9vyfNLMi5Mn
Parts:
- R5701: footprint Resistor_SMD:R_0402_1005Metric -> Resistor_SMD:R_0201_0603Metric; MPN RC0402FR-072K2L -> RC0201FR-072K2L
Changed lines of the file:
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@@
   (property "Reference" "R5701" (at 115.57 82.55 0) (effects (font (size 1.27 1.27)) (justify left)))
   (property "Value" "2.2 kΩ" (at 115.57 85.09 0) (effects (font (size 1.27 1.27)) (justify left)))
-  (property "Footprint" "Resistor_SMD:R_0402_1005Metric" (at 114.3 83.82 0) (effects (font (size 1.27 1.27))) (hide yes))
-  (property "Datasheet" "https://yageogroup.com/en/ProductSearch/PartNumberSearch?part=RC0402FR-072K2L" (at 114.3 83.82 0) (effects (font (size 1.27 1.27))) (hide yes))
-  (property "Description" "Resistor, 2.2 kΩ, 1 %, 1/16 W, 0402" (at 114.3 83.82 0) (effects (font (size 1.27 1.27))) (hide yes))
+  (property "Footprint" "Resistor_SMD:R_0201_0603Metric" (at 114.3 83.82 0) (effects (font (size 1.27 1.27))) (hide yes))
+  (property "Datasheet" "https://yageogroup.com/en/ProductSearch/PartNumberSearch?part=RC0201FR-072K2L" (at 114.3 83.82 0) (effects (font (size 1.27 1.27))) (hide yes))
+  (property "Description" "Resistor, 2.2 kΩ, 1 %, 1/20 W, 0201" (at 114.3 83.82 0) (effects (font (size 1.27 1.27))) (hide yes))
   (property "Manufacturer" "YAGEO" (at 114.3 83.82 0) (effects (font (size 1.27 1.27))) (hide yes))
-  (property "MPN" "RC0402FR-072K2L" (at 114.3 83.82 0) (effects (font (size 1.27 1.27))) (hide yes))
+  (property "MPN" "RC0201FR-072K2L" (at 114.3 83.82 0) (effects (font (size 1.27 1.27))) (hide yes))
   (property "Block" "blk.tpm" (at 114.3 83.82 0) (effects (font (size 1.27 1.27))) (hide yes))
   (pin "1")
