File: board/hardware/t1-main-board/charger-core.kicad_sch (KiCad schematic)
At the start: 29 parts, among them U601 BQ25798RQMR

Commit message: Board in the 62.5 x 95.0 mm body: ADR 0025, outline 59.1 x 91.6, 0201 swaps
ADR 0025 supersedes ADR 0016 for t1 ADR 0006's body: board outline from
the body, 1.2 mm walls and 0.5 mm clearance; height zones and stack
restated unchanged; the speaker on a case shelf (PCB-Z-09); pocket
reliefs at the 4.4 mm jack, the microSD (DM3AT push-push kept) and the
side buttons; the audio 0603 -> 0402 swap gated by t1 V2-A08; reserve
(NFC reader, then TPM) recorded, not applied.

- pcb/geometry.py derives the outline from BODY, WALL and CLEARANCE;
  the pocket, display and fixed parts keep their device-frame positions;
  holes keep their edge distance; the speaker shadow becomes a 1.5 mm
  shelf height area (placement, checks, occupancy).
- build.py reports pocket reliefs and routing room; C904 unfixed (it
  now finds back room, so PCB-Z-04 carries no part).
- Generator: parts.area_swap puts 121 generic 0402 resistors (outside
  audio and VBUS paths, >= 10 ohm) and five 100 nF signal capacitors in
  0201 (BOM v1.16); schematic and board regenerated.
- Result: 1,012/1,012 placed, 98.8 % by the floorplan method (was 111 %),
  factor left 1.68 (was 1.49); DRC 0 errors, ERC 0 errors, 0 check
  findings, pcb tests 20/20, schematic craft Q1 met.
- Specs: PCB constraints v0.17 (M-01, M-02, M-08, Z-02, Z-06 to Z-09,
  R-07), placement v1.1 (section 3, decisions 4 and 13, checks, open
  items with the gated swaps and the reserve), floorplan v1 section 1,
  BOM v1.16.

Co-Authored-By: Claude Opus 5.5 <noreply@anthropic.com>
Claude-Session: https://claude.ai/code/session_01Ei262h3TpgY9vyfNLMi5Mn
Parts:
- R601: footprint Resistor_SMD:R_0402_1005Metric -> Resistor_SMD:R_0201_0603Metric; MPN RC0402FR-076K04L -> RC0201FR-076K04L
- R602, R605: footprint Resistor_SMD:R_0402_1005Metric -> Resistor_SMD:R_0201_0603Metric; MPN RC0402FR-0710KL -> RC0201FR-0710KL
- R603: footprint Resistor_SMD:R_0402_1005Metric -> Resistor_SMD:R_0201_0603Metric; MPN RC0402FR-075K23L -> RC0201FR-075K23L
- R604: footprint Resistor_SMD:R_0402_1005Metric -> Resistor_SMD:R_0201_0603Metric; MPN RC0402FR-0730K1L -> RC0201FR-0730K1L
Changed lines of the file:
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@@
   (property "Reference" "R601" (at 90.17 53.34 0) (effects (font (size 1.27 1.27)) (justify left)))
   (property "Value" "6.04 kΩ" (at 90.17 55.88 0) (effects (font (size 1.27 1.27)) (justify left)))
-  (property "Footprint" "Resistor_SMD:R_0402_1005Metric" (at 88.9 54.61 0) (effects (font (size 1.27 1.27))) (hide yes))
-  (property "Datasheet" "https://yageogroup.com/en/ProductSearch/PartNumberSearch?part=RC0402FR-076K04L" (at 88.9 54.61 0) (effects (font (size 1.27 1.27))) (hide yes))
-  (property "Description" "Resistor, 6.04 kΩ, 1 %, 1/16 W, 0402" (at 88.9 54.61 0) (effects (font (size 1.27 1.27))) (hide yes))
+  (property "Footprint" "Resistor_SMD:R_0201_0603Metric" (at 88.9 54.61 0) (effects (font (size 1.27 1.27))) (hide yes))
+  (property "Datasheet" "https://yageogroup.com/en/ProductSearch/PartNumberSearch?part=RC0201FR-076K04L" (at 88.9 54.61 0) (effects (font (size 1.27 1.27))) (hide yes))
+  (property "Description" "Resistor, 6.04 kΩ, 1 %, 1/20 W, 0201" (at 88.9 54.61 0) (effects (font (size 1.27 1.27))) (hide yes))
   (property "Manufacturer" "YAGEO" (at 88.9 54.61 0) (effects (font (size 1.27 1.27))) (hide yes))
-  (property "MPN" "RC0402FR-076K04L" (at 88.9 54.61 0) (effects (font (size 1.27 1.27))) (hide yes))
+  (property "MPN" "RC0201FR-076K04L" (at 88.9 54.61 0) (effects (font (size 1.27 1.27))) (hide yes))
   (property "Block" "blk.charger-core" (at 88.9 54.61 0) (effects (font (size 1.27 1.27))) (hide yes))
   (pin "1")
@@
   (property "Reference" "R602" (at 104.14 53.34 0) (effects (font (size 1.27 1.27)) (justify left)))
   (property "Value" "10 kΩ" (at 104.14 55.88 0) (effects (font (size 1.27 1.27)) (justify left)))
-  (property "Footprint" "Resistor_SMD:R_0402_1005Metric" (at 102.87 54.61 0) (effects (font (size 1.27 1.27))) (hide yes))
-  (property "Datasheet" "https://yageogroup.com/en/ProductSearch/PartNumberSearch?part=RC0402FR-0710KL" (at 102.87 54.61 0) (effects (font (size 1.27 1.27))) (hide yes))
-  (property "Description" "Resistor, 10 kΩ, 1 %, 1/16 W, 0402" (at 102.87 54.61 0) (effects (font (size 1.27 1.27))) (hide yes))
+  (property "Footprint" "Resistor_SMD:R_0201_0603Metric" (at 102.87 54.61 0) (effects (font (size 1.27 1.27))) (hide yes))
+  (property "Datasheet" "https://yageogroup.com/en/ProductSearch/PartNumberSearch?part=RC0201FR-0710KL" (at 102.87 54.61 0) (effects (font (size 1.27 1.27))) (hide yes))
+  (property "Description" "Resistor, 10 kΩ, 1 %, 1/20 W, 0201" (at 102.87 54.61 0) (effects (font (size 1.27 1.27))) (hide yes))
   (property "Manufacturer" "YAGEO" (at 102.87 54.61 0) (effects (font (size 1.27 1.27))) (hide yes))
-  (property "MPN" "RC0402FR-0710KL" (at 102.87 54.61 0) (effects (font (size 1.27 1.27))) (hide yes))
+  (property "MPN" "RC0201FR-0710KL" (at 102.87 54.61 0) (effects (font (size 1.27 1.27))) (hide yes))
   (property "Block" "blk.charger-core" (at 102.87 54.61 0) (effects (font (size 1.27 1.27))) (hide yes))
   (pin "1")
@@
   (property "Reference" "R603" (at 132.08 53.34 0) (effects (font (size 1.27 1.27)) (justify left)))
   (property "Value" "5.23 kΩ" (at 132.08 55.88 0) (effects (font (size 1.27 1.27)) (justify left)))
-  (property "Footprint" "Resistor_SMD:R_0402_1005Metric" (at 130.81 54.61 0) (effects (font (size 1.27 1.27))) (hide yes))
-  (property "Datasheet" "https://yageogroup.com/en/ProductSearch/PartNumberSearch?part=RC0402FR-075K23L" (at 130.81 54.61 0) (effects (font (size 1.27 1.27))) (hide yes))
-  (property "Description" "Resistor, 5.23 kΩ, 1 %, 1/16 W, 0402" (at 130.81 54.61 0) (effects (font (size 1.27 1.27))) (hide yes))
+  (property "Footprint" "Resistor_SMD:R_0201_0603Metric" (at 130.81 54.61 0) (effects (font (size 1.27 1.27))) (hide yes))
+  (property "Datasheet" "https://yageogroup.com/en/ProductSearch/PartNumberSearch?part=RC0201FR-075K23L" (at 130.81 54.61 0) (effects (font (size 1.27 1.27))) (hide yes))
+  (property "Description" "Resistor, 5.23 kΩ, 1 %, 1/20 W, 0201" (at 130.81 54.61 0) (effects (font (size 1.27 1.27))) (hide yes))
   (property "Manufacturer" "YAGEO" (at 130.81 54.61 0) (effects (font (size 1.27 1.27))) (hide yes))
-  (property "MPN" "RC0402FR-075K23L" (at 130.81 54.61 0) (effects (font (size 1.27 1.27))) (hide yes))
+  (property "MPN" "RC0201FR-075K23L" (at 130.81 54.61 0) (effects (font (size 1.27 1.27))) (hide yes))
   (property "Block" "blk.charger-core" (at 130.81 54.61 0) (effects (font (size 1.27 1.27))) (hide yes))
   (pin "1")
@@
   (property "Reference" "R604" (at 146.05 53.34 0) (effects (font (size 1.27 1.27)) (justify left)))
   (property "Value" "30.1 kΩ" (at 146.05 55.88 0) (effects (font (size 1.27 1.27)) (justify left)))
-  (property "Footprint" "Resistor_SMD:R_0402_1005Metric" (at 144.78 54.61 0) (effects (font (size 1.27 1.27))) (hide yes))
-  (property "Datasheet" "https://yageogroup.com/en/ProductSearch/PartNumberSearch?part=RC0402FR-0730K1L" (at 144.78 54.61 0) (effects (font (size 1.27 1.27))) (hide yes))
-  (property "Description" "Resistor, 30.1 kΩ, 1 %, 1/16 W, 0402" (at 144.78 54.61 0) (effects (font (size 1.27 1.27))) (hide yes))
+  (property "Footprint" "Resistor_SMD:R_0201_0603Metric" (at 144.78 54.61 0) (effects (font (size 1.27 1.27))) (hide yes))
+  (property "Datasheet" "https://yageogroup.com/en/ProductSearch/PartNumberSearch?part=RC0201FR-0730K1L" (at 144.78 54.61 0) (effects (font (size 1.27 1.27))) (hide yes))
+  (property "Description" "Resistor, 30.1 kΩ, 1 %, 1/20 W, 0201" (at 144.78 54.61 0) (effects (font (size 1.27 1.27))) (hide yes))
   (property "Manufacturer" "YAGEO" (at 144.78 54.61 0) (effects (font (size 1.27 1.27))) (hide yes))
-  (property "MPN" "RC0402FR-0730K1L" (at 144.78 54.61 0) (effects (font (size 1.27 1.27))) (hide yes))
+  (property "MPN" "RC0201FR-0730K1L" (at 144.78 54.61 0) (effects (font (size 1.27 1.27))) (hide yes))
   (property "Block" "blk.charger-core" (at 144.78 54.61 0) (effects (font (size 1.27 1.27))) (hide yes))
   (pin "1")
@@
   (property "Reference" "R605" (at 160.02 53.34 0) (effects (font (size 1.27 1.27)) (justify left)))
   (property "Value" "10 kΩ" (at 160.02 55.88 0) (effects (font (size 1.27 1.27)) (justify left)))
-  (property "Footprint" "Resistor_SMD:R_0402_1005Metric" (at 158.75 54.61 0) (effects (font (size 1.27 1.27))) (hide yes))
-  (property "Datasheet" "https://yageogroup.com/en/ProductSearch/PartNumberSearch?part=RC0402FR-0710KL" (at 158.75 54.61 0) (effects (font (size 1.27 1.27))) (hide yes))
-  (property "Description" "Resistor, 10 kΩ, 1 %, 1/16 W, 0402" (at 158.75 54.61 0) (effects (font (size 1.27 1.27))) (hide yes))
+  (property "Footprint" "Resistor_SMD:R_0201_0603Metric" (at 158.75 54.61 0) (effects (font (size 1.27 1.27))) (hide yes))
+  (property "Datasheet" "https://yageogroup.com/en/ProductSearch/PartNumberSearch?part=RC0201FR-0710KL" (at 158.75 54.61 0) (effects (font (size 1.27 1.27))) (hide yes))
+  (property "Description" "Resistor, 10 kΩ, 1 %, 1/20 W, 0201" (at 158.75 54.61 0) (effects (font (size 1.27 1.27))) (hide yes))
   (property "Manufacturer" "YAGEO" (at 158.75 54.61 0) (effects (font (size 1.27 1.27))) (hide yes))
-  (property "MPN" "RC0402FR-0710KL" (at 158.75 54.61 0) (effects (font (size 1.27 1.27))) (hide yes))
+  (property "MPN" "RC0201FR-0710KL" (at 158.75 54.61 0) (effects (font (size 1.27 1.27))) (hide yes))
   (property "Block" "blk.charger-core" (at 158.75 54.61 0) (effects (font (size 1.27 1.27))) (hide yes))
   (pin "1")

Commit message: BOM v1.17: DC-bias gate closed, 7 x 10 uF in 0603 and 2 x 1 uF in 0201
The 1 uF and 10 uF swaps of v1.16 waited for DC-bias figures (DRV-107).
Murata's DC-bias data at each node's highest voltage, -20 to 85 C,
tolerance included, against each circuit's need: the BQ25798 VBUS and
SYS capacitors and the two TPS22945 output capacitors pass and are
swapped; the other 31 positions keep their part. The 10 uF 0603 is in
production. Three findings go to section 7 (items 51-53): the VSYS
converter inputs miss their 3 uF minimum with the present part.

Co-Authored-By: Claude Opus 5.5 <noreply@anthropic.com>
Claude-Session: https://claude.ai/code/session_01Ei262h3TpgY9vyfNLMi5Mn
Parts:
- C605, C606, C612, C613, C614, C615, C616: footprint Capacitor_SMD:C_0805_2012Metric -> Capacitor_SMD:C_0603_1608Metric; MPN GRM21BR61E106KA73L -> GRM188R61E106MA73D
