File: board/hardware/t1-main-board/fp-connector.kicad_sch (KiCad schematic)
At the start: 25 parts, among them J4901 FH35C-51S-0.3SHW, U4901 TPD4E05U06DQAR, U4902 TPD4E05U06DQAR, U4903 TPD4E05U06DQAR, U4904 TPD4E05U06DQAR, U4905 TPD4E05U06DQAR, U4906 TPD4E05U06DQAR, U4907 TPS22950YBHR, U4908 TPS22945DCKR

Commit message: Board: capture blk.current-monitors
Five INA236 on I2C1 (0x40-0x43, 0x48) with their shunts, per power tree
§4.12 and BOM v1 lines 54 and 136. The measured branches are rails of
their own (VSYS_SRC, VSYS_LV_AUDIO, VSYS_AUDIO, VSYS_LV_BL, VSYS_P5V1),
fed through the shunts on this sheet; the charger, audio, backlight and
5.1 V sheets take them. The root's layout may leave a stack level empty,
so the block sits under the notes; IC bboxes hold turned rail values;
passive rows hold a bottom rail's text.

Co-Authored-By: Claude Opus 5.5 <noreply@anthropic.com>
Claude-Session: https://claude.ai/code/session_01Ei262h3TpgY9vyfNLMi5Mn
Parts:
- removed C4901, C4902, C4903, C4904: 1 µF, Capacitor_SMD:C_0402_1005Metric, symbol Device:C
- removed J4901: FH35C-51S-0.3SHW, Hirose:Hirose_FH35C-51S-0.3SHW_1x51-1MP_P0.3mm_Horizontal, symbol Hirose:FH35C-51S-0.3SHW
- removed R4901, R4908: 10 kΩ, Resistor_SMD:R_0402_1005Metric, symbol Device:R
- removed R4902, R4903, R4905: 100 kΩ, Resistor_SMD:R_0402_1005Metric, symbol Device:R
- removed R4904: 3.57 kΩ, Resistor_SMD:R_0402_1005Metric, symbol Device:R
- removed R4906: 100 mΩ, Resistor_SMD:R_0603_1608Metric, symbol Device:R
- removed R4907: 1 Ω, Resistor_SMD:R_0603_1608Metric, symbol Device:R
- removed TP4901: FP_3V3_SRC, TestPoint:TestPoint_Pad_D1.0mm, symbol Connector:TestPoint
- removed TP4902: FP_3V3, TestPoint:TestPoint_Pad_D1.0mm, symbol Connector:TestPoint
- removed TP4903: FP_1V8_SRC, TestPoint:TestPoint_Pad_D1.0mm, symbol Connector:TestPoint
- removed TP4904: FP_1V8, TestPoint:TestPoint_Pad_D1.0mm, symbol Connector:TestPoint
- removed U4901, U4902, U4903, U4904, U4905, U4906: TPD4E05U06DQAR, Texas_Instruments:Texas_DQA0010A_USON-10_1x2.5mm_P0.5mm, symbol Texas_Instruments:TPD4E05U06DQAR
- removed U4907: TPS22950YBHR, Texas_Instruments:Texas_YBH0006_DSBGA-6_0.706x1.106mm_Layout2x3_P0.4mm, symbol Texas_Instruments:TPS22950YBHR
- removed U4908: TPS22945DCKR, Texas_Instruments:Texas_DCK0005A_SC-70-5_1.25x2mm_P0.65mm, symbol Texas_Instruments:TPS22945DCKR
- added C5001, C5002, C5003, C5004: 1 µF, Capacitor_SMD:C_0402_1005Metric, symbol Device:C
- added J5001: FH35C-51S-0.3SHW, Hirose:Hirose_FH35C-51S-0.3SHW_1x51-1MP_P0.3mm_Horizontal, symbol Hirose:FH35C-51S-0.3SHW
- added R5001, R5008: 10 kΩ, Resistor_SMD:R_0402_1005Metric, symbol Device:R
- added R5002, R5003, R5005: 100 kΩ, Resistor_SMD:R_0402_1005Metric, symbol Device:R
- added R5004: 3.57 kΩ, Resistor_SMD:R_0402_1005Metric, symbol Device:R
- added R5006: 100 mΩ, Resistor_SMD:R_0603_1608Metric, symbol Device:R
- added R5007: 1 Ω, Resistor_SMD:R_0603_1608Metric, symbol Device:R
- added TP5001: FP_3V3_SRC, TestPoint:TestPoint_Pad_D1.0mm, symbol Connector:TestPoint
- added TP5002: FP_3V3, TestPoint:TestPoint_Pad_D1.0mm, symbol Connector:TestPoint
- added TP5003: FP_1V8_SRC, TestPoint:TestPoint_Pad_D1.0mm, symbol Connector:TestPoint
- added TP5004: FP_1V8, TestPoint:TestPoint_Pad_D1.0mm, symbol Connector:TestPoint
- added U5001, U5002, U5003, U5004, U5005, U5006: TPD4E05U06DQAR, Texas_Instruments:Texas_DQA0010A_USON-10_1x2.5mm_P0.5mm, symbol Texas_Instruments:TPD4E05U06DQAR
- added U5007: TPS22950YBHR, Texas_Instruments:Texas_YBH0006_DSBGA-6_0.706x1.106mm_Layout2x3_P0.4mm, symbol Texas_Instruments:TPS22950YBHR
- added U5008: TPS22945DCKR, Texas_Instruments:Texas_DCK0005A_SC-70-5_1.25x2mm_P0.65mm, symbol Texas_Instruments:TPS22945DCKR
Connections:
- net BL_LEDA: now also J5001.46 (Pin_46)
- net BL_LEDK: now also J5001.45 (Pin_45)
- net FP3V3_ILIM: now also R5004.1, U5007.C2 (ILIM)
- net FP_1V8: now also J5001.41 (Pin_41), R5007.2, TP5004.1
- net FP_1V8_SRC: now also C5004.1, R5007.1, R5008.1, TP5003.1, U5008.1 (VOUT)
- net FP_3V3: now also J5001.42 (Pin_42), J5001.43 (Pin_43), R5006.2, TP5002.1
- net FP_3V3_SRC: now also C5002.1, R5006.1, TP5001.1, U5007.B2 (VOUT)
- net FP_ALS_INT_N: now also J5001.29 (Pin_29), U5004.1 (D1+)
- net FP_DBI_DC: now also J5001.23 (Pin_23), U5002.4 (D2+)
- net FP_DET_N: now also J5001.36 (Pin_36), R5001.2, U5005.4 (D2+)
- net FP_DSI_CLK_N: now also J5001.15 (Pin_15)
- net FP_DSI_CLK_P: now also J5001.14 (Pin_14)
- net FP_DSI_D0_N: now also J5001.12 (Pin_12)
- net FP_DSI_D0_P: now also J5001.11 (Pin_11)
- net FP_DSI_D1_N: now also J5001.9 (Pin_9)
- net FP_DSI_D1_P: now also J5001.8 (Pin_8)
- net FP_DSI_D2_N: now also J5001.6 (Pin_6)
- net FP_DSI_D2_P: now also J5001.5 (Pin_5)
- net FP_DSI_D3_N: now also J5001.3 (Pin_3)
- net FP_DSI_D3_P: now also J5001.2 (Pin_2)
- net FP_GPIO0: now also J5001.37 (Pin_37), R5002.1, U5005.5 (D2-)
- net FP_GPIO1: now also J5001.38 (Pin_38), R5003.1, U5006.1 (D1+)
- net FP_HID_INT_N: now also J5001.28 (Pin_28), U5003.5 (D2-)
- net FP_I2C_SCL: now also J5001.17 (Pin_17), U5001.1 (D1+)
- net FP_I2C_SDA: now also J5001.18 (Pin_18), U5001.2 (D1-)
- net FP_IO_EN: now also R5005.1, U5007.A1 (ON), U5008.4 (ON)
- net FP_LCD_RST_N: now also J5001.26 (Pin_26), U5003.2 (D1-)
- net FP_LCD_TE: now also J5001.27 (Pin_27), U5003.4 (D2+)
- net FP_SPI_CS_N: now also J5001.22 (Pin_22), U5002.2 (D1-)
- net FP_SPI_MISO: now also J5001.21 (Pin_21), U5002.1 (D1+)
- net FP_SPI_MOSI: now also J5001.20 (Pin_20), U5001.5 (D2-)
- net FP_SPI_SCLK: now also J5001.19 (Pin_19), U5001.4 (D2+)
- net FP_TP_INT: now also J5001.24 (Pin_24), U5002.5 (D2-)
- net FP_TP_RST_N: now also J5001.25 (Pin_25), U5003.1 (D1+)
- net FP_VCI: now also J5001.44 (Pin_44)
- net GND: now also C5001.2, C5002.2, C5003.2, C5004.2, J5001.1 (Pin_1), J5001.10 (Pin_10), J5001.13 (Pin_13), J5001.16 (Pin_16), J5001.33 (Pin_33), J5001.39 (Pin_39), J5001.4 (Pin_4), J5001.7 (Pin_7), R5002.2, R5003.2, R5004.2, R5005.2, R5008.2, U5001.3 (GND), U5001.8 (GND), U5002.3 (GND), U5002.8 (GND), U5003.3 (GND), U5003.8 (GND), U5004.3 (GND), U5004.8 (GND), U5005.3 (GND), U5005.8 (GND), U5006.3 (GND), U5006.8 (GND), U5007.C1 (GND), U5008.2 (GND)
- net LED_B: now also J5001.32 (Pin_32), U5004.5 (D2-)
- net LED_G: now also J5001.31 (Pin_31), U5004.4 (D2+)
- net LED_R: now also J5001.30 (Pin_30), U5004.2 (D1-)
- net MIC_1V8: now also J5001.40 (Pin_40)
- net PDM_CLK0_FP: now also J5001.34 (Pin_34), U5005.1 (D1+)
- net PDM_DATA0: now also J5001.35 (Pin_35), U5005.2 (D1-)
- net vcc3v3_sys: now also C5001.1, R5001.1, U5007.B1 (VIN)
- net vcc_1v8: now also C5003.1, U5008.5 (VIN)

Commit message: Board: capture blk.debug
Debug UART2 (1.8 V) and I2S/DSD pads with ground pads, reset, PMIC and
power-key pads (PCB-T-09), a pad on every spare SoC GPIO whose pinout v1
row names one (the DEBUG bus, on the SoC's right edge), and a rail pad
for each power-tree rail no other sheet probes (PCB-T-02). Each DAC
sheet carries a pad on its MCLK. The spares pinout v1 leaves without a
pad now carry no-connect flags. On the root, facing sheet pins are
joined directly only where the route meets no other symbol.

Co-Authored-By: Claude Opus 5.5 <noreply@anthropic.com>
Claude-Session: https://claude.ai/code/session_01Ei262h3TpgY9vyfNLMi5Mn
Parts:
- removed C5001, C5002, C5003, C5004: 1 µF, Capacitor_SMD:C_0402_1005Metric, symbol Device:C
- removed J5001: FH35C-51S-0.3SHW, Hirose:Hirose_FH35C-51S-0.3SHW_1x51-1MP_P0.3mm_Horizontal, symbol Hirose:FH35C-51S-0.3SHW
- removed R5001, R5008: 10 kΩ, Resistor_SMD:R_0402_1005Metric, symbol Device:R
- removed R5002, R5003, R5005: 100 kΩ, Resistor_SMD:R_0402_1005Metric, symbol Device:R
- removed R5004: 3.57 kΩ, Resistor_SMD:R_0402_1005Metric, symbol Device:R
- removed R5006: 100 mΩ, Resistor_SMD:R_0603_1608Metric, symbol Device:R
- removed R5007: 1 Ω, Resistor_SMD:R_0603_1608Metric, symbol Device:R
- removed TP5001: FP_3V3_SRC, TestPoint:TestPoint_Pad_D1.0mm, symbol Connector:TestPoint
- removed TP5002: FP_3V3, TestPoint:TestPoint_Pad_D1.0mm, symbol Connector:TestPoint
- removed TP5003: FP_1V8_SRC, TestPoint:TestPoint_Pad_D1.0mm, symbol Connector:TestPoint
- removed TP5004: FP_1V8, TestPoint:TestPoint_Pad_D1.0mm, symbol Connector:TestPoint
- removed U5001, U5002, U5003, U5004, U5005, U5006: TPD4E05U06DQAR, Texas_Instruments:Texas_DQA0010A_USON-10_1x2.5mm_P0.5mm, symbol Texas_Instruments:TPD4E05U06DQAR
- removed U5007: TPS22950YBHR, Texas_Instruments:Texas_YBH0006_DSBGA-6_0.706x1.106mm_Layout2x3_P0.4mm, symbol Texas_Instruments:TPS22950YBHR
- removed U5008: TPS22945DCKR, Texas_Instruments:Texas_DCK0005A_SC-70-5_1.25x2mm_P0.65mm, symbol Texas_Instruments:TPS22945DCKR
- added C5101, C5102, C5103, C5104: 1 µF, Capacitor_SMD:C_0402_1005Metric, symbol Device:C
- added J5101: FH35C-51S-0.3SHW, Hirose:Hirose_FH35C-51S-0.3SHW_1x51-1MP_P0.3mm_Horizontal, symbol Hirose:FH35C-51S-0.3SHW
- added R5101, R5108: 10 kΩ, Resistor_SMD:R_0402_1005Metric, symbol Device:R
- added R5102, R5103, R5105: 100 kΩ, Resistor_SMD:R_0402_1005Metric, symbol Device:R
- added R5104: 3.57 kΩ, Resistor_SMD:R_0402_1005Metric, symbol Device:R
- added R5106: 100 mΩ, Resistor_SMD:R_0603_1608Metric, symbol Device:R
- added R5107: 1 Ω, Resistor_SMD:R_0603_1608Metric, symbol Device:R
- added TP5101: FP_3V3_SRC, TestPoint:TestPoint_Pad_D1.0mm, symbol Connector:TestPoint
- added TP5102: FP_3V3, TestPoint:TestPoint_Pad_D1.0mm, symbol Connector:TestPoint
- added TP5103: FP_1V8_SRC, TestPoint:TestPoint_Pad_D1.0mm, symbol Connector:TestPoint
- added TP5104: FP_1V8, TestPoint:TestPoint_Pad_D1.0mm, symbol Connector:TestPoint
- added U5101, U5102, U5103, U5104, U5105, U5106: TPD4E05U06DQAR, Texas_Instruments:Texas_DQA0010A_USON-10_1x2.5mm_P0.5mm, symbol Texas_Instruments:TPD4E05U06DQAR
- added U5107: TPS22950YBHR, Texas_Instruments:Texas_YBH0006_DSBGA-6_0.706x1.106mm_Layout2x3_P0.4mm, symbol Texas_Instruments:TPS22950YBHR
- added U5108: TPS22945DCKR, Texas_Instruments:Texas_DCK0005A_SC-70-5_1.25x2mm_P0.65mm, symbol Texas_Instruments:TPS22945DCKR
Connections:
- net BL_LEDA: now also J5101.46 (Pin_46)
- net BL_LEDK: now also J5101.45 (Pin_45)
- net FP3V3_ILIM: now also R5104.1, U5107.C2 (ILIM)
- net FP_1V8: now also J5101.41 (Pin_41), R5107.2, TP5104.1
- net FP_1V8_SRC: now also C5104.1, R5107.1, R5108.1, TP5103.1, U5108.1 (VOUT)
- net FP_3V3: now also J5101.42 (Pin_42), J5101.43 (Pin_43), R5106.2, TP5102.1
- net FP_3V3_SRC: now also C5102.1, R5106.1, TP5101.1, U5107.B2 (VOUT)
- net FP_ALS_INT_N: now also J5101.29 (Pin_29), U5104.1 (D1+)
- net FP_DBI_DC: now also J5101.23 (Pin_23), U5102.4 (D2+)
- net FP_DET_N: now also J5101.36 (Pin_36), R5101.2, U5105.4 (D2+)
- net FP_DSI_CLK_N: now also J5101.15 (Pin_15)
- net FP_DSI_CLK_P: now also J5101.14 (Pin_14)
- net FP_DSI_D0_N: now also J5101.12 (Pin_12)
- net FP_DSI_D0_P: now also J5101.11 (Pin_11)
- net FP_DSI_D1_N: now also J5101.9 (Pin_9)
- net FP_DSI_D1_P: now also J5101.8 (Pin_8)
- net FP_DSI_D2_N: now also J5101.6 (Pin_6)
- net FP_DSI_D2_P: now also J5101.5 (Pin_5)
- net FP_DSI_D3_N: now also J5101.3 (Pin_3)
- net FP_DSI_D3_P: now also J5101.2 (Pin_2)
- net FP_GPIO0: now also J5101.37 (Pin_37), R5102.1, U5105.5 (D2-)
- net FP_GPIO1: now also J5101.38 (Pin_38), R5103.1, U5106.1 (D1+)
- net FP_HID_INT_N: now also J5101.28 (Pin_28), U5103.5 (D2-)
- net FP_I2C_SCL: now also J5101.17 (Pin_17), U5101.1 (D1+)
- net FP_I2C_SDA: now also J5101.18 (Pin_18), U5101.2 (D1-)
- net FP_IO_EN: now also R5105.1, U5107.A1 (ON), U5108.4 (ON)
- net FP_LCD_RST_N: now also J5101.26 (Pin_26), U5103.2 (D1-)
- net FP_LCD_TE: now also J5101.27 (Pin_27), U5103.4 (D2+)
- net FP_SPI_CS_N: now also J5101.22 (Pin_22), U5102.2 (D1-)
- net FP_SPI_MISO: now also J5101.21 (Pin_21), U5102.1 (D1+)
- net FP_SPI_MOSI: now also J5101.20 (Pin_20), U5101.5 (D2-)
- net FP_SPI_SCLK: now also J5101.19 (Pin_19), U5101.4 (D2+)
- net FP_TP_INT: now also J5101.24 (Pin_24), U5102.5 (D2-)
- net FP_TP_RST_N: now also J5101.25 (Pin_25), U5103.1 (D1+)
- net FP_VCI: now also J5101.44 (Pin_44)
- net GND: now also C5101.2, C5102.2, C5103.2, C5104.2, J5101.1 (Pin_1), J5101.10 (Pin_10), J5101.13 (Pin_13), J5101.16 (Pin_16), J5101.33 (Pin_33), J5101.39 (Pin_39), J5101.4 (Pin_4), J5101.7 (Pin_7), R5102.2, R5103.2, R5104.2, R5105.2, R5108.2, U5101.3 (GND), U5101.8 (GND), U5102.3 (GND), U5102.8 (GND), U5103.3 (GND), U5103.8 (GND), U5104.3 (GND), U5104.8 (GND), U5105.3 (GND), U5105.8 (GND), U5106.3 (GND), U5106.8 (GND), U5107.C1 (GND), U5108.2 (GND)
- net LED_B: now also J5101.32 (Pin_32), U5104.5 (D2-)
- net LED_G: now also J5101.31 (Pin_31), U5104.4 (D2+)
- net LED_R: now also J5101.30 (Pin_30), U5104.2 (D1-)
- net MIC_1V8: now also J5101.40 (Pin_40)
- net PDM_CLK0_FP: now also J5101.34 (Pin_34), U5105.1 (D1+)
- net PDM_DATA0: now also J5101.35 (Pin_35), U5105.2 (D1-)
- net vcc3v3_sys: now also C5101.1, R5101.1, U5107.B1 (VIN)
- net vcc_1v8: now also C5103.1, U5108.5 (VIN)

Commit message: Board: capture blk.mic-ambient and links #34, #35
IM73D122 on PDM CLK1 and SDI1 (BOM v1 line 34, pinout v1 AK2 and 1P2),
LR to ground, 22 Ω clock series, VDD from MIC_1V8 through link #35.
Link #34 on blk.mic-main makes the faceplate branch the rail MIC_1V8_FP
for contact 40 (power tree §4.12, G10). kicad-lib moves to e46bda4 for
the IM73D122, TPS3808G01, SN74LVC1G58 and BAT54 parts.

Co-Authored-By: Claude Opus 5.5 <noreply@anthropic.com>
Claude-Session: https://claude.ai/code/session_01Ei262h3TpgY9vyfNLMi5Mn
Parts:
- removed C5101, C5102, C5103, C5104: 1 µF, Capacitor_SMD:C_0402_1005Metric, symbol Device:C
- removed J5101: FH35C-51S-0.3SHW, Hirose:Hirose_FH35C-51S-0.3SHW_1x51-1MP_P0.3mm_Horizontal, symbol Hirose:FH35C-51S-0.3SHW
- removed R5101, R5108: 10 kΩ, Resistor_SMD:R_0402_1005Metric, symbol Device:R
- removed R5102, R5103, R5105: 100 kΩ, Resistor_SMD:R_0402_1005Metric, symbol Device:R
- removed R5104: 3.57 kΩ, Resistor_SMD:R_0402_1005Metric, symbol Device:R
- removed R5106: 100 mΩ, Resistor_SMD:R_0603_1608Metric, symbol Device:R
- removed R5107: 1 Ω, Resistor_SMD:R_0603_1608Metric, symbol Device:R
- removed TP5101: FP_3V3_SRC, TestPoint:TestPoint_Pad_D1.0mm, symbol Connector:TestPoint
- removed TP5102: FP_3V3, TestPoint:TestPoint_Pad_D1.0mm, symbol Connector:TestPoint
- removed TP5103: FP_1V8_SRC, TestPoint:TestPoint_Pad_D1.0mm, symbol Connector:TestPoint
- removed TP5104: FP_1V8, TestPoint:TestPoint_Pad_D1.0mm, symbol Connector:TestPoint
- removed U5101, U5102, U5103, U5104, U5105, U5106: TPD4E05U06DQAR, Texas_Instruments:Texas_DQA0010A_USON-10_1x2.5mm_P0.5mm, symbol Texas_Instruments:TPD4E05U06DQAR
- removed U5107: TPS22950YBHR, Texas_Instruments:Texas_YBH0006_DSBGA-6_0.706x1.106mm_Layout2x3_P0.4mm, symbol Texas_Instruments:TPS22950YBHR
- removed U5108: TPS22945DCKR, Texas_Instruments:Texas_DCK0005A_SC-70-5_1.25x2mm_P0.65mm, symbol Texas_Instruments:TPS22945DCKR
- added C5201, C5202, C5203, C5204: 1 µF, Capacitor_SMD:C_0402_1005Metric, symbol Device:C
- added J5201: FH35C-51S-0.3SHW, Hirose:Hirose_FH35C-51S-0.3SHW_1x51-1MP_P0.3mm_Horizontal, symbol Hirose:FH35C-51S-0.3SHW
- added R5201, R5208: 10 kΩ, Resistor_SMD:R_0402_1005Metric, symbol Device:R
- added R5202, R5203, R5205: 100 kΩ, Resistor_SMD:R_0402_1005Metric, symbol Device:R
- added R5204: 3.57 kΩ, Resistor_SMD:R_0402_1005Metric, symbol Device:R
- added R5206: 100 mΩ, Resistor_SMD:R_0603_1608Metric, symbol Device:R
- added R5207: 1 Ω, Resistor_SMD:R_0603_1608Metric, symbol Device:R
- added TP5201: FP_3V3_SRC, TestPoint:TestPoint_Pad_D1.0mm, symbol Connector:TestPoint
- added TP5202: FP_3V3, TestPoint:TestPoint_Pad_D1.0mm, symbol Connector:TestPoint
- added TP5203: FP_1V8_SRC, TestPoint:TestPoint_Pad_D1.0mm, symbol Connector:TestPoint
- added TP5204: FP_1V8, TestPoint:TestPoint_Pad_D1.0mm, symbol Connector:TestPoint
- added U5201, U5202, U5203, U5204, U5205, U5206: TPD4E05U06DQAR, Texas_Instruments:Texas_DQA0010A_USON-10_1x2.5mm_P0.5mm, symbol Texas_Instruments:TPD4E05U06DQAR
- added U5207: TPS22950YBHR, Texas_Instruments:Texas_YBH0006_DSBGA-6_0.706x1.106mm_Layout2x3_P0.4mm, symbol Texas_Instruments:TPS22950YBHR
- added U5208: TPS22945DCKR, Texas_Instruments:Texas_DCK0005A_SC-70-5_1.25x2mm_P0.65mm, symbol Texas_Instruments:TPS22945DCKR
Connections:
- net BL_LEDA: now also J5201.46 (Pin_46)
- net BL_LEDK: now also J5201.45 (Pin_45)
- net FP3V3_ILIM: now also R5204.1, U5207.C2 (ILIM)
- net FP_1V8: now also J5201.41 (Pin_41), R5207.2, TP5204.1
- net FP_1V8_SRC: now also C5204.1, R5207.1, R5208.1, TP5203.1, U5208.1 (VOUT)
- net FP_3V3: now also J5201.42 (Pin_42), J5201.43 (Pin_43), R5206.2, TP5202.1
- net FP_3V3_SRC: now also C5202.1, R5206.1, TP5201.1, U5207.B2 (VOUT)
- net FP_ALS_INT_N: now also J5201.29 (Pin_29), U5204.1 (D1+)
- net FP_DBI_DC: now also J5201.23 (Pin_23), U5202.4 (D2+)
- net FP_DET_N: now also J5201.36 (Pin_36), R5201.2, U5205.4 (D2+)
- net FP_DSI_CLK_N: now also J5201.15 (Pin_15)
- net FP_DSI_CLK_P: now also J5201.14 (Pin_14)
- net FP_DSI_D0_N: now also J5201.12 (Pin_12)
- net FP_DSI_D0_P: now also J5201.11 (Pin_11)
- net FP_DSI_D1_N: now also J5201.9 (Pin_9)
- net FP_DSI_D1_P: now also J5201.8 (Pin_8)
- net FP_DSI_D2_N: now also J5201.6 (Pin_6)
- net FP_DSI_D2_P: now also J5201.5 (Pin_5)
- net FP_DSI_D3_N: now also J5201.3 (Pin_3)
- net FP_DSI_D3_P: now also J5201.2 (Pin_2)
- net FP_GPIO0: now also J5201.37 (Pin_37), R5202.1, U5205.5 (D2-)
- net FP_GPIO1: now also J5201.38 (Pin_38), R5203.1, U5206.1 (D1+)
- net FP_HID_INT_N: now also J5201.28 (Pin_28), U5203.5 (D2-)
- net FP_I2C_SCL: now also J5201.17 (Pin_17), U5201.1 (D1+)
- net FP_I2C_SDA: now also J5201.18 (Pin_18), U5201.2 (D1-)
- net FP_IO_EN: now also R5205.1, U5207.A1 (ON), U5208.4 (ON)
- net FP_LCD_RST_N: now also J5201.26 (Pin_26), U5203.2 (D1-)
- net FP_LCD_TE: now also J5201.27 (Pin_27), U5203.4 (D2+)
- net FP_SPI_CS_N: now also J5201.22 (Pin_22), U5202.2 (D1-)
- net FP_SPI_MISO: now also J5201.21 (Pin_21), U5202.1 (D1+)
- net FP_SPI_MOSI: now also J5201.20 (Pin_20), U5201.5 (D2-)
- net FP_SPI_SCLK: now also J5201.19 (Pin_19), U5201.4 (D2+)
- net FP_TP_INT: now also J5201.24 (Pin_24), U5202.5 (D2-)
- net FP_TP_RST_N: now also J5201.25 (Pin_25), U5203.1 (D1+)
- net FP_VCI: now also J5201.44 (Pin_44)
- net GND: now also C5201.2, C5202.2, C5203.2, C5204.2, J5201.1 (Pin_1), J5201.10 (Pin_10), J5201.13 (Pin_13), J5201.16 (Pin_16), J5201.33 (Pin_33), J5201.39 (Pin_39), J5201.4 (Pin_4), J5201.7 (Pin_7), R5202.2, R5203.2, R5204.2, R5205.2, R5208.2, U5201.3 (GND), U5201.8 (GND), U5202.3 (GND), U5202.8 (GND), U5203.3 (GND), U5203.8 (GND), U5204.3 (GND), U5204.8 (GND), U5205.3 (GND), U5205.8 (GND), U5206.3 (GND), U5206.8 (GND), U5207.C1 (GND), U5208.2 (GND)
- net LED_B: now also J5201.32 (Pin_32), U5204.5 (D2-)
- net LED_G: now also J5201.31 (Pin_31), U5204.4 (D2+)
- net LED_R: now also J5201.30 (Pin_30), U5204.2 (D1-)
- net PDM_CLK0_FP: now also J5201.34 (Pin_34), U5205.1 (D1+)
- net PDM_DATA0: now also J5201.35 (Pin_35), U5205.2 (D1-)
- net vcc3v3_sys: now also C5201.1, R5201.1, U5207.B1 (VIN)
- net vcc_1v8: now also C5203.1, U5208.5 (VIN)
- new net MIC_1V8_FP: J5201.40 (Pin_40)
