File: board/hardware/t1-main-board/fp-connector.kicad_sch (KiCad schematic)
At the start: 25 parts, among them J5201 FH35C-51S-0.3SHW, U5201 TPD4E05U06DQAR, U5202 TPD4E05U06DQAR, U5203 TPD4E05U06DQAR, U5204 TPD4E05U06DQAR, U5205 TPD4E05U06DQAR, U5206 TPD4E05U06DQAR, U5207 TPS22950YBHR, U5208 TPS22945DCKR

Commit message: Board: capture blk.maskrom
Power + Vol- at a cold power-on pull eMMC D0 low inside the TPS3808G01
boot window (BOM v1 lines 35, 78, 97, 98; sim/maskrom): SENSE 280k/100k,
CT 390 nF, WINDOW_N with its pad, SN74LVC1G57 and SN74LVC1G58 on
vcca1v8_pmu, BAT54 from PWRON_N, DMG1012T through 1 kΩ to EMMC_D0.
Every block in use now has its sheet; the README states the remaining
single-pin nets.

Co-Authored-By: Claude Opus 5.5 <noreply@anthropic.com>
Claude-Session: https://claude.ai/code/session_01Ei262h3TpgY9vyfNLMi5Mn
Parts:
- removed C5201, C5202, C5203, C5204: 1 µF, Capacitor_SMD:C_0402_1005Metric, symbol Device:C
- removed J5201: FH35C-51S-0.3SHW, Hirose:Hirose_FH35C-51S-0.3SHW_1x51-1MP_P0.3mm_Horizontal, symbol Hirose:FH35C-51S-0.3SHW
- removed R5201, R5208: 10 kΩ, Resistor_SMD:R_0402_1005Metric, symbol Device:R
- removed R5202, R5203, R5205: 100 kΩ, Resistor_SMD:R_0402_1005Metric, symbol Device:R
- removed R5204: 3.57 kΩ, Resistor_SMD:R_0402_1005Metric, symbol Device:R
- removed R5206: 100 mΩ, Resistor_SMD:R_0603_1608Metric, symbol Device:R
- removed R5207: 1 Ω, Resistor_SMD:R_0603_1608Metric, symbol Device:R
- removed TP5201: FP_3V3_SRC, TestPoint:TestPoint_Pad_D1.0mm, symbol Connector:TestPoint
- removed TP5202: FP_3V3, TestPoint:TestPoint_Pad_D1.0mm, symbol Connector:TestPoint
- removed TP5203: FP_1V8_SRC, TestPoint:TestPoint_Pad_D1.0mm, symbol Connector:TestPoint
- removed TP5204: FP_1V8, TestPoint:TestPoint_Pad_D1.0mm, symbol Connector:TestPoint
- removed U5201, U5202, U5203, U5204, U5205, U5206: TPD4E05U06DQAR, Texas_Instruments:Texas_DQA0010A_USON-10_1x2.5mm_P0.5mm, symbol Texas_Instruments:TPD4E05U06DQAR
- removed U5207: TPS22950YBHR, Texas_Instruments:Texas_YBH0006_DSBGA-6_0.706x1.106mm_Layout2x3_P0.4mm, symbol Texas_Instruments:TPS22950YBHR
- removed U5208: TPS22945DCKR, Texas_Instruments:Texas_DCK0005A_SC-70-5_1.25x2mm_P0.65mm, symbol Texas_Instruments:TPS22945DCKR
- added C5301, C5302, C5303, C5304: 1 µF, Capacitor_SMD:C_0402_1005Metric, symbol Device:C
- added J5301: FH35C-51S-0.3SHW, Hirose:Hirose_FH35C-51S-0.3SHW_1x51-1MP_P0.3mm_Horizontal, symbol Hirose:FH35C-51S-0.3SHW
- added R5301, R5308: 10 kΩ, Resistor_SMD:R_0402_1005Metric, symbol Device:R
- added R5302, R5303, R5305: 100 kΩ, Resistor_SMD:R_0402_1005Metric, symbol Device:R
- added R5304: 3.57 kΩ, Resistor_SMD:R_0402_1005Metric, symbol Device:R
- added R5306: 100 mΩ, Resistor_SMD:R_0603_1608Metric, symbol Device:R
- added R5307: 1 Ω, Resistor_SMD:R_0603_1608Metric, symbol Device:R
- added TP5301: FP_3V3_SRC, TestPoint:TestPoint_Pad_D1.0mm, symbol Connector:TestPoint
- added TP5302: FP_3V3, TestPoint:TestPoint_Pad_D1.0mm, symbol Connector:TestPoint
- added TP5303: FP_1V8_SRC, TestPoint:TestPoint_Pad_D1.0mm, symbol Connector:TestPoint
- added TP5304: FP_1V8, TestPoint:TestPoint_Pad_D1.0mm, symbol Connector:TestPoint
- added U5301, U5302, U5303, U5304, U5305, U5306: TPD4E05U06DQAR, Texas_Instruments:Texas_DQA0010A_USON-10_1x2.5mm_P0.5mm, symbol Texas_Instruments:TPD4E05U06DQAR
- added U5307: TPS22950YBHR, Texas_Instruments:Texas_YBH0006_DSBGA-6_0.706x1.106mm_Layout2x3_P0.4mm, symbol Texas_Instruments:TPS22950YBHR
- added U5308: TPS22945DCKR, Texas_Instruments:Texas_DCK0005A_SC-70-5_1.25x2mm_P0.65mm, symbol Texas_Instruments:TPS22945DCKR
Connections:
- net BL_LEDA: now also J5301.46 (Pin_46)
- net BL_LEDK: now also J5301.45 (Pin_45)
- net FP3V3_ILIM: now also R5304.1, U5307.C2 (ILIM)
- net FP_1V8: now also J5301.41 (Pin_41), R5307.2, TP5304.1
- net FP_1V8_SRC: now also C5304.1, R5307.1, R5308.1, TP5303.1, U5308.1 (VOUT)
- net FP_3V3: now also J5301.42 (Pin_42), J5301.43 (Pin_43), R5306.2, TP5302.1
- net FP_3V3_SRC: now also C5302.1, R5306.1, TP5301.1, U5307.B2 (VOUT)
- net FP_ALS_INT_N: now also J5301.29 (Pin_29), U5304.1 (D1+)
- net FP_DBI_DC: now also J5301.23 (Pin_23), U5302.4 (D2+)
- net FP_DET_N: now also J5301.36 (Pin_36), R5301.2, U5305.4 (D2+)
- net FP_DSI_CLK_N: now also J5301.15 (Pin_15)
- net FP_DSI_CLK_P: now also J5301.14 (Pin_14)
- net FP_DSI_D0_N: now also J5301.12 (Pin_12)
- net FP_DSI_D0_P: now also J5301.11 (Pin_11)
- net FP_DSI_D1_N: now also J5301.9 (Pin_9)
- net FP_DSI_D1_P: now also J5301.8 (Pin_8)
- net FP_DSI_D2_N: now also J5301.6 (Pin_6)
- net FP_DSI_D2_P: now also J5301.5 (Pin_5)
- net FP_DSI_D3_N: now also J5301.3 (Pin_3)
- net FP_DSI_D3_P: now also J5301.2 (Pin_2)
- net FP_GPIO0: now also J5301.37 (Pin_37), R5302.1, U5305.5 (D2-)
- net FP_GPIO1: now also J5301.38 (Pin_38), R5303.1, U5306.1 (D1+)
- net FP_HID_INT_N: now also J5301.28 (Pin_28), U5303.5 (D2-)
- net FP_I2C_SCL: now also J5301.17 (Pin_17), U5301.1 (D1+)
- net FP_I2C_SDA: now also J5301.18 (Pin_18), U5301.2 (D1-)
- net FP_IO_EN: now also R5305.1, U5307.A1 (ON), U5308.4 (ON)
- net FP_LCD_RST_N: now also J5301.26 (Pin_26), U5303.2 (D1-)
- net FP_LCD_TE: now also J5301.27 (Pin_27), U5303.4 (D2+)
- net FP_SPI_CS_N: now also J5301.22 (Pin_22), U5302.2 (D1-)
- net FP_SPI_MISO: now also J5301.21 (Pin_21), U5302.1 (D1+)
- net FP_SPI_MOSI: now also J5301.20 (Pin_20), U5301.5 (D2-)
- net FP_SPI_SCLK: now also J5301.19 (Pin_19), U5301.4 (D2+)
- net FP_TP_INT: now also J5301.24 (Pin_24), U5302.5 (D2-)
- net FP_TP_RST_N: now also J5301.25 (Pin_25), U5303.1 (D1+)
- net FP_VCI: now also J5301.44 (Pin_44)
- net GND: now also C5301.2, C5302.2, C5303.2, C5304.2, J5301.1 (Pin_1), J5301.10 (Pin_10), J5301.13 (Pin_13), J5301.16 (Pin_16), J5301.33 (Pin_33), J5301.39 (Pin_39), J5301.4 (Pin_4), J5301.7 (Pin_7), R5302.2, R5303.2, R5304.2, R5305.2, R5308.2, U5301.3 (GND), U5301.8 (GND), U5302.3 (GND), U5302.8 (GND), U5303.3 (GND), U5303.8 (GND), U5304.3 (GND), U5304.8 (GND), U5305.3 (GND), U5305.8 (GND), U5306.3 (GND), U5306.8 (GND), U5307.C1 (GND), U5308.2 (GND)
- net LED_B: now also J5301.32 (Pin_32), U5304.5 (D2-)
- net LED_G: now also J5301.31 (Pin_31), U5304.4 (D2+)
- net LED_R: now also J5301.30 (Pin_30), U5304.2 (D1-)
- net MIC_1V8_FP: now also J5301.40 (Pin_40)
- net PDM_CLK0_FP: now also J5301.34 (Pin_34), U5305.1 (D1+)
- net PDM_DATA0: now also J5301.35 (Pin_35), U5305.2 (D1-)
- net vcc3v3_sys: now also C5301.1, R5301.1, U5307.B1 (VIN)
- net vcc_1v8: now also C5303.1, U5308.5 (VIN)

Commit message: Board on libs v0.2.0: lower-case kebab vendor keys (HL-13)
The libs submodule moves to v0.2.0 (5f24483). Every library nickname in
the generator, the placement tool and the floorplan study follows the
key table (Texas_Instruments -> texas-instruments, OpenDAP_Device ->
opendap-generic, Rockchip and Rockchip_PMIC -> rockchip, ...); the
library tables are written from the files. Schematic and board
regenerated.

Checks: ERC 0 errors (warnings unchanged); DRC 0 errors, 605 warnings,
the same counts by type, schematic parity 0; every placement identical;
craft Q1 met; pcb tests pass; STEP export resolves every libs 3D model
(the 27 parts without a model are KiCad stock lands that have none).

Co-Authored-By: Claude Opus 5.5 <noreply@anthropic.com>
Claude-Session: https://claude.ai/code/session_01Ei262h3TpgY9vyfNLMi5Mn
Parts:
- J5301: footprint Hirose:Hirose_FH35C-51S-0.3SHW_1x51-1MP_P0.3mm_Horizontal -> hirose:Hirose_FH35C-51S-0.3SHW_1x51-1MP_P0.3mm_Horizontal; symbol Hirose:FH35C-51S-0.3SHW -> hirose:FH35C-51S-0.3SHW
- U5301, U5302, U5303, U5304, U5305, U5306: footprint Texas_Instruments:Texas_DQA0010A_USON-10_1x2.5mm_P0.5mm -> texas-instruments:Texas_DQA0010A_USON-10_1x2.5mm_P0.5mm; symbol Texas_Instruments:TPD4E05U06DQAR -> texas-instruments:TPD4E05U06DQAR
- U5307: footprint Texas_Instruments:Texas_YBH0006_DSBGA-6_0.706x1.106mm_Layout2x3_P0.4mm -> texas-instruments:Texas_YBH0006_DSBGA-6_0.706x1.106mm_Layout2x3_P0.4mm; symbol Texas_Instruments:TPS22950YBHR -> texas-instruments:TPS22950YBHR
- U5308: footprint Texas_Instruments:Texas_DCK0005A_SC-70-5_1.25x2mm_P0.65mm -> texas-instruments:Texas_DCK0005A_SC-70-5_1.25x2mm_P0.65mm; symbol Texas_Instruments:TPS22945DCKR -> texas-instruments:TPS22945DCKR

Commit message: Board in the 62.5 x 95.0 mm body: ADR 0025, outline 59.1 x 91.6, 0201 swaps
ADR 0025 supersedes ADR 0016 for t1 ADR 0006's body: board outline from
the body, 1.2 mm walls and 0.5 mm clearance; height zones and stack
restated unchanged; the speaker on a case shelf (PCB-Z-09); pocket
reliefs at the 4.4 mm jack, the microSD (DM3AT push-push kept) and the
side buttons; the audio 0603 -> 0402 swap gated by t1 V2-A08; reserve
(NFC reader, then TPM) recorded, not applied.

- pcb/geometry.py derives the outline from BODY, WALL and CLEARANCE;
  the pocket, display and fixed parts keep their device-frame positions;
  holes keep their edge distance; the speaker shadow becomes a 1.5 mm
  shelf height area (placement, checks, occupancy).
- build.py reports pocket reliefs and routing room; C904 unfixed (it
  now finds back room, so PCB-Z-04 carries no part).
- Generator: parts.area_swap puts 121 generic 0402 resistors (outside
  audio and VBUS paths, >= 10 ohm) and five 100 nF signal capacitors in
  0201 (BOM v1.16); schematic and board regenerated.
- Result: 1,012/1,012 placed, 98.8 % by the floorplan method (was 111 %),
  factor left 1.68 (was 1.49); DRC 0 errors, ERC 0 errors, 0 check
  findings, pcb tests 20/20, schematic craft Q1 met.
- Specs: PCB constraints v0.17 (M-01, M-02, M-08, Z-02, Z-06 to Z-09,
  R-07), placement v1.1 (section 3, decisions 4 and 13, checks, open
  items with the gated swaps and the reserve), floorplan v1 section 1,
  BOM v1.16.

Co-Authored-By: Claude Opus 5.5 <noreply@anthropic.com>
Claude-Session: https://claude.ai/code/session_01Ei262h3TpgY9vyfNLMi5Mn
Parts:
- R5301, R5308: footprint Resistor_SMD:R_0402_1005Metric -> Resistor_SMD:R_0201_0603Metric; MPN RC0402FR-0710KL -> RC0201FR-0710KL
- R5302, R5303, R5305: footprint Resistor_SMD:R_0402_1005Metric -> Resistor_SMD:R_0201_0603Metric; MPN RC0402FR-07100KL -> RC0201FR-07100KL
- R5304: footprint Resistor_SMD:R_0402_1005Metric -> Resistor_SMD:R_0201_0603Metric; MPN RC0402FR-073K57L -> RC0201FR-073K57L
Changed lines of the file:
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@@
   (property "Reference" "R5301" (at 356.87 53.34 0) (effects (font (size 1.27 1.27)) (justify left)))
   (property "Value" "10 kΩ" (at 356.87 55.88 0) (effects (font (size 1.27 1.27)) (justify left)))
-  (property "Footprint" "Resistor_SMD:R_0402_1005Metric" (at 355.6 54.61 0) (effects (font (size 1.27 1.27))) (hide yes))
-  (property "Datasheet" "https://yageogroup.com/en/ProductSearch/PartNumberSearch?part=RC0402FR-0710KL" (at 355.6 54.61 0) (effects (font (size 1.27 1.27))) (hide yes))
-  (property "Description" "Resistor, 10 kΩ, 1 %, 1/16 W, 0402" (at 355.6 54.61 0) (effects (font (size 1.27 1.27))) (hide yes))
+  (property "Footprint" "Resistor_SMD:R_0201_0603Metric" (at 355.6 54.61 0) (effects (font (size 1.27 1.27))) (hide yes))
+  (property "Datasheet" "https://yageogroup.com/en/ProductSearch/PartNumberSearch?part=RC0201FR-0710KL" (at 355.6 54.61 0) (effects (font (size 1.27 1.27))) (hide yes))
+  (property "Description" "Resistor, 10 kΩ, 1 %, 1/20 W, 0201" (at 355.6 54.61 0) (effects (font (size 1.27 1.27))) (hide yes))
   (property "Manufacturer" "YAGEO" (at 355.6 54.61 0) (effects (font (size 1.27 1.27))) (hide yes))
-  (property "MPN" "RC0402FR-0710KL" (at 355.6 54.61 0) (effects (font (size 1.27 1.27))) (hide yes))
+  (property "MPN" "RC0201FR-0710KL" (at 355.6 54.61 0) (effects (font (size 1.27 1.27))) (hide yes))
   (property "Block" "blk.fp-connector" (at 355.6 54.61 0) (effects (font (size 1.27 1.27))) (hide yes))
   (pin "1")
@@
   (property "Reference" "R5302" (at 369.57 53.34 0) (effects (font (size 1.27 1.27)) (justify left)))
   (property "Value" "100 kΩ" (at 369.57 55.88 0) (effects (font (size 1.27 1.27)) (justify left)))
-  (property "Footprint" "Resistor_SMD:R_0402_1005Metric" (at 368.3 54.61 0) (effects (font (size 1.27 1.27))) (hide yes))
-  (property "Datasheet" "https://yageogroup.com/en/ProductSearch/PartNumberSearch?part=RC0402FR-07100KL" (at 368.3 54.61 0) (effects (font (size 1.27 1.27))) (hide yes))
-  (property "Description" "Resistor, 100 kΩ, 1 %, 1/16 W, 0402" (at 368.3 54.61 0) (effects (font (size 1.27 1.27))) (hide yes))
+  (property "Footprint" "Resistor_SMD:R_0201_0603Metric" (at 368.3 54.61 0) (effects (font (size 1.27 1.27))) (hide yes))
+  (property "Datasheet" "https://yageogroup.com/en/ProductSearch/PartNumberSearch?part=RC0201FR-07100KL" (at 368.3 54.61 0) (effects (font (size 1.27 1.27))) (hide yes))
+  (property "Description" "Resistor, 100 kΩ, 1 %, 1/20 W, 0201" (at 368.3 54.61 0) (effects (font (size 1.27 1.27))) (hide yes))
   (property "Manufacturer" "YAGEO" (at 368.3 54.61 0) (effects (font (size 1.27 1.27))) (hide yes))
-  (property "MPN" "RC0402FR-07100KL" (at 368.3 54.61 0) (effects (font (size 1.27 1.27))) (hide yes))
+  (property "MPN" "RC0201FR-07100KL" (at 368.3 54.61 0) (effects (font (size 1.27 1.27))) (hide yes))
   (property "Block" "blk.fp-connector" (at 368.3 54.61 0) (effects (font (size 1.27 1.27))) (hide yes))
   (pin "1")
@@
   (property "Reference" "R5303" (at 383.54 53.34 0) (effects (font (size 1.27 1.27)) (justify left)))
   (property "Value" "100 kΩ" (at 383.54 55.88 0) (effects (font (size 1.27 1.27)) (justify left)))
-  (property "Footprint" "Resistor_SMD:R_0402_1005Metric" (at 382.27 54.61 0) (effects (font (size 1.27 1.27))) (hide yes))
-  (property "Datasheet" "https://yageogroup.com/en/ProductSearch/PartNumberSearch?part=RC0402FR-07100KL" (at 382.27 54.61 0) (effects (font (size 1.27 1.27))) (hide yes))
-  (property "Description" "Resistor, 100 kΩ, 1 %, 1/16 W, 0402" (at 382.27 54.61 0) (effects (font (size 1.27 1.27))) (hide yes))
+  (property "Footprint" "Resistor_SMD:R_0201_0603Metric" (at 382.27 54.61 0) (effects (font (size 1.27 1.27))) (hide yes))
+  (property "Datasheet" "https://yageogroup.com/en/ProductSearch/PartNumberSearch?part=RC0201FR-07100KL" (at 382.27 54.61 0) (effects (font (size 1.27 1.27))) (hide yes))
+  (property "Description" "Resistor, 100 kΩ, 1 %, 1/20 W, 0201" (at 382.27 54.61 0) (effects (font (size 1.27 1.27))) (hide yes))
   (property "Manufacturer" "YAGEO" (at 382.27 54.61 0) (effects (font (size 1.27 1.27))) (hide yes))
-  (property "MPN" "RC0402FR-07100KL" (at 382.27 54.61 0) (effects (font (size 1.27 1.27))) (hide yes))
+  (property "MPN" "RC0201FR-07100KL" (at 382.27 54.61 0) (effects (font (size 1.27 1.27))) (hide yes))
   (property "Block" "blk.fp-connector" (at 382.27 54.61 0) (effects (font (size 1.27 1.27))) (hide yes))
   (pin "1")
@@
   (property "Reference" "R5304" (at 113.03 167.64 0) (effects (font (size 1.27 1.27)) (justify left)))
   (property "Value" "3.57 kΩ" (at 113.03 170.18 0) (effects (font (size 1.27 1.27)) (justify left)))
-  (property "Footprint" "Resistor_SMD:R_0402_1005Metric" (at 111.76 168.91 0) (effects (font (size 1.27 1.27))) (hide yes))
-  (property "Datasheet" "https://yageogroup.com/en/ProductSearch/PartNumberSearch?part=RC0402FR-073K57L" (at 111.76 168.91 0) (effects (font (size 1.27 1.27))) (hide yes))
-  (property "Description" "Resistor, 3.57 kΩ, 1 %, 1/16 W, 0402" (at 111.76 168.91 0) (effects (font (size 1.27 1.27))) (hide yes))
+  (property "Footprint" "Resistor_SMD:R_0201_0603Metric" (at 111.76 168.91 0) (effects (font (size 1.27 1.27))) (hide yes))
+  (property "Datasheet" "https://yageogroup.com/en/ProductSearch/PartNumberSearch?part=RC0201FR-073K57L" (at 111.76 168.91 0) (effects (font (size 1.27 1.27))) (hide yes))
+  (property "Description" "Resistor, 3.57 kΩ, 1 %, 1/20 W, 0201" (at 111.76 168.91 0) (effects (font (size 1.27 1.27))) (hide yes))
   (property "Manufacturer" "YAGEO" (at 111.76 168.91 0) (effects (font (size 1.27 1.27))) (hide yes))
-  (property "MPN" "RC0402FR-073K57L" (at 111.76 168.91 0) (effects (font (size 1.27 1.27))) (hide yes))
+  (property "MPN" "RC0201FR-073K57L" (at 111.76 168.91 0) (effects (font (size 1.27 1.27))) (hide yes))
   (property "Block" "blk.fp-connector" (at 111.76 168.91 0) (effects (font (size 1.27 1.27))) (hide yes))
   (pin "1")
@@
   (property "Reference" "R5305" (at 127 167.64 0) (effects (font (size 1.27 1.27)) (justify left)))
   (property "Value" "100 kΩ" (at 127 170.18 0) (effects (font (size 1.27 1.27)) (justify left)))
-  (property "Footprint" "Resistor_SMD:R_0402_1005Metric" (at 125.73 168.91 0) (effects (font (size 1.27 1.27))) (hide yes))
-  (property "Datasheet" "https://yageogroup.com/en/ProductSearch/PartNumberSearch?part=RC0402FR-07100KL" (at 125.73 168.91 0) (effects (font (size 1.27 1.27))) (hide yes))
-  (property "Description" "Resistor, 100 kΩ, 1 %, 1/16 W, 0402" (at 125.73 168.91 0) (effects (font (size 1.27 1.27))) (hide yes))
+  (property "Footprint" "Resistor_SMD:R_0201_0603Metric" (at 125.73 168.91 0) (effects (font (size 1.27 1.27))) (hide yes))
+  (property "Datasheet" "https://yageogroup.com/en/ProductSearch/PartNumberSearch?part=RC0201FR-07100KL" (at 125.73 168.91 0) (effects (font (size 1.27 1.27))) (hide yes))
+  (property "Description" "Resistor, 100 kΩ, 1 %, 1/20 W, 0201" (at 125.73 168.91 0) (effects (font (size 1.27 1.27))) (hide yes))
   (property "Manufacturer" "YAGEO" (at 125.73 168.91 0) (effects (font (size 1.27 1.27))) (hide yes))
-  (property "MPN" "RC0402FR-07100KL" (at 125.73 168.91 0) (effects (font (size 1.27 1.27))) (hide yes))
+  (property "MPN" "RC0201FR-07100KL" (at 125.73 168.91 0) (effects (font (size 1.27 1.27))) (hide yes))
   (property "Block" "blk.fp-connector" (at 125.73 168.91 0) (effects (font (size 1.27 1.27))) (hide yes))
   (pin "1")
@@
   (property "Reference" "R5308" (at 334.01 167.64 0) (effects (font (size 1.27 1.27)) (justify left)))
   (property "Value" "10 kΩ" (at 334.01 170.18 0) (effects (font (size 1.27 1.27)) (justify left)))
-  (property "Footprint" "Resistor_SMD:R_0402_1005Metric" (at 332.74 168.91 0) (effects (font (size 1.27 1.27))) (hide yes))
-  (property "Datasheet" "https://yageogroup.com/en/ProductSearch/PartNumberSearch?part=RC0402FR-0710KL" (at 332.74 168.91 0) (effects (font (size 1.27 1.27))) (hide yes))
-  (property "Description" "Resistor, 10 kΩ, 1 %, 1/16 W, 0402" (at 332.74 168.91 0) (effects (font (size 1.27 1.27))) (hide yes))
+  (property "Footprint" "Resistor_SMD:R_0201_0603Metric" (at 332.74 168.91 0) (effects (font (size 1.27 1.27))) (hide yes))
+  (property "Datasheet" "https://yageogroup.com/en/ProductSearch/PartNumberSearch?part=RC0201FR-0710KL" (at 332.74 168.91 0) (effects (font (size 1.27 1.27))) (hide yes))
+  (property "Description" "Resistor, 10 kΩ, 1 %, 1/20 W, 0201" (at 332.74 168.91 0) (effects (font (size 1.27 1.27))) (hide yes))
   (property "Manufacturer" "YAGEO" (at 332.74 168.91 0) (effects (font (size 1.27 1.27))) (hide yes))
-  (property "MPN" "RC0402FR-0710KL" (at 332.74 168.91 0) (effects (font (size 1.27 1.27))) (hide yes))
+  (property "MPN" "RC0201FR-0710KL" (at 332.74 168.91 0) (effects (font (size 1.27 1.27))) (hide yes))
   (property "Block" "blk.fp-connector" (at 332.74 168.91 0) (effects (font (size 1.27 1.27))) (hide yes))
   (pin "1")

Commit message: BOM v1.17: DC-bias gate closed, 7 x 10 uF in 0603 and 2 x 1 uF in 0201
The 1 uF and 10 uF swaps of v1.16 waited for DC-bias figures (DRV-107).
Murata's DC-bias data at each node's highest voltage, -20 to 85 C,
tolerance included, against each circuit's need: the BQ25798 VBUS and
SYS capacitors and the two TPS22945 output capacitors pass and are
swapped; the other 31 positions keep their part. The 10 uF 0603 is in
production. Three findings go to section 7 (items 51-53): the VSYS
converter inputs miss their 3 uF minimum with the present part.

Co-Authored-By: Claude Opus 5.5 <noreply@anthropic.com>
Claude-Session: https://claude.ai/code/session_01Ei262h3TpgY9vyfNLMi5Mn
Parts:
- C5304: footprint Capacitor_SMD:C_0402_1005Metric -> Capacitor_SMD:C_0201_0603Metric; MPN GRM155R61A105KE15D -> GRM033R60J105MEA2D
Changed lines of the file:
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@@
   (property "Reference" "C5304" (at 322.58 167.64 0) (effects (font (size 1.27 1.27)) (justify left)))
   (property "Value" "1 µF" (at 322.58 170.18 0) (effects (font (size 1.27 1.27)) (justify left)))
-  (property "Footprint" "Capacitor_SMD:C_0402_1005Metric" (at 320.04 168.91 0) (effects (font (size 1.27 1.27))) (hide yes))
-  (property "Datasheet" "https://www.murata.com/en-us/products/productdetail?partno=GRM155R61A105KE15D" (at 320.04 168.91 0) (effects (font (size 1.27 1.27))) (hide yes))
-  (property "Description" "Capacitor, 1 µF, 10 V, X5R, 0402" (at 320.04 168.91 0) (effects (font (size 1.27 1.27))) (hide yes))
+  (property "Footprint" "Capacitor_SMD:C_0201_0603Metric" (at 320.04 168.91 0) (effects (font (size 1.27 1.27))) (hide yes))
+  (property "Datasheet" "https://www.murata.com/en-us/products/productdetail?partno=GRM033R60J105MEA2D" (at 320.04 168.91 0) (effects (font (size 1.27 1.27))) (hide yes))
+  (property "Description" "Capacitor, 1 µF, 6.3 V, X5R, 0201" (at 320.04 168.91 0) (effects (font (size 1.27 1.27))) (hide yes))
   (property "Manufacturer" "Murata" (at 320.04 168.91 0) (effects (font (size 1.27 1.27))) (hide yes))
-  (property "MPN" "GRM155R61A105KE15D" (at 320.04 168.91 0) (effects (font (size 1.27 1.27))) (hide yes))
+  (property "MPN" "GRM033R60J105MEA2D" (at 320.04 168.91 0) (effects (font (size 1.27 1.27))) (hide yes))
   (property "Block" "blk.fp-connector" (at 320.04 168.91 0) (effects (font (size 1.27 1.27))) (hide yes))
   (pin "1")
