File: board/hardware/t1-main-board/radio-power.kicad_sch (KiCad schematic)
At the start: 25 parts, among them U4701 SN74AXC1T45DCKR, U4702 TPS22919DCKR, U4703 TPS62826DMQR

Commit message: Board: capture blk.current-monitors
Five INA236 on I2C1 (0x40-0x43, 0x48) with their shunts, per power tree
§4.12 and BOM v1 lines 54 and 136. The measured branches are rails of
their own (VSYS_SRC, VSYS_LV_AUDIO, VSYS_AUDIO, VSYS_LV_BL, VSYS_P5V1),
fed through the shunts on this sheet; the charger, audio, backlight and
5.1 V sheets take them. The root's layout may leave a stack level empty,
so the block sits under the notes; IC bboxes hold turned rail values;
passive rows hold a bottom rail's text.

Co-Authored-By: Claude Opus 5.5 <noreply@anthropic.com>
Claude-Session: https://claude.ai/code/session_01Ei262h3TpgY9vyfNLMi5Mn
Parts:
- removed C4701, C4702: 100 nF, Capacitor_SMD:C_0402_1005Metric, symbol Device:C
- removed C4703: 1 µF, Capacitor_SMD:C_0402_1005Metric, symbol Device:C
- removed C4704: 10 µF, Capacitor_SMD:C_0603_1608Metric, symbol Device:C
- removed C4705: 22 µF, Capacitor_SMD:C_0603_1608Metric, symbol Device:C
- removed C4706: 120 pF, Capacitor_SMD:C_0402_1005Metric, symbol Device:C
- removed L4701: 470 nH, T1_Main_Board:L_Wuerth_WE-LHMI_4020, symbol Device:L
- removed R4701, R4702, R4703, R4708: 100 kΩ, Resistor_SMD:R_0402_1005Metric, symbol Device:R
- removed R4704, R4711: 20 mΩ, Resistor_SMD:R_1206_3216Metric, symbol Device:R
- removed R4705: 200 kΩ, Resistor_SMD:R_0603_1608Metric, symbol Device:R
- removed R4706: 100 kΩ, Resistor_SMD:R_0603_1608Metric, symbol Device:R
- removed R4707, R4709: 0 Ω, Resistor_SMD:R_0402_1005Metric, symbol Device:R
- removed R4710: 1 kΩ, Resistor_SMD:R_0603_1608Metric, symbol Device:R
- removed TP4701: WL_3V3_SRC, TestPoint:TestPoint_Pad_D1.0mm, symbol Connector:TestPoint
- removed TP4702: vcc3v3_wl, TestPoint:TestPoint_Pad_D1.0mm, symbol Connector:TestPoint
- removed TP4703: WL_1V8_SRC, TestPoint:TestPoint_Pad_D1.0mm, symbol Connector:TestPoint
- removed TP4704: vcc1v8_wl, TestPoint:TestPoint_Pad_D1.0mm, symbol Connector:TestPoint
- removed U4701: SN74AXC1T45DCKR, Texas_Instruments:Texas_DCK0006A_SC-70-6_1.25x2mm_P0.65mm, symbol Texas_Instruments:SN74AXC1T45DCKR
- removed U4702: TPS22919DCKR, Texas_Instruments:Texas_DCK0006A_SC-70-6_1.25x2mm_P0.65mm, symbol Texas_Instruments:TPS22919DCKR
- removed U4703: TPS62826DMQR, Texas_Instruments:Texas_DMQ0006A_VSON-HR-6_1.5x1.5mm_P0.5mm, symbol Texas_Instruments:TPS62826DMQR
- added C4801, C4802: 100 nF, Capacitor_SMD:C_0402_1005Metric, symbol Device:C
- added C4803: 1 µF, Capacitor_SMD:C_0402_1005Metric, symbol Device:C
- added C4804: 10 µF, Capacitor_SMD:C_0603_1608Metric, symbol Device:C
- added C4805: 22 µF, Capacitor_SMD:C_0603_1608Metric, symbol Device:C
- added C4806: 120 pF, Capacitor_SMD:C_0402_1005Metric, symbol Device:C
- added L4801: 470 nH, T1_Main_Board:L_Wuerth_WE-LHMI_4020, symbol Device:L
- added R4801, R4802, R4803, R4808: 100 kΩ, Resistor_SMD:R_0402_1005Metric, symbol Device:R
- added R4804, R4811: 20 mΩ, Resistor_SMD:R_1206_3216Metric, symbol Device:R
- added R4805: 200 kΩ, Resistor_SMD:R_0603_1608Metric, symbol Device:R
- added R4806: 100 kΩ, Resistor_SMD:R_0603_1608Metric, symbol Device:R
- added R4807, R4809: 0 Ω, Resistor_SMD:R_0402_1005Metric, symbol Device:R
- added R4810: 1 kΩ, Resistor_SMD:R_0603_1608Metric, symbol Device:R
- added TP4801: WL_3V3_SRC, TestPoint:TestPoint_Pad_D1.0mm, symbol Connector:TestPoint
- added TP4802: vcc3v3_wl, TestPoint:TestPoint_Pad_D1.0mm, symbol Connector:TestPoint
- added TP4803: WL_1V8_SRC, TestPoint:TestPoint_Pad_D1.0mm, symbol Connector:TestPoint
- added TP4804: vcc1v8_wl, TestPoint:TestPoint_Pad_D1.0mm, symbol Connector:TestPoint
- added U4801: SN74AXC1T45DCKR, Texas_Instruments:Texas_DCK0006A_SC-70-6_1.25x2mm_P0.65mm, symbol Texas_Instruments:SN74AXC1T45DCKR
- added U4802: TPS22919DCKR, Texas_Instruments:Texas_DCK0006A_SC-70-6_1.25x2mm_P0.65mm, symbol Texas_Instruments:TPS22919DCKR
- added U4803: TPS62826DMQR, Texas_Instruments:Texas_DMQ0006A_VSON-HR-6_1.5x1.5mm_P0.5mm, symbol Texas_Instruments:TPS62826DMQR
Connections:
- net GND: now also C4801.2, C4802.2, C4803.2, C4804.2, C4805.2, R4801.2, R4802.2, R4803.2, R4806.2, R4808.2, R4810.2, U4801.2 (GND), U4802.2 (GND), U4803.4 (GND)
- net VSYS_LV: now also C4804.1, U4803.6 (VIN)
- net WL_1V8_EN: now also R4807.2, R4808.1, R4809.2, U4803.1 (EN)
- net WL_1V8_EN_GPIO: now also R4809.1
- net WL_1V8_FB: now also C4806.2, R4805.2, R4806.1, U4803.3 (FB)
- net WL_1V8_SRC: now also C4805.1, L4801.2, R4811.1, TP4803.1
- net WL_1V8_SW: now also L4801.1, U4803.5 (SW)
- net WL_3V3_SRC: now also R4804.1, TP4801.1, U4802.5 (QOD), U4802.6 (VOUT)
- net WL_PD_HOLD_N: now also R4802.1, U4801.3 (A)
- net WL_PD_N: now also R4801.1, U4801.4 (B)
- net WL_PWR_EN: now also R4803.1, U4802.3 (ON)
- net vcc1v8_wl: now also C4802.1, C4806.1, R4805.1, R4811.2, TP4804.1, U4801.6 (VCCB)
- net vcc3v3_sys: now also C4801.1, C4803.1, U4801.1 (VCCA), U4801.5 (DIR), U4802.1 (IN)
- net vcc3v3_wl: now also R4804.2, R4807.1, R4810.1, TP4802.1

Commit message: Board: capture blk.debug
Debug UART2 (1.8 V) and I2S/DSD pads with ground pads, reset, PMIC and
power-key pads (PCB-T-09), a pad on every spare SoC GPIO whose pinout v1
row names one (the DEBUG bus, on the SoC's right edge), and a rail pad
for each power-tree rail no other sheet probes (PCB-T-02). Each DAC
sheet carries a pad on its MCLK. The spares pinout v1 leaves without a
pad now carry no-connect flags. On the root, facing sheet pins are
joined directly only where the route meets no other symbol.

Co-Authored-By: Claude Opus 5.5 <noreply@anthropic.com>
Claude-Session: https://claude.ai/code/session_01Ei262h3TpgY9vyfNLMi5Mn
Parts:
- removed C4801, C4802: 100 nF, Capacitor_SMD:C_0402_1005Metric, symbol Device:C
- removed C4803: 1 µF, Capacitor_SMD:C_0402_1005Metric, symbol Device:C
- removed C4804: 10 µF, Capacitor_SMD:C_0603_1608Metric, symbol Device:C
- removed C4805: 22 µF, Capacitor_SMD:C_0603_1608Metric, symbol Device:C
- removed C4806: 120 pF, Capacitor_SMD:C_0402_1005Metric, symbol Device:C
- removed L4801: 470 nH, T1_Main_Board:L_Wuerth_WE-LHMI_4020, symbol Device:L
- removed R4801, R4802, R4803, R4808: 100 kΩ, Resistor_SMD:R_0402_1005Metric, symbol Device:R
- removed R4804, R4811: 20 mΩ, Resistor_SMD:R_1206_3216Metric, symbol Device:R
- removed R4805: 200 kΩ, Resistor_SMD:R_0603_1608Metric, symbol Device:R
- removed R4806: 100 kΩ, Resistor_SMD:R_0603_1608Metric, symbol Device:R
- removed R4807, R4809: 0 Ω, Resistor_SMD:R_0402_1005Metric, symbol Device:R
- removed R4810: 1 kΩ, Resistor_SMD:R_0603_1608Metric, symbol Device:R
- removed TP4801: WL_3V3_SRC, TestPoint:TestPoint_Pad_D1.0mm, symbol Connector:TestPoint
- removed TP4802: vcc3v3_wl, TestPoint:TestPoint_Pad_D1.0mm, symbol Connector:TestPoint
- removed TP4803: WL_1V8_SRC, TestPoint:TestPoint_Pad_D1.0mm, symbol Connector:TestPoint
- removed TP4804: vcc1v8_wl, TestPoint:TestPoint_Pad_D1.0mm, symbol Connector:TestPoint
- removed U4801: SN74AXC1T45DCKR, Texas_Instruments:Texas_DCK0006A_SC-70-6_1.25x2mm_P0.65mm, symbol Texas_Instruments:SN74AXC1T45DCKR
- removed U4802: TPS22919DCKR, Texas_Instruments:Texas_DCK0006A_SC-70-6_1.25x2mm_P0.65mm, symbol Texas_Instruments:TPS22919DCKR
- removed U4803: TPS62826DMQR, Texas_Instruments:Texas_DMQ0006A_VSON-HR-6_1.5x1.5mm_P0.5mm, symbol Texas_Instruments:TPS62826DMQR
- added C4901, C4902: 100 nF, Capacitor_SMD:C_0402_1005Metric, symbol Device:C
- added C4903: 1 µF, Capacitor_SMD:C_0402_1005Metric, symbol Device:C
- added C4904: 10 µF, Capacitor_SMD:C_0603_1608Metric, symbol Device:C
- added C4905: 22 µF, Capacitor_SMD:C_0603_1608Metric, symbol Device:C
- added C4906: 120 pF, Capacitor_SMD:C_0402_1005Metric, symbol Device:C
- added L4901: 470 nH, T1_Main_Board:L_Wuerth_WE-LHMI_4020, symbol Device:L
- added R4901, R4902, R4903, R4908: 100 kΩ, Resistor_SMD:R_0402_1005Metric, symbol Device:R
- added R4904, R4911: 20 mΩ, Resistor_SMD:R_1206_3216Metric, symbol Device:R
- added R4905: 200 kΩ, Resistor_SMD:R_0603_1608Metric, symbol Device:R
- added R4906: 100 kΩ, Resistor_SMD:R_0603_1608Metric, symbol Device:R
- added R4907, R4909: 0 Ω, Resistor_SMD:R_0402_1005Metric, symbol Device:R
- added R4910: 1 kΩ, Resistor_SMD:R_0603_1608Metric, symbol Device:R
- added TP4901: WL_3V3_SRC, TestPoint:TestPoint_Pad_D1.0mm, symbol Connector:TestPoint
- added TP4902: vcc3v3_wl, TestPoint:TestPoint_Pad_D1.0mm, symbol Connector:TestPoint
- added TP4903: WL_1V8_SRC, TestPoint:TestPoint_Pad_D1.0mm, symbol Connector:TestPoint
- added TP4904: vcc1v8_wl, TestPoint:TestPoint_Pad_D1.0mm, symbol Connector:TestPoint
- added U4901: SN74AXC1T45DCKR, Texas_Instruments:Texas_DCK0006A_SC-70-6_1.25x2mm_P0.65mm, symbol Texas_Instruments:SN74AXC1T45DCKR
- added U4902: TPS22919DCKR, Texas_Instruments:Texas_DCK0006A_SC-70-6_1.25x2mm_P0.65mm, symbol Texas_Instruments:TPS22919DCKR
- added U4903: TPS62826DMQR, Texas_Instruments:Texas_DMQ0006A_VSON-HR-6_1.5x1.5mm_P0.5mm, symbol Texas_Instruments:TPS62826DMQR
Connections:
- net GND: now also C4901.2, C4902.2, C4903.2, C4904.2, C4905.2, R4901.2, R4902.2, R4903.2, R4906.2, R4908.2, R4910.2, U4901.2 (GND), U4902.2 (GND), U4903.4 (GND)
- net VSYS_LV: now also C4904.1, U4903.6 (VIN)
- net WL_1V8_EN: now also R4907.2, R4908.1, R4909.2, U4903.1 (EN)
- net WL_1V8_EN_GPIO: now also R4909.1
- net WL_1V8_FB: now also C4906.2, R4905.2, R4906.1, U4903.3 (FB)
- net WL_1V8_SRC: now also C4905.1, L4901.2, R4911.1, TP4903.1
- net WL_1V8_SW: now also L4901.1, U4903.5 (SW)
- net WL_3V3_SRC: now also R4904.1, TP4901.1, U4902.5 (QOD), U4902.6 (VOUT)
- net WL_PD_HOLD_N: now also R4902.1, U4901.3 (A)
- net WL_PD_N: now also R4901.1, U4901.4 (B)
- net WL_PWR_EN: now also R4903.1, U4902.3 (ON)
- net vcc1v8_wl: now also C4902.1, C4906.1, R4905.1, R4911.2, TP4904.1, U4901.6 (VCCB)
- net vcc3v3_sys: now also C4901.1, C4903.1, U4901.1 (VCCA), U4901.5 (DIR), U4902.1 (IN)
- net vcc3v3_wl: now also R4904.2, R4907.1, R4910.1, TP4902.1

Commit message: Board: capture blk.mic-ambient and links #34, #35
IM73D122 on PDM CLK1 and SDI1 (BOM v1 line 34, pinout v1 AK2 and 1P2),
LR to ground, 22 Ω clock series, VDD from MIC_1V8 through link #35.
Link #34 on blk.mic-main makes the faceplate branch the rail MIC_1V8_FP
for contact 40 (power tree §4.12, G10). kicad-lib moves to e46bda4 for
the IM73D122, TPS3808G01, SN74LVC1G58 and BAT54 parts.

Co-Authored-By: Claude Opus 5.5 <noreply@anthropic.com>
Claude-Session: https://claude.ai/code/session_01Ei262h3TpgY9vyfNLMi5Mn
Parts:
- removed C4901, C4902: 100 nF, Capacitor_SMD:C_0402_1005Metric, symbol Device:C
- removed C4903: 1 µF, Capacitor_SMD:C_0402_1005Metric, symbol Device:C
- removed C4904: 10 µF, Capacitor_SMD:C_0603_1608Metric, symbol Device:C
- removed C4905: 22 µF, Capacitor_SMD:C_0603_1608Metric, symbol Device:C
- removed C4906: 120 pF, Capacitor_SMD:C_0402_1005Metric, symbol Device:C
- removed L4901: 470 nH, T1_Main_Board:L_Wuerth_WE-LHMI_4020, symbol Device:L
- removed R4901, R4902, R4903, R4908: 100 kΩ, Resistor_SMD:R_0402_1005Metric, symbol Device:R
- removed R4904, R4911: 20 mΩ, Resistor_SMD:R_1206_3216Metric, symbol Device:R
- removed R4905: 200 kΩ, Resistor_SMD:R_0603_1608Metric, symbol Device:R
- removed R4906: 100 kΩ, Resistor_SMD:R_0603_1608Metric, symbol Device:R
- removed R4907, R4909: 0 Ω, Resistor_SMD:R_0402_1005Metric, symbol Device:R
- removed R4910: 1 kΩ, Resistor_SMD:R_0603_1608Metric, symbol Device:R
- removed TP4901: WL_3V3_SRC, TestPoint:TestPoint_Pad_D1.0mm, symbol Connector:TestPoint
- removed TP4902: vcc3v3_wl, TestPoint:TestPoint_Pad_D1.0mm, symbol Connector:TestPoint
- removed TP4903: WL_1V8_SRC, TestPoint:TestPoint_Pad_D1.0mm, symbol Connector:TestPoint
- removed TP4904: vcc1v8_wl, TestPoint:TestPoint_Pad_D1.0mm, symbol Connector:TestPoint
- removed U4901: SN74AXC1T45DCKR, Texas_Instruments:Texas_DCK0006A_SC-70-6_1.25x2mm_P0.65mm, symbol Texas_Instruments:SN74AXC1T45DCKR
- removed U4902: TPS22919DCKR, Texas_Instruments:Texas_DCK0006A_SC-70-6_1.25x2mm_P0.65mm, symbol Texas_Instruments:TPS22919DCKR
- removed U4903: TPS62826DMQR, Texas_Instruments:Texas_DMQ0006A_VSON-HR-6_1.5x1.5mm_P0.5mm, symbol Texas_Instruments:TPS62826DMQR
- added C5001, C5002: 100 nF, Capacitor_SMD:C_0402_1005Metric, symbol Device:C
- added C5003: 1 µF, Capacitor_SMD:C_0402_1005Metric, symbol Device:C
- added C5004: 10 µF, Capacitor_SMD:C_0603_1608Metric, symbol Device:C
- added C5005: 22 µF, Capacitor_SMD:C_0603_1608Metric, symbol Device:C
- added C5006: 120 pF, Capacitor_SMD:C_0402_1005Metric, symbol Device:C
- added L5001: 470 nH, T1_Main_Board:L_Wuerth_WE-LHMI_4020, symbol Device:L
- added R5001, R5002, R5003, R5008: 100 kΩ, Resistor_SMD:R_0402_1005Metric, symbol Device:R
- added R5004, R5011: 20 mΩ, Resistor_SMD:R_1206_3216Metric, symbol Device:R
- added R5005: 200 kΩ, Resistor_SMD:R_0603_1608Metric, symbol Device:R
- added R5006: 100 kΩ, Resistor_SMD:R_0603_1608Metric, symbol Device:R
- added R5007, R5009: 0 Ω, Resistor_SMD:R_0402_1005Metric, symbol Device:R
- added R5010: 1 kΩ, Resistor_SMD:R_0603_1608Metric, symbol Device:R
- added TP5001: WL_3V3_SRC, TestPoint:TestPoint_Pad_D1.0mm, symbol Connector:TestPoint
- added TP5002: vcc3v3_wl, TestPoint:TestPoint_Pad_D1.0mm, symbol Connector:TestPoint
- added TP5003: WL_1V8_SRC, TestPoint:TestPoint_Pad_D1.0mm, symbol Connector:TestPoint
- added TP5004: vcc1v8_wl, TestPoint:TestPoint_Pad_D1.0mm, symbol Connector:TestPoint
- added U5001: SN74AXC1T45DCKR, Texas_Instruments:Texas_DCK0006A_SC-70-6_1.25x2mm_P0.65mm, symbol Texas_Instruments:SN74AXC1T45DCKR
- added U5002: TPS22919DCKR, Texas_Instruments:Texas_DCK0006A_SC-70-6_1.25x2mm_P0.65mm, symbol Texas_Instruments:TPS22919DCKR
- added U5003: TPS62826DMQR, Texas_Instruments:Texas_DMQ0006A_VSON-HR-6_1.5x1.5mm_P0.5mm, symbol Texas_Instruments:TPS62826DMQR
Connections:
- net GND: now also C5001.2, C5002.2, C5003.2, C5004.2, C5005.2, R5001.2, R5002.2, R5003.2, R5006.2, R5008.2, R5010.2, U5001.2 (GND), U5002.2 (GND), U5003.4 (GND)
- net VSYS_LV: now also C5004.1, U5003.6 (VIN)
- net WL_1V8_EN: now also R5007.2, R5008.1, R5009.2, U5003.1 (EN)
- net WL_1V8_EN_GPIO: now also R5009.1
- net WL_1V8_FB: now also C5006.2, R5005.2, R5006.1, U5003.3 (FB)
- net WL_1V8_SRC: now also C5005.1, L5001.2, R5011.1, TP5003.1
- net WL_1V8_SW: now also L5001.1, U5003.5 (SW)
- net WL_3V3_SRC: now also R5004.1, TP5001.1, U5002.5 (QOD), U5002.6 (VOUT)
- net WL_PD_HOLD_N: now also R5002.1, U5001.3 (A)
- net WL_PD_N: now also R5001.1, U5001.4 (B)
- net WL_PWR_EN: now also R5003.1, U5002.3 (ON)
- net vcc1v8_wl: now also C5002.1, C5006.1, R5005.1, R5011.2, TP5004.1, U5001.6 (VCCB)
- net vcc3v3_sys: now also C5001.1, C5003.1, U5001.1 (VCCA), U5001.5 (DIR), U5002.1 (IN)
- net vcc3v3_wl: now also R5004.2, R5007.1, R5010.1, TP5002.1

Commit message: Board: capture blk.maskrom
Power + Vol- at a cold power-on pull eMMC D0 low inside the TPS3808G01
boot window (BOM v1 lines 35, 78, 97, 98; sim/maskrom): SENSE 280k/100k,
CT 390 nF, WINDOW_N with its pad, SN74LVC1G57 and SN74LVC1G58 on
vcca1v8_pmu, BAT54 from PWRON_N, DMG1012T through 1 kΩ to EMMC_D0.
Every block in use now has its sheet; the README states the remaining
single-pin nets.

Co-Authored-By: Claude Opus 5.5 <noreply@anthropic.com>
Claude-Session: https://claude.ai/code/session_01Ei262h3TpgY9vyfNLMi5Mn
Parts:
- removed C5001, C5002: 100 nF, Capacitor_SMD:C_0402_1005Metric, symbol Device:C
- removed C5003: 1 µF, Capacitor_SMD:C_0402_1005Metric, symbol Device:C
- removed C5004: 10 µF, Capacitor_SMD:C_0603_1608Metric, symbol Device:C
- removed C5005: 22 µF, Capacitor_SMD:C_0603_1608Metric, symbol Device:C
- removed C5006: 120 pF, Capacitor_SMD:C_0402_1005Metric, symbol Device:C
- removed L5001: 470 nH, T1_Main_Board:L_Wuerth_WE-LHMI_4020, symbol Device:L
- removed R5001, R5002, R5003, R5008: 100 kΩ, Resistor_SMD:R_0402_1005Metric, symbol Device:R
- removed R5004, R5011: 20 mΩ, Resistor_SMD:R_1206_3216Metric, symbol Device:R
- removed R5005: 200 kΩ, Resistor_SMD:R_0603_1608Metric, symbol Device:R
- removed R5006: 100 kΩ, Resistor_SMD:R_0603_1608Metric, symbol Device:R
- removed R5007, R5009: 0 Ω, Resistor_SMD:R_0402_1005Metric, symbol Device:R
- removed R5010: 1 kΩ, Resistor_SMD:R_0603_1608Metric, symbol Device:R
- removed TP5001: WL_3V3_SRC, TestPoint:TestPoint_Pad_D1.0mm, symbol Connector:TestPoint
- removed TP5002: vcc3v3_wl, TestPoint:TestPoint_Pad_D1.0mm, symbol Connector:TestPoint
- removed TP5003: WL_1V8_SRC, TestPoint:TestPoint_Pad_D1.0mm, symbol Connector:TestPoint
- removed TP5004: vcc1v8_wl, TestPoint:TestPoint_Pad_D1.0mm, symbol Connector:TestPoint
- removed U5001: SN74AXC1T45DCKR, Texas_Instruments:Texas_DCK0006A_SC-70-6_1.25x2mm_P0.65mm, symbol Texas_Instruments:SN74AXC1T45DCKR
- removed U5002: TPS22919DCKR, Texas_Instruments:Texas_DCK0006A_SC-70-6_1.25x2mm_P0.65mm, symbol Texas_Instruments:TPS22919DCKR
- removed U5003: TPS62826DMQR, Texas_Instruments:Texas_DMQ0006A_VSON-HR-6_1.5x1.5mm_P0.5mm, symbol Texas_Instruments:TPS62826DMQR
- added C5101, C5102: 100 nF, Capacitor_SMD:C_0402_1005Metric, symbol Device:C
- added C5103: 1 µF, Capacitor_SMD:C_0402_1005Metric, symbol Device:C
- added C5104: 10 µF, Capacitor_SMD:C_0603_1608Metric, symbol Device:C
- added C5105: 22 µF, Capacitor_SMD:C_0603_1608Metric, symbol Device:C
- added C5106: 120 pF, Capacitor_SMD:C_0402_1005Metric, symbol Device:C
- added L5101: 470 nH, T1_Main_Board:L_Wuerth_WE-LHMI_4020, symbol Device:L
- added R5101, R5102, R5103, R5108: 100 kΩ, Resistor_SMD:R_0402_1005Metric, symbol Device:R
- added R5104, R5111: 20 mΩ, Resistor_SMD:R_1206_3216Metric, symbol Device:R
- added R5105: 200 kΩ, Resistor_SMD:R_0603_1608Metric, symbol Device:R
- added R5106: 100 kΩ, Resistor_SMD:R_0603_1608Metric, symbol Device:R
- added R5107, R5109: 0 Ω, Resistor_SMD:R_0402_1005Metric, symbol Device:R
- added R5110: 1 kΩ, Resistor_SMD:R_0603_1608Metric, symbol Device:R
- added TP5101: WL_3V3_SRC, TestPoint:TestPoint_Pad_D1.0mm, symbol Connector:TestPoint
- added TP5102: vcc3v3_wl, TestPoint:TestPoint_Pad_D1.0mm, symbol Connector:TestPoint
- added TP5103: WL_1V8_SRC, TestPoint:TestPoint_Pad_D1.0mm, symbol Connector:TestPoint
- added TP5104: vcc1v8_wl, TestPoint:TestPoint_Pad_D1.0mm, symbol Connector:TestPoint
- added U5101: SN74AXC1T45DCKR, Texas_Instruments:Texas_DCK0006A_SC-70-6_1.25x2mm_P0.65mm, symbol Texas_Instruments:SN74AXC1T45DCKR
- added U5102: TPS22919DCKR, Texas_Instruments:Texas_DCK0006A_SC-70-6_1.25x2mm_P0.65mm, symbol Texas_Instruments:TPS22919DCKR
- added U5103: TPS62826DMQR, Texas_Instruments:Texas_DMQ0006A_VSON-HR-6_1.5x1.5mm_P0.5mm, symbol Texas_Instruments:TPS62826DMQR
Connections:
- net GND: now also C5101.2, C5102.2, C5103.2, C5104.2, C5105.2, R5101.2, R5102.2, R5103.2, R5106.2, R5108.2, R5110.2, U5101.2 (GND), U5102.2 (GND), U5103.4 (GND)
- net VSYS_LV: now also C5104.1, U5103.6 (VIN)
- net WL_1V8_EN: now also R5107.2, R5108.1, R5109.2, U5103.1 (EN)
- net WL_1V8_EN_GPIO: now also R5109.1
- net WL_1V8_FB: now also C5106.2, R5105.2, R5106.1, U5103.3 (FB)
- net WL_1V8_SRC: now also C5105.1, L5101.2, R5111.1, TP5103.1
- net WL_1V8_SW: now also L5101.1, U5103.5 (SW)
- net WL_3V3_SRC: now also R5104.1, TP5101.1, U5102.5 (QOD), U5102.6 (VOUT)
- net WL_PD_HOLD_N: now also R5102.1, U5101.3 (A)
- net WL_PD_N: now also R5101.1, U5101.4 (B)
- net WL_PWR_EN: now also R5103.1, U5102.3 (ON)
- net vcc1v8_wl: now also C5102.1, C5106.1, R5105.1, R5111.2, TP5104.1, U5101.6 (VCCB)
- net vcc3v3_sys: now also C5101.1, C5103.1, U5101.1 (VCCA), U5101.5 (DIR), U5102.1 (IN)
- net vcc3v3_wl: now also R5104.2, R5107.1, R5110.1, TP5102.1
