File: board/hardware/t1-main-board/radio-power.kicad_sch (KiCad schematic)
At the start: 25 parts, among them U5101 SN74AXC1T45DCKR, U5102 TPS22919DCKR, U5103 TPS62826DMQR

Commit message: Compaction: lower inductors, 0201 decoupling, 0.8 mm signal test pads
A matrix tool (hardware/studies/compaction) checks each candidate against
the design's stresses: same inductance, design peak <= 70 % and the
converter's maximum limit <= 100 % of Isat (30 % drop), height zones,
ratings at least twice the rail, PCB-D-06; sourcing outcome per part.

Applied (placement v1 decision 12, BOM v1.15):
- L601, L4401: XGL4015-102MEC (1.5 mm) for XAL/XGL4020-102MEC (2.1 mm);
- L1001, L5101: XGL4015-471MEC (1.5 mm) for Wurth 744373240047, on the
  stock XxL4020 land (the Wurth land was never drawn);
- L1201 is 1.2 mm (XGL4012, per-MPN heights): it moves next to the SoC;
- 58 x 100 nF decoupling on rails <= 3.3 V in core/IO/radio: 0201;
- 51 test pads on signal nets: 0.8 mm (PCB-D-06 v0.16, JLCPCB guide).
Kept: L901, L2802 (XGL4015 at 103 % of Isat at the limit); no thinner
0805/1206 capacitor passes (obsolete, NRND or unlisted).

Board need 113 % -> 111 % (core band 227 -> 203 %, power band 258 ->
233 %, radio band 19 -> 0 %); only C904 still relies on PCB-Z-04.
ERC 0 errors, craft Q1 met, DRC 0 errors (605 warnings), pcb and study
tests pass, rules test board PASS.

Co-Authored-By: Claude Opus 5.5 <noreply@anthropic.com>
Claude-Session: https://claude.ai/code/session_01Ei262h3TpgY9vyfNLMi5Mn
Parts:
- C5101, C5102: footprint Capacitor_SMD:C_0402_1005Metric -> Capacitor_SMD:C_0201_0603Metric; MPN GRM155R71C104KA88D -> GRM033R61A104KE15D
- L5101: footprint T1_Main_Board:L_Wuerth_WE-LHMI_4020 -> Inductor_SMD:L_Coilcraft_XxL4020; MPN 744373240047 -> XGL4015-471MEC; Manufacturer Wurth Elektronik -> Coilcraft; Second_Source Coilcraft XFL4015-471MEC (land compatibility UNVERIFIED, BO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 -> Wurth 744373240047 (other land, 1.8 mm: bands only; BOM v1 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; Spec Isat 10.4 A -> Isat 10.5 A
Changed lines of the file:
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@@
   (property "Reference" "C5101" (at 110.49 58.42 0) (effects (font (size 1.27 1.27)) (justify left)))
   (property "Value" "100 nF" (at 110.49 60.96 0) (effects (font (size 1.27 1.27)) (justify left)))
-  (property "Footprint" "Capacitor_SMD:C_0402_1005Metric" (at 107.95 59.69 0) (effects (font (size 1.27 1.27))) (hide yes))
-  (property "Datasheet" "https://www.murata.com/en-us/products/productdetail?partno=GRM155R71C104KA88D" (at 107.95 59.69 0) (effects (font (size 1.27 1.27))) (hide yes))
-  (property "Description" "Capacitor, 100 nF, 16 V, X7R, 0402" (at 107.95 59.69 0) (effects (font (size 1.27 1.27))) (hide yes))
+  (property "Footprint" "Capacitor_SMD:C_0201_0603Metric" (at 107.95 59.69 0) (effects (font (size 1.27 1.27))) (hide yes))
+  (property "Datasheet" "https://www.murata.com/en-us/products/productdetail?partno=GRM033R61A104KE15D" (at 107.95 59.69 0) (effects (font (size 1.27 1.27))) (hide yes))
+  (property "Description" "Capacitor, 100 nF, 10 V, X5R, 0201" (at 107.95 59.69 0) (effects (font (size 1.27 1.27))) (hide yes))
   (property "Manufacturer" "Murata" (at 107.95 59.69 0) (effects (font (size 1.27 1.27))) (hide yes))
-  (property "MPN" "GRM155R71C104KA88D" (at 107.95 59.69 0) (effects (font (size 1.27 1.27))) (hide yes))
+  (property "MPN" "GRM033R61A104KE15D" (at 107.95 59.69 0) (effects (font (size 1.27 1.27))) (hide yes))
   (property "Block" "blk.radio-power" (at 107.95 59.69 0) (effects (font (size 1.27 1.27))) (hide yes))
   (pin "1")
@@
   (property "Reference" "C5102" (at 128.27 58.42 0) (effects (font (size 1.27 1.27)) (justify left)))
   (property "Value" "100 nF" (at 128.27 60.96 0) (effects (font (size 1.27 1.27)) (justify left)))
-  (property "Footprint" "Capacitor_SMD:C_0402_1005Metric" (at 125.73 59.69 0) (effects (font (size 1.27 1.27))) (hide yes))
-  (property "Datasheet" "https://www.murata.com/en-us/products/productdetail?partno=GRM155R71C104KA88D" (at 125.73 59.69 0) (effects (font (size 1.27 1.27))) (hide yes))
-  (property "Description" "Capacitor, 100 nF, 16 V, X7R, 0402" (at 125.73 59.69 0) (effects (font (size 1.27 1.27))) (hide yes))
+  (property "Footprint" "Capacitor_SMD:C_0201_0603Metric" (at 125.73 59.69 0) (effects (font (size 1.27 1.27))) (hide yes))
+  (property "Datasheet" "https://www.murata.com/en-us/products/productdetail?partno=GRM033R61A104KE15D" (at 125.73 59.69 0) (effects (font (size 1.27 1.27))) (hide yes))
+  (property "Description" "Capacitor, 100 nF, 10 V, X5R, 0201" (at 125.73 59.69 0) (effects (font (size 1.27 1.27))) (hide yes))
   (property "Manufacturer" "Murata" (at 125.73 59.69 0) (effects (font (size 1.27 1.27))) (hide yes))
-  (property "MPN" "GRM155R71C104KA88D" (at 125.73 59.69 0) (effects (font (size 1.27 1.27))) (hide yes))
+  (property "MPN" "GRM033R61A104KE15D" (at 125.73 59.69 0) (effects (font (size 1.27 1.27))) (hide yes))
   (property "Block" "blk.radio-power" (at 125.73 59.69 0) (effects (font (size 1.27 1.27))) (hide yes))
   (pin "1")
@@
   (property "Reference" "L5101" (at 185.42 115.57 90) (effects (font (size 1.27 1.27))))
   (property "Value" "470 nH" (at 185.42 120.65 90) (effects (font (size 1.27 1.27))))
-  (property "Spec" "Isat 10.4 A" (at 185.42 123.19 90) (effects (font (size 1.27 1.27))))
-  (property "Footprint" "T1_Main_Board:L_Wuerth_WE-LHMI_4020" (at 185.42 118.11 0) (effects (font (size 1.27 1.27))) (hide yes))
-  (property "Datasheet" "https://www.we-online.com/components/products/datasheet/744373240047.pdf" (at 185.42 118.11 0) (effects (font (size 1.27 1.27))) (hide yes))
-  (property "Description" "Power inductor, 0.47 uH, IR 8.7 A, Isat 10.4 A (10 % drop), 4.45 x 4.06 x 1.8 mm" (at 185.42 118.11 0) (effects (font (size 1.27 1.27))) (hide yes))
-  (property "Manufacturer" "Wurth Elektronik" (at 185.42 118.11 0) (effects (font (size 1.27 1.27))) (hide yes))
-  (property "MPN" "744373240047" (at 185.42 118.11 0) (effects (font (size 1.27 1.27))) (hide yes))
-  (property "Second_Source" "Coilcraft XFL4015-471MEC (land compatibility UNVERIFIED, BOM v1 line 106)" (at 185.42 118.11 0) (effects (font (size 1.27 1.27))) (hide yes))
+  (property "Spec" "Isat 10.5 A" (at 185.42 123.19 90) (effects (font (size 1.27 1.27))))
+  (property "Footprint" "Inductor_SMD:L_Coilcraft_XxL4020" (at 185.42 118.11 0) (effects (font (size 1.27 1.27))) (hide yes))
+  (property "Datasheet" "https://coilcraft.com/getmedia/c5d04454-742d-473e-8b80-06c97338c587/xgl4015.pdf" (at 185.42 118.11 0) (effects (font (size 1.27 1.27))) (hide yes))
+  (property "Description" "Power inductor, 0.47 uH 20 %, Isat 10.5 A (30 % drop), Irms 9.6 A, 4.0 x 4.0 x 1.5 mm" (at 185.42 118.11 0) (effects (font (size 1.27 1.27))) (hide yes))
+  (property "Manufacturer" "Coilcraft" (at 185.42 118.11 0) (effects (font (size 1.27 1.27))) (hide yes))
+  (property "MPN" "XGL4015-471MEC" (at 185.42 118.11 0) (effects (font (size 1.27 1.27))) (hide yes))
+  (property "Second_Source" "Wurth 744373240047 (other land, 1.8 mm: bands only; BOM v1 line 106)" (at 185.42 118.11 0) (effects (font (size 1.27 1.27))) (hide yes))
   (property "Block" "blk.radio-power" (at 185.42 118.11 0) (effects (font (size 1.27 1.27))) (hide yes))
   (pin "1")

Commit message: Board on libs v0.2.0: lower-case kebab vendor keys (HL-13)
The libs submodule moves to v0.2.0 (5f24483). Every library nickname in
the generator, the placement tool and the floorplan study follows the
key table (Texas_Instruments -> texas-instruments, OpenDAP_Device ->
opendap-generic, Rockchip and Rockchip_PMIC -> rockchip, ...); the
library tables are written from the files. Schematic and board
regenerated.

Checks: ERC 0 errors (warnings unchanged); DRC 0 errors, 605 warnings,
the same counts by type, schematic parity 0; every placement identical;
craft Q1 met; pcb tests pass; STEP export resolves every libs 3D model
(the 27 parts without a model are KiCad stock lands that have none).

Co-Authored-By: Claude Opus 5.5 <noreply@anthropic.com>
Claude-Session: https://claude.ai/code/session_01Ei262h3TpgY9vyfNLMi5Mn
Parts:
- U5101: footprint Texas_Instruments:Texas_DCK0006A_SC-70-6_1.25x2mm_P0.65mm -> texas-instruments:Texas_DCK0006A_SC-70-6_1.25x2mm_P0.65mm; symbol Texas_Instruments:SN74AXC1T45DCKR -> texas-instruments:SN74AXC1T45DCKR
- U5102: footprint Texas_Instruments:Texas_DCK0006A_SC-70-6_1.25x2mm_P0.65mm -> texas-instruments:Texas_DCK0006A_SC-70-6_1.25x2mm_P0.65mm; symbol Texas_Instruments:TPS22919DCKR -> texas-instruments:TPS22919DCKR
- U5103: footprint Texas_Instruments:Texas_DMQ0006A_VSON-HR-6_1.5x1.5mm_P0.5mm -> texas-instruments:Texas_DMQ0006A_VSON-HR-6_1.5x1.5mm_P0.5mm; symbol Texas_Instruments:TPS62826DMQR -> texas-instruments:TPS62826DMQR
Changed lines of the file:
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@@
 (paper "A3")
 (title_block (title "Radio: rails and PDn hold") (date "2026-10-25") (rev "A") (company "The OpenDAP Project") (comment 1 "blk.radio-power") (comment 2 "AVDD33 switch, AVDD18 buck, links #11 and #12, the PDn hold translator"))
-(symbol (lib_id "Texas_Instruments:SN74AXC1T45DCKR") (at 80.01 71.12 0) (unit 1) (body_style 1) (exclude_from_sim no) (in_bom yes) (on_board yes) (dnp no)
+(symbol (lib_id "texas-instruments:SN74AXC1T45DCKR") (at 80.01 71.12 0) (unit 1) (body_style 1) (exclude_from_sim no) (in_bom yes) (on_board yes) (dnp no)
   (property "Reference" "U5101" (at 83.82 55.88 0) (effects (font (size 1.27 1.27)) (justify left)))
   (property "Value" "SN74AXC1T45DCKR" (at 83.82 53.34 0) (effects (font (size 1.27 1.27)) (justify left)))
-  (property "Footprint" "Texas_Instruments:Texas_DCK0006A_SC-70-6_1.25x2mm_P0.65mm" (at 80.01 71.12 0) (effects (font (size 1.27 1.27))) (hide yes))
+  (property "Footprint" "texas-instruments:Texas_DCK0006A_SC-70-6_1.25x2mm_P0.65mm" (at 80.01 71.12 0) (effects (font (size 1.27 1.27))) (hide yes))
   (property "Datasheet" "https://www.ti.com/lit/ds/symlink/sn74axc1t45.pdf" (at 80.01 71.12 0) (effects (font (size 1.27 1.27))) (hide yes))
   (property "Description" "Single-bit dual-supply bus transceiver, 0.65-3.6 V on each port, direction pin referenced to VCCA, SOT/SC-70-6 (DCK0006A)" (at 80.01 71.12 0) (effects (font (size 1.27 1.27))) (hide yes))
@@
 (rectangle (start 22.86 35.56) (end 167.64 97.79) (stroke (width 0) (type dash)) (fill (type none)))
 (text "PDn hold translator: SN74AXC1T45 (line 148)" (exclude_from_sim no) (at 24.13 34.29 0) (effects (font (size 2.54 2.54)) (justify left bottom)))
-(symbol (lib_id "Texas_Instruments:TPS22919DCKR") (at 201.93 58.42 0) (unit 1) (body_style 1) (exclude_from_sim no) (in_bom yes) (on_board yes) (dnp no)
+(symbol (lib_id "texas-instruments:TPS22919DCKR") (at 201.93 58.42 0) (unit 1) (body_style 1) (exclude_from_sim no) (in_bom yes) (on_board yes) (dnp no)
   (property "Reference" "U5102" (at 194.31 43.18 0) (effects (font (size 1.27 1.27)) (justify left)))
   (property "Value" "TPS22919DCKR" (at 194.31 40.64 0) (effects (font (size 1.27 1.27)) (justify left)))
-  (property "Footprint" "Texas_Instruments:Texas_DCK0006A_SC-70-6_1.25x2mm_P0.65mm" (at 201.93 58.42 0) (effects (font (size 1.27 1.27))) (hide yes))
+  (property "Footprint" "texas-instruments:Texas_DCK0006A_SC-70-6_1.25x2mm_P0.65mm" (at 201.93 58.42 0) (effects (font (size 1.27 1.27))) (hide yes))
   (property "Datasheet" "https://www.ti.com/lit/ds/symlink/tps22919.pdf" (at 201.93 58.42 0) (effects (font (size 1.27 1.27))) (hide yes))
   (property "Description" "Load switch, 1.6-5.5 V, 1.5 A, 90 mOhm, controlled rise time, short-circuit protection, adjustable quick output discharge, SOT/SC-70-6 (DCK0006A)" (at 201.93 58.42 0) (effects (font (size 1.27 1.27))) (hide yes))
@@
   (instances (project "t1-main-board" (path "/7746052e-d7f9-59ad-ba73-bd2b74439529/afc06401-35b4-58d1-93ac-49cd5ed4743d/835da069-84bd-5d4e-910c-ee72eb43e662" (reference "#FLG0032") (unit 1))))
 )
-(symbol (lib_id "Texas_Instruments:TPS62826DMQR") (at 46.99 135.89 0) (unit 1) (body_style 1) (exclude_from_sim no) (in_bom yes) (on_board yes) (dnp no)
+(symbol (lib_id "texas-instruments:TPS62826DMQR") (at 46.99 135.89 0) (unit 1) (body_style 1) (exclude_from_sim no) (in_bom yes) (on_board yes) (dnp no)
   (property "Reference" "U5103" (at 48.26 118.11 0) (effects (font (size 1.27 1.27)) (justify left)))
   (property "Value" "TPS62826DMQR" (at 48.26 115.57 0) (effects (font (size 1.27 1.27)) (justify left)))
-  (property "Footprint" "Texas_Instruments:Texas_DMQ0006A_VSON-HR-6_1.5x1.5mm_P0.5mm" (at 46.99 135.89 0) (effects (font (size 1.27 1.27))) (hide yes))
+  (property "Footprint" "texas-instruments:Texas_DMQ0006A_VSON-HR-6_1.5x1.5mm_P0.5mm" (at 46.99 135.89 0) (effects (font (size 1.27 1.27))) (hide yes))
   (property "Datasheet" "https://www.ti.com/lit/ds/symlink/tps62826.pdf" (at 46.99 135.89 0) (effects (font (size 1.27 1.27))) (hide yes))
   (property "Description" "3 A synchronous step-down converter, 2.4-5.5 V input, 0.6-4.0 V adjustable output, power save mode, power good, 100 % duty cycle, VSON-HR-6 (DMQ0006A) 1.5 x 1.5 mm" (at 46.99 135.89 0) (effects (font (size 1.27 1.27))) (hide yes))

Commit message: Board in the 62.5 x 95.0 mm body: ADR 0025, outline 59.1 x 91.6, 0201 swaps
ADR 0025 supersedes ADR 0016 for t1 ADR 0006's body: board outline from
the body, 1.2 mm walls and 0.5 mm clearance; height zones and stack
restated unchanged; the speaker on a case shelf (PCB-Z-09); pocket
reliefs at the 4.4 mm jack, the microSD (DM3AT push-push kept) and the
side buttons; the audio 0603 -> 0402 swap gated by t1 V2-A08; reserve
(NFC reader, then TPM) recorded, not applied.

- pcb/geometry.py derives the outline from BODY, WALL and CLEARANCE;
  the pocket, display and fixed parts keep their device-frame positions;
  holes keep their edge distance; the speaker shadow becomes a 1.5 mm
  shelf height area (placement, checks, occupancy).
- build.py reports pocket reliefs and routing room; C904 unfixed (it
  now finds back room, so PCB-Z-04 carries no part).
- Generator: parts.area_swap puts 121 generic 0402 resistors (outside
  audio and VBUS paths, >= 10 ohm) and five 100 nF signal capacitors in
  0201 (BOM v1.16); schematic and board regenerated.
- Result: 1,012/1,012 placed, 98.8 % by the floorplan method (was 111 %),
  factor left 1.68 (was 1.49); DRC 0 errors, ERC 0 errors, 0 check
  findings, pcb tests 20/20, schematic craft Q1 met.
- Specs: PCB constraints v0.17 (M-01, M-02, M-08, Z-02, Z-06 to Z-09,
  R-07), placement v1.1 (section 3, decisions 4 and 13, checks, open
  items with the gated swaps and the reserve), floorplan v1 section 1,
  BOM v1.16.

Co-Authored-By: Claude Opus 5.5 <noreply@anthropic.com>
Claude-Session: https://claude.ai/code/session_01Ei262h3TpgY9vyfNLMi5Mn
Parts:
- R5101, R5102, R5103, R5108: footprint Resistor_SMD:R_0402_1005Metric -> Resistor_SMD:R_0201_0603Metric; MPN RC0402FR-07100KL -> RC0201FR-07100KL
Changed lines of the file:
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@@
   (property "Reference" "R5101" (at 140.97 58.42 0) (effects (font (size 1.27 1.27)) (justify left)))
   (property "Value" "100 kΩ" (at 140.97 60.96 0) (effects (font (size 1.27 1.27)) (justify left)))
-  (property "Footprint" "Resistor_SMD:R_0402_1005Metric" (at 139.7 59.69 0) (effects (font (size 1.27 1.27))) (hide yes))
-  (property "Datasheet" "https://yageogroup.com/en/ProductSearch/PartNumberSearch?part=RC0402FR-07100KL" (at 139.7 59.69 0) (effects (font (size 1.27 1.27))) (hide yes))
-  (property "Description" "Resistor, 100 kΩ, 1 %, 1/16 W, 0402" (at 139.7 59.69 0) (effects (font (size 1.27 1.27))) (hide yes))
+  (property "Footprint" "Resistor_SMD:R_0201_0603Metric" (at 139.7 59.69 0) (effects (font (size 1.27 1.27))) (hide yes))
+  (property "Datasheet" "https://yageogroup.com/en/ProductSearch/PartNumberSearch?part=RC0201FR-07100KL" (at 139.7 59.69 0) (effects (font (size 1.27 1.27))) (hide yes))
+  (property "Description" "Resistor, 100 kΩ, 1 %, 1/20 W, 0201" (at 139.7 59.69 0) (effects (font (size 1.27 1.27))) (hide yes))
   (property "Manufacturer" "YAGEO" (at 139.7 59.69 0) (effects (font (size 1.27 1.27))) (hide yes))
-  (property "MPN" "RC0402FR-07100KL" (at 139.7 59.69 0) (effects (font (size 1.27 1.27))) (hide yes))
+  (property "MPN" "RC0201FR-07100KL" (at 139.7 59.69 0) (effects (font (size 1.27 1.27))) (hide yes))
   (property "Block" "blk.radio-power" (at 139.7 59.69 0) (effects (font (size 1.27 1.27))) (hide yes))
   (pin "1")
@@
   (property "Reference" "R5102" (at 154.94 58.42 0) (effects (font (size 1.27 1.27)) (justify left)))
   (property "Value" "100 kΩ" (at 154.94 60.96 0) (effects (font (size 1.27 1.27)) (justify left)))
-  (property "Footprint" "Resistor_SMD:R_0402_1005Metric" (at 153.67 59.69 0) (effects (font (size 1.27 1.27))) (hide yes))
-  (property "Datasheet" "https://yageogroup.com/en/ProductSearch/PartNumberSearch?part=RC0402FR-07100KL" (at 153.67 59.69 0) (effects (font (size 1.27 1.27))) (hide yes))
-  (property "Description" "Resistor, 100 kΩ, 1 %, 1/16 W, 0402" (at 153.67 59.69 0) (effects (font (size 1.27 1.27))) (hide yes))
+  (property "Footprint" "Resistor_SMD:R_0201_0603Metric" (at 153.67 59.69 0) (effects (font (size 1.27 1.27))) (hide yes))
+  (property "Datasheet" "https://yageogroup.com/en/ProductSearch/PartNumberSearch?part=RC0201FR-07100KL" (at 153.67 59.69 0) (effects (font (size 1.27 1.27))) (hide yes))
+  (property "Description" "Resistor, 100 kΩ, 1 %, 1/20 W, 0201" (at 153.67 59.69 0) (effects (font (size 1.27 1.27))) (hide yes))
   (property "Manufacturer" "YAGEO" (at 153.67 59.69 0) (effects (font (size 1.27 1.27))) (hide yes))
-  (property "MPN" "RC0402FR-07100KL" (at 153.67 59.69 0) (effects (font (size 1.27 1.27))) (hide yes))
+  (property "MPN" "RC0201FR-07100KL" (at 153.67 59.69 0) (effects (font (size 1.27 1.27))) (hide yes))
   (property "Block" "blk.radio-power" (at 153.67 59.69 0) (effects (font (size 1.27 1.27))) (hide yes))
   (pin "1")
@@
   (property "Reference" "R5103" (at 246.38 54.61 0) (effects (font (size 1.27 1.27)) (justify left)))
   (property "Value" "100 kΩ" (at 246.38 57.15 0) (effects (font (size 1.27 1.27)) (justify left)))
-  (property "Footprint" "Resistor_SMD:R_0402_1005Metric" (at 245.11 55.88 0) (effects (font (size 1.27 1.27))) (hide yes))
-  (property "Datasheet" "https://yageogroup.com/en/ProductSearch/PartNumberSearch?part=RC0402FR-07100KL" (at 245.11 55.88 0) (effects (font (size 1.27 1.27))) (hide yes))
-  (property "Description" "Resistor, 100 kΩ, 1 %, 1/16 W, 0402" (at 245.11 55.88 0) (effects (font (size 1.27 1.27))) (hide yes))
+  (property "Footprint" "Resistor_SMD:R_0201_0603Metric" (at 245.11 55.88 0) (effects (font (size 1.27 1.27))) (hide yes))
+  (property "Datasheet" "https://yageogroup.com/en/ProductSearch/PartNumberSearch?part=RC0201FR-07100KL" (at 245.11 55.88 0) (effects (font (size 1.27 1.27))) (hide yes))
+  (property "Description" "Resistor, 100 kΩ, 1 %, 1/20 W, 0201" (at 245.11 55.88 0) (effects (font (size 1.27 1.27))) (hide yes))
   (property "Manufacturer" "YAGEO" (at 245.11 55.88 0) (effects (font (size 1.27 1.27))) (hide yes))
-  (property "MPN" "RC0402FR-07100KL" (at 245.11 55.88 0) (effects (font (size 1.27 1.27))) (hide yes))
+  (property "MPN" "RC0201FR-07100KL" (at 245.11 55.88 0) (effects (font (size 1.27 1.27))) (hide yes))
   (property "Block" "blk.radio-power" (at 245.11 55.88 0) (effects (font (size 1.27 1.27))) (hide yes))
   (pin "1")
@@
   (property "Reference" "R5108" (at 87.63 166.37 0) (effects (font (size 1.27 1.27)) (justify left)))
   (property "Value" "100 kΩ" (at 87.63 168.91 0) (effects (font (size 1.27 1.27)) (justify left)))
-  (property "Footprint" "Resistor_SMD:R_0402_1005Metric" (at 86.36 167.64 0) (effects (font (size 1.27 1.27))) (hide yes))
-  (property "Datasheet" "https://yageogroup.com/en/ProductSearch/PartNumberSearch?part=RC0402FR-07100KL" (at 86.36 167.64 0) (effects (font (size 1.27 1.27))) (hide yes))
-  (property "Description" "Resistor, 100 kΩ, 1 %, 1/16 W, 0402" (at 86.36 167.64 0) (effects (font (size 1.27 1.27))) (hide yes))
+  (property "Footprint" "Resistor_SMD:R_0201_0603Metric" (at 86.36 167.64 0) (effects (font (size 1.27 1.27))) (hide yes))
+  (property "Datasheet" "https://yageogroup.com/en/ProductSearch/PartNumberSearch?part=RC0201FR-07100KL" (at 86.36 167.64 0) (effects (font (size 1.27 1.27))) (hide yes))
+  (property "Description" "Resistor, 100 kΩ, 1 %, 1/20 W, 0201" (at 86.36 167.64 0) (effects (font (size 1.27 1.27))) (hide yes))
   (property "Manufacturer" "YAGEO" (at 86.36 167.64 0) (effects (font (size 1.27 1.27))) (hide yes))
-  (property "MPN" "RC0402FR-07100KL" (at 86.36 167.64 0) (effects (font (size 1.27 1.27))) (hide yes))
+  (property "MPN" "RC0201FR-07100KL" (at 86.36 167.64 0) (effects (font (size 1.27 1.27))) (hide yes))
   (property "Block" "blk.radio-power" (at 86.36 167.64 0) (effects (font (size 1.27 1.27))) (hide yes))
   (pin "1")
