File: board/hardware/t1-main-board/pwr-5v1.kicad_sch (KiCad schematic)
At the start: 12 parts, among them U4001 TPS62903RPJR

Commit message: Board: capture blk.current-monitors
Five INA236 on I2C1 (0x40-0x43, 0x48) with their shunts, per power tree
§4.12 and BOM v1 lines 54 and 136. The measured branches are rails of
their own (VSYS_SRC, VSYS_LV_AUDIO, VSYS_AUDIO, VSYS_LV_BL, VSYS_P5V1),
fed through the shunts on this sheet; the charger, audio, backlight and
5.1 V sheets take them. The root's layout may leave a stack level empty,
so the block sits under the notes; IC bboxes hold turned rail values;
passive rows hold a bottom rail's text.

Co-Authored-By: Claude Opus 5.5 <noreply@anthropic.com>
Claude-Session: https://claude.ai/code/session_01Ei262h3TpgY9vyfNLMi5Mn
Parts:
- removed C4001: 10 nF, Capacitor_SMD:C_0402_1005Metric, symbol Device:C
- removed C4002: 10 µF, Capacitor_SMD:C_0805_2012Metric, symbol Device:C
- removed C4003: 22 µF, Capacitor_SMD:C_1210_3225Metric, symbol Device:C
- removed D4001, D4002: BAT54J, Diode_SMD:D_SOD-323F, symbol Diode:BAT54J
- removed L4001: 1 µH, Inductor_SMD:L_Coilcraft_XxL4020, symbol Device:L
- removed R4001: 95.3 kΩ, Resistor_SMD:R_0402_1005Metric, symbol Device:R
- removed R4002: 26.1 kΩ, Resistor_SMD:R_0402_1005Metric, symbol Device:R
- removed R4003: 100 kΩ, Resistor_SMD:R_0402_1005Metric, symbol Device:R
- removed TP4001: P5V1_SRC, TestPoint:TestPoint_Pad_D1.0mm, symbol Connector:TestPoint
- removed TP4002: P5V1_PG, TestPoint:TestPoint_Pad_D1.0mm, symbol Connector:TestPoint
- removed U4001: TPS62903RPJR, Texas_Instruments:Texas_RPJ0009A_VQFN-HR-9_1.5x2mm_P0.5mm, symbol Texas_Instruments:TPS62903RPJR
- added C4101: 10 nF, Capacitor_SMD:C_0402_1005Metric, symbol Device:C
- added C4102: 10 µF, Capacitor_SMD:C_0805_2012Metric, symbol Device:C
- added C4103: 22 µF, Capacitor_SMD:C_1210_3225Metric, symbol Device:C
- added D4101, D4102: BAT54J, Diode_SMD:D_SOD-323F, symbol Diode:BAT54J
- added L4101: 1 µH, Inductor_SMD:L_Coilcraft_XxL4020, symbol Device:L
- added R4101: 95.3 kΩ, Resistor_SMD:R_0402_1005Metric, symbol Device:R
- added R4102: 26.1 kΩ, Resistor_SMD:R_0402_1005Metric, symbol Device:R
- added R4103: 100 kΩ, Resistor_SMD:R_0402_1005Metric, symbol Device:R
- added TP4101: P5V1_SRC, TestPoint:TestPoint_Pad_D1.0mm, symbol Connector:TestPoint
- added TP4102: P5V1_PG, TestPoint:TestPoint_Pad_D1.0mm, symbol Connector:TestPoint
- added U4101: TPS62903RPJR, Texas_Instruments:Texas_RPJ0009A_VQFN-HR-9_1.5x2mm_P0.5mm, symbol Texas_Instruments:TPS62903RPJR
Connections:
- net GND: now also C4101.2, C4102.2, C4103.2, R4101.2, R4102.2, R4103.2, U4101.4 (GND)
- net HAT5V_EN: now also D4101.2 (A)
- net P5V1_EN: now also D4101.1 (K), D4102.1 (K), R4103.1, U4101.5 (EN)
- net P5V1_MODE: now also R4102.1, U4101.7 (MODE/S-CONF)
- net P5V1_PG: now also TP4102.1, U4101.1 (PG)
- net P5V1_SRC: now also C4103.1, L4101.2, TP4101.1, U4101.3 (VOS)
- net P5V1_SS: now also C4101.1, U4101.8 (SS/TR)
- net P5V1_SW: now also L4101.1, U4101.2 (SW)
- net P5V1_VSET: now also R4101.1, U4101.9 (FB/VSET)
- net USB_SRC_ON: now also D4102.2 (A)
- new net VSYS_P5V1: C4102.1, U4101.6 (VIN)

Commit message: Board: capture blk.debug
Debug UART2 (1.8 V) and I2S/DSD pads with ground pads, reset, PMIC and
power-key pads (PCB-T-09), a pad on every spare SoC GPIO whose pinout v1
row names one (the DEBUG bus, on the SoC's right edge), and a rail pad
for each power-tree rail no other sheet probes (PCB-T-02). Each DAC
sheet carries a pad on its MCLK. The spares pinout v1 leaves without a
pad now carry no-connect flags. On the root, facing sheet pins are
joined directly only where the route meets no other symbol.

Co-Authored-By: Claude Opus 5.5 <noreply@anthropic.com>
Claude-Session: https://claude.ai/code/session_01Ei262h3TpgY9vyfNLMi5Mn
Parts:
- removed C4101: 10 nF, Capacitor_SMD:C_0402_1005Metric, symbol Device:C
- removed C4102: 10 µF, Capacitor_SMD:C_0805_2012Metric, symbol Device:C
- removed C4103: 22 µF, Capacitor_SMD:C_1210_3225Metric, symbol Device:C
- removed D4101, D4102: BAT54J, Diode_SMD:D_SOD-323F, symbol Diode:BAT54J
- removed L4101: 1 µH, Inductor_SMD:L_Coilcraft_XxL4020, symbol Device:L
- removed R4101: 95.3 kΩ, Resistor_SMD:R_0402_1005Metric, symbol Device:R
- removed R4102: 26.1 kΩ, Resistor_SMD:R_0402_1005Metric, symbol Device:R
- removed R4103: 100 kΩ, Resistor_SMD:R_0402_1005Metric, symbol Device:R
- removed TP4101: P5V1_SRC, TestPoint:TestPoint_Pad_D1.0mm, symbol Connector:TestPoint
- removed TP4102: P5V1_PG, TestPoint:TestPoint_Pad_D1.0mm, symbol Connector:TestPoint
- removed U4101: TPS62903RPJR, Texas_Instruments:Texas_RPJ0009A_VQFN-HR-9_1.5x2mm_P0.5mm, symbol Texas_Instruments:TPS62903RPJR
- added C4201: 10 nF, Capacitor_SMD:C_0402_1005Metric, symbol Device:C
- added C4202: 10 µF, Capacitor_SMD:C_0805_2012Metric, symbol Device:C
- added C4203: 22 µF, Capacitor_SMD:C_1210_3225Metric, symbol Device:C
- added D4201, D4202: BAT54J, Diode_SMD:D_SOD-323F, symbol Diode:BAT54J
- added L4201: 1 µH, Inductor_SMD:L_Coilcraft_XxL4020, symbol Device:L
- added R4201: 95.3 kΩ, Resistor_SMD:R_0402_1005Metric, symbol Device:R
- added R4202: 26.1 kΩ, Resistor_SMD:R_0402_1005Metric, symbol Device:R
- added R4203: 100 kΩ, Resistor_SMD:R_0402_1005Metric, symbol Device:R
- added TP4201: P5V1_SRC, TestPoint:TestPoint_Pad_D1.0mm, symbol Connector:TestPoint
- added TP4202: P5V1_PG, TestPoint:TestPoint_Pad_D1.0mm, symbol Connector:TestPoint
- added U4201: TPS62903RPJR, Texas_Instruments:Texas_RPJ0009A_VQFN-HR-9_1.5x2mm_P0.5mm, symbol Texas_Instruments:TPS62903RPJR
Connections:
- net GND: now also C4201.2, C4202.2, C4203.2, R4201.2, R4202.2, R4203.2, U4201.4 (GND)
- net HAT5V_EN: now also D4201.2 (A)
- net P5V1_EN: now also D4201.1 (K), D4202.1 (K), R4203.1, U4201.5 (EN)
- net P5V1_MODE: now also R4202.1, U4201.7 (MODE/S-CONF)
- net P5V1_PG: now also TP4202.1, U4201.1 (PG)
- net P5V1_SRC: now also C4203.1, L4201.2, TP4201.1, U4201.3 (VOS)
- net P5V1_SS: now also C4201.1, U4201.8 (SS/TR)
- net P5V1_SW: now also L4201.1, U4201.2 (SW)
- net P5V1_VSET: now also R4201.1, U4201.9 (FB/VSET)
- net USB_SRC_ON: now also D4202.2 (A)
- net VSYS_P5V1: now also C4202.1, U4201.6 (VIN)

Commit message: Board: capture blk.mic-ambient and links #34, #35
IM73D122 on PDM CLK1 and SDI1 (BOM v1 line 34, pinout v1 AK2 and 1P2),
LR to ground, 22 Ω clock series, VDD from MIC_1V8 through link #35.
Link #34 on blk.mic-main makes the faceplate branch the rail MIC_1V8_FP
for contact 40 (power tree §4.12, G10). kicad-lib moves to e46bda4 for
the IM73D122, TPS3808G01, SN74LVC1G58 and BAT54 parts.

Co-Authored-By: Claude Opus 5.5 <noreply@anthropic.com>
Claude-Session: https://claude.ai/code/session_01Ei262h3TpgY9vyfNLMi5Mn
Parts:
- removed C4201: 10 nF, Capacitor_SMD:C_0402_1005Metric, symbol Device:C
- removed C4202: 10 µF, Capacitor_SMD:C_0805_2012Metric, symbol Device:C
- removed C4203: 22 µF, Capacitor_SMD:C_1210_3225Metric, symbol Device:C
- removed D4201, D4202: BAT54J, Diode_SMD:D_SOD-323F, symbol Diode:BAT54J
- removed L4201: 1 µH, Inductor_SMD:L_Coilcraft_XxL4020, symbol Device:L
- removed R4201: 95.3 kΩ, Resistor_SMD:R_0402_1005Metric, symbol Device:R
- removed R4202: 26.1 kΩ, Resistor_SMD:R_0402_1005Metric, symbol Device:R
- removed R4203: 100 kΩ, Resistor_SMD:R_0402_1005Metric, symbol Device:R
- removed TP4201: P5V1_SRC, TestPoint:TestPoint_Pad_D1.0mm, symbol Connector:TestPoint
- removed TP4202: P5V1_PG, TestPoint:TestPoint_Pad_D1.0mm, symbol Connector:TestPoint
- removed U4201: TPS62903RPJR, Texas_Instruments:Texas_RPJ0009A_VQFN-HR-9_1.5x2mm_P0.5mm, symbol Texas_Instruments:TPS62903RPJR
- added C4301: 10 nF, Capacitor_SMD:C_0402_1005Metric, symbol Device:C
- added C4302: 10 µF, Capacitor_SMD:C_0805_2012Metric, symbol Device:C
- added C4303: 22 µF, Capacitor_SMD:C_1210_3225Metric, symbol Device:C
- added D4301, D4302: BAT54J, Diode_SMD:D_SOD-323F, symbol Diode:BAT54J
- added L4301: 1 µH, Inductor_SMD:L_Coilcraft_XxL4020, symbol Device:L
- added R4301: 95.3 kΩ, Resistor_SMD:R_0402_1005Metric, symbol Device:R
- added R4302: 26.1 kΩ, Resistor_SMD:R_0402_1005Metric, symbol Device:R
- added R4303: 100 kΩ, Resistor_SMD:R_0402_1005Metric, symbol Device:R
- added TP4301: P5V1_SRC, TestPoint:TestPoint_Pad_D1.0mm, symbol Connector:TestPoint
- added TP4302: P5V1_PG, TestPoint:TestPoint_Pad_D1.0mm, symbol Connector:TestPoint
- added U4301: TPS62903RPJR, Texas_Instruments:Texas_RPJ0009A_VQFN-HR-9_1.5x2mm_P0.5mm, symbol Texas_Instruments:TPS62903RPJR
Connections:
- net GND: now also C4301.2, C4302.2, C4303.2, R4301.2, R4302.2, R4303.2, U4301.4 (GND)
- net HAT5V_EN: now also D4301.2 (A)
- net P5V1_EN: now also D4301.1 (K), D4302.1 (K), R4303.1, U4301.5 (EN)
- net P5V1_MODE: now also R4302.1, U4301.7 (MODE/S-CONF)
- net P5V1_PG: now also TP4302.1, U4301.1 (PG)
- net P5V1_SRC: now also C4303.1, L4301.2, TP4301.1, U4301.3 (VOS)
- net P5V1_SS: now also C4301.1, U4301.8 (SS/TR)
- net P5V1_SW: now also L4301.1, U4301.2 (SW)
- net P5V1_VSET: now also R4301.1, U4301.9 (FB/VSET)
- net USB_SRC_ON: now also D4302.2 (A)
- net VSYS_P5V1: now also C4302.1, U4301.6 (VIN)

Commit message: Board: capture blk.maskrom
Power + Vol- at a cold power-on pull eMMC D0 low inside the TPS3808G01
boot window (BOM v1 lines 35, 78, 97, 98; sim/maskrom): SENSE 280k/100k,
CT 390 nF, WINDOW_N with its pad, SN74LVC1G57 and SN74LVC1G58 on
vcca1v8_pmu, BAT54 from PWRON_N, DMG1012T through 1 kΩ to EMMC_D0.
Every block in use now has its sheet; the README states the remaining
single-pin nets.

Co-Authored-By: Claude Opus 5.5 <noreply@anthropic.com>
Claude-Session: https://claude.ai/code/session_01Ei262h3TpgY9vyfNLMi5Mn
Parts:
- removed C4301: 10 nF, Capacitor_SMD:C_0402_1005Metric, symbol Device:C
- removed C4302: 10 µF, Capacitor_SMD:C_0805_2012Metric, symbol Device:C
- removed C4303: 22 µF, Capacitor_SMD:C_1210_3225Metric, symbol Device:C
- removed D4301, D4302: BAT54J, Diode_SMD:D_SOD-323F, symbol Diode:BAT54J
- removed L4301: 1 µH, Inductor_SMD:L_Coilcraft_XxL4020, symbol Device:L
- removed R4301: 95.3 kΩ, Resistor_SMD:R_0402_1005Metric, symbol Device:R
- removed R4302: 26.1 kΩ, Resistor_SMD:R_0402_1005Metric, symbol Device:R
- removed R4303: 100 kΩ, Resistor_SMD:R_0402_1005Metric, symbol Device:R
- removed TP4301: P5V1_SRC, TestPoint:TestPoint_Pad_D1.0mm, symbol Connector:TestPoint
- removed TP4302: P5V1_PG, TestPoint:TestPoint_Pad_D1.0mm, symbol Connector:TestPoint
- removed U4301: TPS62903RPJR, Texas_Instruments:Texas_RPJ0009A_VQFN-HR-9_1.5x2mm_P0.5mm, symbol Texas_Instruments:TPS62903RPJR
- added C4401: 10 nF, Capacitor_SMD:C_0402_1005Metric, symbol Device:C
- added C4402: 10 µF, Capacitor_SMD:C_0805_2012Metric, symbol Device:C
- added C4403: 22 µF, Capacitor_SMD:C_1210_3225Metric, symbol Device:C
- added D4401, D4402: BAT54J, Diode_SMD:D_SOD-323F, symbol Diode:BAT54J
- added L4401: 1 µH, Inductor_SMD:L_Coilcraft_XxL4020, symbol Device:L
- added R4401: 95.3 kΩ, Resistor_SMD:R_0402_1005Metric, symbol Device:R
- added R4402: 26.1 kΩ, Resistor_SMD:R_0402_1005Metric, symbol Device:R
- added R4403: 100 kΩ, Resistor_SMD:R_0402_1005Metric, symbol Device:R
- added TP4401: P5V1_SRC, TestPoint:TestPoint_Pad_D1.0mm, symbol Connector:TestPoint
- added TP4402: P5V1_PG, TestPoint:TestPoint_Pad_D1.0mm, symbol Connector:TestPoint
- added U4401: TPS62903RPJR, Texas_Instruments:Texas_RPJ0009A_VQFN-HR-9_1.5x2mm_P0.5mm, symbol Texas_Instruments:TPS62903RPJR
Connections:
- net GND: now also C4401.2, C4402.2, C4403.2, R4401.2, R4402.2, R4403.2, U4401.4 (GND)
- net HAT5V_EN: now also D4401.2 (A)
- net P5V1_EN: now also D4401.1 (K), D4402.1 (K), R4403.1, U4401.5 (EN)
- net P5V1_MODE: now also R4402.1, U4401.7 (MODE/S-CONF)
- net P5V1_PG: now also TP4402.1, U4401.1 (PG)
- net P5V1_SRC: now also C4403.1, L4401.2, TP4401.1, U4401.3 (VOS)
- net P5V1_SS: now also C4401.1, U4401.8 (SS/TR)
- net P5V1_SW: now also L4401.1, U4401.2 (SW)
- net P5V1_VSET: now also R4401.1, U4401.9 (FB/VSET)
- net USB_SRC_ON: now also D4402.2 (A)
- net VSYS_P5V1: now also C4402.1, U4401.6 (VIN)

Commit message: Compaction: lower inductors, 0201 decoupling, 0.8 mm signal test pads
A matrix tool (hardware/studies/compaction) checks each candidate against
the design's stresses: same inductance, design peak <= 70 % and the
converter's maximum limit <= 100 % of Isat (30 % drop), height zones,
ratings at least twice the rail, PCB-D-06; sourcing outcome per part.

Applied (placement v1 decision 12, BOM v1.15):
- L601, L4401: XGL4015-102MEC (1.5 mm) for XAL/XGL4020-102MEC (2.1 mm);
- L1001, L5101: XGL4015-471MEC (1.5 mm) for Wurth 744373240047, on the
  stock XxL4020 land (the Wurth land was never drawn);
- L1201 is 1.2 mm (XGL4012, per-MPN heights): it moves next to the SoC;
- 58 x 100 nF decoupling on rails <= 3.3 V in core/IO/radio: 0201;
- 51 test pads on signal nets: 0.8 mm (PCB-D-06 v0.16, JLCPCB guide).
Kept: L901, L2802 (XGL4015 at 103 % of Isat at the limit); no thinner
0805/1206 capacitor passes (obsolete, NRND or unlisted).

Board need 113 % -> 111 % (core band 227 -> 203 %, power band 258 ->
233 %, radio band 19 -> 0 %); only C904 still relies on PCB-Z-04.
ERC 0 errors, craft Q1 met, DRC 0 errors (605 warnings), pcb and study
tests pass, rules test board PASS.

Co-Authored-By: Claude Opus 5.5 <noreply@anthropic.com>
Claude-Session: https://claude.ai/code/session_01Ei262h3TpgY9vyfNLMi5Mn
Parts:
- L4401: MPN XGL4020-102MEC -> XGL4015-102MEC; MPN_2 (none) -> XGL4012-102MEC; Manufacturer_2 (none) -> Coilcraft; Second_Source (none) -> Coilcraft XGL4012-102MEC (same land, 1.2 mm, Isat 6.6 A at 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; Spec Isat 8.8 A -> Isat 7.3 A
- TP4402: footprint TestPoint:TestPoint_Pad_D1.0mm -> T1_Main_Board:TestPoint_Pad_D0.8mm
Changed lines of the file:
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@@
   (property "Reference" "L4401" (at 168.91 43.18 90) (effects (font (size 1.27 1.27))))
   (property "Value" "1 µH" (at 168.91 48.26 90) (effects (font (size 1.27 1.27))))
-  (property "Spec" "Isat 8.8 A" (at 168.91 50.8 90) (effects (font (size 1.27 1.27))))
+  (property "Spec" "Isat 7.3 A" (at 168.91 50.8 90) (effects (font (size 1.27 1.27))))
   (property "Footprint" "Inductor_SMD:L_Coilcraft_XxL4020" (at 168.91 45.72 0) (effects (font (size 1.27 1.27))) (hide yes))
-  (property "Datasheet" "https://www.coilcraft.com/getmedia/76c9c081-4945-4c85-9129-9356e1ad6734/xgl4020.pdf" (at 168.91 45.72 0) (effects (font (size 1.27 1.27))) (hide yes))
-  (property "Description" "Power inductor, 1.0 uH 20 %, Isat 8.8 A (30 % drop), 4.0 x 4.0 x 2.1 mm" (at 168.91 45.72 0) (effects (font (size 1.27 1.27))) (hide yes))
+  (property "Datasheet" "https://coilcraft.com/getmedia/c5d04454-742d-473e-8b80-06c97338c587/xgl4015.pdf" (at 168.91 45.72 0) (effects (font (size 1.27 1.27))) (hide yes))
+  (property "Description" "Power inductor, 1.0 uH 20 %, Isat 7.3 A (30 % drop), Irms 6.5 A, 4.0 x 4.0 x 1.5 mm" (at 168.91 45.72 0) (effects (font (size 1.27 1.27))) (hide yes))
   (property "Manufacturer" "Coilcraft" (at 168.91 45.72 0) (effects (font (size 1.27 1.27))) (hide yes))
-  (property "MPN" "XGL4020-102MEC" (at 168.91 45.72 0) (effects (font (size 1.27 1.27))) (hide yes))
+  (property "MPN" "XGL4015-102MEC" (at 168.91 45.72 0) (effects (font (size 1.27 1.27))) (hide yes))
+  (property "Second_Source" "Coilcraft XGL4012-102MEC (same land, 1.2 mm, Isat 6.6 A at 30 % drop)" (at 168.91 45.72 0) (effects (font (size 1.27 1.27))) (hide yes))
+  (property "Manufacturer_2" "Coilcraft" (at 168.91 45.72 0) (effects (font (size 1.27 1.27))) (hide yes))
+  (property "MPN_2" "XGL4012-102MEC" (at 168.91 45.72 0) (effects (font (size 1.27 1.27))) (hide yes))
   (property "Block" "blk.pwr-5v1" (at 168.91 45.72 0) (effects (font (size 1.27 1.27))) (hide yes))
   (pin "1")
@@
   (property "Reference" "TP4402" (at 298.45 46.99 0) (effects (font (size 1.27 1.27)) (justify right)))
   (property "Value" "P5V1_PG" (at 298.45 49.53 0) (effects (font (size 1.27 1.27)) (justify right)))
-  (property "Footprint" "TestPoint:TestPoint_Pad_D1.0mm" (at 299.72 52.07 0) (effects (font (size 1.27 1.27))) (hide yes))
+  (property "Footprint" "T1_Main_Board:TestPoint_Pad_D0.8mm" (at 299.72 52.07 0) (effects (font (size 1.27 1.27))) (hide yes))
   (property "Datasheet" "~" (at 299.72 52.07 0) (effects (font (size 1.27 1.27))) (hide yes))
-  (property "Description" "Test pad, 1.0 mm" (at 299.72 52.07 0) (effects (font (size 1.27 1.27))) (hide yes))
+  (property "Description" "Test pad, 0.8 mm, signal net" (at 299.72 52.07 0) (effects (font (size 1.27 1.27))) (hide yes))
   (property "Block" "blk.pwr-5v1" (at 299.72 52.07 0) (effects (font (size 1.27 1.27))) (hide yes))
   (pin "1")

Commit message: Board on libs v0.2.0: lower-case kebab vendor keys (HL-13)
The libs submodule moves to v0.2.0 (5f24483). Every library nickname in
the generator, the placement tool and the floorplan study follows the
key table (Texas_Instruments -> texas-instruments, OpenDAP_Device ->
opendap-generic, Rockchip and Rockchip_PMIC -> rockchip, ...); the
library tables are written from the files. Schematic and board
regenerated.

Checks: ERC 0 errors (warnings unchanged); DRC 0 errors, 605 warnings,
the same counts by type, schematic parity 0; every placement identical;
craft Q1 met; pcb tests pass; STEP export resolves every libs 3D model
(the 27 parts without a model are KiCad stock lands that have none).

Co-Authored-By: Claude Opus 5.5 <noreply@anthropic.com>
Claude-Session: https://claude.ai/code/session_01Ei262h3TpgY9vyfNLMi5Mn
Parts:
- U4401: footprint Texas_Instruments:Texas_RPJ0009A_VQFN-HR-9_1.5x2mm_P0.5mm -> texas-instruments:Texas_RPJ0009A_VQFN-HR-9_1.5x2mm_P0.5mm; symbol Texas_Instruments:TPS62903RPJR -> texas-instruments:TPS62903RPJR
Changed lines of the file:
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@@
 (paper "A3")
 (title_block (title "5.1 V source") (date "2026-10-25") (rev "A") (company "The OpenDAP Project") (comment 1 "blk.pwr-5v1") (comment 2 "TPS62903 buck from VSYS for the HAT and USB-C sources, enabled by either port"))
-(symbol (lib_id "Texas_Instruments:TPS62903RPJR") (at 54.61 63.5 0) (unit 1) (body_style 1) (exclude_from_sim no) (in_bom yes) (on_board yes) (dnp no)
+(symbol (lib_id "texas-instruments:TPS62903RPJR") (at 54.61 63.5 0) (unit 1) (body_style 1) (exclude_from_sim no) (in_bom yes) (on_board yes) (dnp no)
   (property "Reference" "U4401" (at 55.88 45.72 0) (effects (font (size 1.27 1.27)) (justify left)))
   (property "Value" "TPS62903RPJR" (at 55.88 43.18 0) (effects (font (size 1.27 1.27)) (justify left)))
-  (property "Footprint" "Texas_Instruments:Texas_RPJ0009A_VQFN-HR-9_1.5x2mm_P0.5mm" (at 54.61 63.5 0) (effects (font (size 1.27 1.27))) (hide yes))
+  (property "Footprint" "texas-instruments:Texas_RPJ0009A_VQFN-HR-9_1.5x2mm_P0.5mm" (at 54.61 63.5 0) (effects (font (size 1.27 1.27))) (hide yes))
   (property "Datasheet" "https://www.ti.com/lit/ds/symlink/tps62903.pdf" (at 54.61 63.5 0) (effects (font (size 1.27 1.27))) (hide yes))
   (property "Description" "3 A synchronous step-down converter, 3-17 V input, 0.4-5.5 V output, DCS-Control, power good, VQFN-HR-9 (RPJ0009A) 1.5 x 2.0 mm" (at 54.61 63.5 0) (effects (font (size 1.27 1.27))) (hide yes))
