File: board/hardware/t1-main-board/pwr-5v1.kicad_sch (KiCad schematic)
At the start: 12 parts, among them U4401 TPS62903RPJR

Commit message: Board in the 62.5 x 95.0 mm body: ADR 0025, outline 59.1 x 91.6, 0201 swaps
ADR 0025 supersedes ADR 0016 for t1 ADR 0006's body: board outline from
the body, 1.2 mm walls and 0.5 mm clearance; height zones and stack
restated unchanged; the speaker on a case shelf (PCB-Z-09); pocket
reliefs at the 4.4 mm jack, the microSD (DM3AT push-push kept) and the
side buttons; the audio 0603 -> 0402 swap gated by t1 V2-A08; reserve
(NFC reader, then TPM) recorded, not applied.

- pcb/geometry.py derives the outline from BODY, WALL and CLEARANCE;
  the pocket, display and fixed parts keep their device-frame positions;
  holes keep their edge distance; the speaker shadow becomes a 1.5 mm
  shelf height area (placement, checks, occupancy).
- build.py reports pocket reliefs and routing room; C904 unfixed (it
  now finds back room, so PCB-Z-04 carries no part).
- Generator: parts.area_swap puts 121 generic 0402 resistors (outside
  audio and VBUS paths, >= 10 ohm) and five 100 nF signal capacitors in
  0201 (BOM v1.16); schematic and board regenerated.
- Result: 1,012/1,012 placed, 98.8 % by the floorplan method (was 111 %),
  factor left 1.68 (was 1.49); DRC 0 errors, ERC 0 errors, 0 check
  findings, pcb tests 20/20, schematic craft Q1 met.
- Specs: PCB constraints v0.17 (M-01, M-02, M-08, Z-02, Z-06 to Z-09,
  R-07), placement v1.1 (section 3, decisions 4 and 13, checks, open
  items with the gated swaps and the reserve), floorplan v1 section 1,
  BOM v1.16.

Co-Authored-By: Claude Opus 5.5 <noreply@anthropic.com>
Claude-Session: https://claude.ai/code/session_01Ei262h3TpgY9vyfNLMi5Mn
Parts:
- R4401: footprint Resistor_SMD:R_0402_1005Metric -> Resistor_SMD:R_0201_0603Metric; MPN RC0402FR-0795K3L -> RC0201FR-0795K3L
- R4402: footprint Resistor_SMD:R_0402_1005Metric -> Resistor_SMD:R_0201_0603Metric; MPN RC0402FR-0726K1L -> RC0201FR-0726K1L
- R4403: footprint Resistor_SMD:R_0402_1005Metric -> Resistor_SMD:R_0201_0603Metric; MPN RC0402FR-07100KL -> RC0201FR-07100KL
Changed lines of the file:
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@@
   (property "Reference" "R4401" (at 90.17 54.61 0) (effects (font (size 1.27 1.27)) (justify left)))
   (property "Value" "95.3 kΩ" (at 90.17 57.15 0) (effects (font (size 1.27 1.27)) (justify left)))
-  (property "Footprint" "Resistor_SMD:R_0402_1005Metric" (at 88.9 55.88 0) (effects (font (size 1.27 1.27))) (hide yes))
-  (property "Datasheet" "https://yageogroup.com/en/ProductSearch/PartNumberSearch?part=RC0402FR-0795K3L" (at 88.9 55.88 0) (effects (font (size 1.27 1.27))) (hide yes))
-  (property "Description" "Resistor, 95.3 kΩ, 1 %, 1/16 W, 0402" (at 88.9 55.88 0) (effects (font (size 1.27 1.27))) (hide yes))
+  (property "Footprint" "Resistor_SMD:R_0201_0603Metric" (at 88.9 55.88 0) (effects (font (size 1.27 1.27))) (hide yes))
+  (property "Datasheet" "https://yageogroup.com/en/ProductSearch/PartNumberSearch?part=RC0201FR-0795K3L" (at 88.9 55.88 0) (effects (font (size 1.27 1.27))) (hide yes))
+  (property "Description" "Resistor, 95.3 kΩ, 1 %, 1/20 W, 0201" (at 88.9 55.88 0) (effects (font (size 1.27 1.27))) (hide yes))
   (property "Manufacturer" "YAGEO" (at 88.9 55.88 0) (effects (font (size 1.27 1.27))) (hide yes))
-  (property "MPN" "RC0402FR-0795K3L" (at 88.9 55.88 0) (effects (font (size 1.27 1.27))) (hide yes))
+  (property "MPN" "RC0201FR-0795K3L" (at 88.9 55.88 0) (effects (font (size 1.27 1.27))) (hide yes))
   (property "Block" "blk.pwr-5v1" (at 88.9 55.88 0) (effects (font (size 1.27 1.27))) (hide yes))
   (pin "1")
@@
   (property "Reference" "R4402" (at 104.14 54.61 0) (effects (font (size 1.27 1.27)) (justify left)))
   (property "Value" "26.1 kΩ" (at 104.14 57.15 0) (effects (font (size 1.27 1.27)) (justify left)))
-  (property "Footprint" "Resistor_SMD:R_0402_1005Metric" (at 102.87 55.88 0) (effects (font (size 1.27 1.27))) (hide yes))
-  (property "Datasheet" "https://yageogroup.com/en/ProductSearch/PartNumberSearch?part=RC0402FR-0726K1L" (at 102.87 55.88 0) (effects (font (size 1.27 1.27))) (hide yes))
-  (property "Description" "Resistor, 26.1 kΩ, 1 %, 1/16 W, 0402" (at 102.87 55.88 0) (effects (font (size 1.27 1.27))) (hide yes))
+  (property "Footprint" "Resistor_SMD:R_0201_0603Metric" (at 102.87 55.88 0) (effects (font (size 1.27 1.27))) (hide yes))
+  (property "Datasheet" "https://yageogroup.com/en/ProductSearch/PartNumberSearch?part=RC0201FR-0726K1L" (at 102.87 55.88 0) (effects (font (size 1.27 1.27))) (hide yes))
+  (property "Description" "Resistor, 26.1 kΩ, 1 %, 1/20 W, 0201" (at 102.87 55.88 0) (effects (font (size 1.27 1.27))) (hide yes))
   (property "Manufacturer" "YAGEO" (at 102.87 55.88 0) (effects (font (size 1.27 1.27))) (hide yes))
-  (property "MPN" "RC0402FR-0726K1L" (at 102.87 55.88 0) (effects (font (size 1.27 1.27))) (hide yes))
+  (property "MPN" "RC0201FR-0726K1L" (at 102.87 55.88 0) (effects (font (size 1.27 1.27))) (hide yes))
   (property "Block" "blk.pwr-5v1" (at 102.87 55.88 0) (effects (font (size 1.27 1.27))) (hide yes))
   (pin "1")
@@
   (property "Reference" "R4403" (at 133.35 54.61 0) (effects (font (size 1.27 1.27)) (justify left)))
   (property "Value" "100 kΩ" (at 133.35 57.15 0) (effects (font (size 1.27 1.27)) (justify left)))
-  (property "Footprint" "Resistor_SMD:R_0402_1005Metric" (at 132.08 55.88 0) (effects (font (size 1.27 1.27))) (hide yes))
-  (property "Datasheet" "https://yageogroup.com/en/ProductSearch/PartNumberSearch?part=RC0402FR-07100KL" (at 132.08 55.88 0) (effects (font (size 1.27 1.27))) (hide yes))
-  (property "Description" "Resistor, 100 kΩ, 1 %, 1/16 W, 0402" (at 132.08 55.88 0) (effects (font (size 1.27 1.27))) (hide yes))
+  (property "Footprint" "Resistor_SMD:R_0201_0603Metric" (at 132.08 55.88 0) (effects (font (size 1.27 1.27))) (hide yes))
+  (property "Datasheet" "https://yageogroup.com/en/ProductSearch/PartNumberSearch?part=RC0201FR-07100KL" (at 132.08 55.88 0) (effects (font (size 1.27 1.27))) (hide yes))
+  (property "Description" "Resistor, 100 kΩ, 1 %, 1/20 W, 0201" (at 132.08 55.88 0) (effects (font (size 1.27 1.27))) (hide yes))
   (property "Manufacturer" "YAGEO" (at 132.08 55.88 0) (effects (font (size 1.27 1.27))) (hide yes))
-  (property "MPN" "RC0402FR-07100KL" (at 132.08 55.88 0) (effects (font (size 1.27 1.27))) (hide yes))
+  (property "MPN" "RC0201FR-07100KL" (at 132.08 55.88 0) (effects (font (size 1.27 1.27))) (hide yes))
   (property "Block" "blk.pwr-5v1" (at 132.08 55.88 0) (effects (font (size 1.27 1.27))) (hide yes))
   (pin "1")

Commit message: BOM v1.18 item 1: 22 uF 25 V X5R 0805 at the TPS62136 and TPS62903 inputs
C901 and C4402 keep 3.89 uF effective at 8.8 V (-20..85 C, tolerance
included) against the 3 uF minimum; the 10 uF part kept 1.86 uF. Same
land; sourcing pass. Closes BOM §7 item 51.

Co-Authored-By: Claude Opus 5.5 <noreply@anthropic.com>
Claude-Session: https://claude.ai/code/session_01Ei262h3TpgY9vyfNLMi5Mn
Parts:
- C4402: value 10 µF -> 22 µF; MPN GRM21BR61E106KA73L -> GRM21BR61E226ME44L
Changed lines of the file:
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@@
 (symbol (lib_id "Device:C") (at 88.9 87.63 0) (unit 1) (body_style 1) (exclude_from_sim no) (in_bom yes) (on_board yes) (dnp no)
   (property "Reference" "C4402" (at 91.44 86.36 0) (effects (font (size 1.27 1.27)) (justify left)))
-  (property "Value" "10 µF" (at 91.44 88.9 0) (effects (font (size 1.27 1.27)) (justify left)))
+  (property "Value" "22 µF" (at 91.44 88.9 0) (effects (font (size 1.27 1.27)) (justify left)))
   (property "Spec" "25 V X5R" (at 91.44 91.44 0) (effects (font (size 1.27 1.27)) (justify left)))
   (property "Footprint" "Capacitor_SMD:C_0805_2012Metric" (at 88.9 87.63 0) (effects (font (size 1.27 1.27))) (hide yes))
-  (property "Datasheet" "https://www.murata.com/en-us/products/productdetail?partno=GRM21BR61E106KA73L" (at 88.9 87.63 0) (effects (font (size 1.27 1.27))) (hide yes))
-  (property "Description" "Capacitor, 10 µF, 25 V, X5R, 0805" (at 88.9 87.63 0) (effects (font (size 1.27 1.27))) (hide yes))
+  (property "Datasheet" "https://www.murata.com/en-us/products/productdetail?partno=GRM21BR61E226ME44L" (at 88.9 87.63 0) (effects (font (size 1.27 1.27))) (hide yes))
+  (property "Description" "Capacitor, 22 µF, 25 V, X5R, 0805" (at 88.9 87.63 0) (effects (font (size 1.27 1.27))) (hide yes))
   (property "Manufacturer" "Murata" (at 88.9 87.63 0) (effects (font (size 1.27 1.27))) (hide yes))
-  (property "MPN" "GRM21BR61E106KA73L" (at 88.9 87.63 0) (effects (font (size 1.27 1.27))) (hide yes))
+  (property "MPN" "GRM21BR61E226ME44L" (at 88.9 87.63 0) (effects (font (size 1.27 1.27))) (hide yes))
   (property "Block" "blk.pwr-5v1" (at 88.9 87.63 0) (effects (font (size 1.27 1.27))) (hide yes))
   (pin "1")
@@
 (table (column_count 3) (border (external yes) (header yes) (stroke (width 0) (type solid))) (separators (rows yes) (cols yes) (stroke (width 0) (type solid))) (column_widths 38.1 22.86 57.15) (row_heights 5.08 7.62 5.08 7.62) (cells (table_cell "Net" (exclude_from_sim no) (at 22.86 255.27 0) (size 38.1 5.08) (margins 0.9525 0.9525 0.9525 0.9525) (span 1 1) (fill (type none)) (effects (font (size 1.27 1.27) (bold yes)) (justify left top))) (table_cell "Direction" (exclude_from_sim no) (at 60.96 255.27 0) (size 22.86 5.08) (margins 0.9525 0.9525 0.9525 0.9525) (span 1 1) (fill (type none)) (effects (font (size 1.27 1.27) (bold yes)) (justify left top))) (table_cell "Absent state (block not fitted)" (exclude_from_sim no) (at 83.82 255.27 0) (size 57.15 5.08) (margins 0.9525 0.9525 0.9525 0.9525) (span 1 1) (fill (type none)) (effects (font (size 1.27 1.27) (bold yes)) (justify left top))) (table_cell "VSYS_P5V1" (exclude_from_sim no) (at 22.86 260.35 0) (size 38.1 7.62) (margins 0.9525 0.9525 0.9525 0.9525) (span 1 1) (fill (type none)) (effects (font (size 1.27 1.27)) (justify left top))) (table_cell "Supply in" (exclude_from_sim no) (at 60.96 260.35 0) (size 22.86 7.62) (margins 0.9525 0.9525 0.9525 0.9525) (span 1 1) (fill (type none)) (effects (font (size 1.27 1.27)) (justify left top))) (table_cell "VSYS through the HAT INA236 shunt (0x43, blk.current-monitors)" (exclude_from_sim no) (at 83.82 260.35 0) (size 57.15 7.62) (margins 0.9525 0.9525 0.9525 0.9525) (span 1 1) (fill (type none)) (effects (font (size 1.27 1.27)) (justify left top))) (table_cell "HAT5V_EN, USB_SRC_ON" (exclude_from_sim no) (at 22.86 267.97 0) (size 38.1 5.08) (margins 0.9525 0.9525 0.9525 0.9525) (span 1 1) (fill (type none)) (effects (font (size 1.27 1.27)) (justify left top))) (table_cell "Input" (exclude_from_sim no) (at 60.96 267.97 0) (size 22.86 5.08) (margins 0.9525 0.9525 0.9525 0.9525) (span 1 1) (fill (type none)) (effects (font (size 1.27 1.27)) (justify left top))) (table_cell "Expander P02, P03, pulled down: the buck off" (exclude_from_sim no) (at 83.82 267.97 0) (size 57.15 5.08) (margins 0.9525 0.9525 0.9525 0.9525) (span 1 1) (fill (type none)) (effects (font (size 1.27 1.27)) (justify left top))) (table_cell "P5V1_SRC" (exclude_from_sim no) (at 22.86 273.05 0) (size 38.1 7.62) (margins 0.9525 0.9525 0.9525 0.9525) (span 1 1) (fill (type none)) (effects (font (size 1.27 1.27)) (justify left top))) (table_cell "Supply out" (exclude_from_sim no) (at 60.96 273.05 0) (size 22.86 7.62) (margins 0.9525 0.9525 0.9525 0.9525) (span 1 1) (fill (type none)) (effects (font (size 1.27 1.27)) (justify left top))) (table_cell "Off, discharged (output discharge on, MODE 26.1 kΩ)" (exclude_from_sim no) (at 83.82 273.05 0) (size 57.15 7.62) (margins 0.9525 0.9525 0.9525 0.9525) (span 1 1) (fill (type none)) (effects (font (size 1.27 1.27)) (justify left top)))))
 (text "Rails" (exclude_from_sim no) (at 148.59 254 0) (effects (font (size 2.54 2.54)) (justify left bottom)))
-(table (column_count 3) (border (external yes) (header yes) (stroke (width 0) (type solid))) (separators (rows yes) (cols yes) (stroke (width 0) (type solid))) (column_widths 27.94 35.56 55.88) (row_heights 5.08 5.08 5.08) (cells (table_cell "Rail" (exclude_from_sim no) (at 148.59 255.27 0) (size 27.94 5.08) (margins 0.9525 0.9525 0.9525 0.9525) (span 1 1) (fill (type none)) (effects (font (size 1.27 1.27) (bold yes)) (justify left top))) (table_cell "Capacitors" (exclude_from_sim no) (at 176.53 255.27 0) (size 35.56 5.08) (margins 0.9525 0.9525 0.9525 0.9525) (span 1 1) (fill (type none)) (effects (font (size 1.27 1.27) (bold yes)) (justify left top))) (table_cell "Requirement and source" (exclude_from_sim no) (at 212.09 255.27 0) (size 55.88 5.08) (margins 0.9525 0.9525 0.9525 0.9525) (span 1 1) (fill (type none)) (effects (font (size 1.27 1.27) (bold yes)) (justify left top))) (table_cell "VSYS_P5V1" (exclude_from_sim no) (at 148.59 260.35 0) (size 27.94 5.08) (margins 0.9525 0.9525 0.9525 0.9525) (span 1 1) (fill (type none)) (effects (font (size 1.27 1.27)) (justify left top))) (table_cell "10 µF 25 V" (exclude_from_sim no) (at 176.53 260.35 0) (size 35.56 5.08) (margins 0.9525 0.9525 0.9525 0.9525) (span 1 1) (fill (type none)) (effects (font (size 1.27 1.27)) (justify left top))) (table_cell "SLVSES3A Table 8-1" (exclude_from_sim no) (at 212.09 260.35 0) (size 55.88 5.08) (margins 0.9525 0.9525 0.9525 0.9525) (span 1 1) (fill (type none)) (effects (font (size 1.27 1.27)) (justify left top))) (table_cell "P5V1_SRC" (exclude_from_sim no) (at 148.59 265.43 0) (size 27.94 5.08) (margins 0.9525 0.9525 0.9525 0.9525) (span 1 1) (fill (type none)) (effects (font (size 1.27 1.27)) (justify left top))) (table_cell "22 µF 25 V X7R 1210" (exclude_from_sim no) (at 176.53 265.43 0) (size 35.56 5.08) (margins 0.9525 0.9525 0.9525 0.9525) (span 1 1) (fill (type none)) (effects (font (size 1.27 1.27)) (justify left top))) (table_cell "BOM v1 line 121: ≥ 12 µF effective at 5.1 V" (exclude_from_sim no) (at 212.09 265.43 0) (size 55.88 5.08) (margins 0.9525 0.9525 0.9525 0.9525) (span 1 1) (fill (type none)) (effects (font (size 1.27 1.27)) (justify left top)))))
+(table (column_count 3) (border (external yes) (header yes) (stroke (width 0) (type solid))) (separators (rows yes) (cols yes) (stroke (width 0) (type solid))) (column_widths 27.94 35.56 55.88) (row_heights 5.08 7.62 5.08) (cells (table_cell "Rail" (exclude_from_sim no) (at 148.59 255.27 0) (size 27.94 5.08) (margins 0.9525 0.9525 0.9525 0.9525) (span 1 1) (fill (type none)) (effects (font (size 1.27 1.27) (bold yes)) (justify left top))) (table_cell "Capacitors" (exclude_from_sim no) (at 176.53 255.27 0) (size 35.56 5.08) (margins 0.9525 0.9525 0.9525 0.9525) (span 1 1) (fill (type none)) (effects (font (size 1.27 1.27) (bold yes)) (justify left top))) (table_cell "Requirement and source" (exclude_from_sim no) (at 212.09 255.27 0) (size 55.88 5.08) (margins 0.9525 0.9525 0.9525 0.9525) (span 1 1) (fill (type none)) (effects (font (size 1.27 1.27) (bold yes)) (justify left top))) (table_cell "VSYS_P5V1" (exclude_from_sim no) (at 148.59 260.35 0) (size 27.94 7.62) (margins 0.9525 0.9525 0.9525 0.9525) (span 1 1) (fill (type none)) (effects (font (size 1.27 1.27)) (justify left top))) (table_cell "22 µF 25 V" (exclude_from_sim no) (at 176.53 260.35 0) (size 35.56 7.62) (margins 0.9525 0.9525 0.9525 0.9525) (span 1 1) (fill (type none)) (effects (font (size 1.27 1.27)) (justify left top))) (table_cell "SLVSES3A Table 8-1; 3 µF effective minimum (§6.3): 3.9 µF at 8.8 V (BOM v1.18 item 1)" (exclude_from_sim no) (at 212.09 260.35 0) (size 55.88 7.62) (margins 0.9525 0.9525 0.9525 0.9525) (span 1 1) (fill (type none)) (effects (font (size 1.27 1.27)) (justify left top))) (table_cell "P5V1_SRC" (exclude_from_sim no) (at 148.59 267.97 0) (size 27.94 5.08) (margins 0.9525 0.9525 0.9525 0.9525) (span 1 1) (fill (type none)) (effects (font (size 1.27 1.27)) (justify left top))) (table_cell "22 µF 25 V X7R 1210" (exclude_from_sim no) (at 176.53 267.97 0) (size 35.56 5.08) (margins 0.9525 0.9525 0.9525 0.9525) (span 1 1) (fill (type none)) (effects (font (size 1.27 1.27)) (justify left top))) (table_cell "BOM v1 line 121: ≥ 12 µF effective at 5.1 V" (exclude_from_sim no) (at 212.09 267.97 0) (size 55.88 5.08) (margins 0.9525 0.9525 0.9525 0.9525) (span 1 1) (fill (type none)) (effects (font (size 1.27 1.27)) (justify left top)))))
 (wire (pts (xy 72.39 60.96) (xy 73.66 60.96)) (stroke (width 0) (type default)))
 (wire (pts (xy 73.66 60.96) (xy 73.66 59.69)) (stroke (width 0) (type default)))
