File: board/hardware/t1-main-board/haptics.kicad_sch (KiCad schematic)
At the start: 8 parts, among them U5901 DRV2605LDGSR

Commit message: Board: capture blk.current-monitors
Five INA236 on I2C1 (0x40-0x43, 0x48) with their shunts, per power tree
§4.12 and BOM v1 lines 54 and 136. The measured branches are rails of
their own (VSYS_SRC, VSYS_LV_AUDIO, VSYS_AUDIO, VSYS_LV_BL, VSYS_P5V1),
fed through the shunts on this sheet; the charger, audio, backlight and
5.1 V sheets take them. The root's layout may leave a stack level empty,
so the block sits under the notes; IC bboxes hold turned rail values;
passive rows hold a bottom rail's text.

Co-Authored-By: Claude Opus 5.5 <noreply@anthropic.com>
Claude-Session: https://claude.ai/code/session_01Ei262h3TpgY9vyfNLMi5Mn
Parts:
- removed C5901, C5902: 1 µF, Capacitor_SMD:C_0402_1005Metric, symbol Device:C
- removed R5901: 100 mΩ, Resistor_SMD:R_0603_1608Metric, symbol Device:R
- removed TP5901: vcc3v3_sys, TestPoint:TestPoint_Pad_D1.0mm, symbol Connector:TestPoint
- removed TP5902: HAPTIC_VDD, TestPoint:TestPoint_Pad_D1.0mm, symbol Connector:TestPoint
- removed TP5903: LRA_P, TestPoint:TestPoint_Pad_D1.0mm, symbol Connector:TestPoint
- removed TP5904: LRA_N, TestPoint:TestPoint_Pad_D1.0mm, symbol Connector:TestPoint
- removed U5901: DRV2605LDGSR, Texas_Instruments:Texas_DGS0010A_VSSOP-10_3x3mm_P0.5mm, symbol Texas_Instruments:DRV2605LDGSR
- added C6001, C6002: 1 µF, Capacitor_SMD:C_0402_1005Metric, symbol Device:C
- added R6001: 100 mΩ, Resistor_SMD:R_0603_1608Metric, symbol Device:R
- added TP6001: vcc3v3_sys, TestPoint:TestPoint_Pad_D1.0mm, symbol Connector:TestPoint
- added TP6002: HAPTIC_VDD, TestPoint:TestPoint_Pad_D1.0mm, symbol Connector:TestPoint
- added TP6003: LRA_P, TestPoint:TestPoint_Pad_D1.0mm, symbol Connector:TestPoint
- added TP6004: LRA_N, TestPoint:TestPoint_Pad_D1.0mm, symbol Connector:TestPoint
- added U6001: DRV2605LDGSR, Texas_Instruments:Texas_DGS0010A_VSSOP-10_3x3mm_P0.5mm, symbol Texas_Instruments:DRV2605LDGSR
Connections:
- net GND: now also C6001.2, C6002.2, U6001.4 (IN/TRIG), U6001.8 (GND)
- net HAPTIC_EN: now also U6001.5 (EN)
- net HAPTIC_REG: now also C6002.1, U6001.1 (REG)
- net HAPTIC_VDD: now also C6001.1, R6001.2, TP6002.1, U6001.10 (VDD), U6001.6 (VDD/NC)
- net I2C2_SCL: now also U6001.2 (SCL)
- net I2C2_SDA: now also U6001.3 (SDA)
- net LRA_N: now also TP6004.1, U6001.9 (OUT-)
- net LRA_P: now also TP6003.1, U6001.7 (OUT+)
- net vcc3v3_sys: now also R6001.1, TP6001.1
Changed lines of the file:
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@@
 (title_block (title "Haptic driver") (date "2026-10-25") (rev "A") (company "The OpenDAP Project") (comment 1 "blk.haptics") (comment 2 "DRV2605L LRA driver on I2C2 at 0x5A and the actuator contacts"))
 (symbol (lib_id "Texas_Instruments:DRV2605LDGSR") (at 54.61 76.2 0) (unit 1) (body_style 1) (exclude_from_sim no) (in_bom yes) (on_board yes) (dnp no)
-  (property "Reference" "U5901" (at 58.42 54.61 0) (effects (font (size 1.27 1.27)) (justify left)))
+  (property "Reference" "U6001" (at 58.42 54.61 0) (effects (font (size 1.27 1.27)) (justify left)))
   (property "Value" "DRV2605LDGSR" (at 58.42 52.07 0) (effects (font (size 1.27 1.27)) (justify left)))
   (property "Footprint" "Texas_Instruments:Texas_DGS0010A_VSSOP-10_3x3mm_P0.5mm" (at 54.61 76.2 0) (effects (font (size 1.27 1.27))) (hide yes))
@@
   (pin "6")
   (pin "8")
-  (instances (project "t1-main-board" (path "/7746052e-d7f9-59ad-ba73-bd2b74439529/780edba7-5b74-5864-9ee6-3672d6464c18" (reference "U5901") (unit 1))))
+  (instances (project "t1-main-board" (path "/7746052e-d7f9-59ad-ba73-bd2b74439529/780edba7-5b74-5864-9ee6-3672d6464c18" (reference "U6001") (unit 1))))
 )
 (wire (pts (xy 52.07 53.34) (xy 52.07 50.8)) (stroke (width 0) (type default)))
@@
 )
 (symbol (lib_id "Device:C") (at 90.17 57.15 0) (unit 1) (body_style 1) (exclude_from_sim no) (in_bom yes) (on_board yes) (dnp no)
-  (property "Reference" "C5901" (at 92.71 55.88 0) (effects (font (size 1.27 1.27)) (justify left)))
+  (property "Reference" "C6001" (at 92.71 55.88 0) (effects (font (size 1.27 1.27)) (justify left)))
   (property "Value" "1 µF" (at 92.71 58.42 0) (effects (font (size 1.27 1.27)) (justify left)))
   (property "Footprint" "Capacitor_SMD:C_0402_1005Metric" (at 90.17 57.15 0) (effects (font (size 1.27 1.27))) (hide yes))
@@
   (pin "1")
   (pin "2")
-  (instances (project "t1-main-board" (path "/7746052e-d7f9-59ad-ba73-bd2b74439529/780edba7-5b74-5864-9ee6-3672d6464c18" (reference "C5901") (unit 1))))
+  (instances (project "t1-main-board" (path "/7746052e-d7f9-59ad-ba73-bd2b74439529/780edba7-5b74-5864-9ee6-3672d6464c18" (reference "C6001") (unit 1))))
 )
 (wire (pts (xy 90.17 53.34) (xy 90.17 50.8)) (stroke (width 0) (type default)))
@@
 )
 (symbol (lib_id "Device:C") (at 102.87 57.15 0) (unit 1) (body_style 1) (exclude_from_sim no) (in_bom yes) (on_board yes) (dnp no)
-  (property "Reference" "C5902" (at 105.41 55.88 0) (effects (font (size 1.27 1.27)) (justify left)))
+  (property "Reference" "C6002" (at 105.41 55.88 0) (effects (font (size 1.27 1.27)) (justify left)))
   (property "Value" "1 µF" (at 105.41 58.42 0) (effects (font (size 1.27 1.27)) (justify left)))
   (property "Footprint" "Capacitor_SMD:C_0402_1005Metric" (at 102.87 57.15 0) (effects (font (size 1.27 1.27))) (hide yes))
@@
   (pin "1")
   (pin "2")
-  (instances (project "t1-main-board" (path "/7746052e-d7f9-59ad-ba73-bd2b74439529/780edba7-5b74-5864-9ee6-3672d6464c18" (reference "C5902") (unit 1))))
+  (instances (project "t1-main-board" (path "/7746052e-d7f9-59ad-ba73-bd2b74439529/780edba7-5b74-5864-9ee6-3672d6464c18" (reference "C6002") (unit 1))))
 )
 (wire (pts (xy 102.87 53.34) (xy 102.87 50.8)) (stroke (width 0) (type default)))
@@
 (text "DRV2605L at I2C2 0x5A (BOM v1 line 123)" (exclude_from_sim no) (at 24.13 34.29 0) (effects (font (size 2.54 2.54)) (justify left bottom)))
 (symbol (lib_id "Device:R") (at 157.48 50.8 90) (unit 1) (body_style 1) (exclude_from_sim no) (in_bom yes) (on_board yes) (dnp no)
-  (property "Reference" "R5901" (at 154.94 46.99 90) (effects (font (size 1.27 1.27))))
+  (property "Reference" "R6001" (at 154.94 46.99 90) (effects (font (size 1.27 1.27))))
   (property "Value" "100 mΩ" (at 154.94 53.34 90) (effects (font (size 1.27 1.27))))
   (property "Spec" "0603" (at 154.94 55.88 90) (effects (font (size 1.27 1.27))))
@@
   (pin "1")
   (pin "2")
-  (instances (project "t1-main-board" (path "/7746052e-d7f9-59ad-ba73-bd2b74439529/780edba7-5b74-5864-9ee6-3672d6464c18" (reference "R5901") (unit 1) (variant (name "production") (field (name "Value") (value "0 Ω")) (field (name "MPN") (value "RC0603JR-070RL")) (field (name "Manufacturer") (value "YAGEO"))))))
+  (instances (project "t1-main-board" (path "/7746052e-d7f9-59ad-ba73-bd2b74439529/780edba7-5b74-5864-9ee6-3672d6464c18" (reference "R6001") (unit 1) (variant (name "production") (field (name "Value") (value "0 Ω")) (field (name "MPN") (value "RC0603JR-070RL")) (field (name "Manufacturer") (value "YAGEO"))))))
 )
 (rectangle (start 135.89 38.1) (end 179.07 58.42) (stroke (width 0) (type dash)) (fill (type none)))
@@
 (wire (pts (xy 151.13 50.8) (xy 151.13 48.26)) (stroke (width 0) (type default)))
 (symbol (lib_id "Connector:TestPoint") (at 151.13 48.26 0) (unit 1) (body_style 1) (exclude_from_sim no) (in_bom no) (on_board yes) (dnp no)
-  (property "Reference" "TP5901" (at 149.86 43.18 0) (effects (font (size 1.27 1.27)) (justify right)))
+  (property "Reference" "TP6001" (at 149.86 43.18 0) (effects (font (size 1.27 1.27)) (justify right)))
   (property "Value" "vcc3v3_sys" (at 149.86 45.72 0) (effects (font (size 1.27 1.27)) (justify right)))
   (property "Footprint" "TestPoint:TestPoint_Pad_D1.0mm" (at 151.13 48.26 0) (effects (font (size 1.27 1.27))) (hide yes))
@@
   (property "Block" "blk.haptics" (at 151.13 48.26 0) (effects (font (size 1.27 1.27))) (hide yes))
   (pin "1")
-  (instances (project "t1-main-board" (path "/7746052e-d7f9-59ad-ba73-bd2b74439529/780edba7-5b74-5864-9ee6-3672d6464c18" (reference "TP5901") (unit 1))))
+  (instances (project "t1-main-board" (path "/7746052e-d7f9-59ad-ba73-bd2b74439529/780edba7-5b74-5864-9ee6-3672d6464c18" (reference "TP6001") (unit 1))))
 )
 (symbol (lib_id "power:VCC") (at 133.35 50.8 90) (unit 1) (body_style 1) (exclude_from_sim no) (in_bom yes) (on_board yes) (dnp no)
@@
 (wire (pts (xy 163.83 50.8) (xy 163.83 48.26)) (stroke (width 0) (type default)))
 (symbol (lib_id "Connector:TestPoint") (at 163.83 48.26 0) (unit 1) (body_style 1) (exclude_from_sim no) (in_bom no) (on_board yes) (dnp no)
-  (property "Reference" "TP5902" (at 165.1 43.18 0) (effects (font (size 1.27 1.27)) (justify left)))
+  (property "Reference" "TP6002" (at 165.1 43.18 0) (effects (font (size 1.27 1.27)) (justify left)))
   (property "Value" "HAPTIC_VDD" (at 165.1 45.72 0) (effects (font (size 1.27 1.27)) (justify left)))
   (property "Footprint" "TestPoint:TestPoint_Pad_D1.0mm" (at 163.83 48.26 0) (effects (font (size 1.27 1.27))) (hide yes))
@@
   (property "Block" "blk.haptics" (at 163.83 48.26 0) (effects (font (size 1.27 1.27))) (hide yes))
   (pin "1")
-  (instances (project "t1-main-board" (path "/7746052e-d7f9-59ad-ba73-bd2b74439529/780edba7-5b74-5864-9ee6-3672d6464c18" (reference "TP5902") (unit 1))))
+  (instances (project "t1-main-board" (path "/7746052e-d7f9-59ad-ba73-bd2b74439529/780edba7-5b74-5864-9ee6-3672d6464c18" (reference "TP6002") (unit 1))))
 )
 (junction (at 186.69 50.8) (diameter 0) (color 0 0 0 0))
@@
 )
 (symbol (lib_id "Connector:TestPoint") (at 132.08 81.28 0) (unit 1) (body_style 1) (exclude_from_sim no) (in_bom no) (on_board yes) (dnp no)
-  (property "Reference" "TP5903" (at 130.81 76.2 0) (effects (font (size 1.27 1.27)) (justify right)))
+  (property "Reference" "TP6003" (at 130.81 76.2 0) (effects (font (size 1.27 1.27)) (justify right)))
   (property "Value" "LRA_P" (at 130.81 78.74 0) (effects (font (size 1.27 1.27)) (justify right)))
   (property "Footprint" "TestPoint:TestPoint_Pad_D1.0mm" (at 132.08 81.28 0) (effects (font (size 1.27 1.27))) (hide yes))
@@
   (property "Block" "blk.haptics" (at 132.08 81.28 0) (effects (font (size 1.27 1.27))) (hide yes))
   (pin "1")
-  (instances (project "t1-main-board" (path "/7746052e-d7f9-59ad-ba73-bd2b74439529/780edba7-5b74-5864-9ee6-3672d6464c18" (reference "TP5903") (unit 1))))
+  (instances (project "t1-main-board" (path "/7746052e-d7f9-59ad-ba73-bd2b74439529/780edba7-5b74-5864-9ee6-3672d6464c18" (reference "TP6003") (unit 1))))
 )
 (symbol (lib_id "Connector:TestPoint") (at 149.86 81.28 0) (unit 1) (body_style 1) (exclude_from_sim no) (in_bom no) (on_board yes) (dnp no)
-  (property "Reference" "TP5904" (at 148.59 76.2 0) (effects (font (size 1.27 1.27)) (justify right)))
+  (property "Reference" "TP6004" (at 148.59 76.2 0) (effects (font (size 1.27 1.27)) (justify right)))
   (property "Value" "LRA_N" (at 148.59 78.74 0) (effects (font (size 1.27 1.27)) (justify right)))
   (property "Footprint" "TestPoint:TestPoint_Pad_D1.0mm" (at 149.86 81.28 0) (effects (font (size 1.27 1.27))) (hide yes))
@@
   (property "Block" "blk.haptics" (at 149.86 81.28 0) (effects (font (size 1.27 1.27))) (hide yes))
   (pin "1")
-  (instances (project "t1-main-board" (path "/7746052e-d7f9-59ad-ba73-bd2b74439529/780edba7-5b74-5864-9ee6-3672d6464c18" (reference "TP5904") (unit 1))))
+  (instances (project "t1-main-board" (path "/7746052e-d7f9-59ad-ba73-bd2b74439529/780edba7-5b74-5864-9ee6-3672d6464c18" (reference "TP6004") (unit 1))))
 )
 (rectangle (start 120.65 71.12) (end 191.77 92.71) (stroke (width 0) (type dash)) (fill (type none)))

Commit message: Board: capture blk.status-led
LP5521 at 0x32 on I2C2 (BOM v1 line 105) with its charge-pump
capacitors, EN on vcca1v8_pmu, VDD from VSYS_LV through link #22;
LED_R/G/B reach the faceplate connector as the LED bus alias. The
faceplate row of the root is re-packed so five full columns sit left of
the title block.

Co-Authored-By: Claude Opus 5.5 <noreply@anthropic.com>
Claude-Session: https://claude.ai/code/session_01Ei262h3TpgY9vyfNLMi5Mn
Parts:
- removed C6001, C6002: 1 µF, Capacitor_SMD:C_0402_1005Metric, symbol Device:C
- removed R6001: 100 mΩ, Resistor_SMD:R_0603_1608Metric, symbol Device:R
- removed TP6001: vcc3v3_sys, TestPoint:TestPoint_Pad_D1.0mm, symbol Connector:TestPoint
- removed TP6002: HAPTIC_VDD, TestPoint:TestPoint_Pad_D1.0mm, symbol Connector:TestPoint
- removed TP6003: LRA_P, TestPoint:TestPoint_Pad_D1.0mm, symbol Connector:TestPoint
- removed TP6004: LRA_N, TestPoint:TestPoint_Pad_D1.0mm, symbol Connector:TestPoint
- removed U6001: DRV2605LDGSR, Texas_Instruments:Texas_DGS0010A_VSSOP-10_3x3mm_P0.5mm, symbol Texas_Instruments:DRV2605LDGSR
- added C6401, C6402: 1 µF, Capacitor_SMD:C_0402_1005Metric, symbol Device:C
- added R6401: 100 mΩ, Resistor_SMD:R_0603_1608Metric, symbol Device:R
- added TP6401: vcc3v3_sys, TestPoint:TestPoint_Pad_D1.0mm, symbol Connector:TestPoint
- added TP6402: HAPTIC_VDD, TestPoint:TestPoint_Pad_D1.0mm, symbol Connector:TestPoint
- added TP6403: LRA_P, TestPoint:TestPoint_Pad_D1.0mm, symbol Connector:TestPoint
- added TP6404: LRA_N, TestPoint:TestPoint_Pad_D1.0mm, symbol Connector:TestPoint
- added U6401: DRV2605LDGSR, Texas_Instruments:Texas_DGS0010A_VSSOP-10_3x3mm_P0.5mm, symbol Texas_Instruments:DRV2605LDGSR
Connections:
- net GND: now also C6401.2, C6402.2, U6401.4 (IN/TRIG), U6401.8 (GND)
- net HAPTIC_EN: now also U6401.5 (EN)
- net HAPTIC_REG: now also C6402.1, U6401.1 (REG)
- net HAPTIC_VDD: now also C6401.1, R6401.2, TP6402.1, U6401.10 (VDD), U6401.6 (VDD/NC)
- net I2C2_SCL: now also U6401.2 (SCL)
- net I2C2_SDA: now also U6401.3 (SDA)
- net LRA_N: now also TP6404.1, U6401.9 (OUT-)
- net LRA_P: now also TP6403.1, U6401.7 (OUT+)
- net vcc3v3_sys: now also R6401.1, TP6401.1
Changed lines of the file:
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@@
 (title_block (title "Haptic driver") (date "2026-10-25") (rev "A") (company "The OpenDAP Project") (comment 1 "blk.haptics") (comment 2 "DRV2605L LRA driver on I2C2 at 0x5A and the actuator contacts"))
 (symbol (lib_id "Texas_Instruments:DRV2605LDGSR") (at 54.61 76.2 0) (unit 1) (body_style 1) (exclude_from_sim no) (in_bom yes) (on_board yes) (dnp no)
-  (property "Reference" "U6001" (at 58.42 54.61 0) (effects (font (size 1.27 1.27)) (justify left)))
+  (property "Reference" "U6401" (at 58.42 54.61 0) (effects (font (size 1.27 1.27)) (justify left)))
   (property "Value" "DRV2605LDGSR" (at 58.42 52.07 0) (effects (font (size 1.27 1.27)) (justify left)))
   (property "Footprint" "Texas_Instruments:Texas_DGS0010A_VSSOP-10_3x3mm_P0.5mm" (at 54.61 76.2 0) (effects (font (size 1.27 1.27))) (hide yes))
@@
   (pin "6")
   (pin "8")
-  (instances (project "t1-main-board" (path "/7746052e-d7f9-59ad-ba73-bd2b74439529/780edba7-5b74-5864-9ee6-3672d6464c18" (reference "U6001") (unit 1))))
+  (instances (project "t1-main-board" (path "/7746052e-d7f9-59ad-ba73-bd2b74439529/780edba7-5b74-5864-9ee6-3672d6464c18" (reference "U6401") (unit 1))))
 )
 (wire (pts (xy 52.07 53.34) (xy 52.07 50.8)) (stroke (width 0) (type default)))
@@
 )
 (symbol (lib_id "Device:C") (at 90.17 57.15 0) (unit 1) (body_style 1) (exclude_from_sim no) (in_bom yes) (on_board yes) (dnp no)
-  (property "Reference" "C6001" (at 92.71 55.88 0) (effects (font (size 1.27 1.27)) (justify left)))
+  (property "Reference" "C6401" (at 92.71 55.88 0) (effects (font (size 1.27 1.27)) (justify left)))
   (property "Value" "1 µF" (at 92.71 58.42 0) (effects (font (size 1.27 1.27)) (justify left)))
   (property "Footprint" "Capacitor_SMD:C_0402_1005Metric" (at 90.17 57.15 0) (effects (font (size 1.27 1.27))) (hide yes))
@@
   (pin "1")
   (pin "2")
-  (instances (project "t1-main-board" (path "/7746052e-d7f9-59ad-ba73-bd2b74439529/780edba7-5b74-5864-9ee6-3672d6464c18" (reference "C6001") (unit 1))))
+  (instances (project "t1-main-board" (path "/7746052e-d7f9-59ad-ba73-bd2b74439529/780edba7-5b74-5864-9ee6-3672d6464c18" (reference "C6401") (unit 1))))
 )
 (wire (pts (xy 90.17 53.34) (xy 90.17 50.8)) (stroke (width 0) (type default)))
@@
 )
 (symbol (lib_id "Device:C") (at 102.87 57.15 0) (unit 1) (body_style 1) (exclude_from_sim no) (in_bom yes) (on_board yes) (dnp no)
-  (property "Reference" "C6002" (at 105.41 55.88 0) (effects (font (size 1.27 1.27)) (justify left)))
+  (property "Reference" "C6402" (at 105.41 55.88 0) (effects (font (size 1.27 1.27)) (justify left)))
   (property "Value" "1 µF" (at 105.41 58.42 0) (effects (font (size 1.27 1.27)) (justify left)))
   (property "Footprint" "Capacitor_SMD:C_0402_1005Metric" (at 102.87 57.15 0) (effects (font (size 1.27 1.27))) (hide yes))
@@
   (pin "1")
   (pin "2")
-  (instances (project "t1-main-board" (path "/7746052e-d7f9-59ad-ba73-bd2b74439529/780edba7-5b74-5864-9ee6-3672d6464c18" (reference "C6002") (unit 1))))
+  (instances (project "t1-main-board" (path "/7746052e-d7f9-59ad-ba73-bd2b74439529/780edba7-5b74-5864-9ee6-3672d6464c18" (reference "C6402") (unit 1))))
 )
 (wire (pts (xy 102.87 53.34) (xy 102.87 50.8)) (stroke (width 0) (type default)))
@@
 (text "DRV2605L at I2C2 0x5A (BOM v1 line 123)" (exclude_from_sim no) (at 24.13 34.29 0) (effects (font (size 2.54 2.54)) (justify left bottom)))
 (symbol (lib_id "Device:R") (at 157.48 50.8 90) (unit 1) (body_style 1) (exclude_from_sim no) (in_bom yes) (on_board yes) (dnp no)
-  (property "Reference" "R6001" (at 154.94 46.99 90) (effects (font (size 1.27 1.27))))
+  (property "Reference" "R6401" (at 154.94 46.99 90) (effects (font (size 1.27 1.27))))
   (property "Value" "100 mΩ" (at 154.94 53.34 90) (effects (font (size 1.27 1.27))))
   (property "Spec" "0603" (at 154.94 55.88 90) (effects (font (size 1.27 1.27))))
@@
   (pin "1")
   (pin "2")
-  (instances (project "t1-main-board" (path "/7746052e-d7f9-59ad-ba73-bd2b74439529/780edba7-5b74-5864-9ee6-3672d6464c18" (reference "R6001") (unit 1) (variant (name "production") (field (name "Value") (value "0 Ω")) (field (name "MPN") (value "RC0603JR-070RL")) (field (name "Manufacturer") (value "YAGEO"))))))
+  (instances (project "t1-main-board" (path "/7746052e-d7f9-59ad-ba73-bd2b74439529/780edba7-5b74-5864-9ee6-3672d6464c18" (reference "R6401") (unit 1) (variant (name "production") (field (name "Value") (value "0 Ω")) (field (name "MPN") (value "RC0603JR-070RL")) (field (name "Manufacturer") (value "YAGEO"))))))
 )
 (rectangle (start 135.89 38.1) (end 179.07 58.42) (stroke (width 0) (type dash)) (fill (type none)))
@@
 (wire (pts (xy 151.13 50.8) (xy 151.13 48.26)) (stroke (width 0) (type default)))
 (symbol (lib_id "Connector:TestPoint") (at 151.13 48.26 0) (unit 1) (body_style 1) (exclude_from_sim no) (in_bom no) (on_board yes) (dnp no)
-  (property "Reference" "TP6001" (at 149.86 43.18 0) (effects (font (size 1.27 1.27)) (justify right)))
+  (property "Reference" "TP6401" (at 149.86 43.18 0) (effects (font (size 1.27 1.27)) (justify right)))
   (property "Value" "vcc3v3_sys" (at 149.86 45.72 0) (effects (font (size 1.27 1.27)) (justify right)))
   (property "Footprint" "TestPoint:TestPoint_Pad_D1.0mm" (at 151.13 48.26 0) (effects (font (size 1.27 1.27))) (hide yes))
@@
   (property "Block" "blk.haptics" (at 151.13 48.26 0) (effects (font (size 1.27 1.27))) (hide yes))
   (pin "1")
-  (instances (project "t1-main-board" (path "/7746052e-d7f9-59ad-ba73-bd2b74439529/780edba7-5b74-5864-9ee6-3672d6464c18" (reference "TP6001") (unit 1))))
+  (instances (project "t1-main-board" (path "/7746052e-d7f9-59ad-ba73-bd2b74439529/780edba7-5b74-5864-9ee6-3672d6464c18" (reference "TP6401") (unit 1))))
 )
 (symbol (lib_id "power:VCC") (at 133.35 50.8 90) (unit 1) (body_style 1) (exclude_from_sim no) (in_bom yes) (on_board yes) (dnp no)
@@
 (wire (pts (xy 163.83 50.8) (xy 163.83 48.26)) (stroke (width 0) (type default)))
 (symbol (lib_id "Connector:TestPoint") (at 163.83 48.26 0) (unit 1) (body_style 1) (exclude_from_sim no) (in_bom no) (on_board yes) (dnp no)
-  (property "Reference" "TP6002" (at 165.1 43.18 0) (effects (font (size 1.27 1.27)) (justify left)))
+  (property "Reference" "TP6402" (at 165.1 43.18 0) (effects (font (size 1.27 1.27)) (justify left)))
   (property "Value" "HAPTIC_VDD" (at 165.1 45.72 0) (effects (font (size 1.27 1.27)) (justify left)))
   (property "Footprint" "TestPoint:TestPoint_Pad_D1.0mm" (at 163.83 48.26 0) (effects (font (size 1.27 1.27))) (hide yes))
@@
   (property "Block" "blk.haptics" (at 163.83 48.26 0) (effects (font (size 1.27 1.27))) (hide yes))
   (pin "1")
-  (instances (project "t1-main-board" (path "/7746052e-d7f9-59ad-ba73-bd2b74439529/780edba7-5b74-5864-9ee6-3672d6464c18" (reference "TP6002") (unit 1))))
+  (instances (project "t1-main-board" (path "/7746052e-d7f9-59ad-ba73-bd2b74439529/780edba7-5b74-5864-9ee6-3672d6464c18" (reference "TP6402") (unit 1))))
 )
 (junction (at 186.69 50.8) (diameter 0) (color 0 0 0 0))
@@
 )
 (symbol (lib_id "Connector:TestPoint") (at 132.08 81.28 0) (unit 1) (body_style 1) (exclude_from_sim no) (in_bom no) (on_board yes) (dnp no)
-  (property "Reference" "TP6003" (at 130.81 76.2 0) (effects (font (size 1.27 1.27)) (justify right)))
+  (property "Reference" "TP6403" (at 130.81 76.2 0) (effects (font (size 1.27 1.27)) (justify right)))
   (property "Value" "LRA_P" (at 130.81 78.74 0) (effects (font (size 1.27 1.27)) (justify right)))
   (property "Footprint" "TestPoint:TestPoint_Pad_D1.0mm" (at 132.08 81.28 0) (effects (font (size 1.27 1.27))) (hide yes))
@@
   (property "Block" "blk.haptics" (at 132.08 81.28 0) (effects (font (size 1.27 1.27))) (hide yes))
   (pin "1")
-  (instances (project "t1-main-board" (path "/7746052e-d7f9-59ad-ba73-bd2b74439529/780edba7-5b74-5864-9ee6-3672d6464c18" (reference "TP6003") (unit 1))))
+  (instances (project "t1-main-board" (path "/7746052e-d7f9-59ad-ba73-bd2b74439529/780edba7-5b74-5864-9ee6-3672d6464c18" (reference "TP6403") (unit 1))))
 )
 (symbol (lib_id "Connector:TestPoint") (at 149.86 81.28 0) (unit 1) (body_style 1) (exclude_from_sim no) (in_bom no) (on_board yes) (dnp no)
-  (property "Reference" "TP6004" (at 148.59 76.2 0) (effects (font (size 1.27 1.27)) (justify right)))
+  (property "Reference" "TP6404" (at 148.59 76.2 0) (effects (font (size 1.27 1.27)) (justify right)))
   (property "Value" "LRA_N" (at 148.59 78.74 0) (effects (font (size 1.27 1.27)) (justify right)))
   (property "Footprint" "TestPoint:TestPoint_Pad_D1.0mm" (at 149.86 81.28 0) (effects (font (size 1.27 1.27))) (hide yes))
@@
   (property "Block" "blk.haptics" (at 149.86 81.28 0) (effects (font (size 1.27 1.27))) (hide yes))
   (pin "1")
-  (instances (project "t1-main-board" (path "/7746052e-d7f9-59ad-ba73-bd2b74439529/780edba7-5b74-5864-9ee6-3672d6464c18" (reference "TP6004") (unit 1))))
+  (instances (project "t1-main-board" (path "/7746052e-d7f9-59ad-ba73-bd2b74439529/780edba7-5b74-5864-9ee6-3672d6464c18" (reference "TP6404") (unit 1))))
 )
 (rectangle (start 120.65 71.12) (end 191.77 92.71) (stroke (width 0) (type dash)) (fill (type none)))
