File: board/hardware/t1-main-board/haptics.kicad_sch (KiCad schematic)
At the start: 8 parts, among them U6401 DRV2605LDGSR

Commit message: Board: capture blk.debug
Debug UART2 (1.8 V) and I2S/DSD pads with ground pads, reset, PMIC and
power-key pads (PCB-T-09), a pad on every spare SoC GPIO whose pinout v1
row names one (the DEBUG bus, on the SoC's right edge), and a rail pad
for each power-tree rail no other sheet probes (PCB-T-02). Each DAC
sheet carries a pad on its MCLK. The spares pinout v1 leaves without a
pad now carry no-connect flags. On the root, facing sheet pins are
joined directly only where the route meets no other symbol.

Co-Authored-By: Claude Opus 5.5 <noreply@anthropic.com>
Claude-Session: https://claude.ai/code/session_01Ei262h3TpgY9vyfNLMi5Mn
Parts:
- removed C6401, C6402: 1 µF, Capacitor_SMD:C_0402_1005Metric, symbol Device:C
- removed R6401: 100 mΩ, Resistor_SMD:R_0603_1608Metric, symbol Device:R
- removed TP6401: vcc3v3_sys, TestPoint:TestPoint_Pad_D1.0mm, symbol Connector:TestPoint
- removed TP6402: HAPTIC_VDD, TestPoint:TestPoint_Pad_D1.0mm, symbol Connector:TestPoint
- removed TP6403: LRA_P, TestPoint:TestPoint_Pad_D1.0mm, symbol Connector:TestPoint
- removed TP6404: LRA_N, TestPoint:TestPoint_Pad_D1.0mm, symbol Connector:TestPoint
- removed U6401: DRV2605LDGSR, Texas_Instruments:Texas_DGS0010A_VSSOP-10_3x3mm_P0.5mm, symbol Texas_Instruments:DRV2605LDGSR
- added C6501, C6502: 1 µF, Capacitor_SMD:C_0402_1005Metric, symbol Device:C
- added R6501: 100 mΩ, Resistor_SMD:R_0603_1608Metric, symbol Device:R
- added TP6501: vcc3v3_sys, TestPoint:TestPoint_Pad_D1.0mm, symbol Connector:TestPoint
- added TP6502: HAPTIC_VDD, TestPoint:TestPoint_Pad_D1.0mm, symbol Connector:TestPoint
- added TP6503: LRA_P, TestPoint:TestPoint_Pad_D1.0mm, symbol Connector:TestPoint
- added TP6504: LRA_N, TestPoint:TestPoint_Pad_D1.0mm, symbol Connector:TestPoint
- added U6501: DRV2605LDGSR, Texas_Instruments:Texas_DGS0010A_VSSOP-10_3x3mm_P0.5mm, symbol Texas_Instruments:DRV2605LDGSR
Connections:
- net GND: now also C6501.2, C6502.2, U6501.4 (IN/TRIG), U6501.8 (GND)
- net HAPTIC_EN: now also U6501.5 (EN)
- net HAPTIC_REG: now also C6502.1, U6501.1 (REG)
- net HAPTIC_VDD: now also C6501.1, R6501.2, TP6502.1, U6501.10 (VDD), U6501.6 (VDD/NC)
- net I2C2_SCL: now also U6501.2 (SCL)
- net I2C2_SDA: now also U6501.3 (SDA)
- net LRA_N: now also TP6504.1, U6501.9 (OUT-)
- net LRA_P: now also TP6503.1, U6501.7 (OUT+)
- net vcc3v3_sys: now also R6501.1, TP6501.1
Changed lines of the file:
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@@
 (title_block (title "Haptic driver") (date "2026-10-25") (rev "A") (company "The OpenDAP Project") (comment 1 "blk.haptics") (comment 2 "DRV2605L LRA driver on I2C2 at 0x5A and the actuator contacts"))
 (symbol (lib_id "Texas_Instruments:DRV2605LDGSR") (at 54.61 76.2 0) (unit 1) (body_style 1) (exclude_from_sim no) (in_bom yes) (on_board yes) (dnp no)
-  (property "Reference" "U6401" (at 58.42 54.61 0) (effects (font (size 1.27 1.27)) (justify left)))
+  (property "Reference" "U6501" (at 58.42 54.61 0) (effects (font (size 1.27 1.27)) (justify left)))
   (property "Value" "DRV2605LDGSR" (at 58.42 52.07 0) (effects (font (size 1.27 1.27)) (justify left)))
   (property "Footprint" "Texas_Instruments:Texas_DGS0010A_VSSOP-10_3x3mm_P0.5mm" (at 54.61 76.2 0) (effects (font (size 1.27 1.27))) (hide yes))
@@
   (pin "6")
   (pin "8")
-  (instances (project "t1-main-board" (path "/7746052e-d7f9-59ad-ba73-bd2b74439529/780edba7-5b74-5864-9ee6-3672d6464c18" (reference "U6401") (unit 1))))
+  (instances (project "t1-main-board" (path "/7746052e-d7f9-59ad-ba73-bd2b74439529/780edba7-5b74-5864-9ee6-3672d6464c18" (reference "U6501") (unit 1))))
 )
 (wire (pts (xy 52.07 53.34) (xy 52.07 50.8)) (stroke (width 0) (type default)))
@@
 )
 (symbol (lib_id "Device:C") (at 90.17 57.15 0) (unit 1) (body_style 1) (exclude_from_sim no) (in_bom yes) (on_board yes) (dnp no)
-  (property "Reference" "C6401" (at 92.71 55.88 0) (effects (font (size 1.27 1.27)) (justify left)))
+  (property "Reference" "C6501" (at 92.71 55.88 0) (effects (font (size 1.27 1.27)) (justify left)))
   (property "Value" "1 µF" (at 92.71 58.42 0) (effects (font (size 1.27 1.27)) (justify left)))
   (property "Footprint" "Capacitor_SMD:C_0402_1005Metric" (at 90.17 57.15 0) (effects (font (size 1.27 1.27))) (hide yes))
@@
   (pin "1")
   (pin "2")
-  (instances (project "t1-main-board" (path "/7746052e-d7f9-59ad-ba73-bd2b74439529/780edba7-5b74-5864-9ee6-3672d6464c18" (reference "C6401") (unit 1))))
+  (instances (project "t1-main-board" (path "/7746052e-d7f9-59ad-ba73-bd2b74439529/780edba7-5b74-5864-9ee6-3672d6464c18" (reference "C6501") (unit 1))))
 )
 (wire (pts (xy 90.17 53.34) (xy 90.17 50.8)) (stroke (width 0) (type default)))
@@
 )
 (symbol (lib_id "Device:C") (at 102.87 57.15 0) (unit 1) (body_style 1) (exclude_from_sim no) (in_bom yes) (on_board yes) (dnp no)
-  (property "Reference" "C6402" (at 105.41 55.88 0) (effects (font (size 1.27 1.27)) (justify left)))
+  (property "Reference" "C6502" (at 105.41 55.88 0) (effects (font (size 1.27 1.27)) (justify left)))
   (property "Value" "1 µF" (at 105.41 58.42 0) (effects (font (size 1.27 1.27)) (justify left)))
   (property "Footprint" "Capacitor_SMD:C_0402_1005Metric" (at 102.87 57.15 0) (effects (font (size 1.27 1.27))) (hide yes))
@@
   (pin "1")
   (pin "2")
-  (instances (project "t1-main-board" (path "/7746052e-d7f9-59ad-ba73-bd2b74439529/780edba7-5b74-5864-9ee6-3672d6464c18" (reference "C6402") (unit 1))))
+  (instances (project "t1-main-board" (path "/7746052e-d7f9-59ad-ba73-bd2b74439529/780edba7-5b74-5864-9ee6-3672d6464c18" (reference "C6502") (unit 1))))
 )
 (wire (pts (xy 102.87 53.34) (xy 102.87 50.8)) (stroke (width 0) (type default)))
@@
 (text "DRV2605L at I2C2 0x5A (BOM v1 line 123)" (exclude_from_sim no) (at 24.13 34.29 0) (effects (font (size 2.54 2.54)) (justify left bottom)))
 (symbol (lib_id "Device:R") (at 157.48 50.8 90) (unit 1) (body_style 1) (exclude_from_sim no) (in_bom yes) (on_board yes) (dnp no)
-  (property "Reference" "R6401" (at 154.94 46.99 90) (effects (font (size 1.27 1.27))))
+  (property "Reference" "R6501" (at 154.94 46.99 90) (effects (font (size 1.27 1.27))))
   (property "Value" "100 mΩ" (at 154.94 53.34 90) (effects (font (size 1.27 1.27))))
   (property "Spec" "0603" (at 154.94 55.88 90) (effects (font (size 1.27 1.27))))
@@
   (pin "1")
   (pin "2")
-  (instances (project "t1-main-board" (path "/7746052e-d7f9-59ad-ba73-bd2b74439529/780edba7-5b74-5864-9ee6-3672d6464c18" (reference "R6401") (unit 1) (variant (name "production") (field (name "Value") (value "0 Ω")) (field (name "MPN") (value "RC0603JR-070RL")) (field (name "Manufacturer") (value "YAGEO"))))))
+  (instances (project "t1-main-board" (path "/7746052e-d7f9-59ad-ba73-bd2b74439529/780edba7-5b74-5864-9ee6-3672d6464c18" (reference "R6501") (unit 1) (variant (name "production") (field (name "Value") (value "0 Ω")) (field (name "MPN") (value "RC0603JR-070RL")) (field (name "Manufacturer") (value "YAGEO"))))))
 )
 (rectangle (start 135.89 38.1) (end 179.07 58.42) (stroke (width 0) (type dash)) (fill (type none)))
@@
 (wire (pts (xy 151.13 50.8) (xy 151.13 48.26)) (stroke (width 0) (type default)))
 (symbol (lib_id "Connector:TestPoint") (at 151.13 48.26 0) (unit 1) (body_style 1) (exclude_from_sim no) (in_bom no) (on_board yes) (dnp no)
-  (property "Reference" "TP6401" (at 149.86 43.18 0) (effects (font (size 1.27 1.27)) (justify right)))
+  (property "Reference" "TP6501" (at 149.86 43.18 0) (effects (font (size 1.27 1.27)) (justify right)))
   (property "Value" "vcc3v3_sys" (at 149.86 45.72 0) (effects (font (size 1.27 1.27)) (justify right)))
   (property "Footprint" "TestPoint:TestPoint_Pad_D1.0mm" (at 151.13 48.26 0) (effects (font (size 1.27 1.27))) (hide yes))
@@
   (property "Block" "blk.haptics" (at 151.13 48.26 0) (effects (font (size 1.27 1.27))) (hide yes))
   (pin "1")
-  (instances (project "t1-main-board" (path "/7746052e-d7f9-59ad-ba73-bd2b74439529/780edba7-5b74-5864-9ee6-3672d6464c18" (reference "TP6401") (unit 1))))
+  (instances (project "t1-main-board" (path "/7746052e-d7f9-59ad-ba73-bd2b74439529/780edba7-5b74-5864-9ee6-3672d6464c18" (reference "TP6501") (unit 1))))
 )
 (symbol (lib_id "power:VCC") (at 133.35 50.8 90) (unit 1) (body_style 1) (exclude_from_sim no) (in_bom yes) (on_board yes) (dnp no)
@@
 (wire (pts (xy 163.83 50.8) (xy 163.83 48.26)) (stroke (width 0) (type default)))
 (symbol (lib_id "Connector:TestPoint") (at 163.83 48.26 0) (unit 1) (body_style 1) (exclude_from_sim no) (in_bom no) (on_board yes) (dnp no)
-  (property "Reference" "TP6402" (at 165.1 43.18 0) (effects (font (size 1.27 1.27)) (justify left)))
+  (property "Reference" "TP6502" (at 165.1 43.18 0) (effects (font (size 1.27 1.27)) (justify left)))
   (property "Value" "HAPTIC_VDD" (at 165.1 45.72 0) (effects (font (size 1.27 1.27)) (justify left)))
   (property "Footprint" "TestPoint:TestPoint_Pad_D1.0mm" (at 163.83 48.26 0) (effects (font (size 1.27 1.27))) (hide yes))
@@
   (property "Block" "blk.haptics" (at 163.83 48.26 0) (effects (font (size 1.27 1.27))) (hide yes))
   (pin "1")
-  (instances (project "t1-main-board" (path "/7746052e-d7f9-59ad-ba73-bd2b74439529/780edba7-5b74-5864-9ee6-3672d6464c18" (reference "TP6402") (unit 1))))
+  (instances (project "t1-main-board" (path "/7746052e-d7f9-59ad-ba73-bd2b74439529/780edba7-5b74-5864-9ee6-3672d6464c18" (reference "TP6502") (unit 1))))
 )
 (junction (at 186.69 50.8) (diameter 0) (color 0 0 0 0))
@@
 )
 (symbol (lib_id "Connector:TestPoint") (at 132.08 81.28 0) (unit 1) (body_style 1) (exclude_from_sim no) (in_bom no) (on_board yes) (dnp no)
-  (property "Reference" "TP6403" (at 130.81 76.2 0) (effects (font (size 1.27 1.27)) (justify right)))
+  (property "Reference" "TP6503" (at 130.81 76.2 0) (effects (font (size 1.27 1.27)) (justify right)))
   (property "Value" "LRA_P" (at 130.81 78.74 0) (effects (font (size 1.27 1.27)) (justify right)))
   (property "Footprint" "TestPoint:TestPoint_Pad_D1.0mm" (at 132.08 81.28 0) (effects (font (size 1.27 1.27))) (hide yes))
@@
   (property "Block" "blk.haptics" (at 132.08 81.28 0) (effects (font (size 1.27 1.27))) (hide yes))
   (pin "1")
-  (instances (project "t1-main-board" (path "/7746052e-d7f9-59ad-ba73-bd2b74439529/780edba7-5b74-5864-9ee6-3672d6464c18" (reference "TP6403") (unit 1))))
+  (instances (project "t1-main-board" (path "/7746052e-d7f9-59ad-ba73-bd2b74439529/780edba7-5b74-5864-9ee6-3672d6464c18" (reference "TP6503") (unit 1))))
 )
 (symbol (lib_id "Connector:TestPoint") (at 149.86 81.28 0) (unit 1) (body_style 1) (exclude_from_sim no) (in_bom no) (on_board yes) (dnp no)
-  (property "Reference" "TP6404" (at 148.59 76.2 0) (effects (font (size 1.27 1.27)) (justify right)))
+  (property "Reference" "TP6504" (at 148.59 76.2 0) (effects (font (size 1.27 1.27)) (justify right)))
   (property "Value" "LRA_N" (at 148.59 78.74 0) (effects (font (size 1.27 1.27)) (justify right)))
   (property "Footprint" "TestPoint:TestPoint_Pad_D1.0mm" (at 149.86 81.28 0) (effects (font (size 1.27 1.27))) (hide yes))
@@
   (property "Block" "blk.haptics" (at 149.86 81.28 0) (effects (font (size 1.27 1.27))) (hide yes))
   (pin "1")
-  (instances (project "t1-main-board" (path "/7746052e-d7f9-59ad-ba73-bd2b74439529/780edba7-5b74-5864-9ee6-3672d6464c18" (reference "TP6404") (unit 1))))
+  (instances (project "t1-main-board" (path "/7746052e-d7f9-59ad-ba73-bd2b74439529/780edba7-5b74-5864-9ee6-3672d6464c18" (reference "TP6504") (unit 1))))
 )
 (rectangle (start 120.65 71.12) (end 191.77 92.71) (stroke (width 0) (type dash)) (fill (type none)))

Commit message: Board: capture blk.cover-detect
COVER_DET_N on GPIO0_A6 (AJ38, PMUIO1, wake-capable), recorded in
pinout v1 (closes feature blocks G22): board-edge input and ground pads
for the case's actuator, 100 kΩ to vcc3v3_pmu, TPD1E10B06 at the pad
(BOM v1 line 143, PCB-L-10). The line rides the KEYS bus with the
buttons.

Co-Authored-By: Claude Opus 5.5 <noreply@anthropic.com>
Claude-Session: https://claude.ai/code/session_01Ei262h3TpgY9vyfNLMi5Mn
Parts:
- removed C6501, C6502: 1 µF, Capacitor_SMD:C_0402_1005Metric, symbol Device:C
- removed R6501: 100 mΩ, Resistor_SMD:R_0603_1608Metric, symbol Device:R
- removed TP6501: vcc3v3_sys, TestPoint:TestPoint_Pad_D1.0mm, symbol Connector:TestPoint
- removed TP6502: HAPTIC_VDD, TestPoint:TestPoint_Pad_D1.0mm, symbol Connector:TestPoint
- removed TP6503: LRA_P, TestPoint:TestPoint_Pad_D1.0mm, symbol Connector:TestPoint
- removed TP6504: LRA_N, TestPoint:TestPoint_Pad_D1.0mm, symbol Connector:TestPoint
- removed U6501: DRV2605LDGSR, Texas_Instruments:Texas_DGS0010A_VSSOP-10_3x3mm_P0.5mm, symbol Texas_Instruments:DRV2605LDGSR
- added C6601, C6602: 1 µF, Capacitor_SMD:C_0402_1005Metric, symbol Device:C
- added R6601: 100 mΩ, Resistor_SMD:R_0603_1608Metric, symbol Device:R
- added TP6601: vcc3v3_sys, TestPoint:TestPoint_Pad_D1.0mm, symbol Connector:TestPoint
- added TP6602: HAPTIC_VDD, TestPoint:TestPoint_Pad_D1.0mm, symbol Connector:TestPoint
- added TP6603: LRA_P, TestPoint:TestPoint_Pad_D1.0mm, symbol Connector:TestPoint
- added TP6604: LRA_N, TestPoint:TestPoint_Pad_D1.0mm, symbol Connector:TestPoint
- added U6601: DRV2605LDGSR, Texas_Instruments:Texas_DGS0010A_VSSOP-10_3x3mm_P0.5mm, symbol Texas_Instruments:DRV2605LDGSR
Connections:
- net GND: now also C6601.2, C6602.2, U6601.4 (IN/TRIG), U6601.8 (GND)
- net HAPTIC_EN: now also U6601.5 (EN)
- net HAPTIC_REG: now also C6602.1, U6601.1 (REG)
- net HAPTIC_VDD: now also C6601.1, R6601.2, TP6602.1, U6601.10 (VDD), U6601.6 (VDD/NC)
- net I2C2_SCL: now also U6601.2 (SCL)
- net I2C2_SDA: now also U6601.3 (SDA)
- net LRA_N: now also TP6604.1, U6601.9 (OUT-)
- net LRA_P: now also TP6603.1, U6601.7 (OUT+)
- net vcc3v3_sys: now also R6601.1, TP6601.1
Changed lines of the file:
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@@
 (title_block (title "Haptic driver") (date "2026-10-25") (rev "A") (company "The OpenDAP Project") (comment 1 "blk.haptics") (comment 2 "DRV2605L LRA driver on I2C2 at 0x5A and the actuator contacts"))
 (symbol (lib_id "Texas_Instruments:DRV2605LDGSR") (at 54.61 76.2 0) (unit 1) (body_style 1) (exclude_from_sim no) (in_bom yes) (on_board yes) (dnp no)
-  (property "Reference" "U6501" (at 58.42 54.61 0) (effects (font (size 1.27 1.27)) (justify left)))
+  (property "Reference" "U6601" (at 58.42 54.61 0) (effects (font (size 1.27 1.27)) (justify left)))
   (property "Value" "DRV2605LDGSR" (at 58.42 52.07 0) (effects (font (size 1.27 1.27)) (justify left)))
   (property "Footprint" "Texas_Instruments:Texas_DGS0010A_VSSOP-10_3x3mm_P0.5mm" (at 54.61 76.2 0) (effects (font (size 1.27 1.27))) (hide yes))
@@
   (pin "6")
   (pin "8")
-  (instances (project "t1-main-board" (path "/7746052e-d7f9-59ad-ba73-bd2b74439529/780edba7-5b74-5864-9ee6-3672d6464c18" (reference "U6501") (unit 1))))
+  (instances (project "t1-main-board" (path "/7746052e-d7f9-59ad-ba73-bd2b74439529/780edba7-5b74-5864-9ee6-3672d6464c18" (reference "U6601") (unit 1))))
 )
 (wire (pts (xy 52.07 53.34) (xy 52.07 50.8)) (stroke (width 0) (type default)))
@@
 )
 (symbol (lib_id "Device:C") (at 90.17 57.15 0) (unit 1) (body_style 1) (exclude_from_sim no) (in_bom yes) (on_board yes) (dnp no)
-  (property "Reference" "C6501" (at 92.71 55.88 0) (effects (font (size 1.27 1.27)) (justify left)))
+  (property "Reference" "C6601" (at 92.71 55.88 0) (effects (font (size 1.27 1.27)) (justify left)))
   (property "Value" "1 µF" (at 92.71 58.42 0) (effects (font (size 1.27 1.27)) (justify left)))
   (property "Footprint" "Capacitor_SMD:C_0402_1005Metric" (at 90.17 57.15 0) (effects (font (size 1.27 1.27))) (hide yes))
@@
   (pin "1")
   (pin "2")
-  (instances (project "t1-main-board" (path "/7746052e-d7f9-59ad-ba73-bd2b74439529/780edba7-5b74-5864-9ee6-3672d6464c18" (reference "C6501") (unit 1))))
+  (instances (project "t1-main-board" (path "/7746052e-d7f9-59ad-ba73-bd2b74439529/780edba7-5b74-5864-9ee6-3672d6464c18" (reference "C6601") (unit 1))))
 )
 (wire (pts (xy 90.17 53.34) (xy 90.17 50.8)) (stroke (width 0) (type default)))
@@
 )
 (symbol (lib_id "Device:C") (at 102.87 57.15 0) (unit 1) (body_style 1) (exclude_from_sim no) (in_bom yes) (on_board yes) (dnp no)
-  (property "Reference" "C6502" (at 105.41 55.88 0) (effects (font (size 1.27 1.27)) (justify left)))
+  (property "Reference" "C6602" (at 105.41 55.88 0) (effects (font (size 1.27 1.27)) (justify left)))
   (property "Value" "1 µF" (at 105.41 58.42 0) (effects (font (size 1.27 1.27)) (justify left)))
   (property "Footprint" "Capacitor_SMD:C_0402_1005Metric" (at 102.87 57.15 0) (effects (font (size 1.27 1.27))) (hide yes))
@@
   (pin "1")
   (pin "2")
-  (instances (project "t1-main-board" (path "/7746052e-d7f9-59ad-ba73-bd2b74439529/780edba7-5b74-5864-9ee6-3672d6464c18" (reference "C6502") (unit 1))))
+  (instances (project "t1-main-board" (path "/7746052e-d7f9-59ad-ba73-bd2b74439529/780edba7-5b74-5864-9ee6-3672d6464c18" (reference "C6602") (unit 1))))
 )
 (wire (pts (xy 102.87 53.34) (xy 102.87 50.8)) (stroke (width 0) (type default)))
@@
 (text "DRV2605L at I2C2 0x5A (BOM v1 line 123)" (exclude_from_sim no) (at 24.13 34.29 0) (effects (font (size 2.54 2.54)) (justify left bottom)))
 (symbol (lib_id "Device:R") (at 157.48 50.8 90) (unit 1) (body_style 1) (exclude_from_sim no) (in_bom yes) (on_board yes) (dnp no)
-  (property "Reference" "R6501" (at 154.94 46.99 90) (effects (font (size 1.27 1.27))))
+  (property "Reference" "R6601" (at 154.94 46.99 90) (effects (font (size 1.27 1.27))))
   (property "Value" "100 mΩ" (at 154.94 53.34 90) (effects (font (size 1.27 1.27))))
   (property "Spec" "0603" (at 154.94 55.88 90) (effects (font (size 1.27 1.27))))
@@
   (pin "1")
   (pin "2")
-  (instances (project "t1-main-board" (path "/7746052e-d7f9-59ad-ba73-bd2b74439529/780edba7-5b74-5864-9ee6-3672d6464c18" (reference "R6501") (unit 1) (variant (name "production") (field (name "Value") (value "0 Ω")) (field (name "MPN") (value "RC0603JR-070RL")) (field (name "Manufacturer") (value "YAGEO"))))))
+  (instances (project "t1-main-board" (path "/7746052e-d7f9-59ad-ba73-bd2b74439529/780edba7-5b74-5864-9ee6-3672d6464c18" (reference "R6601") (unit 1) (variant (name "production") (field (name "Value") (value "0 Ω")) (field (name "MPN") (value "RC0603JR-070RL")) (field (name "Manufacturer") (value "YAGEO"))))))
 )
 (rectangle (start 135.89 38.1) (end 179.07 58.42) (stroke (width 0) (type dash)) (fill (type none)))
@@
 (wire (pts (xy 151.13 50.8) (xy 151.13 48.26)) (stroke (width 0) (type default)))
 (symbol (lib_id "Connector:TestPoint") (at 151.13 48.26 0) (unit 1) (body_style 1) (exclude_from_sim no) (in_bom no) (on_board yes) (dnp no)
-  (property "Reference" "TP6501" (at 149.86 43.18 0) (effects (font (size 1.27 1.27)) (justify right)))
+  (property "Reference" "TP6601" (at 149.86 43.18 0) (effects (font (size 1.27 1.27)) (justify right)))
   (property "Value" "vcc3v3_sys" (at 149.86 45.72 0) (effects (font (size 1.27 1.27)) (justify right)))
   (property "Footprint" "TestPoint:TestPoint_Pad_D1.0mm" (at 151.13 48.26 0) (effects (font (size 1.27 1.27))) (hide yes))
@@
   (property "Block" "blk.haptics" (at 151.13 48.26 0) (effects (font (size 1.27 1.27))) (hide yes))
   (pin "1")
-  (instances (project "t1-main-board" (path "/7746052e-d7f9-59ad-ba73-bd2b74439529/780edba7-5b74-5864-9ee6-3672d6464c18" (reference "TP6501") (unit 1))))
+  (instances (project "t1-main-board" (path "/7746052e-d7f9-59ad-ba73-bd2b74439529/780edba7-5b74-5864-9ee6-3672d6464c18" (reference "TP6601") (unit 1))))
 )
 (symbol (lib_id "power:VCC") (at 133.35 50.8 90) (unit 1) (body_style 1) (exclude_from_sim no) (in_bom yes) (on_board yes) (dnp no)
@@
 (wire (pts (xy 163.83 50.8) (xy 163.83 48.26)) (stroke (width 0) (type default)))
 (symbol (lib_id "Connector:TestPoint") (at 163.83 48.26 0) (unit 1) (body_style 1) (exclude_from_sim no) (in_bom no) (on_board yes) (dnp no)
-  (property "Reference" "TP6502" (at 165.1 43.18 0) (effects (font (size 1.27 1.27)) (justify left)))
+  (property "Reference" "TP6602" (at 165.1 43.18 0) (effects (font (size 1.27 1.27)) (justify left)))
   (property "Value" "HAPTIC_VDD" (at 165.1 45.72 0) (effects (font (size 1.27 1.27)) (justify left)))
   (property "Footprint" "TestPoint:TestPoint_Pad_D1.0mm" (at 163.83 48.26 0) (effects (font (size 1.27 1.27))) (hide yes))
@@
   (property "Block" "blk.haptics" (at 163.83 48.26 0) (effects (font (size 1.27 1.27))) (hide yes))
   (pin "1")
-  (instances (project "t1-main-board" (path "/7746052e-d7f9-59ad-ba73-bd2b74439529/780edba7-5b74-5864-9ee6-3672d6464c18" (reference "TP6502") (unit 1))))
+  (instances (project "t1-main-board" (path "/7746052e-d7f9-59ad-ba73-bd2b74439529/780edba7-5b74-5864-9ee6-3672d6464c18" (reference "TP6602") (unit 1))))
 )
 (junction (at 186.69 50.8) (diameter 0) (color 0 0 0 0))
@@
 )
 (symbol (lib_id "Connector:TestPoint") (at 132.08 81.28 0) (unit 1) (body_style 1) (exclude_from_sim no) (in_bom no) (on_board yes) (dnp no)
-  (property "Reference" "TP6503" (at 130.81 76.2 0) (effects (font (size 1.27 1.27)) (justify right)))
+  (property "Reference" "TP6603" (at 130.81 76.2 0) (effects (font (size 1.27 1.27)) (justify right)))
   (property "Value" "LRA_P" (at 130.81 78.74 0) (effects (font (size 1.27 1.27)) (justify right)))
   (property "Footprint" "TestPoint:TestPoint_Pad_D1.0mm" (at 132.08 81.28 0) (effects (font (size 1.27 1.27))) (hide yes))
@@
   (property "Block" "blk.haptics" (at 132.08 81.28 0) (effects (font (size 1.27 1.27))) (hide yes))
   (pin "1")
-  (instances (project "t1-main-board" (path "/7746052e-d7f9-59ad-ba73-bd2b74439529/780edba7-5b74-5864-9ee6-3672d6464c18" (reference "TP6503") (unit 1))))
+  (instances (project "t1-main-board" (path "/7746052e-d7f9-59ad-ba73-bd2b74439529/780edba7-5b74-5864-9ee6-3672d6464c18" (reference "TP6603") (unit 1))))
 )
 (symbol (lib_id "Connector:TestPoint") (at 149.86 81.28 0) (unit 1) (body_style 1) (exclude_from_sim no) (in_bom no) (on_board yes) (dnp no)
-  (property "Reference" "TP6504" (at 148.59 76.2 0) (effects (font (size 1.27 1.27)) (justify right)))
+  (property "Reference" "TP6604" (at 148.59 76.2 0) (effects (font (size 1.27 1.27)) (justify right)))
   (property "Value" "LRA_N" (at 148.59 78.74 0) (effects (font (size 1.27 1.27)) (justify right)))
   (property "Footprint" "TestPoint:TestPoint_Pad_D1.0mm" (at 149.86 81.28 0) (effects (font (size 1.27 1.27))) (hide yes))
@@
   (property "Block" "blk.haptics" (at 149.86 81.28 0) (effects (font (size 1.27 1.27))) (hide yes))
   (pin "1")
-  (instances (project "t1-main-board" (path "/7746052e-d7f9-59ad-ba73-bd2b74439529/780edba7-5b74-5864-9ee6-3672d6464c18" (reference "TP6504") (unit 1))))
+  (instances (project "t1-main-board" (path "/7746052e-d7f9-59ad-ba73-bd2b74439529/780edba7-5b74-5864-9ee6-3672d6464c18" (reference "TP6604") (unit 1))))
 )
 (rectangle (start 120.65 71.12) (end 191.77 92.71) (stroke (width 0) (type dash)) (fill (type none)))
