File: board/hardware/t1-main-board/haptics.kicad_sch (KiCad schematic)
At the start: 8 parts, among them U6601 DRV2605LDGSR

Commit message: Board: capture blk.mic-ambient and links #34, #35
IM73D122 on PDM CLK1 and SDI1 (BOM v1 line 34, pinout v1 AK2 and 1P2),
LR to ground, 22 Ω clock series, VDD from MIC_1V8 through link #35.
Link #34 on blk.mic-main makes the faceplate branch the rail MIC_1V8_FP
for contact 40 (power tree §4.12, G10). kicad-lib moves to e46bda4 for
the IM73D122, TPS3808G01, SN74LVC1G58 and BAT54 parts.

Co-Authored-By: Claude Opus 5.5 <noreply@anthropic.com>
Claude-Session: https://claude.ai/code/session_01Ei262h3TpgY9vyfNLMi5Mn
Parts:
- removed C6601, C6602: 1 µF, Capacitor_SMD:C_0402_1005Metric, symbol Device:C
- removed R6601: 100 mΩ, Resistor_SMD:R_0603_1608Metric, symbol Device:R
- removed TP6601: vcc3v3_sys, TestPoint:TestPoint_Pad_D1.0mm, symbol Connector:TestPoint
- removed TP6602: HAPTIC_VDD, TestPoint:TestPoint_Pad_D1.0mm, symbol Connector:TestPoint
- removed TP6603: LRA_P, TestPoint:TestPoint_Pad_D1.0mm, symbol Connector:TestPoint
- removed TP6604: LRA_N, TestPoint:TestPoint_Pad_D1.0mm, symbol Connector:TestPoint
- removed U6601: DRV2605LDGSR, Texas_Instruments:Texas_DGS0010A_VSSOP-10_3x3mm_P0.5mm, symbol Texas_Instruments:DRV2605LDGSR
- added C6701, C6702: 1 µF, Capacitor_SMD:C_0402_1005Metric, symbol Device:C
- added R6701: 100 mΩ, Resistor_SMD:R_0603_1608Metric, symbol Device:R
- added TP6701: vcc3v3_sys, TestPoint:TestPoint_Pad_D1.0mm, symbol Connector:TestPoint
- added TP6702: HAPTIC_VDD, TestPoint:TestPoint_Pad_D1.0mm, symbol Connector:TestPoint
- added TP6703: LRA_P, TestPoint:TestPoint_Pad_D1.0mm, symbol Connector:TestPoint
- added TP6704: LRA_N, TestPoint:TestPoint_Pad_D1.0mm, symbol Connector:TestPoint
- added U6701: DRV2605LDGSR, Texas_Instruments:Texas_DGS0010A_VSSOP-10_3x3mm_P0.5mm, symbol Texas_Instruments:DRV2605LDGSR
Connections:
- net GND: now also C6701.2, C6702.2, U6701.4 (IN/TRIG), U6701.8 (GND)
- net HAPTIC_EN: now also U6701.5 (EN)
- net HAPTIC_REG: now also C6702.1, U6701.1 (REG)
- net HAPTIC_VDD: now also C6701.1, R6701.2, TP6702.1, U6701.10 (VDD), U6701.6 (VDD/NC)
- net I2C2_SCL: now also U6701.2 (SCL)
- net I2C2_SDA: now also U6701.3 (SDA)
- net LRA_N: now also TP6704.1, U6701.9 (OUT-)
- net LRA_P: now also TP6703.1, U6701.7 (OUT+)
- net vcc3v3_sys: now also R6701.1, TP6701.1

Commit message: Board: capture blk.maskrom
Power + Vol- at a cold power-on pull eMMC D0 low inside the TPS3808G01
boot window (BOM v1 lines 35, 78, 97, 98; sim/maskrom): SENSE 280k/100k,
CT 390 nF, WINDOW_N with its pad, SN74LVC1G57 and SN74LVC1G58 on
vcca1v8_pmu, BAT54 from PWRON_N, DMG1012T through 1 kΩ to EMMC_D0.
Every block in use now has its sheet; the README states the remaining
single-pin nets.

Co-Authored-By: Claude Opus 5.5 <noreply@anthropic.com>
Claude-Session: https://claude.ai/code/session_01Ei262h3TpgY9vyfNLMi5Mn
Parts:
- removed C6701, C6702: 1 µF, Capacitor_SMD:C_0402_1005Metric, symbol Device:C
- removed R6701: 100 mΩ, Resistor_SMD:R_0603_1608Metric, symbol Device:R
- removed TP6701: vcc3v3_sys, TestPoint:TestPoint_Pad_D1.0mm, symbol Connector:TestPoint
- removed TP6702: HAPTIC_VDD, TestPoint:TestPoint_Pad_D1.0mm, symbol Connector:TestPoint
- removed TP6703: LRA_P, TestPoint:TestPoint_Pad_D1.0mm, symbol Connector:TestPoint
- removed TP6704: LRA_N, TestPoint:TestPoint_Pad_D1.0mm, symbol Connector:TestPoint
- removed U6701: DRV2605LDGSR, Texas_Instruments:Texas_DGS0010A_VSSOP-10_3x3mm_P0.5mm, symbol Texas_Instruments:DRV2605LDGSR
- added C6801, C6802: 1 µF, Capacitor_SMD:C_0402_1005Metric, symbol Device:C
- added R6801: 100 mΩ, Resistor_SMD:R_0603_1608Metric, symbol Device:R
- added TP6801: vcc3v3_sys, TestPoint:TestPoint_Pad_D1.0mm, symbol Connector:TestPoint
- added TP6802: HAPTIC_VDD, TestPoint:TestPoint_Pad_D1.0mm, symbol Connector:TestPoint
- added TP6803: LRA_P, TestPoint:TestPoint_Pad_D1.0mm, symbol Connector:TestPoint
- added TP6804: LRA_N, TestPoint:TestPoint_Pad_D1.0mm, symbol Connector:TestPoint
- added U6801: DRV2605LDGSR, Texas_Instruments:Texas_DGS0010A_VSSOP-10_3x3mm_P0.5mm, symbol Texas_Instruments:DRV2605LDGSR
Connections:
- net GND: now also C6801.2, C6802.2, U6801.4 (IN/TRIG), U6801.8 (GND)
- net HAPTIC_EN: now also U6801.5 (EN)
- net HAPTIC_REG: now also C6802.1, U6801.1 (REG)
- net HAPTIC_VDD: now also C6801.1, R6801.2, TP6802.1, U6801.10 (VDD), U6801.6 (VDD/NC)
- net I2C2_SCL: now also U6801.2 (SCL)
- net I2C2_SDA: now also U6801.3 (SDA)
- net LRA_N: now also TP6804.1, U6801.9 (OUT-)
- net LRA_P: now also TP6803.1, U6801.7 (OUT+)
- net vcc3v3_sys: now also R6801.1, TP6801.1
Changed lines of the file:
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@@
 (title_block (title "Haptic driver") (date "2026-10-25") (rev "A") (company "The OpenDAP Project") (comment 1 "blk.haptics") (comment 2 "DRV2605L LRA driver on I2C2 at 0x5A and the actuator contacts"))
 (symbol (lib_id "Texas_Instruments:DRV2605LDGSR") (at 54.61 76.2 0) (unit 1) (body_style 1) (exclude_from_sim no) (in_bom yes) (on_board yes) (dnp no)
-  (property "Reference" "U6701" (at 58.42 54.61 0) (effects (font (size 1.27 1.27)) (justify left)))
+  (property "Reference" "U6801" (at 58.42 54.61 0) (effects (font (size 1.27 1.27)) (justify left)))
   (property "Value" "DRV2605LDGSR" (at 58.42 52.07 0) (effects (font (size 1.27 1.27)) (justify left)))
   (property "Footprint" "Texas_Instruments:Texas_DGS0010A_VSSOP-10_3x3mm_P0.5mm" (at 54.61 76.2 0) (effects (font (size 1.27 1.27))) (hide yes))
@@
   (pin "6")
   (pin "8")
-  (instances (project "t1-main-board" (path "/7746052e-d7f9-59ad-ba73-bd2b74439529/780edba7-5b74-5864-9ee6-3672d6464c18" (reference "U6701") (unit 1))))
+  (instances (project "t1-main-board" (path "/7746052e-d7f9-59ad-ba73-bd2b74439529/780edba7-5b74-5864-9ee6-3672d6464c18" (reference "U6801") (unit 1))))
 )
 (wire (pts (xy 52.07 53.34) (xy 52.07 50.8)) (stroke (width 0) (type default)))
@@
 )
 (symbol (lib_id "Device:C") (at 90.17 57.15 0) (unit 1) (body_style 1) (exclude_from_sim no) (in_bom yes) (on_board yes) (dnp no)
-  (property "Reference" "C6701" (at 92.71 55.88 0) (effects (font (size 1.27 1.27)) (justify left)))
+  (property "Reference" "C6801" (at 92.71 55.88 0) (effects (font (size 1.27 1.27)) (justify left)))
   (property "Value" "1 µF" (at 92.71 58.42 0) (effects (font (size 1.27 1.27)) (justify left)))
   (property "Footprint" "Capacitor_SMD:C_0402_1005Metric" (at 90.17 57.15 0) (effects (font (size 1.27 1.27))) (hide yes))
@@
   (pin "1")
   (pin "2")
-  (instances (project "t1-main-board" (path "/7746052e-d7f9-59ad-ba73-bd2b74439529/780edba7-5b74-5864-9ee6-3672d6464c18" (reference "C6701") (unit 1))))
+  (instances (project "t1-main-board" (path "/7746052e-d7f9-59ad-ba73-bd2b74439529/780edba7-5b74-5864-9ee6-3672d6464c18" (reference "C6801") (unit 1))))
 )
 (wire (pts (xy 90.17 53.34) (xy 90.17 50.8)) (stroke (width 0) (type default)))
@@
 )
 (symbol (lib_id "Device:C") (at 102.87 57.15 0) (unit 1) (body_style 1) (exclude_from_sim no) (in_bom yes) (on_board yes) (dnp no)
-  (property "Reference" "C6702" (at 105.41 55.88 0) (effects (font (size 1.27 1.27)) (justify left)))
+  (property "Reference" "C6802" (at 105.41 55.88 0) (effects (font (size 1.27 1.27)) (justify left)))
   (property "Value" "1 µF" (at 105.41 58.42 0) (effects (font (size 1.27 1.27)) (justify left)))
   (property "Footprint" "Capacitor_SMD:C_0402_1005Metric" (at 102.87 57.15 0) (effects (font (size 1.27 1.27))) (hide yes))
@@
   (pin "1")
   (pin "2")
-  (instances (project "t1-main-board" (path "/7746052e-d7f9-59ad-ba73-bd2b74439529/780edba7-5b74-5864-9ee6-3672d6464c18" (reference "C6702") (unit 1))))
+  (instances (project "t1-main-board" (path "/7746052e-d7f9-59ad-ba73-bd2b74439529/780edba7-5b74-5864-9ee6-3672d6464c18" (reference "C6802") (unit 1))))
 )
 (wire (pts (xy 102.87 53.34) (xy 102.87 50.8)) (stroke (width 0) (type default)))
@@
 (text "DRV2605L at I2C2 0x5A (BOM v1 line 123)" (exclude_from_sim no) (at 24.13 34.29 0) (effects (font (size 2.54 2.54)) (justify left bottom)))
 (symbol (lib_id "Device:R") (at 157.48 50.8 90) (unit 1) (body_style 1) (exclude_from_sim no) (in_bom yes) (on_board yes) (dnp no)
-  (property "Reference" "R6701" (at 154.94 46.99 90) (effects (font (size 1.27 1.27))))
+  (property "Reference" "R6801" (at 154.94 46.99 90) (effects (font (size 1.27 1.27))))
   (property "Value" "100 mΩ" (at 154.94 53.34 90) (effects (font (size 1.27 1.27))))
   (property "Spec" "0603" (at 154.94 55.88 90) (effects (font (size 1.27 1.27))))
@@
   (pin "1")
   (pin "2")
-  (instances (project "t1-main-board" (path "/7746052e-d7f9-59ad-ba73-bd2b74439529/780edba7-5b74-5864-9ee6-3672d6464c18" (reference "R6701") (unit 1) (variant (name "production") (field (name "Value") (value "0 Ω")) (field (name "MPN") (value "RC0603JR-070RL")) (field (name "Manufacturer") (value "YAGEO"))))))
+  (instances (project "t1-main-board" (path "/7746052e-d7f9-59ad-ba73-bd2b74439529/780edba7-5b74-5864-9ee6-3672d6464c18" (reference "R6801") (unit 1) (variant (name "production") (field (name "Value") (value "0 Ω")) (field (name "MPN") (value "RC0603JR-070RL")) (field (name "Manufacturer") (value "YAGEO"))))))
 )
 (rectangle (start 135.89 38.1) (end 179.07 58.42) (stroke (width 0) (type dash)) (fill (type none)))
@@
 (wire (pts (xy 151.13 50.8) (xy 151.13 48.26)) (stroke (width 0) (type default)))
 (symbol (lib_id "Connector:TestPoint") (at 151.13 48.26 0) (unit 1) (body_style 1) (exclude_from_sim no) (in_bom no) (on_board yes) (dnp no)
-  (property "Reference" "TP6701" (at 149.86 43.18 0) (effects (font (size 1.27 1.27)) (justify right)))
+  (property "Reference" "TP6801" (at 149.86 43.18 0) (effects (font (size 1.27 1.27)) (justify right)))
   (property "Value" "vcc3v3_sys" (at 149.86 45.72 0) (effects (font (size 1.27 1.27)) (justify right)))
   (property "Footprint" "TestPoint:TestPoint_Pad_D1.0mm" (at 151.13 48.26 0) (effects (font (size 1.27 1.27))) (hide yes))
@@
   (property "Block" "blk.haptics" (at 151.13 48.26 0) (effects (font (size 1.27 1.27))) (hide yes))
   (pin "1")
-  (instances (project "t1-main-board" (path "/7746052e-d7f9-59ad-ba73-bd2b74439529/780edba7-5b74-5864-9ee6-3672d6464c18" (reference "TP6701") (unit 1))))
+  (instances (project "t1-main-board" (path "/7746052e-d7f9-59ad-ba73-bd2b74439529/780edba7-5b74-5864-9ee6-3672d6464c18" (reference "TP6801") (unit 1))))
 )
 (symbol (lib_id "power:VCC") (at 133.35 50.8 90) (unit 1) (body_style 1) (exclude_from_sim no) (in_bom yes) (on_board yes) (dnp no)
@@
 (wire (pts (xy 163.83 50.8) (xy 163.83 48.26)) (stroke (width 0) (type default)))
 (symbol (lib_id "Connector:TestPoint") (at 163.83 48.26 0) (unit 1) (body_style 1) (exclude_from_sim no) (in_bom no) (on_board yes) (dnp no)
-  (property "Reference" "TP6702" (at 165.1 43.18 0) (effects (font (size 1.27 1.27)) (justify left)))
+  (property "Reference" "TP6802" (at 165.1 43.18 0) (effects (font (size 1.27 1.27)) (justify left)))
   (property "Value" "HAPTIC_VDD" (at 165.1 45.72 0) (effects (font (size 1.27 1.27)) (justify left)))
   (property "Footprint" "TestPoint:TestPoint_Pad_D1.0mm" (at 163.83 48.26 0) (effects (font (size 1.27 1.27))) (hide yes))
@@
   (property "Block" "blk.haptics" (at 163.83 48.26 0) (effects (font (size 1.27 1.27))) (hide yes))
   (pin "1")
-  (instances (project "t1-main-board" (path "/7746052e-d7f9-59ad-ba73-bd2b74439529/780edba7-5b74-5864-9ee6-3672d6464c18" (reference "TP6702") (unit 1))))
+  (instances (project "t1-main-board" (path "/7746052e-d7f9-59ad-ba73-bd2b74439529/780edba7-5b74-5864-9ee6-3672d6464c18" (reference "TP6802") (unit 1))))
 )
 (junction (at 186.69 50.8) (diameter 0) (color 0 0 0 0))
@@
 )
 (symbol (lib_id "Connector:TestPoint") (at 132.08 81.28 0) (unit 1) (body_style 1) (exclude_from_sim no) (in_bom no) (on_board yes) (dnp no)
-  (property "Reference" "TP6703" (at 130.81 76.2 0) (effects (font (size 1.27 1.27)) (justify right)))
+  (property "Reference" "TP6803" (at 130.81 76.2 0) (effects (font (size 1.27 1.27)) (justify right)))
   (property "Value" "LRA_P" (at 130.81 78.74 0) (effects (font (size 1.27 1.27)) (justify right)))
   (property "Footprint" "TestPoint:TestPoint_Pad_D1.0mm" (at 132.08 81.28 0) (effects (font (size 1.27 1.27))) (hide yes))
@@
   (property "Block" "blk.haptics" (at 132.08 81.28 0) (effects (font (size 1.27 1.27))) (hide yes))
   (pin "1")
-  (instances (project "t1-main-board" (path "/7746052e-d7f9-59ad-ba73-bd2b74439529/780edba7-5b74-5864-9ee6-3672d6464c18" (reference "TP6703") (unit 1))))
+  (instances (project "t1-main-board" (path "/7746052e-d7f9-59ad-ba73-bd2b74439529/780edba7-5b74-5864-9ee6-3672d6464c18" (reference "TP6803") (unit 1))))
 )
 (symbol (lib_id "Connector:TestPoint") (at 149.86 81.28 0) (unit 1) (body_style 1) (exclude_from_sim no) (in_bom no) (on_board yes) (dnp no)
-  (property "Reference" "TP6704" (at 148.59 76.2 0) (effects (font (size 1.27 1.27)) (justify right)))
+  (property "Reference" "TP6804" (at 148.59 76.2 0) (effects (font (size 1.27 1.27)) (justify right)))
   (property "Value" "LRA_N" (at 148.59 78.74 0) (effects (font (size 1.27 1.27)) (justify right)))
   (property "Footprint" "TestPoint:TestPoint_Pad_D1.0mm" (at 149.86 81.28 0) (effects (font (size 1.27 1.27))) (hide yes))
@@
   (property "Block" "blk.haptics" (at 149.86 81.28 0) (effects (font (size 1.27 1.27))) (hide yes))
   (pin "1")
-  (instances (project "t1-main-board" (path "/7746052e-d7f9-59ad-ba73-bd2b74439529/780edba7-5b74-5864-9ee6-3672d6464c18" (reference "TP6704") (unit 1))))
+  (instances (project "t1-main-board" (path "/7746052e-d7f9-59ad-ba73-bd2b74439529/780edba7-5b74-5864-9ee6-3672d6464c18" (reference "TP6804") (unit 1))))
 )
 (rectangle (start 120.65 71.12) (end 191.77 92.71) (stroke (width 0) (type dash)) (fill (type none)))

Commit message: Board on libs v0.2.0: lower-case kebab vendor keys (HL-13)
The libs submodule moves to v0.2.0 (5f24483). Every library nickname in
the generator, the placement tool and the floorplan study follows the
key table (Texas_Instruments -> texas-instruments, OpenDAP_Device ->
opendap-generic, Rockchip and Rockchip_PMIC -> rockchip, ...); the
library tables are written from the files. Schematic and board
regenerated.

Checks: ERC 0 errors (warnings unchanged); DRC 0 errors, 605 warnings,
the same counts by type, schematic parity 0; every placement identical;
craft Q1 met; pcb tests pass; STEP export resolves every libs 3D model
(the 27 parts without a model are KiCad stock lands that have none).

Co-Authored-By: Claude Opus 5.5 <noreply@anthropic.com>
Claude-Session: https://claude.ai/code/session_01Ei262h3TpgY9vyfNLMi5Mn
Parts:
- U6801: footprint Texas_Instruments:Texas_DGS0010A_VSSOP-10_3x3mm_P0.5mm -> texas-instruments:Texas_DGS0010A_VSSOP-10_3x3mm_P0.5mm; symbol Texas_Instruments:DRV2605LDGSR -> texas-instruments:DRV2605LDGSR
Changed lines of the file:
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@@
 (paper "A4")
 (title_block (title "Haptic driver") (date "2026-10-25") (rev "A") (company "The OpenDAP Project") (comment 1 "blk.haptics") (comment 2 "DRV2605L LRA driver on I2C2 at 0x5A and the actuator contacts"))
-(symbol (lib_id "Texas_Instruments:DRV2605LDGSR") (at 54.61 76.2 0) (unit 1) (body_style 1) (exclude_from_sim no) (in_bom yes) (on_board yes) (dnp no)
+(symbol (lib_id "texas-instruments:DRV2605LDGSR") (at 54.61 76.2 0) (unit 1) (body_style 1) (exclude_from_sim no) (in_bom yes) (on_board yes) (dnp no)
   (property "Reference" "U6801" (at 58.42 54.61 0) (effects (font (size 1.27 1.27)) (justify left)))
   (property "Value" "DRV2605LDGSR" (at 58.42 52.07 0) (effects (font (size 1.27 1.27)) (justify left)))
-  (property "Footprint" "Texas_Instruments:Texas_DGS0010A_VSSOP-10_3x3mm_P0.5mm" (at 54.61 76.2 0) (effects (font (size 1.27 1.27))) (hide yes))
+  (property "Footprint" "texas-instruments:Texas_DGS0010A_VSSOP-10_3x3mm_P0.5mm" (at 54.61 76.2 0) (effects (font (size 1.27 1.27))) (hide yes))
   (property "Datasheet" "https://www.ti.com/lit/ds/symlink/drv2605l.pdf" (at 54.61 76.2 0) (effects (font (size 1.27 1.27))) (hide yes))
   (property "Description" "Haptic driver for LRA and ERM actuators, closed-loop auto-resonance, licensed effect library, I2C, 2-5.2 V, VSSOP-10 (DGS0010A)" (at 54.61 76.2 0) (effects (font (size 1.27 1.27))) (hide yes))

Commit message: BOM v1.18 item 2: successors of the discontinued 1 uF 0402
GRM155R61A105KE15D is to be discontinued. 44 positions take
GRM155C71A105KE11D (1 uF 10 V X7S); the eight TPS7A20 positions take
GRM155R61C225KE11D (2.2 uF 16 V X5R) to keep the 0.47 uF effective
minimum with 10 % to spare at up to 3.8 V. Same land; sourcing pass.
Closes BOM §7 item 52; new item 55 lists the other capture parts outside
Murata's product data or near end of life.

Co-Authored-By: Claude Opus 5.5 <noreply@anthropic.com>
Claude-Session: https://claude.ai/code/session_01Ei262h3TpgY9vyfNLMi5Mn
Parts:
- C6801, C6802: MPN GRM155R61A105KE15D -> GRM155C71A105KE11D
Changed lines of the file:
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@@
   (property "Value" "1 µF" (at 92.71 58.42 0) (effects (font (size 1.27 1.27)) (justify left)))
   (property "Footprint" "Capacitor_SMD:C_0402_1005Metric" (at 90.17 57.15 0) (effects (font (size 1.27 1.27))) (hide yes))
-  (property "Datasheet" "https://www.murata.com/en-us/products/productdetail?partno=GRM155R61A105KE15D" (at 90.17 57.15 0) (effects (font (size 1.27 1.27))) (hide yes))
-  (property "Description" "Capacitor, 1 µF, 10 V, X5R, 0402" (at 90.17 57.15 0) (effects (font (size 1.27 1.27))) (hide yes))
+  (property "Datasheet" "https://www.murata.com/en-us/products/productdetail?partno=GRM155C71A105KE11D" (at 90.17 57.15 0) (effects (font (size 1.27 1.27))) (hide yes))
+  (property "Description" "Capacitor, 1 µF, 10 V, X7S, 0402" (at 90.17 57.15 0) (effects (font (size 1.27 1.27))) (hide yes))
   (property "Manufacturer" "Murata" (at 90.17 57.15 0) (effects (font (size 1.27 1.27))) (hide yes))
-  (property "MPN" "GRM155R61A105KE15D" (at 90.17 57.15 0) (effects (font (size 1.27 1.27))) (hide yes))
+  (property "MPN" "GRM155C71A105KE11D" (at 90.17 57.15 0) (effects (font (size 1.27 1.27))) (hide yes))
   (property "Block" "blk.haptics" (at 90.17 57.15 0) (effects (font (size 1.27 1.27))) (hide yes))
   (pin "1")
@@
   (property "Value" "1 µF" (at 105.41 58.42 0) (effects (font (size 1.27 1.27)) (justify left)))
   (property "Footprint" "Capacitor_SMD:C_0402_1005Metric" (at 102.87 57.15 0) (effects (font (size 1.27 1.27))) (hide yes))
-  (property "Datasheet" "https://www.murata.com/en-us/products/productdetail?partno=GRM155R61A105KE15D" (at 102.87 57.15 0) (effects (font (size 1.27 1.27))) (hide yes))
-  (property "Description" "Capacitor, 1 µF, 10 V, X5R, 0402" (at 102.87 57.15 0) (effects (font (size 1.27 1.27))) (hide yes))
+  (property "Datasheet" "https://www.murata.com/en-us/products/productdetail?partno=GRM155C71A105KE11D" (at 102.87 57.15 0) (effects (font (size 1.27 1.27))) (hide yes))
+  (property "Description" "Capacitor, 1 µF, 10 V, X7S, 0402" (at 102.87 57.15 0) (effects (font (size 1.27 1.27))) (hide yes))
   (property "Manufacturer" "Murata" (at 102.87 57.15 0) (effects (font (size 1.27 1.27))) (hide yes))
-  (property "MPN" "GRM155R61A105KE15D" (at 102.87 57.15 0) (effects (font (size 1.27 1.27))) (hide yes))
+  (property "MPN" "GRM155C71A105KE11D" (at 102.87 57.15 0) (effects (font (size 1.27 1.27))) (hide yes))
   (property "Block" "blk.haptics" (at 102.87 57.15 0) (effects (font (size 1.27 1.27))) (hide yes))
   (pin "1")
