File: board/hardware/t1-main-board/nfc-reader.kicad_sch (KiCad schematic)
At the start: 34 parts, among them U5401 PN7160A1HN-C100E, U5402 TPS22919DCKR, Y5401 27.12 MHz

Commit message: Board: capture blk.current-monitors
Five INA236 on I2C1 (0x40-0x43, 0x48) with their shunts, per power tree
§4.12 and BOM v1 lines 54 and 136. The measured branches are rails of
their own (VSYS_SRC, VSYS_LV_AUDIO, VSYS_AUDIO, VSYS_LV_BL, VSYS_P5V1),
fed through the shunts on this sheet; the charger, audio, backlight and
5.1 V sheets take them. The root's layout may leave a stack level empty,
so the block sits under the notes; IC bboxes hold turned rail values;
passive rows hold a bottom rail's text.

Co-Authored-By: Claude Opus 5.5 <noreply@anthropic.com>
Claude-Session: https://claude.ai/code/session_01Ei262h3TpgY9vyfNLMi5Mn
Parts:
- removed C5401, C5403: 4.7 µF, Capacitor_SMD:C_0402_1005Metric, symbol Device:C
- removed C5402, C5409: 100 nF, Capacitor_SMD:C_0402_1005Metric, symbol Device:C
- removed C5404, C5405, C5406, C5407: 2.2 µF, Capacitor_SMD:C_0402_1005Metric, symbol Device:C
- removed C5408, C5412: 1 µF, Capacitor_SMD:C_0402_1005Metric, symbol Device:C
- removed C5410, C5411: 15 pF, Capacitor_SMD:C_0402_1005Metric, symbol Device:C
- removed C5413, C5416: 330 pF, Capacitor_SMD:C_0402_1005Metric, symbol Device:C
- removed C5414, C5417: 68 pF, Capacitor_SMD:C_0402_1005Metric, symbol Device:C
- removed C5415, C5418: 100 pF, Capacitor_SMD:C_0402_1005Metric, symbol Device:C
- removed C5419, C5420: 1 nF, Capacitor_SMD:C_0402_1005Metric, symbol Device:C
- removed L5401, L5402: 160 nH, Inductor_SMD:L_0603_1608Metric, symbol Device:L
- removed R5401: 100 mΩ, Resistor_SMD:R_0603_1608Metric, symbol Device:R
- removed R5402, R5403: 2.7 Ω, Resistor_SMD:R_0402_1005Metric, symbol Device:R
- removed R5404, R5405: 2.2 kΩ, Resistor_SMD:R_0402_1005Metric, symbol Device:R
- removed TP5401: NFC_VBAT_SRC, TestPoint:TestPoint_Pad_D1.0mm, symbol Connector:TestPoint
- removed TP5402: NFC_VBAT, TestPoint:TestPoint_Pad_D1.0mm, symbol Connector:TestPoint
- removed TP5403: NFC_ANT_P, TestPoint:TestPoint_Pad_D1.0mm, symbol Connector:TestPoint
- removed TP5404: NFC_ANT_N, TestPoint:TestPoint_Pad_D1.0mm, symbol Connector:TestPoint
- removed U5401: PN7160A1HN-C100E, NXP:NXP_SOT618-1_HVQFN-40-1EP_6x6mm_P0.5mm_EP4.1x4.1mm, symbol NXP:PN7160A1HN-C100E
- removed U5402: TPS22919DCKR, Texas_Instruments:Texas_DCK0006A_SC-70-6_1.25x2mm_P0.65mm, symbol Texas_Instruments:TPS22919DCKR
- removed Y5401: 27.12 MHz, Crystal:Crystal_SMD_2016-4Pin_2.0x1.6mm, symbol OpenDAP_Device:Crystal_GND24
- added C5501, C5503: 4.7 µF, Capacitor_SMD:C_0402_1005Metric, symbol Device:C
- added C5502, C5509: 100 nF, Capacitor_SMD:C_0402_1005Metric, symbol Device:C
- added C5504, C5505, C5506, C5507: 2.2 µF, Capacitor_SMD:C_0402_1005Metric, symbol Device:C
- added C5508, C5512: 1 µF, Capacitor_SMD:C_0402_1005Metric, symbol Device:C
- added C5510, C5511: 15 pF, Capacitor_SMD:C_0402_1005Metric, symbol Device:C
- added C5513, C5516: 330 pF, Capacitor_SMD:C_0402_1005Metric, symbol Device:C
- added C5514, C5517: 68 pF, Capacitor_SMD:C_0402_1005Metric, symbol Device:C
- added C5515, C5518: 100 pF, Capacitor_SMD:C_0402_1005Metric, symbol Device:C
- added C5519, C5520: 1 nF, Capacitor_SMD:C_0402_1005Metric, symbol Device:C
- added L5501, L5502: 160 nH, Inductor_SMD:L_0603_1608Metric, symbol Device:L
- added R5501: 100 mΩ, Resistor_SMD:R_0603_1608Metric, symbol Device:R
- added R5502, R5503: 2.7 Ω, Resistor_SMD:R_0402_1005Metric, symbol Device:R
- added R5504, R5505: 2.2 kΩ, Resistor_SMD:R_0402_1005Metric, symbol Device:R
- added TP5501: NFC_VBAT_SRC, TestPoint:TestPoint_Pad_D1.0mm, symbol Connector:TestPoint
- added TP5502: NFC_VBAT, TestPoint:TestPoint_Pad_D1.0mm, symbol Connector:TestPoint
- added TP5503: NFC_ANT_P, TestPoint:TestPoint_Pad_D1.0mm, symbol Connector:TestPoint
- added TP5504: NFC_ANT_N, TestPoint:TestPoint_Pad_D1.0mm, symbol Connector:TestPoint
- added U5501: PN7160A1HN-C100E, NXP:NXP_SOT618-1_HVQFN-40-1EP_6x6mm_P0.5mm_EP4.1x4.1mm, symbol NXP:PN7160A1HN-C100E
- added U5502: TPS22919DCKR, Texas_Instruments:Texas_DCK0006A_SC-70-6_1.25x2mm_P0.65mm, symbol Texas_Instruments:TPS22919DCKR
- added Y5501: 27.12 MHz, Crystal:Crystal_SMD_2016-4Pin_2.0x1.6mm, symbol OpenDAP_Device:Crystal_GND24
Connections:
- net GND: now also C5501.2, C5502.2, C5503.2, C5504.2, C5505.2, C5506.2, C5507.2, C5508.2, C5509.2, C5510.2, C5511.2, C5512.2, C5513.2, C5515.2, C5516.2, C5518.2, U5501.1 (I2C_ADR0/SPI_NSS), U5501.20 (VSS(TX)), U5501.3 (I2C_ADR1/SPI_MOSI), U5501.39 (WKUP_REQ), U5501.4 (VSS(PAD)), U5501.9 (VSS(A)), U5501.EP (VSS), U5502.2 (GND), Y5501.2, Y5501.4
- net I2C2_SCL: now also U5501.7 (I2C_SCL/SPI_SCK)
- net I2C2_SDA: now also U5501.5 (I2C_SDA/SPI_MISO)
- net NFC_ANT_N: now also R5503.2, TP5504.1
- net NFC_ANT_P: now also R5502.2, TP5503.1
- net NFC_DWL_REQ: now also U5501.2 (DWL_REQ)
- net NFC_EMC_N: now also C5516.1, C5517.1, L5502.2, R5505.1
- net NFC_EMC_P: now also C5513.1, C5514.1, L5501.2, R5504.1
- net NFC_IRQ: now also U5501.8 (IRQ)
- net NFC_MATCH_N: now also C5517.2, C5518.1, R5503.1
- net NFC_MATCH_P: now also C5514.2, C5515.1, R5502.1
- net NFC_PWR_EN: now also U5502.3 (ON)
- net NFC_RXN: now also C5520.2, U5501.15 (RXN)
- net NFC_RXN_R: now also C5520.1, R5505.2
- net NFC_RXP: now also C5519.2, U5501.16 (RXP)
- net NFC_RXP_R: now also C5519.1, R5504.2
- net NFC_TVDD: now also C5504.1, C5505.1, U5501.14 (VDD(TX)), U5501.18 (TVDD_IN), U5501.22 (TVDD_IN2)
- net NFC_TX1: now also L5501.1, U5501.21 (TX1)
- net NFC_TX2: now also L5502.1, U5501.19 (TX2)
- net NFC_VBAT: now also C5501.1, C5502.1, C5503.1, R5501.2, TP5502.1, U5501.12 (VBAT2), U5501.13 (VDD(UP)), U5501.28 (VBAT)
- net NFC_VBAT_SRC: now also R5501.1, TP5501.1, U5502.5 (QOD), U5502.6 (VOUT)
- net NFC_VDD: now also C5506.1, C5507.1, U5501.26 (VDD(A)), U5501.27 (VDD), U5501.31 (VDD(D))
- net NFC_VEN: now also U5501.10 (VEN)
- net NFC_VMID: now also C5509.1, U5501.17 (VDD(VMID))
- net NFC_XTAL1: now also C5510.1, U5501.30 (NFC_CLK_XTAL1), Y5501.1
- net NFC_XTAL2: now also C5511.1, U5501.29 (XTAL2), Y5501.3
- net VSYS_LV: now also C5512.1, U5502.1 (IN)
- net vcca1v8_pmu: now also C5508.1, U5501.6 (VDD(PAD))

Commit message: Board: capture blk.debug
Debug UART2 (1.8 V) and I2S/DSD pads with ground pads, reset, PMIC and
power-key pads (PCB-T-09), a pad on every spare SoC GPIO whose pinout v1
row names one (the DEBUG bus, on the SoC's right edge), and a rail pad
for each power-tree rail no other sheet probes (PCB-T-02). Each DAC
sheet carries a pad on its MCLK. The spares pinout v1 leaves without a
pad now carry no-connect flags. On the root, facing sheet pins are
joined directly only where the route meets no other symbol.

Co-Authored-By: Claude Opus 5.5 <noreply@anthropic.com>
Claude-Session: https://claude.ai/code/session_01Ei262h3TpgY9vyfNLMi5Mn
Parts:
- removed C5501, C5503: 4.7 µF, Capacitor_SMD:C_0402_1005Metric, symbol Device:C
- removed C5502, C5509: 100 nF, Capacitor_SMD:C_0402_1005Metric, symbol Device:C
- removed C5504, C5505, C5506, C5507: 2.2 µF, Capacitor_SMD:C_0402_1005Metric, symbol Device:C
- removed C5508, C5512: 1 µF, Capacitor_SMD:C_0402_1005Metric, symbol Device:C
- removed C5510, C5511: 15 pF, Capacitor_SMD:C_0402_1005Metric, symbol Device:C
- removed C5513, C5516: 330 pF, Capacitor_SMD:C_0402_1005Metric, symbol Device:C
- removed C5514, C5517: 68 pF, Capacitor_SMD:C_0402_1005Metric, symbol Device:C
- removed C5515, C5518: 100 pF, Capacitor_SMD:C_0402_1005Metric, symbol Device:C
- removed C5519, C5520: 1 nF, Capacitor_SMD:C_0402_1005Metric, symbol Device:C
- removed L5501, L5502: 160 nH, Inductor_SMD:L_0603_1608Metric, symbol Device:L
- removed R5501: 100 mΩ, Resistor_SMD:R_0603_1608Metric, symbol Device:R
- removed R5502, R5503: 2.7 Ω, Resistor_SMD:R_0402_1005Metric, symbol Device:R
- removed R5504, R5505: 2.2 kΩ, Resistor_SMD:R_0402_1005Metric, symbol Device:R
- removed TP5501: NFC_VBAT_SRC, TestPoint:TestPoint_Pad_D1.0mm, symbol Connector:TestPoint
- removed TP5502: NFC_VBAT, TestPoint:TestPoint_Pad_D1.0mm, symbol Connector:TestPoint
- removed TP5503: NFC_ANT_P, TestPoint:TestPoint_Pad_D1.0mm, symbol Connector:TestPoint
- removed TP5504: NFC_ANT_N, TestPoint:TestPoint_Pad_D1.0mm, symbol Connector:TestPoint
- removed U5501: PN7160A1HN-C100E, NXP:NXP_SOT618-1_HVQFN-40-1EP_6x6mm_P0.5mm_EP4.1x4.1mm, symbol NXP:PN7160A1HN-C100E
- removed U5502: TPS22919DCKR, Texas_Instruments:Texas_DCK0006A_SC-70-6_1.25x2mm_P0.65mm, symbol Texas_Instruments:TPS22919DCKR
- removed Y5501: 27.12 MHz, Crystal:Crystal_SMD_2016-4Pin_2.0x1.6mm, symbol OpenDAP_Device:Crystal_GND24
- added C5601, C5603: 4.7 µF, Capacitor_SMD:C_0402_1005Metric, symbol Device:C
- added C5602, C5609: 100 nF, Capacitor_SMD:C_0402_1005Metric, symbol Device:C
- added C5604, C5605, C5606, C5607: 2.2 µF, Capacitor_SMD:C_0402_1005Metric, symbol Device:C
- added C5608, C5612: 1 µF, Capacitor_SMD:C_0402_1005Metric, symbol Device:C
- added C5610, C5611: 15 pF, Capacitor_SMD:C_0402_1005Metric, symbol Device:C
- added C5613, C5616: 330 pF, Capacitor_SMD:C_0402_1005Metric, symbol Device:C
- added C5614, C5617: 68 pF, Capacitor_SMD:C_0402_1005Metric, symbol Device:C
- added C5615, C5618: 100 pF, Capacitor_SMD:C_0402_1005Metric, symbol Device:C
- added C5619, C5620: 1 nF, Capacitor_SMD:C_0402_1005Metric, symbol Device:C
- added L5601, L5602: 160 nH, Inductor_SMD:L_0603_1608Metric, symbol Device:L
- added R5601: 100 mΩ, Resistor_SMD:R_0603_1608Metric, symbol Device:R
- added R5602, R5603: 2.7 Ω, Resistor_SMD:R_0402_1005Metric, symbol Device:R
- added R5604, R5605: 2.2 kΩ, Resistor_SMD:R_0402_1005Metric, symbol Device:R
- added TP5601: NFC_VBAT_SRC, TestPoint:TestPoint_Pad_D1.0mm, symbol Connector:TestPoint
- added TP5602: NFC_VBAT, TestPoint:TestPoint_Pad_D1.0mm, symbol Connector:TestPoint
- added TP5603: NFC_ANT_P, TestPoint:TestPoint_Pad_D1.0mm, symbol Connector:TestPoint
- added TP5604: NFC_ANT_N, TestPoint:TestPoint_Pad_D1.0mm, symbol Connector:TestPoint
- added U5601: PN7160A1HN-C100E, NXP:NXP_SOT618-1_HVQFN-40-1EP_6x6mm_P0.5mm_EP4.1x4.1mm, symbol NXP:PN7160A1HN-C100E
- added U5602: TPS22919DCKR, Texas_Instruments:Texas_DCK0006A_SC-70-6_1.25x2mm_P0.65mm, symbol Texas_Instruments:TPS22919DCKR
- added Y5601: 27.12 MHz, Crystal:Crystal_SMD_2016-4Pin_2.0x1.6mm, symbol OpenDAP_Device:Crystal_GND24
Connections:
- net GND: now also C5601.2, C5602.2, C5603.2, C5604.2, C5605.2, C5606.2, C5607.2, C5608.2, C5609.2, C5610.2, C5611.2, C5612.2, C5613.2, C5615.2, C5616.2, C5618.2, U5601.1 (I2C_ADR0/SPI_NSS), U5601.20 (VSS(TX)), U5601.3 (I2C_ADR1/SPI_MOSI), U5601.39 (WKUP_REQ), U5601.4 (VSS(PAD)), U5601.9 (VSS(A)), U5601.EP (VSS), U5602.2 (GND), Y5601.2, Y5601.4
- net I2C2_SCL: now also U5601.7 (I2C_SCL/SPI_SCK)
- net I2C2_SDA: now also U5601.5 (I2C_SDA/SPI_MISO)
- net NFC_ANT_N: now also R5603.2, TP5604.1
- net NFC_ANT_P: now also R5602.2, TP5603.1
- net NFC_DWL_REQ: now also U5601.2 (DWL_REQ)
- net NFC_EMC_N: now also C5616.1, C5617.1, L5602.2, R5605.1
- net NFC_EMC_P: now also C5613.1, C5614.1, L5601.2, R5604.1
- net NFC_IRQ: now also U5601.8 (IRQ)
- net NFC_MATCH_N: now also C5617.2, C5618.1, R5603.1
- net NFC_MATCH_P: now also C5614.2, C5615.1, R5602.1
- net NFC_PWR_EN: now also U5602.3 (ON)
- net NFC_RXN: now also C5620.2, U5601.15 (RXN)
- net NFC_RXN_R: now also C5620.1, R5605.2
- net NFC_RXP: now also C5619.2, U5601.16 (RXP)
- net NFC_RXP_R: now also C5619.1, R5604.2
- net NFC_TVDD: now also C5604.1, C5605.1, U5601.14 (VDD(TX)), U5601.18 (TVDD_IN), U5601.22 (TVDD_IN2)
- net NFC_TX1: now also L5601.1, U5601.21 (TX1)
- net NFC_TX2: now also L5602.1, U5601.19 (TX2)
- net NFC_VBAT: now also C5601.1, C5602.1, C5603.1, R5601.2, TP5602.1, U5601.12 (VBAT2), U5601.13 (VDD(UP)), U5601.28 (VBAT)
- net NFC_VBAT_SRC: now also R5601.1, TP5601.1, U5602.5 (QOD), U5602.6 (VOUT)
- net NFC_VDD: now also C5606.1, C5607.1, U5601.26 (VDD(A)), U5601.27 (VDD), U5601.31 (VDD(D))
- net NFC_VEN: now also U5601.10 (VEN)
- net NFC_VMID: now also C5609.1, U5601.17 (VDD(VMID))
- net NFC_XTAL1: now also C5610.1, U5601.30 (NFC_CLK_XTAL1), Y5601.1
- net NFC_XTAL2: now also C5611.1, U5601.29 (XTAL2), Y5601.3
- net VSYS_LV: now also C5612.1, U5602.1 (IN)
- net vcca1v8_pmu: now also C5608.1, U5601.6 (VDD(PAD))

Commit message: Board: capture blk.mic-ambient and links #34, #35
IM73D122 on PDM CLK1 and SDI1 (BOM v1 line 34, pinout v1 AK2 and 1P2),
LR to ground, 22 Ω clock series, VDD from MIC_1V8 through link #35.
Link #34 on blk.mic-main makes the faceplate branch the rail MIC_1V8_FP
for contact 40 (power tree §4.12, G10). kicad-lib moves to e46bda4 for
the IM73D122, TPS3808G01, SN74LVC1G58 and BAT54 parts.

Co-Authored-By: Claude Opus 5.5 <noreply@anthropic.com>
Claude-Session: https://claude.ai/code/session_01Ei262h3TpgY9vyfNLMi5Mn
Parts:
- removed C5601, C5603: 4.7 µF, Capacitor_SMD:C_0402_1005Metric, symbol Device:C
- removed C5602, C5609: 100 nF, Capacitor_SMD:C_0402_1005Metric, symbol Device:C
- removed C5604, C5605, C5606, C5607: 2.2 µF, Capacitor_SMD:C_0402_1005Metric, symbol Device:C
- removed C5608, C5612: 1 µF, Capacitor_SMD:C_0402_1005Metric, symbol Device:C
- removed C5610, C5611: 15 pF, Capacitor_SMD:C_0402_1005Metric, symbol Device:C
- removed C5613, C5616: 330 pF, Capacitor_SMD:C_0402_1005Metric, symbol Device:C
- removed C5614, C5617: 68 pF, Capacitor_SMD:C_0402_1005Metric, symbol Device:C
- removed C5615, C5618: 100 pF, Capacitor_SMD:C_0402_1005Metric, symbol Device:C
- removed C5619, C5620: 1 nF, Capacitor_SMD:C_0402_1005Metric, symbol Device:C
- removed L5601, L5602: 160 nH, Inductor_SMD:L_0603_1608Metric, symbol Device:L
- removed R5601: 100 mΩ, Resistor_SMD:R_0603_1608Metric, symbol Device:R
- removed R5602, R5603: 2.7 Ω, Resistor_SMD:R_0402_1005Metric, symbol Device:R
- removed R5604, R5605: 2.2 kΩ, Resistor_SMD:R_0402_1005Metric, symbol Device:R
- removed TP5601: NFC_VBAT_SRC, TestPoint:TestPoint_Pad_D1.0mm, symbol Connector:TestPoint
- removed TP5602: NFC_VBAT, TestPoint:TestPoint_Pad_D1.0mm, symbol Connector:TestPoint
- removed TP5603: NFC_ANT_P, TestPoint:TestPoint_Pad_D1.0mm, symbol Connector:TestPoint
- removed TP5604: NFC_ANT_N, TestPoint:TestPoint_Pad_D1.0mm, symbol Connector:TestPoint
- removed U5601: PN7160A1HN-C100E, NXP:NXP_SOT618-1_HVQFN-40-1EP_6x6mm_P0.5mm_EP4.1x4.1mm, symbol NXP:PN7160A1HN-C100E
- removed U5602: TPS22919DCKR, Texas_Instruments:Texas_DCK0006A_SC-70-6_1.25x2mm_P0.65mm, symbol Texas_Instruments:TPS22919DCKR
- removed Y5601: 27.12 MHz, Crystal:Crystal_SMD_2016-4Pin_2.0x1.6mm, symbol OpenDAP_Device:Crystal_GND24
- added C5701, C5703: 4.7 µF, Capacitor_SMD:C_0402_1005Metric, symbol Device:C
- added C5702, C5709: 100 nF, Capacitor_SMD:C_0402_1005Metric, symbol Device:C
- added C5704, C5705, C5706, C5707: 2.2 µF, Capacitor_SMD:C_0402_1005Metric, symbol Device:C
- added C5708, C5712: 1 µF, Capacitor_SMD:C_0402_1005Metric, symbol Device:C
- added C5710, C5711: 15 pF, Capacitor_SMD:C_0402_1005Metric, symbol Device:C
- added C5713, C5716: 330 pF, Capacitor_SMD:C_0402_1005Metric, symbol Device:C
- added C5714, C5717: 68 pF, Capacitor_SMD:C_0402_1005Metric, symbol Device:C
- added C5715, C5718: 100 pF, Capacitor_SMD:C_0402_1005Metric, symbol Device:C
- added C5719, C5720: 1 nF, Capacitor_SMD:C_0402_1005Metric, symbol Device:C
- added L5701, L5702: 160 nH, Inductor_SMD:L_0603_1608Metric, symbol Device:L
- added R5701: 100 mΩ, Resistor_SMD:R_0603_1608Metric, symbol Device:R
- added R5702, R5703: 2.7 Ω, Resistor_SMD:R_0402_1005Metric, symbol Device:R
- added R5704, R5705: 2.2 kΩ, Resistor_SMD:R_0402_1005Metric, symbol Device:R
- added TP5701: NFC_VBAT_SRC, TestPoint:TestPoint_Pad_D1.0mm, symbol Connector:TestPoint
- added TP5702: NFC_VBAT, TestPoint:TestPoint_Pad_D1.0mm, symbol Connector:TestPoint
- added TP5703: NFC_ANT_P, TestPoint:TestPoint_Pad_D1.0mm, symbol Connector:TestPoint
- added TP5704: NFC_ANT_N, TestPoint:TestPoint_Pad_D1.0mm, symbol Connector:TestPoint
- added U5701: PN7160A1HN-C100E, NXP:NXP_SOT618-1_HVQFN-40-1EP_6x6mm_P0.5mm_EP4.1x4.1mm, symbol NXP:PN7160A1HN-C100E
- added U5702: TPS22919DCKR, Texas_Instruments:Texas_DCK0006A_SC-70-6_1.25x2mm_P0.65mm, symbol Texas_Instruments:TPS22919DCKR
- added Y5701: 27.12 MHz, Crystal:Crystal_SMD_2016-4Pin_2.0x1.6mm, symbol OpenDAP_Device:Crystal_GND24
Connections:
- net GND: now also C5701.2, C5702.2, C5703.2, C5704.2, C5705.2, C5706.2, C5707.2, C5708.2, C5709.2, C5710.2, C5711.2, C5712.2, C5713.2, C5715.2, C5716.2, C5718.2, U5701.1 (I2C_ADR0/SPI_NSS), U5701.20 (VSS(TX)), U5701.3 (I2C_ADR1/SPI_MOSI), U5701.39 (WKUP_REQ), U5701.4 (VSS(PAD)), U5701.9 (VSS(A)), U5701.EP (VSS), U5702.2 (GND), Y5701.2, Y5701.4
- net I2C2_SCL: now also U5701.7 (I2C_SCL/SPI_SCK)
- net I2C2_SDA: now also U5701.5 (I2C_SDA/SPI_MISO)
- net NFC_ANT_N: now also R5703.2, TP5704.1
- net NFC_ANT_P: now also R5702.2, TP5703.1
- net NFC_DWL_REQ: now also U5701.2 (DWL_REQ)
- net NFC_EMC_N: now also C5716.1, C5717.1, L5702.2, R5705.1
- net NFC_EMC_P: now also C5713.1, C5714.1, L5701.2, R5704.1
- net NFC_IRQ: now also U5701.8 (IRQ)
- net NFC_MATCH_N: now also C5717.2, C5718.1, R5703.1
- net NFC_MATCH_P: now also C5714.2, C5715.1, R5702.1
- net NFC_PWR_EN: now also U5702.3 (ON)
- net NFC_RXN: now also C5720.2, U5701.15 (RXN)
- net NFC_RXN_R: now also C5720.1, R5705.2
- net NFC_RXP: now also C5719.2, U5701.16 (RXP)
- net NFC_RXP_R: now also C5719.1, R5704.2
- net NFC_TVDD: now also C5704.1, C5705.1, U5701.14 (VDD(TX)), U5701.18 (TVDD_IN), U5701.22 (TVDD_IN2)
- net NFC_TX1: now also L5701.1, U5701.21 (TX1)
- net NFC_TX2: now also L5702.1, U5701.19 (TX2)
- net NFC_VBAT: now also C5701.1, C5702.1, C5703.1, R5701.2, TP5702.1, U5701.12 (VBAT2), U5701.13 (VDD(UP)), U5701.28 (VBAT)
- net NFC_VBAT_SRC: now also R5701.1, TP5701.1, U5702.5 (QOD), U5702.6 (VOUT)
- net NFC_VDD: now also C5706.1, C5707.1, U5701.26 (VDD(A)), U5701.27 (VDD), U5701.31 (VDD(D))
- net NFC_VEN: now also U5701.10 (VEN)
- net NFC_VMID: now also C5709.1, U5701.17 (VDD(VMID))
- net NFC_XTAL1: now also C5710.1, U5701.30 (NFC_CLK_XTAL1), Y5701.1
- net NFC_XTAL2: now also C5711.1, U5701.29 (XTAL2), Y5701.3
- net VSYS_LV: now also C5712.1, U5702.1 (IN)
- net vcca1v8_pmu: now also C5708.1, U5701.6 (VDD(PAD))

Commit message: Board: capture blk.maskrom
Power + Vol- at a cold power-on pull eMMC D0 low inside the TPS3808G01
boot window (BOM v1 lines 35, 78, 97, 98; sim/maskrom): SENSE 280k/100k,
CT 390 nF, WINDOW_N with its pad, SN74LVC1G57 and SN74LVC1G58 on
vcca1v8_pmu, BAT54 from PWRON_N, DMG1012T through 1 kΩ to EMMC_D0.
Every block in use now has its sheet; the README states the remaining
single-pin nets.

Co-Authored-By: Claude Opus 5.5 <noreply@anthropic.com>
Claude-Session: https://claude.ai/code/session_01Ei262h3TpgY9vyfNLMi5Mn
Parts:
- removed C5701, C5703: 4.7 µF, Capacitor_SMD:C_0402_1005Metric, symbol Device:C
- removed C5702, C5709: 100 nF, Capacitor_SMD:C_0402_1005Metric, symbol Device:C
- removed C5704, C5705, C5706, C5707: 2.2 µF, Capacitor_SMD:C_0402_1005Metric, symbol Device:C
- removed C5708, C5712: 1 µF, Capacitor_SMD:C_0402_1005Metric, symbol Device:C
- removed C5710, C5711: 15 pF, Capacitor_SMD:C_0402_1005Metric, symbol Device:C
- removed C5713, C5716: 330 pF, Capacitor_SMD:C_0402_1005Metric, symbol Device:C
- removed C5714, C5717: 68 pF, Capacitor_SMD:C_0402_1005Metric, symbol Device:C
- removed C5715, C5718: 100 pF, Capacitor_SMD:C_0402_1005Metric, symbol Device:C
- removed C5719, C5720: 1 nF, Capacitor_SMD:C_0402_1005Metric, symbol Device:C
- removed L5701, L5702: 160 nH, Inductor_SMD:L_0603_1608Metric, symbol Device:L
- removed R5701: 100 mΩ, Resistor_SMD:R_0603_1608Metric, symbol Device:R
- removed R5702, R5703: 2.7 Ω, Resistor_SMD:R_0402_1005Metric, symbol Device:R
- removed R5704, R5705: 2.2 kΩ, Resistor_SMD:R_0402_1005Metric, symbol Device:R
- removed TP5701: NFC_VBAT_SRC, TestPoint:TestPoint_Pad_D1.0mm, symbol Connector:TestPoint
- removed TP5702: NFC_VBAT, TestPoint:TestPoint_Pad_D1.0mm, symbol Connector:TestPoint
- removed TP5703: NFC_ANT_P, TestPoint:TestPoint_Pad_D1.0mm, symbol Connector:TestPoint
- removed TP5704: NFC_ANT_N, TestPoint:TestPoint_Pad_D1.0mm, symbol Connector:TestPoint
- removed U5701: PN7160A1HN-C100E, NXP:NXP_SOT618-1_HVQFN-40-1EP_6x6mm_P0.5mm_EP4.1x4.1mm, symbol NXP:PN7160A1HN-C100E
- removed U5702: TPS22919DCKR, Texas_Instruments:Texas_DCK0006A_SC-70-6_1.25x2mm_P0.65mm, symbol Texas_Instruments:TPS22919DCKR
- removed Y5701: 27.12 MHz, Crystal:Crystal_SMD_2016-4Pin_2.0x1.6mm, symbol OpenDAP_Device:Crystal_GND24
- added C5801, C5803: 4.7 µF, Capacitor_SMD:C_0402_1005Metric, symbol Device:C
- added C5802, C5809: 100 nF, Capacitor_SMD:C_0402_1005Metric, symbol Device:C
- added C5804, C5805, C5806, C5807: 2.2 µF, Capacitor_SMD:C_0402_1005Metric, symbol Device:C
- added C5808, C5812: 1 µF, Capacitor_SMD:C_0402_1005Metric, symbol Device:C
- added C5810, C5811: 15 pF, Capacitor_SMD:C_0402_1005Metric, symbol Device:C
- added C5813, C5816: 330 pF, Capacitor_SMD:C_0402_1005Metric, symbol Device:C
- added C5814, C5817: 68 pF, Capacitor_SMD:C_0402_1005Metric, symbol Device:C
- added C5815, C5818: 100 pF, Capacitor_SMD:C_0402_1005Metric, symbol Device:C
- added C5819, C5820: 1 nF, Capacitor_SMD:C_0402_1005Metric, symbol Device:C
- added L5801, L5802: 160 nH, Inductor_SMD:L_0603_1608Metric, symbol Device:L
- added R5801: 100 mΩ, Resistor_SMD:R_0603_1608Metric, symbol Device:R
- added R5802, R5803: 2.7 Ω, Resistor_SMD:R_0402_1005Metric, symbol Device:R
- added R5804, R5805: 2.2 kΩ, Resistor_SMD:R_0402_1005Metric, symbol Device:R
- added TP5801: NFC_VBAT_SRC, TestPoint:TestPoint_Pad_D1.0mm, symbol Connector:TestPoint
- added TP5802: NFC_VBAT, TestPoint:TestPoint_Pad_D1.0mm, symbol Connector:TestPoint
- added TP5803: NFC_ANT_P, TestPoint:TestPoint_Pad_D1.0mm, symbol Connector:TestPoint
- added TP5804: NFC_ANT_N, TestPoint:TestPoint_Pad_D1.0mm, symbol Connector:TestPoint
- added U5801: PN7160A1HN-C100E, NXP:NXP_SOT618-1_HVQFN-40-1EP_6x6mm_P0.5mm_EP4.1x4.1mm, symbol NXP:PN7160A1HN-C100E
- added U5802: TPS22919DCKR, Texas_Instruments:Texas_DCK0006A_SC-70-6_1.25x2mm_P0.65mm, symbol Texas_Instruments:TPS22919DCKR
- added Y5801: 27.12 MHz, Crystal:Crystal_SMD_2016-4Pin_2.0x1.6mm, symbol OpenDAP_Device:Crystal_GND24
Connections:
- net GND: now also C5801.2, C5802.2, C5803.2, C5804.2, C5805.2, C5806.2, C5807.2, C5808.2, C5809.2, C5810.2, C5811.2, C5812.2, C5813.2, C5815.2, C5816.2, C5818.2, U5801.1 (I2C_ADR0/SPI_NSS), U5801.20 (VSS(TX)), U5801.3 (I2C_ADR1/SPI_MOSI), U5801.39 (WKUP_REQ), U5801.4 (VSS(PAD)), U5801.9 (VSS(A)), U5801.EP (VSS), U5802.2 (GND), Y5801.2, Y5801.4
- net I2C2_SCL: now also U5801.7 (I2C_SCL/SPI_SCK)
- net I2C2_SDA: now also U5801.5 (I2C_SDA/SPI_MISO)
- net NFC_ANT_N: now also R5803.2, TP5804.1
- net NFC_ANT_P: now also R5802.2, TP5803.1
- net NFC_DWL_REQ: now also U5801.2 (DWL_REQ)
- net NFC_EMC_N: now also C5816.1, C5817.1, L5802.2, R5805.1
- net NFC_EMC_P: now also C5813.1, C5814.1, L5801.2, R5804.1
- net NFC_IRQ: now also U5801.8 (IRQ)
- net NFC_MATCH_N: now also C5817.2, C5818.1, R5803.1
- net NFC_MATCH_P: now also C5814.2, C5815.1, R5802.1
- net NFC_PWR_EN: now also U5802.3 (ON)
- net NFC_RXN: now also C5820.2, U5801.15 (RXN)
- net NFC_RXN_R: now also C5820.1, R5805.2
- net NFC_RXP: now also C5819.2, U5801.16 (RXP)
- net NFC_RXP_R: now also C5819.1, R5804.2
- net NFC_TVDD: now also C5804.1, C5805.1, U5801.14 (VDD(TX)), U5801.18 (TVDD_IN), U5801.22 (TVDD_IN2)
- net NFC_TX1: now also L5801.1, U5801.21 (TX1)
- net NFC_TX2: now also L5802.1, U5801.19 (TX2)
- net NFC_VBAT: now also C5801.1, C5802.1, C5803.1, R5801.2, TP5802.1, U5801.12 (VBAT2), U5801.13 (VDD(UP)), U5801.28 (VBAT)
- net NFC_VBAT_SRC: now also R5801.1, TP5801.1, U5802.5 (QOD), U5802.6 (VOUT)
- net NFC_VDD: now also C5806.1, C5807.1, U5801.26 (VDD(A)), U5801.27 (VDD), U5801.31 (VDD(D))
- net NFC_VEN: now also U5801.10 (VEN)
- net NFC_VMID: now also C5809.1, U5801.17 (VDD(VMID))
- net NFC_XTAL1: now also C5810.1, U5801.30 (NFC_CLK_XTAL1), Y5801.1
- net NFC_XTAL2: now also C5811.1, U5801.29 (XTAL2), Y5801.3
- net VSYS_LV: now also C5812.1, U5802.1 (IN)
- net vcca1v8_pmu: now also C5808.1, U5801.6 (VDD(PAD))
