File: board/hardware/t1-main-board/board-id.kicad_sch (KiCad schematic)
At the start: 2 parts, among them U5801 AT24C02D-STUM-T

Commit message: Board: capture blk.current-monitors
Five INA236 on I2C1 (0x40-0x43, 0x48) with their shunts, per power tree
§4.12 and BOM v1 lines 54 and 136. The measured branches are rails of
their own (VSYS_SRC, VSYS_LV_AUDIO, VSYS_AUDIO, VSYS_LV_BL, VSYS_P5V1),
fed through the shunts on this sheet; the charger, audio, backlight and
5.1 V sheets take them. The root's layout may leave a stack level empty,
so the block sits under the notes; IC bboxes hold turned rail values;
passive rows hold a bottom rail's text.

Co-Authored-By: Claude Opus 5.5 <noreply@anthropic.com>
Claude-Session: https://claude.ai/code/session_01Ei262h3TpgY9vyfNLMi5Mn
Parts:
- removed C5801: 100 nF, Capacitor_SMD:C_0402_1005Metric, symbol Device:C
- removed U5801: AT24C02D-STUM-T, Microchip:Microchip_5TS1_SOT-23-5_1.6x2.9mm_P0.95mm, symbol Microchip:AT24C02D-STUM-T
- added C5901: 100 nF, Capacitor_SMD:C_0402_1005Metric, symbol Device:C
- added U5901: AT24C02D-STUM-T, Microchip:Microchip_5TS1_SOT-23-5_1.6x2.9mm_P0.95mm, symbol Microchip:AT24C02D-STUM-T
Connections:
- net GND: now also C5901.2, U5901.2 (GND), U5901.5 (WP)
- net I2C2_SCL: now also U5901.1 (SCL)
- net I2C2_SDA: now also U5901.3 (SDA)
- net vcca1v8_pmu: now also C5901.1, U5901.4 (VCC)
Changed lines of the file:
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@@
 (title_block (title "Board EEPROM") (date "2026-10-25") (rev "A") (company "The OpenDAP Project") (comment 1 "blk.board-id") (comment 2 "AT24C02D board identity EEPROM on I2C2 at 0x50"))
 (symbol (lib_id "Microchip:AT24C02D-STUM-T") (at 45.72 63.5 0) (unit 1) (body_style 1) (exclude_from_sim no) (in_bom yes) (on_board yes) (dnp no)
-  (property "Reference" "U5801" (at 52.07 50.8 0) (effects (font (size 1.27 1.27)) (justify left)))
+  (property "Reference" "U5901" (at 52.07 50.8 0) (effects (font (size 1.27 1.27)) (justify left)))
   (property "Value" "AT24C02D-STUM-T" (at 52.07 48.26 0) (effects (font (size 1.27 1.27)) (justify left)))
   (property "Footprint" "Microchip:Microchip_5TS1_SOT-23-5_1.6x2.9mm_P0.95mm" (at 45.72 63.5 0) (effects (font (size 1.27 1.27))) (hide yes))
@@
   (pin "4")
   (pin "2")
-  (instances (project "t1-main-board" (path "/7746052e-d7f9-59ad-ba73-bd2b74439529/5b273614-fd04-534a-8238-3227aff193cb" (reference "U5801") (unit 1))))
+  (instances (project "t1-main-board" (path "/7746052e-d7f9-59ad-ba73-bd2b74439529/5b273614-fd04-534a-8238-3227aff193cb" (reference "U5901") (unit 1))))
 )
 (wire (pts (xy 38.1 60.96) (xy 35.56 60.96)) (stroke (width 0) (type default)))
@@
 )
 (symbol (lib_id "Device:C") (at 80.01 48.26 0) (unit 1) (body_style 1) (exclude_from_sim no) (in_bom yes) (on_board yes) (dnp no)
-  (property "Reference" "C5801" (at 82.55 46.99 0) (effects (font (size 1.27 1.27)) (justify left)))
+  (property "Reference" "C5901" (at 82.55 46.99 0) (effects (font (size 1.27 1.27)) (justify left)))
   (property "Value" "100 nF" (at 82.55 49.53 0) (effects (font (size 1.27 1.27)) (justify left)))
   (property "Footprint" "Capacitor_SMD:C_0402_1005Metric" (at 80.01 48.26 0) (effects (font (size 1.27 1.27))) (hide yes))
@@
   (pin "1")
   (pin "2")
-  (instances (project "t1-main-board" (path "/7746052e-d7f9-59ad-ba73-bd2b74439529/5b273614-fd04-534a-8238-3227aff193cb" (reference "C5801") (unit 1))))
+  (instances (project "t1-main-board" (path "/7746052e-d7f9-59ad-ba73-bd2b74439529/5b273614-fd04-534a-8238-3227aff193cb" (reference "C5901") (unit 1))))
 )
 (wire (pts (xy 80.01 44.45) (xy 80.01 41.91)) (stroke (width 0) (type default)))

Commit message: Board: capture blk.status-led
LP5521 at 0x32 on I2C2 (BOM v1 line 105) with its charge-pump
capacitors, EN on vcca1v8_pmu, VDD from VSYS_LV through link #22;
LED_R/G/B reach the faceplate connector as the LED bus alias. The
faceplate row of the root is re-packed so five full columns sit left of
the title block.

Co-Authored-By: Claude Opus 5.5 <noreply@anthropic.com>
Claude-Session: https://claude.ai/code/session_01Ei262h3TpgY9vyfNLMi5Mn
Parts:
- removed C5901: 100 nF, Capacitor_SMD:C_0402_1005Metric, symbol Device:C
- removed U5901: AT24C02D-STUM-T, Microchip:Microchip_5TS1_SOT-23-5_1.6x2.9mm_P0.95mm, symbol Microchip:AT24C02D-STUM-T
- added C5301: 100 nF, Capacitor_SMD:C_0402_1005Metric, symbol Device:C
- added U5301: AT24C02D-STUM-T, Microchip:Microchip_5TS1_SOT-23-5_1.6x2.9mm_P0.95mm, symbol Microchip:AT24C02D-STUM-T
Connections:
- net GND: now also C5301.2, U5301.2 (GND), U5301.5 (WP)
- net I2C2_SCL: now also U5301.1 (SCL)
- net I2C2_SDA: now also U5301.3 (SDA)
- net vcca1v8_pmu: now also C5301.1, U5301.4 (VCC)
Changed lines of the file:
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@@
 (title_block (title "Board EEPROM") (date "2026-10-25") (rev "A") (company "The OpenDAP Project") (comment 1 "blk.board-id") (comment 2 "AT24C02D board identity EEPROM on I2C2 at 0x50"))
 (symbol (lib_id "Microchip:AT24C02D-STUM-T") (at 45.72 63.5 0) (unit 1) (body_style 1) (exclude_from_sim no) (in_bom yes) (on_board yes) (dnp no)
-  (property "Reference" "U5901" (at 52.07 50.8 0) (effects (font (size 1.27 1.27)) (justify left)))
+  (property "Reference" "U5301" (at 52.07 50.8 0) (effects (font (size 1.27 1.27)) (justify left)))
   (property "Value" "AT24C02D-STUM-T" (at 52.07 48.26 0) (effects (font (size 1.27 1.27)) (justify left)))
   (property "Footprint" "Microchip:Microchip_5TS1_SOT-23-5_1.6x2.9mm_P0.95mm" (at 45.72 63.5 0) (effects (font (size 1.27 1.27))) (hide yes))
@@
   (pin "4")
   (pin "2")
-  (instances (project "t1-main-board" (path "/7746052e-d7f9-59ad-ba73-bd2b74439529/5b273614-fd04-534a-8238-3227aff193cb" (reference "U5901") (unit 1))))
+  (instances (project "t1-main-board" (path "/7746052e-d7f9-59ad-ba73-bd2b74439529/5b273614-fd04-534a-8238-3227aff193cb" (reference "U5301") (unit 1))))
 )
 (wire (pts (xy 38.1 60.96) (xy 35.56 60.96)) (stroke (width 0) (type default)))
@@
 )
 (symbol (lib_id "Device:C") (at 80.01 48.26 0) (unit 1) (body_style 1) (exclude_from_sim no) (in_bom yes) (on_board yes) (dnp no)
-  (property "Reference" "C5901" (at 82.55 46.99 0) (effects (font (size 1.27 1.27)) (justify left)))
+  (property "Reference" "C5301" (at 82.55 46.99 0) (effects (font (size 1.27 1.27)) (justify left)))
   (property "Value" "100 nF" (at 82.55 49.53 0) (effects (font (size 1.27 1.27)) (justify left)))
   (property "Footprint" "Capacitor_SMD:C_0402_1005Metric" (at 80.01 48.26 0) (effects (font (size 1.27 1.27))) (hide yes))
@@
   (pin "1")
   (pin "2")
-  (instances (project "t1-main-board" (path "/7746052e-d7f9-59ad-ba73-bd2b74439529/5b273614-fd04-534a-8238-3227aff193cb" (reference "C5901") (unit 1))))
+  (instances (project "t1-main-board" (path "/7746052e-d7f9-59ad-ba73-bd2b74439529/5b273614-fd04-534a-8238-3227aff193cb" (reference "C5301") (unit 1))))
 )
 (wire (pts (xy 80.01 44.45) (xy 80.01 41.91)) (stroke (width 0) (type default)))

Commit message: Board: capture blk.debug
Debug UART2 (1.8 V) and I2S/DSD pads with ground pads, reset, PMIC and
power-key pads (PCB-T-09), a pad on every spare SoC GPIO whose pinout v1
row names one (the DEBUG bus, on the SoC's right edge), and a rail pad
for each power-tree rail no other sheet probes (PCB-T-02). Each DAC
sheet carries a pad on its MCLK. The spares pinout v1 leaves without a
pad now carry no-connect flags. On the root, facing sheet pins are
joined directly only where the route meets no other symbol.

Co-Authored-By: Claude Opus 5.5 <noreply@anthropic.com>
Claude-Session: https://claude.ai/code/session_01Ei262h3TpgY9vyfNLMi5Mn
Parts:
- removed C5301: 100 nF, Capacitor_SMD:C_0402_1005Metric, symbol Device:C
- removed U5301: AT24C02D-STUM-T, Microchip:Microchip_5TS1_SOT-23-5_1.6x2.9mm_P0.95mm, symbol Microchip:AT24C02D-STUM-T
- added C5401: 100 nF, Capacitor_SMD:C_0402_1005Metric, symbol Device:C
- added U5401: AT24C02D-STUM-T, Microchip:Microchip_5TS1_SOT-23-5_1.6x2.9mm_P0.95mm, symbol Microchip:AT24C02D-STUM-T
Connections:
- net GND: now also C5401.2, U5401.2 (GND), U5401.5 (WP)
- net I2C2_SCL: now also U5401.1 (SCL)
- net I2C2_SDA: now also U5401.3 (SDA)
- net vcca1v8_pmu: now also C5401.1, U5401.4 (VCC)
Changed lines of the file:
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@@
 (title_block (title "Board EEPROM") (date "2026-10-25") (rev "A") (company "The OpenDAP Project") (comment 1 "blk.board-id") (comment 2 "AT24C02D board identity EEPROM on I2C2 at 0x50"))
 (symbol (lib_id "Microchip:AT24C02D-STUM-T") (at 45.72 63.5 0) (unit 1) (body_style 1) (exclude_from_sim no) (in_bom yes) (on_board yes) (dnp no)
-  (property "Reference" "U5301" (at 52.07 50.8 0) (effects (font (size 1.27 1.27)) (justify left)))
+  (property "Reference" "U5401" (at 52.07 50.8 0) (effects (font (size 1.27 1.27)) (justify left)))
   (property "Value" "AT24C02D-STUM-T" (at 52.07 48.26 0) (effects (font (size 1.27 1.27)) (justify left)))
   (property "Footprint" "Microchip:Microchip_5TS1_SOT-23-5_1.6x2.9mm_P0.95mm" (at 45.72 63.5 0) (effects (font (size 1.27 1.27))) (hide yes))
@@
   (pin "4")
   (pin "2")
-  (instances (project "t1-main-board" (path "/7746052e-d7f9-59ad-ba73-bd2b74439529/5b273614-fd04-534a-8238-3227aff193cb" (reference "U5301") (unit 1))))
+  (instances (project "t1-main-board" (path "/7746052e-d7f9-59ad-ba73-bd2b74439529/5b273614-fd04-534a-8238-3227aff193cb" (reference "U5401") (unit 1))))
 )
 (wire (pts (xy 38.1 60.96) (xy 35.56 60.96)) (stroke (width 0) (type default)))
@@
 )
 (symbol (lib_id "Device:C") (at 80.01 48.26 0) (unit 1) (body_style 1) (exclude_from_sim no) (in_bom yes) (on_board yes) (dnp no)
-  (property "Reference" "C5301" (at 82.55 46.99 0) (effects (font (size 1.27 1.27)) (justify left)))
+  (property "Reference" "C5401" (at 82.55 46.99 0) (effects (font (size 1.27 1.27)) (justify left)))
   (property "Value" "100 nF" (at 82.55 49.53 0) (effects (font (size 1.27 1.27)) (justify left)))
   (property "Footprint" "Capacitor_SMD:C_0402_1005Metric" (at 80.01 48.26 0) (effects (font (size 1.27 1.27))) (hide yes))
@@
   (pin "1")
   (pin "2")
-  (instances (project "t1-main-board" (path "/7746052e-d7f9-59ad-ba73-bd2b74439529/5b273614-fd04-534a-8238-3227aff193cb" (reference "C5301") (unit 1))))
+  (instances (project "t1-main-board" (path "/7746052e-d7f9-59ad-ba73-bd2b74439529/5b273614-fd04-534a-8238-3227aff193cb" (reference "C5401") (unit 1))))
 )
 (wire (pts (xy 80.01 44.45) (xy 80.01 41.91)) (stroke (width 0) (type default)))

Commit message: Board: capture blk.mic-ambient and links #34, #35
IM73D122 on PDM CLK1 and SDI1 (BOM v1 line 34, pinout v1 AK2 and 1P2),
LR to ground, 22 Ω clock series, VDD from MIC_1V8 through link #35.
Link #34 on blk.mic-main makes the faceplate branch the rail MIC_1V8_FP
for contact 40 (power tree §4.12, G10). kicad-lib moves to e46bda4 for
the IM73D122, TPS3808G01, SN74LVC1G58 and BAT54 parts.

Co-Authored-By: Claude Opus 5.5 <noreply@anthropic.com>
Claude-Session: https://claude.ai/code/session_01Ei262h3TpgY9vyfNLMi5Mn
Parts:
- removed C5401: 100 nF, Capacitor_SMD:C_0402_1005Metric, symbol Device:C
- removed U5401: AT24C02D-STUM-T, Microchip:Microchip_5TS1_SOT-23-5_1.6x2.9mm_P0.95mm, symbol Microchip:AT24C02D-STUM-T
- added C5501: 100 nF, Capacitor_SMD:C_0402_1005Metric, symbol Device:C
- added U5501: AT24C02D-STUM-T, Microchip:Microchip_5TS1_SOT-23-5_1.6x2.9mm_P0.95mm, symbol Microchip:AT24C02D-STUM-T
Connections:
- net GND: now also C5501.2, U5501.2 (GND), U5501.5 (WP)
- net I2C2_SCL: now also U5501.1 (SCL)
- net I2C2_SDA: now also U5501.3 (SDA)
- net vcca1v8_pmu: now also C5501.1, U5501.4 (VCC)
Changed lines of the file:
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@@
 (title_block (title "Board EEPROM") (date "2026-10-25") (rev "A") (company "The OpenDAP Project") (comment 1 "blk.board-id") (comment 2 "AT24C02D board identity EEPROM on I2C2 at 0x50"))
 (symbol (lib_id "Microchip:AT24C02D-STUM-T") (at 45.72 63.5 0) (unit 1) (body_style 1) (exclude_from_sim no) (in_bom yes) (on_board yes) (dnp no)
-  (property "Reference" "U5401" (at 52.07 50.8 0) (effects (font (size 1.27 1.27)) (justify left)))
+  (property "Reference" "U5501" (at 52.07 50.8 0) (effects (font (size 1.27 1.27)) (justify left)))
   (property "Value" "AT24C02D-STUM-T" (at 52.07 48.26 0) (effects (font (size 1.27 1.27)) (justify left)))
   (property "Footprint" "Microchip:Microchip_5TS1_SOT-23-5_1.6x2.9mm_P0.95mm" (at 45.72 63.5 0) (effects (font (size 1.27 1.27))) (hide yes))
@@
   (pin "4")
   (pin "2")
-  (instances (project "t1-main-board" (path "/7746052e-d7f9-59ad-ba73-bd2b74439529/5b273614-fd04-534a-8238-3227aff193cb" (reference "U5401") (unit 1))))
+  (instances (project "t1-main-board" (path "/7746052e-d7f9-59ad-ba73-bd2b74439529/5b273614-fd04-534a-8238-3227aff193cb" (reference "U5501") (unit 1))))
 )
 (wire (pts (xy 38.1 60.96) (xy 35.56 60.96)) (stroke (width 0) (type default)))
@@
 (wire (pts (xy 38.1 68.58) (xy 35.56 68.58)) (stroke (width 0) (type default)))
 (symbol (lib_id "power:GND") (at 35.56 68.58 0) (unit 1) (body_style 1) (exclude_from_sim no) (in_bom yes) (on_board yes) (dnp no)
-  (property "Reference" "#PWR0769" (at 35.56 68.58 0) (effects (font (size 1.27 1.27))) (hide yes))
+  (property "Reference" "#PWR0771" (at 35.56 68.58 0) (effects (font (size 1.27 1.27))) (hide yes))
   (property "Value" "GND" (at 35.56 72.39 0) (effects (font (size 1.27 1.27))))
   (property "Footprint" "" (at 35.56 68.58 0) (effects (font (size 1.27 1.27))) (hide yes))
   (property "Datasheet" "" (at 35.56 68.58 0) (effects (font (size 1.27 1.27))) (hide yes))
   (pin "1")
-  (instances (project "t1-main-board" (path "/7746052e-d7f9-59ad-ba73-bd2b74439529/5b273614-fd04-534a-8238-3227aff193cb" (reference "#PWR0769") (unit 1))))
+  (instances (project "t1-main-board" (path "/7746052e-d7f9-59ad-ba73-bd2b74439529/5b273614-fd04-534a-8238-3227aff193cb" (reference "#PWR0771") (unit 1))))
 )
 (wire (pts (xy 45.72 45.72) (xy 45.72 43.18)) (stroke (width 0) (type default)))
 (symbol (lib_id "power:VCC") (at 45.72 43.18 0) (unit 1) (body_style 1) (exclude_from_sim no) (in_bom yes) (on_board yes) (dnp no)
-  (property "Reference" "#PWR0770" (at 45.72 43.18 0) (effects (font (size 1.27 1.27))) (hide yes))
+  (property "Reference" "#PWR0772" (at 45.72 43.18 0) (effects (font (size 1.27 1.27))) (hide yes))
   (property "Value" "vcca1v8_pmu" (at 45.72 39.37 0) (effects (font (size 1.27 1.27))))
   (property "Footprint" "" (at 45.72 43.18 0) (effects (font (size 1.27 1.27))) (hide yes))
   (property "Datasheet" "" (at 45.72 43.18 0) (effects (font (size 1.27 1.27))) (hide yes))
   (pin "1")
-  (instances (project "t1-main-board" (path "/7746052e-d7f9-59ad-ba73-bd2b74439529/5b273614-fd04-534a-8238-3227aff193cb" (reference "#PWR0770") (unit 1))))
+  (instances (project "t1-main-board" (path "/7746052e-d7f9-59ad-ba73-bd2b74439529/5b273614-fd04-534a-8238-3227aff193cb" (reference "#PWR0772") (unit 1))))
 )
 (wire (pts (xy 45.72 81.28) (xy 45.72 83.82)) (stroke (width 0) (type default)))
 (symbol (lib_id "power:GND") (at 45.72 83.82 0) (unit 1) (body_style 1) (exclude_from_sim no) (in_bom yes) (on_board yes) (dnp no)
-  (property "Reference" "#PWR0771" (at 45.72 83.82 0) (effects (font (size 1.27 1.27))) (hide yes))
+  (property "Reference" "#PWR0773" (at 45.72 83.82 0) (effects (font (size 1.27 1.27))) (hide yes))
   (property "Value" "GND" (at 45.72 87.63 0) (effects (font (size 1.27 1.27))))
   (property "Footprint" "" (at 45.72 83.82 0) (effects (font (size 1.27 1.27))) (hide yes))
   (property "Datasheet" "" (at 45.72 83.82 0) (effects (font (size 1.27 1.27))) (hide yes))
   (pin "1")
-  (instances (project "t1-main-board" (path "/7746052e-d7f9-59ad-ba73-bd2b74439529/5b273614-fd04-534a-8238-3227aff193cb" (reference "#PWR0771") (unit 1))))
+  (instances (project "t1-main-board" (path "/7746052e-d7f9-59ad-ba73-bd2b74439529/5b273614-fd04-534a-8238-3227aff193cb" (reference "#PWR0773") (unit 1))))
 )
 (symbol (lib_id "Device:C") (at 80.01 48.26 0) (unit 1) (body_style 1) (exclude_from_sim no) (in_bom yes) (on_board yes) (dnp no)
-  (property "Reference" "C5401" (at 82.55 46.99 0) (effects (font (size 1.27 1.27)) (justify left)))
+  (property "Reference" "C5501" (at 82.55 46.99 0) (effects (font (size 1.27 1.27)) (justify left)))
   (property "Value" "100 nF" (at 82.55 49.53 0) (effects (font (size 1.27 1.27)) (justify left)))
   (property "Footprint" "Capacitor_SMD:C_0402_1005Metric" (at 80.01 48.26 0) (effects (font (size 1.27 1.27))) (hide yes))
@@
   (pin "1")
   (pin "2")
-  (instances (project "t1-main-board" (path "/7746052e-d7f9-59ad-ba73-bd2b74439529/5b273614-fd04-534a-8238-3227aff193cb" (reference "C5401") (unit 1))))
+  (instances (project "t1-main-board" (path "/7746052e-d7f9-59ad-ba73-bd2b74439529/5b273614-fd04-534a-8238-3227aff193cb" (reference "C5501") (unit 1))))
 )
 (wire (pts (xy 80.01 44.45) (xy 80.01 41.91)) (stroke (width 0) (type default)))
 (wire (pts (xy 80.01 52.07) (xy 80.01 54.61)) (stroke (width 0) (type default)))
 (symbol (lib_id "power:GND") (at 80.01 54.61 0) (unit 1) (body_style 1) (exclude_from_sim no) (in_bom yes) (on_board yes) (dnp no)
-  (property "Reference" "#PWR0772" (at 80.01 54.61 0) (effects (font (size 1.27 1.27))) (hide yes))
+  (property "Reference" "#PWR0774" (at 80.01 54.61 0) (effects (font (size 1.27 1.27))) (hide yes))
   (property "Value" "GND" (at 80.01 58.42 0) (effects (font (size 1.27 1.27))))
   (property "Footprint" "" (at 80.01 54.61 0) (effects (font (size 1.27 1.27))) (hide yes))
   (property "Datasheet" "" (at 80.01 54.61 0) (effects (font (size 1.27 1.27))) (hide yes))
   (pin "1")
-  (instances (project "t1-main-board" (path "/7746052e-d7f9-59ad-ba73-bd2b74439529/5b273614-fd04-534a-8238-3227aff193cb" (reference "#PWR0772") (unit 1))))
+  (instances (project "t1-main-board" (path "/7746052e-d7f9-59ad-ba73-bd2b74439529/5b273614-fd04-534a-8238-3227aff193cb" (reference "#PWR0774") (unit 1))))
 )
 (symbol (lib_id "power:VCC") (at 80.01 41.91 0) (unit 1) (body_style 1) (exclude_from_sim no) (in_bom yes) (on_board yes) (dnp no)
-  (property "Reference" "#PWR0773" (at 80.01 41.91 0) (effects (font (size 1.27 1.27))) (hide yes))
+  (property "Reference" "#PWR0775" (at 80.01 41.91 0) (effects (font (size 1.27 1.27))) (hide yes))
   (property "Value" "vcca1v8_pmu" (at 80.01 38.1 0) (effects (font (size 1.27 1.27))))
   (property "Footprint" "" (at 80.01 41.91 0) (effects (font (size 1.27 1.27))) (hide yes))
   (property "Datasheet" "" (at 80.01 41.91 0) (effects (font (size 1.27 1.27))) (hide yes))
   (pin "1")
-  (instances (project "t1-main-board" (path "/7746052e-d7f9-59ad-ba73-bd2b74439529/5b273614-fd04-534a-8238-3227aff193cb" (reference "#PWR0773") (unit 1))))
+  (instances (project "t1-main-board" (path "/7746052e-d7f9-59ad-ba73-bd2b74439529/5b273614-fd04-534a-8238-3227aff193cb" (reference "#PWR0775") (unit 1))))
 )
 (rectangle (start 22.86 35.56) (end 93.98 92.71) (stroke (width 0) (type dash)) (fill (type none)))

Commit message: Board: capture blk.maskrom
Power + Vol- at a cold power-on pull eMMC D0 low inside the TPS3808G01
boot window (BOM v1 lines 35, 78, 97, 98; sim/maskrom): SENSE 280k/100k,
CT 390 nF, WINDOW_N with its pad, SN74LVC1G57 and SN74LVC1G58 on
vcca1v8_pmu, BAT54 from PWRON_N, DMG1012T through 1 kΩ to EMMC_D0.
Every block in use now has its sheet; the README states the remaining
single-pin nets.

Co-Authored-By: Claude Opus 5.5 <noreply@anthropic.com>
Claude-Session: https://claude.ai/code/session_01Ei262h3TpgY9vyfNLMi5Mn
Parts:
- removed C5501: 100 nF, Capacitor_SMD:C_0402_1005Metric, symbol Device:C
- removed U5501: AT24C02D-STUM-T, Microchip:Microchip_5TS1_SOT-23-5_1.6x2.9mm_P0.95mm, symbol Microchip:AT24C02D-STUM-T
- added C5601: 100 nF, Capacitor_SMD:C_0402_1005Metric, symbol Device:C
- added U5601: AT24C02D-STUM-T, Microchip:Microchip_5TS1_SOT-23-5_1.6x2.9mm_P0.95mm, symbol Microchip:AT24C02D-STUM-T
Connections:
- net GND: now also C5601.2, U5601.2 (GND), U5601.5 (WP)
- net I2C2_SCL: now also U5601.1 (SCL)
- net I2C2_SDA: now also U5601.3 (SDA)
- net vcca1v8_pmu: now also C5601.1, U5601.4 (VCC)
Changed lines of the file:
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@@
 (title_block (title "Board EEPROM") (date "2026-10-25") (rev "A") (company "The OpenDAP Project") (comment 1 "blk.board-id") (comment 2 "AT24C02D board identity EEPROM on I2C2 at 0x50"))
 (symbol (lib_id "Microchip:AT24C02D-STUM-T") (at 45.72 63.5 0) (unit 1) (body_style 1) (exclude_from_sim no) (in_bom yes) (on_board yes) (dnp no)
-  (property "Reference" "U5501" (at 52.07 50.8 0) (effects (font (size 1.27 1.27)) (justify left)))
+  (property "Reference" "U5601" (at 52.07 50.8 0) (effects (font (size 1.27 1.27)) (justify left)))
   (property "Value" "AT24C02D-STUM-T" (at 52.07 48.26 0) (effects (font (size 1.27 1.27)) (justify left)))
   (property "Footprint" "Microchip:Microchip_5TS1_SOT-23-5_1.6x2.9mm_P0.95mm" (at 45.72 63.5 0) (effects (font (size 1.27 1.27))) (hide yes))
@@
   (pin "4")
   (pin "2")
-  (instances (project "t1-main-board" (path "/7746052e-d7f9-59ad-ba73-bd2b74439529/5b273614-fd04-534a-8238-3227aff193cb" (reference "U5501") (unit 1))))
+  (instances (project "t1-main-board" (path "/7746052e-d7f9-59ad-ba73-bd2b74439529/5b273614-fd04-534a-8238-3227aff193cb" (reference "U5601") (unit 1))))
 )
 (wire (pts (xy 38.1 60.96) (xy 35.56 60.96)) (stroke (width 0) (type default)))
@@
 )
 (symbol (lib_id "Device:C") (at 80.01 48.26 0) (unit 1) (body_style 1) (exclude_from_sim no) (in_bom yes) (on_board yes) (dnp no)
-  (property "Reference" "C5501" (at 82.55 46.99 0) (effects (font (size 1.27 1.27)) (justify left)))
+  (property "Reference" "C5601" (at 82.55 46.99 0) (effects (font (size 1.27 1.27)) (justify left)))
   (property "Value" "100 nF" (at 82.55 49.53 0) (effects (font (size 1.27 1.27)) (justify left)))
   (property "Footprint" "Capacitor_SMD:C_0402_1005Metric" (at 80.01 48.26 0) (effects (font (size 1.27 1.27))) (hide yes))
@@
   (pin "1")
   (pin "2")
-  (instances (project "t1-main-board" (path "/7746052e-d7f9-59ad-ba73-bd2b74439529/5b273614-fd04-534a-8238-3227aff193cb" (reference "C5501") (unit 1))))
+  (instances (project "t1-main-board" (path "/7746052e-d7f9-59ad-ba73-bd2b74439529/5b273614-fd04-534a-8238-3227aff193cb" (reference "C5601") (unit 1))))
 )
 (wire (pts (xy 80.01 44.45) (xy 80.01 41.91)) (stroke (width 0) (type default)))
