File: board/hardware/t1-main-board/board-id.kicad_sch (KiCad schematic)
At the start: 2 parts, among them U5601 AT24C02D-STUM-T

Commit message: Compaction: lower inductors, 0201 decoupling, 0.8 mm signal test pads
A matrix tool (hardware/studies/compaction) checks each candidate against
the design's stresses: same inductance, design peak <= 70 % and the
converter's maximum limit <= 100 % of Isat (30 % drop), height zones,
ratings at least twice the rail, PCB-D-06; sourcing outcome per part.

Applied (placement v1 decision 12, BOM v1.15):
- L601, L4401: XGL4015-102MEC (1.5 mm) for XAL/XGL4020-102MEC (2.1 mm);
- L1001, L5101: XGL4015-471MEC (1.5 mm) for Wurth 744373240047, on the
  stock XxL4020 land (the Wurth land was never drawn);
- L1201 is 1.2 mm (XGL4012, per-MPN heights): it moves next to the SoC;
- 58 x 100 nF decoupling on rails <= 3.3 V in core/IO/radio: 0201;
- 51 test pads on signal nets: 0.8 mm (PCB-D-06 v0.16, JLCPCB guide).
Kept: L901, L2802 (XGL4015 at 103 % of Isat at the limit); no thinner
0805/1206 capacitor passes (obsolete, NRND or unlisted).

Board need 113 % -> 111 % (core band 227 -> 203 %, power band 258 ->
233 %, radio band 19 -> 0 %); only C904 still relies on PCB-Z-04.
ERC 0 errors, craft Q1 met, DRC 0 errors (605 warnings), pcb and study
tests pass, rules test board PASS.

Co-Authored-By: Claude Opus 5.5 <noreply@anthropic.com>
Claude-Session: https://claude.ai/code/session_01Ei262h3TpgY9vyfNLMi5Mn
Parts:
- C5601: footprint Capacitor_SMD:C_0402_1005Metric -> Capacitor_SMD:C_0201_0603Metric; MPN GRM155R71C104KA88D -> GRM033R61A104KE15D
Changed lines of the file:
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@@
   (property "Reference" "C5601" (at 82.55 46.99 0) (effects (font (size 1.27 1.27)) (justify left)))
   (property "Value" "100 nF" (at 82.55 49.53 0) (effects (font (size 1.27 1.27)) (justify left)))
-  (property "Footprint" "Capacitor_SMD:C_0402_1005Metric" (at 80.01 48.26 0) (effects (font (size 1.27 1.27))) (hide yes))
-  (property "Datasheet" "https://www.murata.com/en-us/products/productdetail?partno=GRM155R71C104KA88D" (at 80.01 48.26 0) (effects (font (size 1.27 1.27))) (hide yes))
-  (property "Description" "Capacitor, 100 nF, 16 V, X7R, 0402" (at 80.01 48.26 0) (effects (font (size 1.27 1.27))) (hide yes))
+  (property "Footprint" "Capacitor_SMD:C_0201_0603Metric" (at 80.01 48.26 0) (effects (font (size 1.27 1.27))) (hide yes))
+  (property "Datasheet" "https://www.murata.com/en-us/products/productdetail?partno=GRM033R61A104KE15D" (at 80.01 48.26 0) (effects (font (size 1.27 1.27))) (hide yes))
+  (property "Description" "Capacitor, 100 nF, 10 V, X5R, 0201" (at 80.01 48.26 0) (effects (font (size 1.27 1.27))) (hide yes))
   (property "Manufacturer" "Murata" (at 80.01 48.26 0) (effects (font (size 1.27 1.27))) (hide yes))
-  (property "MPN" "GRM155R71C104KA88D" (at 80.01 48.26 0) (effects (font (size 1.27 1.27))) (hide yes))
+  (property "MPN" "GRM033R61A104KE15D" (at 80.01 48.26 0) (effects (font (size 1.27 1.27))) (hide yes))
   (property "Block" "blk.board-id" (at 80.01 48.26 0) (effects (font (size 1.27 1.27))) (hide yes))
   (pin "1")

Commit message: Board on libs v0.2.0: lower-case kebab vendor keys (HL-13)
The libs submodule moves to v0.2.0 (5f24483). Every library nickname in
the generator, the placement tool and the floorplan study follows the
key table (Texas_Instruments -> texas-instruments, OpenDAP_Device ->
opendap-generic, Rockchip and Rockchip_PMIC -> rockchip, ...); the
library tables are written from the files. Schematic and board
regenerated.

Checks: ERC 0 errors (warnings unchanged); DRC 0 errors, 605 warnings,
the same counts by type, schematic parity 0; every placement identical;
craft Q1 met; pcb tests pass; STEP export resolves every libs 3D model
(the 27 parts without a model are KiCad stock lands that have none).

Co-Authored-By: Claude Opus 5.5 <noreply@anthropic.com>
Claude-Session: https://claude.ai/code/session_01Ei262h3TpgY9vyfNLMi5Mn
Parts:
- U5601: footprint Microchip:Microchip_5TS1_SOT-23-5_1.6x2.9mm_P0.95mm -> microchip:Microchip_5TS1_SOT-23-5_1.6x2.9mm_P0.95mm; symbol Microchip:AT24C02D-STUM-T -> microchip:AT24C02D-STUM-T
Changed lines of the file:
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@@
 (paper "A4")
 (title_block (title "Board EEPROM") (date "2026-10-25") (rev "A") (company "The OpenDAP Project") (comment 1 "blk.board-id") (comment 2 "AT24C02D board identity EEPROM on I2C2 at 0x50"))
-(symbol (lib_id "Microchip:AT24C02D-STUM-T") (at 45.72 63.5 0) (unit 1) (body_style 1) (exclude_from_sim no) (in_bom yes) (on_board yes) (dnp no)
+(symbol (lib_id "microchip:AT24C02D-STUM-T") (at 45.72 63.5 0) (unit 1) (body_style 1) (exclude_from_sim no) (in_bom yes) (on_board yes) (dnp no)
   (property "Reference" "U5601" (at 52.07 50.8 0) (effects (font (size 1.27 1.27)) (justify left)))
   (property "Value" "AT24C02D-STUM-T" (at 52.07 48.26 0) (effects (font (size 1.27 1.27)) (justify left)))
-  (property "Footprint" "Microchip:Microchip_5TS1_SOT-23-5_1.6x2.9mm_P0.95mm" (at 45.72 63.5 0) (effects (font (size 1.27 1.27))) (hide yes))
+  (property "Footprint" "microchip:Microchip_5TS1_SOT-23-5_1.6x2.9mm_P0.95mm" (at 45.72 63.5 0) (effects (font (size 1.27 1.27))) (hide yes))
   (property "Datasheet" "https://ww1.microchip.com/downloads/aemDocuments/documents/MPD/ProductDocuments/DataSheets/AT24C01D-AT24C02D-I2C-Compatible-Two-Wire-Serial-EEPROM-1-Kbit-2-Kbit-DS20006064.pdf" (at 45.72 63.5 0) (effects (font (size 1.27 1.27))) (hide yes))
   (property "Description" "Serial EEPROM, 2 kbit (256 x 8), I2C 1 MHz at 2.5-3.6 V / 400 kHz at 1.7-3.6 V, 8-byte page, write protect, fixed address 0x50, 5-lead SOT23 (5TS1)" (at 45.72 63.5 0) (effects (font (size 1.27 1.27))) (hide yes))
