File: board/hardware/t1-main-board/speaker.kicad_sch (KiCad schematic)
At the start: 10 parts, among them U6101 MAX98357AETE

Commit message: Board: capture blk.current-monitors
Five INA236 on I2C1 (0x40-0x43, 0x48) with their shunts, per power tree
§4.12 and BOM v1 lines 54 and 136. The measured branches are rails of
their own (VSYS_SRC, VSYS_LV_AUDIO, VSYS_AUDIO, VSYS_LV_BL, VSYS_P5V1),
fed through the shunts on this sheet; the charger, audio, backlight and
5.1 V sheets take them. The root's layout may leave a stack level empty,
so the block sits under the notes; IC bboxes hold turned rail values;
passive rows hold a bottom rail's text.

Co-Authored-By: Claude Opus 5.5 <noreply@anthropic.com>
Claude-Session: https://claude.ai/code/session_01Ei262h3TpgY9vyfNLMi5Mn
Parts:
- removed C6101: 10 µF, Capacitor_SMD:C_0603_1608Metric, symbol Device:C
- removed C6102: 100 nF, Capacitor_SMD:C_0402_1005Metric, symbol Device:C
- removed R6101: 100 kΩ, Resistor_SMD:R_0402_1005Metric, symbol Device:R
- removed R6102: 100 mΩ, Resistor_SMD:R_0603_1608Metric, symbol Device:R
- removed R6103: 0 Ω, Resistor_SMD:R_0402_1005Metric, symbol Device:R
- removed TP6101: VSYS_LV, TestPoint:TestPoint_Pad_D1.0mm, symbol Connector:TestPoint
- removed TP6102: SPK_VDD, TestPoint:TestPoint_Pad_D1.0mm, symbol Connector:TestPoint
- removed TP6103: SPK_P, TestPoint:TestPoint_Pad_D1.0mm, symbol Connector:TestPoint
- removed TP6104: SPK_N, TestPoint:TestPoint_Pad_D1.0mm, symbol Connector:TestPoint
- removed U6101: MAX98357AETE, Analog_Devices:Maxim_T1633-4_TQFN-16-1EP_3x3mm_P0.5mm_EP1.1x1.1mm, symbol Analog_Devices:MAX98357AETE
- added C6201: 10 µF, Capacitor_SMD:C_0603_1608Metric, symbol Device:C
- added C6202: 100 nF, Capacitor_SMD:C_0402_1005Metric, symbol Device:C
- added R6201: 100 kΩ, Resistor_SMD:R_0402_1005Metric, symbol Device:R
- added R6202: 100 mΩ, Resistor_SMD:R_0603_1608Metric, symbol Device:R
- added R6203: 0 Ω, Resistor_SMD:R_0402_1005Metric, symbol Device:R
- added TP6201: VSYS_LV, TestPoint:TestPoint_Pad_D1.0mm, symbol Connector:TestPoint
- added TP6202: SPK_VDD, TestPoint:TestPoint_Pad_D1.0mm, symbol Connector:TestPoint
- added TP6203: SPK_P, TestPoint:TestPoint_Pad_D1.0mm, symbol Connector:TestPoint
- added TP6204: SPK_N, TestPoint:TestPoint_Pad_D1.0mm, symbol Connector:TestPoint
- added U6201: MAX98357AETE, Analog_Devices:Maxim_T1633-4_TQFN-16-1EP_3x3mm_P0.5mm_EP1.1x1.1mm, symbol Analog_Devices:MAX98357AETE
Connections:
- net GND: now also C6201.2, C6202.2, U6201.11 (GND), U6201.15 (GND), U6201.3 (GND), U6201.EP
- net SPK_BCLK: now also U6201.16 (BCLK)
- net SPK_GAIN: now also R6201.2, U6201.2 (GAIN_SLOT)
- net SPK_LRCK: now also U6201.14 (LRCLK)
- net SPK_N: now also TP6204.1, U6201.10 (OUTN)
- net SPK_P: now also TP6203.1, U6201.9 (OUTP)
- net SPK_SD: now also R6203.2, U6201.4 (SD_MODE)
- net SPK_SDIN: now also U6201.1 (DIN)
- net SPK_SD_MODE: now also R6203.1
- net SPK_VDD: now also C6201.1, C6202.1, R6201.1, R6202.2, TP6202.1, U6201.7 (VDD), U6201.8 (VDD)
- net VSYS_LV: now also R6202.1, TP6201.1

Commit message: Board: capture blk.status-led
LP5521 at 0x32 on I2C2 (BOM v1 line 105) with its charge-pump
capacitors, EN on vcca1v8_pmu, VDD from VSYS_LV through link #22;
LED_R/G/B reach the faceplate connector as the LED bus alias. The
faceplate row of the root is re-packed so five full columns sit left of
the title block.

Co-Authored-By: Claude Opus 5.5 <noreply@anthropic.com>
Claude-Session: https://claude.ai/code/session_01Ei262h3TpgY9vyfNLMi5Mn
Parts:
- removed C6201: 10 µF, Capacitor_SMD:C_0603_1608Metric, symbol Device:C
- removed C6202: 100 nF, Capacitor_SMD:C_0402_1005Metric, symbol Device:C
- removed R6201: 100 kΩ, Resistor_SMD:R_0402_1005Metric, symbol Device:R
- removed R6202: 100 mΩ, Resistor_SMD:R_0603_1608Metric, symbol Device:R
- removed R6203: 0 Ω, Resistor_SMD:R_0402_1005Metric, symbol Device:R
- removed TP6201: VSYS_LV, TestPoint:TestPoint_Pad_D1.0mm, symbol Connector:TestPoint
- removed TP6202: SPK_VDD, TestPoint:TestPoint_Pad_D1.0mm, symbol Connector:TestPoint
- removed TP6203: SPK_P, TestPoint:TestPoint_Pad_D1.0mm, symbol Connector:TestPoint
- removed TP6204: SPK_N, TestPoint:TestPoint_Pad_D1.0mm, symbol Connector:TestPoint
- removed U6201: MAX98357AETE, Analog_Devices:Maxim_T1633-4_TQFN-16-1EP_3x3mm_P0.5mm_EP1.1x1.1mm, symbol Analog_Devices:MAX98357AETE
- added C5201: 10 µF, Capacitor_SMD:C_0603_1608Metric, symbol Device:C
- added C5202: 100 nF, Capacitor_SMD:C_0402_1005Metric, symbol Device:C
- added R5201: 100 kΩ, Resistor_SMD:R_0402_1005Metric, symbol Device:R
- added R5202: 100 mΩ, Resistor_SMD:R_0603_1608Metric, symbol Device:R
- added R5203: 0 Ω, Resistor_SMD:R_0402_1005Metric, symbol Device:R
- added TP5201: VSYS_LV, TestPoint:TestPoint_Pad_D1.0mm, symbol Connector:TestPoint
- added TP5202: SPK_VDD, TestPoint:TestPoint_Pad_D1.0mm, symbol Connector:TestPoint
- added TP5203: SPK_P, TestPoint:TestPoint_Pad_D1.0mm, symbol Connector:TestPoint
- added TP5204: SPK_N, TestPoint:TestPoint_Pad_D1.0mm, symbol Connector:TestPoint
- added U5201: MAX98357AETE, Analog_Devices:Maxim_T1633-4_TQFN-16-1EP_3x3mm_P0.5mm_EP1.1x1.1mm, symbol Analog_Devices:MAX98357AETE
Connections:
- net GND: now also C5201.2, C5202.2, U5201.11 (GND), U5201.15 (GND), U5201.3 (GND), U5201.EP
- net SPK_BCLK: now also U5201.16 (BCLK)
- net SPK_GAIN: now also R5201.2, U5201.2 (GAIN_SLOT)
- net SPK_LRCK: now also U5201.14 (LRCLK)
- net SPK_N: now also TP5204.1, U5201.10 (OUTN)
- net SPK_P: now also TP5203.1, U5201.9 (OUTP)
- net SPK_SD: now also R5203.2, U5201.4 (SD_MODE)
- net SPK_SDIN: now also U5201.1 (DIN)
- net SPK_SD_MODE: now also R5203.1
- net SPK_VDD: now also C5201.1, C5202.1, R5201.1, R5202.2, TP5202.1, U5201.7 (VDD), U5201.8 (VDD)
- net VSYS_LV: now also R5202.1, TP5201.1

Commit message: Board: capture blk.debug
Debug UART2 (1.8 V) and I2S/DSD pads with ground pads, reset, PMIC and
power-key pads (PCB-T-09), a pad on every spare SoC GPIO whose pinout v1
row names one (the DEBUG bus, on the SoC's right edge), and a rail pad
for each power-tree rail no other sheet probes (PCB-T-02). Each DAC
sheet carries a pad on its MCLK. The spares pinout v1 leaves without a
pad now carry no-connect flags. On the root, facing sheet pins are
joined directly only where the route meets no other symbol.

Co-Authored-By: Claude Opus 5.5 <noreply@anthropic.com>
Claude-Session: https://claude.ai/code/session_01Ei262h3TpgY9vyfNLMi5Mn
Parts:
- removed C5201: 10 µF, Capacitor_SMD:C_0603_1608Metric, symbol Device:C
- removed C5202: 100 nF, Capacitor_SMD:C_0402_1005Metric, symbol Device:C
- removed R5201: 100 kΩ, Resistor_SMD:R_0402_1005Metric, symbol Device:R
- removed R5202: 100 mΩ, Resistor_SMD:R_0603_1608Metric, symbol Device:R
- removed R5203: 0 Ω, Resistor_SMD:R_0402_1005Metric, symbol Device:R
- removed TP5201: VSYS_LV, TestPoint:TestPoint_Pad_D1.0mm, symbol Connector:TestPoint
- removed TP5202: SPK_VDD, TestPoint:TestPoint_Pad_D1.0mm, symbol Connector:TestPoint
- removed TP5203: SPK_P, TestPoint:TestPoint_Pad_D1.0mm, symbol Connector:TestPoint
- removed TP5204: SPK_N, TestPoint:TestPoint_Pad_D1.0mm, symbol Connector:TestPoint
- removed U5201: MAX98357AETE, Analog_Devices:Maxim_T1633-4_TQFN-16-1EP_3x3mm_P0.5mm_EP1.1x1.1mm, symbol Analog_Devices:MAX98357AETE
- added C5301: 10 µF, Capacitor_SMD:C_0603_1608Metric, symbol Device:C
- added C5302: 100 nF, Capacitor_SMD:C_0402_1005Metric, symbol Device:C
- added R5301: 100 kΩ, Resistor_SMD:R_0402_1005Metric, symbol Device:R
- added R5302: 100 mΩ, Resistor_SMD:R_0603_1608Metric, symbol Device:R
- added R5303: 0 Ω, Resistor_SMD:R_0402_1005Metric, symbol Device:R
- added TP5301: VSYS_LV, TestPoint:TestPoint_Pad_D1.0mm, symbol Connector:TestPoint
- added TP5302: SPK_VDD, TestPoint:TestPoint_Pad_D1.0mm, symbol Connector:TestPoint
- added TP5303: SPK_P, TestPoint:TestPoint_Pad_D1.0mm, symbol Connector:TestPoint
- added TP5304: SPK_N, TestPoint:TestPoint_Pad_D1.0mm, symbol Connector:TestPoint
- added U5301: MAX98357AETE, Analog_Devices:Maxim_T1633-4_TQFN-16-1EP_3x3mm_P0.5mm_EP1.1x1.1mm, symbol Analog_Devices:MAX98357AETE
Connections:
- net GND: now also C5301.2, C5302.2, U5301.11 (GND), U5301.15 (GND), U5301.3 (GND), U5301.EP
- net SPK_BCLK: now also U5301.16 (BCLK)
- net SPK_GAIN: now also R5301.2, U5301.2 (GAIN_SLOT)
- net SPK_LRCK: now also U5301.14 (LRCLK)
- net SPK_N: now also TP5304.1, U5301.10 (OUTN)
- net SPK_P: now also TP5303.1, U5301.9 (OUTP)
- net SPK_SD: now also R5303.2, U5301.4 (SD_MODE)
- net SPK_SDIN: now also U5301.1 (DIN)
- net SPK_SD_MODE: now also R5303.1
- net SPK_VDD: now also C5301.1, C5302.1, R5301.1, R5302.2, TP5302.1, U5301.7 (VDD), U5301.8 (VDD)
- net VSYS_LV: now also R5302.1, TP5301.1

Commit message: Board: capture blk.mic-ambient and links #34, #35
IM73D122 on PDM CLK1 and SDI1 (BOM v1 line 34, pinout v1 AK2 and 1P2),
LR to ground, 22 Ω clock series, VDD from MIC_1V8 through link #35.
Link #34 on blk.mic-main makes the faceplate branch the rail MIC_1V8_FP
for contact 40 (power tree §4.12, G10). kicad-lib moves to e46bda4 for
the IM73D122, TPS3808G01, SN74LVC1G58 and BAT54 parts.

Co-Authored-By: Claude Opus 5.5 <noreply@anthropic.com>
Claude-Session: https://claude.ai/code/session_01Ei262h3TpgY9vyfNLMi5Mn
Parts:
- removed C5301: 10 µF, Capacitor_SMD:C_0603_1608Metric, symbol Device:C
- removed C5302: 100 nF, Capacitor_SMD:C_0402_1005Metric, symbol Device:C
- removed R5301: 100 kΩ, Resistor_SMD:R_0402_1005Metric, symbol Device:R
- removed R5302: 100 mΩ, Resistor_SMD:R_0603_1608Metric, symbol Device:R
- removed R5303: 0 Ω, Resistor_SMD:R_0402_1005Metric, symbol Device:R
- removed TP5301: VSYS_LV, TestPoint:TestPoint_Pad_D1.0mm, symbol Connector:TestPoint
- removed TP5302: SPK_VDD, TestPoint:TestPoint_Pad_D1.0mm, symbol Connector:TestPoint
- removed TP5303: SPK_P, TestPoint:TestPoint_Pad_D1.0mm, symbol Connector:TestPoint
- removed TP5304: SPK_N, TestPoint:TestPoint_Pad_D1.0mm, symbol Connector:TestPoint
- removed U5301: MAX98357AETE, Analog_Devices:Maxim_T1633-4_TQFN-16-1EP_3x3mm_P0.5mm_EP1.1x1.1mm, symbol Analog_Devices:MAX98357AETE
- added C5401: 10 µF, Capacitor_SMD:C_0603_1608Metric, symbol Device:C
- added C5402: 100 nF, Capacitor_SMD:C_0402_1005Metric, symbol Device:C
- added R5401: 100 kΩ, Resistor_SMD:R_0402_1005Metric, symbol Device:R
- added R5402: 100 mΩ, Resistor_SMD:R_0603_1608Metric, symbol Device:R
- added R5403: 0 Ω, Resistor_SMD:R_0402_1005Metric, symbol Device:R
- added TP5401: VSYS_LV, TestPoint:TestPoint_Pad_D1.0mm, symbol Connector:TestPoint
- added TP5402: SPK_VDD, TestPoint:TestPoint_Pad_D1.0mm, symbol Connector:TestPoint
- added TP5403: SPK_P, TestPoint:TestPoint_Pad_D1.0mm, symbol Connector:TestPoint
- added TP5404: SPK_N, TestPoint:TestPoint_Pad_D1.0mm, symbol Connector:TestPoint
- added U5401: MAX98357AETE, Analog_Devices:Maxim_T1633-4_TQFN-16-1EP_3x3mm_P0.5mm_EP1.1x1.1mm, symbol Analog_Devices:MAX98357AETE
Connections:
- net GND: now also C5401.2, C5402.2, U5401.11 (GND), U5401.15 (GND), U5401.3 (GND), U5401.EP
- net SPK_BCLK: now also U5401.16 (BCLK)
- net SPK_GAIN: now also R5401.2, U5401.2 (GAIN_SLOT)
- net SPK_LRCK: now also U5401.14 (LRCLK)
- net SPK_N: now also TP5404.1, U5401.10 (OUTN)
- net SPK_P: now also TP5403.1, U5401.9 (OUTP)
- net SPK_SD: now also R5403.2, U5401.4 (SD_MODE)
- net SPK_SDIN: now also U5401.1 (DIN)
- net SPK_SD_MODE: now also R5403.1
- net SPK_VDD: now also C5401.1, C5402.1, R5401.1, R5402.2, TP5402.1, U5401.7 (VDD), U5401.8 (VDD)
- net VSYS_LV: now also R5402.1, TP5401.1

Commit message: Board: capture blk.maskrom
Power + Vol- at a cold power-on pull eMMC D0 low inside the TPS3808G01
boot window (BOM v1 lines 35, 78, 97, 98; sim/maskrom): SENSE 280k/100k,
CT 390 nF, WINDOW_N with its pad, SN74LVC1G57 and SN74LVC1G58 on
vcca1v8_pmu, BAT54 from PWRON_N, DMG1012T through 1 kΩ to EMMC_D0.
Every block in use now has its sheet; the README states the remaining
single-pin nets.

Co-Authored-By: Claude Opus 5.5 <noreply@anthropic.com>
Claude-Session: https://claude.ai/code/session_01Ei262h3TpgY9vyfNLMi5Mn
Parts:
- removed C5401: 10 µF, Capacitor_SMD:C_0603_1608Metric, symbol Device:C
- removed C5402: 100 nF, Capacitor_SMD:C_0402_1005Metric, symbol Device:C
- removed R5401: 100 kΩ, Resistor_SMD:R_0402_1005Metric, symbol Device:R
- removed R5402: 100 mΩ, Resistor_SMD:R_0603_1608Metric, symbol Device:R
- removed R5403: 0 Ω, Resistor_SMD:R_0402_1005Metric, symbol Device:R
- removed TP5401: VSYS_LV, TestPoint:TestPoint_Pad_D1.0mm, symbol Connector:TestPoint
- removed TP5402: SPK_VDD, TestPoint:TestPoint_Pad_D1.0mm, symbol Connector:TestPoint
- removed TP5403: SPK_P, TestPoint:TestPoint_Pad_D1.0mm, symbol Connector:TestPoint
- removed TP5404: SPK_N, TestPoint:TestPoint_Pad_D1.0mm, symbol Connector:TestPoint
- removed U5401: MAX98357AETE, Analog_Devices:Maxim_T1633-4_TQFN-16-1EP_3x3mm_P0.5mm_EP1.1x1.1mm, symbol Analog_Devices:MAX98357AETE
- added C5501: 10 µF, Capacitor_SMD:C_0603_1608Metric, symbol Device:C
- added C5502: 100 nF, Capacitor_SMD:C_0402_1005Metric, symbol Device:C
- added R5501: 100 kΩ, Resistor_SMD:R_0402_1005Metric, symbol Device:R
- added R5502: 100 mΩ, Resistor_SMD:R_0603_1608Metric, symbol Device:R
- added R5503: 0 Ω, Resistor_SMD:R_0402_1005Metric, symbol Device:R
- added TP5501: VSYS_LV, TestPoint:TestPoint_Pad_D1.0mm, symbol Connector:TestPoint
- added TP5502: SPK_VDD, TestPoint:TestPoint_Pad_D1.0mm, symbol Connector:TestPoint
- added TP5503: SPK_P, TestPoint:TestPoint_Pad_D1.0mm, symbol Connector:TestPoint
- added TP5504: SPK_N, TestPoint:TestPoint_Pad_D1.0mm, symbol Connector:TestPoint
- added U5501: MAX98357AETE, Analog_Devices:Maxim_T1633-4_TQFN-16-1EP_3x3mm_P0.5mm_EP1.1x1.1mm, symbol Analog_Devices:MAX98357AETE
Connections:
- net GND: now also C5501.2, C5502.2, U5501.11 (GND), U5501.15 (GND), U5501.3 (GND), U5501.EP
- net SPK_BCLK: now also U5501.16 (BCLK)
- net SPK_GAIN: now also R5501.2, U5501.2 (GAIN_SLOT)
- net SPK_LRCK: now also U5501.14 (LRCLK)
- net SPK_N: now also TP5504.1, U5501.10 (OUTN)
- net SPK_P: now also TP5503.1, U5501.9 (OUTP)
- net SPK_SD: now also R5503.2, U5501.4 (SD_MODE)
- net SPK_SDIN: now also U5501.1 (DIN)
- net SPK_SD_MODE: now also R5503.1
- net SPK_VDD: now also C5501.1, C5502.1, R5501.1, R5502.2, TP5502.1, U5501.7 (VDD), U5501.8 (VDD)
- net VSYS_LV: now also R5502.1, TP5501.1

Commit message: Board on libs v0.2.0: lower-case kebab vendor keys (HL-13)
The libs submodule moves to v0.2.0 (5f24483). Every library nickname in
the generator, the placement tool and the floorplan study follows the
key table (Texas_Instruments -> texas-instruments, OpenDAP_Device ->
opendap-generic, Rockchip and Rockchip_PMIC -> rockchip, ...); the
library tables are written from the files. Schematic and board
regenerated.

Checks: ERC 0 errors (warnings unchanged); DRC 0 errors, 605 warnings,
the same counts by type, schematic parity 0; every placement identical;
craft Q1 met; pcb tests pass; STEP export resolves every libs 3D model
(the 27 parts without a model are KiCad stock lands that have none).

Co-Authored-By: Claude Opus 5.5 <noreply@anthropic.com>
Claude-Session: https://claude.ai/code/session_01Ei262h3TpgY9vyfNLMi5Mn
Parts:
- U5501: footprint Analog_Devices:Maxim_T1633-4_TQFN-16-1EP_3x3mm_P0.5mm_EP1.1x1.1mm -> analog-devices:Maxim_T1633-4_TQFN-16-1EP_3x3mm_P0.5mm_EP1.1x1.1mm; symbol Analog_Devices:MAX98357AETE -> analog-devices:MAX98357AETE
Changed lines of the file:
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@@
 (paper "A4")
 (title_block (title "Speaker amplifier") (date "2026-10-25") (rev "A") (company "The OpenDAP Project") (comment 1 "blk.speaker") (comment 2 "MAX98357A on I2S3, SD_MODE shutdown, speaker spring-contact pads"))
-(symbol (lib_id "Analog_Devices:MAX98357AETE") (at 53.34 72.39 0) (unit 1) (body_style 1) (exclude_from_sim no) (in_bom yes) (on_board yes) (dnp no)
+(symbol (lib_id "analog-devices:MAX98357AETE") (at 53.34 72.39 0) (unit 1) (body_style 1) (exclude_from_sim no) (in_bom yes) (on_board yes) (dnp no)
   (property "Reference" "U5501" (at 57.15 50.8 0) (effects (font (size 1.27 1.27)) (justify left)))
   (property "Value" "MAX98357AETE" (at 57.15 48.26 0) (effects (font (size 1.27 1.27)) (justify left)))
-  (property "Footprint" "Analog_Devices:Maxim_T1633-4_TQFN-16-1EP_3x3mm_P0.5mm_EP1.1x1.1mm" (at 53.34 72.39 0) (effects (font (size 1.27 1.27))) (hide yes))
+  (property "Footprint" "analog-devices:Maxim_T1633-4_TQFN-16-1EP_3x3mm_P0.5mm_EP1.1x1.1mm" (at 53.34 72.39 0) (effects (font (size 1.27 1.27))) (hide yes))
   (property "Datasheet" "https://www.analog.com/media/en/technical-documentation/data-sheets/MAX98357A-MAX98357B.pdf" (at 53.34 72.39 0) (effects (font (size 1.27 1.27))) (hide yes))
   (property "Description" "Mono filterless Class D amplifier, PCM input (I2S, left-justified, 8-slot TDM), no MCLK, pin-selected gain, 2.5-5.5 V supply, 16-pin TQFN (T1633+4) 3 x 3 mm with exposed pad" (at 53.34 72.39 0) (effects (font (size 1.27 1.27))) (hide yes))

Commit message: Board in the 62.5 x 95.0 mm body: ADR 0025, outline 59.1 x 91.6, 0201 swaps
ADR 0025 supersedes ADR 0016 for t1 ADR 0006's body: board outline from
the body, 1.2 mm walls and 0.5 mm clearance; height zones and stack
restated unchanged; the speaker on a case shelf (PCB-Z-09); pocket
reliefs at the 4.4 mm jack, the microSD (DM3AT push-push kept) and the
side buttons; the audio 0603 -> 0402 swap gated by t1 V2-A08; reserve
(NFC reader, then TPM) recorded, not applied.

- pcb/geometry.py derives the outline from BODY, WALL and CLEARANCE;
  the pocket, display and fixed parts keep their device-frame positions;
  holes keep their edge distance; the speaker shadow becomes a 1.5 mm
  shelf height area (placement, checks, occupancy).
- build.py reports pocket reliefs and routing room; C904 unfixed (it
  now finds back room, so PCB-Z-04 carries no part).
- Generator: parts.area_swap puts 121 generic 0402 resistors (outside
  audio and VBUS paths, >= 10 ohm) and five 100 nF signal capacitors in
  0201 (BOM v1.16); schematic and board regenerated.
- Result: 1,012/1,012 placed, 98.8 % by the floorplan method (was 111 %),
  factor left 1.68 (was 1.49); DRC 0 errors, ERC 0 errors, 0 check
  findings, pcb tests 20/20, schematic craft Q1 met.
- Specs: PCB constraints v0.17 (M-01, M-02, M-08, Z-02, Z-06 to Z-09,
  R-07), placement v1.1 (section 3, decisions 4 and 13, checks, open
  items with the gated swaps and the reserve), floorplan v1 section 1,
  BOM v1.16.

Co-Authored-By: Claude Opus 5.5 <noreply@anthropic.com>
Claude-Session: https://claude.ai/code/session_01Ei262h3TpgY9vyfNLMi5Mn
Parts:
- R5501: footprint Resistor_SMD:R_0402_1005Metric -> Resistor_SMD:R_0201_0603Metric; MPN RC0402FR-07100KL -> RC0201FR-07100KL
Changed lines of the file:
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@@
   (property "Reference" "R5501" (at 114.3 52.07 0) (effects (font (size 1.27 1.27)) (justify left)))
   (property "Value" "100 kΩ" (at 114.3 54.61 0) (effects (font (size 1.27 1.27)) (justify left)))
-  (property "Footprint" "Resistor_SMD:R_0402_1005Metric" (at 113.03 53.34 0) (effects (font (size 1.27 1.27))) (hide yes))
-  (property "Datasheet" "https://yageogroup.com/en/ProductSearch/PartNumberSearch?part=RC0402FR-07100KL" (at 113.03 53.34 0) (effects (font (size 1.27 1.27))) (hide yes))
-  (property "Description" "Resistor, 100 kΩ, 1 %, 1/16 W, 0402" (at 113.03 53.34 0) (effects (font (size 1.27 1.27))) (hide yes))
+  (property "Footprint" "Resistor_SMD:R_0201_0603Metric" (at 113.03 53.34 0) (effects (font (size 1.27 1.27))) (hide yes))
+  (property "Datasheet" "https://yageogroup.com/en/ProductSearch/PartNumberSearch?part=RC0201FR-07100KL" (at 113.03 53.34 0) (effects (font (size 1.27 1.27))) (hide yes))
+  (property "Description" "Resistor, 100 kΩ, 1 %, 1/20 W, 0201" (at 113.03 53.34 0) (effects (font (size 1.27 1.27))) (hide yes))
   (property "Manufacturer" "YAGEO" (at 113.03 53.34 0) (effects (font (size 1.27 1.27))) (hide yes))
-  (property "MPN" "RC0402FR-07100KL" (at 113.03 53.34 0) (effects (font (size 1.27 1.27))) (hide yes))
+  (property "MPN" "RC0201FR-07100KL" (at 113.03 53.34 0) (effects (font (size 1.27 1.27))) (hide yes))
   (property "Block" "blk.speaker" (at 113.03 53.34 0) (effects (font (size 1.27 1.27))) (hide yes))
   (pin "1")
