File: board/hardware/t1-main-board/usb-c.kicad_sch (KiCad schematic)
At the start: 17 parts, among them J4201 USB4105-GF-A, U4201 TVS2200DRVR, U4202 TPD8S300ARUKR, U4203 TPD4E05U06DQAR, U4204 FUSB302BMPX

Commit message: Board: capture blk.current-monitors
Five INA236 on I2C1 (0x40-0x43, 0x48) with their shunts, per power tree
§4.12 and BOM v1 lines 54 and 136. The measured branches are rails of
their own (VSYS_SRC, VSYS_LV_AUDIO, VSYS_AUDIO, VSYS_LV_BL, VSYS_P5V1),
fed through the shunts on this sheet; the charger, audio, backlight and
5.1 V sheets take them. The root's layout may leave a stack level empty,
so the block sits under the notes; IC bboxes hold turned rail values;
passive rows hold a bottom rail's text.

Co-Authored-By: Claude Opus 5.5 <noreply@anthropic.com>
Claude-Session: https://claude.ai/code/session_01Ei262h3TpgY9vyfNLMi5Mn
Parts:
- removed C4201: 100 nF, Capacitor_SMD:C_0603_1608Metric, symbol Device:C
- removed C4202, C4203: 1 µF, Capacitor_SMD:C_0402_1005Metric, symbol Device:C
- removed C4204: 100 nF, Capacitor_SMD:C_0402_1005Metric, symbol Device:C
- removed J4201: USB4105-GF-A, GCT:GCT_USB4105-GF-A_USB-C_Receptacle_USB2.0_Horizontal, symbol GCT:USB4105-GF-A
- removed R4201, R4204: 10 kΩ, Resistor_SMD:R_0402_1005Metric, symbol Device:R
- removed R4202, R4203: 2.2 Ω, Resistor_SMD:R_0402_1005Metric, symbol Device:R
- removed R4205: 15 kΩ, Resistor_SMD:R_0402_1005Metric, symbol Device:R
- removed TP4201: USBC_SBU1, TestPoint:TestPoint_Pad_D1.0mm, symbol Connector:TestPoint
- removed TP4202: USBC_SBU2, TestPoint:TestPoint_Pad_D1.0mm, symbol Connector:TestPoint
- removed TP4203: USBC_PROT_FLT_N, TestPoint:TestPoint_Pad_D1.0mm, symbol Connector:TestPoint
- removed U4201: TVS2200DRVR, Texas_Instruments:Texas_DRV0006A_WSON-6-1EP_2x2mm_P0.65mm_EP1x1.6mm, symbol Texas_Instruments:TVS2200DRVR
- removed U4202: TPD8S300ARUKR, Texas_Instruments:Texas_RUK0020B_WQFN-20-1EP_3x3mm_P0.4mm_EP1.7x1.7mm, symbol Texas_Instruments:TPD8S300ARUKR
- removed U4203: TPD4E05U06DQAR, Texas_Instruments:Texas_DQA0010A_USON-10_1x2.5mm_P0.5mm, symbol Texas_Instruments:TPD4E05U06DQAR
- removed U4204: FUSB302BMPX, onsemi:onsemi_510BR_WQFN-14-1EP_2.5x2.5mm_P0.5mm_EP1.45x1.45mm, symbol onsemi:FUSB302BMPX
- added C4301: 100 nF, Capacitor_SMD:C_0603_1608Metric, symbol Device:C
- added C4302, C4303: 1 µF, Capacitor_SMD:C_0402_1005Metric, symbol Device:C
- added C4304: 100 nF, Capacitor_SMD:C_0402_1005Metric, symbol Device:C
- added J4301: USB4105-GF-A, GCT:GCT_USB4105-GF-A_USB-C_Receptacle_USB2.0_Horizontal, symbol GCT:USB4105-GF-A
- added R4301, R4304: 10 kΩ, Resistor_SMD:R_0402_1005Metric, symbol Device:R
- added R4302, R4303: 2.2 Ω, Resistor_SMD:R_0402_1005Metric, symbol Device:R
- added R4305: 15 kΩ, Resistor_SMD:R_0402_1005Metric, symbol Device:R
- added TP4301: USBC_SBU1, TestPoint:TestPoint_Pad_D1.0mm, symbol Connector:TestPoint
- added TP4302: USBC_SBU2, TestPoint:TestPoint_Pad_D1.0mm, symbol Connector:TestPoint
- added TP4303: USBC_PROT_FLT_N, TestPoint:TestPoint_Pad_D1.0mm, symbol Connector:TestPoint
- added U4301: TVS2200DRVR, Texas_Instruments:Texas_DRV0006A_WSON-6-1EP_2x2mm_P0.65mm_EP1x1.6mm, symbol Texas_Instruments:TVS2200DRVR
- added U4302: TPD8S300ARUKR, Texas_Instruments:Texas_RUK0020B_WQFN-20-1EP_3x3mm_P0.4mm_EP1.7x1.7mm, symbol Texas_Instruments:TPD8S300ARUKR
- added U4303: TPD4E05U06DQAR, Texas_Instruments:Texas_DQA0010A_USON-10_1x2.5mm_P0.5mm, symbol Texas_Instruments:TPD4E05U06DQAR
- added U4304: FUSB302BMPX, onsemi:onsemi_510BR_WQFN-14-1EP_2.5x2.5mm_P0.5mm_EP1.45x1.45mm, symbol onsemi:FUSB302BMPX
Connections:
- net GND: now also C4301.2, C4302.2, C4303.2, C4304.2, J4301.A1 (GND), J4301.A12 (GND), J4301.B1 (GND), J4301.B12 (GND), J4301.S1 (GND), R4305.2, U4301.1 (GND), U4301.2 (GND), U4301.3 (GND), U4301.7 (GND), U4302.13 (GND), U4302.16 (D4), U4302.17 (D3), U4302.18 (GND), U4302.19 (D2), U4302.20 (D1), U4302.21 (GND), U4302.8 (GND), U4303.3 (GND), U4303.8 (GND), U4304.15 (GND), U4304.8 (GND), U4304.9 (GND)
- net I2C1_SCL: now also U4304.6 (SCL)
- net I2C1_SDA: now also U4304.7 (SDA)
- net USBC_CC1: now also U4302.12 (CC1), U4304.10 (CC1), U4304.11 (CC1)
- net USBC_CC2: now also U4302.11 (CC2), U4304.1 (CC2), U4304.14 (CC2)
- net USBC_C_CC1: now also J4301.A5 (CC1), U4302.4 (C_CC1), U4302.7 (RPD_G1)
- net USBC_C_CC2: now also J4301.B5 (CC2), U4302.5 (C_CC2), U4302.6 (RPD_G2)
- net USBC_C_SBU1: now also J4301.A8 (SBU1), U4302.1 (C_SBU1)
- net USBC_C_SBU2: now also J4301.B8 (SBU2), U4302.2 (C_SBU2)
- net USBC_DM: now also R4303.2
- net USBC_DM_C: now also J4301.A7 (Dn1), J4301.B7 (Dn2), R4303.1, U4303.2 (D1-)
- net USBC_DP: now also R4302.2
- net USBC_DP_C: now also J4301.A6 (Dp1), J4301.B6 (Dp2), R4302.1, U4303.1 (D1+)
- net USBC_INT_N: now also U4304.5 (INT_N)
- net USBC_PROT_FLT_N: now also R4301.2, TP4303.1, U4302.9 (FLT)
- net USBC_SBU1: now also TP4301.1, U4302.15 (SBU1)
- net USBC_SBU2: now also TP4302.1, U4302.14 (SBU2)
- net USBC_VBIAS: now also C4301.1, U4302.3 (VBIAS)
- net USBC_VBUS: now also J4301.A4 (VBUS), J4301.A9 (VBUS), J4301.B4 (VBUS), J4301.B9 (VBUS), R4304.1, U4301.4 (IN), U4301.5 (IN), U4301.6 (IN), U4304.2 (VBUS)
- net USBC_VBUSDET: now also R4304.2, R4305.1
- net vcc3v3_pmu: now also C4302.1, C4303.1, C4304.1, R4301.1, U4302.10 (VPWR), U4304.3 (VDD), U4304.4 (VDD)

Commit message: Board: capture blk.debug
Debug UART2 (1.8 V) and I2S/DSD pads with ground pads, reset, PMIC and
power-key pads (PCB-T-09), a pad on every spare SoC GPIO whose pinout v1
row names one (the DEBUG bus, on the SoC's right edge), and a rail pad
for each power-tree rail no other sheet probes (PCB-T-02). Each DAC
sheet carries a pad on its MCLK. The spares pinout v1 leaves without a
pad now carry no-connect flags. On the root, facing sheet pins are
joined directly only where the route meets no other symbol.

Co-Authored-By: Claude Opus 5.5 <noreply@anthropic.com>
Claude-Session: https://claude.ai/code/session_01Ei262h3TpgY9vyfNLMi5Mn
Parts:
- removed C4301: 100 nF, Capacitor_SMD:C_0603_1608Metric, symbol Device:C
- removed C4302, C4303: 1 µF, Capacitor_SMD:C_0402_1005Metric, symbol Device:C
- removed C4304: 100 nF, Capacitor_SMD:C_0402_1005Metric, symbol Device:C
- removed J4301: USB4105-GF-A, GCT:GCT_USB4105-GF-A_USB-C_Receptacle_USB2.0_Horizontal, symbol GCT:USB4105-GF-A
- removed R4301, R4304: 10 kΩ, Resistor_SMD:R_0402_1005Metric, symbol Device:R
- removed R4302, R4303: 2.2 Ω, Resistor_SMD:R_0402_1005Metric, symbol Device:R
- removed R4305: 15 kΩ, Resistor_SMD:R_0402_1005Metric, symbol Device:R
- removed TP4301: USBC_SBU1, TestPoint:TestPoint_Pad_D1.0mm, symbol Connector:TestPoint
- removed TP4302: USBC_SBU2, TestPoint:TestPoint_Pad_D1.0mm, symbol Connector:TestPoint
- removed TP4303: USBC_PROT_FLT_N, TestPoint:TestPoint_Pad_D1.0mm, symbol Connector:TestPoint
- removed U4301: TVS2200DRVR, Texas_Instruments:Texas_DRV0006A_WSON-6-1EP_2x2mm_P0.65mm_EP1x1.6mm, symbol Texas_Instruments:TVS2200DRVR
- removed U4302: TPD8S300ARUKR, Texas_Instruments:Texas_RUK0020B_WQFN-20-1EP_3x3mm_P0.4mm_EP1.7x1.7mm, symbol Texas_Instruments:TPD8S300ARUKR
- removed U4303: TPD4E05U06DQAR, Texas_Instruments:Texas_DQA0010A_USON-10_1x2.5mm_P0.5mm, symbol Texas_Instruments:TPD4E05U06DQAR
- removed U4304: FUSB302BMPX, onsemi:onsemi_510BR_WQFN-14-1EP_2.5x2.5mm_P0.5mm_EP1.45x1.45mm, symbol onsemi:FUSB302BMPX
- added C4401: 100 nF, Capacitor_SMD:C_0603_1608Metric, symbol Device:C
- added C4402, C4403: 1 µF, Capacitor_SMD:C_0402_1005Metric, symbol Device:C
- added C4404: 100 nF, Capacitor_SMD:C_0402_1005Metric, symbol Device:C
- added J4401: USB4105-GF-A, GCT:GCT_USB4105-GF-A_USB-C_Receptacle_USB2.0_Horizontal, symbol GCT:USB4105-GF-A
- added R4401, R4404: 10 kΩ, Resistor_SMD:R_0402_1005Metric, symbol Device:R
- added R4402, R4403: 2.2 Ω, Resistor_SMD:R_0402_1005Metric, symbol Device:R
- added R4405: 15 kΩ, Resistor_SMD:R_0402_1005Metric, symbol Device:R
- added TP4401: USBC_SBU1, TestPoint:TestPoint_Pad_D1.0mm, symbol Connector:TestPoint
- added TP4402: USBC_SBU2, TestPoint:TestPoint_Pad_D1.0mm, symbol Connector:TestPoint
- added TP4403: USBC_PROT_FLT_N, TestPoint:TestPoint_Pad_D1.0mm, symbol Connector:TestPoint
- added U4401: TVS2200DRVR, Texas_Instruments:Texas_DRV0006A_WSON-6-1EP_2x2mm_P0.65mm_EP1x1.6mm, symbol Texas_Instruments:TVS2200DRVR
- added U4402: TPD8S300ARUKR, Texas_Instruments:Texas_RUK0020B_WQFN-20-1EP_3x3mm_P0.4mm_EP1.7x1.7mm, symbol Texas_Instruments:TPD8S300ARUKR
- added U4403: TPD4E05U06DQAR, Texas_Instruments:Texas_DQA0010A_USON-10_1x2.5mm_P0.5mm, symbol Texas_Instruments:TPD4E05U06DQAR
- added U4404: FUSB302BMPX, onsemi:onsemi_510BR_WQFN-14-1EP_2.5x2.5mm_P0.5mm_EP1.45x1.45mm, symbol onsemi:FUSB302BMPX
Connections:
- net GND: now also C4401.2, C4402.2, C4403.2, C4404.2, J4401.A1 (GND), J4401.A12 (GND), J4401.B1 (GND), J4401.B12 (GND), J4401.S1 (GND), R4405.2, U4401.1 (GND), U4401.2 (GND), U4401.3 (GND), U4401.7 (GND), U4402.13 (GND), U4402.16 (D4), U4402.17 (D3), U4402.18 (GND), U4402.19 (D2), U4402.20 (D1), U4402.21 (GND), U4402.8 (GND), U4403.3 (GND), U4403.8 (GND), U4404.15 (GND), U4404.8 (GND), U4404.9 (GND)
- net I2C1_SCL: now also U4404.6 (SCL)
- net I2C1_SDA: now also U4404.7 (SDA)
- net USBC_CC1: now also U4402.12 (CC1), U4404.10 (CC1), U4404.11 (CC1)
- net USBC_CC2: now also U4402.11 (CC2), U4404.1 (CC2), U4404.14 (CC2)
- net USBC_C_CC1: now also J4401.A5 (CC1), U4402.4 (C_CC1), U4402.7 (RPD_G1)
- net USBC_C_CC2: now also J4401.B5 (CC2), U4402.5 (C_CC2), U4402.6 (RPD_G2)
- net USBC_C_SBU1: now also J4401.A8 (SBU1), U4402.1 (C_SBU1)
- net USBC_C_SBU2: now also J4401.B8 (SBU2), U4402.2 (C_SBU2)
- net USBC_DM: now also R4403.2
- net USBC_DM_C: now also J4401.A7 (Dn1), J4401.B7 (Dn2), R4403.1, U4403.2 (D1-)
- net USBC_DP: now also R4402.2
- net USBC_DP_C: now also J4401.A6 (Dp1), J4401.B6 (Dp2), R4402.1, U4403.1 (D1+)
- net USBC_INT_N: now also U4404.5 (INT_N)
- net USBC_PROT_FLT_N: now also R4401.2, TP4403.1, U4402.9 (FLT)
- net USBC_SBU1: now also TP4401.1, U4402.15 (SBU1)
- net USBC_SBU2: now also TP4402.1, U4402.14 (SBU2)
- net USBC_VBIAS: now also C4401.1, U4402.3 (VBIAS)
- net USBC_VBUS: now also J4401.A4 (VBUS), J4401.A9 (VBUS), J4401.B4 (VBUS), J4401.B9 (VBUS), R4404.1, U4401.4 (IN), U4401.5 (IN), U4401.6 (IN), U4404.2 (VBUS)
- net USBC_VBUSDET: now also R4404.2, R4405.1
- net vcc3v3_pmu: now also C4402.1, C4403.1, C4404.1, R4401.1, U4402.10 (VPWR), U4404.3 (VDD), U4404.4 (VDD)

Commit message: Board: capture blk.mic-ambient and links #34, #35
IM73D122 on PDM CLK1 and SDI1 (BOM v1 line 34, pinout v1 AK2 and 1P2),
LR to ground, 22 Ω clock series, VDD from MIC_1V8 through link #35.
Link #34 on blk.mic-main makes the faceplate branch the rail MIC_1V8_FP
for contact 40 (power tree §4.12, G10). kicad-lib moves to e46bda4 for
the IM73D122, TPS3808G01, SN74LVC1G58 and BAT54 parts.

Co-Authored-By: Claude Opus 5.5 <noreply@anthropic.com>
Claude-Session: https://claude.ai/code/session_01Ei262h3TpgY9vyfNLMi5Mn
Parts:
- removed C4401: 100 nF, Capacitor_SMD:C_0603_1608Metric, symbol Device:C
- removed C4402, C4403: 1 µF, Capacitor_SMD:C_0402_1005Metric, symbol Device:C
- removed C4404: 100 nF, Capacitor_SMD:C_0402_1005Metric, symbol Device:C
- removed J4401: USB4105-GF-A, GCT:GCT_USB4105-GF-A_USB-C_Receptacle_USB2.0_Horizontal, symbol GCT:USB4105-GF-A
- removed R4401, R4404: 10 kΩ, Resistor_SMD:R_0402_1005Metric, symbol Device:R
- removed R4402, R4403: 2.2 Ω, Resistor_SMD:R_0402_1005Metric, symbol Device:R
- removed R4405: 15 kΩ, Resistor_SMD:R_0402_1005Metric, symbol Device:R
- removed TP4401: USBC_SBU1, TestPoint:TestPoint_Pad_D1.0mm, symbol Connector:TestPoint
- removed TP4402: USBC_SBU2, TestPoint:TestPoint_Pad_D1.0mm, symbol Connector:TestPoint
- removed TP4403: USBC_PROT_FLT_N, TestPoint:TestPoint_Pad_D1.0mm, symbol Connector:TestPoint
- removed U4401: TVS2200DRVR, Texas_Instruments:Texas_DRV0006A_WSON-6-1EP_2x2mm_P0.65mm_EP1x1.6mm, symbol Texas_Instruments:TVS2200DRVR
- removed U4402: TPD8S300ARUKR, Texas_Instruments:Texas_RUK0020B_WQFN-20-1EP_3x3mm_P0.4mm_EP1.7x1.7mm, symbol Texas_Instruments:TPD8S300ARUKR
- removed U4403: TPD4E05U06DQAR, Texas_Instruments:Texas_DQA0010A_USON-10_1x2.5mm_P0.5mm, symbol Texas_Instruments:TPD4E05U06DQAR
- removed U4404: FUSB302BMPX, onsemi:onsemi_510BR_WQFN-14-1EP_2.5x2.5mm_P0.5mm_EP1.45x1.45mm, symbol onsemi:FUSB302BMPX
- added C4501: 100 nF, Capacitor_SMD:C_0603_1608Metric, symbol Device:C
- added C4502, C4503: 1 µF, Capacitor_SMD:C_0402_1005Metric, symbol Device:C
- added C4504: 100 nF, Capacitor_SMD:C_0402_1005Metric, symbol Device:C
- added J4501: USB4105-GF-A, GCT:GCT_USB4105-GF-A_USB-C_Receptacle_USB2.0_Horizontal, symbol GCT:USB4105-GF-A
- added R4501, R4504: 10 kΩ, Resistor_SMD:R_0402_1005Metric, symbol Device:R
- added R4502, R4503: 2.2 Ω, Resistor_SMD:R_0402_1005Metric, symbol Device:R
- added R4505: 15 kΩ, Resistor_SMD:R_0402_1005Metric, symbol Device:R
- added TP4501: USBC_SBU1, TestPoint:TestPoint_Pad_D1.0mm, symbol Connector:TestPoint
- added TP4502: USBC_SBU2, TestPoint:TestPoint_Pad_D1.0mm, symbol Connector:TestPoint
- added TP4503: USBC_PROT_FLT_N, TestPoint:TestPoint_Pad_D1.0mm, symbol Connector:TestPoint
- added U4501: TVS2200DRVR, Texas_Instruments:Texas_DRV0006A_WSON-6-1EP_2x2mm_P0.65mm_EP1x1.6mm, symbol Texas_Instruments:TVS2200DRVR
- added U4502: TPD8S300ARUKR, Texas_Instruments:Texas_RUK0020B_WQFN-20-1EP_3x3mm_P0.4mm_EP1.7x1.7mm, symbol Texas_Instruments:TPD8S300ARUKR
- added U4503: TPD4E05U06DQAR, Texas_Instruments:Texas_DQA0010A_USON-10_1x2.5mm_P0.5mm, symbol Texas_Instruments:TPD4E05U06DQAR
- added U4504: FUSB302BMPX, onsemi:onsemi_510BR_WQFN-14-1EP_2.5x2.5mm_P0.5mm_EP1.45x1.45mm, symbol onsemi:FUSB302BMPX
Connections:
- net GND: now also C4501.2, C4502.2, C4503.2, C4504.2, J4501.A1 (GND), J4501.A12 (GND), J4501.B1 (GND), J4501.B12 (GND), J4501.S1 (GND), R4505.2, U4501.1 (GND), U4501.2 (GND), U4501.3 (GND), U4501.7 (GND), U4502.13 (GND), U4502.16 (D4), U4502.17 (D3), U4502.18 (GND), U4502.19 (D2), U4502.20 (D1), U4502.21 (GND), U4502.8 (GND), U4503.3 (GND), U4503.8 (GND), U4504.15 (GND), U4504.8 (GND), U4504.9 (GND)
- net I2C1_SCL: now also U4504.6 (SCL)
- net I2C1_SDA: now also U4504.7 (SDA)
- net USBC_CC1: now also U4502.12 (CC1), U4504.10 (CC1), U4504.11 (CC1)
- net USBC_CC2: now also U4502.11 (CC2), U4504.1 (CC2), U4504.14 (CC2)
- net USBC_C_CC1: now also J4501.A5 (CC1), U4502.4 (C_CC1), U4502.7 (RPD_G1)
- net USBC_C_CC2: now also J4501.B5 (CC2), U4502.5 (C_CC2), U4502.6 (RPD_G2)
- net USBC_C_SBU1: now also J4501.A8 (SBU1), U4502.1 (C_SBU1)
- net USBC_C_SBU2: now also J4501.B8 (SBU2), U4502.2 (C_SBU2)
- net USBC_DM: now also R4503.2
- net USBC_DM_C: now also J4501.A7 (Dn1), J4501.B7 (Dn2), R4503.1, U4503.2 (D1-)
- net USBC_DP: now also R4502.2
- net USBC_DP_C: now also J4501.A6 (Dp1), J4501.B6 (Dp2), R4502.1, U4503.1 (D1+)
- net USBC_INT_N: now also U4504.5 (INT_N)
- net USBC_PROT_FLT_N: now also R4501.2, TP4503.1, U4502.9 (FLT)
- net USBC_SBU1: now also TP4501.1, U4502.15 (SBU1)
- net USBC_SBU2: now also TP4502.1, U4502.14 (SBU2)
- net USBC_VBIAS: now also C4501.1, U4502.3 (VBIAS)
- net USBC_VBUS: now also J4501.A4 (VBUS), J4501.A9 (VBUS), J4501.B4 (VBUS), J4501.B9 (VBUS), R4504.1, U4501.4 (IN), U4501.5 (IN), U4501.6 (IN), U4504.2 (VBUS)
- net USBC_VBUSDET: now also R4504.2, R4505.1
- net vcc3v3_pmu: now also C4502.1, C4503.1, C4504.1, R4501.1, U4502.10 (VPWR), U4504.3 (VDD), U4504.4 (VDD)

Commit message: Board: capture blk.maskrom
Power + Vol- at a cold power-on pull eMMC D0 low inside the TPS3808G01
boot window (BOM v1 lines 35, 78, 97, 98; sim/maskrom): SENSE 280k/100k,
CT 390 nF, WINDOW_N with its pad, SN74LVC1G57 and SN74LVC1G58 on
vcca1v8_pmu, BAT54 from PWRON_N, DMG1012T through 1 kΩ to EMMC_D0.
Every block in use now has its sheet; the README states the remaining
single-pin nets.

Co-Authored-By: Claude Opus 5.5 <noreply@anthropic.com>
Claude-Session: https://claude.ai/code/session_01Ei262h3TpgY9vyfNLMi5Mn
Parts:
- removed C4501: 100 nF, Capacitor_SMD:C_0603_1608Metric, symbol Device:C
- removed C4502, C4503: 1 µF, Capacitor_SMD:C_0402_1005Metric, symbol Device:C
- removed C4504: 100 nF, Capacitor_SMD:C_0402_1005Metric, symbol Device:C
- removed J4501: USB4105-GF-A, GCT:GCT_USB4105-GF-A_USB-C_Receptacle_USB2.0_Horizontal, symbol GCT:USB4105-GF-A
- removed R4501, R4504: 10 kΩ, Resistor_SMD:R_0402_1005Metric, symbol Device:R
- removed R4502, R4503: 2.2 Ω, Resistor_SMD:R_0402_1005Metric, symbol Device:R
- removed R4505: 15 kΩ, Resistor_SMD:R_0402_1005Metric, symbol Device:R
- removed TP4501: USBC_SBU1, TestPoint:TestPoint_Pad_D1.0mm, symbol Connector:TestPoint
- removed TP4502: USBC_SBU2, TestPoint:TestPoint_Pad_D1.0mm, symbol Connector:TestPoint
- removed TP4503: USBC_PROT_FLT_N, TestPoint:TestPoint_Pad_D1.0mm, symbol Connector:TestPoint
- removed U4501: TVS2200DRVR, Texas_Instruments:Texas_DRV0006A_WSON-6-1EP_2x2mm_P0.65mm_EP1x1.6mm, symbol Texas_Instruments:TVS2200DRVR
- removed U4502: TPD8S300ARUKR, Texas_Instruments:Texas_RUK0020B_WQFN-20-1EP_3x3mm_P0.4mm_EP1.7x1.7mm, symbol Texas_Instruments:TPD8S300ARUKR
- removed U4503: TPD4E05U06DQAR, Texas_Instruments:Texas_DQA0010A_USON-10_1x2.5mm_P0.5mm, symbol Texas_Instruments:TPD4E05U06DQAR
- removed U4504: FUSB302BMPX, onsemi:onsemi_510BR_WQFN-14-1EP_2.5x2.5mm_P0.5mm_EP1.45x1.45mm, symbol onsemi:FUSB302BMPX
- added C4601: 100 nF, Capacitor_SMD:C_0603_1608Metric, symbol Device:C
- added C4602, C4603: 1 µF, Capacitor_SMD:C_0402_1005Metric, symbol Device:C
- added C4604: 100 nF, Capacitor_SMD:C_0402_1005Metric, symbol Device:C
- added J4601: USB4105-GF-A, GCT:GCT_USB4105-GF-A_USB-C_Receptacle_USB2.0_Horizontal, symbol GCT:USB4105-GF-A
- added R4601, R4604: 10 kΩ, Resistor_SMD:R_0402_1005Metric, symbol Device:R
- added R4602, R4603: 2.2 Ω, Resistor_SMD:R_0402_1005Metric, symbol Device:R
- added R4605: 15 kΩ, Resistor_SMD:R_0402_1005Metric, symbol Device:R
- added TP4601: USBC_SBU1, TestPoint:TestPoint_Pad_D1.0mm, symbol Connector:TestPoint
- added TP4602: USBC_SBU2, TestPoint:TestPoint_Pad_D1.0mm, symbol Connector:TestPoint
- added TP4603: USBC_PROT_FLT_N, TestPoint:TestPoint_Pad_D1.0mm, symbol Connector:TestPoint
- added U4601: TVS2200DRVR, Texas_Instruments:Texas_DRV0006A_WSON-6-1EP_2x2mm_P0.65mm_EP1x1.6mm, symbol Texas_Instruments:TVS2200DRVR
- added U4602: TPD8S300ARUKR, Texas_Instruments:Texas_RUK0020B_WQFN-20-1EP_3x3mm_P0.4mm_EP1.7x1.7mm, symbol Texas_Instruments:TPD8S300ARUKR
- added U4603: TPD4E05U06DQAR, Texas_Instruments:Texas_DQA0010A_USON-10_1x2.5mm_P0.5mm, symbol Texas_Instruments:TPD4E05U06DQAR
- added U4604: FUSB302BMPX, onsemi:onsemi_510BR_WQFN-14-1EP_2.5x2.5mm_P0.5mm_EP1.45x1.45mm, symbol onsemi:FUSB302BMPX
Connections:
- net GND: now also C4601.2, C4602.2, C4603.2, C4604.2, J4601.A1 (GND), J4601.A12 (GND), J4601.B1 (GND), J4601.B12 (GND), J4601.S1 (GND), R4605.2, U4601.1 (GND), U4601.2 (GND), U4601.3 (GND), U4601.7 (GND), U4602.13 (GND), U4602.16 (D4), U4602.17 (D3), U4602.18 (GND), U4602.19 (D2), U4602.20 (D1), U4602.21 (GND), U4602.8 (GND), U4603.3 (GND), U4603.8 (GND), U4604.15 (GND), U4604.8 (GND), U4604.9 (GND)
- net I2C1_SCL: now also U4604.6 (SCL)
- net I2C1_SDA: now also U4604.7 (SDA)
- net USBC_CC1: now also U4602.12 (CC1), U4604.10 (CC1), U4604.11 (CC1)
- net USBC_CC2: now also U4602.11 (CC2), U4604.1 (CC2), U4604.14 (CC2)
- net USBC_C_CC1: now also J4601.A5 (CC1), U4602.4 (C_CC1), U4602.7 (RPD_G1)
- net USBC_C_CC2: now also J4601.B5 (CC2), U4602.5 (C_CC2), U4602.6 (RPD_G2)
- net USBC_C_SBU1: now also J4601.A8 (SBU1), U4602.1 (C_SBU1)
- net USBC_C_SBU2: now also J4601.B8 (SBU2), U4602.2 (C_SBU2)
- net USBC_DM: now also R4603.2
- net USBC_DM_C: now also J4601.A7 (Dn1), J4601.B7 (Dn2), R4603.1, U4603.2 (D1-)
- net USBC_DP: now also R4602.2
- net USBC_DP_C: now also J4601.A6 (Dp1), J4601.B6 (Dp2), R4602.1, U4603.1 (D1+)
- net USBC_INT_N: now also U4604.5 (INT_N)
- net USBC_PROT_FLT_N: now also R4601.2, TP4603.1, U4602.9 (FLT)
- net USBC_SBU1: now also TP4601.1, U4602.15 (SBU1)
- net USBC_SBU2: now also TP4602.1, U4602.14 (SBU2)
- net USBC_VBIAS: now also C4601.1, U4602.3 (VBIAS)
- net USBC_VBUS: now also J4601.A4 (VBUS), J4601.A9 (VBUS), J4601.B4 (VBUS), J4601.B9 (VBUS), R4604.1, U4601.4 (IN), U4601.5 (IN), U4601.6 (IN), U4604.2 (VBUS)
- net USBC_VBUSDET: now also R4604.2, R4605.1
- net vcc3v3_pmu: now also C4602.1, C4603.1, C4604.1, R4601.1, U4602.10 (VPWR), U4604.3 (VDD), U4604.4 (VDD)
