File: board/hardware/t1-main-board/usb-c.kicad_sch (KiCad schematic)
At the start: 17 parts, among them J4601 USB4105-GF-A, U4601 TVS2200DRVR, U4602 TPD8S300ARUKR, U4603 TPD4E05U06DQAR, U4604 FUSB302BMPX

Commit message: Compaction: lower inductors, 0201 decoupling, 0.8 mm signal test pads
A matrix tool (hardware/studies/compaction) checks each candidate against
the design's stresses: same inductance, design peak <= 70 % and the
converter's maximum limit <= 100 % of Isat (30 % drop), height zones,
ratings at least twice the rail, PCB-D-06; sourcing outcome per part.

Applied (placement v1 decision 12, BOM v1.15):
- L601, L4401: XGL4015-102MEC (1.5 mm) for XAL/XGL4020-102MEC (2.1 mm);
- L1001, L5101: XGL4015-471MEC (1.5 mm) for Wurth 744373240047, on the
  stock XxL4020 land (the Wurth land was never drawn);
- L1201 is 1.2 mm (XGL4012, per-MPN heights): it moves next to the SoC;
- 58 x 100 nF decoupling on rails <= 3.3 V in core/IO/radio: 0201;
- 51 test pads on signal nets: 0.8 mm (PCB-D-06 v0.16, JLCPCB guide).
Kept: L901, L2802 (XGL4015 at 103 % of Isat at the limit); no thinner
0805/1206 capacitor passes (obsolete, NRND or unlisted).

Board need 113 % -> 111 % (core band 227 -> 203 %, power band 258 ->
233 %, radio band 19 -> 0 %); only C904 still relies on PCB-Z-04.
ERC 0 errors, craft Q1 met, DRC 0 errors (605 warnings), pcb and study
tests pass, rules test board PASS.

Co-Authored-By: Claude Opus 5.5 <noreply@anthropic.com>
Claude-Session: https://claude.ai/code/session_01Ei262h3TpgY9vyfNLMi5Mn
Parts:
- C4604: footprint Capacitor_SMD:C_0402_1005Metric -> Capacitor_SMD:C_0201_0603Metric; MPN GRM155R71C104KA88D -> GRM033R61A104KE15D
- TP4601, TP4602, TP4603: footprint TestPoint:TestPoint_Pad_D1.0mm -> T1_Main_Board:TestPoint_Pad_D0.8mm
Changed lines of the file:
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@@
   (property "Reference" "TP4601" (at 36.83 143.51 0) (effects (font (size 1.27 1.27)) (justify right)))
   (property "Value" "USBC_SBU1" (at 36.83 146.05 0) (effects (font (size 1.27 1.27)) (justify right)))
-  (property "Footprint" "TestPoint:TestPoint_Pad_D1.0mm" (at 38.1 148.59 0) (effects (font (size 1.27 1.27))) (hide yes))
+  (property "Footprint" "T1_Main_Board:TestPoint_Pad_D0.8mm" (at 38.1 148.59 0) (effects (font (size 1.27 1.27))) (hide yes))
   (property "Datasheet" "~" (at 38.1 148.59 0) (effects (font (size 1.27 1.27))) (hide yes))
-  (property "Description" "Test pad, 1.0 mm" (at 38.1 148.59 0) (effects (font (size 1.27 1.27))) (hide yes))
+  (property "Description" "Test pad, 0.8 mm, signal net" (at 38.1 148.59 0) (effects (font (size 1.27 1.27))) (hide yes))
   (property "Block" "blk.usb-c" (at 38.1 148.59 0) (effects (font (size 1.27 1.27))) (hide yes))
   (pin "1")
@@
   (property "Reference" "TP4602" (at 67.31 143.51 0) (effects (font (size 1.27 1.27)) (justify right)))
   (property "Value" "USBC_SBU2" (at 67.31 146.05 0) (effects (font (size 1.27 1.27)) (justify right)))
-  (property "Footprint" "TestPoint:TestPoint_Pad_D1.0mm" (at 68.58 148.59 0) (effects (font (size 1.27 1.27))) (hide yes))
+  (property "Footprint" "T1_Main_Board:TestPoint_Pad_D0.8mm" (at 68.58 148.59 0) (effects (font (size 1.27 1.27))) (hide yes))
   (property "Datasheet" "~" (at 68.58 148.59 0) (effects (font (size 1.27 1.27))) (hide yes))
-  (property "Description" "Test pad, 1.0 mm" (at 68.58 148.59 0) (effects (font (size 1.27 1.27))) (hide yes))
+  (property "Description" "Test pad, 0.8 mm, signal net" (at 68.58 148.59 0) (effects (font (size 1.27 1.27))) (hide yes))
   (property "Block" "blk.usb-c" (at 68.58 148.59 0) (effects (font (size 1.27 1.27))) (hide yes))
   (pin "1")
@@
   (property "Reference" "TP4603" (at 97.79 143.51 0) (effects (font (size 1.27 1.27)) (justify right)))
   (property "Value" "USBC_PROT_FLT_N" (at 97.79 146.05 0) (effects (font (size 1.27 1.27)) (justify right)))
-  (property "Footprint" "TestPoint:TestPoint_Pad_D1.0mm" (at 99.06 148.59 0) (effects (font (size 1.27 1.27))) (hide yes))
+  (property "Footprint" "T1_Main_Board:TestPoint_Pad_D0.8mm" (at 99.06 148.59 0) (effects (font (size 1.27 1.27))) (hide yes))
   (property "Datasheet" "~" (at 99.06 148.59 0) (effects (font (size 1.27 1.27))) (hide yes))
-  (property "Description" "Test pad, 1.0 mm" (at 99.06 148.59 0) (effects (font (size 1.27 1.27))) (hide yes))
+  (property "Description" "Test pad, 0.8 mm, signal net" (at 99.06 148.59 0) (effects (font (size 1.27 1.27))) (hide yes))
   (property "Block" "blk.usb-c" (at 99.06 148.59 0) (effects (font (size 1.27 1.27))) (hide yes))
   (pin "1")
@@
   (property "Reference" "C4604" (at 198.12 149.86 0) (effects (font (size 1.27 1.27)) (justify left)))
   (property "Value" "100 nF" (at 198.12 152.4 0) (effects (font (size 1.27 1.27)) (justify left)))
-  (property "Footprint" "Capacitor_SMD:C_0402_1005Metric" (at 195.58 151.13 0) (effects (font (size 1.27 1.27))) (hide yes))
-  (property "Datasheet" "https://www.murata.com/en-us/products/productdetail?partno=GRM155R71C104KA88D" (at 195.58 151.13 0) (effects (font (size 1.27 1.27))) (hide yes))
-  (property "Description" "Capacitor, 100 nF, 16 V, X7R, 0402" (at 195.58 151.13 0) (effects (font (size 1.27 1.27))) (hide yes))
+  (property "Footprint" "Capacitor_SMD:C_0201_0603Metric" (at 195.58 151.13 0) (effects (font (size 1.27 1.27))) (hide yes))
+  (property "Datasheet" "https://www.murata.com/en-us/products/productdetail?partno=GRM033R61A104KE15D" (at 195.58 151.13 0) (effects (font (size 1.27 1.27))) (hide yes))
+  (property "Description" "Capacitor, 100 nF, 10 V, X5R, 0201" (at 195.58 151.13 0) (effects (font (size 1.27 1.27))) (hide yes))
   (property "Manufacturer" "Murata" (at 195.58 151.13 0) (effects (font (size 1.27 1.27))) (hide yes))
-  (property "MPN" "GRM155R71C104KA88D" (at 195.58 151.13 0) (effects (font (size 1.27 1.27))) (hide yes))
+  (property "MPN" "GRM033R61A104KE15D" (at 195.58 151.13 0) (effects (font (size 1.27 1.27))) (hide yes))
   (property "Block" "blk.usb-c" (at 195.58 151.13 0) (effects (font (size 1.27 1.27))) (hide yes))
   (pin "1")

Commit message: Board on libs v0.2.0: lower-case kebab vendor keys (HL-13)
The libs submodule moves to v0.2.0 (5f24483). Every library nickname in
the generator, the placement tool and the floorplan study follows the
key table (Texas_Instruments -> texas-instruments, OpenDAP_Device ->
opendap-generic, Rockchip and Rockchip_PMIC -> rockchip, ...); the
library tables are written from the files. Schematic and board
regenerated.

Checks: ERC 0 errors (warnings unchanged); DRC 0 errors, 605 warnings,
the same counts by type, schematic parity 0; every placement identical;
craft Q1 met; pcb tests pass; STEP export resolves every libs 3D model
(the 27 parts without a model are KiCad stock lands that have none).

Co-Authored-By: Claude Opus 5.5 <noreply@anthropic.com>
Claude-Session: https://claude.ai/code/session_01Ei262h3TpgY9vyfNLMi5Mn
Parts:
- J4601: footprint GCT:GCT_USB4105-GF-A_USB-C_Receptacle_USB2.0_Horizontal -> gct:GCT_USB4105-GF-A_USB-C_Receptacle_USB2.0_Horizontal; symbol GCT:USB4105-GF-A -> gct:USB4105-GF-A
- U4601: footprint Texas_Instruments:Texas_DRV0006A_WSON-6-1EP_2x2mm_P0.65mm_EP1x1.6mm -> texas-instruments:Texas_DRV0006A_WSON-6-1EP_2x2mm_P0.65mm_EP1x1.6mm; symbol Texas_Instruments:TVS2200DRVR -> texas-instruments:TVS2200DRVR
- U4602: footprint Texas_Instruments:Texas_RUK0020B_WQFN-20-1EP_3x3mm_P0.4mm_EP1.7x1.7mm -> texas-instruments:Texas_RUK0020B_WQFN-20-1EP_3x3mm_P0.4mm_EP1.7x1.7mm; symbol Texas_Instruments:TPD8S300ARUKR -> texas-instruments:TPD8S300ARUKR
- U4603: footprint Texas_Instruments:Texas_DQA0010A_USON-10_1x2.5mm_P0.5mm -> texas-instruments:Texas_DQA0010A_USON-10_1x2.5mm_P0.5mm; symbol Texas_Instruments:TPD4E05U06DQAR -> texas-instruments:TPD4E05U06DQAR
Changed lines of the file:
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@@
 (paper "A3")
 (title_block (title "Main USB-C port") (date "2026-10-25") (rev "A") (company "The OpenDAP Project") (comment 1 "blk.usb-c") (comment 2 "USB4105 receptacle, VBUS TVS, CC/SBU protection, D± ESD and the FUSB302B port controller"))
-(symbol (lib_id "GCT:USB4105-GF-A") (at 57.15 86.36 0) (unit 1) (body_style 1) (exclude_from_sim no) (in_bom yes) (on_board yes) (dnp no)
+(symbol (lib_id "gct:USB4105-GF-A") (at 57.15 86.36 0) (unit 1) (body_style 1) (exclude_from_sim no) (in_bom yes) (on_board yes) (dnp no)
   (property "Reference" "J4601" (at 68.58 66.04 0) (effects (font (size 1.27 1.27)) (justify left)))
   (property "Value" "USB4105-GF-A" (at 68.58 63.5 0) (effects (font (size 1.27 1.27)) (justify left)))
-  (property "Footprint" "GCT:GCT_USB4105-GF-A_USB-C_Receptacle_USB2.0_Horizontal" (at 57.15 86.36 0) (effects (font (size 1.27 1.27))) (hide yes))
+  (property "Footprint" "gct:GCT_USB4105-GF-A_USB-C_Receptacle_USB2.0_Horizontal" (at 57.15 86.36 0) (effects (font (size 1.27 1.27))) (hide yes))
   (property "Datasheet" "https://gct.co/files/drawings/usb4105.pdf" (at 57.15 86.36 0) (effects (font (size 1.27 1.27))) (hide yes))
   (property "Description" "USB Type-C receptacle for USB 2.0, 16 contacts, SMT, PCB top mount, 4 shell stakes, 5 A VBUS" (at 57.15 86.36 0) (effects (font (size 1.27 1.27))) (hide yes))
@@
 (rectangle (start 22.86 35.56) (end 128.27 125.73) (stroke (width 0) (type dash)) (fill (type none)))
 (text "Receptacle: GCT USB4105-GF-A (BOM v1 line 61)" (exclude_from_sim no) (at 24.13 34.29 0) (effects (font (size 2.54 2.54)) (justify left bottom)))
-(symbol (lib_id "Texas_Instruments:TVS2200DRVR") (at 161.29 55.88 0) (unit 1) (body_style 1) (exclude_from_sim no) (in_bom yes) (on_board yes) (dnp no)
+(symbol (lib_id "texas-instruments:TVS2200DRVR") (at 161.29 55.88 0) (unit 1) (body_style 1) (exclude_from_sim no) (in_bom yes) (on_board yes) (dnp no)
   (property "Reference" "U4601" (at 153.67 43.18 0) (effects (font (size 1.27 1.27)) (justify left)))
   (property "Value" "TVS2200DRVR" (at 153.67 40.64 0) (effects (font (size 1.27 1.27)) (justify left)))
-  (property "Footprint" "Texas_Instruments:Texas_DRV0006A_WSON-6-1EP_2x2mm_P0.65mm_EP1x1.6mm" (at 161.29 55.88 0) (effects (font (size 1.27 1.27))) (hide yes))
+  (property "Footprint" "texas-instruments:Texas_DRV0006A_WSON-6-1EP_2x2mm_P0.65mm_EP1x1.6mm" (at 161.29 55.88 0) (effects (font (size 1.27 1.27))) (hide yes))
   (property "Datasheet" "https://www.ti.com/lit/ds/symlink/tvs2200.pdf" (at 161.29 55.88 0) (effects (font (size 1.27 1.27))) (hide yes))
   (property "Description" "Unidirectional flat-clamp surge protection device, 22 V stand-off, 40 A 8/20 us, IEC 61000-4-2 level 4, WSON-6 (DRV0006A) 2 x 2 mm" (at 161.29 55.88 0) (effects (font (size 1.27 1.27))) (hide yes))
@@
 (rectangle (start 133.35 35.56) (end 215.9 80.01) (stroke (width 0) (type dash)) (fill (type none)))
 (text "VBUS TVS, 22 V flat clamp (line 64)" (exclude_from_sim no) (at 134.62 34.29 0) (effects (font (size 2.54 2.54)) (justify left bottom)))
-(symbol (lib_id "Texas_Instruments:TPD8S300ARUKR") (at 252.73 86.36 0) (unit 1) (body_style 1) (exclude_from_sim no) (in_bom yes) (on_board yes) (dnp no)
+(symbol (lib_id "texas-instruments:TPD8S300ARUKR") (at 252.73 86.36 0) (unit 1) (body_style 1) (exclude_from_sim no) (in_bom yes) (on_board yes) (dnp no)
   (property "Reference" "U4602" (at 256.54 57.15 0) (effects (font (size 1.27 1.27)) (justify left)))
   (property "Value" "TPD8S300ARUKR" (at 256.54 54.61 0) (effects (font (size 1.27 1.27)) (justify left)))
-  (property "Footprint" "Texas_Instruments:Texas_RUK0020B_WQFN-20-1EP_3x3mm_P0.4mm_EP1.7x1.7mm" (at 252.73 86.36 0) (effects (font (size 1.27 1.27))) (hide yes))
+  (property "Footprint" "texas-instruments:Texas_RUK0020B_WQFN-20-1EP_3x3mm_P0.4mm_EP1.7x1.7mm" (at 252.73 86.36 0) (effects (font (size 1.27 1.27))) (hide yes))
   (property "Datasheet" "https://www.ti.com/lit/ds/symlink/tpd8s300a.pdf" (at 252.73 86.36 0) (effects (font (size 1.27 1.27))) (hide yes))
   (property "Description" "USB Type-C port protector, 20 V short-to-VBUS overvoltage protection on CC1, CC2, SBU1, SBU2, 8-channel IEC 61000-4-2 ESD, dead-battery Rd, WQFN-20 (RUK0020B) 3 x 3 mm" (at 252.73 86.36 0) (effects (font (size 1.27 1.27))) (hide yes))
@@
 (rectangle (start 220.98 35.56) (end 337.82 128.27) (stroke (width 0) (type dash)) (fill (type none)))
 (text "CC and SBU protection: TPD8S300A (line 63)" (exclude_from_sim no) (at 222.25 34.29 0) (effects (font (size 2.54 2.54)) (justify left bottom)))
-(symbol (lib_id "Texas_Instruments:TPD4E05U06DQAR") (at 369.57 59.69 0) (unit 1) (body_style 1) (exclude_from_sim no) (in_bom yes) (on_board yes) (dnp no)
+(symbol (lib_id "texas-instruments:TPD4E05U06DQAR") (at 369.57 59.69 0) (unit 1) (body_style 1) (exclude_from_sim no) (in_bom yes) (on_board yes) (dnp no)
   (property "Reference" "U4603" (at 363.22 43.18 0) (effects (font (size 1.27 1.27)) (justify left)))
   (property "Value" "TPD4E05U06DQAR" (at 363.22 40.64 0) (effects (font (size 1.27 1.27)) (justify left)))
-  (property "Footprint" "Texas_Instruments:Texas_DQA0010A_USON-10_1x2.5mm_P0.5mm" (at 369.57 59.69 0) (effects (font (size 1.27 1.27))) (hide yes))
+  (property "Footprint" "texas-instruments:Texas_DQA0010A_USON-10_1x2.5mm_P0.5mm" (at 369.57 59.69 0) (effects (font (size 1.27 1.27))) (hide yes))
   (property "Datasheet" "https://www.ti.com/lit/ds/symlink/tpd4e05u06.pdf" (at 369.57 59.69 0) (effects (font (size 1.27 1.27))) (hide yes))
   (property "Description" "4-channel ESD protection, 0.5 pF, 5.5 V stand-off, IEC 61000-4-2 level 4, flow-through routing, USON-10 (DQA0010A) 1 x 2.5 mm" (at 369.57 59.69 0) (effects (font (size 1.27 1.27))) (hide yes))

Commit message: BOM v1.18 item 2: successors of the discontinued 1 uF 0402
GRM155R61A105KE15D is to be discontinued. 44 positions take
GRM155C71A105KE11D (1 uF 10 V X7S); the eight TPS7A20 positions take
GRM155R61C225KE11D (2.2 uF 16 V X5R) to keep the 0.47 uF effective
minimum with 10 % to spare at up to 3.8 V. Same land; sourcing pass.
Closes BOM §7 item 52; new item 55 lists the other capture parts outside
Murata's product data or near end of life.

Co-Authored-By: Claude Opus 5.5 <noreply@anthropic.com>
Claude-Session: https://claude.ai/code/session_01Ei262h3TpgY9vyfNLMi5Mn
Parts:
- C4602, C4603: MPN GRM155R61A105KE15D -> GRM155C71A105KE11D
Changed lines of the file:
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@@
   (property "Value" "1 µF" (at 314.96 58.42 0) (effects (font (size 1.27 1.27)) (justify left)))
   (property "Footprint" "Capacitor_SMD:C_0402_1005Metric" (at 312.42 57.15 0) (effects (font (size 1.27 1.27))) (hide yes))
-  (property "Datasheet" "https://www.murata.com/en-us/products/productdetail?partno=GRM155R61A105KE15D" (at 312.42 57.15 0) (effects (font (size 1.27 1.27))) (hide yes))
-  (property "Description" "Capacitor, 1 µF, 10 V, X5R, 0402" (at 312.42 57.15 0) (effects (font (size 1.27 1.27))) (hide yes))
+  (property "Datasheet" "https://www.murata.com/en-us/products/productdetail?partno=GRM155C71A105KE11D" (at 312.42 57.15 0) (effects (font (size 1.27 1.27))) (hide yes))
+  (property "Description" "Capacitor, 1 µF, 10 V, X7S, 0402" (at 312.42 57.15 0) (effects (font (size 1.27 1.27))) (hide yes))
   (property "Manufacturer" "Murata" (at 312.42 57.15 0) (effects (font (size 1.27 1.27))) (hide yes))
-  (property "MPN" "GRM155R61A105KE15D" (at 312.42 57.15 0) (effects (font (size 1.27 1.27))) (hide yes))
+  (property "MPN" "GRM155C71A105KE11D" (at 312.42 57.15 0) (effects (font (size 1.27 1.27))) (hide yes))
   (property "Block" "blk.usb-c" (at 312.42 57.15 0) (effects (font (size 1.27 1.27))) (hide yes))
   (pin "1")
@@
   (property "Value" "1 µF" (at 185.42 152.4 0) (effects (font (size 1.27 1.27)) (justify left)))
   (property "Footprint" "Capacitor_SMD:C_0402_1005Metric" (at 182.88 151.13 0) (effects (font (size 1.27 1.27))) (hide yes))
-  (property "Datasheet" "https://www.murata.com/en-us/products/productdetail?partno=GRM155R61A105KE15D" (at 182.88 151.13 0) (effects (font (size 1.27 1.27))) (hide yes))
-  (property "Description" "Capacitor, 1 µF, 10 V, X5R, 0402" (at 182.88 151.13 0) (effects (font (size 1.27 1.27))) (hide yes))
+  (property "Datasheet" "https://www.murata.com/en-us/products/productdetail?partno=GRM155C71A105KE11D" (at 182.88 151.13 0) (effects (font (size 1.27 1.27))) (hide yes))
+  (property "Description" "Capacitor, 1 µF, 10 V, X7S, 0402" (at 182.88 151.13 0) (effects (font (size 1.27 1.27))) (hide yes))
   (property "Manufacturer" "Murata" (at 182.88 151.13 0) (effects (font (size 1.27 1.27))) (hide yes))
-  (property "MPN" "GRM155R61A105KE15D" (at 182.88 151.13 0) (effects (font (size 1.27 1.27))) (hide yes))
+  (property "MPN" "GRM155C71A105KE11D" (at 182.88 151.13 0) (effects (font (size 1.27 1.27))) (hide yes))
   (property "Block" "blk.usb-c" (at 182.88 151.13 0) (effects (font (size 1.27 1.27))) (hide yes))
   (pin "1")
