File: board/hardware/t1-main-board/hat-5v.kicad_sch (KiCad schematic)
At the start: 12 parts, among them Q4401 DMG1012T, U4401 TPS259470ARPWR, U4402 FUSB302B01MPX

Commit message: Board: capture blk.current-monitors
Five INA236 on I2C1 (0x40-0x43, 0x48) with their shunts, per power tree
§4.12 and BOM v1 lines 54 and 136. The measured branches are rails of
their own (VSYS_SRC, VSYS_LV_AUDIO, VSYS_AUDIO, VSYS_LV_BL, VSYS_P5V1),
fed through the shunts on this sheet; the charger, audio, backlight and
5.1 V sheets take them. The root's layout may leave a stack level empty,
so the block sits under the notes; IC bboxes hold turned rail values;
passive rows hold a bottom rail's text.

Co-Authored-By: Claude Opus 5.5 <noreply@anthropic.com>
Claude-Session: https://claude.ai/code/session_01Ei262h3TpgY9vyfNLMi5Mn
Parts:
- removed C4401, C4402, C4404: 1 µF, Capacitor_SMD:C_0402_1005Metric, symbol Device:C
- removed C4403: 1 nF, Capacitor_SMD:C_0402_1005Metric, symbol Device:C
- removed C4405: 100 nF, Capacitor_SMD:C_0402_1005Metric, symbol Device:C
- removed Q4401: DMG1012T, Package_TO_SOT_SMD:SOT-523, symbol Transistor_FET:DMG1012T
- removed R4401: 1.87 kΩ, Resistor_SMD:R_0402_1005Metric, symbol Device:R
- removed R4402: 10 kΩ, Resistor_SMD:R_0402_1005Metric, symbol Device:R
- removed R4403: 100 Ω, Resistor_SMD:R_0805_2012Metric, symbol Device:R
- removed R4404: 100 kΩ, Resistor_SMD:R_0402_1005Metric, symbol Device:R
- removed U4401: TPS259470ARPWR, Texas_Instruments:Texas_RPW0010A_VQFN-HR-10_2x2mm_P0.45mm, symbol Texas_Instruments:TPS259470ARPWR
- removed U4402: FUSB302B01MPX, onsemi:onsemi_510BR_WQFN-14-1EP_2.5x2.5mm_P0.5mm_EP1.45x1.45mm, symbol onsemi:FUSB302B01MPX
- added C4501, C4502, C4504: 1 µF, Capacitor_SMD:C_0402_1005Metric, symbol Device:C
- added C4503: 1 nF, Capacitor_SMD:C_0402_1005Metric, symbol Device:C
- added C4505: 100 nF, Capacitor_SMD:C_0402_1005Metric, symbol Device:C
- added Q4501: DMG1012T, Package_TO_SOT_SMD:SOT-523, symbol Transistor_FET:DMG1012T
- added R4501: 1.87 kΩ, Resistor_SMD:R_0402_1005Metric, symbol Device:R
- added R4502: 10 kΩ, Resistor_SMD:R_0402_1005Metric, symbol Device:R
- added R4503: 100 Ω, Resistor_SMD:R_0805_2012Metric, symbol Device:R
- added R4504: 100 kΩ, Resistor_SMD:R_0402_1005Metric, symbol Device:R
- added U4501: TPS259470ARPWR, Texas_Instruments:Texas_RPW0010A_VQFN-HR-10_2x2mm_P0.45mm, symbol Texas_Instruments:TPS259470ARPWR
- added U4502: FUSB302B01MPX, onsemi:onsemi_510BR_WQFN-14-1EP_2.5x2.5mm_P0.5mm_EP1.45x1.45mm, symbol onsemi:FUSB302B01MPX
Connections:
- net EFUSE_HAT5V_FLT_N: now also U4501.4 (FLT)
- net EFUSE_HAT5V_IMON: now also C4503.1, R4502.2
- net EFUSE_HAT5V_IMON_ILM: now also R4501.1, R4502.1, U4501.9 (ILM)
- net GND: now also C4501.2, C4502.2, C4503.2, C4504.2, C4505.2, Q4501.2 (S), R4501.2, R4504.2, U4501.2 (OVLO), U4501.8 (GND), U4502.15 (GND), U4502.8 (GND), U4502.9 (GND)
- net HAT5V_EN: now also U4501.1 (EN/UVLO)
- net HAT_5V: now also C4502.1, R4503.1, U4501.6 (OUT), U4502.2 (VBUS)
- net HAT_CC: now also U4502.10 (CC1), U4502.11 (CC1)
- net HAT_DISCH_D: now also Q4501.3 (D), R4503.2
- net HAT_PD_INT_N: now also U4502.5 (INT_N)
- net HAT_VBUS_DISCH: now also Q4501.1 (G), R4504.1
- net I2C1_SCL: now also U4502.6 (SCL)
- net I2C1_SDA: now also U4502.7 (SDA)
- net P5V1_LIM: now also C4501.1, U4501.5 (IN)
- net vcc3v3_pmu: now also C4504.1, C4505.1, U4502.3 (VDD), U4502.4 (VDD)

Commit message: Board: capture blk.debug
Debug UART2 (1.8 V) and I2S/DSD pads with ground pads, reset, PMIC and
power-key pads (PCB-T-09), a pad on every spare SoC GPIO whose pinout v1
row names one (the DEBUG bus, on the SoC's right edge), and a rail pad
for each power-tree rail no other sheet probes (PCB-T-02). Each DAC
sheet carries a pad on its MCLK. The spares pinout v1 leaves without a
pad now carry no-connect flags. On the root, facing sheet pins are
joined directly only where the route meets no other symbol.

Co-Authored-By: Claude Opus 5.5 <noreply@anthropic.com>
Claude-Session: https://claude.ai/code/session_01Ei262h3TpgY9vyfNLMi5Mn
Parts:
- removed C4501, C4502, C4504: 1 µF, Capacitor_SMD:C_0402_1005Metric, symbol Device:C
- removed C4503: 1 nF, Capacitor_SMD:C_0402_1005Metric, symbol Device:C
- removed C4505: 100 nF, Capacitor_SMD:C_0402_1005Metric, symbol Device:C
- removed Q4501: DMG1012T, Package_TO_SOT_SMD:SOT-523, symbol Transistor_FET:DMG1012T
- removed R4501: 1.87 kΩ, Resistor_SMD:R_0402_1005Metric, symbol Device:R
- removed R4502: 10 kΩ, Resistor_SMD:R_0402_1005Metric, symbol Device:R
- removed R4503: 100 Ω, Resistor_SMD:R_0805_2012Metric, symbol Device:R
- removed R4504: 100 kΩ, Resistor_SMD:R_0402_1005Metric, symbol Device:R
- removed U4501: TPS259470ARPWR, Texas_Instruments:Texas_RPW0010A_VQFN-HR-10_2x2mm_P0.45mm, symbol Texas_Instruments:TPS259470ARPWR
- removed U4502: FUSB302B01MPX, onsemi:onsemi_510BR_WQFN-14-1EP_2.5x2.5mm_P0.5mm_EP1.45x1.45mm, symbol onsemi:FUSB302B01MPX
- added C4601, C4602, C4604: 1 µF, Capacitor_SMD:C_0402_1005Metric, symbol Device:C
- added C4603: 1 nF, Capacitor_SMD:C_0402_1005Metric, symbol Device:C
- added C4605: 100 nF, Capacitor_SMD:C_0402_1005Metric, symbol Device:C
- added Q4601: DMG1012T, Package_TO_SOT_SMD:SOT-523, symbol Transistor_FET:DMG1012T
- added R4601: 1.87 kΩ, Resistor_SMD:R_0402_1005Metric, symbol Device:R
- added R4602: 10 kΩ, Resistor_SMD:R_0402_1005Metric, symbol Device:R
- added R4603: 100 Ω, Resistor_SMD:R_0805_2012Metric, symbol Device:R
- added R4604: 100 kΩ, Resistor_SMD:R_0402_1005Metric, symbol Device:R
- added U4601: TPS259470ARPWR, Texas_Instruments:Texas_RPW0010A_VQFN-HR-10_2x2mm_P0.45mm, symbol Texas_Instruments:TPS259470ARPWR
- added U4602: FUSB302B01MPX, onsemi:onsemi_510BR_WQFN-14-1EP_2.5x2.5mm_P0.5mm_EP1.45x1.45mm, symbol onsemi:FUSB302B01MPX
Connections:
- net EFUSE_HAT5V_FLT_N: now also U4601.4 (FLT)
- net EFUSE_HAT5V_IMON: now also C4603.1, R4602.2
- net EFUSE_HAT5V_IMON_ILM: now also R4601.1, R4602.1, U4601.9 (ILM)
- net GND: now also C4601.2, C4602.2, C4603.2, C4604.2, C4605.2, Q4601.2 (S), R4601.2, R4604.2, U4601.2 (OVLO), U4601.8 (GND), U4602.15 (GND), U4602.8 (GND), U4602.9 (GND)
- net HAT5V_EN: now also U4601.1 (EN/UVLO)
- net HAT_5V: now also C4602.1, R4603.1, U4601.6 (OUT), U4602.2 (VBUS)
- net HAT_CC: now also U4602.10 (CC1), U4602.11 (CC1)
- net HAT_DISCH_D: now also Q4601.3 (D), R4603.2
- net HAT_PD_INT_N: now also U4602.5 (INT_N)
- net HAT_VBUS_DISCH: now also Q4601.1 (G), R4604.1
- net I2C1_SCL: now also U4602.6 (SCL)
- net I2C1_SDA: now also U4602.7 (SDA)
- net P5V1_LIM: now also C4601.1, U4601.5 (IN)
- net vcc3v3_pmu: now also C4604.1, C4605.1, U4602.3 (VDD), U4602.4 (VDD)

Commit message: Board: capture blk.mic-ambient and links #34, #35
IM73D122 on PDM CLK1 and SDI1 (BOM v1 line 34, pinout v1 AK2 and 1P2),
LR to ground, 22 Ω clock series, VDD from MIC_1V8 through link #35.
Link #34 on blk.mic-main makes the faceplate branch the rail MIC_1V8_FP
for contact 40 (power tree §4.12, G10). kicad-lib moves to e46bda4 for
the IM73D122, TPS3808G01, SN74LVC1G58 and BAT54 parts.

Co-Authored-By: Claude Opus 5.5 <noreply@anthropic.com>
Claude-Session: https://claude.ai/code/session_01Ei262h3TpgY9vyfNLMi5Mn
Parts:
- removed C4601, C4602, C4604: 1 µF, Capacitor_SMD:C_0402_1005Metric, symbol Device:C
- removed C4603: 1 nF, Capacitor_SMD:C_0402_1005Metric, symbol Device:C
- removed C4605: 100 nF, Capacitor_SMD:C_0402_1005Metric, symbol Device:C
- removed Q4601: DMG1012T, Package_TO_SOT_SMD:SOT-523, symbol Transistor_FET:DMG1012T
- removed R4601: 1.87 kΩ, Resistor_SMD:R_0402_1005Metric, symbol Device:R
- removed R4602: 10 kΩ, Resistor_SMD:R_0402_1005Metric, symbol Device:R
- removed R4603: 100 Ω, Resistor_SMD:R_0805_2012Metric, symbol Device:R
- removed R4604: 100 kΩ, Resistor_SMD:R_0402_1005Metric, symbol Device:R
- removed U4601: TPS259470ARPWR, Texas_Instruments:Texas_RPW0010A_VQFN-HR-10_2x2mm_P0.45mm, symbol Texas_Instruments:TPS259470ARPWR
- removed U4602: FUSB302B01MPX, onsemi:onsemi_510BR_WQFN-14-1EP_2.5x2.5mm_P0.5mm_EP1.45x1.45mm, symbol onsemi:FUSB302B01MPX
- added C4701, C4702, C4704: 1 µF, Capacitor_SMD:C_0402_1005Metric, symbol Device:C
- added C4703: 1 nF, Capacitor_SMD:C_0402_1005Metric, symbol Device:C
- added C4705: 100 nF, Capacitor_SMD:C_0402_1005Metric, symbol Device:C
- added Q4701: DMG1012T, Package_TO_SOT_SMD:SOT-523, symbol Transistor_FET:DMG1012T
- added R4701: 1.87 kΩ, Resistor_SMD:R_0402_1005Metric, symbol Device:R
- added R4702: 10 kΩ, Resistor_SMD:R_0402_1005Metric, symbol Device:R
- added R4703: 100 Ω, Resistor_SMD:R_0805_2012Metric, symbol Device:R
- added R4704: 100 kΩ, Resistor_SMD:R_0402_1005Metric, symbol Device:R
- added U4701: TPS259470ARPWR, Texas_Instruments:Texas_RPW0010A_VQFN-HR-10_2x2mm_P0.45mm, symbol Texas_Instruments:TPS259470ARPWR
- added U4702: FUSB302B01MPX, onsemi:onsemi_510BR_WQFN-14-1EP_2.5x2.5mm_P0.5mm_EP1.45x1.45mm, symbol onsemi:FUSB302B01MPX
Connections:
- net EFUSE_HAT5V_FLT_N: now also U4701.4 (FLT)
- net EFUSE_HAT5V_IMON: now also C4703.1, R4702.2
- net EFUSE_HAT5V_IMON_ILM: now also R4701.1, R4702.1, U4701.9 (ILM)
- net GND: now also C4701.2, C4702.2, C4703.2, C4704.2, C4705.2, Q4701.2 (S), R4701.2, R4704.2, U4701.2 (OVLO), U4701.8 (GND), U4702.15 (GND), U4702.8 (GND), U4702.9 (GND)
- net HAT5V_EN: now also U4701.1 (EN/UVLO)
- net HAT_5V: now also C4702.1, R4703.1, U4701.6 (OUT), U4702.2 (VBUS)
- net HAT_CC: now also U4702.10 (CC1), U4702.11 (CC1)
- net HAT_DISCH_D: now also Q4701.3 (D), R4703.2
- net HAT_PD_INT_N: now also U4702.5 (INT_N)
- net HAT_VBUS_DISCH: now also Q4701.1 (G), R4704.1
- net I2C1_SCL: now also U4702.6 (SCL)
- net I2C1_SDA: now also U4702.7 (SDA)
- net P5V1_LIM: now also C4701.1, U4701.5 (IN)
- net vcc3v3_pmu: now also C4704.1, C4705.1, U4702.3 (VDD), U4702.4 (VDD)

Commit message: Board: capture blk.maskrom
Power + Vol- at a cold power-on pull eMMC D0 low inside the TPS3808G01
boot window (BOM v1 lines 35, 78, 97, 98; sim/maskrom): SENSE 280k/100k,
CT 390 nF, WINDOW_N with its pad, SN74LVC1G57 and SN74LVC1G58 on
vcca1v8_pmu, BAT54 from PWRON_N, DMG1012T through 1 kΩ to EMMC_D0.
Every block in use now has its sheet; the README states the remaining
single-pin nets.

Co-Authored-By: Claude Opus 5.5 <noreply@anthropic.com>
Claude-Session: https://claude.ai/code/session_01Ei262h3TpgY9vyfNLMi5Mn
Parts:
- removed C4701, C4702, C4704: 1 µF, Capacitor_SMD:C_0402_1005Metric, symbol Device:C
- removed C4703: 1 nF, Capacitor_SMD:C_0402_1005Metric, symbol Device:C
- removed C4705: 100 nF, Capacitor_SMD:C_0402_1005Metric, symbol Device:C
- removed Q4701: DMG1012T, Package_TO_SOT_SMD:SOT-523, symbol Transistor_FET:DMG1012T
- removed R4701: 1.87 kΩ, Resistor_SMD:R_0402_1005Metric, symbol Device:R
- removed R4702: 10 kΩ, Resistor_SMD:R_0402_1005Metric, symbol Device:R
- removed R4703: 100 Ω, Resistor_SMD:R_0805_2012Metric, symbol Device:R
- removed R4704: 100 kΩ, Resistor_SMD:R_0402_1005Metric, symbol Device:R
- removed U4701: TPS259470ARPWR, Texas_Instruments:Texas_RPW0010A_VQFN-HR-10_2x2mm_P0.45mm, symbol Texas_Instruments:TPS259470ARPWR
- removed U4702: FUSB302B01MPX, onsemi:onsemi_510BR_WQFN-14-1EP_2.5x2.5mm_P0.5mm_EP1.45x1.45mm, symbol onsemi:FUSB302B01MPX
- added C4801, C4802, C4804: 1 µF, Capacitor_SMD:C_0402_1005Metric, symbol Device:C
- added C4803: 1 nF, Capacitor_SMD:C_0402_1005Metric, symbol Device:C
- added C4805: 100 nF, Capacitor_SMD:C_0402_1005Metric, symbol Device:C
- added Q4801: DMG1012T, Package_TO_SOT_SMD:SOT-523, symbol Transistor_FET:DMG1012T
- added R4801: 1.87 kΩ, Resistor_SMD:R_0402_1005Metric, symbol Device:R
- added R4802: 10 kΩ, Resistor_SMD:R_0402_1005Metric, symbol Device:R
- added R4803: 100 Ω, Resistor_SMD:R_0805_2012Metric, symbol Device:R
- added R4804: 100 kΩ, Resistor_SMD:R_0402_1005Metric, symbol Device:R
- added U4801: TPS259470ARPWR, Texas_Instruments:Texas_RPW0010A_VQFN-HR-10_2x2mm_P0.45mm, symbol Texas_Instruments:TPS259470ARPWR
- added U4802: FUSB302B01MPX, onsemi:onsemi_510BR_WQFN-14-1EP_2.5x2.5mm_P0.5mm_EP1.45x1.45mm, symbol onsemi:FUSB302B01MPX
Connections:
- net EFUSE_HAT5V_FLT_N: now also U4801.4 (FLT)
- net EFUSE_HAT5V_IMON: now also C4803.1, R4802.2
- net EFUSE_HAT5V_IMON_ILM: now also R4801.1, R4802.1, U4801.9 (ILM)
- net GND: now also C4801.2, C4802.2, C4803.2, C4804.2, C4805.2, Q4801.2 (S), R4801.2, R4804.2, U4801.2 (OVLO), U4801.8 (GND), U4802.15 (GND), U4802.8 (GND), U4802.9 (GND)
- net HAT5V_EN: now also U4801.1 (EN/UVLO)
- net HAT_5V: now also C4802.1, R4803.1, U4801.6 (OUT), U4802.2 (VBUS)
- net HAT_CC: now also U4802.10 (CC1), U4802.11 (CC1)
- net HAT_DISCH_D: now also Q4801.3 (D), R4803.2
- net HAT_PD_INT_N: now also U4802.5 (INT_N)
- net HAT_VBUS_DISCH: now also Q4801.1 (G), R4804.1
- net I2C1_SCL: now also U4802.6 (SCL)
- net I2C1_SDA: now also U4802.7 (SDA)
- net P5V1_LIM: now also C4801.1, U4801.5 (IN)
- net vcc3v3_pmu: now also C4804.1, C4805.1, U4802.3 (VDD), U4802.4 (VDD)

Commit message: Board on libs v0.2.0: lower-case kebab vendor keys (HL-13)
The libs submodule moves to v0.2.0 (5f24483). Every library nickname in
the generator, the placement tool and the floorplan study follows the
key table (Texas_Instruments -> texas-instruments, OpenDAP_Device ->
opendap-generic, Rockchip and Rockchip_PMIC -> rockchip, ...); the
library tables are written from the files. Schematic and board
regenerated.

Checks: ERC 0 errors (warnings unchanged); DRC 0 errors, 605 warnings,
the same counts by type, schematic parity 0; every placement identical;
craft Q1 met; pcb tests pass; STEP export resolves every libs 3D model
(the 27 parts without a model are KiCad stock lands that have none).

Co-Authored-By: Claude Opus 5.5 <noreply@anthropic.com>
Claude-Session: https://claude.ai/code/session_01Ei262h3TpgY9vyfNLMi5Mn
Parts:
- U4801: footprint Texas_Instruments:Texas_RPW0010A_VQFN-HR-10_2x2mm_P0.45mm -> texas-instruments:Texas_RPW0010A_VQFN-HR-10_2x2mm_P0.45mm; symbol Texas_Instruments:TPS259470ARPWR -> texas-instruments:TPS259470ARPWR
Changed lines of the file:
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@@
 (paper "A3")
 (title_block (title "HAT port VBUS and USB PD") (date "2026-10-25") (rev "A") (company "The OpenDAP Project") (comment 1 "blk.hat-5v") (comment 2 "eFuse #A to the HAT VBUS, the FUSB302B01 port controller and the VBUS discharge"))
-(symbol (lib_id "Texas_Instruments:TPS259470ARPWR") (at 53.34 82.55 0) (unit 1) (body_style 1) (exclude_from_sim no) (in_bom yes) (on_board yes) (dnp no)
+(symbol (lib_id "texas-instruments:TPS259470ARPWR") (at 53.34 82.55 0) (unit 1) (body_style 1) (exclude_from_sim no) (in_bom yes) (on_board yes) (dnp no)
   (property "Reference" "U4801" (at 41.91 60.96 0) (effects (font (size 1.27 1.27)) (justify left)))
   (property "Value" "TPS259470ARPWR" (at 41.91 58.42 0) (effects (font (size 1.27 1.27)) (justify left)))
-  (property "Footprint" "Texas_Instruments:Texas_RPW0010A_VQFN-HR-10_2x2mm_P0.45mm" (at 53.34 82.55 0) (effects (font (size 1.27 1.27))) (hide yes))
+  (property "Footprint" "texas-instruments:Texas_RPW0010A_VQFN-HR-10_2x2mm_P0.45mm" (at 53.34 82.55 0) (effects (font (size 1.27 1.27))) (hide yes))
   (property "Datasheet" "https://www.ti.com/lit/ds/symlink/tps25947.pdf" (at 53.34 82.55 0) (effects (font (size 1.27 1.27))) (hide yes))
   (property "Description" "eFuse, 2.7-23 V, 5.5 A, 28 mOhm, true reverse-current blocking, adjustable UVLO/OVLO and current limit, AUXOFF and FLT outputs, auto-retry, VQFN-HR-10 (RPW0010A) 2 x 2 mm" (at 53.34 82.55 0) (effects (font (size 1.27 1.27))) (hide yes))

Commit message: BOM v1.18 item 2: successors of the discontinued 1 uF 0402
GRM155R61A105KE15D is to be discontinued. 44 positions take
GRM155C71A105KE11D (1 uF 10 V X7S); the eight TPS7A20 positions take
GRM155R61C225KE11D (2.2 uF 16 V X5R) to keep the 0.47 uF effective
minimum with 10 % to spare at up to 3.8 V. Same land; sourcing pass.
Closes BOM §7 item 52; new item 55 lists the other capture parts outside
Murata's product data or near end of life.

Co-Authored-By: Claude Opus 5.5 <noreply@anthropic.com>
Claude-Session: https://claude.ai/code/session_01Ei262h3TpgY9vyfNLMi5Mn
Parts:
- C4804: MPN GRM155R61A105KE15D -> GRM155C71A105KE11D
Changed lines of the file:
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@@
   (property "Value" "1 µF" (at 252.73 49.53 0) (effects (font (size 1.27 1.27)) (justify left)))
   (property "Footprint" "Capacitor_SMD:C_0402_1005Metric" (at 250.19 48.26 0) (effects (font (size 1.27 1.27))) (hide yes))
-  (property "Datasheet" "https://www.murata.com/en-us/products/productdetail?partno=GRM155R61A105KE15D" (at 250.19 48.26 0) (effects (font (size 1.27 1.27))) (hide yes))
-  (property "Description" "Capacitor, 1 µF, 10 V, X5R, 0402" (at 250.19 48.26 0) (effects (font (size 1.27 1.27))) (hide yes))
+  (property "Datasheet" "https://www.murata.com/en-us/products/productdetail?partno=GRM155C71A105KE11D" (at 250.19 48.26 0) (effects (font (size 1.27 1.27))) (hide yes))
+  (property "Description" "Capacitor, 1 µF, 10 V, X7S, 0402" (at 250.19 48.26 0) (effects (font (size 1.27 1.27))) (hide yes))
   (property "Manufacturer" "Murata" (at 250.19 48.26 0) (effects (font (size 1.27 1.27))) (hide yes))
-  (property "MPN" "GRM155R61A105KE15D" (at 250.19 48.26 0) (effects (font (size 1.27 1.27))) (hide yes))
+  (property "MPN" "GRM155C71A105KE11D" (at 250.19 48.26 0) (effects (font (size 1.27 1.27))) (hide yes))
   (property "Block" "blk.hat-5v" (at 250.19 48.26 0) (effects (font (size 1.27 1.27))) (hide yes))
   (pin "1")
