File: board/hardware/t1-main-board/pmic.kicad_sch (KiCad schematic)
At the start: 48 parts, among them U1101 RK809-5, Y1101 32.768 kHz

Commit message: Compaction: lower inductors, 0201 decoupling, 0.8 mm signal test pads
A matrix tool (hardware/studies/compaction) checks each candidate against
the design's stresses: same inductance, design peak <= 70 % and the
converter's maximum limit <= 100 % of Isat (30 % drop), height zones,
ratings at least twice the rail, PCB-D-06; sourcing outcome per part.

Applied (placement v1 decision 12, BOM v1.15):
- L601, L4401: XGL4015-102MEC (1.5 mm) for XAL/XGL4020-102MEC (2.1 mm);
- L1001, L5101: XGL4015-471MEC (1.5 mm) for Wurth 744373240047, on the
  stock XxL4020 land (the Wurth land was never drawn);
- L1201 is 1.2 mm (XGL4012, per-MPN heights): it moves next to the SoC;
- 58 x 100 nF decoupling on rails <= 3.3 V in core/IO/radio: 0201;
- 51 test pads on signal nets: 0.8 mm (PCB-D-06 v0.16, JLCPCB guide).
Kept: L901, L2802 (XGL4015 at 103 % of Isat at the limit); no thinner
0805/1206 capacitor passes (obsolete, NRND or unlisted).

Board need 113 % -> 111 % (core band 227 -> 203 %, power band 258 ->
233 %, radio band 19 -> 0 %); only C904 still relies on PCB-Z-04.
ERC 0 errors, craft Q1 met, DRC 0 errors (605 warnings), pcb and study
tests pass, rules test board PASS.

Co-Authored-By: Claude Opus 5.5 <noreply@anthropic.com>
Claude-Session: https://claude.ai/code/session_01Ei262h3TpgY9vyfNLMi5Mn
Parts:
- TP1101, TP1102: footprint TestPoint:TestPoint_Pad_D1.0mm -> T1_Main_Board:TestPoint_Pad_D0.8mm
Changed lines of the file:
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@@
   (property "Reference" "TP1101" (at 354.33 129.54 0) (effects (font (size 1.27 1.27)) (justify left)))
   (property "Value" "PMIC_BATDIV" (at 354.33 132.08 0) (effects (font (size 1.27 1.27)) (justify left)))
-  (property "Footprint" "TestPoint:TestPoint_Pad_D1.0mm" (at 353.06 134.62 0) (effects (font (size 1.27 1.27))) (hide yes))
+  (property "Footprint" "T1_Main_Board:TestPoint_Pad_D0.8mm" (at 353.06 134.62 0) (effects (font (size 1.27 1.27))) (hide yes))
   (property "Datasheet" "~" (at 353.06 134.62 0) (effects (font (size 1.27 1.27))) (hide yes))
-  (property "Description" "Test pad, 1.0 mm" (at 353.06 134.62 0) (effects (font (size 1.27 1.27))) (hide yes))
+  (property "Description" "Test pad, 0.8 mm, signal net" (at 353.06 134.62 0) (effects (font (size 1.27 1.27))) (hide yes))
   (property "Block" "blk.pmic" (at 353.06 134.62 0) (effects (font (size 1.27 1.27))) (hide yes))
   (pin "1")
@@
   (property "Reference" "TP1102" (at 384.81 129.54 0) (effects (font (size 1.27 1.27)) (justify left)))
   (property "Value" "PMIC_SNS" (at 384.81 132.08 0) (effects (font (size 1.27 1.27)) (justify left)))
-  (property "Footprint" "TestPoint:TestPoint_Pad_D1.0mm" (at 383.54 134.62 0) (effects (font (size 1.27 1.27))) (hide yes))
+  (property "Footprint" "T1_Main_Board:TestPoint_Pad_D0.8mm" (at 383.54 134.62 0) (effects (font (size 1.27 1.27))) (hide yes))
   (property "Datasheet" "~" (at 383.54 134.62 0) (effects (font (size 1.27 1.27))) (hide yes))
-  (property "Description" "Test pad, 1.0 mm" (at 383.54 134.62 0) (effects (font (size 1.27 1.27))) (hide yes))
+  (property "Description" "Test pad, 0.8 mm, signal net" (at 383.54 134.62 0) (effects (font (size 1.27 1.27))) (hide yes))
   (property "Block" "blk.pmic" (at 383.54 134.62 0) (effects (font (size 1.27 1.27))) (hide yes))
   (pin "1")

Commit message: Board on libs v0.2.0: lower-case kebab vendor keys (HL-13)
The libs submodule moves to v0.2.0 (5f24483). Every library nickname in
the generator, the placement tool and the floorplan study follows the
key table (Texas_Instruments -> texas-instruments, OpenDAP_Device ->
opendap-generic, Rockchip and Rockchip_PMIC -> rockchip, ...); the
library tables are written from the files. Schematic and board
regenerated.

Checks: ERC 0 errors (warnings unchanged); DRC 0 errors, 605 warnings,
the same counts by type, schematic parity 0; every placement identical;
craft Q1 met; pcb tests pass; STEP export resolves every libs 3D model
(the 27 parts without a model are KiCad stock lands that have none).

Co-Authored-By: Claude Opus 5.5 <noreply@anthropic.com>
Claude-Session: https://claude.ai/code/session_01Ei262h3TpgY9vyfNLMi5Mn
Parts:
- U1101: footprint Rockchip_PMIC:QFN-68-1EP_7x7mm_P0.35mm_EP5.49x5.49mm_ThermalVias -> rockchip:QFN-68-1EP_7x7mm_P0.35mm_EP5.49x5.49mm_ThermalVias; symbol Rockchip_PMIC:RK809-5 -> rockchip:RK809-5; Manufacturer_2 Rockchip -> rockchip
- Y1101: symbol OpenDAP_Device:Crystal -> opendap-generic:Crystal
Changed lines of the file:
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@@
 (rectangle (start 22.86 27.94) (end 203.2 193.04) (stroke (width 0) (type dash)) (fill (type none)))
 (text "RK809-5" (exclude_from_sim no) (at 24.13 26.67 0) (effects (font (size 2.54 2.54)) (justify left bottom)))
-(symbol (lib_id "Rockchip_PMIC:RK809-5") (at 68.58 81.28 0) (unit 1) (body_style 1) (exclude_from_sim no) (in_bom yes) (on_board yes) (dnp no)
+(symbol (lib_id "rockchip:RK809-5") (at 68.58 81.28 0) (unit 1) (body_style 1) (exclude_from_sim no) (in_bom yes) (on_board yes) (dnp no)
   (property "Reference" "U1101" (at 59.69 113.03 0) (effects (font (size 1.27 1.27)) (justify left)))
   (property "Value" "RK809-5" (at 59.69 110.49 0) (effects (font (size 1.27 1.27)) (justify left)))
-  (property "Footprint" "Rockchip_PMIC:QFN-68-1EP_7x7mm_P0.35mm_EP5.49x5.49mm_ThermalVias" (at 68.58 81.28 0) (effects (font (size 1.27 1.27))) (hide yes))
+  (property "Footprint" "rockchip:QFN-68-1EP_7x7mm_P0.35mm_EP5.49x5.49mm_ThermalVias" (at 68.58 81.28 0) (effects (font (size 1.27 1.27))) (hide yes))
   (property "Datasheet" "https://rockchip.fr/RK809%20datasheet%20V1.01.pdf" (at 68.58 81.28 0) (effects (font (size 1.27 1.27))) (hide yes))
   (property "Description" "PMIC: five synchronous bucks, nine LDOs, two power switches, RTC with 32.768 kHz output, fuel gauge, audio codec; QFN68 7 x 7 mm, 0.35 mm pitch, exposed ground pad" (at 68.58 81.28 0) (effects (font (size 1.27 1.27))) (hide yes))
@@
   (property "Second_Source" "Rockchip RK809-5A (BOM v1 line 2)" (at 68.58 81.28 0) (effects (font (size 1.27 1.27))) (hide yes))
   (property "Block" "blk.pmic" (at 68.58 81.28 0) (effects (font (size 1.27 1.27))) (hide yes))
-  (property "Manufacturer_2" "Rockchip" (at 68.58 81.28 0) (effects (font (size 1.27 1.27))) (hide yes))
+  (property "Manufacturer_2" "rockchip" (at 68.58 81.28 0) (effects (font (size 1.27 1.27))) (hide yes))
   (property "MPN_2" "RK809-5A" (at 68.58 81.28 0) (effects (font (size 1.27 1.27))) (hide yes))
   (pin "12")
@@
   (instances (project "t1-main-board" (path "/7746052e-d7f9-59ad-ba73-bd2b74439529/17ca007d-d661-5052-8fa8-f3468133f957" (reference "#PWR0091") (unit 1))))
 )
-(symbol (lib_id "Rockchip_PMIC:RK809-5") (at 68.58 162.56 0) (unit 2) (body_style 1) (exclude_from_sim no) (in_bom yes) (on_board yes) (dnp no)
+(symbol (lib_id "rockchip:RK809-5") (at 68.58 162.56 0) (unit 2) (body_style 1) (exclude_from_sim no) (in_bom yes) (on_board yes) (dnp no)
   (property "Reference" "U1101" (at 59.69 191.77 0) (effects (font (size 1.27 1.27)) (justify left)))
   (property "Value" "RK809-5" (at 59.69 189.23 0) (effects (font (size 1.27 1.27)) (justify left)))
-  (property "Footprint" "Rockchip_PMIC:QFN-68-1EP_7x7mm_P0.35mm_EP5.49x5.49mm_ThermalVias" (at 68.58 162.56 0) (effects (font (size 1.27 1.27))) (hide yes))
+  (property "Footprint" "rockchip:QFN-68-1EP_7x7mm_P0.35mm_EP5.49x5.49mm_ThermalVias" (at 68.58 162.56 0) (effects (font (size 1.27 1.27))) (hide yes))
   (property "Datasheet" "https://rockchip.fr/RK809%20datasheet%20V1.01.pdf" (at 68.58 162.56 0) (effects (font (size 1.27 1.27))) (hide yes))
   (property "Description" "PMIC: five synchronous bucks, nine LDOs, two power switches, RTC with 32.768 kHz output, fuel gauge, audio codec; QFN68 7 x 7 mm, 0.35 mm pitch, exposed ground pad" (at 68.58 162.56 0) (effects (font (size 1.27 1.27))) (hide yes))
@@
   (property "Second_Source" "Rockchip RK809-5A (BOM v1 line 2)" (at 68.58 162.56 0) (effects (font (size 1.27 1.27))) (hide yes))
   (property "Block" "blk.pmic" (at 68.58 162.56 0) (effects (font (size 1.27 1.27))) (hide yes))
-  (property "Manufacturer_2" "Rockchip" (at 68.58 162.56 0) (effects (font (size 1.27 1.27))) (hide yes))
+  (property "Manufacturer_2" "rockchip" (at 68.58 162.56 0) (effects (font (size 1.27 1.27))) (hide yes))
   (property "MPN_2" "RK809-5A" (at 68.58 162.56 0) (effects (font (size 1.27 1.27))) (hide yes))
   (pin "23")
@@
   (instances (project "t1-main-board" (path "/7746052e-d7f9-59ad-ba73-bd2b74439529/17ca007d-d661-5052-8fa8-f3468133f957" (reference "#PWR0102") (unit 1))))
 )
-(symbol (lib_id "Rockchip_PMIC:RK809-5") (at 160.02 81.28 0) (unit 3) (body_style 1) (exclude_from_sim no) (in_bom yes) (on_board yes) (dnp no)
+(symbol (lib_id "rockchip:RK809-5") (at 160.02 81.28 0) (unit 3) (body_style 1) (exclude_from_sim no) (in_bom yes) (on_board yes) (dnp no)
   (property "Reference" "U1101" (at 148.59 52.07 0) (effects (font (size 1.27 1.27)) (justify left)))
   (property "Value" "RK809-5" (at 148.59 49.53 0) (effects (font (size 1.27 1.27)) (justify left)))
-  (property "Footprint" "Rockchip_PMIC:QFN-68-1EP_7x7mm_P0.35mm_EP5.49x5.49mm_ThermalVias" (at 160.02 81.28 0) (effects (font (size 1.27 1.27))) (hide yes))
+  (property "Footprint" "rockchip:QFN-68-1EP_7x7mm_P0.35mm_EP5.49x5.49mm_ThermalVias" (at 160.02 81.28 0) (effects (font (size 1.27 1.27))) (hide yes))
   (property "Datasheet" "https://rockchip.fr/RK809%20datasheet%20V1.01.pdf" (at 160.02 81.28 0) (effects (font (size 1.27 1.27))) (hide yes))
   (property "Description" "PMIC: five synchronous bucks, nine LDOs, two power switches, RTC with 32.768 kHz output, fuel gauge, audio codec; QFN68 7 x 7 mm, 0.35 mm pitch, exposed ground pad" (at 160.02 81.28 0) (effects (font (size 1.27 1.27))) (hide yes))
@@
   (property "Second_Source" "Rockchip RK809-5A (BOM v1 line 2)" (at 160.02 81.28 0) (effects (font (size 1.27 1.27))) (hide yes))
   (property "Block" "blk.pmic" (at 160.02 81.28 0) (effects (font (size 1.27 1.27))) (hide yes))
-  (property "Manufacturer_2" "Rockchip" (at 160.02 81.28 0) (effects (font (size 1.27 1.27))) (hide yes))
+  (property "Manufacturer_2" "rockchip" (at 160.02 81.28 0) (effects (font (size 1.27 1.27))) (hide yes))
   (property "MPN_2" "RK809-5A" (at 160.02 81.28 0) (effects (font (size 1.27 1.27))) (hide yes))
   (pin "1")
@@
 (wire (pts (xy 175.26 78.74) (xy 177.8 78.74)) (stroke (width 0) (type default)))
 (wire (pts (xy 175.26 81.28) (xy 177.8 81.28)) (stroke (width 0) (type default)))
-(symbol (lib_id "Rockchip_PMIC:RK809-5") (at 160.02 154.94 0) (unit 4) (body_style 1) (exclude_from_sim no) (in_bom yes) (on_board yes) (dnp no)
+(symbol (lib_id "rockchip:RK809-5") (at 160.02 154.94 0) (unit 4) (body_style 1) (exclude_from_sim no) (in_bom yes) (on_board yes) (dnp no)
   (property "Reference" "U1101" (at 146.05 186.69 0) (effects (font (size 1.27 1.27)) (justify left)))
   (property "Value" "RK809-5" (at 146.05 184.15 0) (effects (font (size 1.27 1.27)) (justify left)))
-  (property "Footprint" "Rockchip_PMIC:QFN-68-1EP_7x7mm_P0.35mm_EP5.49x5.49mm_ThermalVias" (at 160.02 154.94 0) (effects (font (size 1.27 1.27))) (hide yes))
+  (property "Footprint" "rockchip:QFN-68-1EP_7x7mm_P0.35mm_EP5.49x5.49mm_ThermalVias" (at 160.02 154.94 0) (effects (font (size 1.27 1.27))) (hide yes))
   (property "Datasheet" "https://rockchip.fr/RK809%20datasheet%20V1.01.pdf" (at 160.02 154.94 0) (effects (font (size 1.27 1.27))) (hide yes))
   (property "Description" "PMIC: five synchronous bucks, nine LDOs, two power switches, RTC with 32.768 kHz output, fuel gauge, audio codec; QFN68 7 x 7 mm, 0.35 mm pitch, exposed ground pad" (at 160.02 154.94 0) (effects (font (size 1.27 1.27))) (hide yes))
@@
   (property "Second_Source" "Rockchip RK809-5A (BOM v1 line 2)" (at 160.02 154.94 0) (effects (font (size 1.27 1.27))) (hide yes))
   (property "Block" "blk.pmic" (at 160.02 154.94 0) (effects (font (size 1.27 1.27))) (hide yes))
-  (property "Manufacturer_2" "Rockchip" (at 160.02 154.94 0) (effects (font (size 1.27 1.27))) (hide yes))
+  (property "Manufacturer_2" "rockchip" (at 160.02 154.94 0) (effects (font (size 1.27 1.27))) (hide yes))
   (property "MPN_2" "RK809-5A" (at 160.02 154.94 0) (effects (font (size 1.27 1.27))) (hide yes))
   (pin "14")
@@
 (junction (at 375.92 80.01) (diameter 0) (color 0 0 0 0))
 (wire (pts (xy 375.92 80.01) (xy 375.92 92.71)) (stroke (width 0) (type default)))
-(symbol (lib_id "OpenDAP_Device:Crystal") (at 370.84 111.76 0) (unit 1) (body_style 1) (exclude_from_sim no) (in_bom yes) (on_board yes) (dnp no)
+(symbol (lib_id "opendap-generic:Crystal") (at 370.84 111.76 0) (unit 1) (body_style 1) (exclude_from_sim no) (in_bom yes) (on_board yes) (dnp no)
   (property "Reference" "Y1101" (at 367.03 106.68 0) (effects (font (size 1.27 1.27)) (justify left)))
   (property "Value" "32.768 kHz" (at 367.03 116.84 0) (effects (font (size 1.27 1.27)) (justify left)))
