File: board/hardware/t1-main-board/pmic.kicad_sch (KiCad schematic)
At the start: 48 parts, among them U1101 RK809-5, Y1101 32.768 kHz

Commit message: Board in the 62.5 x 95.0 mm body: ADR 0025, outline 59.1 x 91.6, 0201 swaps
ADR 0025 supersedes ADR 0016 for t1 ADR 0006's body: board outline from
the body, 1.2 mm walls and 0.5 mm clearance; height zones and stack
restated unchanged; the speaker on a case shelf (PCB-Z-09); pocket
reliefs at the 4.4 mm jack, the microSD (DM3AT push-push kept) and the
side buttons; the audio 0603 -> 0402 swap gated by t1 V2-A08; reserve
(NFC reader, then TPM) recorded, not applied.

- pcb/geometry.py derives the outline from BODY, WALL and CLEARANCE;
  the pocket, display and fixed parts keep their device-frame positions;
  holes keep their edge distance; the speaker shadow becomes a 1.5 mm
  shelf height area (placement, checks, occupancy).
- build.py reports pocket reliefs and routing room; C904 unfixed (it
  now finds back room, so PCB-Z-04 carries no part).
- Generator: parts.area_swap puts 121 generic 0402 resistors (outside
  audio and VBUS paths, >= 10 ohm) and five 100 nF signal capacitors in
  0201 (BOM v1.16); schematic and board regenerated.
- Result: 1,012/1,012 placed, 98.8 % by the floorplan method (was 111 %),
  factor left 1.68 (was 1.49); DRC 0 errors, ERC 0 errors, 0 check
  findings, pcb tests 20/20, schematic craft Q1 met.
- Specs: PCB constraints v0.17 (M-01, M-02, M-08, Z-02, Z-06 to Z-09,
  R-07), placement v1.1 (section 3, decisions 4 and 13, checks, open
  items with the gated swaps and the reserve), floorplan v1 section 1,
  BOM v1.16.

Co-Authored-By: Claude Opus 5.5 <noreply@anthropic.com>
Claude-Session: https://claude.ai/code/session_01Ei262h3TpgY9vyfNLMi5Mn
Parts:
- C1114, C1115: footprint Capacitor_SMD:C_0402_1005Metric -> Capacitor_SMD:C_0201_0603Metric; MPN GRM155R71C104KA88D -> GRM033R61A104KE15D
- R1101: footprint Resistor_SMD:R_0402_1005Metric -> Resistor_SMD:R_0201_0603Metric; MPN RC0402FR-0747KL -> RC0201FR-0747KL
- R1102: footprint Resistor_SMD:R_0402_1005Metric -> Resistor_SMD:R_0201_0603Metric; MPN RC0402FR-07120KL -> RC0201FR-07120KL
- R1103: footprint Resistor_SMD:R_0402_1005Metric -> Resistor_SMD:R_0201_0603Metric; MPN RC0402FR-07100KL -> RC0201FR-07100KL
- R1104: footprint Resistor_SMD:R_0402_1005Metric -> Resistor_SMD:R_0201_0603Metric; MPN RC0402FR-0722KL -> RC0201FR-0722KL
Changed lines of the file:
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@@
   (property "Reference" "R1101" (at 313.69 82.55 0) (effects (font (size 1.27 1.27)) (justify left)))
   (property "Value" "47 kΩ" (at 313.69 85.09 0) (effects (font (size 1.27 1.27)) (justify left)))
-  (property "Footprint" "Resistor_SMD:R_0402_1005Metric" (at 312.42 83.82 0) (effects (font (size 1.27 1.27))) (hide yes))
-  (property "Datasheet" "https://yageogroup.com/en/ProductSearch/PartNumberSearch?part=RC0402FR-0747KL" (at 312.42 83.82 0) (effects (font (size 1.27 1.27))) (hide yes))
-  (property "Description" "Resistor, 47 kΩ, 1 %, 1/16 W, 0402" (at 312.42 83.82 0) (effects (font (size 1.27 1.27))) (hide yes))
+  (property "Footprint" "Resistor_SMD:R_0201_0603Metric" (at 312.42 83.82 0) (effects (font (size 1.27 1.27))) (hide yes))
+  (property "Datasheet" "https://yageogroup.com/en/ProductSearch/PartNumberSearch?part=RC0201FR-0747KL" (at 312.42 83.82 0) (effects (font (size 1.27 1.27))) (hide yes))
+  (property "Description" "Resistor, 47 kΩ, 1 %, 1/20 W, 0201" (at 312.42 83.82 0) (effects (font (size 1.27 1.27))) (hide yes))
   (property "Manufacturer" "YAGEO" (at 312.42 83.82 0) (effects (font (size 1.27 1.27))) (hide yes))
-  (property "MPN" "RC0402FR-0747KL" (at 312.42 83.82 0) (effects (font (size 1.27 1.27))) (hide yes))
+  (property "MPN" "RC0201FR-0747KL" (at 312.42 83.82 0) (effects (font (size 1.27 1.27))) (hide yes))
   (property "Block" "blk.pmic" (at 312.42 83.82 0) (effects (font (size 1.27 1.27))) (hide yes))
   (pin "1")
@@
   (property "Reference" "R1102" (at 313.69 95.25 0) (effects (font (size 1.27 1.27)) (justify left)))
   (property "Value" "120 kΩ" (at 313.69 97.79 0) (effects (font (size 1.27 1.27)) (justify left)))
-  (property "Footprint" "Resistor_SMD:R_0402_1005Metric" (at 312.42 96.52 0) (effects (font (size 1.27 1.27))) (hide yes))
-  (property "Datasheet" "https://yageogroup.com/en/ProductSearch/PartNumberSearch?part=RC0402FR-07120KL" (at 312.42 96.52 0) (effects (font (size 1.27 1.27))) (hide yes))
-  (property "Description" "Resistor, 120 kΩ, 1 %, 1/16 W, 0402" (at 312.42 96.52 0) (effects (font (size 1.27 1.27))) (hide yes))
+  (property "Footprint" "Resistor_SMD:R_0201_0603Metric" (at 312.42 96.52 0) (effects (font (size 1.27 1.27))) (hide yes))
+  (property "Datasheet" "https://yageogroup.com/en/ProductSearch/PartNumberSearch?part=RC0201FR-07120KL" (at 312.42 96.52 0) (effects (font (size 1.27 1.27))) (hide yes))
+  (property "Description" "Resistor, 120 kΩ, 1 %, 1/20 W, 0201" (at 312.42 96.52 0) (effects (font (size 1.27 1.27))) (hide yes))
   (property "Manufacturer" "YAGEO" (at 312.42 96.52 0) (effects (font (size 1.27 1.27))) (hide yes))
-  (property "MPN" "RC0402FR-07120KL" (at 312.42 96.52 0) (effects (font (size 1.27 1.27))) (hide yes))
+  (property "MPN" "RC0201FR-07120KL" (at 312.42 96.52 0) (effects (font (size 1.27 1.27))) (hide yes))
   (property "Block" "blk.pmic" (at 312.42 96.52 0) (effects (font (size 1.27 1.27))) (hide yes))
   (pin "1")
@@
   (property "Reference" "C1114" (at 350.52 73.66 0) (effects (font (size 1.27 1.27)) (justify left)))
   (property "Value" "100 nF" (at 350.52 76.2 0) (effects (font (size 1.27 1.27)) (justify left)))
-  (property "Footprint" "Capacitor_SMD:C_0402_1005Metric" (at 347.98 74.93 0) (effects (font (size 1.27 1.27))) (hide yes))
-  (property "Datasheet" "https://www.murata.com/en-us/products/productdetail?partno=GRM155R71C104KA88D" (at 347.98 74.93 0) (effects (font (size 1.27 1.27))) (hide yes))
-  (property "Description" "Capacitor, 100 nF, 16 V, X7R, 0402" (at 347.98 74.93 0) (effects (font (size 1.27 1.27))) (hide yes))
+  (property "Footprint" "Capacitor_SMD:C_0201_0603Metric" (at 347.98 74.93 0) (effects (font (size 1.27 1.27))) (hide yes))
+  (property "Datasheet" "https://www.murata.com/en-us/products/productdetail?partno=GRM033R61A104KE15D" (at 347.98 74.93 0) (effects (font (size 1.27 1.27))) (hide yes))
+  (property "Description" "Capacitor, 100 nF, 10 V, X5R, 0201" (at 347.98 74.93 0) (effects (font (size 1.27 1.27))) (hide yes))
   (property "Manufacturer" "Murata" (at 347.98 74.93 0) (effects (font (size 1.27 1.27))) (hide yes))
-  (property "MPN" "GRM155R71C104KA88D" (at 347.98 74.93 0) (effects (font (size 1.27 1.27))) (hide yes))
+  (property "MPN" "GRM033R61A104KE15D" (at 347.98 74.93 0) (effects (font (size 1.27 1.27))) (hide yes))
   (property "Block" "blk.pmic" (at 347.98 74.93 0) (effects (font (size 1.27 1.27))) (hide yes))
   (pin "1")
@@
   (property "Reference" "R1103" (at 369.57 71.12 0) (effects (font (size 1.27 1.27)) (justify left)))
   (property "Value" "100 kΩ" (at 369.57 73.66 0) (effects (font (size 1.27 1.27)) (justify left)))
-  (property "Footprint" "Resistor_SMD:R_0402_1005Metric" (at 368.3 72.39 0) (effects (font (size 1.27 1.27))) (hide yes))
-  (property "Datasheet" "https://yageogroup.com/en/ProductSearch/PartNumberSearch?part=RC0402FR-07100KL" (at 368.3 72.39 0) (effects (font (size 1.27 1.27))) (hide yes))
-  (property "Description" "Resistor, 100 kΩ, 1 %, 1/16 W, 0402" (at 368.3 72.39 0) (effects (font (size 1.27 1.27))) (hide yes))
+  (property "Footprint" "Resistor_SMD:R_0201_0603Metric" (at 368.3 72.39 0) (effects (font (size 1.27 1.27))) (hide yes))
+  (property "Datasheet" "https://yageogroup.com/en/ProductSearch/PartNumberSearch?part=RC0201FR-07100KL" (at 368.3 72.39 0) (effects (font (size 1.27 1.27))) (hide yes))
+  (property "Description" "Resistor, 100 kΩ, 1 %, 1/20 W, 0201" (at 368.3 72.39 0) (effects (font (size 1.27 1.27))) (hide yes))
   (property "Manufacturer" "YAGEO" (at 368.3 72.39 0) (effects (font (size 1.27 1.27))) (hide yes))
-  (property "MPN" "RC0402FR-07100KL" (at 368.3 72.39 0) (effects (font (size 1.27 1.27))) (hide yes))
+  (property "MPN" "RC0201FR-07100KL" (at 368.3 72.39 0) (effects (font (size 1.27 1.27))) (hide yes))
   (property "Block" "blk.pmic" (at 368.3 72.39 0) (effects (font (size 1.27 1.27))) (hide yes))
   (pin "1")
@@
   (property "Reference" "R1104" (at 369.57 86.36 0) (effects (font (size 1.27 1.27)) (justify left)))
   (property "Value" "22 kΩ" (at 369.57 88.9 0) (effects (font (size 1.27 1.27)) (justify left)))
-  (property "Footprint" "Resistor_SMD:R_0402_1005Metric" (at 368.3 87.63 0) (effects (font (size 1.27 1.27))) (hide yes))
-  (property "Datasheet" "https://yageogroup.com/en/ProductSearch/PartNumberSearch?part=RC0402FR-0722KL" (at 368.3 87.63 0) (effects (font (size 1.27 1.27))) (hide yes))
-  (property "Description" "Resistor, 22 kΩ, 1 %, 1/16 W, 0402" (at 368.3 87.63 0) (effects (font (size 1.27 1.27))) (hide yes))
+  (property "Footprint" "Resistor_SMD:R_0201_0603Metric" (at 368.3 87.63 0) (effects (font (size 1.27 1.27))) (hide yes))
+  (property "Datasheet" "https://yageogroup.com/en/ProductSearch/PartNumberSearch?part=RC0201FR-0722KL" (at 368.3 87.63 0) (effects (font (size 1.27 1.27))) (hide yes))
+  (property "Description" "Resistor, 22 kΩ, 1 %, 1/20 W, 0201" (at 368.3 87.63 0) (effects (font (size 1.27 1.27))) (hide yes))
   (property "Manufacturer" "YAGEO" (at 368.3 87.63 0) (effects (font (size 1.27 1.27))) (hide yes))
-  (property "MPN" "RC0402FR-0722KL" (at 368.3 87.63 0) (effects (font (size 1.27 1.27))) (hide yes))
+  (property "MPN" "RC0201FR-0722KL" (at 368.3 87.63 0) (effects (font (size 1.27 1.27))) (hide yes))
   (property "Block" "blk.pmic" (at 368.3 87.63 0) (effects (font (size 1.27 1.27))) (hide yes))
   (pin "1")
@@
   (property "Reference" "C1115" (at 383.54 86.36 0) (effects (font (size 1.27 1.27)) (justify left)))
   (property "Value" "100 nF" (at 383.54 88.9 0) (effects (font (size 1.27 1.27)) (justify left)))
-  (property "Footprint" "Capacitor_SMD:C_0402_1005Metric" (at 381 87.63 0) (effects (font (size 1.27 1.27))) (hide yes))
-  (property "Datasheet" "https://www.murata.com/en-us/products/productdetail?partno=GRM155R71C104KA88D" (at 381 87.63 0) (effects (font (size 1.27 1.27))) (hide yes))
-  (property "Description" "Capacitor, 100 nF, 16 V, X7R, 0402" (at 381 87.63 0) (effects (font (size 1.27 1.27))) (hide yes))
+  (property "Footprint" "Capacitor_SMD:C_0201_0603Metric" (at 381 87.63 0) (effects (font (size 1.27 1.27))) (hide yes))
+  (property "Datasheet" "https://www.murata.com/en-us/products/productdetail?partno=GRM033R61A104KE15D" (at 381 87.63 0) (effects (font (size 1.27 1.27))) (hide yes))
+  (property "Description" "Capacitor, 100 nF, 10 V, X5R, 0201" (at 381 87.63 0) (effects (font (size 1.27 1.27))) (hide yes))
   (property "Manufacturer" "Murata" (at 381 87.63 0) (effects (font (size 1.27 1.27))) (hide yes))
-  (property "MPN" "GRM155R71C104KA88D" (at 381 87.63 0) (effects (font (size 1.27 1.27))) (hide yes))
+  (property "MPN" "GRM033R61A104KE15D" (at 381 87.63 0) (effects (font (size 1.27 1.27))) (hide yes))
   (property "Block" "blk.pmic" (at 381 87.63 0) (effects (font (size 1.27 1.27))) (hide yes))
   (pin "1")

Commit message: BOM v1.18 item 2: successors of the discontinued 1 uF 0402
GRM155R61A105KE15D is to be discontinued. 44 positions take
GRM155C71A105KE11D (1 uF 10 V X7S); the eight TPS7A20 positions take
GRM155R61C225KE11D (2.2 uF 16 V X5R) to keep the 0.47 uF effective
minimum with 10 % to spare at up to 3.8 V. Same land; sourcing pass.
Closes BOM §7 item 52; new item 55 lists the other capture parts outside
Murata's product data or near end of life.

Co-Authored-By: Claude Opus 5.5 <noreply@anthropic.com>
Claude-Session: https://claude.ai/code/session_01Ei262h3TpgY9vyfNLMi5Mn
Parts:
- C1110, C1111, C1112, C1113, C1122, C1123, C1124, C1125, C1126, C1127, C1128, C1129, C1130, C1131, C1132, C1133, C1134, C1135: MPN GRM155R61A105KE15D -> GRM155C71A105KE11D

Commit message: Placement v1.3: capacitor proximity rule, checked and met
pcb/proximity.py assigns every converter's input and output capacitors
(from pin functions and types) and every IC's decoupling (block rule and
the generator's new Decoupling field) and checks each within its bound
of the pins it serves (input 3, output 5, decoupling 4, bulk 6 mm); the
build fails otherwise. The placer places each IC's capacitors right
after it, keeps room for them, reorders, swaps and repairs; a search
radius bug (mm used as cells) that blocked rotations is fixed. RK809
moved 1.2 mm right and 1.1 mm down off the radio zone edge.

Fixes found: C901 was 29 mm from U901; 136 of 237 capacitors were beyond
their bound. Now 248 checked, none beyond. BOM v1.18 items 3 (revised:
3 x GRM219R61C226ME15L per LDO position), 5 (C4403 as 2 x 0805) and 6.
Tests: test_proximity (6).

Co-Authored-By: Claude Opus 5.5 <noreply@anthropic.com>
Claude-Session: https://claude.ai/code/session_01Ei262h3TpgY9vyfNLMi5Mn
Parts:
- C1116, C1117, C1118, C1119, C1120: Decoupling (none) -> VSYS_LV
- C1121, C1122, C1123, C1124, C1125: Decoupling (none) -> vcc3v3_sys
- C1126: Decoupling (none) -> vdda0v9_image
- C1127: Decoupling (none) -> vdda_0v9
- C1128: Decoupling (none) -> vdda0v9_pmu
- C1129: Decoupling (none) -> FP_VCI_SRC
- C1130: Decoupling (none) -> vccio_sd
- C1131: Decoupling (none) -> vcc3v3_pmu
- C1132: Decoupling (none) -> vcca_1v8
- C1133: Decoupling (none) -> vcca1v8_pmu
- C1134: Decoupling (none) -> vcca1v8_image
- C1135: Decoupling (none) -> vcc3v3_sd
Changed lines of the file:
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@@
   (property "MPN" "GRM188R61A106KE69D" (at 33.02 219.71 0) (effects (font (size 1.27 1.27))) (hide yes))
   (property "Block" "blk.pmic" (at 33.02 219.71 0) (effects (font (size 1.27 1.27))) (hide yes))
+  (property "Decoupling" "VSYS_LV" (at 33.02 219.71 0) (effects (font (size 1.27 1.27))) (hide yes))
   (pin "1")
   (pin "2")
@@
   (property "MPN" "GRM188R61A106KE69D" (at 48.26 219.71 0) (effects (font (size 1.27 1.27))) (hide yes))
   (property "Block" "blk.pmic" (at 48.26 219.71 0) (effects (font (size 1.27 1.27))) (hide yes))
+  (property "Decoupling" "VSYS_LV" (at 48.26 219.71 0) (effects (font (size 1.27 1.27))) (hide yes))
   (pin "1")
   (pin "2")
@@
   (property "MPN" "GRM188R61A106KE69D" (at 63.5 219.71 0) (effects (font (size 1.27 1.27))) (hide yes))
   (property "Block" "blk.pmic" (at 63.5 219.71 0) (effects (font (size 1.27 1.27))) (hide yes))
+  (property "Decoupling" "VSYS_LV" (at 63.5 219.71 0) (effects (font (size 1.27 1.27))) (hide yes))
   (pin "1")
   (pin "2")
@@
   (property "MPN" "GRM188R61A106KE69D" (at 78.74 219.71 0) (effects (font (size 1.27 1.27))) (hide yes))
   (property "Block" "blk.pmic" (at 78.74 219.71 0) (effects (font (size 1.27 1.27))) (hide yes))
+  (property "Decoupling" "VSYS_LV" (at 78.74 219.71 0) (effects (font (size 1.27 1.27))) (hide yes))
   (pin "1")
   (pin "2")
@@
   (property "MPN" "GRM188R61A106KE69D" (at 93.98 219.71 0) (effects (font (size 1.27 1.27))) (hide yes))
   (property "Block" "blk.pmic" (at 93.98 219.71 0) (effects (font (size 1.27 1.27))) (hide yes))
+  (property "Decoupling" "VSYS_LV" (at 93.98 219.71 0) (effects (font (size 1.27 1.27))) (hide yes))
   (pin "1")
   (pin "2")
@@
   (property "MPN" "GRM188R61A106KE69D" (at 109.22 219.71 0) (effects (font (size 1.27 1.27))) (hide yes))
   (property "Block" "blk.pmic" (at 109.22 219.71 0) (effects (font (size 1.27 1.27))) (hide yes))
+  (property "Decoupling" "vcc3v3_sys" (at 109.22 219.71 0) (effects (font (size 1.27 1.27))) (hide yes))
   (pin "1")
   (pin "2")
@@
   (property "MPN" "GRM155C71A105KE11D" (at 124.46 219.71 0) (effects (font (size 1.27 1.27))) (hide yes))
   (property "Block" "blk.pmic" (at 124.46 219.71 0) (effects (font (size 1.27 1.27))) (hide yes))
+  (property "Decoupling" "vcc3v3_sys" (at 124.46 219.71 0) (effects (font (size 1.27 1.27))) (hide yes))
   (pin "1")
   (pin "2")
@@
   (property "MPN" "GRM155C71A105KE11D" (at 139.7 219.71 0) (effects (font (size 1.27 1.27))) (hide yes))
   (property "Block" "blk.pmic" (at 139.7 219.71 0) (effects (font (size 1.27 1.27))) (hide yes))
+  (property "Decoupling" "vcc3v3_sys" (at 139.7 219.71 0) (effects (font (size 1.27 1.27))) (hide yes))
   (pin "1")
   (pin "2")
@@
   (property "MPN" "GRM155C71A105KE11D" (at 154.94 219.71 0) (effects (font (size 1.27 1.27))) (hide yes))
   (property "Block" "blk.pmic" (at 154.94 219.71 0) (effects (font (size 1.27 1.27))) (hide yes))
+  (property "Decoupling" "vcc3v3_sys" (at 154.94 219.71 0) (effects (font (size 1.27 1.27))) (hide yes))
   (pin "1")
   (pin "2")
@@
   (property "MPN" "GRM155C71A105KE11D" (at 170.18 219.71 0) (effects (font (size 1.27 1.27))) (hide yes))
   (property "Block" "blk.pmic" (at 170.18 219.71 0) (effects (font (size 1.27 1.27))) (hide yes))
+  (property "Decoupling" "vcc3v3_sys" (at 170.18 219.71 0) (effects (font (size 1.27 1.27))) (hide yes))
   (pin "1")
   (pin "2")
@@
   (property "MPN" "GRM155C71A105KE11D" (at 223.52 181.61 0) (effects (font (size 1.27 1.27))) (hide yes))
   (property "Block" "blk.pmic" (at 223.52 181.61 0) (effects (font (size 1.27 1.27))) (hide yes))
+  (property "Decoupling" "vdda0v9_image" (at 223.52 181.61 0) (effects (font (size 1.27 1.27))) (hide yes))
   (pin "1")
   (pin "2")
@@
   (property "MPN" "GRM155C71A105KE11D" (at 241.3 181.61 0) (effects (font (size 1.27 1.27))) (hide yes))
   (property "Block" "blk.pmic" (at 241.3 181.61 0) (effects (font (size 1.27 1.27))) (hide yes))
+  (property "Decoupling" "vdda_0v9" (at 241.3 181.61 0) (effects (font (size 1.27 1.27))) (hide yes))
   (pin "1")
   (pin "2")
@@
   (property "MPN" "GRM155C71A105KE11D" (at 259.08 181.61 0) (effects (font (size 1.27 1.27))) (hide yes))
   (property "Block" "blk.pmic" (at 259.08 181.61 0) (effects (font (size 1.27 1.27))) (hide yes))
+  (property "Decoupling" "vdda0v9_pmu" (at 259.08 181.61 0) (effects (font (size 1.27 1.27))) (hide yes))
   (pin "1")
   (pin "2")
@@
   (property "MPN" "GRM155C71A105KE11D" (at 276.86 181.61 0) (effects (font (size 1.27 1.27))) (hide yes))
   (property "Block" "blk.pmic" (at 276.86 181.61 0) (effects (font (size 1.27 1.27))) (hide yes))
+  (property "Decoupling" "FP_VCI_SRC" (at 276.86 181.61 0) (effects (font (size 1.27 1.27))) (hide yes))
   (pin "1")
   (pin "2")
@@
   (property "MPN" "GRM155C71A105KE11D" (at 294.64 181.61 0) (effects (font (size 1.27 1.27))) (hide yes))
   (property "Block" "blk.pmic" (at 294.64 181.61 0) (effects (font (size 1.27 1.27))) (hide yes))
+  (property "Decoupling" "vccio_sd" (at 294.64 181.61 0) (effects (font (size 1.27 1.27))) (hide yes))
   (pin "1")
   (pin "2")
@@
   (property "MPN" "GRM155C71A105KE11D" (at 312.42 181.61 0) (effects (font (size 1.27 1.27))) (hide yes))
   (property "Block" "blk.pmic" (at 312.42 181.61 0) (effects (font (size 1.27 1.27))) (hide yes))
+  (property "Decoupling" "vcc3v3_pmu" (at 312.42 181.61 0) (effects (font (size 1.27 1.27))) (hide yes))
   (pin "1")
   (pin "2")
@@
   (property "MPN" "GRM155C71A105KE11D" (at 330.2 181.61 0) (effects (font (size 1.27 1.27))) (hide yes))
   (property "Block" "blk.pmic" (at 330.2 181.61 0) (effects (font (size 1.27 1.27))) (hide yes))
+  (property "Decoupling" "vcca_1v8" (at 330.2 181.61 0) (effects (font (size 1.27 1.27))) (hide yes))
   (pin "1")
   (pin "2")
@@
   (property "MPN" "GRM155C71A105KE11D" (at 347.98 181.61 0) (effects (font (size 1.27 1.27))) (hide yes))
   (property "Block" "blk.pmic" (at 347.98 181.61 0) (effects (font (size 1.27 1.27))) (hide yes))
+  (property "Decoupling" "vcca1v8_pmu" (at 347.98 181.61 0) (effects (font (size 1.27 1.27))) (hide yes))
   (pin "1")
   (pin "2")
@@
   (property "MPN" "GRM155C71A105KE11D" (at 365.76 181.61 0) (effects (font (size 1.27 1.27))) (hide yes))
   (property "Block" "blk.pmic" (at 365.76 181.61 0) (effects (font (size 1.27 1.27))) (hide yes))
+  (property "Decoupling" "vcca1v8_image" (at 365.76 181.61 0) (effects (font (size 1.27 1.27))) (hide yes))
   (pin "1")
   (pin "2")
@@
   (property "MPN" "GRM155C71A105KE11D" (at 383.54 181.61 0) (effects (font (size 1.27 1.27))) (hide yes))
   (property "Block" "blk.pmic" (at 383.54 181.61 0) (effects (font (size 1.27 1.27))) (hide yes))
-  (pin "1")
-  (pin "2")
+  (property "Decoupling" "vcc3v3_sd" (at 383.54 181.61 0) (effects (font (size 1.27 1.27))) (hide yes))
+  (pin "1")
+  (pin "2")
