File: board/hardware/t1-main-board/radio-module.kicad_sch (KiCad schematic)
At the start: 11 parts, among them U4601 LBES5PL2EL-923

Commit message: Board: capture blk.current-monitors
Five INA236 on I2C1 (0x40-0x43, 0x48) with their shunts, per power tree
§4.12 and BOM v1 lines 54 and 136. The measured branches are rails of
their own (VSYS_SRC, VSYS_LV_AUDIO, VSYS_AUDIO, VSYS_LV_BL, VSYS_P5V1),
fed through the shunts on this sheet; the charger, audio, backlight and
5.1 V sheets take them. The root's layout may leave a stack level empty,
so the block sits under the notes; IC bboxes hold turned rail values;
passive rows hold a bottom rail's text.

Co-Authored-By: Claude Opus 5.5 <noreply@anthropic.com>
Claude-Session: https://claude.ai/code/session_01Ei262h3TpgY9vyfNLMi5Mn
Parts:
- removed C4601, C4602, C4603: 10 µF, Capacitor_SMD:C_0603_1608Metric, symbol Device:C
- removed C4604: 100 nF, Capacitor_SMD:C_0402_1005Metric, symbol Device:C
- removed R4601, R4602, R4603, R4604, R4605, R4606: 0 Ω, Resistor_SMD:R_0402_1005Metric, symbol Device:R
- removed U4601: LBES5PL2EL-923, Murata:Murata_Type2EL_LGA-107_8.8x7.7mm, symbol Murata:LBES5PL2EL-923
- added C4701, C4702, C4703: 10 µF, Capacitor_SMD:C_0603_1608Metric, symbol Device:C
- added C4704: 100 nF, Capacitor_SMD:C_0402_1005Metric, symbol Device:C
- added R4701, R4702, R4703, R4704, R4705, R4706: 0 Ω, Resistor_SMD:R_0402_1005Metric, symbol Device:R
- added U4701: LBES5PL2EL-923, Murata:Murata_Type2EL_LGA-107_8.8x7.7mm, symbol Murata:LBES5PL2EL-923
Connections:
- net BT_UART_CTS: now also U4701.50 (UART_CTS)
- net BT_UART_RTS: now also U4701.52 (UART_RTS)
- net BT_UART_RXD: now also U4701.51 (UART_RX)
- net BT_UART_TXD: now also U4701.49 (UART_TX)
- net BT_WAKE_IN: now also U4701.75 (BT15.4_WAKE_IN)
- net BT_WAKE_OUT: now also U4701.76 (BT15.4_WAKE_OUT)
- net GND: now also C4701.2, C4702.2, C4703.2, C4704.2, U4701.1 (GND), U4701.100 (GND), U4701.101 (GND), U4701.102 (GND), U4701.103 (GND), U4701.104 (GND), U4701.105 (GND), U4701.106 (GND), U4701.107 (GND), U4701.11 (GND), U4701.14 (GND), U4701.16 (GND), U4701.17 (GND), U4701.19 (GND), U4701.2 (GND), U4701.20 (GND), U4701.21 (GND), U4701.22 (GND), U4701.28 (GND), U4701.29 (GND), U4701.32 (GND), U4701.39 (GND), U4701.41 (GND), U4701.43 (GND), U4701.53 (GND), U4701.62 (GND), U4701.67 (GND), U4701.68 (GND), U4701.71 (GND), U4701.81 (GND), U4701.82 (GND), U4701.83 (GND), U4701.84 (GND), U4701.85 (GND), U4701.86 (GND), U4701.87 (GND), U4701.88 (GND), U4701.89 (GND), U4701.9 (GND), U4701.90 (GND), U4701.91 (GND), U4701.92 (GND), U4701.93 (GND), U4701.94 (GND), U4701.95 (GND), U4701.96 (GND), U4701.97 (GND), U4701.98 (GND), U4701.99 (GND)
- net WL_ANT0: now also U4701.15 (ANT0)
- net WL_ANT1: now also U4701.23 (ANT1)
- net WL_BT_IN: now also U4701.18 (BT_15.4_IN)
- net WL_PD_N: now also U4701.10 (PDn)
- net WL_SD_CLK: now also R4702.1
- net WL_SD_CLK_M: now also R4702.2, U4701.44 (SD_CLK)
- net WL_SD_CMD: now also R4701.1
- net WL_SD_CMD_M: now also R4701.2, U4701.42 (SD_CMD)
- net WL_SD_D0: now also R4703.1
- net WL_SD_D0_M: now also R4703.2, U4701.48 (SD_DAT[0])
- net WL_SD_D1: now also R4704.1
- net WL_SD_D1_M: now also R4704.2, U4701.45 (SD_DAT[1])
- net WL_SD_D2: now also R4705.1
- net WL_SD_D2_M: now also R4705.2, U4701.47 (SD_DAT[2])
- net WL_SD_D3: now also R4706.1
- net WL_SD_D3_M: now also R4706.2, U4701.46 (SD_DAT[3])
- net WL_WAKE_OUT: now also U4701.73 (WL_WAKE_OUT)
- net vcc1v8_wl: now also C4702.1, U4701.30 (AVDD18_2), U4701.31 (AVDD18_1)
- net vcc3v3_wl: now also C4701.1, U4701.12 (AVDD33_1), U4701.13 (AVDD33_2)
- net vcc_1v8: now also C4703.1, C4704.1, U4701.40 (SD_VIO), U4701.54 (VIO), U4701.55 (CONFIG_HOST[0]), U4701.56 (CONFIG_HOST[1])

Commit message: Board: capture blk.debug
Debug UART2 (1.8 V) and I2S/DSD pads with ground pads, reset, PMIC and
power-key pads (PCB-T-09), a pad on every spare SoC GPIO whose pinout v1
row names one (the DEBUG bus, on the SoC's right edge), and a rail pad
for each power-tree rail no other sheet probes (PCB-T-02). Each DAC
sheet carries a pad on its MCLK. The spares pinout v1 leaves without a
pad now carry no-connect flags. On the root, facing sheet pins are
joined directly only where the route meets no other symbol.

Co-Authored-By: Claude Opus 5.5 <noreply@anthropic.com>
Claude-Session: https://claude.ai/code/session_01Ei262h3TpgY9vyfNLMi5Mn
Parts:
- removed C4701, C4702, C4703: 10 µF, Capacitor_SMD:C_0603_1608Metric, symbol Device:C
- removed C4704: 100 nF, Capacitor_SMD:C_0402_1005Metric, symbol Device:C
- removed R4701, R4702, R4703, R4704, R4705, R4706: 0 Ω, Resistor_SMD:R_0402_1005Metric, symbol Device:R
- removed U4701: LBES5PL2EL-923, Murata:Murata_Type2EL_LGA-107_8.8x7.7mm, symbol Murata:LBES5PL2EL-923
- added C4801, C4802, C4803: 10 µF, Capacitor_SMD:C_0603_1608Metric, symbol Device:C
- added C4804: 100 nF, Capacitor_SMD:C_0402_1005Metric, symbol Device:C
- added R4801, R4802, R4803, R4804, R4805, R4806: 0 Ω, Resistor_SMD:R_0402_1005Metric, symbol Device:R
- added U4801: LBES5PL2EL-923, Murata:Murata_Type2EL_LGA-107_8.8x7.7mm, symbol Murata:LBES5PL2EL-923
Connections:
- net BT_UART_CTS: now also U4801.50 (UART_CTS)
- net BT_UART_RTS: now also U4801.52 (UART_RTS)
- net BT_UART_RXD: now also U4801.51 (UART_RX)
- net BT_UART_TXD: now also U4801.49 (UART_TX)
- net BT_WAKE_IN: now also U4801.75 (BT15.4_WAKE_IN)
- net BT_WAKE_OUT: now also U4801.76 (BT15.4_WAKE_OUT)
- net GND: now also C4801.2, C4802.2, C4803.2, C4804.2, U4801.1 (GND), U4801.100 (GND), U4801.101 (GND), U4801.102 (GND), U4801.103 (GND), U4801.104 (GND), U4801.105 (GND), U4801.106 (GND), U4801.107 (GND), U4801.11 (GND), U4801.14 (GND), U4801.16 (GND), U4801.17 (GND), U4801.19 (GND), U4801.2 (GND), U4801.20 (GND), U4801.21 (GND), U4801.22 (GND), U4801.28 (GND), U4801.29 (GND), U4801.32 (GND), U4801.39 (GND), U4801.41 (GND), U4801.43 (GND), U4801.53 (GND), U4801.62 (GND), U4801.67 (GND), U4801.68 (GND), U4801.71 (GND), U4801.81 (GND), U4801.82 (GND), U4801.83 (GND), U4801.84 (GND), U4801.85 (GND), U4801.86 (GND), U4801.87 (GND), U4801.88 (GND), U4801.89 (GND), U4801.9 (GND), U4801.90 (GND), U4801.91 (GND), U4801.92 (GND), U4801.93 (GND), U4801.94 (GND), U4801.95 (GND), U4801.96 (GND), U4801.97 (GND), U4801.98 (GND), U4801.99 (GND)
- net WL_ANT0: now also U4801.15 (ANT0)
- net WL_ANT1: now also U4801.23 (ANT1)
- net WL_BT_IN: now also U4801.18 (BT_15.4_IN)
- net WL_PD_N: now also U4801.10 (PDn)
- net WL_SD_CLK: now also R4802.1
- net WL_SD_CLK_M: now also R4802.2, U4801.44 (SD_CLK)
- net WL_SD_CMD: now also R4801.1
- net WL_SD_CMD_M: now also R4801.2, U4801.42 (SD_CMD)
- net WL_SD_D0: now also R4803.1
- net WL_SD_D0_M: now also R4803.2, U4801.48 (SD_DAT[0])
- net WL_SD_D1: now also R4804.1
- net WL_SD_D1_M: now also R4804.2, U4801.45 (SD_DAT[1])
- net WL_SD_D2: now also R4805.1
- net WL_SD_D2_M: now also R4805.2, U4801.47 (SD_DAT[2])
- net WL_SD_D3: now also R4806.1
- net WL_SD_D3_M: now also R4806.2, U4801.46 (SD_DAT[3])
- net WL_WAKE_OUT: now also U4801.73 (WL_WAKE_OUT)
- net vcc1v8_wl: now also C4802.1, U4801.30 (AVDD18_2), U4801.31 (AVDD18_1)
- net vcc3v3_wl: now also C4801.1, U4801.12 (AVDD33_1), U4801.13 (AVDD33_2)
- net vcc_1v8: now also C4803.1, C4804.1, U4801.40 (SD_VIO), U4801.54 (VIO), U4801.55 (CONFIG_HOST[0]), U4801.56 (CONFIG_HOST[1])

Commit message: Board: capture blk.mic-ambient and links #34, #35
IM73D122 on PDM CLK1 and SDI1 (BOM v1 line 34, pinout v1 AK2 and 1P2),
LR to ground, 22 Ω clock series, VDD from MIC_1V8 through link #35.
Link #34 on blk.mic-main makes the faceplate branch the rail MIC_1V8_FP
for contact 40 (power tree §4.12, G10). kicad-lib moves to e46bda4 for
the IM73D122, TPS3808G01, SN74LVC1G58 and BAT54 parts.

Co-Authored-By: Claude Opus 5.5 <noreply@anthropic.com>
Claude-Session: https://claude.ai/code/session_01Ei262h3TpgY9vyfNLMi5Mn
Parts:
- removed C4801, C4802, C4803: 10 µF, Capacitor_SMD:C_0603_1608Metric, symbol Device:C
- removed C4804: 100 nF, Capacitor_SMD:C_0402_1005Metric, symbol Device:C
- removed R4801, R4802, R4803, R4804, R4805, R4806: 0 Ω, Resistor_SMD:R_0402_1005Metric, symbol Device:R
- removed U4801: LBES5PL2EL-923, Murata:Murata_Type2EL_LGA-107_8.8x7.7mm, symbol Murata:LBES5PL2EL-923
- added C4901, C4902, C4903: 10 µF, Capacitor_SMD:C_0603_1608Metric, symbol Device:C
- added C4904: 100 nF, Capacitor_SMD:C_0402_1005Metric, symbol Device:C
- added R4901, R4902, R4903, R4904, R4905, R4906: 0 Ω, Resistor_SMD:R_0402_1005Metric, symbol Device:R
- added U4901: LBES5PL2EL-923, Murata:Murata_Type2EL_LGA-107_8.8x7.7mm, symbol Murata:LBES5PL2EL-923
Connections:
- net BT_UART_CTS: now also U4901.50 (UART_CTS)
- net BT_UART_RTS: now also U4901.52 (UART_RTS)
- net BT_UART_RXD: now also U4901.51 (UART_RX)
- net BT_UART_TXD: now also U4901.49 (UART_TX)
- net BT_WAKE_IN: now also U4901.75 (BT15.4_WAKE_IN)
- net BT_WAKE_OUT: now also U4901.76 (BT15.4_WAKE_OUT)
- net GND: now also C4901.2, C4902.2, C4903.2, C4904.2, U4901.1 (GND), U4901.100 (GND), U4901.101 (GND), U4901.102 (GND), U4901.103 (GND), U4901.104 (GND), U4901.105 (GND), U4901.106 (GND), U4901.107 (GND), U4901.11 (GND), U4901.14 (GND), U4901.16 (GND), U4901.17 (GND), U4901.19 (GND), U4901.2 (GND), U4901.20 (GND), U4901.21 (GND), U4901.22 (GND), U4901.28 (GND), U4901.29 (GND), U4901.32 (GND), U4901.39 (GND), U4901.41 (GND), U4901.43 (GND), U4901.53 (GND), U4901.62 (GND), U4901.67 (GND), U4901.68 (GND), U4901.71 (GND), U4901.81 (GND), U4901.82 (GND), U4901.83 (GND), U4901.84 (GND), U4901.85 (GND), U4901.86 (GND), U4901.87 (GND), U4901.88 (GND), U4901.89 (GND), U4901.9 (GND), U4901.90 (GND), U4901.91 (GND), U4901.92 (GND), U4901.93 (GND), U4901.94 (GND), U4901.95 (GND), U4901.96 (GND), U4901.97 (GND), U4901.98 (GND), U4901.99 (GND)
- net WL_ANT0: now also U4901.15 (ANT0)
- net WL_ANT1: now also U4901.23 (ANT1)
- net WL_BT_IN: now also U4901.18 (BT_15.4_IN)
- net WL_PD_N: now also U4901.10 (PDn)
- net WL_SD_CLK: now also R4902.1
- net WL_SD_CLK_M: now also R4902.2, U4901.44 (SD_CLK)
- net WL_SD_CMD: now also R4901.1
- net WL_SD_CMD_M: now also R4901.2, U4901.42 (SD_CMD)
- net WL_SD_D0: now also R4903.1
- net WL_SD_D0_M: now also R4903.2, U4901.48 (SD_DAT[0])
- net WL_SD_D1: now also R4904.1
- net WL_SD_D1_M: now also R4904.2, U4901.45 (SD_DAT[1])
- net WL_SD_D2: now also R4905.1
- net WL_SD_D2_M: now also R4905.2, U4901.47 (SD_DAT[2])
- net WL_SD_D3: now also R4906.1
- net WL_SD_D3_M: now also R4906.2, U4901.46 (SD_DAT[3])
- net WL_WAKE_OUT: now also U4901.73 (WL_WAKE_OUT)
- net vcc1v8_wl: now also C4902.1, U4901.30 (AVDD18_2), U4901.31 (AVDD18_1)
- net vcc3v3_wl: now also C4901.1, U4901.12 (AVDD33_1), U4901.13 (AVDD33_2)
- net vcc_1v8: now also C4903.1, C4904.1, U4901.40 (SD_VIO), U4901.54 (VIO), U4901.55 (CONFIG_HOST[0]), U4901.56 (CONFIG_HOST[1])

Commit message: Board: capture blk.maskrom
Power + Vol- at a cold power-on pull eMMC D0 low inside the TPS3808G01
boot window (BOM v1 lines 35, 78, 97, 98; sim/maskrom): SENSE 280k/100k,
CT 390 nF, WINDOW_N with its pad, SN74LVC1G57 and SN74LVC1G58 on
vcca1v8_pmu, BAT54 from PWRON_N, DMG1012T through 1 kΩ to EMMC_D0.
Every block in use now has its sheet; the README states the remaining
single-pin nets.

Co-Authored-By: Claude Opus 5.5 <noreply@anthropic.com>
Claude-Session: https://claude.ai/code/session_01Ei262h3TpgY9vyfNLMi5Mn
Parts:
- removed C4901, C4902, C4903: 10 µF, Capacitor_SMD:C_0603_1608Metric, symbol Device:C
- removed C4904: 100 nF, Capacitor_SMD:C_0402_1005Metric, symbol Device:C
- removed R4901, R4902, R4903, R4904, R4905, R4906: 0 Ω, Resistor_SMD:R_0402_1005Metric, symbol Device:R
- removed U4901: LBES5PL2EL-923, Murata:Murata_Type2EL_LGA-107_8.8x7.7mm, symbol Murata:LBES5PL2EL-923
- added C5001, C5002, C5003: 10 µF, Capacitor_SMD:C_0603_1608Metric, symbol Device:C
- added C5004: 100 nF, Capacitor_SMD:C_0402_1005Metric, symbol Device:C
- added R5001, R5002, R5003, R5004, R5005, R5006: 0 Ω, Resistor_SMD:R_0402_1005Metric, symbol Device:R
- added U5001: LBES5PL2EL-923, Murata:Murata_Type2EL_LGA-107_8.8x7.7mm, symbol Murata:LBES5PL2EL-923
Connections:
- net BT_UART_CTS: now also U5001.50 (UART_CTS)
- net BT_UART_RTS: now also U5001.52 (UART_RTS)
- net BT_UART_RXD: now also U5001.51 (UART_RX)
- net BT_UART_TXD: now also U5001.49 (UART_TX)
- net BT_WAKE_IN: now also U5001.75 (BT15.4_WAKE_IN)
- net BT_WAKE_OUT: now also U5001.76 (BT15.4_WAKE_OUT)
- net GND: now also C5001.2, C5002.2, C5003.2, C5004.2, U5001.1 (GND), U5001.100 (GND), U5001.101 (GND), U5001.102 (GND), U5001.103 (GND), U5001.104 (GND), U5001.105 (GND), U5001.106 (GND), U5001.107 (GND), U5001.11 (GND), U5001.14 (GND), U5001.16 (GND), U5001.17 (GND), U5001.19 (GND), U5001.2 (GND), U5001.20 (GND), U5001.21 (GND), U5001.22 (GND), U5001.28 (GND), U5001.29 (GND), U5001.32 (GND), U5001.39 (GND), U5001.41 (GND), U5001.43 (GND), U5001.53 (GND), U5001.62 (GND), U5001.67 (GND), U5001.68 (GND), U5001.71 (GND), U5001.81 (GND), U5001.82 (GND), U5001.83 (GND), U5001.84 (GND), U5001.85 (GND), U5001.86 (GND), U5001.87 (GND), U5001.88 (GND), U5001.89 (GND), U5001.9 (GND), U5001.90 (GND), U5001.91 (GND), U5001.92 (GND), U5001.93 (GND), U5001.94 (GND), U5001.95 (GND), U5001.96 (GND), U5001.97 (GND), U5001.98 (GND), U5001.99 (GND)
- net WL_ANT0: now also U5001.15 (ANT0)
- net WL_ANT1: now also U5001.23 (ANT1)
- net WL_BT_IN: now also U5001.18 (BT_15.4_IN)
- net WL_PD_N: now also U5001.10 (PDn)
- net WL_SD_CLK: now also R5002.1
- net WL_SD_CLK_M: now also R5002.2, U5001.44 (SD_CLK)
- net WL_SD_CMD: now also R5001.1
- net WL_SD_CMD_M: now also R5001.2, U5001.42 (SD_CMD)
- net WL_SD_D0: now also R5003.1
- net WL_SD_D0_M: now also R5003.2, U5001.48 (SD_DAT[0])
- net WL_SD_D1: now also R5004.1
- net WL_SD_D1_M: now also R5004.2, U5001.45 (SD_DAT[1])
- net WL_SD_D2: now also R5005.1
- net WL_SD_D2_M: now also R5005.2, U5001.47 (SD_DAT[2])
- net WL_SD_D3: now also R5006.1
- net WL_SD_D3_M: now also R5006.2, U5001.46 (SD_DAT[3])
- net WL_WAKE_OUT: now also U5001.73 (WL_WAKE_OUT)
- net vcc1v8_wl: now also C5002.1, U5001.30 (AVDD18_2), U5001.31 (AVDD18_1)
- net vcc3v3_wl: now also C5001.1, U5001.12 (AVDD33_1), U5001.13 (AVDD33_2)
- net vcc_1v8: now also C5003.1, C5004.1, U5001.40 (SD_VIO), U5001.54 (VIO), U5001.55 (CONFIG_HOST[0]), U5001.56 (CONFIG_HOST[1])

Commit message: Compaction: lower inductors, 0201 decoupling, 0.8 mm signal test pads
A matrix tool (hardware/studies/compaction) checks each candidate against
the design's stresses: same inductance, design peak <= 70 % and the
converter's maximum limit <= 100 % of Isat (30 % drop), height zones,
ratings at least twice the rail, PCB-D-06; sourcing outcome per part.

Applied (placement v1 decision 12, BOM v1.15):
- L601, L4401: XGL4015-102MEC (1.5 mm) for XAL/XGL4020-102MEC (2.1 mm);
- L1001, L5101: XGL4015-471MEC (1.5 mm) for Wurth 744373240047, on the
  stock XxL4020 land (the Wurth land was never drawn);
- L1201 is 1.2 mm (XGL4012, per-MPN heights): it moves next to the SoC;
- 58 x 100 nF decoupling on rails <= 3.3 V in core/IO/radio: 0201;
- 51 test pads on signal nets: 0.8 mm (PCB-D-06 v0.16, JLCPCB guide).
Kept: L901, L2802 (XGL4015 at 103 % of Isat at the limit); no thinner
0805/1206 capacitor passes (obsolete, NRND or unlisted).

Board need 113 % -> 111 % (core band 227 -> 203 %, power band 258 ->
233 %, radio band 19 -> 0 %); only C904 still relies on PCB-Z-04.
ERC 0 errors, craft Q1 met, DRC 0 errors (605 warnings), pcb and study
tests pass, rules test board PASS.

Co-Authored-By: Claude Opus 5.5 <noreply@anthropic.com>
Claude-Session: https://claude.ai/code/session_01Ei262h3TpgY9vyfNLMi5Mn
Parts:
- C5004: footprint Capacitor_SMD:C_0402_1005Metric -> Capacitor_SMD:C_0201_0603Metric; MPN GRM155R71C104KA88D -> GRM033R61A104KE15D
Changed lines of the file:
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@@
   (property "Reference" "C5004" (at 91.44 180.34 0) (effects (font (size 1.27 1.27)) (justify left)))
   (property "Value" "100 nF" (at 91.44 182.88 0) (effects (font (size 1.27 1.27)) (justify left)))
-  (property "Footprint" "Capacitor_SMD:C_0402_1005Metric" (at 88.9 181.61 0) (effects (font (size 1.27 1.27))) (hide yes))
-  (property "Datasheet" "https://www.murata.com/en-us/products/productdetail?partno=GRM155R71C104KA88D" (at 88.9 181.61 0) (effects (font (size 1.27 1.27))) (hide yes))
-  (property "Description" "Capacitor, 100 nF, 16 V, X7R, 0402" (at 88.9 181.61 0) (effects (font (size 1.27 1.27))) (hide yes))
+  (property "Footprint" "Capacitor_SMD:C_0201_0603Metric" (at 88.9 181.61 0) (effects (font (size 1.27 1.27))) (hide yes))
+  (property "Datasheet" "https://www.murata.com/en-us/products/productdetail?partno=GRM033R61A104KE15D" (at 88.9 181.61 0) (effects (font (size 1.27 1.27))) (hide yes))
+  (property "Description" "Capacitor, 100 nF, 10 V, X5R, 0201" (at 88.9 181.61 0) (effects (font (size 1.27 1.27))) (hide yes))
   (property "Manufacturer" "Murata" (at 88.9 181.61 0) (effects (font (size 1.27 1.27))) (hide yes))
-  (property "MPN" "GRM155R71C104KA88D" (at 88.9 181.61 0) (effects (font (size 1.27 1.27))) (hide yes))
+  (property "MPN" "GRM033R61A104KE15D" (at 88.9 181.61 0) (effects (font (size 1.27 1.27))) (hide yes))
   (property "Block" "blk.radio-module" (at 88.9 181.61 0) (effects (font (size 1.27 1.27))) (hide yes))
   (pin "1")
