File: board/hardware/t1-main-board/radio-module.kicad_sch (KiCad schematic)
At the start: 11 parts, among them U5001 LBES5PL2EL-923

Commit message: Board on libs v0.2.0: lower-case kebab vendor keys (HL-13)
The libs submodule moves to v0.2.0 (5f24483). Every library nickname in
the generator, the placement tool and the floorplan study follows the
key table (Texas_Instruments -> texas-instruments, OpenDAP_Device ->
opendap-generic, Rockchip and Rockchip_PMIC -> rockchip, ...); the
library tables are written from the files. Schematic and board
regenerated.

Checks: ERC 0 errors (warnings unchanged); DRC 0 errors, 605 warnings,
the same counts by type, schematic parity 0; every placement identical;
craft Q1 met; pcb tests pass; STEP export resolves every libs 3D model
(the 27 parts without a model are KiCad stock lands that have none).

Co-Authored-By: Claude Opus 5.5 <noreply@anthropic.com>
Claude-Session: https://claude.ai/code/session_01Ei262h3TpgY9vyfNLMi5Mn
Parts:
- U5001: footprint Murata:Murata_Type2EL_LGA-107_8.8x7.7mm -> murata:Murata_Type2EL_LGA-107_8.8x7.7mm; symbol Murata:LBES5PL2EL-923 -> murata:LBES5PL2EL-923
Changed lines of the file:
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@@
 (paper "A3")
 (title_block (title "Radio: module") (date "2026-10-25") (rev "A") (company "The OpenDAP Project") (comment 1 "blk.radio-module") (comment 2 "Murata Type 2EL by unit, its decoupling and the SDIO series positions"))
-(symbol (lib_id "Murata:LBES5PL2EL-923") (at 43.18 78.74 0) (unit 1) (body_style 1) (exclude_from_sim no) (in_bom yes) (on_board yes) (dnp no)
+(symbol (lib_id "murata:LBES5PL2EL-923") (at 43.18 78.74 0) (unit 1) (body_style 1) (exclude_from_sim no) (in_bom yes) (on_board yes) (dnp no)
   (property "Reference" "U5001" (at 30.48 93.98 0) (effects (font (size 1.27 1.27)) (justify left)))
   (property "Value" "LBES5PL2EL-923" (at 30.48 91.44 0) (effects (font (size 1.27 1.27)) (justify left)))
-  (property "Footprint" "Murata:Murata_Type2EL_LGA-107_8.8x7.7mm" (at 43.18 78.74 0) (effects (font (size 1.27 1.27))) (hide yes))
+  (property "Footprint" "murata:Murata_Type2EL_LGA-107_8.8x7.7mm" (at 43.18 78.74 0) (effects (font (size 1.27 1.27))) (hide yes))
   (property "Datasheet" "https://www.murata.com/en-us/products/connectivitymodule/wi-fi-bluetooth/overview/lineup/type2el" (at 43.18 78.74 0) (effects (font (size 1.27 1.27))) (hide yes))
   (property "Description" "Murata Type 2EL module, NXP IW612: Wi-Fi 6 802.11a/b/g/n/ac/ax 1x1 2.4/5 GHz (SDIO 3.0), Bluetooth 5.4 BR/EDR/LE (UART, PCM), IEEE 802.15.4 (SPI), LGA-107 8.8 x 7.7 x 1.3 mm" (at 43.18 78.74 0) (effects (font (size 1.27 1.27))) (hide yes))
@@
   (instances (project "t1-main-board" (path "/7746052e-d7f9-59ad-ba73-bd2b74439529/afc06401-35b4-58d1-93ac-49cd5ed4743d/b6a27376-5f97-5e53-a107-ffdaf8725f86" (reference "#PWR0654") (unit 1))))
 )
-(symbol (lib_id "Murata:LBES5PL2EL-923") (at 100.33 81.28 0) (unit 2) (body_style 1) (exclude_from_sim no) (in_bom yes) (on_board yes) (dnp no)
+(symbol (lib_id "murata:LBES5PL2EL-923") (at 100.33 81.28 0) (unit 2) (body_style 1) (exclude_from_sim no) (in_bom yes) (on_board yes) (dnp no)
   (property "Reference" "U5001" (at 85.09 48.26 0) (effects (font (size 1.27 1.27)) (justify left)))
   (property "Value" "LBES5PL2EL-923" (at 85.09 45.72 0) (effects (font (size 1.27 1.27)) (justify left)))
-  (property "Footprint" "Murata:Murata_Type2EL_LGA-107_8.8x7.7mm" (at 100.33 81.28 0) (effects (font (size 1.27 1.27))) (hide yes))
+  (property "Footprint" "murata:Murata_Type2EL_LGA-107_8.8x7.7mm" (at 100.33 81.28 0) (effects (font (size 1.27 1.27))) (hide yes))
   (property "Datasheet" "https://www.murata.com/en-us/products/connectivitymodule/wi-fi-bluetooth/overview/lineup/type2el" (at 100.33 81.28 0) (effects (font (size 1.27 1.27))) (hide yes))
   (property "Description" "Murata Type 2EL module, NXP IW612: Wi-Fi 6 802.11a/b/g/n/ac/ax 1x1 2.4/5 GHz (SDIO 3.0), Bluetooth 5.4 BR/EDR/LE (UART, PCM), IEEE 802.15.4 (SPI), LGA-107 8.8 x 7.7 x 1.3 mm" (at 100.33 81.28 0) (effects (font (size 1.27 1.27))) (hide yes))
@@
 (no_connect (at 120.65 71.12))
 (no_connect (at 120.65 76.2))
-(symbol (lib_id "Murata:LBES5PL2EL-923") (at 160.02 63.5 0) (unit 3) (body_style 1) (exclude_from_sim no) (in_bom yes) (on_board yes) (dnp no)
+(symbol (lib_id "murata:LBES5PL2EL-923") (at 160.02 63.5 0) (unit 3) (body_style 1) (exclude_from_sim no) (in_bom yes) (on_board yes) (dnp no)
   (property "Reference" "U5001" (at 144.78 48.26 0) (effects (font (size 1.27 1.27)) (justify left)))
   (property "Value" "LBES5PL2EL-923" (at 144.78 45.72 0) (effects (font (size 1.27 1.27)) (justify left)))
-  (property "Footprint" "Murata:Murata_Type2EL_LGA-107_8.8x7.7mm" (at 160.02 63.5 0) (effects (font (size 1.27 1.27))) (hide yes))
+  (property "Footprint" "murata:Murata_Type2EL_LGA-107_8.8x7.7mm" (at 160.02 63.5 0) (effects (font (size 1.27 1.27))) (hide yes))
   (property "Datasheet" "https://www.murata.com/en-us/products/connectivitymodule/wi-fi-bluetooth/overview/lineup/type2el" (at 160.02 63.5 0) (effects (font (size 1.27 1.27))) (hide yes))
   (property "Description" "Murata Type 2EL module, NXP IW612: Wi-Fi 6 802.11a/b/g/n/ac/ax 1x1 2.4/5 GHz (SDIO 3.0), Bluetooth 5.4 BR/EDR/LE (UART, PCM), IEEE 802.15.4 (SPI), LGA-107 8.8 x 7.7 x 1.3 mm" (at 160.02 63.5 0) (effects (font (size 1.27 1.27))) (hide yes))
@@
 (no_connect (at 180.34 71.12))
 (no_connect (at 180.34 73.66))
-(symbol (lib_id "Murata:LBES5PL2EL-923") (at 240.03 66.04 0) (unit 4) (body_style 1) (exclude_from_sim no) (in_bom yes) (on_board yes) (dnp no)
+(symbol (lib_id "murata:LBES5PL2EL-923") (at 240.03 66.04 0) (unit 4) (body_style 1) (exclude_from_sim no) (in_bom yes) (on_board yes) (dnp no)
   (property "Reference" "U5001" (at 222.25 48.26 0) (effects (font (size 1.27 1.27)) (justify left)))
   (property "Value" "LBES5PL2EL-923" (at 222.25 45.72 0) (effects (font (size 1.27 1.27)) (justify left)))
-  (property "Footprint" "Murata:Murata_Type2EL_LGA-107_8.8x7.7mm" (at 240.03 66.04 0) (effects (font (size 1.27 1.27))) (hide yes))
+  (property "Footprint" "murata:Murata_Type2EL_LGA-107_8.8x7.7mm" (at 240.03 66.04 0) (effects (font (size 1.27 1.27))) (hide yes))
   (property "Datasheet" "https://www.murata.com/en-us/products/connectivitymodule/wi-fi-bluetooth/overview/lineup/type2el" (at 240.03 66.04 0) (effects (font (size 1.27 1.27))) (hide yes))
   (property "Description" "Murata Type 2EL module, NXP IW612: Wi-Fi 6 802.11a/b/g/n/ac/ax 1x1 2.4/5 GHz (SDIO 3.0), Bluetooth 5.4 BR/EDR/LE (UART, PCM), IEEE 802.15.4 (SPI), LGA-107 8.8 x 7.7 x 1.3 mm" (at 240.03 66.04 0) (effects (font (size 1.27 1.27))) (hide yes))
@@
 (wire (pts (xy 262.89 63.5) (xy 265.43 63.5)) (stroke (width 0) (type default)))
 (no_connect (at 262.89 68.58))
-(symbol (lib_id "Murata:LBES5PL2EL-923") (at 43.18 137.16 0) (unit 5) (body_style 1) (exclude_from_sim no) (in_bom yes) (on_board yes) (dnp no)
+(symbol (lib_id "murata:LBES5PL2EL-923") (at 43.18 137.16 0) (unit 5) (body_style 1) (exclude_from_sim no) (in_bom yes) (on_board yes) (dnp no)
   (property "Reference" "U5001" (at 35.56 124.46 0) (effects (font (size 1.27 1.27)) (justify left)))
   (property "Value" "LBES5PL2EL-923" (at 35.56 121.92 0) (effects (font (size 1.27 1.27)) (justify left)))
-  (property "Footprint" "Murata:Murata_Type2EL_LGA-107_8.8x7.7mm" (at 43.18 137.16 0) (effects (font (size 1.27 1.27))) (hide yes))
+  (property "Footprint" "murata:Murata_Type2EL_LGA-107_8.8x7.7mm" (at 43.18 137.16 0) (effects (font (size 1.27 1.27))) (hide yes))
   (property "Datasheet" "https://www.murata.com/en-us/products/connectivitymodule/wi-fi-bluetooth/overview/lineup/type2el" (at 43.18 137.16 0) (effects (font (size 1.27 1.27))) (hide yes))
   (property "Description" "Murata Type 2EL module, NXP IW612: Wi-Fi 6 802.11a/b/g/n/ac/ax 1x1 2.4/5 GHz (SDIO 3.0), Bluetooth 5.4 BR/EDR/LE (UART, PCM), IEEE 802.15.4 (SPI), LGA-107 8.8 x 7.7 x 1.3 mm" (at 43.18 137.16 0) (effects (font (size 1.27 1.27))) (hide yes))
@@
 (no_connect (at 55.88 142.24))
 (no_connect (at 55.88 144.78))
-(symbol (lib_id "Murata:LBES5PL2EL-923") (at 127 134.62 0) (unit 6) (body_style 1) (exclude_from_sim no) (in_bom yes) (on_board yes) (dnp no)
+(symbol (lib_id "murata:LBES5PL2EL-923") (at 127 134.62 0) (unit 6) (body_style 1) (exclude_from_sim no) (in_bom yes) (on_board yes) (dnp no)
   (property "Reference" "U5001" (at 63.5 124.46 0) (effects (font (size 1.27 1.27)) (justify left)))
   (property "Value" "LBES5PL2EL-923" (at 63.5 121.92 0) (effects (font (size 1.27 1.27)) (justify left)))
-  (property "Footprint" "Murata:Murata_Type2EL_LGA-107_8.8x7.7mm" (at 127 134.62 0) (effects (font (size 1.27 1.27))) (hide yes))
+  (property "Footprint" "murata:Murata_Type2EL_LGA-107_8.8x7.7mm" (at 127 134.62 0) (effects (font (size 1.27 1.27))) (hide yes))
   (property "Datasheet" "https://www.murata.com/en-us/products/connectivitymodule/wi-fi-bluetooth/overview/lineup/type2el" (at 127 134.62 0) (effects (font (size 1.27 1.27))) (hide yes))
   (property "Description" "Murata Type 2EL module, NXP IW612: Wi-Fi 6 802.11a/b/g/n/ac/ax 1x1 2.4/5 GHz (SDIO 3.0), Bluetooth 5.4 BR/EDR/LE (UART, PCM), IEEE 802.15.4 (SPI), LGA-107 8.8 x 7.7 x 1.3 mm" (at 127 134.62 0) (effects (font (size 1.27 1.27))) (hide yes))
