File: board/hardware/t1-main-board/status-led.kicad_sch (KiCad schematic)
At the start: 8 parts, among them U6201 LP5521YQX

Commit message: Board: capture blk.debug
Debug UART2 (1.8 V) and I2S/DSD pads with ground pads, reset, PMIC and
power-key pads (PCB-T-09), a pad on every spare SoC GPIO whose pinout v1
row names one (the DEBUG bus, on the SoC's right edge), and a rail pad
for each power-tree rail no other sheet probes (PCB-T-02). Each DAC
sheet carries a pad on its MCLK. The spares pinout v1 leaves without a
pad now carry no-connect flags. On the root, facing sheet pins are
joined directly only where the route meets no other symbol.

Co-Authored-By: Claude Opus 5.5 <noreply@anthropic.com>
Claude-Session: https://claude.ai/code/session_01Ei262h3TpgY9vyfNLMi5Mn
Parts:
- removed C6201, C6202: 1 µF, Capacitor_SMD:C_0402_1005Metric, symbol Device:C
- removed C6203, C6204: 470 nF, Capacitor_SMD:C_0402_1005Metric, symbol Device:C
- removed R6201: 100 mΩ, Resistor_SMD:R_0603_1608Metric, symbol Device:R
- removed TP6201: VSYS_LV, TestPoint:TestPoint_Pad_D1.0mm, symbol Connector:TestPoint
- removed TP6202: LED_VDD, TestPoint:TestPoint_Pad_D1.0mm, symbol Connector:TestPoint
- removed U6201: LP5521YQX, Texas_Instruments:Texas_NJA0024A_WQFN-24-1EP_4x5mm_P0.5mm_EP2.4x3.4mm_ThermalVias, symbol Texas_Instruments:LP5521YQX
- added C6301, C6302: 1 µF, Capacitor_SMD:C_0402_1005Metric, symbol Device:C
- added C6303, C6304: 470 nF, Capacitor_SMD:C_0402_1005Metric, symbol Device:C
- added R6301: 100 mΩ, Resistor_SMD:R_0603_1608Metric, symbol Device:R
- added TP6301: VSYS_LV, TestPoint:TestPoint_Pad_D1.0mm, symbol Connector:TestPoint
- added TP6302: LED_VDD, TestPoint:TestPoint_Pad_D1.0mm, symbol Connector:TestPoint
- added U6301: LP5521YQX, Texas_Instruments:Texas_NJA0024A_WQFN-24-1EP_4x5mm_P0.5mm_EP2.4x3.4mm_ThermalVias, symbol Texas_Instruments:LP5521YQX
Connections:
- net GND: now also C6301.2, C6302.2, U6301.20 (ADDR_SEL0), U6301.21 (ADDR_SEL1), U6301.25 (EP), U6301.4 (GND), U6301.5 (CLK_32K), U6301.7 (TRIG)
- net I2C2_SCL: now also U6301.15 (SCL)
- net I2C2_SDA: now also U6301.13 (SDA)
- net LED_B: now also U6301.19 (B)
- net LED_CFLY1N: now also C6303.2, U6301.24 (CFLY1N)
- net LED_CFLY1P: now also C6303.1, U6301.2 (CFLY1P)
- net LED_CFLY2N: now also C6304.2, U6301.23 (CFLY2N)
- net LED_CFLY2P: now also C6304.1, U6301.1 (CFLY2P)
- net LED_G: now also U6301.18 (G)
- net LED_R: now also U6301.17 (R)
- net LED_VDD: now also C6301.1, R6301.2, TP6302.1, U6301.3 (VDD)
- net LED_VOUT: now also C6302.1, U6301.22 (VOUT)
- net VSYS_LV: now also R6301.1, TP6301.1
- net vcca1v8_pmu: now also U6301.14 (EN)
Changed lines of the file:
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@@
 (title_block (title "Status LED driver") (date "2026-10-25") (rev "A") (company "The OpenDAP Project") (comment 1 "blk.status-led") (comment 2 "LP5521 RGB LED driver on I2C2 at 0x32: charge pump, LED_R/G/B to the faceplate, link #22"))
 (symbol (lib_id "Texas_Instruments:LP5521YQX") (at 58.42 82.55 0) (unit 1) (body_style 1) (exclude_from_sim no) (in_bom yes) (on_board yes) (dnp no)
-  (property "Reference" "U6201" (at 59.69 50.8 0) (effects (font (size 1.27 1.27)) (justify left)))
+  (property "Reference" "U6301" (at 59.69 50.8 0) (effects (font (size 1.27 1.27)) (justify left)))
   (property "Value" "LP5521YQX" (at 59.69 48.26 0) (effects (font (size 1.27 1.27)) (justify left)))
   (property "Footprint" "Texas_Instruments:Texas_NJA0024A_WQFN-24-1EP_4x5mm_P0.5mm_EP2.4x3.4mm_ThermalVias" (at 58.42 82.55 0) (effects (font (size 1.27 1.27))) (hide yes))
@@
   (pin "4")
   (pin "25")
-  (instances (project "t1-main-board" (path "/7746052e-d7f9-59ad-ba73-bd2b74439529/7565c505-141d-591d-ab0e-49e98d8f1d5a" (reference "U6201") (unit 1))))
+  (instances (project "t1-main-board" (path "/7746052e-d7f9-59ad-ba73-bd2b74439529/7565c505-141d-591d-ab0e-49e98d8f1d5a" (reference "U6301") (unit 1))))
 )
 (wire (pts (xy 55.88 115.57) (xy 55.88 118.11)) (stroke (width 0) (type default)))
@@
 )
 (symbol (lib_id "Device:C") (at 91.44 54.61 0) (unit 1) (body_style 1) (exclude_from_sim no) (in_bom yes) (on_board yes) (dnp no)
-  (property "Reference" "C6201" (at 93.98 53.34 0) (effects (font (size 1.27 1.27)) (justify left)))
+  (property "Reference" "C6301" (at 93.98 53.34 0) (effects (font (size 1.27 1.27)) (justify left)))
   (property "Value" "1 µF" (at 93.98 55.88 0) (effects (font (size 1.27 1.27)) (justify left)))
   (property "Footprint" "Capacitor_SMD:C_0402_1005Metric" (at 91.44 54.61 0) (effects (font (size 1.27 1.27))) (hide yes))
@@
   (pin "1")
   (pin "2")
-  (instances (project "t1-main-board" (path "/7746052e-d7f9-59ad-ba73-bd2b74439529/7565c505-141d-591d-ab0e-49e98d8f1d5a" (reference "C6201") (unit 1))))
+  (instances (project "t1-main-board" (path "/7746052e-d7f9-59ad-ba73-bd2b74439529/7565c505-141d-591d-ab0e-49e98d8f1d5a" (reference "C6301") (unit 1))))
 )
 (wire (pts (xy 91.44 50.8) (xy 91.44 48.26)) (stroke (width 0) (type default)))
@@
 )
 (symbol (lib_id "Device:C") (at 104.14 54.61 0) (unit 1) (body_style 1) (exclude_from_sim no) (in_bom yes) (on_board yes) (dnp no)
-  (property "Reference" "C6202" (at 106.68 53.34 0) (effects (font (size 1.27 1.27)) (justify left)))
+  (property "Reference" "C6302" (at 106.68 53.34 0) (effects (font (size 1.27 1.27)) (justify left)))
   (property "Value" "1 µF" (at 106.68 55.88 0) (effects (font (size 1.27 1.27)) (justify left)))
   (property "Spec" "10 V X5R" (at 106.68 58.42 0) (effects (font (size 1.27 1.27)) (justify left)))
@@
   (pin "1")
   (pin "2")
-  (instances (project "t1-main-board" (path "/7746052e-d7f9-59ad-ba73-bd2b74439529/7565c505-141d-591d-ab0e-49e98d8f1d5a" (reference "C6202") (unit 1))))
+  (instances (project "t1-main-board" (path "/7746052e-d7f9-59ad-ba73-bd2b74439529/7565c505-141d-591d-ab0e-49e98d8f1d5a" (reference "C6302") (unit 1))))
 )
 (wire (pts (xy 104.14 50.8) (xy 104.14 48.26)) (stroke (width 0) (type default)))
@@
 )
 (symbol (lib_id "Device:C") (at 91.44 88.9 0) (unit 1) (body_style 1) (exclude_from_sim no) (in_bom yes) (on_board yes) (dnp no)
-  (property "Reference" "C6203" (at 93.98 87.63 0) (effects (font (size 1.27 1.27)) (justify left)))
+  (property "Reference" "C6303" (at 93.98 87.63 0) (effects (font (size 1.27 1.27)) (justify left)))
   (property "Value" "470 nF" (at 93.98 90.17 0) (effects (font (size 1.27 1.27)) (justify left)))
   (property "Spec" "10 V X5R" (at 93.98 92.71 0) (effects (font (size 1.27 1.27)) (justify left)))
@@
   (pin "1")
   (pin "2")
-  (instances (project "t1-main-board" (path "/7746052e-d7f9-59ad-ba73-bd2b74439529/7565c505-141d-591d-ab0e-49e98d8f1d5a" (reference "C6203") (unit 1))))
+  (instances (project "t1-main-board" (path "/7746052e-d7f9-59ad-ba73-bd2b74439529/7565c505-141d-591d-ab0e-49e98d8f1d5a" (reference "C6303") (unit 1))))
 )
 (wire (pts (xy 91.44 85.09) (xy 91.44 82.55)) (stroke (width 0) (type default)))
 (symbol (lib_id "Device:C") (at 106.68 88.9 0) (unit 1) (body_style 1) (exclude_from_sim no) (in_bom yes) (on_board yes) (dnp no)
-  (property "Reference" "C6204" (at 109.22 87.63 0) (effects (font (size 1.27 1.27)) (justify left)))
+  (property "Reference" "C6304" (at 109.22 87.63 0) (effects (font (size 1.27 1.27)) (justify left)))
   (property "Value" "470 nF" (at 109.22 90.17 0) (effects (font (size 1.27 1.27)) (justify left)))
   (property "Spec" "10 V X5R" (at 109.22 92.71 0) (effects (font (size 1.27 1.27)) (justify left)))
@@
   (pin "1")
   (pin "2")
-  (instances (project "t1-main-board" (path "/7746052e-d7f9-59ad-ba73-bd2b74439529/7565c505-141d-591d-ab0e-49e98d8f1d5a" (reference "C6204") (unit 1))))
+  (instances (project "t1-main-board" (path "/7746052e-d7f9-59ad-ba73-bd2b74439529/7565c505-141d-591d-ab0e-49e98d8f1d5a" (reference "C6304") (unit 1))))
 )
 (wire (pts (xy 106.68 85.09) (xy 106.68 82.55)) (stroke (width 0) (type default)))
@@
 (text "LP5521 at I2C2 0x32 (BOM v1 line 105; SNVS441I Figure 26)" (exclude_from_sim no) (at 24.13 34.29 0) (effects (font (size 2.54 2.54)) (justify left bottom)))
 (symbol (lib_id "Device:R") (at 190.5 50.8 90) (unit 1) (body_style 1) (exclude_from_sim no) (in_bom yes) (on_board yes) (dnp no)
-  (property "Reference" "R6201" (at 187.96 46.99 90) (effects (font (size 1.27 1.27))))
+  (property "Reference" "R6301" (at 187.96 46.99 90) (effects (font (size 1.27 1.27))))
   (property "Value" "100 mΩ" (at 187.96 53.34 90) (effects (font (size 1.27 1.27))))
   (property "Spec" "0603" (at 187.96 55.88 90) (effects (font (size 1.27 1.27))))
@@
   (pin "1")
   (pin "2")
-  (instances (project "t1-main-board" (path "/7746052e-d7f9-59ad-ba73-bd2b74439529/7565c505-141d-591d-ab0e-49e98d8f1d5a" (reference "R6201") (unit 1) (variant (name "production") (field (name "Value") (value "0 Ω")) (field (name "MPN") (value "RC0603JR-070RL")) (field (name "Manufacturer") (value "YAGEO"))))))
+  (instances (project "t1-main-board" (path "/7746052e-d7f9-59ad-ba73-bd2b74439529/7565c505-141d-591d-ab0e-49e98d8f1d5a" (reference "R6301") (unit 1) (variant (name "production") (field (name "Value") (value "0 Ω")) (field (name "MPN") (value "RC0603JR-070RL")) (field (name "Manufacturer") (value "YAGEO"))))))
 )
 (rectangle (start 172.72 38.1) (end 208.28 58.42) (stroke (width 0) (type dash)) (fill (type none)))
@@
 (wire (pts (xy 184.15 50.8) (xy 184.15 48.26)) (stroke (width 0) (type default)))
 (symbol (lib_id "Connector:TestPoint") (at 184.15 48.26 0) (unit 1) (body_style 1) (exclude_from_sim no) (in_bom no) (on_board yes) (dnp no)
-  (property "Reference" "TP6201" (at 182.88 43.18 0) (effects (font (size 1.27 1.27)) (justify right)))
+  (property "Reference" "TP6301" (at 182.88 43.18 0) (effects (font (size 1.27 1.27)) (justify right)))
   (property "Value" "VSYS_LV" (at 182.88 45.72 0) (effects (font (size 1.27 1.27)) (justify right)))
   (property "Footprint" "TestPoint:TestPoint_Pad_D1.0mm" (at 184.15 48.26 0) (effects (font (size 1.27 1.27))) (hide yes))
@@
   (property "Block" "blk.status-led" (at 184.15 48.26 0) (effects (font (size 1.27 1.27))) (hide yes))
   (pin "1")
-  (instances (project "t1-main-board" (path "/7746052e-d7f9-59ad-ba73-bd2b74439529/7565c505-141d-591d-ab0e-49e98d8f1d5a" (reference "TP6201") (unit 1))))
+  (instances (project "t1-main-board" (path "/7746052e-d7f9-59ad-ba73-bd2b74439529/7565c505-141d-591d-ab0e-49e98d8f1d5a" (reference "TP6301") (unit 1))))
 )
 (symbol (lib_id "power:VCC") (at 170.18 50.8 90) (unit 1) (body_style 1) (exclude_from_sim no) (in_bom yes) (on_board yes) (dnp no)
@@
 (wire (pts (xy 196.85 50.8) (xy 196.85 48.26)) (stroke (width 0) (type default)))
 (symbol (lib_id "Connector:TestPoint") (at 196.85 48.26 0) (unit 1) (body_style 1) (exclude_from_sim no) (in_bom no) (on_board yes) (dnp no)
-  (property "Reference" "TP6202" (at 198.12 43.18 0) (effects (font (size 1.27 1.27)) (justify left)))
+  (property "Reference" "TP6302" (at 198.12 43.18 0) (effects (font (size 1.27 1.27)) (justify left)))
   (property "Value" "LED_VDD" (at 198.12 45.72 0) (effects (font (size 1.27 1.27)) (justify left)))
   (property "Footprint" "TestPoint:TestPoint_Pad_D1.0mm" (at 196.85 48.26 0) (effects (font (size 1.27 1.27))) (hide yes))
@@
   (property "Block" "blk.status-led" (at 196.85 48.26 0) (effects (font (size 1.27 1.27))) (hide yes))
   (pin "1")
-  (instances (project "t1-main-board" (path "/7746052e-d7f9-59ad-ba73-bd2b74439529/7565c505-141d-591d-ab0e-49e98d8f1d5a" (reference "TP6202") (unit 1))))
+  (instances (project "t1-main-board" (path "/7746052e-d7f9-59ad-ba73-bd2b74439529/7565c505-141d-591d-ab0e-49e98d8f1d5a" (reference "TP6302") (unit 1))))
 )
 (junction (at 215.9 50.8) (diameter 0) (color 0 0 0 0))

Commit message: Board: capture blk.cover-detect
COVER_DET_N on GPIO0_A6 (AJ38, PMUIO1, wake-capable), recorded in
pinout v1 (closes feature blocks G22): board-edge input and ground pads
for the case's actuator, 100 kΩ to vcc3v3_pmu, TPD1E10B06 at the pad
(BOM v1 line 143, PCB-L-10). The line rides the KEYS bus with the
buttons.

Co-Authored-By: Claude Opus 5.5 <noreply@anthropic.com>
Claude-Session: https://claude.ai/code/session_01Ei262h3TpgY9vyfNLMi5Mn
Parts:
- removed C6301, C6302: 1 µF, Capacitor_SMD:C_0402_1005Metric, symbol Device:C
- removed C6303, C6304: 470 nF, Capacitor_SMD:C_0402_1005Metric, symbol Device:C
- removed R6301: 100 mΩ, Resistor_SMD:R_0603_1608Metric, symbol Device:R
- removed TP6301: VSYS_LV, TestPoint:TestPoint_Pad_D1.0mm, symbol Connector:TestPoint
- removed TP6302: LED_VDD, TestPoint:TestPoint_Pad_D1.0mm, symbol Connector:TestPoint
- removed U6301: LP5521YQX, Texas_Instruments:Texas_NJA0024A_WQFN-24-1EP_4x5mm_P0.5mm_EP2.4x3.4mm_ThermalVias, symbol Texas_Instruments:LP5521YQX
- added C6401, C6402: 1 µF, Capacitor_SMD:C_0402_1005Metric, symbol Device:C
- added C6403, C6404: 470 nF, Capacitor_SMD:C_0402_1005Metric, symbol Device:C
- added R6401: 100 mΩ, Resistor_SMD:R_0603_1608Metric, symbol Device:R
- added TP6401: VSYS_LV, TestPoint:TestPoint_Pad_D1.0mm, symbol Connector:TestPoint
- added TP6402: LED_VDD, TestPoint:TestPoint_Pad_D1.0mm, symbol Connector:TestPoint
- added U6401: LP5521YQX, Texas_Instruments:Texas_NJA0024A_WQFN-24-1EP_4x5mm_P0.5mm_EP2.4x3.4mm_ThermalVias, symbol Texas_Instruments:LP5521YQX
Connections:
- net GND: now also C6401.2, C6402.2, U6401.20 (ADDR_SEL0), U6401.21 (ADDR_SEL1), U6401.25 (EP), U6401.4 (GND), U6401.5 (CLK_32K), U6401.7 (TRIG)
- net I2C2_SCL: now also U6401.15 (SCL)
- net I2C2_SDA: now also U6401.13 (SDA)
- net LED_B: now also U6401.19 (B)
- net LED_CFLY1N: now also C6403.2, U6401.24 (CFLY1N)
- net LED_CFLY1P: now also C6403.1, U6401.2 (CFLY1P)
- net LED_CFLY2N: now also C6404.2, U6401.23 (CFLY2N)
- net LED_CFLY2P: now also C6404.1, U6401.1 (CFLY2P)
- net LED_G: now also U6401.18 (G)
- net LED_R: now also U6401.17 (R)
- net LED_VDD: now also C6401.1, R6401.2, TP6402.1, U6401.3 (VDD)
- net LED_VOUT: now also C6402.1, U6401.22 (VOUT)
- net VSYS_LV: now also R6401.1, TP6401.1
- net vcca1v8_pmu: now also U6401.14 (EN)
Changed lines of the file:
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@@
 (title_block (title "Status LED driver") (date "2026-10-25") (rev "A") (company "The OpenDAP Project") (comment 1 "blk.status-led") (comment 2 "LP5521 RGB LED driver on I2C2 at 0x32: charge pump, LED_R/G/B to the faceplate, link #22"))
 (symbol (lib_id "Texas_Instruments:LP5521YQX") (at 58.42 82.55 0) (unit 1) (body_style 1) (exclude_from_sim no) (in_bom yes) (on_board yes) (dnp no)
-  (property "Reference" "U6301" (at 59.69 50.8 0) (effects (font (size 1.27 1.27)) (justify left)))
+  (property "Reference" "U6401" (at 59.69 50.8 0) (effects (font (size 1.27 1.27)) (justify left)))
   (property "Value" "LP5521YQX" (at 59.69 48.26 0) (effects (font (size 1.27 1.27)) (justify left)))
   (property "Footprint" "Texas_Instruments:Texas_NJA0024A_WQFN-24-1EP_4x5mm_P0.5mm_EP2.4x3.4mm_ThermalVias" (at 58.42 82.55 0) (effects (font (size 1.27 1.27))) (hide yes))
@@
   (pin "4")
   (pin "25")
-  (instances (project "t1-main-board" (path "/7746052e-d7f9-59ad-ba73-bd2b74439529/7565c505-141d-591d-ab0e-49e98d8f1d5a" (reference "U6301") (unit 1))))
+  (instances (project "t1-main-board" (path "/7746052e-d7f9-59ad-ba73-bd2b74439529/7565c505-141d-591d-ab0e-49e98d8f1d5a" (reference "U6401") (unit 1))))
 )
 (wire (pts (xy 55.88 115.57) (xy 55.88 118.11)) (stroke (width 0) (type default)))
@@
 )
 (symbol (lib_id "Device:C") (at 91.44 54.61 0) (unit 1) (body_style 1) (exclude_from_sim no) (in_bom yes) (on_board yes) (dnp no)
-  (property "Reference" "C6301" (at 93.98 53.34 0) (effects (font (size 1.27 1.27)) (justify left)))
+  (property "Reference" "C6401" (at 93.98 53.34 0) (effects (font (size 1.27 1.27)) (justify left)))
   (property "Value" "1 µF" (at 93.98 55.88 0) (effects (font (size 1.27 1.27)) (justify left)))
   (property "Footprint" "Capacitor_SMD:C_0402_1005Metric" (at 91.44 54.61 0) (effects (font (size 1.27 1.27))) (hide yes))
@@
   (pin "1")
   (pin "2")
-  (instances (project "t1-main-board" (path "/7746052e-d7f9-59ad-ba73-bd2b74439529/7565c505-141d-591d-ab0e-49e98d8f1d5a" (reference "C6301") (unit 1))))
+  (instances (project "t1-main-board" (path "/7746052e-d7f9-59ad-ba73-bd2b74439529/7565c505-141d-591d-ab0e-49e98d8f1d5a" (reference "C6401") (unit 1))))
 )
 (wire (pts (xy 91.44 50.8) (xy 91.44 48.26)) (stroke (width 0) (type default)))
@@
 )
 (symbol (lib_id "Device:C") (at 104.14 54.61 0) (unit 1) (body_style 1) (exclude_from_sim no) (in_bom yes) (on_board yes) (dnp no)
-  (property "Reference" "C6302" (at 106.68 53.34 0) (effects (font (size 1.27 1.27)) (justify left)))
+  (property "Reference" "C6402" (at 106.68 53.34 0) (effects (font (size 1.27 1.27)) (justify left)))
   (property "Value" "1 µF" (at 106.68 55.88 0) (effects (font (size 1.27 1.27)) (justify left)))
   (property "Spec" "10 V X5R" (at 106.68 58.42 0) (effects (font (size 1.27 1.27)) (justify left)))
@@
   (pin "1")
   (pin "2")
-  (instances (project "t1-main-board" (path "/7746052e-d7f9-59ad-ba73-bd2b74439529/7565c505-141d-591d-ab0e-49e98d8f1d5a" (reference "C6302") (unit 1))))
+  (instances (project "t1-main-board" (path "/7746052e-d7f9-59ad-ba73-bd2b74439529/7565c505-141d-591d-ab0e-49e98d8f1d5a" (reference "C6402") (unit 1))))
 )
 (wire (pts (xy 104.14 50.8) (xy 104.14 48.26)) (stroke (width 0) (type default)))
@@
 )
 (symbol (lib_id "Device:C") (at 91.44 88.9 0) (unit 1) (body_style 1) (exclude_from_sim no) (in_bom yes) (on_board yes) (dnp no)
-  (property "Reference" "C6303" (at 93.98 87.63 0) (effects (font (size 1.27 1.27)) (justify left)))
+  (property "Reference" "C6403" (at 93.98 87.63 0) (effects (font (size 1.27 1.27)) (justify left)))
   (property "Value" "470 nF" (at 93.98 90.17 0) (effects (font (size 1.27 1.27)) (justify left)))
   (property "Spec" "10 V X5R" (at 93.98 92.71 0) (effects (font (size 1.27 1.27)) (justify left)))
@@
   (pin "1")
   (pin "2")
-  (instances (project "t1-main-board" (path "/7746052e-d7f9-59ad-ba73-bd2b74439529/7565c505-141d-591d-ab0e-49e98d8f1d5a" (reference "C6303") (unit 1))))
+  (instances (project "t1-main-board" (path "/7746052e-d7f9-59ad-ba73-bd2b74439529/7565c505-141d-591d-ab0e-49e98d8f1d5a" (reference "C6403") (unit 1))))
 )
 (wire (pts (xy 91.44 85.09) (xy 91.44 82.55)) (stroke (width 0) (type default)))
 (symbol (lib_id "Device:C") (at 106.68 88.9 0) (unit 1) (body_style 1) (exclude_from_sim no) (in_bom yes) (on_board yes) (dnp no)
-  (property "Reference" "C6304" (at 109.22 87.63 0) (effects (font (size 1.27 1.27)) (justify left)))
+  (property "Reference" "C6404" (at 109.22 87.63 0) (effects (font (size 1.27 1.27)) (justify left)))
   (property "Value" "470 nF" (at 109.22 90.17 0) (effects (font (size 1.27 1.27)) (justify left)))
   (property "Spec" "10 V X5R" (at 109.22 92.71 0) (effects (font (size 1.27 1.27)) (justify left)))
@@
   (pin "1")
   (pin "2")
-  (instances (project "t1-main-board" (path "/7746052e-d7f9-59ad-ba73-bd2b74439529/7565c505-141d-591d-ab0e-49e98d8f1d5a" (reference "C6304") (unit 1))))
+  (instances (project "t1-main-board" (path "/7746052e-d7f9-59ad-ba73-bd2b74439529/7565c505-141d-591d-ab0e-49e98d8f1d5a" (reference "C6404") (unit 1))))
 )
 (wire (pts (xy 106.68 85.09) (xy 106.68 82.55)) (stroke (width 0) (type default)))
@@
 (text "LP5521 at I2C2 0x32 (BOM v1 line 105; SNVS441I Figure 26)" (exclude_from_sim no) (at 24.13 34.29 0) (effects (font (size 2.54 2.54)) (justify left bottom)))
 (symbol (lib_id "Device:R") (at 190.5 50.8 90) (unit 1) (body_style 1) (exclude_from_sim no) (in_bom yes) (on_board yes) (dnp no)
-  (property "Reference" "R6301" (at 187.96 46.99 90) (effects (font (size 1.27 1.27))))
+  (property "Reference" "R6401" (at 187.96 46.99 90) (effects (font (size 1.27 1.27))))
   (property "Value" "100 mΩ" (at 187.96 53.34 90) (effects (font (size 1.27 1.27))))
   (property "Spec" "0603" (at 187.96 55.88 90) (effects (font (size 1.27 1.27))))
@@
   (pin "1")
   (pin "2")
-  (instances (project "t1-main-board" (path "/7746052e-d7f9-59ad-ba73-bd2b74439529/7565c505-141d-591d-ab0e-49e98d8f1d5a" (reference "R6301") (unit 1) (variant (name "production") (field (name "Value") (value "0 Ω")) (field (name "MPN") (value "RC0603JR-070RL")) (field (name "Manufacturer") (value "YAGEO"))))))
+  (instances (project "t1-main-board" (path "/7746052e-d7f9-59ad-ba73-bd2b74439529/7565c505-141d-591d-ab0e-49e98d8f1d5a" (reference "R6401") (unit 1) (variant (name "production") (field (name "Value") (value "0 Ω")) (field (name "MPN") (value "RC0603JR-070RL")) (field (name "Manufacturer") (value "YAGEO"))))))
 )
 (rectangle (start 172.72 38.1) (end 208.28 58.42) (stroke (width 0) (type dash)) (fill (type none)))
@@
 (wire (pts (xy 184.15 50.8) (xy 184.15 48.26)) (stroke (width 0) (type default)))
 (symbol (lib_id "Connector:TestPoint") (at 184.15 48.26 0) (unit 1) (body_style 1) (exclude_from_sim no) (in_bom no) (on_board yes) (dnp no)
-  (property "Reference" "TP6301" (at 182.88 43.18 0) (effects (font (size 1.27 1.27)) (justify right)))
+  (property "Reference" "TP6401" (at 182.88 43.18 0) (effects (font (size 1.27 1.27)) (justify right)))
   (property "Value" "VSYS_LV" (at 182.88 45.72 0) (effects (font (size 1.27 1.27)) (justify right)))
   (property "Footprint" "TestPoint:TestPoint_Pad_D1.0mm" (at 184.15 48.26 0) (effects (font (size 1.27 1.27))) (hide yes))
@@
   (property "Block" "blk.status-led" (at 184.15 48.26 0) (effects (font (size 1.27 1.27))) (hide yes))
   (pin "1")
-  (instances (project "t1-main-board" (path "/7746052e-d7f9-59ad-ba73-bd2b74439529/7565c505-141d-591d-ab0e-49e98d8f1d5a" (reference "TP6301") (unit 1))))
+  (instances (project "t1-main-board" (path "/7746052e-d7f9-59ad-ba73-bd2b74439529/7565c505-141d-591d-ab0e-49e98d8f1d5a" (reference "TP6401") (unit 1))))
 )
 (symbol (lib_id "power:VCC") (at 170.18 50.8 90) (unit 1) (body_style 1) (exclude_from_sim no) (in_bom yes) (on_board yes) (dnp no)
@@
 (wire (pts (xy 196.85 50.8) (xy 196.85 48.26)) (stroke (width 0) (type default)))
 (symbol (lib_id "Connector:TestPoint") (at 196.85 48.26 0) (unit 1) (body_style 1) (exclude_from_sim no) (in_bom no) (on_board yes) (dnp no)
-  (property "Reference" "TP6302" (at 198.12 43.18 0) (effects (font (size 1.27 1.27)) (justify left)))
+  (property "Reference" "TP6402" (at 198.12 43.18 0) (effects (font (size 1.27 1.27)) (justify left)))
   (property "Value" "LED_VDD" (at 198.12 45.72 0) (effects (font (size 1.27 1.27)) (justify left)))
   (property "Footprint" "TestPoint:TestPoint_Pad_D1.0mm" (at 196.85 48.26 0) (effects (font (size 1.27 1.27))) (hide yes))
@@
   (property "Block" "blk.status-led" (at 196.85 48.26 0) (effects (font (size 1.27 1.27))) (hide yes))
   (pin "1")
-  (instances (project "t1-main-board" (path "/7746052e-d7f9-59ad-ba73-bd2b74439529/7565c505-141d-591d-ab0e-49e98d8f1d5a" (reference "TP6302") (unit 1))))
+  (instances (project "t1-main-board" (path "/7746052e-d7f9-59ad-ba73-bd2b74439529/7565c505-141d-591d-ab0e-49e98d8f1d5a" (reference "TP6402") (unit 1))))
 )
 (junction (at 215.9 50.8) (diameter 0) (color 0 0 0 0))
