File: board/hardware/t1-main-board/status-led.kicad_sch (KiCad schematic)
At the start: 8 parts, among them U6401 LP5521YQX

Commit message: Board: capture blk.mic-ambient and links #34, #35
IM73D122 on PDM CLK1 and SDI1 (BOM v1 line 34, pinout v1 AK2 and 1P2),
LR to ground, 22 Ω clock series, VDD from MIC_1V8 through link #35.
Link #34 on blk.mic-main makes the faceplate branch the rail MIC_1V8_FP
for contact 40 (power tree §4.12, G10). kicad-lib moves to e46bda4 for
the IM73D122, TPS3808G01, SN74LVC1G58 and BAT54 parts.

Co-Authored-By: Claude Opus 5.5 <noreply@anthropic.com>
Claude-Session: https://claude.ai/code/session_01Ei262h3TpgY9vyfNLMi5Mn
Parts:
- removed C6401, C6402: 1 µF, Capacitor_SMD:C_0402_1005Metric, symbol Device:C
- removed C6403, C6404: 470 nF, Capacitor_SMD:C_0402_1005Metric, symbol Device:C
- removed R6401: 100 mΩ, Resistor_SMD:R_0603_1608Metric, symbol Device:R
- removed TP6401: VSYS_LV, TestPoint:TestPoint_Pad_D1.0mm, symbol Connector:TestPoint
- removed TP6402: LED_VDD, TestPoint:TestPoint_Pad_D1.0mm, symbol Connector:TestPoint
- removed U6401: LP5521YQX, Texas_Instruments:Texas_NJA0024A_WQFN-24-1EP_4x5mm_P0.5mm_EP2.4x3.4mm_ThermalVias, symbol Texas_Instruments:LP5521YQX
- added C6501, C6502: 1 µF, Capacitor_SMD:C_0402_1005Metric, symbol Device:C
- added C6503, C6504: 470 nF, Capacitor_SMD:C_0402_1005Metric, symbol Device:C
- added R6501: 100 mΩ, Resistor_SMD:R_0603_1608Metric, symbol Device:R
- added TP6501: VSYS_LV, TestPoint:TestPoint_Pad_D1.0mm, symbol Connector:TestPoint
- added TP6502: LED_VDD, TestPoint:TestPoint_Pad_D1.0mm, symbol Connector:TestPoint
- added U6501: LP5521YQX, Texas_Instruments:Texas_NJA0024A_WQFN-24-1EP_4x5mm_P0.5mm_EP2.4x3.4mm_ThermalVias, symbol Texas_Instruments:LP5521YQX
Connections:
- net GND: now also C6501.2, C6502.2, U6501.20 (ADDR_SEL0), U6501.21 (ADDR_SEL1), U6501.25 (EP), U6501.4 (GND), U6501.5 (CLK_32K), U6501.7 (TRIG)
- net I2C2_SCL: now also U6501.15 (SCL)
- net I2C2_SDA: now also U6501.13 (SDA)
- net LED_B: now also U6501.19 (B)
- net LED_CFLY1N: now also C6503.2, U6501.24 (CFLY1N)
- net LED_CFLY1P: now also C6503.1, U6501.2 (CFLY1P)
- net LED_CFLY2N: now also C6504.2, U6501.23 (CFLY2N)
- net LED_CFLY2P: now also C6504.1, U6501.1 (CFLY2P)
- net LED_G: now also U6501.18 (G)
- net LED_R: now also U6501.17 (R)
- net LED_VDD: now also C6501.1, R6501.2, TP6502.1, U6501.3 (VDD)
- net LED_VOUT: now also C6502.1, U6501.22 (VOUT)
- net VSYS_LV: now also R6501.1, TP6501.1
- net vcca1v8_pmu: now also U6501.14 (EN)

Commit message: Board: capture blk.maskrom
Power + Vol- at a cold power-on pull eMMC D0 low inside the TPS3808G01
boot window (BOM v1 lines 35, 78, 97, 98; sim/maskrom): SENSE 280k/100k,
CT 390 nF, WINDOW_N with its pad, SN74LVC1G57 and SN74LVC1G58 on
vcca1v8_pmu, BAT54 from PWRON_N, DMG1012T through 1 kΩ to EMMC_D0.
Every block in use now has its sheet; the README states the remaining
single-pin nets.

Co-Authored-By: Claude Opus 5.5 <noreply@anthropic.com>
Claude-Session: https://claude.ai/code/session_01Ei262h3TpgY9vyfNLMi5Mn
Parts:
- removed C6501, C6502: 1 µF, Capacitor_SMD:C_0402_1005Metric, symbol Device:C
- removed C6503, C6504: 470 nF, Capacitor_SMD:C_0402_1005Metric, symbol Device:C
- removed R6501: 100 mΩ, Resistor_SMD:R_0603_1608Metric, symbol Device:R
- removed TP6501: VSYS_LV, TestPoint:TestPoint_Pad_D1.0mm, symbol Connector:TestPoint
- removed TP6502: LED_VDD, TestPoint:TestPoint_Pad_D1.0mm, symbol Connector:TestPoint
- removed U6501: LP5521YQX, Texas_Instruments:Texas_NJA0024A_WQFN-24-1EP_4x5mm_P0.5mm_EP2.4x3.4mm_ThermalVias, symbol Texas_Instruments:LP5521YQX
- added C6601, C6602: 1 µF, Capacitor_SMD:C_0402_1005Metric, symbol Device:C
- added C6603, C6604: 470 nF, Capacitor_SMD:C_0402_1005Metric, symbol Device:C
- added R6601: 100 mΩ, Resistor_SMD:R_0603_1608Metric, symbol Device:R
- added TP6601: VSYS_LV, TestPoint:TestPoint_Pad_D1.0mm, symbol Connector:TestPoint
- added TP6602: LED_VDD, TestPoint:TestPoint_Pad_D1.0mm, symbol Connector:TestPoint
- added U6601: LP5521YQX, Texas_Instruments:Texas_NJA0024A_WQFN-24-1EP_4x5mm_P0.5mm_EP2.4x3.4mm_ThermalVias, symbol Texas_Instruments:LP5521YQX
Connections:
- net GND: now also C6601.2, C6602.2, U6601.20 (ADDR_SEL0), U6601.21 (ADDR_SEL1), U6601.25 (EP), U6601.4 (GND), U6601.5 (CLK_32K), U6601.7 (TRIG)
- net I2C2_SCL: now also U6601.15 (SCL)
- net I2C2_SDA: now also U6601.13 (SDA)
- net LED_B: now also U6601.19 (B)
- net LED_CFLY1N: now also C6603.2, U6601.24 (CFLY1N)
- net LED_CFLY1P: now also C6603.1, U6601.2 (CFLY1P)
- net LED_CFLY2N: now also C6604.2, U6601.23 (CFLY2N)
- net LED_CFLY2P: now also C6604.1, U6601.1 (CFLY2P)
- net LED_G: now also U6601.18 (G)
- net LED_R: now also U6601.17 (R)
- net LED_VDD: now also C6601.1, R6601.2, TP6602.1, U6601.3 (VDD)
- net LED_VOUT: now also C6602.1, U6601.22 (VOUT)
- net VSYS_LV: now also R6601.1, TP6601.1
- net vcca1v8_pmu: now also U6601.14 (EN)
Changed lines of the file:
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@@
 (title_block (title "Status LED driver") (date "2026-10-25") (rev "A") (company "The OpenDAP Project") (comment 1 "blk.status-led") (comment 2 "LP5521 RGB LED driver on I2C2 at 0x32: charge pump, LED_R/G/B to the faceplate, link #22"))
 (symbol (lib_id "Texas_Instruments:LP5521YQX") (at 58.42 82.55 0) (unit 1) (body_style 1) (exclude_from_sim no) (in_bom yes) (on_board yes) (dnp no)
-  (property "Reference" "U6501" (at 59.69 50.8 0) (effects (font (size 1.27 1.27)) (justify left)))
+  (property "Reference" "U6601" (at 59.69 50.8 0) (effects (font (size 1.27 1.27)) (justify left)))
   (property "Value" "LP5521YQX" (at 59.69 48.26 0) (effects (font (size 1.27 1.27)) (justify left)))
   (property "Footprint" "Texas_Instruments:Texas_NJA0024A_WQFN-24-1EP_4x5mm_P0.5mm_EP2.4x3.4mm_ThermalVias" (at 58.42 82.55 0) (effects (font (size 1.27 1.27))) (hide yes))
@@
   (pin "4")
   (pin "25")
-  (instances (project "t1-main-board" (path "/7746052e-d7f9-59ad-ba73-bd2b74439529/7565c505-141d-591d-ab0e-49e98d8f1d5a" (reference "U6501") (unit 1))))
+  (instances (project "t1-main-board" (path "/7746052e-d7f9-59ad-ba73-bd2b74439529/7565c505-141d-591d-ab0e-49e98d8f1d5a" (reference "U6601") (unit 1))))
 )
 (wire (pts (xy 55.88 115.57) (xy 55.88 118.11)) (stroke (width 0) (type default)))
@@
 )
 (symbol (lib_id "Device:C") (at 91.44 54.61 0) (unit 1) (body_style 1) (exclude_from_sim no) (in_bom yes) (on_board yes) (dnp no)
-  (property "Reference" "C6501" (at 93.98 53.34 0) (effects (font (size 1.27 1.27)) (justify left)))
+  (property "Reference" "C6601" (at 93.98 53.34 0) (effects (font (size 1.27 1.27)) (justify left)))
   (property "Value" "1 µF" (at 93.98 55.88 0) (effects (font (size 1.27 1.27)) (justify left)))
   (property "Footprint" "Capacitor_SMD:C_0402_1005Metric" (at 91.44 54.61 0) (effects (font (size 1.27 1.27))) (hide yes))
@@
   (pin "1")
   (pin "2")
-  (instances (project "t1-main-board" (path "/7746052e-d7f9-59ad-ba73-bd2b74439529/7565c505-141d-591d-ab0e-49e98d8f1d5a" (reference "C6501") (unit 1))))
+  (instances (project "t1-main-board" (path "/7746052e-d7f9-59ad-ba73-bd2b74439529/7565c505-141d-591d-ab0e-49e98d8f1d5a" (reference "C6601") (unit 1))))
 )
 (wire (pts (xy 91.44 50.8) (xy 91.44 48.26)) (stroke (width 0) (type default)))
@@
 )
 (symbol (lib_id "Device:C") (at 104.14 54.61 0) (unit 1) (body_style 1) (exclude_from_sim no) (in_bom yes) (on_board yes) (dnp no)
-  (property "Reference" "C6502" (at 106.68 53.34 0) (effects (font (size 1.27 1.27)) (justify left)))
+  (property "Reference" "C6602" (at 106.68 53.34 0) (effects (font (size 1.27 1.27)) (justify left)))
   (property "Value" "1 µF" (at 106.68 55.88 0) (effects (font (size 1.27 1.27)) (justify left)))
   (property "Spec" "10 V X5R" (at 106.68 58.42 0) (effects (font (size 1.27 1.27)) (justify left)))
@@
   (pin "1")
   (pin "2")
-  (instances (project "t1-main-board" (path "/7746052e-d7f9-59ad-ba73-bd2b74439529/7565c505-141d-591d-ab0e-49e98d8f1d5a" (reference "C6502") (unit 1))))
+  (instances (project "t1-main-board" (path "/7746052e-d7f9-59ad-ba73-bd2b74439529/7565c505-141d-591d-ab0e-49e98d8f1d5a" (reference "C6602") (unit 1))))
 )
 (wire (pts (xy 104.14 50.8) (xy 104.14 48.26)) (stroke (width 0) (type default)))
@@
 )
 (symbol (lib_id "Device:C") (at 91.44 88.9 0) (unit 1) (body_style 1) (exclude_from_sim no) (in_bom yes) (on_board yes) (dnp no)
-  (property "Reference" "C6503" (at 93.98 87.63 0) (effects (font (size 1.27 1.27)) (justify left)))
+  (property "Reference" "C6603" (at 93.98 87.63 0) (effects (font (size 1.27 1.27)) (justify left)))
   (property "Value" "470 nF" (at 93.98 90.17 0) (effects (font (size 1.27 1.27)) (justify left)))
   (property "Spec" "10 V X5R" (at 93.98 92.71 0) (effects (font (size 1.27 1.27)) (justify left)))
@@
   (pin "1")
   (pin "2")
-  (instances (project "t1-main-board" (path "/7746052e-d7f9-59ad-ba73-bd2b74439529/7565c505-141d-591d-ab0e-49e98d8f1d5a" (reference "C6503") (unit 1))))
+  (instances (project "t1-main-board" (path "/7746052e-d7f9-59ad-ba73-bd2b74439529/7565c505-141d-591d-ab0e-49e98d8f1d5a" (reference "C6603") (unit 1))))
 )
 (wire (pts (xy 91.44 85.09) (xy 91.44 82.55)) (stroke (width 0) (type default)))
 (symbol (lib_id "Device:C") (at 106.68 88.9 0) (unit 1) (body_style 1) (exclude_from_sim no) (in_bom yes) (on_board yes) (dnp no)
-  (property "Reference" "C6504" (at 109.22 87.63 0) (effects (font (size 1.27 1.27)) (justify left)))
+  (property "Reference" "C6604" (at 109.22 87.63 0) (effects (font (size 1.27 1.27)) (justify left)))
   (property "Value" "470 nF" (at 109.22 90.17 0) (effects (font (size 1.27 1.27)) (justify left)))
   (property "Spec" "10 V X5R" (at 109.22 92.71 0) (effects (font (size 1.27 1.27)) (justify left)))
@@
   (pin "1")
   (pin "2")
-  (instances (project "t1-main-board" (path "/7746052e-d7f9-59ad-ba73-bd2b74439529/7565c505-141d-591d-ab0e-49e98d8f1d5a" (reference "C6504") (unit 1))))
+  (instances (project "t1-main-board" (path "/7746052e-d7f9-59ad-ba73-bd2b74439529/7565c505-141d-591d-ab0e-49e98d8f1d5a" (reference "C6604") (unit 1))))
 )
 (wire (pts (xy 106.68 85.09) (xy 106.68 82.55)) (stroke (width 0) (type default)))
@@
 (text "LP5521 at I2C2 0x32 (BOM v1 line 105; SNVS441I Figure 26)" (exclude_from_sim no) (at 24.13 34.29 0) (effects (font (size 2.54 2.54)) (justify left bottom)))
 (symbol (lib_id "Device:R") (at 190.5 50.8 90) (unit 1) (body_style 1) (exclude_from_sim no) (in_bom yes) (on_board yes) (dnp no)
-  (property "Reference" "R6501" (at 187.96 46.99 90) (effects (font (size 1.27 1.27))))
+  (property "Reference" "R6601" (at 187.96 46.99 90) (effects (font (size 1.27 1.27))))
   (property "Value" "100 mΩ" (at 187.96 53.34 90) (effects (font (size 1.27 1.27))))
   (property "Spec" "0603" (at 187.96 55.88 90) (effects (font (size 1.27 1.27))))
@@
   (pin "1")
   (pin "2")
-  (instances (project "t1-main-board" (path "/7746052e-d7f9-59ad-ba73-bd2b74439529/7565c505-141d-591d-ab0e-49e98d8f1d5a" (reference "R6501") (unit 1) (variant (name "production") (field (name "Value") (value "0 Ω")) (field (name "MPN") (value "RC0603JR-070RL")) (field (name "Manufacturer") (value "YAGEO"))))))
+  (instances (project "t1-main-board" (path "/7746052e-d7f9-59ad-ba73-bd2b74439529/7565c505-141d-591d-ab0e-49e98d8f1d5a" (reference "R6601") (unit 1) (variant (name "production") (field (name "Value") (value "0 Ω")) (field (name "MPN") (value "RC0603JR-070RL")) (field (name "Manufacturer") (value "YAGEO"))))))
 )
 (rectangle (start 172.72 38.1) (end 208.28 58.42) (stroke (width 0) (type dash)) (fill (type none)))
@@
 (wire (pts (xy 184.15 50.8) (xy 184.15 48.26)) (stroke (width 0) (type default)))
 (symbol (lib_id "Connector:TestPoint") (at 184.15 48.26 0) (unit 1) (body_style 1) (exclude_from_sim no) (in_bom no) (on_board yes) (dnp no)
-  (property "Reference" "TP6501" (at 182.88 43.18 0) (effects (font (size 1.27 1.27)) (justify right)))
+  (property "Reference" "TP6601" (at 182.88 43.18 0) (effects (font (size 1.27 1.27)) (justify right)))
   (property "Value" "VSYS_LV" (at 182.88 45.72 0) (effects (font (size 1.27 1.27)) (justify right)))
   (property "Footprint" "TestPoint:TestPoint_Pad_D1.0mm" (at 184.15 48.26 0) (effects (font (size 1.27 1.27))) (hide yes))
@@
   (property "Block" "blk.status-led" (at 184.15 48.26 0) (effects (font (size 1.27 1.27))) (hide yes))
   (pin "1")
-  (instances (project "t1-main-board" (path "/7746052e-d7f9-59ad-ba73-bd2b74439529/7565c505-141d-591d-ab0e-49e98d8f1d5a" (reference "TP6501") (unit 1))))
+  (instances (project "t1-main-board" (path "/7746052e-d7f9-59ad-ba73-bd2b74439529/7565c505-141d-591d-ab0e-49e98d8f1d5a" (reference "TP6601") (unit 1))))
 )
 (symbol (lib_id "power:VCC") (at 170.18 50.8 90) (unit 1) (body_style 1) (exclude_from_sim no) (in_bom yes) (on_board yes) (dnp no)
@@
 (wire (pts (xy 196.85 50.8) (xy 196.85 48.26)) (stroke (width 0) (type default)))
 (symbol (lib_id "Connector:TestPoint") (at 196.85 48.26 0) (unit 1) (body_style 1) (exclude_from_sim no) (in_bom no) (on_board yes) (dnp no)
-  (property "Reference" "TP6502" (at 198.12 43.18 0) (effects (font (size 1.27 1.27)) (justify left)))
+  (property "Reference" "TP6602" (at 198.12 43.18 0) (effects (font (size 1.27 1.27)) (justify left)))
   (property "Value" "LED_VDD" (at 198.12 45.72 0) (effects (font (size 1.27 1.27)) (justify left)))
   (property "Footprint" "TestPoint:TestPoint_Pad_D1.0mm" (at 196.85 48.26 0) (effects (font (size 1.27 1.27))) (hide yes))
@@
   (property "Block" "blk.status-led" (at 196.85 48.26 0) (effects (font (size 1.27 1.27))) (hide yes))
   (pin "1")
-  (instances (project "t1-main-board" (path "/7746052e-d7f9-59ad-ba73-bd2b74439529/7565c505-141d-591d-ab0e-49e98d8f1d5a" (reference "TP6502") (unit 1))))
+  (instances (project "t1-main-board" (path "/7746052e-d7f9-59ad-ba73-bd2b74439529/7565c505-141d-591d-ab0e-49e98d8f1d5a" (reference "TP6602") (unit 1))))
 )
 (junction (at 215.9 50.8) (diameter 0) (color 0 0 0 0))

Commit message: Board on libs v0.2.0: lower-case kebab vendor keys (HL-13)
The libs submodule moves to v0.2.0 (5f24483). Every library nickname in
the generator, the placement tool and the floorplan study follows the
key table (Texas_Instruments -> texas-instruments, OpenDAP_Device ->
opendap-generic, Rockchip and Rockchip_PMIC -> rockchip, ...); the
library tables are written from the files. Schematic and board
regenerated.

Checks: ERC 0 errors (warnings unchanged); DRC 0 errors, 605 warnings,
the same counts by type, schematic parity 0; every placement identical;
craft Q1 met; pcb tests pass; STEP export resolves every libs 3D model
(the 27 parts without a model are KiCad stock lands that have none).

Co-Authored-By: Claude Opus 5.5 <noreply@anthropic.com>
Claude-Session: https://claude.ai/code/session_01Ei262h3TpgY9vyfNLMi5Mn
Parts:
- U6601: footprint Texas_Instruments:Texas_NJA0024A_WQFN-24-1EP_4x5mm_P0.5mm_EP2.4x3.4mm_ThermalVias -> texas-instruments:Texas_NJA0024A_WQFN-24-1EP_4x5mm_P0.5mm_EP2.4x3.4mm_ThermalVias; symbol Texas_Instruments:LP5521YQX -> texas-instruments:LP5521YQX
Changed lines of the file:
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@@
 (paper "A4")
 (title_block (title "Status LED driver") (date "2026-10-25") (rev "A") (company "The OpenDAP Project") (comment 1 "blk.status-led") (comment 2 "LP5521 RGB LED driver on I2C2 at 0x32: charge pump, LED_R/G/B to the faceplate, link #22"))
-(symbol (lib_id "Texas_Instruments:LP5521YQX") (at 58.42 82.55 0) (unit 1) (body_style 1) (exclude_from_sim no) (in_bom yes) (on_board yes) (dnp no)
+(symbol (lib_id "texas-instruments:LP5521YQX") (at 58.42 82.55 0) (unit 1) (body_style 1) (exclude_from_sim no) (in_bom yes) (on_board yes) (dnp no)
   (property "Reference" "U6601" (at 59.69 50.8 0) (effects (font (size 1.27 1.27)) (justify left)))
   (property "Value" "LP5521YQX" (at 59.69 48.26 0) (effects (font (size 1.27 1.27)) (justify left)))
-  (property "Footprint" "Texas_Instruments:Texas_NJA0024A_WQFN-24-1EP_4x5mm_P0.5mm_EP2.4x3.4mm_ThermalVias" (at 58.42 82.55 0) (effects (font (size 1.27 1.27))) (hide yes))
+  (property "Footprint" "texas-instruments:Texas_NJA0024A_WQFN-24-1EP_4x5mm_P0.5mm_EP2.4x3.4mm_ThermalVias" (at 58.42 82.55 0) (effects (font (size 1.27 1.27))) (hide yes))
   (property "Datasheet" "https://www.ti.com/lit/ds/symlink/lp5521.pdf" (at 58.42 82.55 0) (effects (font (size 1.27 1.27))) (hide yes))
   (property "Description" "Three-channel RGB LED driver, 25.5 mA programmable current sources, 8-bit PWM, program engines, adaptive 1x/1.5x charge pump, I2C, WQFN-24 (NJA0024A) 4 x 5 mm with exposed pad" (at 58.42 82.55 0) (effects (font (size 1.27 1.27))) (hide yes))

Commit message: BOM v1.18 item 2: successors of the discontinued 1 uF 0402
GRM155R61A105KE15D is to be discontinued. 44 positions take
GRM155C71A105KE11D (1 uF 10 V X7S); the eight TPS7A20 positions take
GRM155R61C225KE11D (2.2 uF 16 V X5R) to keep the 0.47 uF effective
minimum with 10 % to spare at up to 3.8 V. Same land; sourcing pass.
Closes BOM §7 item 52; new item 55 lists the other capture parts outside
Murata's product data or near end of life.

Co-Authored-By: Claude Opus 5.5 <noreply@anthropic.com>
Claude-Session: https://claude.ai/code/session_01Ei262h3TpgY9vyfNLMi5Mn
Parts:
- C6601: MPN GRM155R61A105KE15D -> GRM155C71A105KE11D
- C6602: MPN GRM155R61A105KE15D -> GRM155C71A105KE11D; Spec 10 V X5R -> 10 V X7S
Changed lines of the file:
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@@
   (property "Value" "1 µF" (at 93.98 55.88 0) (effects (font (size 1.27 1.27)) (justify left)))
   (property "Footprint" "Capacitor_SMD:C_0402_1005Metric" (at 91.44 54.61 0) (effects (font (size 1.27 1.27))) (hide yes))
-  (property "Datasheet" "https://www.murata.com/en-us/products/productdetail?partno=GRM155R61A105KE15D" (at 91.44 54.61 0) (effects (font (size 1.27 1.27))) (hide yes))
-  (property "Description" "Capacitor, 1 µF, 10 V, X5R, 0402" (at 91.44 54.61 0) (effects (font (size 1.27 1.27))) (hide yes))
+  (property "Datasheet" "https://www.murata.com/en-us/products/productdetail?partno=GRM155C71A105KE11D" (at 91.44 54.61 0) (effects (font (size 1.27 1.27))) (hide yes))
+  (property "Description" "Capacitor, 1 µF, 10 V, X7S, 0402" (at 91.44 54.61 0) (effects (font (size 1.27 1.27))) (hide yes))
   (property "Manufacturer" "Murata" (at 91.44 54.61 0) (effects (font (size 1.27 1.27))) (hide yes))
-  (property "MPN" "GRM155R61A105KE15D" (at 91.44 54.61 0) (effects (font (size 1.27 1.27))) (hide yes))
+  (property "MPN" "GRM155C71A105KE11D" (at 91.44 54.61 0) (effects (font (size 1.27 1.27))) (hide yes))
   (property "Block" "blk.status-led" (at 91.44 54.61 0) (effects (font (size 1.27 1.27))) (hide yes))
   (pin "1")
@@
   (property "Reference" "C6602" (at 106.68 53.34 0) (effects (font (size 1.27 1.27)) (justify left)))
   (property "Value" "1 µF" (at 106.68 55.88 0) (effects (font (size 1.27 1.27)) (justify left)))
-  (property "Spec" "10 V X5R" (at 106.68 58.42 0) (effects (font (size 1.27 1.27)) (justify left)))
+  (property "Spec" "10 V X7S" (at 106.68 58.42 0) (effects (font (size 1.27 1.27)) (justify left)))
   (property "Footprint" "Capacitor_SMD:C_0402_1005Metric" (at 104.14 54.61 0) (effects (font (size 1.27 1.27))) (hide yes))
-  (property "Datasheet" "https://www.murata.com/en-us/products/productdetail?partno=GRM155R61A105KE15D" (at 104.14 54.61 0) (effects (font (size 1.27 1.27))) (hide yes))
-  (property "Description" "Capacitor, 1 µF, 10 V, X5R, 0402" (at 104.14 54.61 0) (effects (font (size 1.27 1.27))) (hide yes))
+  (property "Datasheet" "https://www.murata.com/en-us/products/productdetail?partno=GRM155C71A105KE11D" (at 104.14 54.61 0) (effects (font (size 1.27 1.27))) (hide yes))
+  (property "Description" "Capacitor, 1 µF, 10 V, X7S, 0402" (at 104.14 54.61 0) (effects (font (size 1.27 1.27))) (hide yes))
   (property "Manufacturer" "Murata" (at 104.14 54.61 0) (effects (font (size 1.27 1.27))) (hide yes))
-  (property "MPN" "GRM155R61A105KE15D" (at 104.14 54.61 0) (effects (font (size 1.27 1.27))) (hide yes))
+  (property "MPN" "GRM155C71A105KE11D" (at 104.14 54.61 0) (effects (font (size 1.27 1.27))) (hide yes))
   (property "Block" "blk.status-led" (at 104.14 54.61 0) (effects (font (size 1.27 1.27))) (hide yes))
   (pin "1")
