File: board/hardware/t1-main-board/usb-vbus-out.kicad_sch (KiCad schematic)
At the start: 11 parts, among them U4101 TPS259470ARPWR, U4102 TPS259470ARPWR

Commit message: Board: capture blk.current-monitors
Five INA236 on I2C1 (0x40-0x43, 0x48) with their shunts, per power tree
§4.12 and BOM v1 lines 54 and 136. The measured branches are rails of
their own (VSYS_SRC, VSYS_LV_AUDIO, VSYS_AUDIO, VSYS_LV_BL, VSYS_P5V1),
fed through the shunts on this sheet; the charger, audio, backlight and
5.1 V sheets take them. The root's layout may leave a stack level empty,
so the block sits under the notes; IC bboxes hold turned rail values;
passive rows hold a bottom rail's text.

Co-Authored-By: Claude Opus 5.5 <noreply@anthropic.com>
Claude-Session: https://claude.ai/code/session_01Ei262h3TpgY9vyfNLMi5Mn
Parts:
- removed C4101, C4102, C4103, C4104: 1 µF, Capacitor_SMD:C_0402_1005Metric, symbol Device:C
- removed C4105: 1 nF, Capacitor_SMD:C_0402_1005Metric, symbol Device:C
- removed R4101: 1.47 kΩ, Resistor_SMD:R_0402_1005Metric, symbol Device:R
- removed R4102: 1.87 kΩ, Resistor_SMD:R_0402_1005Metric, symbol Device:R
- removed R4103: 10 kΩ, Resistor_SMD:R_0402_1005Metric, symbol Device:R
- removed TP4101: EFUSE_5V_IMON_ILM, TestPoint:TestPoint_Pad_D1.0mm, symbol Connector:TestPoint
- removed U4101, U4102: TPS259470ARPWR, Texas_Instruments:Texas_RPW0010A_VQFN-HR-10_2x2mm_P0.45mm, symbol Texas_Instruments:TPS259470ARPWR
- added C4201, C4202, C4203, C4204: 1 µF, Capacitor_SMD:C_0402_1005Metric, symbol Device:C
- added C4205: 1 nF, Capacitor_SMD:C_0402_1005Metric, symbol Device:C
- added R4201: 1.47 kΩ, Resistor_SMD:R_0402_1005Metric, symbol Device:R
- added R4202: 1.87 kΩ, Resistor_SMD:R_0402_1005Metric, symbol Device:R
- added R4203: 10 kΩ, Resistor_SMD:R_0402_1005Metric, symbol Device:R
- added TP4201: EFUSE_5V_IMON_ILM, TestPoint:TestPoint_Pad_D1.0mm, symbol Connector:TestPoint
- added U4201, U4202: TPS259470ARPWR, Texas_Instruments:Texas_RPW0010A_VQFN-HR-10_2x2mm_P0.45mm, symbol Texas_Instruments:TPS259470ARPWR
Connections:
- net EFUSE_5V_FLT_N: now also U4201.4 (FLT)
- net EFUSE_5V_IMON_ILM: now also R4201.1, TP4201.1, U4201.9 (ILM)
- net EFUSE_VBUS_FLT_N: now also U4202.4 (FLT)
- net EFUSE_VBUS_IMON: now also C4205.1, R4203.2
- net EFUSE_VBUS_IMON_ILM: now also R4202.1, R4203.1, U4202.9 (ILM)
- net GND: now also C4201.2, C4202.2, C4203.2, C4204.2, C4205.2, R4201.2, R4202.2, U4201.2 (OVLO), U4201.8 (GND), U4202.2 (OVLO), U4202.8 (GND)
- net P5V1_LIM: now also C4202.1, C4203.1, U4201.6 (OUT), U4202.5 (IN)
- net P5V1_SRC: now also C4201.1, U4201.1 (EN/UVLO), U4201.5 (IN)
- net USBC_VBUS: now also C4204.1, U4202.6 (OUT)
- net USB_SRC_ON: now also U4202.1 (EN/UVLO)

Commit message: Board: capture blk.debug
Debug UART2 (1.8 V) and I2S/DSD pads with ground pads, reset, PMIC and
power-key pads (PCB-T-09), a pad on every spare SoC GPIO whose pinout v1
row names one (the DEBUG bus, on the SoC's right edge), and a rail pad
for each power-tree rail no other sheet probes (PCB-T-02). Each DAC
sheet carries a pad on its MCLK. The spares pinout v1 leaves without a
pad now carry no-connect flags. On the root, facing sheet pins are
joined directly only where the route meets no other symbol.

Co-Authored-By: Claude Opus 5.5 <noreply@anthropic.com>
Claude-Session: https://claude.ai/code/session_01Ei262h3TpgY9vyfNLMi5Mn
Parts:
- removed C4201, C4202, C4203, C4204: 1 µF, Capacitor_SMD:C_0402_1005Metric, symbol Device:C
- removed C4205: 1 nF, Capacitor_SMD:C_0402_1005Metric, symbol Device:C
- removed R4201: 1.47 kΩ, Resistor_SMD:R_0402_1005Metric, symbol Device:R
- removed R4202: 1.87 kΩ, Resistor_SMD:R_0402_1005Metric, symbol Device:R
- removed R4203: 10 kΩ, Resistor_SMD:R_0402_1005Metric, symbol Device:R
- removed TP4201: EFUSE_5V_IMON_ILM, TestPoint:TestPoint_Pad_D1.0mm, symbol Connector:TestPoint
- removed U4201, U4202: TPS259470ARPWR, Texas_Instruments:Texas_RPW0010A_VQFN-HR-10_2x2mm_P0.45mm, symbol Texas_Instruments:TPS259470ARPWR
- added C4301, C4302, C4303, C4304: 1 µF, Capacitor_SMD:C_0402_1005Metric, symbol Device:C
- added C4305: 1 nF, Capacitor_SMD:C_0402_1005Metric, symbol Device:C
- added R4301: 1.47 kΩ, Resistor_SMD:R_0402_1005Metric, symbol Device:R
- added R4302: 1.87 kΩ, Resistor_SMD:R_0402_1005Metric, symbol Device:R
- added R4303: 10 kΩ, Resistor_SMD:R_0402_1005Metric, symbol Device:R
- added TP4301: EFUSE_5V_IMON_ILM, TestPoint:TestPoint_Pad_D1.0mm, symbol Connector:TestPoint
- added U4301, U4302: TPS259470ARPWR, Texas_Instruments:Texas_RPW0010A_VQFN-HR-10_2x2mm_P0.45mm, symbol Texas_Instruments:TPS259470ARPWR
Connections:
- net EFUSE_5V_FLT_N: now also U4301.4 (FLT)
- net EFUSE_5V_IMON_ILM: now also R4301.1, TP4301.1, U4301.9 (ILM)
- net EFUSE_VBUS_FLT_N: now also U4302.4 (FLT)
- net EFUSE_VBUS_IMON: now also C4305.1, R4303.2
- net EFUSE_VBUS_IMON_ILM: now also R4302.1, R4303.1, U4302.9 (ILM)
- net GND: now also C4301.2, C4302.2, C4303.2, C4304.2, C4305.2, R4301.2, R4302.2, U4301.2 (OVLO), U4301.8 (GND), U4302.2 (OVLO), U4302.8 (GND)
- net P5V1_LIM: now also C4302.1, C4303.1, U4301.6 (OUT), U4302.5 (IN)
- net P5V1_SRC: now also C4301.1, U4301.1 (EN/UVLO), U4301.5 (IN)
- net USBC_VBUS: now also C4304.1, U4302.6 (OUT)
- net USB_SRC_ON: now also U4302.1 (EN/UVLO)

Commit message: Board: capture blk.mic-ambient and links #34, #35
IM73D122 on PDM CLK1 and SDI1 (BOM v1 line 34, pinout v1 AK2 and 1P2),
LR to ground, 22 Ω clock series, VDD from MIC_1V8 through link #35.
Link #34 on blk.mic-main makes the faceplate branch the rail MIC_1V8_FP
for contact 40 (power tree §4.12, G10). kicad-lib moves to e46bda4 for
the IM73D122, TPS3808G01, SN74LVC1G58 and BAT54 parts.

Co-Authored-By: Claude Opus 5.5 <noreply@anthropic.com>
Claude-Session: https://claude.ai/code/session_01Ei262h3TpgY9vyfNLMi5Mn
Parts:
- removed C4301, C4302, C4303, C4304: 1 µF, Capacitor_SMD:C_0402_1005Metric, symbol Device:C
- removed C4305: 1 nF, Capacitor_SMD:C_0402_1005Metric, symbol Device:C
- removed R4301: 1.47 kΩ, Resistor_SMD:R_0402_1005Metric, symbol Device:R
- removed R4302: 1.87 kΩ, Resistor_SMD:R_0402_1005Metric, symbol Device:R
- removed R4303: 10 kΩ, Resistor_SMD:R_0402_1005Metric, symbol Device:R
- removed TP4301: EFUSE_5V_IMON_ILM, TestPoint:TestPoint_Pad_D1.0mm, symbol Connector:TestPoint
- removed U4301, U4302: TPS259470ARPWR, Texas_Instruments:Texas_RPW0010A_VQFN-HR-10_2x2mm_P0.45mm, symbol Texas_Instruments:TPS259470ARPWR
- added C4401, C4402, C4403, C4404: 1 µF, Capacitor_SMD:C_0402_1005Metric, symbol Device:C
- added C4405: 1 nF, Capacitor_SMD:C_0402_1005Metric, symbol Device:C
- added R4401: 1.47 kΩ, Resistor_SMD:R_0402_1005Metric, symbol Device:R
- added R4402: 1.87 kΩ, Resistor_SMD:R_0402_1005Metric, symbol Device:R
- added R4403: 10 kΩ, Resistor_SMD:R_0402_1005Metric, symbol Device:R
- added TP4401: EFUSE_5V_IMON_ILM, TestPoint:TestPoint_Pad_D1.0mm, symbol Connector:TestPoint
- added U4401, U4402: TPS259470ARPWR, Texas_Instruments:Texas_RPW0010A_VQFN-HR-10_2x2mm_P0.45mm, symbol Texas_Instruments:TPS259470ARPWR
Connections:
- net EFUSE_5V_FLT_N: now also U4401.4 (FLT)
- net EFUSE_5V_IMON_ILM: now also R4401.1, TP4401.1, U4401.9 (ILM)
- net EFUSE_VBUS_FLT_N: now also U4402.4 (FLT)
- net EFUSE_VBUS_IMON: now also C4405.1, R4403.2
- net EFUSE_VBUS_IMON_ILM: now also R4402.1, R4403.1, U4402.9 (ILM)
- net GND: now also C4401.2, C4402.2, C4403.2, C4404.2, C4405.2, R4401.2, R4402.2, U4401.2 (OVLO), U4401.8 (GND), U4402.2 (OVLO), U4402.8 (GND)
- net P5V1_LIM: now also C4402.1, C4403.1, U4401.6 (OUT), U4402.5 (IN)
- net P5V1_SRC: now also C4401.1, U4401.1 (EN/UVLO), U4401.5 (IN)
- net USBC_VBUS: now also C4404.1, U4402.6 (OUT)
- net USB_SRC_ON: now also U4402.1 (EN/UVLO)

Commit message: Board: capture blk.maskrom
Power + Vol- at a cold power-on pull eMMC D0 low inside the TPS3808G01
boot window (BOM v1 lines 35, 78, 97, 98; sim/maskrom): SENSE 280k/100k,
CT 390 nF, WINDOW_N with its pad, SN74LVC1G57 and SN74LVC1G58 on
vcca1v8_pmu, BAT54 from PWRON_N, DMG1012T through 1 kΩ to EMMC_D0.
Every block in use now has its sheet; the README states the remaining
single-pin nets.

Co-Authored-By: Claude Opus 5.5 <noreply@anthropic.com>
Claude-Session: https://claude.ai/code/session_01Ei262h3TpgY9vyfNLMi5Mn
Parts:
- removed C4401, C4402, C4403, C4404: 1 µF, Capacitor_SMD:C_0402_1005Metric, symbol Device:C
- removed C4405: 1 nF, Capacitor_SMD:C_0402_1005Metric, symbol Device:C
- removed R4401: 1.47 kΩ, Resistor_SMD:R_0402_1005Metric, symbol Device:R
- removed R4402: 1.87 kΩ, Resistor_SMD:R_0402_1005Metric, symbol Device:R
- removed R4403: 10 kΩ, Resistor_SMD:R_0402_1005Metric, symbol Device:R
- removed TP4401: EFUSE_5V_IMON_ILM, TestPoint:TestPoint_Pad_D1.0mm, symbol Connector:TestPoint
- removed U4401, U4402: TPS259470ARPWR, Texas_Instruments:Texas_RPW0010A_VQFN-HR-10_2x2mm_P0.45mm, symbol Texas_Instruments:TPS259470ARPWR
- added C4501, C4502, C4503, C4504: 1 µF, Capacitor_SMD:C_0402_1005Metric, symbol Device:C
- added C4505: 1 nF, Capacitor_SMD:C_0402_1005Metric, symbol Device:C
- added R4501: 1.47 kΩ, Resistor_SMD:R_0402_1005Metric, symbol Device:R
- added R4502: 1.87 kΩ, Resistor_SMD:R_0402_1005Metric, symbol Device:R
- added R4503: 10 kΩ, Resistor_SMD:R_0402_1005Metric, symbol Device:R
- added TP4501: EFUSE_5V_IMON_ILM, TestPoint:TestPoint_Pad_D1.0mm, symbol Connector:TestPoint
- added U4501, U4502: TPS259470ARPWR, Texas_Instruments:Texas_RPW0010A_VQFN-HR-10_2x2mm_P0.45mm, symbol Texas_Instruments:TPS259470ARPWR
Connections:
- net EFUSE_5V_FLT_N: now also U4501.4 (FLT)
- net EFUSE_5V_IMON_ILM: now also R4501.1, TP4501.1, U4501.9 (ILM)
- net EFUSE_VBUS_FLT_N: now also U4502.4 (FLT)
- net EFUSE_VBUS_IMON: now also C4505.1, R4503.2
- net EFUSE_VBUS_IMON_ILM: now also R4502.1, R4503.1, U4502.9 (ILM)
- net GND: now also C4501.2, C4502.2, C4503.2, C4504.2, C4505.2, R4501.2, R4502.2, U4501.2 (OVLO), U4501.8 (GND), U4502.2 (OVLO), U4502.8 (GND)
- net P5V1_LIM: now also C4502.1, C4503.1, U4501.6 (OUT), U4502.5 (IN)
- net P5V1_SRC: now also C4501.1, U4501.1 (EN/UVLO), U4501.5 (IN)
- net USBC_VBUS: now also C4504.1, U4502.6 (OUT)
- net USB_SRC_ON: now also U4502.1 (EN/UVLO)

Commit message: Compaction: lower inductors, 0201 decoupling, 0.8 mm signal test pads
A matrix tool (hardware/studies/compaction) checks each candidate against
the design's stresses: same inductance, design peak <= 70 % and the
converter's maximum limit <= 100 % of Isat (30 % drop), height zones,
ratings at least twice the rail, PCB-D-06; sourcing outcome per part.

Applied (placement v1 decision 12, BOM v1.15):
- L601, L4401: XGL4015-102MEC (1.5 mm) for XAL/XGL4020-102MEC (2.1 mm);
- L1001, L5101: XGL4015-471MEC (1.5 mm) for Wurth 744373240047, on the
  stock XxL4020 land (the Wurth land was never drawn);
- L1201 is 1.2 mm (XGL4012, per-MPN heights): it moves next to the SoC;
- 58 x 100 nF decoupling on rails <= 3.3 V in core/IO/radio: 0201;
- 51 test pads on signal nets: 0.8 mm (PCB-D-06 v0.16, JLCPCB guide).
Kept: L901, L2802 (XGL4015 at 103 % of Isat at the limit); no thinner
0805/1206 capacitor passes (obsolete, NRND or unlisted).

Board need 113 % -> 111 % (core band 227 -> 203 %, power band 258 ->
233 %, radio band 19 -> 0 %); only C904 still relies on PCB-Z-04.
ERC 0 errors, craft Q1 met, DRC 0 errors (605 warnings), pcb and study
tests pass, rules test board PASS.

Co-Authored-By: Claude Opus 5.5 <noreply@anthropic.com>
Claude-Session: https://claude.ai/code/session_01Ei262h3TpgY9vyfNLMi5Mn
Parts:
- TP4501: footprint TestPoint:TestPoint_Pad_D1.0mm -> T1_Main_Board:TestPoint_Pad_D0.8mm
Changed lines of the file:
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@@
   (property "Reference" "TP4501" (at 104.14 83.82 0) (effects (font (size 1.27 1.27)) (justify right)))
   (property "Value" "EFUSE_5V_IMON_ILM" (at 104.14 86.36 0) (effects (font (size 1.27 1.27)) (justify right)))
-  (property "Footprint" "TestPoint:TestPoint_Pad_D1.0mm" (at 105.41 88.9 0) (effects (font (size 1.27 1.27))) (hide yes))
+  (property "Footprint" "T1_Main_Board:TestPoint_Pad_D0.8mm" (at 105.41 88.9 0) (effects (font (size 1.27 1.27))) (hide yes))
   (property "Datasheet" "~" (at 105.41 88.9 0) (effects (font (size 1.27 1.27))) (hide yes))
-  (property "Description" "Test pad, 1.0 mm" (at 105.41 88.9 0) (effects (font (size 1.27 1.27))) (hide yes))
+  (property "Description" "Test pad, 0.8 mm, signal net" (at 105.41 88.9 0) (effects (font (size 1.27 1.27))) (hide yes))
   (property "Block" "blk.usb-vbus-out" (at 105.41 88.9 0) (effects (font (size 1.27 1.27))) (hide yes))
   (pin "1")

Commit message: Board on libs v0.2.0: lower-case kebab vendor keys (HL-13)
The libs submodule moves to v0.2.0 (5f24483). Every library nickname in
the generator, the placement tool and the floorplan study follows the
key table (Texas_Instruments -> texas-instruments, OpenDAP_Device ->
opendap-generic, Rockchip and Rockchip_PMIC -> rockchip, ...); the
library tables are written from the files. Schematic and board
regenerated.

Checks: ERC 0 errors (warnings unchanged); DRC 0 errors, 605 warnings,
the same counts by type, schematic parity 0; every placement identical;
craft Q1 met; pcb tests pass; STEP export resolves every libs 3D model
(the 27 parts without a model are KiCad stock lands that have none).

Co-Authored-By: Claude Opus 5.5 <noreply@anthropic.com>
Claude-Session: https://claude.ai/code/session_01Ei262h3TpgY9vyfNLMi5Mn
Parts:
- U4501, U4502: footprint Texas_Instruments:Texas_RPW0010A_VQFN-HR-10_2x2mm_P0.45mm -> texas-instruments:Texas_RPW0010A_VQFN-HR-10_2x2mm_P0.45mm; symbol Texas_Instruments:TPS259470ARPWR -> texas-instruments:TPS259470ARPWR
Changed lines of the file:
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@@
 (paper "A3")
 (title_block (title "USB-C source path") (date "2026-10-25") (rev "A") (company "The OpenDAP Project") (comment 1 "blk.usb-vbus-out") (comment 2 "eFuse #D, the shared 5.1 V limiter, and eFuse #C to the USB-C VBUS"))
-(symbol (lib_id "Texas_Instruments:TPS259470ARPWR") (at 53.34 80.01 0) (unit 1) (body_style 1) (exclude_from_sim no) (in_bom yes) (on_board yes) (dnp no)
+(symbol (lib_id "texas-instruments:TPS259470ARPWR") (at 53.34 80.01 0) (unit 1) (body_style 1) (exclude_from_sim no) (in_bom yes) (on_board yes) (dnp no)
   (property "Reference" "U4501" (at 41.91 58.42 0) (effects (font (size 1.27 1.27)) (justify left)))
   (property "Value" "TPS259470ARPWR" (at 41.91 55.88 0) (effects (font (size 1.27 1.27)) (justify left)))
-  (property "Footprint" "Texas_Instruments:Texas_RPW0010A_VQFN-HR-10_2x2mm_P0.45mm" (at 53.34 80.01 0) (effects (font (size 1.27 1.27))) (hide yes))
+  (property "Footprint" "texas-instruments:Texas_RPW0010A_VQFN-HR-10_2x2mm_P0.45mm" (at 53.34 80.01 0) (effects (font (size 1.27 1.27))) (hide yes))
   (property "Datasheet" "https://www.ti.com/lit/ds/symlink/tps25947.pdf" (at 53.34 80.01 0) (effects (font (size 1.27 1.27))) (hide yes))
   (property "Description" "eFuse, 2.7-23 V, 5.5 A, 28 mOhm, true reverse-current blocking, adjustable UVLO/OVLO and current limit, AUXOFF and FLT outputs, auto-retry, VQFN-HR-10 (RPW0010A) 2 x 2 mm" (at 53.34 80.01 0) (effects (font (size 1.27 1.27))) (hide yes))
@@
 (rectangle (start 22.86 35.56) (end 167.64 114.3) (stroke (width 0) (type dash)) (fill (type none)))
 (text "eFuse #D, shared limiter, RILM 1.47 kΩ (BOM v1 line 44, v1.14)" (exclude_from_sim no) (at 24.13 34.29 0) (effects (font (size 2.54 2.54)) (justify left bottom)))
-(symbol (lib_id "Texas_Instruments:TPS259470ARPWR") (at 205.74 81.28 0) (unit 1) (body_style 1) (exclude_from_sim no) (in_bom yes) (on_board yes) (dnp no)
+(symbol (lib_id "texas-instruments:TPS259470ARPWR") (at 205.74 81.28 0) (unit 1) (body_style 1) (exclude_from_sim no) (in_bom yes) (on_board yes) (dnp no)
   (property "Reference" "U4502" (at 194.31 59.69 0) (effects (font (size 1.27 1.27)) (justify left)))
   (property "Value" "TPS259470ARPWR" (at 194.31 57.15 0) (effects (font (size 1.27 1.27)) (justify left)))
-  (property "Footprint" "Texas_Instruments:Texas_RPW0010A_VQFN-HR-10_2x2mm_P0.45mm" (at 205.74 81.28 0) (effects (font (size 1.27 1.27))) (hide yes))
+  (property "Footprint" "texas-instruments:Texas_RPW0010A_VQFN-HR-10_2x2mm_P0.45mm" (at 205.74 81.28 0) (effects (font (size 1.27 1.27))) (hide yes))
   (property "Datasheet" "https://www.ti.com/lit/ds/symlink/tps25947.pdf" (at 205.74 81.28 0) (effects (font (size 1.27 1.27))) (hide yes))
   (property "Description" "eFuse, 2.7-23 V, 5.5 A, 28 mOhm, true reverse-current blocking, adjustable UVLO/OVLO and current limit, AUXOFF and FLT outputs, auto-retry, VQFN-HR-10 (RPW0010A) 2 x 2 mm" (at 205.74 81.28 0) (effects (font (size 1.27 1.27))) (hide yes))
