File: board/hardware/t1-main-board/fp-display.kicad_sch (KiCad schematic)
At the start: 7 parts, among them U6001 TPS22945DCKR

Commit message: NFC reader withdrawn from the board, every model (BRD-057)
Maintainer decision 2026-10-27, reason: board area. blk.nfc-reader (#42)
withdrawn: PN7160, front end, crystal, antenna contacts, NFC_VBAT switch
and link #18 removed (35 parts). BRD-057 reworded: NFC as the dynamic tag
only; blk.nfc-tag stays. Pinout v1: 1N20, A37, B38 become unconnected
spares, expander P05 a spare. BOM v1.18 item 7 (line 50: 5 switches,
lines 127-128 withdrawn), power tree v0.10, variant files, feature blocks.

Sheets after the removed one move up a page; references renumbered in
plan.py, parts.py and the specs (J6201 -> J6101 and others).

Placement v1.4: 990 parts placed, board need 96.9 % (99.1 % before),
factor 1.72; 243 capacitors within bound; DRC 0 errors; ERC 0 errors;
craft Q1 met; overlaps 0; pcb tests pass; STEP exported.

Co-Authored-By: Claude Opus 5.5 <noreply@anthropic.com>
Claude-Session: https://claude.ai/code/session_01Ei262h3TpgY9vyfNLMi5Mn
Parts:
- removed C6001, C6002: 1 µF, Capacitor_SMD:C_0402_1005Metric, symbol Device:C
- removed R6001: 10 kΩ, Resistor_SMD:R_0201_0603Metric, symbol Device:R
- removed R6002: 100 mΩ, Resistor_SMD:R_0603_1608Metric, symbol Device:R
- removed TP6001: FP_VCI_OUT, TestPoint:TestPoint_Pad_D1.0mm, symbol Connector:TestPoint
- removed TP6002: FP_VCI, TestPoint:TestPoint_Pad_D1.0mm, symbol Connector:TestPoint
- removed U6001: TPS22945DCKR, texas-instruments:Texas_DCK0005A_SC-70-5_1.25x2mm_P0.65mm, symbol texas-instruments:TPS22945DCKR
- added C5901, C5902: 1 µF, Capacitor_SMD:C_0402_1005Metric, symbol Device:C
- added R5901: 10 kΩ, Resistor_SMD:R_0201_0603Metric, symbol Device:R
- added R5902: 100 mΩ, Resistor_SMD:R_0603_1608Metric, symbol Device:R
- added TP5901: FP_VCI_OUT, TestPoint:TestPoint_Pad_D1.0mm, symbol Connector:TestPoint
- added TP5902: FP_VCI, TestPoint:TestPoint_Pad_D1.0mm, symbol Connector:TestPoint
- added U5901: TPS22945DCKR, texas-instruments:Texas_DCK0005A_SC-70-5_1.25x2mm_P0.65mm, symbol texas-instruments:TPS22945DCKR
Connections:
- net FP_IO_EN: now also U5901.4 (ON)
- net FP_VCI: now also R5902.2, TP5902.1
- net FP_VCI_OUT: now also C5902.1, R5901.1, R5902.1, TP5901.1, U5901.1 (VOUT)
- net FP_VCI_SRC: now also C5901.1, U5901.5 (VIN)
- net GND: now also C5901.2, C5902.2, R5901.2, U5901.2 (GND)
Changed lines of the file:
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@@
 (title_block (title "Faceplate display supply") (date "2026-10-25") (rev "A") (company "The OpenDAP Project") (comment 1 "blk.fp-display") (comment 2 "FP_VCI current-limited switch after RK809 LDO4; DSI lanes pass to the connector"))
 (symbol (lib_id "texas-instruments:TPS22945DCKR") (at 48.26 60.96 0) (unit 1) (body_style 1) (exclude_from_sim no) (in_bom yes) (on_board yes) (dnp no)
-  (property "Reference" "U6001" (at 49.53 45.72 0) (effects (font (size 1.27 1.27)) (justify left)))
+  (property "Reference" "U5901" (at 49.53 45.72 0) (effects (font (size 1.27 1.27)) (justify left)))
   (property "Value" "TPS22945DCKR" (at 49.53 43.18 0) (effects (font (size 1.27 1.27)) (justify left)))
   (property "Footprint" "texas-instruments:Texas_DCK0005A_SC-70-5_1.25x2mm_P0.65mm" (at 48.26 60.96 0) (effects (font (size 1.27 1.27))) (hide yes))
@@
   (pin "5")
   (pin "2")
-  (instances (project "t1-main-board" (path "/7746052e-d7f9-59ad-ba73-bd2b74439529/996ec8da-1510-50ce-b9cf-a8f3bb19efac" (reference "U6001") (unit 1))))
+  (instances (project "t1-main-board" (path "/7746052e-d7f9-59ad-ba73-bd2b74439529/996ec8da-1510-50ce-b9cf-a8f3bb19efac" (reference "U5901") (unit 1))))
 )
 (wire (pts (xy 38.1 60.96) (xy 35.56 60.96)) (stroke (width 0) (type default)))
@@
 )
 (symbol (lib_id "Device:C") (at 78.74 57.15 0) (unit 1) (body_style 1) (exclude_from_sim no) (in_bom yes) (on_board yes) (dnp no)
-  (property "Reference" "C6001" (at 81.28 55.88 0) (effects (font (size 1.27 1.27)) (justify left)))
+  (property "Reference" "C5901" (at 81.28 55.88 0) (effects (font (size 1.27 1.27)) (justify left)))
   (property "Value" "1 µF" (at 81.28 58.42 0) (effects (font (size 1.27 1.27)) (justify left)))
   (property "Footprint" "Capacitor_SMD:C_0402_1005Metric" (at 78.74 57.15 0) (effects (font (size 1.27 1.27))) (hide yes))
@@
   (pin "1")
   (pin "2")
-  (instances (project "t1-main-board" (path "/7746052e-d7f9-59ad-ba73-bd2b74439529/996ec8da-1510-50ce-b9cf-a8f3bb19efac" (reference "C6001") (unit 1))))
+  (instances (project "t1-main-board" (path "/7746052e-d7f9-59ad-ba73-bd2b74439529/996ec8da-1510-50ce-b9cf-a8f3bb19efac" (reference "C5901") (unit 1))))
 )
 (wire (pts (xy 78.74 53.34) (xy 78.74 50.8)) (stroke (width 0) (type default)))
@@
 )
 (symbol (lib_id "Device:C") (at 91.44 57.15 0) (unit 1) (body_style 1) (exclude_from_sim no) (in_bom yes) (on_board yes) (dnp no)
-  (property "Reference" "C6002" (at 93.98 55.88 0) (effects (font (size 1.27 1.27)) (justify left)))
+  (property "Reference" "C5902" (at 93.98 55.88 0) (effects (font (size 1.27 1.27)) (justify left)))
   (property "Value" "1 µF" (at 93.98 58.42 0) (effects (font (size 1.27 1.27)) (justify left)))
   (property "Footprint" "Capacitor_SMD:C_0402_1005Metric" (at 91.44 57.15 0) (effects (font (size 1.27 1.27))) (hide yes))
@@
   (pin "1")
   (pin "2")
-  (instances (project "t1-main-board" (path "/7746052e-d7f9-59ad-ba73-bd2b74439529/996ec8da-1510-50ce-b9cf-a8f3bb19efac" (reference "C6002") (unit 1))))
+  (instances (project "t1-main-board" (path "/7746052e-d7f9-59ad-ba73-bd2b74439529/996ec8da-1510-50ce-b9cf-a8f3bb19efac" (reference "C5902") (unit 1))))
 )
 (wire (pts (xy 91.44 53.34) (xy 91.44 50.8)) (stroke (width 0) (type default)))
@@
 )
 (symbol (lib_id "Device:R") (at 104.14 57.15 0) (unit 1) (body_style 1) (exclude_from_sim no) (in_bom yes) (on_board yes) (dnp no)
-  (property "Reference" "R6001" (at 105.41 55.88 0) (effects (font (size 1.27 1.27)) (justify left)))
+  (property "Reference" "R5901" (at 105.41 55.88 0) (effects (font (size 1.27 1.27)) (justify left)))
   (property "Value" "10 kΩ" (at 105.41 58.42 0) (effects (font (size 1.27 1.27)) (justify left)))
   (property "Footprint" "Resistor_SMD:R_0201_0603Metric" (at 104.14 57.15 0) (effects (font (size 1.27 1.27))) (hide yes))
@@
   (pin "1")
   (pin "2")
-  (instances (project "t1-main-board" (path "/7746052e-d7f9-59ad-ba73-bd2b74439529/996ec8da-1510-50ce-b9cf-a8f3bb19efac" (reference "R6001") (unit 1))))
+  (instances (project "t1-main-board" (path "/7746052e-d7f9-59ad-ba73-bd2b74439529/996ec8da-1510-50ce-b9cf-a8f3bb19efac" (reference "R5901") (unit 1))))
 )
 (wire (pts (xy 104.14 53.34) (xy 104.14 50.8)) (stroke (width 0) (type default)))
@@
 (text "FP_VCI: TPS22945 after RK809 LDO4 (BOM v1 line 146)" (exclude_from_sim no) (at 24.13 34.29 0) (effects (font (size 2.54 2.54)) (justify left bottom)))
 (symbol (lib_id "Device:R") (at 184.15 50.8 90) (unit 1) (body_style 1) (exclude_from_sim no) (in_bom yes) (on_board yes) (dnp no)
-  (property "Reference" "R6002" (at 181.61 46.99 90) (effects (font (size 1.27 1.27))))
+  (property "Reference" "R5902" (at 181.61 46.99 90) (effects (font (size 1.27 1.27))))
   (property "Value" "100 mΩ" (at 181.61 53.34 90) (effects (font (size 1.27 1.27))))
   (property "Spec" "0603" (at 181.61 55.88 90) (effects (font (size 1.27 1.27))))
@@
   (pin "1")
   (pin "2")
-  (instances (project "t1-main-board" (path "/7746052e-d7f9-59ad-ba73-bd2b74439529/996ec8da-1510-50ce-b9cf-a8f3bb19efac" (reference "R6002") (unit 1) (variant (name "production") (field (name "Value") (value "0 Ω")) (field (name "MPN") (value "RC0603JR-070RL")) (field (name "Manufacturer") (value "YAGEO"))))))
+  (instances (project "t1-main-board" (path "/7746052e-d7f9-59ad-ba73-bd2b74439529/996ec8da-1510-50ce-b9cf-a8f3bb19efac" (reference "R5902") (unit 1) (variant (name "production") (field (name "Value") (value "0 Ω")) (field (name "MPN") (value "RC0603JR-070RL")) (field (name "Manufacturer") (value "YAGEO"))))))
 )
 (rectangle (start 162.56 38.1) (end 200.66 58.42) (stroke (width 0) (type dash)) (fill (type none)))
@@
 (wire (pts (xy 177.8 50.8) (xy 177.8 48.26)) (stroke (width 0) (type default)))
 (symbol (lib_id "Connector:TestPoint") (at 177.8 48.26 0) (unit 1) (body_style 1) (exclude_from_sim no) (in_bom no) (on_board yes) (dnp no)
-  (property "Reference" "TP6001" (at 176.53 43.18 0) (effects (font (size 1.27 1.27)) (justify right)))
+  (property "Reference" "TP5901" (at 176.53 43.18 0) (effects (font (size 1.27 1.27)) (justify right)))
   (property "Value" "FP_VCI_OUT" (at 176.53 45.72 0) (effects (font (size 1.27 1.27)) (justify right)))
   (property "Footprint" "TestPoint:TestPoint_Pad_D1.0mm" (at 177.8 48.26 0) (effects (font (size 1.27 1.27))) (hide yes))
@@
   (property "Block" "blk.fp-display" (at 177.8 48.26 0) (effects (font (size 1.27 1.27))) (hide yes))
   (pin "1")
-  (instances (project "t1-main-board" (path "/7746052e-d7f9-59ad-ba73-bd2b74439529/996ec8da-1510-50ce-b9cf-a8f3bb19efac" (reference "TP6001") (unit 1))))
+  (instances (project "t1-main-board" (path "/7746052e-d7f9-59ad-ba73-bd2b74439529/996ec8da-1510-50ce-b9cf-a8f3bb19efac" (reference "TP5901") (unit 1))))
 )
 (wire (pts (xy 187.96 50.8) (xy 213.36 50.8)) (stroke (width 0) (type default)))
@@
 (wire (pts (xy 190.5 50.8) (xy 190.5 48.26)) (stroke (width 0) (type default)))
 (symbol (lib_id "Connector:TestPoint") (at 190.5 48.26 0) (unit 1) (body_style 1) (exclude_from_sim no) (in_bom no) (on_board yes) (dnp no)
-  (property "Reference" "TP6002" (at 191.77 43.18 0) (effects (font (size 1.27 1.27)) (justify left)))
+  (property "Reference" "TP5902" (at 191.77 43.18 0) (effects (font (size 1.27 1.27)) (justify left)))
   (property "Value" "FP_VCI" (at 191.77 45.72 0) (effects (font (size 1.27 1.27)) (justify left)))
   (property "Footprint" "TestPoint:TestPoint_Pad_D1.0mm" (at 190.5 48.26 0) (effects (font (size 1.27 1.27))) (hide yes))
@@
   (property "Block" "blk.fp-display" (at 190.5 48.26 0) (effects (font (size 1.27 1.27))) (hide yes))
   (pin "1")
-  (instances (project "t1-main-board" (path "/7746052e-d7f9-59ad-ba73-bd2b74439529/996ec8da-1510-50ce-b9cf-a8f3bb19efac" (reference "TP6002") (unit 1))))
+  (instances (project "t1-main-board" (path "/7746052e-d7f9-59ad-ba73-bd2b74439529/996ec8da-1510-50ce-b9cf-a8f3bb19efac" (reference "TP5902") (unit 1))))
 )
 (symbol (lib_id "power:VCC") (at 213.36 50.8 270) (unit 1) (body_style 1) (exclude_from_sim no) (in_bom yes) (on_board yes) (dnp no)
