File: board/hardware/t1-main-board/antennas.kicad_sch (KiCad schematic)
At the start: 9 parts, among them J4801 U.FL-R-SMT-1, J4802 U.FL-R-SMT-1

Commit message: Board: capture blk.current-monitors
Five INA236 on I2C1 (0x40-0x43, 0x48) with their shunts, per power tree
§4.12 and BOM v1 lines 54 and 136. The measured branches are rails of
their own (VSYS_SRC, VSYS_LV_AUDIO, VSYS_AUDIO, VSYS_LV_BL, VSYS_P5V1),
fed through the shunts on this sheet; the charger, audio, backlight and
5.1 V sheets take them. The root's layout may leave a stack level empty,
so the block sits under the notes; IC bboxes hold turned rail values;
passive rows hold a bottom rail's text.

Co-Authored-By: Claude Opus 5.5 <noreply@anthropic.com>
Claude-Session: https://claude.ai/code/session_01Ei262h3TpgY9vyfNLMi5Mn
Parts:
- removed C4801, C4802, C4803, C4804: DNP, Capacitor_SMD:C_0201_0603Metric, symbol Device:C
- removed C4805: 10 pF, Capacitor_SMD:C_0201_0603Metric, symbol Device:C
- removed J4801, J4802: U.FL-R-SMT-1, Hirose:Hirose_U.FL-R-SMT-1_Vertical, symbol Hirose:U.FL-R-SMT-1
- removed R4801, R4802: 0 Ω, Resistor_SMD:R_0201_0603Metric, symbol Device:R
- added C4901, C4902, C4903, C4904: DNP, Capacitor_SMD:C_0201_0603Metric, symbol Device:C
- added C4905: 10 pF, Capacitor_SMD:C_0201_0603Metric, symbol Device:C
- added J4901, J4902: U.FL-R-SMT-1, Hirose:Hirose_U.FL-R-SMT-1_Vertical, symbol Hirose:U.FL-R-SMT-1
- added R4901, R4902: 0 Ω, Resistor_SMD:R_0201_0603Metric, symbol Device:R
Connections:
- net GND: now also C4901.2, C4902.2, C4903.2, C4904.2, J4901.2 (GND), J4902.2 (GND)
- net WL_ANT0: now also C4901.1, R4901.1
- net WL_ANT0_J: now also C4902.1, J4901.1 (SIG), R4901.2
- net WL_ANT1: now also C4903.1, C4905.2, R4902.1
- net WL_ANT1_J: now also C4904.1, J4902.1 (SIG), R4902.2
- net WL_BT_IN: now also C4905.1
Changed lines of the file:
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@@
 (title_block (title "Antenna feeds") (date "2026-10-25") (rev "A") (company "The OpenDAP Project") (comment 1 "blk.antennas") (comment 2 "ANT0 and ANT1 paths as Murata's copy: matching positions, U.FL, the 10 pF shared link"))
 (symbol (lib_id "Device:R") (at 40.64 48.26 90) (unit 1) (body_style 1) (exclude_from_sim no) (in_bom yes) (on_board yes) (dnp no)
-  (property "Reference" "R4801" (at 40.64 45.72 90) (effects (font (size 1.27 1.27))))
+  (property "Reference" "R4901" (at 40.64 45.72 90) (effects (font (size 1.27 1.27))))
   (property "Value" "0 Ω" (at 40.64 50.8 90) (effects (font (size 1.27 1.27))))
   (property "Footprint" "Resistor_SMD:R_0201_0603Metric" (at 40.64 48.26 0) (effects (font (size 1.27 1.27))) (hide yes))
@@
   (pin "1")
   (pin "2")
-  (instances (project "t1-main-board" (path "/7746052e-d7f9-59ad-ba73-bd2b74439529/cd42149b-9c25-54cb-87d6-a01fc7fce92f" (reference "R4801") (unit 1))))
+  (instances (project "t1-main-board" (path "/7746052e-d7f9-59ad-ba73-bd2b74439529/cd42149b-9c25-54cb-87d6-a01fc7fce92f" (reference "R4901") (unit 1))))
 )
 (wire (pts (xy 36.83 48.26) (xy 34.29 48.26)) (stroke (width 0) (type default)))
 (wire (pts (xy 44.45 48.26) (xy 46.99 48.26)) (stroke (width 0) (type default)))
 (symbol (lib_id "Device:C") (at 33.02 78.74 0) (unit 1) (body_style 1) (exclude_from_sim no) (in_bom no) (on_board yes) (dnp yes)
-  (property "Reference" "C4801" (at 35.56 77.47 0) (effects (font (size 1.27 1.27)) (justify left)))
+  (property "Reference" "C4901" (at 35.56 77.47 0) (effects (font (size 1.27 1.27)) (justify left)))
   (property "Value" "DNP" (at 35.56 80.01 0) (effects (font (size 1.27 1.27)) (justify left)))
   (property "Footprint" "Capacitor_SMD:C_0201_0603Metric" (at 33.02 78.74 0) (effects (font (size 1.27 1.27))) (hide yes))
@@
   (pin "1")
   (pin "2")
-  (instances (project "t1-main-board" (path "/7746052e-d7f9-59ad-ba73-bd2b74439529/cd42149b-9c25-54cb-87d6-a01fc7fce92f" (reference "C4801") (unit 1))))
+  (instances (project "t1-main-board" (path "/7746052e-d7f9-59ad-ba73-bd2b74439529/cd42149b-9c25-54cb-87d6-a01fc7fce92f" (reference "C4901") (unit 1))))
 )
 (wire (pts (xy 33.02 74.93) (xy 33.02 72.39)) (stroke (width 0) (type default)))
@@
 )
 (symbol (lib_id "Device:C") (at 45.72 78.74 0) (unit 1) (body_style 1) (exclude_from_sim no) (in_bom no) (on_board yes) (dnp yes)
-  (property "Reference" "C4802" (at 48.26 77.47 0) (effects (font (size 1.27 1.27)) (justify left)))
+  (property "Reference" "C4902" (at 48.26 77.47 0) (effects (font (size 1.27 1.27)) (justify left)))
   (property "Value" "DNP" (at 48.26 80.01 0) (effects (font (size 1.27 1.27)) (justify left)))
   (property "Footprint" "Capacitor_SMD:C_0201_0603Metric" (at 45.72 78.74 0) (effects (font (size 1.27 1.27))) (hide yes))
@@
   (pin "1")
   (pin "2")
-  (instances (project "t1-main-board" (path "/7746052e-d7f9-59ad-ba73-bd2b74439529/cd42149b-9c25-54cb-87d6-a01fc7fce92f" (reference "C4802") (unit 1))))
+  (instances (project "t1-main-board" (path "/7746052e-d7f9-59ad-ba73-bd2b74439529/cd42149b-9c25-54cb-87d6-a01fc7fce92f" (reference "C4902") (unit 1))))
 )
 (wire (pts (xy 45.72 74.93) (xy 45.72 72.39)) (stroke (width 0) (type default)))
@@
 )
 (symbol (lib_id "Hirose:U.FL-R-SMT-1") (at 78.74 53.34 0) (unit 1) (body_style 1) (exclude_from_sim no) (in_bom yes) (on_board yes) (dnp no)
-  (property "Reference" "J4801" (at 73.66 43.18 0) (effects (font (size 1.27 1.27)) (justify left)))
+  (property "Reference" "J4901" (at 73.66 43.18 0) (effects (font (size 1.27 1.27)) (justify left)))
   (property "Value" "U.FL-R-SMT-1" (at 73.66 40.64 0) (effects (font (size 1.27 1.27)) (justify left)))
   (property "Footprint" "Hirose:Hirose_U.FL-R-SMT-1_Vertical" (at 78.74 53.34 0) (effects (font (size 1.27 1.27))) (hide yes))
@@
   (pin "1")
   (pin "2")
-  (instances (project "t1-main-board" (path "/7746052e-d7f9-59ad-ba73-bd2b74439529/cd42149b-9c25-54cb-87d6-a01fc7fce92f" (reference "J4801") (unit 1))))
+  (instances (project "t1-main-board" (path "/7746052e-d7f9-59ad-ba73-bd2b74439529/cd42149b-9c25-54cb-87d6-a01fc7fce92f" (reference "J4901") (unit 1))))
 )
 (wire (pts (xy 71.12 50.8) (xy 68.58 50.8)) (stroke (width 0) (type default)))
@@
 (text "ANT0: Wi-Fi 2.4 / 5 GHz and Bluetooth (shared, ADR 0018)" (exclude_from_sim no) (at 24.13 34.29 0) (effects (font (size 2.54 2.54)) (justify left bottom)))
 (symbol (lib_id "Device:R") (at 176.53 48.26 90) (unit 1) (body_style 1) (exclude_from_sim no) (in_bom yes) (on_board yes) (dnp yes)
-  (property "Reference" "R4802" (at 176.53 45.72 90) (effects (font (size 1.27 1.27))))
+  (property "Reference" "R4902" (at 176.53 45.72 90) (effects (font (size 1.27 1.27))))
   (property "Value" "0 Ω" (at 176.53 50.8 90) (effects (font (size 1.27 1.27))))
   (property "Footprint" "Resistor_SMD:R_0201_0603Metric" (at 176.53 48.26 0) (effects (font (size 1.27 1.27))) (hide yes))
@@
   (pin "1")
   (pin "2")
-  (instances (project "t1-main-board" (path "/7746052e-d7f9-59ad-ba73-bd2b74439529/cd42149b-9c25-54cb-87d6-a01fc7fce92f" (reference "R4802") (unit 1))))
+  (instances (project "t1-main-board" (path "/7746052e-d7f9-59ad-ba73-bd2b74439529/cd42149b-9c25-54cb-87d6-a01fc7fce92f" (reference "R4902") (unit 1))))
 )
 (wire (pts (xy 172.72 48.26) (xy 170.18 48.26)) (stroke (width 0) (type default)))
 (wire (pts (xy 180.34 48.26) (xy 182.88 48.26)) (stroke (width 0) (type default)))
 (symbol (lib_id "Device:C") (at 168.91 78.74 0) (unit 1) (body_style 1) (exclude_from_sim no) (in_bom no) (on_board yes) (dnp yes)
-  (property "Reference" "C4803" (at 171.45 77.47 0) (effects (font (size 1.27 1.27)) (justify left)))
+  (property "Reference" "C4903" (at 171.45 77.47 0) (effects (font (size 1.27 1.27)) (justify left)))
   (property "Value" "DNP" (at 171.45 80.01 0) (effects (font (size 1.27 1.27)) (justify left)))
   (property "Footprint" "Capacitor_SMD:C_0201_0603Metric" (at 168.91 78.74 0) (effects (font (size 1.27 1.27))) (hide yes))
@@
   (pin "1")
   (pin "2")
-  (instances (project "t1-main-board" (path "/7746052e-d7f9-59ad-ba73-bd2b74439529/cd42149b-9c25-54cb-87d6-a01fc7fce92f" (reference "C4803") (unit 1))))
+  (instances (project "t1-main-board" (path "/7746052e-d7f9-59ad-ba73-bd2b74439529/cd42149b-9c25-54cb-87d6-a01fc7fce92f" (reference "C4903") (unit 1))))
 )
 (wire (pts (xy 168.91 74.93) (xy 168.91 72.39)) (stroke (width 0) (type default)))
@@
 )
 (symbol (lib_id "Device:C") (at 181.61 78.74 0) (unit 1) (body_style 1) (exclude_from_sim no) (in_bom no) (on_board yes) (dnp yes)
-  (property "Reference" "C4804" (at 184.15 77.47 0) (effects (font (size 1.27 1.27)) (justify left)))
+  (property "Reference" "C4904" (at 184.15 77.47 0) (effects (font (size 1.27 1.27)) (justify left)))
   (property "Value" "DNP" (at 184.15 80.01 0) (effects (font (size 1.27 1.27)) (justify left)))
   (property "Footprint" "Capacitor_SMD:C_0201_0603Metric" (at 181.61 78.74 0) (effects (font (size 1.27 1.27))) (hide yes))
@@
   (pin "1")
   (pin "2")
-  (instances (project "t1-main-board" (path "/7746052e-d7f9-59ad-ba73-bd2b74439529/cd42149b-9c25-54cb-87d6-a01fc7fce92f" (reference "C4804") (unit 1))))
+  (instances (project "t1-main-board" (path "/7746052e-d7f9-59ad-ba73-bd2b74439529/cd42149b-9c25-54cb-87d6-a01fc7fce92f" (reference "C4904") (unit 1))))
 )
 (wire (pts (xy 181.61 74.93) (xy 181.61 72.39)) (stroke (width 0) (type default)))
@@
 )
 (symbol (lib_id "Hirose:U.FL-R-SMT-1") (at 214.63 53.34 0) (unit 1) (body_style 1) (exclude_from_sim no) (in_bom yes) (on_board yes) (dnp no)
-  (property "Reference" "J4802" (at 209.55 43.18 0) (effects (font (size 1.27 1.27)) (justify left)))
+  (property "Reference" "J4902" (at 209.55 43.18 0) (effects (font (size 1.27 1.27)) (justify left)))
   (property "Value" "U.FL-R-SMT-1" (at 209.55 40.64 0) (effects (font (size 1.27 1.27)) (justify left)))
   (property "Footprint" "Hirose:Hirose_U.FL-R-SMT-1_Vertical" (at 214.63 53.34 0) (effects (font (size 1.27 1.27))) (hide yes))
@@
   (pin "1")
   (pin "2")
-  (instances (project "t1-main-board" (path "/7746052e-d7f9-59ad-ba73-bd2b74439529/cd42149b-9c25-54cb-87d6-a01fc7fce92f" (reference "J4802") (unit 1))))
+  (instances (project "t1-main-board" (path "/7746052e-d7f9-59ad-ba73-bd2b74439529/cd42149b-9c25-54cb-87d6-a01fc7fce92f" (reference "J4902") (unit 1))))
 )
 (wire (pts (xy 207.01 50.8) (xy 204.47 50.8)) (stroke (width 0) (type default)))
@@
 (text "ANT1: dedicated configuration, not fitted (ADR 0018 item 4)" (exclude_from_sim no) (at 160.02 34.29 0) (effects (font (size 2.54 2.54)) (justify left bottom)))
 (symbol (lib_id "Device:C") (at 41.91 114.3 90) (unit 1) (body_style 1) (exclude_from_sim no) (in_bom yes) (on_board yes) (dnp no)
-  (property "Reference" "C4805" (at 41.91 110.49 90) (effects (font (size 1.27 1.27))))
+  (property "Reference" "C4905" (at 41.91 110.49 90) (effects (font (size 1.27 1.27))))
   (property "Value" "10 pF" (at 41.91 118.11 90) (effects (font (size 1.27 1.27))))
   (property "Spec" "50 V C0G" (at 41.91 120.65 90) (effects (font (size 1.27 1.27))))
@@
   (pin "1")
   (pin "2")
-  (instances (project "t1-main-board" (path "/7746052e-d7f9-59ad-ba73-bd2b74439529/cd42149b-9c25-54cb-87d6-a01fc7fce92f" (reference "C4805") (unit 1))))
+  (instances (project "t1-main-board" (path "/7746052e-d7f9-59ad-ba73-bd2b74439529/cd42149b-9c25-54cb-87d6-a01fc7fce92f" (reference "C4905") (unit 1))))
 )
 (wire (pts (xy 38.1 114.3) (xy 35.56 114.3)) (stroke (width 0) (type default)))

Commit message: Board: capture blk.debug
Debug UART2 (1.8 V) and I2S/DSD pads with ground pads, reset, PMIC and
power-key pads (PCB-T-09), a pad on every spare SoC GPIO whose pinout v1
row names one (the DEBUG bus, on the SoC's right edge), and a rail pad
for each power-tree rail no other sheet probes (PCB-T-02). Each DAC
sheet carries a pad on its MCLK. The spares pinout v1 leaves without a
pad now carry no-connect flags. On the root, facing sheet pins are
joined directly only where the route meets no other symbol.

Co-Authored-By: Claude Opus 5.5 <noreply@anthropic.com>
Claude-Session: https://claude.ai/code/session_01Ei262h3TpgY9vyfNLMi5Mn
Parts:
- removed C4901, C4902, C4903, C4904: DNP, Capacitor_SMD:C_0201_0603Metric, symbol Device:C
- removed C4905: 10 pF, Capacitor_SMD:C_0201_0603Metric, symbol Device:C
- removed J4901, J4902: U.FL-R-SMT-1, Hirose:Hirose_U.FL-R-SMT-1_Vertical, symbol Hirose:U.FL-R-SMT-1
- removed R4901, R4902: 0 Ω, Resistor_SMD:R_0201_0603Metric, symbol Device:R
- added C5001, C5002, C5003, C5004: DNP, Capacitor_SMD:C_0201_0603Metric, symbol Device:C
- added C5005: 10 pF, Capacitor_SMD:C_0201_0603Metric, symbol Device:C
- added J5001, J5002: U.FL-R-SMT-1, Hirose:Hirose_U.FL-R-SMT-1_Vertical, symbol Hirose:U.FL-R-SMT-1
- added R5001, R5002: 0 Ω, Resistor_SMD:R_0201_0603Metric, symbol Device:R
Connections:
- net GND: now also C5001.2, C5002.2, C5003.2, C5004.2, J5001.2 (GND), J5002.2 (GND)
- net WL_ANT0: now also C5001.1, R5001.1
- net WL_ANT0_J: now also C5002.1, J5001.1 (SIG), R5001.2
- net WL_ANT1: now also C5003.1, C5005.2, R5002.1
- net WL_ANT1_J: now also C5004.1, J5002.1 (SIG), R5002.2
- net WL_BT_IN: now also C5005.1
Changed lines of the file:
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@@
 (title_block (title "Antenna feeds") (date "2026-10-25") (rev "A") (company "The OpenDAP Project") (comment 1 "blk.antennas") (comment 2 "ANT0 and ANT1 paths as Murata's copy: matching positions, U.FL, the 10 pF shared link"))
 (symbol (lib_id "Device:R") (at 40.64 48.26 90) (unit 1) (body_style 1) (exclude_from_sim no) (in_bom yes) (on_board yes) (dnp no)
-  (property "Reference" "R4901" (at 40.64 45.72 90) (effects (font (size 1.27 1.27))))
+  (property "Reference" "R5001" (at 40.64 45.72 90) (effects (font (size 1.27 1.27))))
   (property "Value" "0 Ω" (at 40.64 50.8 90) (effects (font (size 1.27 1.27))))
   (property "Footprint" "Resistor_SMD:R_0201_0603Metric" (at 40.64 48.26 0) (effects (font (size 1.27 1.27))) (hide yes))
@@
   (pin "1")
   (pin "2")
-  (instances (project "t1-main-board" (path "/7746052e-d7f9-59ad-ba73-bd2b74439529/cd42149b-9c25-54cb-87d6-a01fc7fce92f" (reference "R4901") (unit 1))))
+  (instances (project "t1-main-board" (path "/7746052e-d7f9-59ad-ba73-bd2b74439529/cd42149b-9c25-54cb-87d6-a01fc7fce92f" (reference "R5001") (unit 1))))
 )
 (wire (pts (xy 36.83 48.26) (xy 34.29 48.26)) (stroke (width 0) (type default)))
 (wire (pts (xy 44.45 48.26) (xy 46.99 48.26)) (stroke (width 0) (type default)))
 (symbol (lib_id "Device:C") (at 33.02 78.74 0) (unit 1) (body_style 1) (exclude_from_sim no) (in_bom no) (on_board yes) (dnp yes)
-  (property "Reference" "C4901" (at 35.56 77.47 0) (effects (font (size 1.27 1.27)) (justify left)))
+  (property "Reference" "C5001" (at 35.56 77.47 0) (effects (font (size 1.27 1.27)) (justify left)))
   (property "Value" "DNP" (at 35.56 80.01 0) (effects (font (size 1.27 1.27)) (justify left)))
   (property "Footprint" "Capacitor_SMD:C_0201_0603Metric" (at 33.02 78.74 0) (effects (font (size 1.27 1.27))) (hide yes))
@@
   (pin "1")
   (pin "2")
-  (instances (project "t1-main-board" (path "/7746052e-d7f9-59ad-ba73-bd2b74439529/cd42149b-9c25-54cb-87d6-a01fc7fce92f" (reference "C4901") (unit 1))))
+  (instances (project "t1-main-board" (path "/7746052e-d7f9-59ad-ba73-bd2b74439529/cd42149b-9c25-54cb-87d6-a01fc7fce92f" (reference "C5001") (unit 1))))
 )
 (wire (pts (xy 33.02 74.93) (xy 33.02 72.39)) (stroke (width 0) (type default)))
@@
 )
 (symbol (lib_id "Device:C") (at 45.72 78.74 0) (unit 1) (body_style 1) (exclude_from_sim no) (in_bom no) (on_board yes) (dnp yes)
-  (property "Reference" "C4902" (at 48.26 77.47 0) (effects (font (size 1.27 1.27)) (justify left)))
+  (property "Reference" "C5002" (at 48.26 77.47 0) (effects (font (size 1.27 1.27)) (justify left)))
   (property "Value" "DNP" (at 48.26 80.01 0) (effects (font (size 1.27 1.27)) (justify left)))
   (property "Footprint" "Capacitor_SMD:C_0201_0603Metric" (at 45.72 78.74 0) (effects (font (size 1.27 1.27))) (hide yes))
@@
   (pin "1")
   (pin "2")
-  (instances (project "t1-main-board" (path "/7746052e-d7f9-59ad-ba73-bd2b74439529/cd42149b-9c25-54cb-87d6-a01fc7fce92f" (reference "C4902") (unit 1))))
+  (instances (project "t1-main-board" (path "/7746052e-d7f9-59ad-ba73-bd2b74439529/cd42149b-9c25-54cb-87d6-a01fc7fce92f" (reference "C5002") (unit 1))))
 )
 (wire (pts (xy 45.72 74.93) (xy 45.72 72.39)) (stroke (width 0) (type default)))
@@
 )
 (symbol (lib_id "Hirose:U.FL-R-SMT-1") (at 78.74 53.34 0) (unit 1) (body_style 1) (exclude_from_sim no) (in_bom yes) (on_board yes) (dnp no)
-  (property "Reference" "J4901" (at 73.66 43.18 0) (effects (font (size 1.27 1.27)) (justify left)))
+  (property "Reference" "J5001" (at 73.66 43.18 0) (effects (font (size 1.27 1.27)) (justify left)))
   (property "Value" "U.FL-R-SMT-1" (at 73.66 40.64 0) (effects (font (size 1.27 1.27)) (justify left)))
   (property "Footprint" "Hirose:Hirose_U.FL-R-SMT-1_Vertical" (at 78.74 53.34 0) (effects (font (size 1.27 1.27))) (hide yes))
@@
   (pin "1")
   (pin "2")
-  (instances (project "t1-main-board" (path "/7746052e-d7f9-59ad-ba73-bd2b74439529/cd42149b-9c25-54cb-87d6-a01fc7fce92f" (reference "J4901") (unit 1))))
+  (instances (project "t1-main-board" (path "/7746052e-d7f9-59ad-ba73-bd2b74439529/cd42149b-9c25-54cb-87d6-a01fc7fce92f" (reference "J5001") (unit 1))))
 )
 (wire (pts (xy 71.12 50.8) (xy 68.58 50.8)) (stroke (width 0) (type default)))
@@
 (text "ANT0: Wi-Fi 2.4 / 5 GHz and Bluetooth (shared, ADR 0018)" (exclude_from_sim no) (at 24.13 34.29 0) (effects (font (size 2.54 2.54)) (justify left bottom)))
 (symbol (lib_id "Device:R") (at 176.53 48.26 90) (unit 1) (body_style 1) (exclude_from_sim no) (in_bom yes) (on_board yes) (dnp yes)
-  (property "Reference" "R4902" (at 176.53 45.72 90) (effects (font (size 1.27 1.27))))
+  (property "Reference" "R5002" (at 176.53 45.72 90) (effects (font (size 1.27 1.27))))
   (property "Value" "0 Ω" (at 176.53 50.8 90) (effects (font (size 1.27 1.27))))
   (property "Footprint" "Resistor_SMD:R_0201_0603Metric" (at 176.53 48.26 0) (effects (font (size 1.27 1.27))) (hide yes))
@@
   (pin "1")
   (pin "2")
-  (instances (project "t1-main-board" (path "/7746052e-d7f9-59ad-ba73-bd2b74439529/cd42149b-9c25-54cb-87d6-a01fc7fce92f" (reference "R4902") (unit 1))))
+  (instances (project "t1-main-board" (path "/7746052e-d7f9-59ad-ba73-bd2b74439529/cd42149b-9c25-54cb-87d6-a01fc7fce92f" (reference "R5002") (unit 1))))
 )
 (wire (pts (xy 172.72 48.26) (xy 170.18 48.26)) (stroke (width 0) (type default)))
 (wire (pts (xy 180.34 48.26) (xy 182.88 48.26)) (stroke (width 0) (type default)))
 (symbol (lib_id "Device:C") (at 168.91 78.74 0) (unit 1) (body_style 1) (exclude_from_sim no) (in_bom no) (on_board yes) (dnp yes)
-  (property "Reference" "C4903" (at 171.45 77.47 0) (effects (font (size 1.27 1.27)) (justify left)))
+  (property "Reference" "C5003" (at 171.45 77.47 0) (effects (font (size 1.27 1.27)) (justify left)))
   (property "Value" "DNP" (at 171.45 80.01 0) (effects (font (size 1.27 1.27)) (justify left)))
   (property "Footprint" "Capacitor_SMD:C_0201_0603Metric" (at 168.91 78.74 0) (effects (font (size 1.27 1.27))) (hide yes))
@@
   (pin "1")
   (pin "2")
-  (instances (project "t1-main-board" (path "/7746052e-d7f9-59ad-ba73-bd2b74439529/cd42149b-9c25-54cb-87d6-a01fc7fce92f" (reference "C4903") (unit 1))))
+  (instances (project "t1-main-board" (path "/7746052e-d7f9-59ad-ba73-bd2b74439529/cd42149b-9c25-54cb-87d6-a01fc7fce92f" (reference "C5003") (unit 1))))
 )
 (wire (pts (xy 168.91 74.93) (xy 168.91 72.39)) (stroke (width 0) (type default)))
@@
 )
 (symbol (lib_id "Device:C") (at 181.61 78.74 0) (unit 1) (body_style 1) (exclude_from_sim no) (in_bom no) (on_board yes) (dnp yes)
-  (property "Reference" "C4904" (at 184.15 77.47 0) (effects (font (size 1.27 1.27)) (justify left)))
+  (property "Reference" "C5004" (at 184.15 77.47 0) (effects (font (size 1.27 1.27)) (justify left)))
   (property "Value" "DNP" (at 184.15 80.01 0) (effects (font (size 1.27 1.27)) (justify left)))
   (property "Footprint" "Capacitor_SMD:C_0201_0603Metric" (at 181.61 78.74 0) (effects (font (size 1.27 1.27))) (hide yes))
@@
   (pin "1")
   (pin "2")
-  (instances (project "t1-main-board" (path "/7746052e-d7f9-59ad-ba73-bd2b74439529/cd42149b-9c25-54cb-87d6-a01fc7fce92f" (reference "C4904") (unit 1))))
+  (instances (project "t1-main-board" (path "/7746052e-d7f9-59ad-ba73-bd2b74439529/cd42149b-9c25-54cb-87d6-a01fc7fce92f" (reference "C5004") (unit 1))))
 )
 (wire (pts (xy 181.61 74.93) (xy 181.61 72.39)) (stroke (width 0) (type default)))
@@
 )
 (symbol (lib_id "Hirose:U.FL-R-SMT-1") (at 214.63 53.34 0) (unit 1) (body_style 1) (exclude_from_sim no) (in_bom yes) (on_board yes) (dnp no)
-  (property "Reference" "J4902" (at 209.55 43.18 0) (effects (font (size 1.27 1.27)) (justify left)))
+  (property "Reference" "J5002" (at 209.55 43.18 0) (effects (font (size 1.27 1.27)) (justify left)))
   (property "Value" "U.FL-R-SMT-1" (at 209.55 40.64 0) (effects (font (size 1.27 1.27)) (justify left)))
   (property "Footprint" "Hirose:Hirose_U.FL-R-SMT-1_Vertical" (at 214.63 53.34 0) (effects (font (size 1.27 1.27))) (hide yes))
@@
   (pin "1")
   (pin "2")
-  (instances (project "t1-main-board" (path "/7746052e-d7f9-59ad-ba73-bd2b74439529/cd42149b-9c25-54cb-87d6-a01fc7fce92f" (reference "J4902") (unit 1))))
+  (instances (project "t1-main-board" (path "/7746052e-d7f9-59ad-ba73-bd2b74439529/cd42149b-9c25-54cb-87d6-a01fc7fce92f" (reference "J5002") (unit 1))))
 )
 (wire (pts (xy 207.01 50.8) (xy 204.47 50.8)) (stroke (width 0) (type default)))
@@
 (text "ANT1: dedicated configuration, not fitted (ADR 0018 item 4)" (exclude_from_sim no) (at 160.02 34.29 0) (effects (font (size 2.54 2.54)) (justify left bottom)))
 (symbol (lib_id "Device:C") (at 41.91 114.3 90) (unit 1) (body_style 1) (exclude_from_sim no) (in_bom yes) (on_board yes) (dnp no)
-  (property "Reference" "C4905" (at 41.91 110.49 90) (effects (font (size 1.27 1.27))))
+  (property "Reference" "C5005" (at 41.91 110.49 90) (effects (font (size 1.27 1.27))))
   (property "Value" "10 pF" (at 41.91 118.11 90) (effects (font (size 1.27 1.27))))
   (property "Spec" "50 V C0G" (at 41.91 120.65 90) (effects (font (size 1.27 1.27))))
@@
   (pin "1")
   (pin "2")
-  (instances (project "t1-main-board" (path "/7746052e-d7f9-59ad-ba73-bd2b74439529/cd42149b-9c25-54cb-87d6-a01fc7fce92f" (reference "C4905") (unit 1))))
+  (instances (project "t1-main-board" (path "/7746052e-d7f9-59ad-ba73-bd2b74439529/cd42149b-9c25-54cb-87d6-a01fc7fce92f" (reference "C5005") (unit 1))))
 )
 (wire (pts (xy 38.1 114.3) (xy 35.56 114.3)) (stroke (width 0) (type default)))
