File: board/hardware/t1-main-board/antennas.kicad_sch (KiCad schematic)
At the start: 9 parts, among them J5001 U.FL-R-SMT-1, J5002 U.FL-R-SMT-1

Commit message: Board: capture blk.mic-ambient and links #34, #35
IM73D122 on PDM CLK1 and SDI1 (BOM v1 line 34, pinout v1 AK2 and 1P2),
LR to ground, 22 Ω clock series, VDD from MIC_1V8 through link #35.
Link #34 on blk.mic-main makes the faceplate branch the rail MIC_1V8_FP
for contact 40 (power tree §4.12, G10). kicad-lib moves to e46bda4 for
the IM73D122, TPS3808G01, SN74LVC1G58 and BAT54 parts.

Co-Authored-By: Claude Opus 5.5 <noreply@anthropic.com>
Claude-Session: https://claude.ai/code/session_01Ei262h3TpgY9vyfNLMi5Mn
Parts:
- removed C5001, C5002, C5003, C5004: DNP, Capacitor_SMD:C_0201_0603Metric, symbol Device:C
- removed C5005: 10 pF, Capacitor_SMD:C_0201_0603Metric, symbol Device:C
- removed J5001, J5002: U.FL-R-SMT-1, Hirose:Hirose_U.FL-R-SMT-1_Vertical, symbol Hirose:U.FL-R-SMT-1
- removed R5001, R5002: 0 Ω, Resistor_SMD:R_0201_0603Metric, symbol Device:R
- added C5101, C5102, C5103, C5104: DNP, Capacitor_SMD:C_0201_0603Metric, symbol Device:C
- added C5105: 10 pF, Capacitor_SMD:C_0201_0603Metric, symbol Device:C
- added J5101, J5102: U.FL-R-SMT-1, Hirose:Hirose_U.FL-R-SMT-1_Vertical, symbol Hirose:U.FL-R-SMT-1
- added R5101, R5102: 0 Ω, Resistor_SMD:R_0201_0603Metric, symbol Device:R
Connections:
- net GND: now also C5101.2, C5102.2, C5103.2, C5104.2, J5101.2 (GND), J5102.2 (GND)
- net WL_ANT0: now also C5101.1, R5101.1
- net WL_ANT0_J: now also C5102.1, J5101.1 (SIG), R5101.2
- net WL_ANT1: now also C5103.1, C5105.2, R5102.1
- net WL_ANT1_J: now also C5104.1, J5102.1 (SIG), R5102.2
- net WL_BT_IN: now also C5105.1
Changed lines of the file:
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@@
 (title_block (title "Antenna feeds") (date "2026-10-25") (rev "A") (company "The OpenDAP Project") (comment 1 "blk.antennas") (comment 2 "ANT0 and ANT1 paths as Murata's copy: matching positions, U.FL, the 10 pF shared link"))
 (symbol (lib_id "Device:R") (at 40.64 48.26 90) (unit 1) (body_style 1) (exclude_from_sim no) (in_bom yes) (on_board yes) (dnp no)
-  (property "Reference" "R5001" (at 40.64 45.72 90) (effects (font (size 1.27 1.27))))
+  (property "Reference" "R5101" (at 40.64 45.72 90) (effects (font (size 1.27 1.27))))
   (property "Value" "0 Ω" (at 40.64 50.8 90) (effects (font (size 1.27 1.27))))
   (property "Footprint" "Resistor_SMD:R_0201_0603Metric" (at 40.64 48.26 0) (effects (font (size 1.27 1.27))) (hide yes))
@@
   (pin "1")
   (pin "2")
-  (instances (project "t1-main-board" (path "/7746052e-d7f9-59ad-ba73-bd2b74439529/cd42149b-9c25-54cb-87d6-a01fc7fce92f" (reference "R5001") (unit 1))))
+  (instances (project "t1-main-board" (path "/7746052e-d7f9-59ad-ba73-bd2b74439529/cd42149b-9c25-54cb-87d6-a01fc7fce92f" (reference "R5101") (unit 1))))
 )
 (wire (pts (xy 36.83 48.26) (xy 34.29 48.26)) (stroke (width 0) (type default)))
 (wire (pts (xy 44.45 48.26) (xy 46.99 48.26)) (stroke (width 0) (type default)))
 (symbol (lib_id "Device:C") (at 33.02 78.74 0) (unit 1) (body_style 1) (exclude_from_sim no) (in_bom no) (on_board yes) (dnp yes)
-  (property "Reference" "C5001" (at 35.56 77.47 0) (effects (font (size 1.27 1.27)) (justify left)))
+  (property "Reference" "C5101" (at 35.56 77.47 0) (effects (font (size 1.27 1.27)) (justify left)))
   (property "Value" "DNP" (at 35.56 80.01 0) (effects (font (size 1.27 1.27)) (justify left)))
   (property "Footprint" "Capacitor_SMD:C_0201_0603Metric" (at 33.02 78.74 0) (effects (font (size 1.27 1.27))) (hide yes))
@@
   (pin "1")
   (pin "2")
-  (instances (project "t1-main-board" (path "/7746052e-d7f9-59ad-ba73-bd2b74439529/cd42149b-9c25-54cb-87d6-a01fc7fce92f" (reference "C5001") (unit 1))))
+  (instances (project "t1-main-board" (path "/7746052e-d7f9-59ad-ba73-bd2b74439529/cd42149b-9c25-54cb-87d6-a01fc7fce92f" (reference "C5101") (unit 1))))
 )
 (wire (pts (xy 33.02 74.93) (xy 33.02 72.39)) (stroke (width 0) (type default)))
@@
 )
 (symbol (lib_id "Device:C") (at 45.72 78.74 0) (unit 1) (body_style 1) (exclude_from_sim no) (in_bom no) (on_board yes) (dnp yes)
-  (property "Reference" "C5002" (at 48.26 77.47 0) (effects (font (size 1.27 1.27)) (justify left)))
+  (property "Reference" "C5102" (at 48.26 77.47 0) (effects (font (size 1.27 1.27)) (justify left)))
   (property "Value" "DNP" (at 48.26 80.01 0) (effects (font (size 1.27 1.27)) (justify left)))
   (property "Footprint" "Capacitor_SMD:C_0201_0603Metric" (at 45.72 78.74 0) (effects (font (size 1.27 1.27))) (hide yes))
@@
   (pin "1")
   (pin "2")
-  (instances (project "t1-main-board" (path "/7746052e-d7f9-59ad-ba73-bd2b74439529/cd42149b-9c25-54cb-87d6-a01fc7fce92f" (reference "C5002") (unit 1))))
+  (instances (project "t1-main-board" (path "/7746052e-d7f9-59ad-ba73-bd2b74439529/cd42149b-9c25-54cb-87d6-a01fc7fce92f" (reference "C5102") (unit 1))))
 )
 (wire (pts (xy 45.72 74.93) (xy 45.72 72.39)) (stroke (width 0) (type default)))
@@
 )
 (symbol (lib_id "Hirose:U.FL-R-SMT-1") (at 78.74 53.34 0) (unit 1) (body_style 1) (exclude_from_sim no) (in_bom yes) (on_board yes) (dnp no)
-  (property "Reference" "J5001" (at 73.66 43.18 0) (effects (font (size 1.27 1.27)) (justify left)))
+  (property "Reference" "J5101" (at 73.66 43.18 0) (effects (font (size 1.27 1.27)) (justify left)))
   (property "Value" "U.FL-R-SMT-1" (at 73.66 40.64 0) (effects (font (size 1.27 1.27)) (justify left)))
   (property "Footprint" "Hirose:Hirose_U.FL-R-SMT-1_Vertical" (at 78.74 53.34 0) (effects (font (size 1.27 1.27))) (hide yes))
@@
   (pin "1")
   (pin "2")
-  (instances (project "t1-main-board" (path "/7746052e-d7f9-59ad-ba73-bd2b74439529/cd42149b-9c25-54cb-87d6-a01fc7fce92f" (reference "J5001") (unit 1))))
+  (instances (project "t1-main-board" (path "/7746052e-d7f9-59ad-ba73-bd2b74439529/cd42149b-9c25-54cb-87d6-a01fc7fce92f" (reference "J5101") (unit 1))))
 )
 (wire (pts (xy 71.12 50.8) (xy 68.58 50.8)) (stroke (width 0) (type default)))
@@
 (text "ANT0: Wi-Fi 2.4 / 5 GHz and Bluetooth (shared, ADR 0018)" (exclude_from_sim no) (at 24.13 34.29 0) (effects (font (size 2.54 2.54)) (justify left bottom)))
 (symbol (lib_id "Device:R") (at 176.53 48.26 90) (unit 1) (body_style 1) (exclude_from_sim no) (in_bom yes) (on_board yes) (dnp yes)
-  (property "Reference" "R5002" (at 176.53 45.72 90) (effects (font (size 1.27 1.27))))
+  (property "Reference" "R5102" (at 176.53 45.72 90) (effects (font (size 1.27 1.27))))
   (property "Value" "0 Ω" (at 176.53 50.8 90) (effects (font (size 1.27 1.27))))
   (property "Footprint" "Resistor_SMD:R_0201_0603Metric" (at 176.53 48.26 0) (effects (font (size 1.27 1.27))) (hide yes))
@@
   (pin "1")
   (pin "2")
-  (instances (project "t1-main-board" (path "/7746052e-d7f9-59ad-ba73-bd2b74439529/cd42149b-9c25-54cb-87d6-a01fc7fce92f" (reference "R5002") (unit 1))))
+  (instances (project "t1-main-board" (path "/7746052e-d7f9-59ad-ba73-bd2b74439529/cd42149b-9c25-54cb-87d6-a01fc7fce92f" (reference "R5102") (unit 1))))
 )
 (wire (pts (xy 172.72 48.26) (xy 170.18 48.26)) (stroke (width 0) (type default)))
 (wire (pts (xy 180.34 48.26) (xy 182.88 48.26)) (stroke (width 0) (type default)))
 (symbol (lib_id "Device:C") (at 168.91 78.74 0) (unit 1) (body_style 1) (exclude_from_sim no) (in_bom no) (on_board yes) (dnp yes)
-  (property "Reference" "C5003" (at 171.45 77.47 0) (effects (font (size 1.27 1.27)) (justify left)))
+  (property "Reference" "C5103" (at 171.45 77.47 0) (effects (font (size 1.27 1.27)) (justify left)))
   (property "Value" "DNP" (at 171.45 80.01 0) (effects (font (size 1.27 1.27)) (justify left)))
   (property "Footprint" "Capacitor_SMD:C_0201_0603Metric" (at 168.91 78.74 0) (effects (font (size 1.27 1.27))) (hide yes))
@@
   (pin "1")
   (pin "2")
-  (instances (project "t1-main-board" (path "/7746052e-d7f9-59ad-ba73-bd2b74439529/cd42149b-9c25-54cb-87d6-a01fc7fce92f" (reference "C5003") (unit 1))))
+  (instances (project "t1-main-board" (path "/7746052e-d7f9-59ad-ba73-bd2b74439529/cd42149b-9c25-54cb-87d6-a01fc7fce92f" (reference "C5103") (unit 1))))
 )
 (wire (pts (xy 168.91 74.93) (xy 168.91 72.39)) (stroke (width 0) (type default)))
@@
 )
 (symbol (lib_id "Device:C") (at 181.61 78.74 0) (unit 1) (body_style 1) (exclude_from_sim no) (in_bom no) (on_board yes) (dnp yes)
-  (property "Reference" "C5004" (at 184.15 77.47 0) (effects (font (size 1.27 1.27)) (justify left)))
+  (property "Reference" "C5104" (at 184.15 77.47 0) (effects (font (size 1.27 1.27)) (justify left)))
   (property "Value" "DNP" (at 184.15 80.01 0) (effects (font (size 1.27 1.27)) (justify left)))
   (property "Footprint" "Capacitor_SMD:C_0201_0603Metric" (at 181.61 78.74 0) (effects (font (size 1.27 1.27))) (hide yes))
@@
   (pin "1")
   (pin "2")
-  (instances (project "t1-main-board" (path "/7746052e-d7f9-59ad-ba73-bd2b74439529/cd42149b-9c25-54cb-87d6-a01fc7fce92f" (reference "C5004") (unit 1))))
+  (instances (project "t1-main-board" (path "/7746052e-d7f9-59ad-ba73-bd2b74439529/cd42149b-9c25-54cb-87d6-a01fc7fce92f" (reference "C5104") (unit 1))))
 )
 (wire (pts (xy 181.61 74.93) (xy 181.61 72.39)) (stroke (width 0) (type default)))
@@
 )
 (symbol (lib_id "Hirose:U.FL-R-SMT-1") (at 214.63 53.34 0) (unit 1) (body_style 1) (exclude_from_sim no) (in_bom yes) (on_board yes) (dnp no)
-  (property "Reference" "J5002" (at 209.55 43.18 0) (effects (font (size 1.27 1.27)) (justify left)))
+  (property "Reference" "J5102" (at 209.55 43.18 0) (effects (font (size 1.27 1.27)) (justify left)))
   (property "Value" "U.FL-R-SMT-1" (at 209.55 40.64 0) (effects (font (size 1.27 1.27)) (justify left)))
   (property "Footprint" "Hirose:Hirose_U.FL-R-SMT-1_Vertical" (at 214.63 53.34 0) (effects (font (size 1.27 1.27))) (hide yes))
@@
   (pin "1")
   (pin "2")
-  (instances (project "t1-main-board" (path "/7746052e-d7f9-59ad-ba73-bd2b74439529/cd42149b-9c25-54cb-87d6-a01fc7fce92f" (reference "J5002") (unit 1))))
+  (instances (project "t1-main-board" (path "/7746052e-d7f9-59ad-ba73-bd2b74439529/cd42149b-9c25-54cb-87d6-a01fc7fce92f" (reference "J5102") (unit 1))))
 )
 (wire (pts (xy 207.01 50.8) (xy 204.47 50.8)) (stroke (width 0) (type default)))
@@
 (text "ANT1: dedicated configuration, not fitted (ADR 0018 item 4)" (exclude_from_sim no) (at 160.02 34.29 0) (effects (font (size 2.54 2.54)) (justify left bottom)))
 (symbol (lib_id "Device:C") (at 41.91 114.3 90) (unit 1) (body_style 1) (exclude_from_sim no) (in_bom yes) (on_board yes) (dnp no)
-  (property "Reference" "C5005" (at 41.91 110.49 90) (effects (font (size 1.27 1.27))))
+  (property "Reference" "C5105" (at 41.91 110.49 90) (effects (font (size 1.27 1.27))))
   (property "Value" "10 pF" (at 41.91 118.11 90) (effects (font (size 1.27 1.27))))
   (property "Spec" "50 V C0G" (at 41.91 120.65 90) (effects (font (size 1.27 1.27))))
@@
   (pin "1")
   (pin "2")
-  (instances (project "t1-main-board" (path "/7746052e-d7f9-59ad-ba73-bd2b74439529/cd42149b-9c25-54cb-87d6-a01fc7fce92f" (reference "C5005") (unit 1))))
+  (instances (project "t1-main-board" (path "/7746052e-d7f9-59ad-ba73-bd2b74439529/cd42149b-9c25-54cb-87d6-a01fc7fce92f" (reference "C5105") (unit 1))))
 )
 (wire (pts (xy 38.1 114.3) (xy 35.56 114.3)) (stroke (width 0) (type default)))

Commit message: Board: capture blk.maskrom
Power + Vol- at a cold power-on pull eMMC D0 low inside the TPS3808G01
boot window (BOM v1 lines 35, 78, 97, 98; sim/maskrom): SENSE 280k/100k,
CT 390 nF, WINDOW_N with its pad, SN74LVC1G57 and SN74LVC1G58 on
vcca1v8_pmu, BAT54 from PWRON_N, DMG1012T through 1 kΩ to EMMC_D0.
Every block in use now has its sheet; the README states the remaining
single-pin nets.

Co-Authored-By: Claude Opus 5.5 <noreply@anthropic.com>
Claude-Session: https://claude.ai/code/session_01Ei262h3TpgY9vyfNLMi5Mn
Parts:
- removed C5101, C5102, C5103, C5104: DNP, Capacitor_SMD:C_0201_0603Metric, symbol Device:C
- removed C5105: 10 pF, Capacitor_SMD:C_0201_0603Metric, symbol Device:C
- removed J5101, J5102: U.FL-R-SMT-1, Hirose:Hirose_U.FL-R-SMT-1_Vertical, symbol Hirose:U.FL-R-SMT-1
- removed R5101, R5102: 0 Ω, Resistor_SMD:R_0201_0603Metric, symbol Device:R
- added C5201, C5202, C5203, C5204: DNP, Capacitor_SMD:C_0201_0603Metric, symbol Device:C
- added C5205: 10 pF, Capacitor_SMD:C_0201_0603Metric, symbol Device:C
- added J5201, J5202: U.FL-R-SMT-1, Hirose:Hirose_U.FL-R-SMT-1_Vertical, symbol Hirose:U.FL-R-SMT-1
- added R5201, R5202: 0 Ω, Resistor_SMD:R_0201_0603Metric, symbol Device:R
Connections:
- net GND: now also C5201.2, C5202.2, C5203.2, C5204.2, J5201.2 (GND), J5202.2 (GND)
- net WL_ANT0: now also C5201.1, R5201.1
- net WL_ANT0_J: now also C5202.1, J5201.1 (SIG), R5201.2
- net WL_ANT1: now also C5203.1, C5205.2, R5202.1
- net WL_ANT1_J: now also C5204.1, J5202.1 (SIG), R5202.2
- net WL_BT_IN: now also C5205.1
Changed lines of the file:
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@@
 (title_block (title "Antenna feeds") (date "2026-10-25") (rev "A") (company "The OpenDAP Project") (comment 1 "blk.antennas") (comment 2 "ANT0 and ANT1 paths as Murata's copy: matching positions, U.FL, the 10 pF shared link"))
 (symbol (lib_id "Device:R") (at 40.64 48.26 90) (unit 1) (body_style 1) (exclude_from_sim no) (in_bom yes) (on_board yes) (dnp no)
-  (property "Reference" "R5101" (at 40.64 45.72 90) (effects (font (size 1.27 1.27))))
+  (property "Reference" "R5201" (at 40.64 45.72 90) (effects (font (size 1.27 1.27))))
   (property "Value" "0 Ω" (at 40.64 50.8 90) (effects (font (size 1.27 1.27))))
   (property "Footprint" "Resistor_SMD:R_0201_0603Metric" (at 40.64 48.26 0) (effects (font (size 1.27 1.27))) (hide yes))
@@
   (pin "1")
   (pin "2")
-  (instances (project "t1-main-board" (path "/7746052e-d7f9-59ad-ba73-bd2b74439529/cd42149b-9c25-54cb-87d6-a01fc7fce92f" (reference "R5101") (unit 1))))
+  (instances (project "t1-main-board" (path "/7746052e-d7f9-59ad-ba73-bd2b74439529/cd42149b-9c25-54cb-87d6-a01fc7fce92f" (reference "R5201") (unit 1))))
 )
 (wire (pts (xy 36.83 48.26) (xy 34.29 48.26)) (stroke (width 0) (type default)))
 (wire (pts (xy 44.45 48.26) (xy 46.99 48.26)) (stroke (width 0) (type default)))
 (symbol (lib_id "Device:C") (at 33.02 78.74 0) (unit 1) (body_style 1) (exclude_from_sim no) (in_bom no) (on_board yes) (dnp yes)
-  (property "Reference" "C5101" (at 35.56 77.47 0) (effects (font (size 1.27 1.27)) (justify left)))
+  (property "Reference" "C5201" (at 35.56 77.47 0) (effects (font (size 1.27 1.27)) (justify left)))
   (property "Value" "DNP" (at 35.56 80.01 0) (effects (font (size 1.27 1.27)) (justify left)))
   (property "Footprint" "Capacitor_SMD:C_0201_0603Metric" (at 33.02 78.74 0) (effects (font (size 1.27 1.27))) (hide yes))
@@
   (pin "1")
   (pin "2")
-  (instances (project "t1-main-board" (path "/7746052e-d7f9-59ad-ba73-bd2b74439529/cd42149b-9c25-54cb-87d6-a01fc7fce92f" (reference "C5101") (unit 1))))
+  (instances (project "t1-main-board" (path "/7746052e-d7f9-59ad-ba73-bd2b74439529/cd42149b-9c25-54cb-87d6-a01fc7fce92f" (reference "C5201") (unit 1))))
 )
 (wire (pts (xy 33.02 74.93) (xy 33.02 72.39)) (stroke (width 0) (type default)))
@@
 )
 (symbol (lib_id "Device:C") (at 45.72 78.74 0) (unit 1) (body_style 1) (exclude_from_sim no) (in_bom no) (on_board yes) (dnp yes)
-  (property "Reference" "C5102" (at 48.26 77.47 0) (effects (font (size 1.27 1.27)) (justify left)))
+  (property "Reference" "C5202" (at 48.26 77.47 0) (effects (font (size 1.27 1.27)) (justify left)))
   (property "Value" "DNP" (at 48.26 80.01 0) (effects (font (size 1.27 1.27)) (justify left)))
   (property "Footprint" "Capacitor_SMD:C_0201_0603Metric" (at 45.72 78.74 0) (effects (font (size 1.27 1.27))) (hide yes))
@@
   (pin "1")
   (pin "2")
-  (instances (project "t1-main-board" (path "/7746052e-d7f9-59ad-ba73-bd2b74439529/cd42149b-9c25-54cb-87d6-a01fc7fce92f" (reference "C5102") (unit 1))))
+  (instances (project "t1-main-board" (path "/7746052e-d7f9-59ad-ba73-bd2b74439529/cd42149b-9c25-54cb-87d6-a01fc7fce92f" (reference "C5202") (unit 1))))
 )
 (wire (pts (xy 45.72 74.93) (xy 45.72 72.39)) (stroke (width 0) (type default)))
@@
 )
 (symbol (lib_id "Hirose:U.FL-R-SMT-1") (at 78.74 53.34 0) (unit 1) (body_style 1) (exclude_from_sim no) (in_bom yes) (on_board yes) (dnp no)
-  (property "Reference" "J5101" (at 73.66 43.18 0) (effects (font (size 1.27 1.27)) (justify left)))
+  (property "Reference" "J5201" (at 73.66 43.18 0) (effects (font (size 1.27 1.27)) (justify left)))
   (property "Value" "U.FL-R-SMT-1" (at 73.66 40.64 0) (effects (font (size 1.27 1.27)) (justify left)))
   (property "Footprint" "Hirose:Hirose_U.FL-R-SMT-1_Vertical" (at 78.74 53.34 0) (effects (font (size 1.27 1.27))) (hide yes))
@@
   (pin "1")
   (pin "2")
-  (instances (project "t1-main-board" (path "/7746052e-d7f9-59ad-ba73-bd2b74439529/cd42149b-9c25-54cb-87d6-a01fc7fce92f" (reference "J5101") (unit 1))))
+  (instances (project "t1-main-board" (path "/7746052e-d7f9-59ad-ba73-bd2b74439529/cd42149b-9c25-54cb-87d6-a01fc7fce92f" (reference "J5201") (unit 1))))
 )
 (wire (pts (xy 71.12 50.8) (xy 68.58 50.8)) (stroke (width 0) (type default)))
@@
 (text "ANT0: Wi-Fi 2.4 / 5 GHz and Bluetooth (shared, ADR 0018)" (exclude_from_sim no) (at 24.13 34.29 0) (effects (font (size 2.54 2.54)) (justify left bottom)))
 (symbol (lib_id "Device:R") (at 176.53 48.26 90) (unit 1) (body_style 1) (exclude_from_sim no) (in_bom yes) (on_board yes) (dnp yes)
-  (property "Reference" "R5102" (at 176.53 45.72 90) (effects (font (size 1.27 1.27))))
+  (property "Reference" "R5202" (at 176.53 45.72 90) (effects (font (size 1.27 1.27))))
   (property "Value" "0 Ω" (at 176.53 50.8 90) (effects (font (size 1.27 1.27))))
   (property "Footprint" "Resistor_SMD:R_0201_0603Metric" (at 176.53 48.26 0) (effects (font (size 1.27 1.27))) (hide yes))
@@
   (pin "1")
   (pin "2")
-  (instances (project "t1-main-board" (path "/7746052e-d7f9-59ad-ba73-bd2b74439529/cd42149b-9c25-54cb-87d6-a01fc7fce92f" (reference "R5102") (unit 1))))
+  (instances (project "t1-main-board" (path "/7746052e-d7f9-59ad-ba73-bd2b74439529/cd42149b-9c25-54cb-87d6-a01fc7fce92f" (reference "R5202") (unit 1))))
 )
 (wire (pts (xy 172.72 48.26) (xy 170.18 48.26)) (stroke (width 0) (type default)))
 (wire (pts (xy 180.34 48.26) (xy 182.88 48.26)) (stroke (width 0) (type default)))
 (symbol (lib_id "Device:C") (at 168.91 78.74 0) (unit 1) (body_style 1) (exclude_from_sim no) (in_bom no) (on_board yes) (dnp yes)
-  (property "Reference" "C5103" (at 171.45 77.47 0) (effects (font (size 1.27 1.27)) (justify left)))
+  (property "Reference" "C5203" (at 171.45 77.47 0) (effects (font (size 1.27 1.27)) (justify left)))
   (property "Value" "DNP" (at 171.45 80.01 0) (effects (font (size 1.27 1.27)) (justify left)))
   (property "Footprint" "Capacitor_SMD:C_0201_0603Metric" (at 168.91 78.74 0) (effects (font (size 1.27 1.27))) (hide yes))
@@
   (pin "1")
   (pin "2")
-  (instances (project "t1-main-board" (path "/7746052e-d7f9-59ad-ba73-bd2b74439529/cd42149b-9c25-54cb-87d6-a01fc7fce92f" (reference "C5103") (unit 1))))
+  (instances (project "t1-main-board" (path "/7746052e-d7f9-59ad-ba73-bd2b74439529/cd42149b-9c25-54cb-87d6-a01fc7fce92f" (reference "C5203") (unit 1))))
 )
 (wire (pts (xy 168.91 74.93) (xy 168.91 72.39)) (stroke (width 0) (type default)))
@@
 )
 (symbol (lib_id "Device:C") (at 181.61 78.74 0) (unit 1) (body_style 1) (exclude_from_sim no) (in_bom no) (on_board yes) (dnp yes)
-  (property "Reference" "C5104" (at 184.15 77.47 0) (effects (font (size 1.27 1.27)) (justify left)))
+  (property "Reference" "C5204" (at 184.15 77.47 0) (effects (font (size 1.27 1.27)) (justify left)))
   (property "Value" "DNP" (at 184.15 80.01 0) (effects (font (size 1.27 1.27)) (justify left)))
   (property "Footprint" "Capacitor_SMD:C_0201_0603Metric" (at 181.61 78.74 0) (effects (font (size 1.27 1.27))) (hide yes))
@@
   (pin "1")
   (pin "2")
-  (instances (project "t1-main-board" (path "/7746052e-d7f9-59ad-ba73-bd2b74439529/cd42149b-9c25-54cb-87d6-a01fc7fce92f" (reference "C5104") (unit 1))))
+  (instances (project "t1-main-board" (path "/7746052e-d7f9-59ad-ba73-bd2b74439529/cd42149b-9c25-54cb-87d6-a01fc7fce92f" (reference "C5204") (unit 1))))
 )
 (wire (pts (xy 181.61 74.93) (xy 181.61 72.39)) (stroke (width 0) (type default)))
@@
 )
 (symbol (lib_id "Hirose:U.FL-R-SMT-1") (at 214.63 53.34 0) (unit 1) (body_style 1) (exclude_from_sim no) (in_bom yes) (on_board yes) (dnp no)
-  (property "Reference" "J5102" (at 209.55 43.18 0) (effects (font (size 1.27 1.27)) (justify left)))
+  (property "Reference" "J5202" (at 209.55 43.18 0) (effects (font (size 1.27 1.27)) (justify left)))
   (property "Value" "U.FL-R-SMT-1" (at 209.55 40.64 0) (effects (font (size 1.27 1.27)) (justify left)))
   (property "Footprint" "Hirose:Hirose_U.FL-R-SMT-1_Vertical" (at 214.63 53.34 0) (effects (font (size 1.27 1.27))) (hide yes))
@@
   (pin "1")
   (pin "2")
-  (instances (project "t1-main-board" (path "/7746052e-d7f9-59ad-ba73-bd2b74439529/cd42149b-9c25-54cb-87d6-a01fc7fce92f" (reference "J5102") (unit 1))))
+  (instances (project "t1-main-board" (path "/7746052e-d7f9-59ad-ba73-bd2b74439529/cd42149b-9c25-54cb-87d6-a01fc7fce92f" (reference "J5202") (unit 1))))
 )
 (wire (pts (xy 207.01 50.8) (xy 204.47 50.8)) (stroke (width 0) (type default)))
@@
 (text "ANT1: dedicated configuration, not fitted (ADR 0018 item 4)" (exclude_from_sim no) (at 160.02 34.29 0) (effects (font (size 2.54 2.54)) (justify left bottom)))
 (symbol (lib_id "Device:C") (at 41.91 114.3 90) (unit 1) (body_style 1) (exclude_from_sim no) (in_bom yes) (on_board yes) (dnp no)
-  (property "Reference" "C5105" (at 41.91 110.49 90) (effects (font (size 1.27 1.27))))
+  (property "Reference" "C5205" (at 41.91 110.49 90) (effects (font (size 1.27 1.27))))
   (property "Value" "10 pF" (at 41.91 118.11 90) (effects (font (size 1.27 1.27))))
   (property "Spec" "50 V C0G" (at 41.91 120.65 90) (effects (font (size 1.27 1.27))))
@@
   (pin "1")
   (pin "2")
-  (instances (project "t1-main-board" (path "/7746052e-d7f9-59ad-ba73-bd2b74439529/cd42149b-9c25-54cb-87d6-a01fc7fce92f" (reference "C5105") (unit 1))))
+  (instances (project "t1-main-board" (path "/7746052e-d7f9-59ad-ba73-bd2b74439529/cd42149b-9c25-54cb-87d6-a01fc7fce92f" (reference "C5205") (unit 1))))
 )
 (wire (pts (xy 38.1 114.3) (xy 35.56 114.3)) (stroke (width 0) (type default)))
