File: board/hardware/t1-main-board/antennas.kicad_sch (KiCad schematic)
At the start: 9 parts, among them J5201 U.FL-R-SMT-1, J5202 U.FL-R-SMT-1

Commit message: Board on libs v0.2.0: lower-case kebab vendor keys (HL-13)
The libs submodule moves to v0.2.0 (5f24483). Every library nickname in
the generator, the placement tool and the floorplan study follows the
key table (Texas_Instruments -> texas-instruments, OpenDAP_Device ->
opendap-generic, Rockchip and Rockchip_PMIC -> rockchip, ...); the
library tables are written from the files. Schematic and board
regenerated.

Checks: ERC 0 errors (warnings unchanged); DRC 0 errors, 605 warnings,
the same counts by type, schematic parity 0; every placement identical;
craft Q1 met; pcb tests pass; STEP export resolves every libs 3D model
(the 27 parts without a model are KiCad stock lands that have none).

Co-Authored-By: Claude Opus 5.5 <noreply@anthropic.com>
Claude-Session: https://claude.ai/code/session_01Ei262h3TpgY9vyfNLMi5Mn
Parts:
- J5201, J5202: footprint Hirose:Hirose_U.FL-R-SMT-1_Vertical -> hirose:Hirose_U.FL-R-SMT-1_Vertical; symbol Hirose:U.FL-R-SMT-1 -> hirose:U.FL-R-SMT-1
Changed lines of the file:
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@@
   (instances (project "t1-main-board" (path "/7746052e-d7f9-59ad-ba73-bd2b74439529/cd42149b-9c25-54cb-87d6-a01fc7fce92f" (reference "#PWR0693") (unit 1))))
 )
-(symbol (lib_id "Hirose:U.FL-R-SMT-1") (at 78.74 53.34 0) (unit 1) (body_style 1) (exclude_from_sim no) (in_bom yes) (on_board yes) (dnp no)
+(symbol (lib_id "hirose:U.FL-R-SMT-1") (at 78.74 53.34 0) (unit 1) (body_style 1) (exclude_from_sim no) (in_bom yes) (on_board yes) (dnp no)
   (property "Reference" "J5201" (at 73.66 43.18 0) (effects (font (size 1.27 1.27)) (justify left)))
   (property "Value" "U.FL-R-SMT-1" (at 73.66 40.64 0) (effects (font (size 1.27 1.27)) (justify left)))
-  (property "Footprint" "Hirose:Hirose_U.FL-R-SMT-1_Vertical" (at 78.74 53.34 0) (effects (font (size 1.27 1.27))) (hide yes))
+  (property "Footprint" "hirose:Hirose_U.FL-R-SMT-1_Vertical" (at 78.74 53.34 0) (effects (font (size 1.27 1.27))) (hide yes))
   (property "Datasheet" "https://www.hirose.com/en/product/series/U.FL" (at 78.74 53.34 0) (effects (font (size 1.27 1.27))) (hide yes))
   (property "Description" "U.FL ultra-small SMT coaxial receptacle, 50 ohm, DC to 6 GHz, 2.6 x 2.6 mm, 1.25 mm high" (at 78.74 53.34 0) (effects (font (size 1.27 1.27))) (hide yes))
@@
   (instances (project "t1-main-board" (path "/7746052e-d7f9-59ad-ba73-bd2b74439529/cd42149b-9c25-54cb-87d6-a01fc7fce92f" (reference "#PWR0696") (unit 1))))
 )
-(symbol (lib_id "Hirose:U.FL-R-SMT-1") (at 214.63 53.34 0) (unit 1) (body_style 1) (exclude_from_sim no) (in_bom yes) (on_board yes) (dnp no)
+(symbol (lib_id "hirose:U.FL-R-SMT-1") (at 214.63 53.34 0) (unit 1) (body_style 1) (exclude_from_sim no) (in_bom yes) (on_board yes) (dnp no)
   (property "Reference" "J5202" (at 209.55 43.18 0) (effects (font (size 1.27 1.27)) (justify left)))
   (property "Value" "U.FL-R-SMT-1" (at 209.55 40.64 0) (effects (font (size 1.27 1.27)) (justify left)))
-  (property "Footprint" "Hirose:Hirose_U.FL-R-SMT-1_Vertical" (at 214.63 53.34 0) (effects (font (size 1.27 1.27))) (hide yes))
+  (property "Footprint" "hirose:Hirose_U.FL-R-SMT-1_Vertical" (at 214.63 53.34 0) (effects (font (size 1.27 1.27))) (hide yes))
   (property "Datasheet" "https://www.hirose.com/en/product/series/U.FL" (at 214.63 53.34 0) (effects (font (size 1.27 1.27))) (hide yes))
   (property "Description" "U.FL ultra-small SMT coaxial receptacle, 50 ohm, DC to 6 GHz, 2.6 x 2.6 mm, 1.25 mm high" (at 214.63 53.34 0) (effects (font (size 1.27 1.27))) (hide yes))
