File: board/hardware/t1-main-board/debug.kicad_sch (KiCad schematic)
At the start: 57 parts

Commit message: Board: capture blk.cover-detect
COVER_DET_N on GPIO0_A6 (AJ38, PMUIO1, wake-capable), recorded in
pinout v1 (closes feature blocks G22): board-edge input and ground pads
for the case's actuator, 100 kΩ to vcc3v3_pmu, TPD1E10B06 at the pad
(BOM v1 line 143, PCB-L-10). The line rides the KEYS bus with the
buttons.

Co-Authored-By: Claude Opus 5.5 <noreply@anthropic.com>
Claude-Session: https://claude.ai/code/session_01Ei262h3TpgY9vyfNLMi5Mn
Parts:
- removed TP4157: VSYS_P5V1, TestPoint:TestPoint_Pad_D1.0mm, symbol Connector:TestPoint
- TP4114: value SPARE_0A6 -> SPARE_1A0
- TP4115: value SPARE_1A0 -> SPARE_1A1
- TP4116: value SPARE_1A1 -> SPARE_1A3
- TP4117: value SPARE_1A3 -> SPARE_1A4
- TP4118: value SPARE_1A4 -> SPARE_1A5
- TP4119: value SPARE_1A5 -> SPARE_1A6
- TP4120: value SPARE_1A6 -> SPARE_1A7
- TP4121: value SPARE_1A7 -> SPARE_1B3
- TP4122: value SPARE_1B3 -> SPARE_1D0
- TP4123: value SPARE_1D0 -> SPARE_1D1
- TP4124: value SPARE_1D1 -> SPARE_1D3
- TP4125: value SPARE_1D3 -> SPARE_2B1
- TP4126: value SPARE_2B1 -> SPARE_2B2
- TP4127: value SPARE_2B2 -> SPARE_3B7
- TP4128: value SPARE_3B7 -> SPARE_3C0
- TP4129: value SPARE_3C0 -> SPARE_3C4
- TP4130: value SPARE_3C4 -> SPARE_3C5
- TP4131: value SPARE_3C5 -> SPARE_4C7
- TP4132: value SPARE_4C7 -> SPARE_4D0
- TP4133: value SPARE_4D0 -> SPARE_4D1
- TP4134: value SPARE_4D1 -> vdd_gpu
- TP4135: value vdd_gpu -> vdd_npu
- TP4136: value vdd_npu -> vccio6_1v8
- TP4137: value vccio6_1v8 -> vdda0v9_image
- TP4138: value vdda0v9_image -> vdda_0v9
- TP4139: value vdda_0v9 -> vdda0v9_pmu
- TP4140: value vdda0v9_pmu -> vccio_sd
- TP4141: value vccio_sd -> vcc3v3_pmu
- TP4142: value vcc3v3_pmu -> vcca_1v8
- TP4143: value vcca_1v8 -> vcca1v8_image
- TP4144: value vcca1v8_image -> DAC_VP
- TP4145: value DAC_VP -> DAC1_VA
- TP4146: value DAC1_VA -> DAC2_VA
- TP4147: value DAC2_VA -> MCLK_3V1
- TP4148: value MCLK_3V1 -> MCLK_1V8
- TP4149: value MCLK_1V8 -> AUDIO_P7V0
- TP4150: value AUDIO_P7V0 -> AUDIO_N7V0
- TP4151: value AUDIO_N7V0 -> BAT_N
- TP4152: value BAT_N -> FP_VCI_SRC
- TP4153: value FP_VCI_SRC -> VSYS_SRC
- TP4154: value VSYS_SRC -> VSYS_AUDIO
- TP4155: value VSYS_AUDIO -> VSYS_LV_BL
- TP4156: value VSYS_LV_BL -> VSYS_P5V1
Connections:
- net SPARE_0A6 is gone; now on net SPARE_1A0: TP4114.1
- net AUDIO_N7V0: now also TP4150.1; no longer TP4151.1
- net AUDIO_P7V0: now also TP4149.1; no longer TP4150.1
- net BAT_N: now also TP4151.1; no longer TP4152.1
- net DAC1_VA: now also TP4145.1; no longer TP4146.1
- net DAC2_VA: now also TP4146.1; no longer TP4147.1
- net DAC_VP: now also TP4144.1; no longer TP4145.1
- net FP_VCI_SRC: now also TP4152.1; no longer TP4153.1
- net MCLK_1V8: now also TP4148.1; no longer TP4149.1
- net MCLK_3V1: now also TP4147.1; no longer TP4148.1
- net SPARE_1A0: no longer TP4115.1
- net SPARE_1A1: now also TP4115.1; no longer TP4116.1
- net SPARE_1A3: now also TP4116.1; no longer TP4117.1
- net SPARE_1A4: now also TP4117.1; no longer TP4118.1
- net SPARE_1A5: now also TP4118.1; no longer TP4119.1
- net SPARE_1A6: now also TP4119.1; no longer TP4120.1
- net SPARE_1A7: now also TP4120.1; no longer TP4121.1
- net SPARE_1B3: now also TP4121.1; no longer TP4122.1
- net SPARE_1D0: now also TP4122.1; no longer TP4123.1
- net SPARE_1D1: now also TP4123.1; no longer TP4124.1
- net SPARE_1D3: now also TP4124.1; no longer TP4125.1
- net SPARE_2B1: now also TP4125.1; no longer TP4126.1
- net SPARE_2B2: now also TP4126.1; no longer TP4127.1
- net SPARE_3B7: now also TP4127.1; no longer TP4128.1
- net SPARE_3C0: now also TP4128.1; no longer TP4129.1
- net SPARE_3C4: now also TP4129.1; no longer TP4130.1
- net SPARE_3C5: now also TP4130.1; no longer TP4131.1
- net SPARE_4C7: now also TP4131.1; no longer TP4132.1
- net SPARE_4D0: now also TP4132.1; no longer TP4133.1
- net SPARE_4D1: now also TP4133.1; no longer TP4134.1
- net VSYS_AUDIO: now also TP4154.1; no longer TP4155.1
- net VSYS_LV_BL: now also TP4155.1; no longer TP4156.1
- net VSYS_P5V1: now also TP4156.1
- net VSYS_SRC: now also TP4153.1; no longer TP4154.1
- net vcc3v3_pmu: now also TP4141.1; no longer TP4142.1
- net vcca1v8_image: now also TP4143.1; no longer TP4144.1
- net vcca_1v8: now also TP4142.1; no longer TP4143.1
- net vccio6_1v8: now also TP4136.1; no longer TP4137.1
- net vccio_sd: now also TP4140.1; no longer TP4141.1
- net vdd_gpu: now also TP4134.1; no longer TP4135.1
- net vdd_npu: now also TP4135.1; no longer TP4136.1
- net vdda0v9_image: now also TP4137.1; no longer TP4138.1
- net vdda0v9_pmu: now also TP4139.1; no longer TP4140.1
- net vdda_0v9: now also TP4138.1; no longer TP4139.1
Other:
- moved on the sheet: TP4124, TP4125, TP4126, TP4127, TP4128, TP4129, TP4130, TP4131, TP4132, TP4133, TP4134, TP4135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

Commit message: Board: capture blk.mic-ambient and links #34, #35
IM73D122 on PDM CLK1 and SDI1 (BOM v1 line 34, pinout v1 AK2 and 1P2),
LR to ground, 22 Ω clock series, VDD from MIC_1V8 through link #35.
Link #34 on blk.mic-main makes the faceplate branch the rail MIC_1V8_FP
for contact 40 (power tree §4.12, G10). kicad-lib moves to e46bda4 for
the IM73D122, TPS3808G01, SN74LVC1G58 and BAT54 parts.

Co-Authored-By: Claude Opus 5.5 <noreply@anthropic.com>
Claude-Session: https://claude.ai/code/session_01Ei262h3TpgY9vyfNLMi5Mn
Parts:
- removed TP4101: DBG_UART_TX, TestPoint:TestPoint_Pad_D1.0mm, symbol Connector:TestPoint
- removed TP4102: DBG_UART_RX, TestPoint:TestPoint_Pad_D1.0mm, symbol Connector:TestPoint
- removed TP4103, TP4109: GND, TestPoint:TestPoint_Pad_D1.0mm, symbol Connector:TestPoint
- removed TP4104: I2S_BCLK, TestPoint:TestPoint_Pad_D1.0mm, symbol Connector:TestPoint
- removed TP4105: I2S_LRCK, TestPoint:TestPoint_Pad_D1.0mm, symbol Connector:TestPoint
- removed TP4106: I2S_SDO0, TestPoint:TestPoint_Pad_D1.0mm, symbol Connector:TestPoint
- removed TP4107: DSD_L, TestPoint:TestPoint_Pad_D1.0mm, symbol Connector:TestPoint
- removed TP4108: DSD_R, TestPoint:TestPoint_Pad_D1.0mm, symbol Connector:TestPoint
- removed TP4110: SOC_RESET_N, TestPoint:TestPoint_Pad_D1.0mm, symbol Connector:TestPoint
- removed TP4111: PMIC_INT_N, TestPoint:TestPoint_Pad_D1.0mm, symbol Connector:TestPoint
- removed TP4112: PMIC_SLEEP, TestPoint:TestPoint_Pad_D1.0mm, symbol Connector:TestPoint
- removed TP4113: PWRON_N, TestPoint:TestPoint_Pad_D1.0mm, symbol Connector:TestPoint
- removed TP4114: SPARE_1A0, TestPoint:TestPoint_Pad_D1.0mm, symbol Connector:TestPoint
- removed TP4115: SPARE_1A1, TestPoint:TestPoint_Pad_D1.0mm, symbol Connector:TestPoint
- removed TP4116: SPARE_1A3, TestPoint:TestPoint_Pad_D1.0mm, symbol Connector:TestPoint
- removed TP4117: SPARE_1A4, TestPoint:TestPoint_Pad_D1.0mm, symbol Connector:TestPoint
- removed TP4118: SPARE_1A5, TestPoint:TestPoint_Pad_D1.0mm, symbol Connector:TestPoint
- removed TP4119: SPARE_1A6, TestPoint:TestPoint_Pad_D1.0mm, symbol Connector:TestPoint
- removed TP4120: SPARE_1A7, TestPoint:TestPoint_Pad_D1.0mm, symbol Connector:TestPoint
- removed TP4121: SPARE_1B3, TestPoint:TestPoint_Pad_D1.0mm, symbol Connector:TestPoint
- removed TP4122: SPARE_1D0, TestPoint:TestPoint_Pad_D1.0mm, symbol Connector:TestPoint
- removed TP4123: SPARE_1D1, TestPoint:TestPoint_Pad_D1.0mm, symbol Connector:TestPoint
- removed TP4124: SPARE_1D3, TestPoint:TestPoint_Pad_D1.0mm, symbol Connector:TestPoint
- removed TP4125: SPARE_2B1, TestPoint:TestPoint_Pad_D1.0mm, symbol Connector:TestPoint
- removed TP4126: SPARE_2B2, TestPoint:TestPoint_Pad_D1.0mm, symbol Connector:TestPoint
- removed TP4127: SPARE_3B7, TestPoint:TestPoint_Pad_D1.0mm, symbol Connector:TestPoint
- removed TP4128: SPARE_3C0, TestPoint:TestPoint_Pad_D1.0mm, symbol Connector:TestPoint
- removed TP4129: SPARE_3C4, TestPoint:TestPoint_Pad_D1.0mm, symbol Connector:TestPoint
- removed TP4130: SPARE_3C5, TestPoint:TestPoint_Pad_D1.0mm, symbol Connector:TestPoint
- removed TP4131: SPARE_4C7, TestPoint:TestPoint_Pad_D1.0mm, symbol Connector:TestPoint
- removed TP4132: SPARE_4D0, TestPoint:TestPoint_Pad_D1.0mm, symbol Connector:TestPoint
- removed TP4133: SPARE_4D1, TestPoint:TestPoint_Pad_D1.0mm, symbol Connector:TestPoint
- removed TP4134: vdd_gpu, TestPoint:TestPoint_Pad_D1.0mm, symbol Connector:TestPoint
- removed TP4135: vdd_npu, TestPoint:TestPoint_Pad_D1.0mm, symbol Connector:TestPoint
- removed TP4136: vccio6_1v8, TestPoint:TestPoint_Pad_D1.0mm, symbol Connector:TestPoint
- removed TP4137: vdda0v9_image, TestPoint:TestPoint_Pad_D1.0mm, symbol Connector:TestPoint
- removed TP4138: vdda_0v9, TestPoint:TestPoint_Pad_D1.0mm, symbol Connector:TestPoint
- removed TP4139: vdda0v9_pmu, TestPoint:TestPoint_Pad_D1.0mm, symbol Connector:TestPoint
- removed TP4140: vccio_sd, TestPoint:TestPoint_Pad_D1.0mm, symbol Connector:TestPoint
- removed TP4141: vcc3v3_pmu, TestPoint:TestPoint_Pad_D1.0mm, symbol Connector:TestPoint
- removed TP4142: vcca_1v8, TestPoint:TestPoint_Pad_D1.0mm, symbol Connector:TestPoint
- removed TP4143: vcca1v8_image, TestPoint:TestPoint_Pad_D1.0mm, symbol Connector:TestPoint
- removed TP4144: DAC_VP, TestPoint:TestPoint_Pad_D1.0mm, symbol Connector:TestPoint
- removed TP4145: DAC1_VA, TestPoint:TestPoint_Pad_D1.0mm, symbol Connector:TestPoint
- removed TP4146: DAC2_VA, TestPoint:TestPoint_Pad_D1.0mm, symbol Connector:TestPoint
- removed TP4147: MCLK_3V1, TestPoint:TestPoint_Pad_D1.0mm, symbol Connector:TestPoint
- removed TP4148: MCLK_1V8, TestPoint:TestPoint_Pad_D1.0mm, symbol Connector:TestPoint
- removed TP4149: AUDIO_P7V0, TestPoint:TestPoint_Pad_D1.0mm, symbol Connector:TestPoint
- removed TP4150: AUDIO_N7V0, TestPoint:TestPoint_Pad_D1.0mm, symbol Connector:TestPoint
- removed TP4151: BAT_N, TestPoint:TestPoint_Pad_D1.0mm, symbol Connector:TestPoint
- removed TP4152: FP_VCI_SRC, TestPoint:TestPoint_Pad_D1.0mm, symbol Connector:TestPoint
- removed TP4153: VSYS_SRC, TestPoint:TestPoint_Pad_D1.0mm, symbol Connector:TestPoint
- removed TP4154: VSYS_AUDIO, TestPoint:TestPoint_Pad_D1.0mm, symbol Connector:TestPoint
- removed TP4155: VSYS_LV_BL, TestPoint:TestPoint_Pad_D1.0mm, symbol Connector:TestPoint
- removed TP4156: VSYS_P5V1, TestPoint:TestPoint_Pad_D1.0mm, symbol Connector:TestPoint
- added TP4201: DBG_UART_TX, TestPoint:TestPoint_Pad_D1.0mm, symbol Connector:TestPoint
- added TP4202: DBG_UART_RX, TestPoint:TestPoint_Pad_D1.0mm, symbol Connector:TestPoint
- added TP4203, TP4209: GND, TestPoint:TestPoint_Pad_D1.0mm, symbol Connector:TestPoint
- added TP4204: I2S_BCLK, TestPoint:TestPoint_Pad_D1.0mm, symbol Connector:TestPoint
- added TP4205: I2S_LRCK, TestPoint:TestPoint_Pad_D1.0mm, symbol Connector:TestPoint
- added TP4206: I2S_SDO0, TestPoint:TestPoint_Pad_D1.0mm, symbol Connector:TestPoint
- added TP4207: DSD_L, TestPoint:TestPoint_Pad_D1.0mm, symbol Connector:TestPoint
- added TP4208: DSD_R, TestPoint:TestPoint_Pad_D1.0mm, symbol Connector:TestPoint
- added TP4210: SOC_RESET_N, TestPoint:TestPoint_Pad_D1.0mm, symbol Connector:TestPoint
- added TP4211: PMIC_INT_N, TestPoint:TestPoint_Pad_D1.0mm, symbol Connector:TestPoint
- added TP4212: PMIC_SLEEP, TestPoint:TestPoint_Pad_D1.0mm, symbol Connector:TestPoint
- added TP4213: PWRON_N, TestPoint:TestPoint_Pad_D1.0mm, symbol Connector:TestPoint
- added TP4214: SPARE_1A0, TestPoint:TestPoint_Pad_D1.0mm, symbol Connector:TestPoint
- added TP4215: SPARE_1A1, TestPoint:TestPoint_Pad_D1.0mm, symbol Connector:TestPoint
- added TP4216: SPARE_1A3, TestPoint:TestPoint_Pad_D1.0mm, symbol Connector:TestPoint
- added TP4217: SPARE_1A4, TestPoint:TestPoint_Pad_D1.0mm, symbol Connector:TestPoint
- added TP4218: SPARE_1A5, TestPoint:TestPoint_Pad_D1.0mm, symbol Connector:TestPoint
- added TP4219: SPARE_1A6, TestPoint:TestPoint_Pad_D1.0mm, symbol Connector:TestPoint
- added TP4220: SPARE_1A7, TestPoint:TestPoint_Pad_D1.0mm, symbol Connector:TestPoint
- added TP4221: SPARE_1B3, TestPoint:TestPoint_Pad_D1.0mm, symbol Connector:TestPoint
- added TP4222: SPARE_1D0, TestPoint:TestPoint_Pad_D1.0mm, symbol Connector:TestPoint
- added TP4223: SPARE_1D1, TestPoint:TestPoint_Pad_D1.0mm, symbol Connector:TestPoint
- added TP4224: SPARE_1D3, TestPoint:TestPoint_Pad_D1.0mm, symbol Connector:TestPoint
- added TP4225: SPARE_2B1, TestPoint:TestPoint_Pad_D1.0mm, symbol Connector:TestPoint
- added TP4226: SPARE_2B2, TestPoint:TestPoint_Pad_D1.0mm, symbol Connector:TestPoint
- added TP4227: SPARE_3B7, TestPoint:TestPoint_Pad_D1.0mm, symbol Connector:TestPoint
- added TP4228: SPARE_3C0, TestPoint:TestPoint_Pad_D1.0mm, symbol Connector:TestPoint
- added TP4229: SPARE_3C4, TestPoint:TestPoint_Pad_D1.0mm, symbol Connector:TestPoint
- added TP4230: SPARE_3C5, TestPoint:TestPoint_Pad_D1.0mm, symbol Connector:TestPoint
- added TP4231: SPARE_4C7, TestPoint:TestPoint_Pad_D1.0mm, symbol Connector:TestPoint
- added TP4232: SPARE_4D0, TestPoint:TestPoint_Pad_D1.0mm, symbol Connector:TestPoint
- added TP4233: SPARE_4D1, TestPoint:TestPoint_Pad_D1.0mm, symbol Connector:TestPoint
- added TP4234: vdd_gpu, TestPoint:TestPoint_Pad_D1.0mm, symbol Connector:TestPoint
- added TP4235: vdd_npu, TestPoint:TestPoint_Pad_D1.0mm, symbol Connector:TestPoint
- added TP4236: vccio6_1v8, TestPoint:TestPoint_Pad_D1.0mm, symbol Connector:TestPoint
- added TP4237: vdda0v9_image, TestPoint:TestPoint_Pad_D1.0mm, symbol Connector:TestPoint
- added TP4238: vdda_0v9, TestPoint:TestPoint_Pad_D1.0mm, symbol Connector:TestPoint
- added TP4239: vdda0v9_pmu, TestPoint:TestPoint_Pad_D1.0mm, symbol Connector:TestPoint
- added TP4240: vccio_sd, TestPoint:TestPoint_Pad_D1.0mm, symbol Connector:TestPoint
- added TP4241: vcc3v3_pmu, TestPoint:TestPoint_Pad_D1.0mm, symbol Connector:TestPoint
- added TP4242: vcca_1v8, TestPoint:TestPoint_Pad_D1.0mm, symbol Connector:TestPoint
- added TP4243: vcca1v8_image, TestPoint:TestPoint_Pad_D1.0mm, symbol Connector:TestPoint
- added TP4244: DAC_VP, TestPoint:TestPoint_Pad_D1.0mm, symbol Connector:TestPoint
- added TP4245: DAC1_VA, TestPoint:TestPoint_Pad_D1.0mm, symbol Connector:TestPoint
- added TP4246: DAC2_VA, TestPoint:TestPoint_Pad_D1.0mm, symbol Connector:TestPoint
- added TP4247: MCLK_3V1, TestPoint:TestPoint_Pad_D1.0mm, symbol Connector:TestPoint
- added TP4248: MCLK_1V8, TestPoint:TestPoint_Pad_D1.0mm, symbol Connector:TestPoint
- added TP4249: AUDIO_P7V0, TestPoint:TestPoint_Pad_D1.0mm, symbol Connector:TestPoint
- added TP4250: AUDIO_N7V0, TestPoint:TestPoint_Pad_D1.0mm, symbol Connector:TestPoint
- added TP4251: BAT_N, TestPoint:TestPoint_Pad_D1.0mm, symbol Connector:TestPoint
- added TP4252: FP_VCI_SRC, TestPoint:TestPoint_Pad_D1.0mm, symbol Connector:TestPoint
- added TP4253: VSYS_SRC, TestPoint:TestPoint_Pad_D1.0mm, symbol Connector:TestPoint
- added TP4254: VSYS_AUDIO, TestPoint:TestPoint_Pad_D1.0mm, symbol Connector:TestPoint
- added TP4255: VSYS_LV_BL, TestPoint:TestPoint_Pad_D1.0mm, symbol Connector:TestPoint
- added TP4256: VSYS_P5V1, TestPoint:TestPoint_Pad_D1.0mm, symbol Connector:TestPoint
Connections:
- net AUDIO_N7V0: now also TP4250.1
- net AUDIO_P7V0: now also TP4249.1
- net BAT_N: now also TP4251.1
- net DAC1_VA: now also TP4245.1
- net DAC2_VA: now also TP4246.1
- net DAC_VP: now also TP4244.1
- net DBG_UART_RX: now also TP4202.1
- net DBG_UART_TX: now also TP4201.1
- net DSD_L: now also TP4207.1
- net DSD_R: now also TP4208.1
- net FP_VCI_SRC: now also TP4252.1
- net GND: now also TP4203.1, TP4209.1
- net I2S_BCLK: now also TP4204.1
- net I2S_LRCK: now also TP4205.1
- net I2S_SDO0: now also TP4206.1
- net MCLK_1V8: now also TP4248.1
- net MCLK_3V1: now also TP4247.1
- net PMIC_INT_N: now also TP4211.1
- net PMIC_SLEEP: now also TP4212.1
- net PWRON_N: now also TP4213.1
- net SOC_RESET_N: now also TP4210.1
- net SPARE_1A0: now also TP4214.1
- net SPARE_1A1: now also TP4215.1
- net SPARE_1A3: now also TP4216.1
- net SPARE_1A4: now also TP4217.1
- net SPARE_1A5: now also TP4218.1
- net SPARE_1A6: now also TP4219.1
- net SPARE_1A7: now also TP4220.1
- net SPARE_1B3: now also TP4221.1
- net SPARE_1D0: now also TP4222.1
- net SPARE_1D1: now also TP4223.1
- net SPARE_1D3: now also TP4224.1
- net SPARE_2B1: now also TP4225.1
- net SPARE_2B2: now also TP4226.1
- net SPARE_3B7: now also TP4227.1
- net SPARE_3C0: now also TP4228.1
- net SPARE_3C4: now also TP4229.1
- net SPARE_3C5: now also TP4230.1
- net SPARE_4C7: now also TP4231.1
- net SPARE_4D0: now also TP4232.1
- net SPARE_4D1: now also TP4233.1
- net VSYS_AUDIO: now also TP4254.1
- net VSYS_LV_BL: now also TP4255.1
- net VSYS_P5V1: now also TP4256.1
- net VSYS_SRC: now also TP4253.1
- net vcc3v3_pmu: now also TP4241.1
- net vcca1v8_image: now also TP4243.1
- net vcca_1v8: now also TP4242.1
- net vccio6_1v8: now also TP4236.1
- net vccio_sd: now also TP4240.1
- net vdd_gpu: now also TP4234.1
- net vdd_npu: now also TP4235.1
- net vdda0v9_image: now also TP4237.1
- net vdda0v9_pmu: now also TP4239.1
- net vdda_0v9: now also TP4238.1

Commit message: Board: capture blk.maskrom
Power + Vol- at a cold power-on pull eMMC D0 low inside the TPS3808G01
boot window (BOM v1 lines 35, 78, 97, 98; sim/maskrom): SENSE 280k/100k,
CT 390 nF, WINDOW_N with its pad, SN74LVC1G57 and SN74LVC1G58 on
vcca1v8_pmu, BAT54 from PWRON_N, DMG1012T through 1 kΩ to EMMC_D0.
Every block in use now has its sheet; the README states the remaining
single-pin nets.

Co-Authored-By: Claude Opus 5.5 <noreply@anthropic.com>
Claude-Session: https://claude.ai/code/session_01Ei262h3TpgY9vyfNLMi5Mn
Parts:
- removed TP4201: DBG_UART_TX, TestPoint:TestPoint_Pad_D1.0mm, symbol Connector:TestPoint
- removed TP4202: DBG_UART_RX, TestPoint:TestPoint_Pad_D1.0mm, symbol Connector:TestPoint
- removed TP4203, TP4209: GND, TestPoint:TestPoint_Pad_D1.0mm, symbol Connector:TestPoint
- removed TP4204: I2S_BCLK, TestPoint:TestPoint_Pad_D1.0mm, symbol Connector:TestPoint
- removed TP4205: I2S_LRCK, TestPoint:TestPoint_Pad_D1.0mm, symbol Connector:TestPoint
- removed TP4206: I2S_SDO0, TestPoint:TestPoint_Pad_D1.0mm, symbol Connector:TestPoint
- removed TP4207: DSD_L, TestPoint:TestPoint_Pad_D1.0mm, symbol Connector:TestPoint
- removed TP4208: DSD_R, TestPoint:TestPoint_Pad_D1.0mm, symbol Connector:TestPoint
- removed TP4210: SOC_RESET_N, TestPoint:TestPoint_Pad_D1.0mm, symbol Connector:TestPoint
- removed TP4211: PMIC_INT_N, TestPoint:TestPoint_Pad_D1.0mm, symbol Connector:TestPoint
- removed TP4212: PMIC_SLEEP, TestPoint:TestPoint_Pad_D1.0mm, symbol Connector:TestPoint
- removed TP4213: PWRON_N, TestPoint:TestPoint_Pad_D1.0mm, symbol Connector:TestPoint
- removed TP4214: SPARE_1A0, TestPoint:TestPoint_Pad_D1.0mm, symbol Connector:TestPoint
- removed TP4215: SPARE_1A1, TestPoint:TestPoint_Pad_D1.0mm, symbol Connector:TestPoint
- removed TP4216: SPARE_1A3, TestPoint:TestPoint_Pad_D1.0mm, symbol Connector:TestPoint
- removed TP4217: SPARE_1A4, TestPoint:TestPoint_Pad_D1.0mm, symbol Connector:TestPoint
- removed TP4218: SPARE_1A5, TestPoint:TestPoint_Pad_D1.0mm, symbol Connector:TestPoint
- removed TP4219: SPARE_1A6, TestPoint:TestPoint_Pad_D1.0mm, symbol Connector:TestPoint
- removed TP4220: SPARE_1A7, TestPoint:TestPoint_Pad_D1.0mm, symbol Connector:TestPoint
- removed TP4221: SPARE_1B3, TestPoint:TestPoint_Pad_D1.0mm, symbol Connector:TestPoint
- removed TP4222: SPARE_1D0, TestPoint:TestPoint_Pad_D1.0mm, symbol Connector:TestPoint
- removed TP4223: SPARE_1D1, TestPoint:TestPoint_Pad_D1.0mm, symbol Connector:TestPoint
- removed TP4224: SPARE_1D3, TestPoint:TestPoint_Pad_D1.0mm, symbol Connector:TestPoint
- removed TP4225: SPARE_2B1, TestPoint:TestPoint_Pad_D1.0mm, symbol Connector:TestPoint
- removed TP4226: SPARE_2B2, TestPoint:TestPoint_Pad_D1.0mm, symbol Connector:TestPoint
- removed TP4227: SPARE_3B7, TestPoint:TestPoint_Pad_D1.0mm, symbol Connector:TestPoint
- removed TP4228: SPARE_3C0, TestPoint:TestPoint_Pad_D1.0mm, symbol Connector:TestPoint
- removed TP4229: SPARE_3C4, TestPoint:TestPoint_Pad_D1.0mm, symbol Connector:TestPoint
- removed TP4230: SPARE_3C5, TestPoint:TestPoint_Pad_D1.0mm, symbol Connector:TestPoint
- removed TP4231: SPARE_4C7, TestPoint:TestPoint_Pad_D1.0mm, symbol Connector:TestPoint
- removed TP4232: SPARE_4D0, TestPoint:TestPoint_Pad_D1.0mm, symbol Connector:TestPoint
- removed TP4233: SPARE_4D1, TestPoint:TestPoint_Pad_D1.0mm, symbol Connector:TestPoint
- removed TP4234: vdd_gpu, TestPoint:TestPoint_Pad_D1.0mm, symbol Connector:TestPoint
- removed TP4235: vdd_npu, TestPoint:TestPoint_Pad_D1.0mm, symbol Connector:TestPoint
- removed TP4236: vccio6_1v8, TestPoint:TestPoint_Pad_D1.0mm, symbol Connector:TestPoint
- removed TP4237: vdda0v9_image, TestPoint:TestPoint_Pad_D1.0mm, symbol Connector:TestPoint
- removed TP4238: vdda_0v9, TestPoint:TestPoint_Pad_D1.0mm, symbol Connector:TestPoint
- removed TP4239: vdda0v9_pmu, TestPoint:TestPoint_Pad_D1.0mm, symbol Connector:TestPoint
- removed TP4240: vccio_sd, TestPoint:TestPoint_Pad_D1.0mm, symbol Connector:TestPoint
- removed TP4241: vcc3v3_pmu, TestPoint:TestPoint_Pad_D1.0mm, symbol Connector:TestPoint
- removed TP4242: vcca_1v8, TestPoint:TestPoint_Pad_D1.0mm, symbol Connector:TestPoint
- removed TP4243: vcca1v8_image, TestPoint:TestPoint_Pad_D1.0mm, symbol Connector:TestPoint
- removed TP4244: DAC_VP, TestPoint:TestPoint_Pad_D1.0mm, symbol Connector:TestPoint
- removed TP4245: DAC1_VA, TestPoint:TestPoint_Pad_D1.0mm, symbol Connector:TestPoint
- removed TP4246: DAC2_VA, TestPoint:TestPoint_Pad_D1.0mm, symbol Connector:TestPoint
- removed TP4247: MCLK_3V1, TestPoint:TestPoint_Pad_D1.0mm, symbol Connector:TestPoint
- removed TP4248: MCLK_1V8, TestPoint:TestPoint_Pad_D1.0mm, symbol Connector:TestPoint
- removed TP4249: AUDIO_P7V0, TestPoint:TestPoint_Pad_D1.0mm, symbol Connector:TestPoint
- removed TP4250: AUDIO_N7V0, TestPoint:TestPoint_Pad_D1.0mm, symbol Connector:TestPoint
- removed TP4251: BAT_N, TestPoint:TestPoint_Pad_D1.0mm, symbol Connector:TestPoint
- removed TP4252: FP_VCI_SRC, TestPoint:TestPoint_Pad_D1.0mm, symbol Connector:TestPoint
- removed TP4253: VSYS_SRC, TestPoint:TestPoint_Pad_D1.0mm, symbol Connector:TestPoint
- removed TP4254: VSYS_AUDIO, TestPoint:TestPoint_Pad_D1.0mm, symbol Connector:TestPoint
- removed TP4255: VSYS_LV_BL, TestPoint:TestPoint_Pad_D1.0mm, symbol Connector:TestPoint
- removed TP4256: VSYS_P5V1, TestPoint:TestPoint_Pad_D1.0mm, symbol Connector:TestPoint
- added TP4301: DBG_UART_TX, TestPoint:TestPoint_Pad_D1.0mm, symbol Connector:TestPoint
- added TP4302: DBG_UART_RX, TestPoint:TestPoint_Pad_D1.0mm, symbol Connector:TestPoint
- added TP4303, TP4309: GND, TestPoint:TestPoint_Pad_D1.0mm, symbol Connector:TestPoint
- added TP4304: I2S_BCLK, TestPoint:TestPoint_Pad_D1.0mm, symbol Connector:TestPoint
- added TP4305: I2S_LRCK, TestPoint:TestPoint_Pad_D1.0mm, symbol Connector:TestPoint
- added TP4306: I2S_SDO0, TestPoint:TestPoint_Pad_D1.0mm, symbol Connector:TestPoint
- added TP4307: DSD_L, TestPoint:TestPoint_Pad_D1.0mm, symbol Connector:TestPoint
- added TP4308: DSD_R, TestPoint:TestPoint_Pad_D1.0mm, symbol Connector:TestPoint
- added TP4310: SOC_RESET_N, TestPoint:TestPoint_Pad_D1.0mm, symbol Connector:TestPoint
- added TP4311: PMIC_INT_N, TestPoint:TestPoint_Pad_D1.0mm, symbol Connector:TestPoint
- added TP4312: PMIC_SLEEP, TestPoint:TestPoint_Pad_D1.0mm, symbol Connector:TestPoint
- added TP4313: PWRON_N, TestPoint:TestPoint_Pad_D1.0mm, symbol Connector:TestPoint
- added TP4314: SPARE_1A0, TestPoint:TestPoint_Pad_D1.0mm, symbol Connector:TestPoint
- added TP4315: SPARE_1A1, TestPoint:TestPoint_Pad_D1.0mm, symbol Connector:TestPoint
- added TP4316: SPARE_1A3, TestPoint:TestPoint_Pad_D1.0mm, symbol Connector:TestPoint
- added TP4317: SPARE_1A4, TestPoint:TestPoint_Pad_D1.0mm, symbol Connector:TestPoint
- added TP4318: SPARE_1A5, TestPoint:TestPoint_Pad_D1.0mm, symbol Connector:TestPoint
- added TP4319: SPARE_1A6, TestPoint:TestPoint_Pad_D1.0mm, symbol Connector:TestPoint
- added TP4320: SPARE_1A7, TestPoint:TestPoint_Pad_D1.0mm, symbol Connector:TestPoint
- added TP4321: SPARE_1B3, TestPoint:TestPoint_Pad_D1.0mm, symbol Connector:TestPoint
- added TP4322: SPARE_1D0, TestPoint:TestPoint_Pad_D1.0mm, symbol Connector:TestPoint
- added TP4323: SPARE_1D1, TestPoint:TestPoint_Pad_D1.0mm, symbol Connector:TestPoint
- added TP4324: SPARE_1D3, TestPoint:TestPoint_Pad_D1.0mm, symbol Connector:TestPoint
- added TP4325: SPARE_2B1, TestPoint:TestPoint_Pad_D1.0mm, symbol Connector:TestPoint
- added TP4326: SPARE_2B2, TestPoint:TestPoint_Pad_D1.0mm, symbol Connector:TestPoint
- added TP4327: SPARE_3B7, TestPoint:TestPoint_Pad_D1.0mm, symbol Connector:TestPoint
- added TP4328: SPARE_3C0, TestPoint:TestPoint_Pad_D1.0mm, symbol Connector:TestPoint
- added TP4329: SPARE_3C4, TestPoint:TestPoint_Pad_D1.0mm, symbol Connector:TestPoint
- added TP4330: SPARE_3C5, TestPoint:TestPoint_Pad_D1.0mm, symbol Connector:TestPoint
- added TP4331: SPARE_4C7, TestPoint:TestPoint_Pad_D1.0mm, symbol Connector:TestPoint
- added TP4332: SPARE_4D0, TestPoint:TestPoint_Pad_D1.0mm, symbol Connector:TestPoint
- added TP4333: SPARE_4D1, TestPoint:TestPoint_Pad_D1.0mm, symbol Connector:TestPoint
- added TP4334: vdd_gpu, TestPoint:TestPoint_Pad_D1.0mm, symbol Connector:TestPoint
- added TP4335: vdd_npu, TestPoint:TestPoint_Pad_D1.0mm, symbol Connector:TestPoint
- added TP4336: vccio6_1v8, TestPoint:TestPoint_Pad_D1.0mm, symbol Connector:TestPoint
- added TP4337: vdda0v9_image, TestPoint:TestPoint_Pad_D1.0mm, symbol Connector:TestPoint
- added TP4338: vdda_0v9, TestPoint:TestPoint_Pad_D1.0mm, symbol Connector:TestPoint
- added TP4339: vdda0v9_pmu, TestPoint:TestPoint_Pad_D1.0mm, symbol Connector:TestPoint
- added TP4340: vccio_sd, TestPoint:TestPoint_Pad_D1.0mm, symbol Connector:TestPoint
- added TP4341: vcc3v3_pmu, TestPoint:TestPoint_Pad_D1.0mm, symbol Connector:TestPoint
- added TP4342: vcca_1v8, TestPoint:TestPoint_Pad_D1.0mm, symbol Connector:TestPoint
- added TP4343: vcca1v8_image, TestPoint:TestPoint_Pad_D1.0mm, symbol Connector:TestPoint
- added TP4344: DAC_VP, TestPoint:TestPoint_Pad_D1.0mm, symbol Connector:TestPoint
- added TP4345: DAC1_VA, TestPoint:TestPoint_Pad_D1.0mm, symbol Connector:TestPoint
- added TP4346: DAC2_VA, TestPoint:TestPoint_Pad_D1.0mm, symbol Connector:TestPoint
- added TP4347: MCLK_3V1, TestPoint:TestPoint_Pad_D1.0mm, symbol Connector:TestPoint
- added TP4348: MCLK_1V8, TestPoint:TestPoint_Pad_D1.0mm, symbol Connector:TestPoint
- added TP4349: AUDIO_P7V0, TestPoint:TestPoint_Pad_D1.0mm, symbol Connector:TestPoint
- added TP4350: AUDIO_N7V0, TestPoint:TestPoint_Pad_D1.0mm, symbol Connector:TestPoint
- added TP4351: BAT_N, TestPoint:TestPoint_Pad_D1.0mm, symbol Connector:TestPoint
- added TP4352: FP_VCI_SRC, TestPoint:TestPoint_Pad_D1.0mm, symbol Connector:TestPoint
- added TP4353: VSYS_SRC, TestPoint:TestPoint_Pad_D1.0mm, symbol Connector:TestPoint
- added TP4354: VSYS_AUDIO, TestPoint:TestPoint_Pad_D1.0mm, symbol Connector:TestPoint
- added TP4355: VSYS_LV_BL, TestPoint:TestPoint_Pad_D1.0mm, symbol Connector:TestPoint
- added TP4356: VSYS_P5V1, TestPoint:TestPoint_Pad_D1.0mm, symbol Connector:TestPoint
Connections:
- net AUDIO_N7V0: now also TP4350.1
- net AUDIO_P7V0: now also TP4349.1
- net BAT_N: now also TP4351.1
- net DAC1_VA: now also TP4345.1
- net DAC2_VA: now also TP4346.1
- net DAC_VP: now also TP4344.1
- net DBG_UART_RX: now also TP4302.1
- net DBG_UART_TX: now also TP4301.1
- net DSD_L: now also TP4307.1
- net DSD_R: now also TP4308.1
- net FP_VCI_SRC: now also TP4352.1
- net GND: now also TP4303.1, TP4309.1
- net I2S_BCLK: now also TP4304.1
- net I2S_LRCK: now also TP4305.1
- net I2S_SDO0: now also TP4306.1
- net MCLK_1V8: now also TP4348.1
- net MCLK_3V1: now also TP4347.1
- net PMIC_INT_N: now also TP4311.1
- net PMIC_SLEEP: now also TP4312.1
- net PWRON_N: now also TP4313.1
- net SOC_RESET_N: now also TP4310.1
- net SPARE_1A0: now also TP4314.1
- net SPARE_1A1: now also TP4315.1
- net SPARE_1A3: now also TP4316.1
- net SPARE_1A4: now also TP4317.1
- net SPARE_1A5: now also TP4318.1
- net SPARE_1A6: now also TP4319.1
- net SPARE_1A7: now also TP4320.1
- net SPARE_1B3: now also TP4321.1
- net SPARE_1D0: now also TP4322.1
- net SPARE_1D1: now also TP4323.1
- net SPARE_1D3: now also TP4324.1
- net SPARE_2B1: now also TP4325.1
- net SPARE_2B2: now also TP4326.1
- net SPARE_3B7: now also TP4327.1
- net SPARE_3C0: now also TP4328.1
- net SPARE_3C4: now also TP4329.1
- net SPARE_3C5: now also TP4330.1
- net SPARE_4C7: now also TP4331.1
- net SPARE_4D0: now also TP4332.1
- net SPARE_4D1: now also TP4333.1
- net VSYS_AUDIO: now also TP4354.1
- net VSYS_LV_BL: now also TP4355.1
- net VSYS_P5V1: now also TP4356.1
- net VSYS_SRC: now also TP4353.1
- net vcc3v3_pmu: now also TP4341.1
- net vcca1v8_image: now also TP4343.1
- net vcca_1v8: now also TP4342.1
- net vccio6_1v8: now also TP4336.1
- net vccio_sd: now also TP4340.1
- net vdd_gpu: now also TP4334.1
- net vdd_npu: now also TP4335.1
- net vdda0v9_image: now also TP4337.1
- net vdda0v9_pmu: now also TP4339.1
- net vdda_0v9: now also TP4338.1

Commit message: Compaction: lower inductors, 0201 decoupling, 0.8 mm signal test pads
A matrix tool (hardware/studies/compaction) checks each candidate against
the design's stresses: same inductance, design peak <= 70 % and the
converter's maximum limit <= 100 % of Isat (30 % drop), height zones,
ratings at least twice the rail, PCB-D-06; sourcing outcome per part.

Applied (placement v1 decision 12, BOM v1.15):
- L601, L4401: XGL4015-102MEC (1.5 mm) for XAL/XGL4020-102MEC (2.1 mm);
- L1001, L5101: XGL4015-471MEC (1.5 mm) for Wurth 744373240047, on the
  stock XxL4020 land (the Wurth land was never drawn);
- L1201 is 1.2 mm (XGL4012, per-MPN heights): it moves next to the SoC;
- 58 x 100 nF decoupling on rails <= 3.3 V in core/IO/radio: 0201;
- 51 test pads on signal nets: 0.8 mm (PCB-D-06 v0.16, JLCPCB guide).
Kept: L901, L2802 (XGL4015 at 103 % of Isat at the limit); no thinner
0805/1206 capacitor passes (obsolete, NRND or unlisted).

Board need 113 % -> 111 % (core band 227 -> 203 %, power band 258 ->
233 %, radio band 19 -> 0 %); only C904 still relies on PCB-Z-04.
ERC 0 errors, craft Q1 met, DRC 0 errors (605 warnings), pcb and study
tests pass, rules test board PASS.

Co-Authored-By: Claude Opus 5.5 <noreply@anthropic.com>
Claude-Session: https://claude.ai/code/session_01Ei262h3TpgY9vyfNLMi5Mn
Parts:
- TP4301, TP4302, TP4304, TP4305, TP4306, TP4307, TP4308, TP4310, TP4311, TP4312, TP4313, TP4314, TP4315, TP4316, TP4317, TP4318, TP4319, TP4320, TP4321, TP4322, TP4323, TP4324, TP4325, TP4326, TP4327, TP4328, TP4329, TP4330, TP4331, TP4332, TP4333: footprint TestPoint:TestPoint_Pad_D1.0mm -> T1_Main_Board:TestPoint_Pad_D0.8mm
