File: board/hardware/t1-main-board/fp-backlight.kicad_sch (KiCad schematic)
At the start: 7 parts, among them U5001 TPS61160DRVR

Commit message: Board: capture blk.current-monitors
Five INA236 on I2C1 (0x40-0x43, 0x48) with their shunts, per power tree
§4.12 and BOM v1 lines 54 and 136. The measured branches are rails of
their own (VSYS_SRC, VSYS_LV_AUDIO, VSYS_AUDIO, VSYS_LV_BL, VSYS_P5V1),
fed through the shunts on this sheet; the charger, audio, backlight and
5.1 V sheets take them. The root's layout may leave a stack level empty,
so the block sits under the notes; IC bboxes hold turned rail values;
passive rows hold a bottom rail's text.

Co-Authored-By: Claude Opus 5.5 <noreply@anthropic.com>
Claude-Session: https://claude.ai/code/session_01Ei262h3TpgY9vyfNLMi5Mn
Parts:
- removed C5001: 4.7 µF, Capacitor_SMD:C_0603_1608Metric, symbol Device:C
- removed C5002: 220 nF, Capacitor_SMD:C_0402_1005Metric, symbol Device:C
- removed C5003: 1 µF, Capacitor_SMD:C_0603_1608Metric, symbol Device:C
- removed D5001: PMEG6010CEH, Diode_SMD:D_SOD-123F, symbol Diode:PMEG6010CEH
- removed L5001: 22 µH, T1_Main_Board:L_Murata_LQH3NP_3x3mm, symbol Device:L
- removed R5001: 3.32 Ω, Resistor_SMD:R_0603_1608Metric, symbol Device:R
- removed U5001: TPS61160DRVR, Texas_Instruments:Texas_DRV0006A_WSON-6-1EP_2x2mm_P0.65mm_EP1x1.6mm, symbol Texas_Instruments:TPS61160DRVR
- added C5101: 4.7 µF, Capacitor_SMD:C_0603_1608Metric, symbol Device:C
- added C5102: 220 nF, Capacitor_SMD:C_0402_1005Metric, symbol Device:C
- added C5103: 1 µF, Capacitor_SMD:C_0603_1608Metric, symbol Device:C
- added D5101: PMEG6010CEH, Diode_SMD:D_SOD-123F, symbol Diode:PMEG6010CEH
- added L5101: 22 µH, T1_Main_Board:L_Murata_LQH3NP_3x3mm, symbol Device:L
- added R5101: 3.32 Ω, Resistor_SMD:R_0603_1608Metric, symbol Device:R
- added U5101: TPS61160DRVR, Texas_Instruments:Texas_DRV0006A_WSON-6-1EP_2x2mm_P0.65mm_EP1x1.6mm, symbol Texas_Instruments:TPS61160DRVR
Connections:
- net BL_COMP: now also C5102.1, U5101.2 (COMP)
- net BL_LEDA: now also C5103.1, D5101.1 (K)
- net BL_LEDK: now also R5101.1, U5101.1 (FB)
- net BL_PWM: now also U5101.5 (CTRL)
- net BL_SW: now also D5101.2 (A), L5101.2, U5101.4 (SW)
- net GND: now also C5101.2, C5102.2, C5103.2, R5101.2, U5101.3 (GND), U5101.7 (EP)
- new net VSYS_LV_BL: C5101.1, L5101.1, U5101.6 (VIN)

Commit message: Board: capture blk.debug
Debug UART2 (1.8 V) and I2S/DSD pads with ground pads, reset, PMIC and
power-key pads (PCB-T-09), a pad on every spare SoC GPIO whose pinout v1
row names one (the DEBUG bus, on the SoC's right edge), and a rail pad
for each power-tree rail no other sheet probes (PCB-T-02). Each DAC
sheet carries a pad on its MCLK. The spares pinout v1 leaves without a
pad now carry no-connect flags. On the root, facing sheet pins are
joined directly only where the route meets no other symbol.

Co-Authored-By: Claude Opus 5.5 <noreply@anthropic.com>
Claude-Session: https://claude.ai/code/session_01Ei262h3TpgY9vyfNLMi5Mn
Parts:
- removed C5101: 4.7 µF, Capacitor_SMD:C_0603_1608Metric, symbol Device:C
- removed C5102: 220 nF, Capacitor_SMD:C_0402_1005Metric, symbol Device:C
- removed C5103: 1 µF, Capacitor_SMD:C_0603_1608Metric, symbol Device:C
- removed D5101: PMEG6010CEH, Diode_SMD:D_SOD-123F, symbol Diode:PMEG6010CEH
- removed L5101: 22 µH, T1_Main_Board:L_Murata_LQH3NP_3x3mm, symbol Device:L
- removed R5101: 3.32 Ω, Resistor_SMD:R_0603_1608Metric, symbol Device:R
- removed U5101: TPS61160DRVR, Texas_Instruments:Texas_DRV0006A_WSON-6-1EP_2x2mm_P0.65mm_EP1x1.6mm, symbol Texas_Instruments:TPS61160DRVR
- added C5201: 4.7 µF, Capacitor_SMD:C_0603_1608Metric, symbol Device:C
- added C5202: 220 nF, Capacitor_SMD:C_0402_1005Metric, symbol Device:C
- added C5203: 1 µF, Capacitor_SMD:C_0603_1608Metric, symbol Device:C
- added D5201: PMEG6010CEH, Diode_SMD:D_SOD-123F, symbol Diode:PMEG6010CEH
- added L5201: 22 µH, T1_Main_Board:L_Murata_LQH3NP_3x3mm, symbol Device:L
- added R5201: 3.32 Ω, Resistor_SMD:R_0603_1608Metric, symbol Device:R
- added U5201: TPS61160DRVR, Texas_Instruments:Texas_DRV0006A_WSON-6-1EP_2x2mm_P0.65mm_EP1x1.6mm, symbol Texas_Instruments:TPS61160DRVR
Connections:
- net BL_COMP: now also C5202.1, U5201.2 (COMP)
- net BL_LEDA: now also C5203.1, D5201.1 (K)
- net BL_LEDK: now also R5201.1, U5201.1 (FB)
- net BL_PWM: now also U5201.5 (CTRL)
- net BL_SW: now also D5201.2 (A), L5201.2, U5201.4 (SW)
- net GND: now also C5201.2, C5202.2, C5203.2, R5201.2, U5201.3 (GND), U5201.7 (EP)
- net VSYS_LV_BL: now also C5201.1, L5201.1, U5201.6 (VIN)
Changed lines of the file:
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@@
 (title_block (title "Faceplate backlight") (date "2026-10-25") (rev "A") (company "The OpenDAP Project") (comment 1 "blk.fp-backlight") (comment 2 "TPS61160 boost LED driver, 60 mA, open-LED threshold below 30 V"))
 (symbol (lib_id "Texas_Instruments:TPS61160DRVR") (at 45.72 60.96 0) (unit 1) (body_style 1) (exclude_from_sim no) (in_bom yes) (on_board yes) (dnp no)
-  (property "Reference" "U5101" (at 46.99 45.72 0) (effects (font (size 1.27 1.27)) (justify left)))
+  (property "Reference" "U5201" (at 46.99 45.72 0) (effects (font (size 1.27 1.27)) (justify left)))
   (property "Value" "TPS61160DRVR" (at 46.99 43.18 0) (effects (font (size 1.27 1.27)) (justify left)))
   (property "Footprint" "Texas_Instruments:Texas_DRV0006A_WSON-6-1EP_2x2mm_P0.65mm_EP1x1.6mm" (at 45.72 60.96 0) (effects (font (size 1.27 1.27))) (hide yes))
@@
   (pin "3")
   (pin "7")
-  (instances (project "t1-main-board" (path "/7746052e-d7f9-59ad-ba73-bd2b74439529/d5d538fb-ce80-5e4a-9a88-723f34af818e" (reference "U5101") (unit 1))))
+  (instances (project "t1-main-board" (path "/7746052e-d7f9-59ad-ba73-bd2b74439529/d5d538fb-ce80-5e4a-9a88-723f34af818e" (reference "U5201") (unit 1))))
 )
 (wire (pts (xy 43.18 76.2) (xy 43.18 78.74)) (stroke (width 0) (type default)))
@@
 )
 (symbol (lib_id "Device:C") (at 72.39 53.34 0) (unit 1) (body_style 1) (exclude_from_sim no) (in_bom yes) (on_board yes) (dnp no)
-  (property "Reference" "C5101" (at 74.93 52.07 0) (effects (font (size 1.27 1.27)) (justify left)))
+  (property "Reference" "C5201" (at 74.93 52.07 0) (effects (font (size 1.27 1.27)) (justify left)))
   (property "Value" "4.7 µF" (at 74.93 54.61 0) (effects (font (size 1.27 1.27)) (justify left)))
   (property "Spec" "10 V X5R" (at 74.93 57.15 0) (effects (font (size 1.27 1.27)) (justify left)))
@@
   (pin "1")
   (pin "2")
-  (instances (project "t1-main-board" (path "/7746052e-d7f9-59ad-ba73-bd2b74439529/d5d538fb-ce80-5e4a-9a88-723f34af818e" (reference "C5101") (unit 1))))
+  (instances (project "t1-main-board" (path "/7746052e-d7f9-59ad-ba73-bd2b74439529/d5d538fb-ce80-5e4a-9a88-723f34af818e" (reference "C5201") (unit 1))))
 )
 (wire (pts (xy 72.39 49.53) (xy 72.39 46.99)) (stroke (width 0) (type default)))
@@
 )
 (symbol (lib_id "Device:C") (at 87.63 53.34 0) (unit 1) (body_style 1) (exclude_from_sim no) (in_bom yes) (on_board yes) (dnp no)
-  (property "Reference" "C5102" (at 90.17 52.07 0) (effects (font (size 1.27 1.27)) (justify left)))
+  (property "Reference" "C5202" (at 90.17 52.07 0) (effects (font (size 1.27 1.27)) (justify left)))
   (property "Value" "220 nF" (at 90.17 54.61 0) (effects (font (size 1.27 1.27)) (justify left)))
   (property "Spec" "10 V X5R" (at 90.17 57.15 0) (effects (font (size 1.27 1.27)) (justify left)))
@@
   (pin "1")
   (pin "2")
-  (instances (project "t1-main-board" (path "/7746052e-d7f9-59ad-ba73-bd2b74439529/d5d538fb-ce80-5e4a-9a88-723f34af818e" (reference "C5102") (unit 1))))
+  (instances (project "t1-main-board" (path "/7746052e-d7f9-59ad-ba73-bd2b74439529/d5d538fb-ce80-5e4a-9a88-723f34af818e" (reference "C5202") (unit 1))))
 )
 (wire (pts (xy 87.63 49.53) (xy 87.63 46.99)) (stroke (width 0) (type default)))
@@
 )
 (symbol (lib_id "Device:R") (at 102.87 53.34 0) (unit 1) (body_style 1) (exclude_from_sim no) (in_bom yes) (on_board yes) (dnp no)
-  (property "Reference" "R5101" (at 104.14 52.07 0) (effects (font (size 1.27 1.27)) (justify left)))
+  (property "Reference" "R5201" (at 104.14 52.07 0) (effects (font (size 1.27 1.27)) (justify left)))
   (property "Value" "3.32 Ω" (at 104.14 54.61 0) (effects (font (size 1.27 1.27)) (justify left)))
   (property "Footprint" "Resistor_SMD:R_0603_1608Metric" (at 102.87 53.34 0) (effects (font (size 1.27 1.27))) (hide yes))
@@
   (pin "1")
   (pin "2")
-  (instances (project "t1-main-board" (path "/7746052e-d7f9-59ad-ba73-bd2b74439529/d5d538fb-ce80-5e4a-9a88-723f34af818e" (reference "R5101") (unit 1))))
+  (instances (project "t1-main-board" (path "/7746052e-d7f9-59ad-ba73-bd2b74439529/d5d538fb-ce80-5e4a-9a88-723f34af818e" (reference "R5201") (unit 1))))
 )
 (wire (pts (xy 102.87 49.53) (xy 102.87 46.99)) (stroke (width 0) (type default)))
@@
 (text "TPS61160, RSET 3.32 Ω for 60 mA (BOM v1 line 51)" (exclude_from_sim no) (at 24.13 34.29 0) (effects (font (size 2.54 2.54)) (justify left bottom)))
 (symbol (lib_id "Device:L") (at 162.56 45.72 90) (unit 1) (body_style 1) (exclude_from_sim no) (in_bom yes) (on_board yes) (dnp no)
-  (property "Reference" "L5101" (at 162.56 43.18 90) (effects (font (size 1.27 1.27))))
+  (property "Reference" "L5201" (at 162.56 43.18 90) (effects (font (size 1.27 1.27))))
   (property "Value" "22 µH" (at 162.56 48.26 90) (effects (font (size 1.27 1.27))))
   (property "Footprint" "T1_Main_Board:L_Murata_LQH3NP_3x3mm" (at 162.56 45.72 0) (effects (font (size 1.27 1.27))) (hide yes))
@@
   (pin "1")
   (pin "2")
-  (instances (project "t1-main-board" (path "/7746052e-d7f9-59ad-ba73-bd2b74439529/d5d538fb-ce80-5e4a-9a88-723f34af818e" (reference "L5101") (unit 1))))
+  (instances (project "t1-main-board" (path "/7746052e-d7f9-59ad-ba73-bd2b74439529/d5d538fb-ce80-5e4a-9a88-723f34af818e" (reference "L5201") (unit 1))))
 )
 (wire (pts (xy 158.75 45.72) (xy 156.21 45.72)) (stroke (width 0) (type default)))
@@
 (wire (pts (xy 166.37 45.72) (xy 168.91 45.72)) (stroke (width 0) (type default)))
 (symbol (lib_id "Diode:PMEG6010CEH") (at 170.18 60.96 180) (unit 1) (body_style 1) (exclude_from_sim no) (in_bom yes) (on_board yes) (dnp no)
-  (property "Reference" "D5101" (at 170.18 54.61 0) (effects (font (size 1.27 1.27)) (justify left)))
+  (property "Reference" "D5201" (at 170.18 54.61 0) (effects (font (size 1.27 1.27)) (justify left)))
   (property "Value" "PMEG6010CEH" (at 170.18 57.15 0) (effects (font (size 1.27 1.27)) (justify left)))
   (property "Footprint" "Diode_SMD:D_SOD-123F" (at 170.18 60.96 0) (effects (font (size 1.27 1.27))) (hide yes))
@@
   (pin "1")
   (pin "2")
-  (instances (project "t1-main-board" (path "/7746052e-d7f9-59ad-ba73-bd2b74439529/d5d538fb-ce80-5e4a-9a88-723f34af818e" (reference "D5101") (unit 1))))
+  (instances (project "t1-main-board" (path "/7746052e-d7f9-59ad-ba73-bd2b74439529/d5d538fb-ce80-5e4a-9a88-723f34af818e" (reference "D5201") (unit 1))))
 )
 (wire (pts (xy 173.99 60.96) (xy 179.07 60.96)) (stroke (width 0) (type default)))
 (wire (pts (xy 166.37 60.96) (xy 161.29 60.96)) (stroke (width 0) (type default)))
 (symbol (lib_id "Device:C") (at 154.94 81.28 0) (unit 1) (body_style 1) (exclude_from_sim no) (in_bom yes) (on_board yes) (dnp no)
-  (property "Reference" "C5103" (at 157.48 80.01 0) (effects (font (size 1.27 1.27)) (justify left)))
+  (property "Reference" "C5203" (at 157.48 80.01 0) (effects (font (size 1.27 1.27)) (justify left)))
   (property "Value" "1 µF" (at 157.48 82.55 0) (effects (font (size 1.27 1.27)) (justify left)))
   (property "Spec" "50 V X7R" (at 157.48 85.09 0) (effects (font (size 1.27 1.27)) (justify left)))
@@
   (pin "1")
   (pin "2")
-  (instances (project "t1-main-board" (path "/7746052e-d7f9-59ad-ba73-bd2b74439529/d5d538fb-ce80-5e4a-9a88-723f34af818e" (reference "C5103") (unit 1))))
+  (instances (project "t1-main-board" (path "/7746052e-d7f9-59ad-ba73-bd2b74439529/d5d538fb-ce80-5e4a-9a88-723f34af818e" (reference "C5203") (unit 1))))
 )
 (wire (pts (xy 154.94 77.47) (xy 154.94 74.93)) (stroke (width 0) (type default)))

Commit message: Board: capture blk.mic-ambient and links #34, #35
IM73D122 on PDM CLK1 and SDI1 (BOM v1 line 34, pinout v1 AK2 and 1P2),
LR to ground, 22 Ω clock series, VDD from MIC_1V8 through link #35.
Link #34 on blk.mic-main makes the faceplate branch the rail MIC_1V8_FP
for contact 40 (power tree §4.12, G10). kicad-lib moves to e46bda4 for
the IM73D122, TPS3808G01, SN74LVC1G58 and BAT54 parts.

Co-Authored-By: Claude Opus 5.5 <noreply@anthropic.com>
Claude-Session: https://claude.ai/code/session_01Ei262h3TpgY9vyfNLMi5Mn
Parts:
- removed C5201: 4.7 µF, Capacitor_SMD:C_0603_1608Metric, symbol Device:C
- removed C5202: 220 nF, Capacitor_SMD:C_0402_1005Metric, symbol Device:C
- removed C5203: 1 µF, Capacitor_SMD:C_0603_1608Metric, symbol Device:C
- removed D5201: PMEG6010CEH, Diode_SMD:D_SOD-123F, symbol Diode:PMEG6010CEH
- removed L5201: 22 µH, T1_Main_Board:L_Murata_LQH3NP_3x3mm, symbol Device:L
- removed R5201: 3.32 Ω, Resistor_SMD:R_0603_1608Metric, symbol Device:R
- removed U5201: TPS61160DRVR, Texas_Instruments:Texas_DRV0006A_WSON-6-1EP_2x2mm_P0.65mm_EP1x1.6mm, symbol Texas_Instruments:TPS61160DRVR
- added C5301: 4.7 µF, Capacitor_SMD:C_0603_1608Metric, symbol Device:C
- added C5302: 220 nF, Capacitor_SMD:C_0402_1005Metric, symbol Device:C
- added C5303: 1 µF, Capacitor_SMD:C_0603_1608Metric, symbol Device:C
- added D5301: PMEG6010CEH, Diode_SMD:D_SOD-123F, symbol Diode:PMEG6010CEH
- added L5301: 22 µH, T1_Main_Board:L_Murata_LQH3NP_3x3mm, symbol Device:L
- added R5301: 3.32 Ω, Resistor_SMD:R_0603_1608Metric, symbol Device:R
- added U5301: TPS61160DRVR, Texas_Instruments:Texas_DRV0006A_WSON-6-1EP_2x2mm_P0.65mm_EP1x1.6mm, symbol Texas_Instruments:TPS61160DRVR
Connections:
- net BL_COMP: now also C5302.1, U5301.2 (COMP)
- net BL_LEDA: now also C5303.1, D5301.1 (K)
- net BL_LEDK: now also R5301.1, U5301.1 (FB)
- net BL_PWM: now also U5301.5 (CTRL)
- net BL_SW: now also D5301.2 (A), L5301.2, U5301.4 (SW)
- net GND: now also C5301.2, C5302.2, C5303.2, R5301.2, U5301.3 (GND), U5301.7 (EP)
- net VSYS_LV_BL: now also C5301.1, L5301.1, U5301.6 (VIN)
Changed lines of the file:
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@@
 (title_block (title "Faceplate backlight") (date "2026-10-25") (rev "A") (company "The OpenDAP Project") (comment 1 "blk.fp-backlight") (comment 2 "TPS61160 boost LED driver, 60 mA, open-LED threshold below 30 V"))
 (symbol (lib_id "Texas_Instruments:TPS61160DRVR") (at 45.72 60.96 0) (unit 1) (body_style 1) (exclude_from_sim no) (in_bom yes) (on_board yes) (dnp no)
-  (property "Reference" "U5201" (at 46.99 45.72 0) (effects (font (size 1.27 1.27)) (justify left)))
+  (property "Reference" "U5301" (at 46.99 45.72 0) (effects (font (size 1.27 1.27)) (justify left)))
   (property "Value" "TPS61160DRVR" (at 46.99 43.18 0) (effects (font (size 1.27 1.27)) (justify left)))
   (property "Footprint" "Texas_Instruments:Texas_DRV0006A_WSON-6-1EP_2x2mm_P0.65mm_EP1x1.6mm" (at 45.72 60.96 0) (effects (font (size 1.27 1.27))) (hide yes))
@@
   (pin "3")
   (pin "7")
-  (instances (project "t1-main-board" (path "/7746052e-d7f9-59ad-ba73-bd2b74439529/d5d538fb-ce80-5e4a-9a88-723f34af818e" (reference "U5201") (unit 1))))
+  (instances (project "t1-main-board" (path "/7746052e-d7f9-59ad-ba73-bd2b74439529/d5d538fb-ce80-5e4a-9a88-723f34af818e" (reference "U5301") (unit 1))))
 )
 (wire (pts (xy 43.18 76.2) (xy 43.18 78.74)) (stroke (width 0) (type default)))
@@
 )
 (symbol (lib_id "Device:C") (at 72.39 53.34 0) (unit 1) (body_style 1) (exclude_from_sim no) (in_bom yes) (on_board yes) (dnp no)
-  (property "Reference" "C5201" (at 74.93 52.07 0) (effects (font (size 1.27 1.27)) (justify left)))
+  (property "Reference" "C5301" (at 74.93 52.07 0) (effects (font (size 1.27 1.27)) (justify left)))
   (property "Value" "4.7 µF" (at 74.93 54.61 0) (effects (font (size 1.27 1.27)) (justify left)))
   (property "Spec" "10 V X5R" (at 74.93 57.15 0) (effects (font (size 1.27 1.27)) (justify left)))
@@
   (pin "1")
   (pin "2")
-  (instances (project "t1-main-board" (path "/7746052e-d7f9-59ad-ba73-bd2b74439529/d5d538fb-ce80-5e4a-9a88-723f34af818e" (reference "C5201") (unit 1))))
+  (instances (project "t1-main-board" (path "/7746052e-d7f9-59ad-ba73-bd2b74439529/d5d538fb-ce80-5e4a-9a88-723f34af818e" (reference "C5301") (unit 1))))
 )
 (wire (pts (xy 72.39 49.53) (xy 72.39 46.99)) (stroke (width 0) (type default)))
@@
 )
 (symbol (lib_id "Device:C") (at 87.63 53.34 0) (unit 1) (body_style 1) (exclude_from_sim no) (in_bom yes) (on_board yes) (dnp no)
-  (property "Reference" "C5202" (at 90.17 52.07 0) (effects (font (size 1.27 1.27)) (justify left)))
+  (property "Reference" "C5302" (at 90.17 52.07 0) (effects (font (size 1.27 1.27)) (justify left)))
   (property "Value" "220 nF" (at 90.17 54.61 0) (effects (font (size 1.27 1.27)) (justify left)))
   (property "Spec" "10 V X5R" (at 90.17 57.15 0) (effects (font (size 1.27 1.27)) (justify left)))
@@
   (pin "1")
   (pin "2")
-  (instances (project "t1-main-board" (path "/7746052e-d7f9-59ad-ba73-bd2b74439529/d5d538fb-ce80-5e4a-9a88-723f34af818e" (reference "C5202") (unit 1))))
+  (instances (project "t1-main-board" (path "/7746052e-d7f9-59ad-ba73-bd2b74439529/d5d538fb-ce80-5e4a-9a88-723f34af818e" (reference "C5302") (unit 1))))
 )
 (wire (pts (xy 87.63 49.53) (xy 87.63 46.99)) (stroke (width 0) (type default)))
@@
 )
 (symbol (lib_id "Device:R") (at 102.87 53.34 0) (unit 1) (body_style 1) (exclude_from_sim no) (in_bom yes) (on_board yes) (dnp no)
-  (property "Reference" "R5201" (at 104.14 52.07 0) (effects (font (size 1.27 1.27)) (justify left)))
+  (property "Reference" "R5301" (at 104.14 52.07 0) (effects (font (size 1.27 1.27)) (justify left)))
   (property "Value" "3.32 Ω" (at 104.14 54.61 0) (effects (font (size 1.27 1.27)) (justify left)))
   (property "Footprint" "Resistor_SMD:R_0603_1608Metric" (at 102.87 53.34 0) (effects (font (size 1.27 1.27))) (hide yes))
@@
   (pin "1")
   (pin "2")
-  (instances (project "t1-main-board" (path "/7746052e-d7f9-59ad-ba73-bd2b74439529/d5d538fb-ce80-5e4a-9a88-723f34af818e" (reference "R5201") (unit 1))))
+  (instances (project "t1-main-board" (path "/7746052e-d7f9-59ad-ba73-bd2b74439529/d5d538fb-ce80-5e4a-9a88-723f34af818e" (reference "R5301") (unit 1))))
 )
 (wire (pts (xy 102.87 49.53) (xy 102.87 46.99)) (stroke (width 0) (type default)))
@@
 (text "TPS61160, RSET 3.32 Ω for 60 mA (BOM v1 line 51)" (exclude_from_sim no) (at 24.13 34.29 0) (effects (font (size 2.54 2.54)) (justify left bottom)))
 (symbol (lib_id "Device:L") (at 162.56 45.72 90) (unit 1) (body_style 1) (exclude_from_sim no) (in_bom yes) (on_board yes) (dnp no)
-  (property "Reference" "L5201" (at 162.56 43.18 90) (effects (font (size 1.27 1.27))))
+  (property "Reference" "L5301" (at 162.56 43.18 90) (effects (font (size 1.27 1.27))))
   (property "Value" "22 µH" (at 162.56 48.26 90) (effects (font (size 1.27 1.27))))
   (property "Footprint" "T1_Main_Board:L_Murata_LQH3NP_3x3mm" (at 162.56 45.72 0) (effects (font (size 1.27 1.27))) (hide yes))
@@
   (pin "1")
   (pin "2")
-  (instances (project "t1-main-board" (path "/7746052e-d7f9-59ad-ba73-bd2b74439529/d5d538fb-ce80-5e4a-9a88-723f34af818e" (reference "L5201") (unit 1))))
+  (instances (project "t1-main-board" (path "/7746052e-d7f9-59ad-ba73-bd2b74439529/d5d538fb-ce80-5e4a-9a88-723f34af818e" (reference "L5301") (unit 1))))
 )
 (wire (pts (xy 158.75 45.72) (xy 156.21 45.72)) (stroke (width 0) (type default)))
@@
 (wire (pts (xy 166.37 45.72) (xy 168.91 45.72)) (stroke (width 0) (type default)))
 (symbol (lib_id "Diode:PMEG6010CEH") (at 170.18 60.96 180) (unit 1) (body_style 1) (exclude_from_sim no) (in_bom yes) (on_board yes) (dnp no)
-  (property "Reference" "D5201" (at 170.18 54.61 0) (effects (font (size 1.27 1.27)) (justify left)))
+  (property "Reference" "D5301" (at 170.18 54.61 0) (effects (font (size 1.27 1.27)) (justify left)))
   (property "Value" "PMEG6010CEH" (at 170.18 57.15 0) (effects (font (size 1.27 1.27)) (justify left)))
   (property "Footprint" "Diode_SMD:D_SOD-123F" (at 170.18 60.96 0) (effects (font (size 1.27 1.27))) (hide yes))
@@
   (pin "1")
   (pin "2")
-  (instances (project "t1-main-board" (path "/7746052e-d7f9-59ad-ba73-bd2b74439529/d5d538fb-ce80-5e4a-9a88-723f34af818e" (reference "D5201") (unit 1))))
+  (instances (project "t1-main-board" (path "/7746052e-d7f9-59ad-ba73-bd2b74439529/d5d538fb-ce80-5e4a-9a88-723f34af818e" (reference "D5301") (unit 1))))
 )
 (wire (pts (xy 173.99 60.96) (xy 179.07 60.96)) (stroke (width 0) (type default)))
 (wire (pts (xy 166.37 60.96) (xy 161.29 60.96)) (stroke (width 0) (type default)))
 (symbol (lib_id "Device:C") (at 154.94 81.28 0) (unit 1) (body_style 1) (exclude_from_sim no) (in_bom yes) (on_board yes) (dnp no)
-  (property "Reference" "C5203" (at 157.48 80.01 0) (effects (font (size 1.27 1.27)) (justify left)))
+  (property "Reference" "C5303" (at 157.48 80.01 0) (effects (font (size 1.27 1.27)) (justify left)))
   (property "Value" "1 µF" (at 157.48 82.55 0) (effects (font (size 1.27 1.27)) (justify left)))
   (property "Spec" "50 V X7R" (at 157.48 85.09 0) (effects (font (size 1.27 1.27)) (justify left)))
@@
   (pin "1")
   (pin "2")
-  (instances (project "t1-main-board" (path "/7746052e-d7f9-59ad-ba73-bd2b74439529/d5d538fb-ce80-5e4a-9a88-723f34af818e" (reference "C5203") (unit 1))))
+  (instances (project "t1-main-board" (path "/7746052e-d7f9-59ad-ba73-bd2b74439529/d5d538fb-ce80-5e4a-9a88-723f34af818e" (reference "C5303") (unit 1))))
 )
 (wire (pts (xy 154.94 77.47) (xy 154.94 74.93)) (stroke (width 0) (type default)))
