File: board/hardware/t1-main-board/fp-backlight.kicad_sch (KiCad schematic)
At the start: 7 parts, among them U5301 TPS61160DRVR

Commit message: Board: capture blk.maskrom
Power + Vol- at a cold power-on pull eMMC D0 low inside the TPS3808G01
boot window (BOM v1 lines 35, 78, 97, 98; sim/maskrom): SENSE 280k/100k,
CT 390 nF, WINDOW_N with its pad, SN74LVC1G57 and SN74LVC1G58 on
vcca1v8_pmu, BAT54 from PWRON_N, DMG1012T through 1 kΩ to EMMC_D0.
Every block in use now has its sheet; the README states the remaining
single-pin nets.

Co-Authored-By: Claude Opus 5.5 <noreply@anthropic.com>
Claude-Session: https://claude.ai/code/session_01Ei262h3TpgY9vyfNLMi5Mn
Parts:
- removed C5301: 4.7 µF, Capacitor_SMD:C_0603_1608Metric, symbol Device:C
- removed C5302: 220 nF, Capacitor_SMD:C_0402_1005Metric, symbol Device:C
- removed C5303: 1 µF, Capacitor_SMD:C_0603_1608Metric, symbol Device:C
- removed D5301: PMEG6010CEH, Diode_SMD:D_SOD-123F, symbol Diode:PMEG6010CEH
- removed L5301: 22 µH, T1_Main_Board:L_Murata_LQH3NP_3x3mm, symbol Device:L
- removed R5301: 3.32 Ω, Resistor_SMD:R_0603_1608Metric, symbol Device:R
- removed U5301: TPS61160DRVR, Texas_Instruments:Texas_DRV0006A_WSON-6-1EP_2x2mm_P0.65mm_EP1x1.6mm, symbol Texas_Instruments:TPS61160DRVR
- added C5401: 4.7 µF, Capacitor_SMD:C_0603_1608Metric, symbol Device:C
- added C5402: 220 nF, Capacitor_SMD:C_0402_1005Metric, symbol Device:C
- added C5403: 1 µF, Capacitor_SMD:C_0603_1608Metric, symbol Device:C
- added D5401: PMEG6010CEH, Diode_SMD:D_SOD-123F, symbol Diode:PMEG6010CEH
- added L5401: 22 µH, T1_Main_Board:L_Murata_LQH3NP_3x3mm, symbol Device:L
- added R5401: 3.32 Ω, Resistor_SMD:R_0603_1608Metric, symbol Device:R
- added U5401: TPS61160DRVR, Texas_Instruments:Texas_DRV0006A_WSON-6-1EP_2x2mm_P0.65mm_EP1x1.6mm, symbol Texas_Instruments:TPS61160DRVR
Connections:
- net BL_COMP: now also C5402.1, U5401.2 (COMP)
- net BL_LEDA: now also C5403.1, D5401.1 (K)
- net BL_LEDK: now also R5401.1, U5401.1 (FB)
- net BL_PWM: now also U5401.5 (CTRL)
- net BL_SW: now also D5401.2 (A), L5401.2, U5401.4 (SW)
- net GND: now also C5401.2, C5402.2, C5403.2, R5401.2, U5401.3 (GND), U5401.7 (EP)
- net VSYS_LV_BL: now also C5401.1, L5401.1, U5401.6 (VIN)
Changed lines of the file:
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@@
 (title_block (title "Faceplate backlight") (date "2026-10-25") (rev "A") (company "The OpenDAP Project") (comment 1 "blk.fp-backlight") (comment 2 "TPS61160 boost LED driver, 60 mA, open-LED threshold below 30 V"))
 (symbol (lib_id "Texas_Instruments:TPS61160DRVR") (at 45.72 60.96 0) (unit 1) (body_style 1) (exclude_from_sim no) (in_bom yes) (on_board yes) (dnp no)
-  (property "Reference" "U5301" (at 46.99 45.72 0) (effects (font (size 1.27 1.27)) (justify left)))
+  (property "Reference" "U5401" (at 46.99 45.72 0) (effects (font (size 1.27 1.27)) (justify left)))
   (property "Value" "TPS61160DRVR" (at 46.99 43.18 0) (effects (font (size 1.27 1.27)) (justify left)))
   (property "Footprint" "Texas_Instruments:Texas_DRV0006A_WSON-6-1EP_2x2mm_P0.65mm_EP1x1.6mm" (at 45.72 60.96 0) (effects (font (size 1.27 1.27))) (hide yes))
@@
   (pin "3")
   (pin "7")
-  (instances (project "t1-main-board" (path "/7746052e-d7f9-59ad-ba73-bd2b74439529/d5d538fb-ce80-5e4a-9a88-723f34af818e" (reference "U5301") (unit 1))))
+  (instances (project "t1-main-board" (path "/7746052e-d7f9-59ad-ba73-bd2b74439529/d5d538fb-ce80-5e4a-9a88-723f34af818e" (reference "U5401") (unit 1))))
 )
 (wire (pts (xy 43.18 76.2) (xy 43.18 78.74)) (stroke (width 0) (type default)))
@@
 )
 (symbol (lib_id "Device:C") (at 72.39 53.34 0) (unit 1) (body_style 1) (exclude_from_sim no) (in_bom yes) (on_board yes) (dnp no)
-  (property "Reference" "C5301" (at 74.93 52.07 0) (effects (font (size 1.27 1.27)) (justify left)))
+  (property "Reference" "C5401" (at 74.93 52.07 0) (effects (font (size 1.27 1.27)) (justify left)))
   (property "Value" "4.7 µF" (at 74.93 54.61 0) (effects (font (size 1.27 1.27)) (justify left)))
   (property "Spec" "10 V X5R" (at 74.93 57.15 0) (effects (font (size 1.27 1.27)) (justify left)))
@@
   (pin "1")
   (pin "2")
-  (instances (project "t1-main-board" (path "/7746052e-d7f9-59ad-ba73-bd2b74439529/d5d538fb-ce80-5e4a-9a88-723f34af818e" (reference "C5301") (unit 1))))
+  (instances (project "t1-main-board" (path "/7746052e-d7f9-59ad-ba73-bd2b74439529/d5d538fb-ce80-5e4a-9a88-723f34af818e" (reference "C5401") (unit 1))))
 )
 (wire (pts (xy 72.39 49.53) (xy 72.39 46.99)) (stroke (width 0) (type default)))
@@
 )
 (symbol (lib_id "Device:C") (at 87.63 53.34 0) (unit 1) (body_style 1) (exclude_from_sim no) (in_bom yes) (on_board yes) (dnp no)
-  (property "Reference" "C5302" (at 90.17 52.07 0) (effects (font (size 1.27 1.27)) (justify left)))
+  (property "Reference" "C5402" (at 90.17 52.07 0) (effects (font (size 1.27 1.27)) (justify left)))
   (property "Value" "220 nF" (at 90.17 54.61 0) (effects (font (size 1.27 1.27)) (justify left)))
   (property "Spec" "10 V X5R" (at 90.17 57.15 0) (effects (font (size 1.27 1.27)) (justify left)))
@@
   (pin "1")
   (pin "2")
-  (instances (project "t1-main-board" (path "/7746052e-d7f9-59ad-ba73-bd2b74439529/d5d538fb-ce80-5e4a-9a88-723f34af818e" (reference "C5302") (unit 1))))
+  (instances (project "t1-main-board" (path "/7746052e-d7f9-59ad-ba73-bd2b74439529/d5d538fb-ce80-5e4a-9a88-723f34af818e" (reference "C5402") (unit 1))))
 )
 (wire (pts (xy 87.63 49.53) (xy 87.63 46.99)) (stroke (width 0) (type default)))
@@
 )
 (symbol (lib_id "Device:R") (at 102.87 53.34 0) (unit 1) (body_style 1) (exclude_from_sim no) (in_bom yes) (on_board yes) (dnp no)
-  (property "Reference" "R5301" (at 104.14 52.07 0) (effects (font (size 1.27 1.27)) (justify left)))
+  (property "Reference" "R5401" (at 104.14 52.07 0) (effects (font (size 1.27 1.27)) (justify left)))
   (property "Value" "3.32 Ω" (at 104.14 54.61 0) (effects (font (size 1.27 1.27)) (justify left)))
   (property "Footprint" "Resistor_SMD:R_0603_1608Metric" (at 102.87 53.34 0) (effects (font (size 1.27 1.27))) (hide yes))
@@
   (pin "1")
   (pin "2")
-  (instances (project "t1-main-board" (path "/7746052e-d7f9-59ad-ba73-bd2b74439529/d5d538fb-ce80-5e4a-9a88-723f34af818e" (reference "R5301") (unit 1))))
+  (instances (project "t1-main-board" (path "/7746052e-d7f9-59ad-ba73-bd2b74439529/d5d538fb-ce80-5e4a-9a88-723f34af818e" (reference "R5401") (unit 1))))
 )
 (wire (pts (xy 102.87 49.53) (xy 102.87 46.99)) (stroke (width 0) (type default)))
@@
 (text "TPS61160, RSET 3.32 Ω for 60 mA (BOM v1 line 51)" (exclude_from_sim no) (at 24.13 34.29 0) (effects (font (size 2.54 2.54)) (justify left bottom)))
 (symbol (lib_id "Device:L") (at 162.56 45.72 90) (unit 1) (body_style 1) (exclude_from_sim no) (in_bom yes) (on_board yes) (dnp no)
-  (property "Reference" "L5301" (at 162.56 43.18 90) (effects (font (size 1.27 1.27))))
+  (property "Reference" "L5401" (at 162.56 43.18 90) (effects (font (size 1.27 1.27))))
   (property "Value" "22 µH" (at 162.56 48.26 90) (effects (font (size 1.27 1.27))))
   (property "Footprint" "T1_Main_Board:L_Murata_LQH3NP_3x3mm" (at 162.56 45.72 0) (effects (font (size 1.27 1.27))) (hide yes))
@@
   (pin "1")
   (pin "2")
-  (instances (project "t1-main-board" (path "/7746052e-d7f9-59ad-ba73-bd2b74439529/d5d538fb-ce80-5e4a-9a88-723f34af818e" (reference "L5301") (unit 1))))
+  (instances (project "t1-main-board" (path "/7746052e-d7f9-59ad-ba73-bd2b74439529/d5d538fb-ce80-5e4a-9a88-723f34af818e" (reference "L5401") (unit 1))))
 )
 (wire (pts (xy 158.75 45.72) (xy 156.21 45.72)) (stroke (width 0) (type default)))
@@
 (wire (pts (xy 166.37 45.72) (xy 168.91 45.72)) (stroke (width 0) (type default)))
 (symbol (lib_id "Diode:PMEG6010CEH") (at 170.18 60.96 180) (unit 1) (body_style 1) (exclude_from_sim no) (in_bom yes) (on_board yes) (dnp no)
-  (property "Reference" "D5301" (at 170.18 54.61 0) (effects (font (size 1.27 1.27)) (justify left)))
+  (property "Reference" "D5401" (at 170.18 54.61 0) (effects (font (size 1.27 1.27)) (justify left)))
   (property "Value" "PMEG6010CEH" (at 170.18 57.15 0) (effects (font (size 1.27 1.27)) (justify left)))
   (property "Footprint" "Diode_SMD:D_SOD-123F" (at 170.18 60.96 0) (effects (font (size 1.27 1.27))) (hide yes))
@@
   (pin "1")
   (pin "2")
-  (instances (project "t1-main-board" (path "/7746052e-d7f9-59ad-ba73-bd2b74439529/d5d538fb-ce80-5e4a-9a88-723f34af818e" (reference "D5301") (unit 1))))
+  (instances (project "t1-main-board" (path "/7746052e-d7f9-59ad-ba73-bd2b74439529/d5d538fb-ce80-5e4a-9a88-723f34af818e" (reference "D5401") (unit 1))))
 )
 (wire (pts (xy 173.99 60.96) (xy 179.07 60.96)) (stroke (width 0) (type default)))
 (wire (pts (xy 166.37 60.96) (xy 161.29 60.96)) (stroke (width 0) (type default)))
 (symbol (lib_id "Device:C") (at 154.94 81.28 0) (unit 1) (body_style 1) (exclude_from_sim no) (in_bom yes) (on_board yes) (dnp no)
-  (property "Reference" "C5303" (at 157.48 80.01 0) (effects (font (size 1.27 1.27)) (justify left)))
+  (property "Reference" "C5403" (at 157.48 80.01 0) (effects (font (size 1.27 1.27)) (justify left)))
   (property "Value" "1 µF" (at 157.48 82.55 0) (effects (font (size 1.27 1.27)) (justify left)))
   (property "Spec" "50 V X7R" (at 157.48 85.09 0) (effects (font (size 1.27 1.27)) (justify left)))
@@
   (pin "1")
   (pin "2")
-  (instances (project "t1-main-board" (path "/7746052e-d7f9-59ad-ba73-bd2b74439529/d5d538fb-ce80-5e4a-9a88-723f34af818e" (reference "C5303") (unit 1))))
+  (instances (project "t1-main-board" (path "/7746052e-d7f9-59ad-ba73-bd2b74439529/d5d538fb-ce80-5e4a-9a88-723f34af818e" (reference "C5403") (unit 1))))
 )
 (wire (pts (xy 154.94 77.47) (xy 154.94 74.93)) (stroke (width 0) (type default)))

Commit message: Board on libs v0.2.0: lower-case kebab vendor keys (HL-13)
The libs submodule moves to v0.2.0 (5f24483). Every library nickname in
the generator, the placement tool and the floorplan study follows the
key table (Texas_Instruments -> texas-instruments, OpenDAP_Device ->
opendap-generic, Rockchip and Rockchip_PMIC -> rockchip, ...); the
library tables are written from the files. Schematic and board
regenerated.

Checks: ERC 0 errors (warnings unchanged); DRC 0 errors, 605 warnings,
the same counts by type, schematic parity 0; every placement identical;
craft Q1 met; pcb tests pass; STEP export resolves every libs 3D model
(the 27 parts without a model are KiCad stock lands that have none).

Co-Authored-By: Claude Opus 5.5 <noreply@anthropic.com>
Claude-Session: https://claude.ai/code/session_01Ei262h3TpgY9vyfNLMi5Mn
Parts:
- U5401: footprint Texas_Instruments:Texas_DRV0006A_WSON-6-1EP_2x2mm_P0.65mm_EP1x1.6mm -> texas-instruments:Texas_DRV0006A_WSON-6-1EP_2x2mm_P0.65mm_EP1x1.6mm; symbol Texas_Instruments:TPS61160DRVR -> texas-instruments:TPS61160DRVR
Changed lines of the file:
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@@
 (paper "A4")
 (title_block (title "Faceplate backlight") (date "2026-10-25") (rev "A") (company "The OpenDAP Project") (comment 1 "blk.fp-backlight") (comment 2 "TPS61160 boost LED driver, 60 mA, open-LED threshold below 30 V"))
-(symbol (lib_id "Texas_Instruments:TPS61160DRVR") (at 45.72 60.96 0) (unit 1) (body_style 1) (exclude_from_sim no) (in_bom yes) (on_board yes) (dnp no)
+(symbol (lib_id "texas-instruments:TPS61160DRVR") (at 45.72 60.96 0) (unit 1) (body_style 1) (exclude_from_sim no) (in_bom yes) (on_board yes) (dnp no)
   (property "Reference" "U5401" (at 46.99 45.72 0) (effects (font (size 1.27 1.27)) (justify left)))
   (property "Value" "TPS61160DRVR" (at 46.99 43.18 0) (effects (font (size 1.27 1.27)) (justify left)))
-  (property "Footprint" "Texas_Instruments:Texas_DRV0006A_WSON-6-1EP_2x2mm_P0.65mm_EP1x1.6mm" (at 45.72 60.96 0) (effects (font (size 1.27 1.27))) (hide yes))
+  (property "Footprint" "texas-instruments:Texas_DRV0006A_WSON-6-1EP_2x2mm_P0.65mm_EP1x1.6mm" (at 45.72 60.96 0) (effects (font (size 1.27 1.27))) (hide yes))
   (property "Datasheet" "https://www.ti.com/lit/ds/symlink/tps61160.pdf" (at 45.72 60.96 0) (effects (font (size 1.27 1.27))) (hide yes))
   (property "Description" "White LED boost driver, 2.7-18 V in, 0.7 A switch, 600 kHz, 200 mV FB, 26 V open-LED protection, PWM and EasyScale dimming, WSON-6 2 x 2 mm (DRV0006A) with exposed pad" (at 45.72 60.96 0) (effects (font (size 1.27 1.27))) (hide yes))
