File: board/hardware/t1-main-board/rp2354-core.kicad_sch (KiCad schematic)
At the start: 20 parts, among them Q3501 DMG1012T, U3501 RP2354A, Y3501 12 MHz

Commit message: Compaction: lower inductors, 0201 decoupling, 0.8 mm signal test pads
A matrix tool (hardware/studies/compaction) checks each candidate against
the design's stresses: same inductance, design peak <= 70 % and the
converter's maximum limit <= 100 % of Isat (30 % drop), height zones,
ratings at least twice the rail, PCB-D-06; sourcing outcome per part.

Applied (placement v1 decision 12, BOM v1.15):
- L601, L4401: XGL4015-102MEC (1.5 mm) for XAL/XGL4020-102MEC (2.1 mm);
- L1001, L5101: XGL4015-471MEC (1.5 mm) for Wurth 744373240047, on the
  stock XxL4020 land (the Wurth land was never drawn);
- L1201 is 1.2 mm (XGL4012, per-MPN heights): it moves next to the SoC;
- 58 x 100 nF decoupling on rails <= 3.3 V in core/IO/radio: 0201;
- 51 test pads on signal nets: 0.8 mm (PCB-D-06 v0.16, JLCPCB guide).
Kept: L901, L2802 (XGL4015 at 103 % of Isat at the limit); no thinner
0805/1206 capacitor passes (obsolete, NRND or unlisted).

Board need 113 % -> 111 % (core band 227 -> 203 %, power band 258 ->
233 %, radio band 19 -> 0 %); only C904 still relies on PCB-Z-04.
ERC 0 errors, craft Q1 met, DRC 0 errors (605 warnings), pcb and study
tests pass, rules test board PASS.

Co-Authored-By: Claude Opus 5.5 <noreply@anthropic.com>
Claude-Session: https://claude.ai/code/session_01Ei262h3TpgY9vyfNLMi5Mn
Parts:
- C3501: footprint Capacitor_SMD:C_0402_1005Metric -> Capacitor_SMD:C_0201_0603Metric; MPN GRM155R71C104KA88D -> GRM033R61A104KE15D
- TP3501, TP3502, TP3503, TP3504, TP3505: footprint TestPoint:TestPoint_Pad_D1.0mm -> T1_Main_Board:TestPoint_Pad_D0.8mm
Changed lines of the file:
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@@
   (property "Reference" "C3501" (at 323.85 64.77 0) (effects (font (size 1.27 1.27)) (justify left)))
   (property "Value" "100 nF" (at 323.85 67.31 0) (effects (font (size 1.27 1.27)) (justify left)))
-  (property "Footprint" "Capacitor_SMD:C_0402_1005Metric" (at 321.31 66.04 0) (effects (font (size 1.27 1.27))) (hide yes))
-  (property "Datasheet" "https://www.murata.com/en-us/products/productdetail?partno=GRM155R71C104KA88D" (at 321.31 66.04 0) (effects (font (size 1.27 1.27))) (hide yes))
-  (property "Description" "Capacitor, 100 nF, 16 V, X7R, 0402" (at 321.31 66.04 0) (effects (font (size 1.27 1.27))) (hide yes))
+  (property "Footprint" "Capacitor_SMD:C_0201_0603Metric" (at 321.31 66.04 0) (effects (font (size 1.27 1.27))) (hide yes))
+  (property "Datasheet" "https://www.murata.com/en-us/products/productdetail?partno=GRM033R61A104KE15D" (at 321.31 66.04 0) (effects (font (size 1.27 1.27))) (hide yes))
+  (property "Description" "Capacitor, 100 nF, 10 V, X5R, 0201" (at 321.31 66.04 0) (effects (font (size 1.27 1.27))) (hide yes))
   (property "Manufacturer" "Murata" (at 321.31 66.04 0) (effects (font (size 1.27 1.27))) (hide yes))
-  (property "MPN" "GRM155R71C104KA88D" (at 321.31 66.04 0) (effects (font (size 1.27 1.27))) (hide yes))
+  (property "MPN" "GRM033R61A104KE15D" (at 321.31 66.04 0) (effects (font (size 1.27 1.27))) (hide yes))
   (property "Block" "blk.rp2354-core" (at 321.31 66.04 0) (effects (font (size 1.27 1.27))) (hide yes))
   (pin "1")
@@
   (property "Reference" "TP3501" (at 280.67 97.79 0) (effects (font (size 1.27 1.27)) (justify right)))
   (property "Value" "RP_SWCLK" (at 280.67 100.33 0) (effects (font (size 1.27 1.27)) (justify right)))
-  (property "Footprint" "TestPoint:TestPoint_Pad_D1.0mm" (at 281.94 102.87 0) (effects (font (size 1.27 1.27))) (hide yes))
+  (property "Footprint" "T1_Main_Board:TestPoint_Pad_D0.8mm" (at 281.94 102.87 0) (effects (font (size 1.27 1.27))) (hide yes))
   (property "Datasheet" "~" (at 281.94 102.87 0) (effects (font (size 1.27 1.27))) (hide yes))
-  (property "Description" "Test pad, 1.0 mm" (at 281.94 102.87 0) (effects (font (size 1.27 1.27))) (hide yes))
+  (property "Description" "Test pad, 0.8 mm, signal net" (at 281.94 102.87 0) (effects (font (size 1.27 1.27))) (hide yes))
   (property "Block" "blk.rp2354-core" (at 281.94 102.87 0) (effects (font (size 1.27 1.27))) (hide yes))
   (pin "1")
@@
   (property "Reference" "TP3502" (at 298.45 97.79 0) (effects (font (size 1.27 1.27)) (justify right)))
   (property "Value" "RP_SWDIO" (at 298.45 100.33 0) (effects (font (size 1.27 1.27)) (justify right)))
-  (property "Footprint" "TestPoint:TestPoint_Pad_D1.0mm" (at 299.72 102.87 0) (effects (font (size 1.27 1.27))) (hide yes))
+  (property "Footprint" "T1_Main_Board:TestPoint_Pad_D0.8mm" (at 299.72 102.87 0) (effects (font (size 1.27 1.27))) (hide yes))
   (property "Datasheet" "~" (at 299.72 102.87 0) (effects (font (size 1.27 1.27))) (hide yes))
-  (property "Description" "Test pad, 1.0 mm" (at 299.72 102.87 0) (effects (font (size 1.27 1.27))) (hide yes))
+  (property "Description" "Test pad, 0.8 mm, signal net" (at 299.72 102.87 0) (effects (font (size 1.27 1.27))) (hide yes))
   (property "Block" "blk.rp2354-core" (at 299.72 102.87 0) (effects (font (size 1.27 1.27))) (hide yes))
   (pin "1")
@@
   (property "Reference" "TP3503" (at 316.23 97.79 0) (effects (font (size 1.27 1.27)) (justify right)))
   (property "Value" "RP_RUN" (at 316.23 100.33 0) (effects (font (size 1.27 1.27)) (justify right)))
-  (property "Footprint" "TestPoint:TestPoint_Pad_D1.0mm" (at 317.5 102.87 0) (effects (font (size 1.27 1.27))) (hide yes))
+  (property "Footprint" "T1_Main_Board:TestPoint_Pad_D0.8mm" (at 317.5 102.87 0) (effects (font (size 1.27 1.27))) (hide yes))
   (property "Datasheet" "~" (at 317.5 102.87 0) (effects (font (size 1.27 1.27))) (hide yes))
-  (property "Description" "Test pad, 1.0 mm" (at 317.5 102.87 0) (effects (font (size 1.27 1.27))) (hide yes))
+  (property "Description" "Test pad, 0.8 mm, signal net" (at 317.5 102.87 0) (effects (font (size 1.27 1.27))) (hide yes))
   (property "Block" "blk.rp2354-core" (at 317.5 102.87 0) (effects (font (size 1.27 1.27))) (hide yes))
   (pin "1")
@@
   (property "Reference" "TP3504" (at 334.01 97.79 0) (effects (font (size 1.27 1.27)) (justify right)))
   (property "Value" "RP_QSPI_SS" (at 334.01 100.33 0) (effects (font (size 1.27 1.27)) (justify right)))
-  (property "Footprint" "TestPoint:TestPoint_Pad_D1.0mm" (at 335.28 102.87 0) (effects (font (size 1.27 1.27))) (hide yes))
+  (property "Footprint" "T1_Main_Board:TestPoint_Pad_D0.8mm" (at 335.28 102.87 0) (effects (font (size 1.27 1.27))) (hide yes))
   (property "Datasheet" "~" (at 335.28 102.87 0) (effects (font (size 1.27 1.27))) (hide yes))
-  (property "Description" "Test pad, 1.0 mm" (at 335.28 102.87 0) (effects (font (size 1.27 1.27))) (hide yes))
+  (property "Description" "Test pad, 0.8 mm, signal net" (at 335.28 102.87 0) (effects (font (size 1.27 1.27))) (hide yes))
   (property "Block" "blk.rp2354-core" (at 335.28 102.87 0) (effects (font (size 1.27 1.27))) (hide yes))
   (pin "1")
@@
   (property "Reference" "TP3505" (at 351.79 97.79 0) (effects (font (size 1.27 1.27)) (justify right)))
   (property "Value" "RP_SPARE" (at 351.79 100.33 0) (effects (font (size 1.27 1.27)) (justify right)))
-  (property "Footprint" "TestPoint:TestPoint_Pad_D1.0mm" (at 353.06 102.87 0) (effects (font (size 1.27 1.27))) (hide yes))
+  (property "Footprint" "T1_Main_Board:TestPoint_Pad_D0.8mm" (at 353.06 102.87 0) (effects (font (size 1.27 1.27))) (hide yes))
   (property "Datasheet" "~" (at 353.06 102.87 0) (effects (font (size 1.27 1.27))) (hide yes))
-  (property "Description" "Test pad, 1.0 mm" (at 353.06 102.87 0) (effects (font (size 1.27 1.27))) (hide yes))
+  (property "Description" "Test pad, 0.8 mm, signal net" (at 353.06 102.87 0) (effects (font (size 1.27 1.27))) (hide yes))
   (property "Block" "blk.rp2354-core" (at 353.06 102.87 0) (effects (font (size 1.27 1.27))) (hide yes))
   (pin "1")

Commit message: Board on libs v0.2.0: lower-case kebab vendor keys (HL-13)
The libs submodule moves to v0.2.0 (5f24483). Every library nickname in
the generator, the placement tool and the floorplan study follows the
key table (Texas_Instruments -> texas-instruments, OpenDAP_Device ->
opendap-generic, Rockchip and Rockchip_PMIC -> rockchip, ...); the
library tables are written from the files. Schematic and board
regenerated.

Checks: ERC 0 errors (warnings unchanged); DRC 0 errors, 605 warnings,
the same counts by type, schematic parity 0; every placement identical;
craft Q1 met; pcb tests pass; STEP export resolves every libs 3D model
(the 27 parts without a model are KiCad stock lands that have none).

Co-Authored-By: Claude Opus 5.5 <noreply@anthropic.com>
Claude-Session: https://claude.ai/code/session_01Ei262h3TpgY9vyfNLMi5Mn
Parts:
- U3501: footprint Raspberry_Pi:QFN-60-1EP_7x7mm_P0.4mm_EP3.4x3.4mm_ThermalVias -> raspberry-pi:QFN-60-1EP_7x7mm_P0.4mm_EP3.4x3.4mm_ThermalVias; symbol Raspberry_Pi:RP2354A -> raspberry-pi:RP2354A
- Y3501: footprint ECS:Oscillator_SMD_ECS_ECS-2016MV-4Pin_2.0x1.6mm -> ecs:Oscillator_SMD_ECS_ECS-2016MV-4Pin_2.0x1.6mm; symbol ECS:ECS-2016MV-120-BN-TR -> ecs:ECS-2016MV-120-BN-TR
Changed lines of the file:
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@@
 (paper "A3")
 (title_block (title "Coprocessor: RP2354A") (date "2026-10-25") (rev "A") (company "The OpenDAP Project") (comment 1 "blk.rp2354-core") (comment 2 "System and GPIO units, 12 MHz oscillator, BOOTSEL, USB series, I2S taps, test pads"))
-(symbol (lib_id "Raspberry_Pi:RP2354A") (at 54.61 72.39 0) (unit 1) (body_style 1) (exclude_from_sim no) (in_bom yes) (on_board yes) (dnp no)
+(symbol (lib_id "raspberry-pi:RP2354A") (at 54.61 72.39 0) (unit 1) (body_style 1) (exclude_from_sim no) (in_bom yes) (on_board yes) (dnp no)
   (property "Reference" "U3501" (at 45.72 43.18 0) (effects (font (size 1.27 1.27)) (justify left)))
   (property "Value" "RP2354A" (at 45.72 40.64 0) (effects (font (size 1.27 1.27)) (justify left)))
-  (property "Footprint" "Raspberry_Pi:QFN-60-1EP_7x7mm_P0.4mm_EP3.4x3.4mm_ThermalVias" (at 54.61 72.39 0) (effects (font (size 1.27 1.27))) (hide yes))
+  (property "Footprint" "raspberry-pi:QFN-60-1EP_7x7mm_P0.4mm_EP3.4x3.4mm_ThermalVias" (at 54.61 72.39 0) (effects (font (size 1.27 1.27))) (hide yes))
   (property "Datasheet" "https://datasheets.raspberrypi.com/rp2350/rp2350-datasheet.pdf" (at 54.61 72.39 0) (effects (font (size 1.27 1.27))) (hide yes))
   (property "Description" "RP2350 microcontroller with 2 MB of QSPI flash stacked in the package, 30 GPIOs, QFN-60 7 x 7 mm, 0.4 mm pitch, exposed GND pad" (at 54.61 72.39 0) (effects (font (size 1.27 1.27))) (hide yes))
@@
 (rectangle (start 22.86 35.56) (end 167.64 105.41) (stroke (width 0) (type dash)) (fill (type none)))
 (text "RP2354A system: RUN, SWD, clock, BOOTSEL, USB (BOM v1 line 12)" (exclude_from_sim no) (at 24.13 34.29 0) (effects (font (size 2.54 2.54)) (justify left bottom)))
-(symbol (lib_id "Raspberry_Pi:RP2354A") (at 186.69 92.71 0) (unit 2) (body_style 1) (exclude_from_sim no) (in_bom yes) (on_board yes) (dnp no)
+(symbol (lib_id "raspberry-pi:RP2354A") (at 186.69 92.71 0) (unit 2) (body_style 1) (exclude_from_sim no) (in_bom yes) (on_board yes) (dnp no)
   (property "Reference" "U3501" (at 175.26 43.18 0) (effects (font (size 1.27 1.27)) (justify left)))
   (property "Value" "RP2354A" (at 175.26 40.64 0) (effects (font (size 1.27 1.27)) (justify left)))
-  (property "Footprint" "Raspberry_Pi:QFN-60-1EP_7x7mm_P0.4mm_EP3.4x3.4mm_ThermalVias" (at 186.69 92.71 0) (effects (font (size 1.27 1.27))) (hide yes))
+  (property "Footprint" "raspberry-pi:QFN-60-1EP_7x7mm_P0.4mm_EP3.4x3.4mm_ThermalVias" (at 186.69 92.71 0) (effects (font (size 1.27 1.27))) (hide yes))
   (property "Datasheet" "https://datasheets.raspberrypi.com/rp2350/rp2350-datasheet.pdf" (at 186.69 92.71 0) (effects (font (size 1.27 1.27))) (hide yes))
   (property "Description" "RP2350 microcontroller with 2 MB of QSPI flash stacked in the package, 30 GPIOs, QFN-60 7 x 7 mm, 0.4 mm pitch, exposed GND pad" (at 186.69 92.71 0) (effects (font (size 1.27 1.27))) (hide yes))
@@
 (rectangle (start 172.72 35.56) (end 262.89 142.24) (stroke (width 0) (type dash)) (fill (type none)))
 (text "RP2354A GPIO (pinout v1 §3 allocation)" (exclude_from_sim no) (at 173.99 34.29 0) (effects (font (size 2.54 2.54)) (justify left bottom)))
-(symbol (lib_id "ECS:ECS-2016MV-120-BN-TR") (at 283.21 58.42 0) (unit 1) (body_style 1) (exclude_from_sim no) (in_bom yes) (on_board yes) (dnp no)
+(symbol (lib_id "ecs:ECS-2016MV-120-BN-TR") (at 283.21 58.42 0) (unit 1) (body_style 1) (exclude_from_sim no) (in_bom yes) (on_board yes) (dnp no)
   (property "Reference" "Y3501" (at 284.48 45.72 0) (effects (font (size 1.27 1.27)) (justify left)))
   (property "Value" "12 MHz" (at 284.48 43.18 0) (effects (font (size 1.27 1.27)) (justify left)))
-  (property "Footprint" "ECS:Oscillator_SMD_ECS_ECS-2016MV-4Pin_2.0x1.6mm" (at 283.21 58.42 0) (effects (font (size 1.27 1.27))) (hide yes))
+  (property "Footprint" "ecs:Oscillator_SMD_ECS_ECS-2016MV-4Pin_2.0x1.6mm" (at 283.21 58.42 0) (effects (font (size 1.27 1.27))) (hide yes))
   (property "Datasheet" "https://ecsxtal.com/store/pdf/ECS-2016MV.pdf" (at 283.21 58.42 0) (effects (font (size 1.27 1.27))) (hide yes))
   (property "Description" "12.000 MHz HCMOS crystal oscillator, ECS-2016MV MultiVolt (1.6-3.6 V), +/-50 ppm, -40 to +85 C, tri-state, 2.0 x 1.6 mm, 4 pads" (at 283.21 58.42 0) (effects (font (size 1.27 1.27))) (hide yes))
