File: board/hardware/t1-main-board/soc-ddr.kicad_sch (KiCad schematic)
At the start: 2 parts, among them U1301 RK3566

Commit message: Board on libs v0.2.0: lower-case kebab vendor keys (HL-13)
The libs submodule moves to v0.2.0 (5f24483). Every library nickname in
the generator, the placement tool and the floorplan study follows the
key table (Texas_Instruments -> texas-instruments, OpenDAP_Device ->
opendap-generic, Rockchip and Rockchip_PMIC -> rockchip, ...); the
library tables are written from the files. Schematic and board
regenerated.

Checks: ERC 0 errors (warnings unchanged); DRC 0 errors, 605 warnings,
the same counts by type, schematic parity 0; every placement identical;
craft Q1 met; pcb tests pass; STEP export resolves every libs 3D model
(the 27 parts without a model are KiCad stock lands that have none).

Co-Authored-By: Claude Opus 5.5 <noreply@anthropic.com>
Claude-Session: https://claude.ai/code/session_01Ei262h3TpgY9vyfNLMi5Mn
Parts:
- U1301: footprint Rockchip:Rockchip_FCCSP-565L_15.5x14.4mm_P0.4mm_P0.65mm_Ball0.25mm_Pad0.25mm_NSMD -> rockchip:Rockchip_FCCSP-565L_15.5x14.4mm_P0.4mm_P0.65mm_Ball0.25mm_Pad0.25mm_NSMD; symbol Rockchip:RK3566 -> rockchip:RK3566
Changed lines of the file:
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@@
 (paper "A3")
 (title_block (title "SoC: LPDDR4X interface") (date "2026-10-25") (rev "A") (company "The OpenDAP Project") (comment 1 "blk.soc-ddr") (comment 2 "RK3566 DDR PHY units: channels A and B, reset and ZQ calibration"))
-(symbol (lib_id "Rockchip:RK3566") (at 120.65 69.85 0) (unit 1) (body_style 1) (exclude_from_sim no) (in_bom yes) (on_board yes) (dnp no)
+(symbol (lib_id "rockchip:RK3566") (at 120.65 69.85 0) (unit 1) (body_style 1) (exclude_from_sim no) (in_bom yes) (on_board yes) (dnp no)
   (property "Reference" "U1301" (at 48.26 35.56 0) (effects (font (size 1.27 1.27)) (justify left)))
   (property "Value" "RK3566" (at 48.26 33.02 0) (effects (font (size 1.27 1.27)) (justify left)))
-  (property "Footprint" "Rockchip:Rockchip_FCCSP-565L_15.5x14.4mm_P0.4mm_P0.65mm_Ball0.25mm_Pad0.25mm_NSMD" (at 120.65 69.85 0) (effects (font (size 1.27 1.27))) (hide yes))
+  (property "Footprint" "rockchip:Rockchip_FCCSP-565L_15.5x14.4mm_P0.4mm_P0.65mm_Ball0.25mm_Pad0.25mm_NSMD" (at 120.65 69.85 0) (effects (font (size 1.27 1.27))) (hide yes))
   (property "Datasheet" "https://dl.xkwy2018.com/downloads/RK3568/Rockchip-RK3566-Datasheet-V1.1-20210305.pdf" (at 120.65 69.85 0) (effects (font (size 1.27 1.27))) (hide yes))
   (property "Description" "Quad-core Arm Cortex-A55 application processor, LPDDR4X/DDR4 32-bit, eMMC 5.1, FCCSP565L 15.5 x 14.4 mm" (at 120.65 69.85 0) (effects (font (size 1.27 1.27))) (hide yes))
@@
 (wire (pts (xy 199.39 72.39) (xy 201.93 72.39)) (stroke (width 0) (type default)))
 (no_connect (at 199.39 74.93))
-(symbol (lib_id "Rockchip:RK3566") (at 120.65 148.59 0) (unit 2) (body_style 1) (exclude_from_sim no) (in_bom yes) (on_board yes) (dnp no)
+(symbol (lib_id "rockchip:RK3566") (at 120.65 148.59 0) (unit 2) (body_style 1) (exclude_from_sim no) (in_bom yes) (on_board yes) (dnp no)
   (property "Reference" "U1301" (at 48.26 114.3 0) (effects (font (size 1.27 1.27)) (justify left)))
   (property "Value" "RK3566" (at 48.26 111.76 0) (effects (font (size 1.27 1.27)) (justify left)))
-  (property "Footprint" "Rockchip:Rockchip_FCCSP-565L_15.5x14.4mm_P0.4mm_P0.65mm_Ball0.25mm_Pad0.25mm_NSMD" (at 120.65 148.59 0) (effects (font (size 1.27 1.27))) (hide yes))
+  (property "Footprint" "rockchip:Rockchip_FCCSP-565L_15.5x14.4mm_P0.4mm_P0.65mm_Ball0.25mm_Pad0.25mm_NSMD" (at 120.65 148.59 0) (effects (font (size 1.27 1.27))) (hide yes))
   (property "Datasheet" "https://dl.xkwy2018.com/downloads/RK3568/Rockchip-RK3566-Datasheet-V1.1-20210305.pdf" (at 120.65 148.59 0) (effects (font (size 1.27 1.27))) (hide yes))
   (property "Description" "Quad-core Arm Cortex-A55 application processor, LPDDR4X/DDR4 32-bit, eMMC 5.1, FCCSP565L 15.5 x 14.4 mm" (at 120.65 148.59 0) (effects (font (size 1.27 1.27))) (hide yes))
@@
 (no_connect (at 199.39 151.13))
 (wire (pts (xy 199.39 153.67) (xy 201.93 153.67)) (stroke (width 0) (type default)))
-(symbol (lib_id "Rockchip:RK3566") (at 255.27 125.73 0) (unit 3) (body_style 1) (exclude_from_sim no) (in_bom yes) (on_board yes) (dnp no)
+(symbol (lib_id "rockchip:RK3566") (at 255.27 125.73 0) (unit 3) (body_style 1) (exclude_from_sim no) (in_bom yes) (on_board yes) (dnp no)
   (property "Reference" "U1301" (at 226.06 114.3 0) (effects (font (size 1.27 1.27)) (justify left)))
   (property "Value" "RK3566" (at 226.06 111.76 0) (effects (font (size 1.27 1.27)) (justify left)))
-  (property "Footprint" "Rockchip:Rockchip_FCCSP-565L_15.5x14.4mm_P0.4mm_P0.65mm_Ball0.25mm_Pad0.25mm_NSMD" (at 255.27 125.73 0) (effects (font (size 1.27 1.27))) (hide yes))
+  (property "Footprint" "rockchip:Rockchip_FCCSP-565L_15.5x14.4mm_P0.4mm_P0.65mm_Ball0.25mm_Pad0.25mm_NSMD" (at 255.27 125.73 0) (effects (font (size 1.27 1.27))) (hide yes))
   (property "Datasheet" "https://dl.xkwy2018.com/downloads/RK3568/Rockchip-RK3566-Datasheet-V1.1-20210305.pdf" (at 255.27 125.73 0) (effects (font (size 1.27 1.27))) (hide yes))
   (property "Description" "Quad-core Arm Cortex-A55 application processor, LPDDR4X/DDR4 32-bit, eMMC 5.1, FCCSP565L 15.5 x 14.4 mm" (at 255.27 125.73 0) (effects (font (size 1.27 1.27))) (hide yes))

Commit message: Board in the 62.5 x 95.0 mm body: ADR 0025, outline 59.1 x 91.6, 0201 swaps
ADR 0025 supersedes ADR 0016 for t1 ADR 0006's body: board outline from
the body, 1.2 mm walls and 0.5 mm clearance; height zones and stack
restated unchanged; the speaker on a case shelf (PCB-Z-09); pocket
reliefs at the 4.4 mm jack, the microSD (DM3AT push-push kept) and the
side buttons; the audio 0603 -> 0402 swap gated by t1 V2-A08; reserve
(NFC reader, then TPM) recorded, not applied.

- pcb/geometry.py derives the outline from BODY, WALL and CLEARANCE;
  the pocket, display and fixed parts keep their device-frame positions;
  holes keep their edge distance; the speaker shadow becomes a 1.5 mm
  shelf height area (placement, checks, occupancy).
- build.py reports pocket reliefs and routing room; C904 unfixed (it
  now finds back room, so PCB-Z-04 carries no part).
- Generator: parts.area_swap puts 121 generic 0402 resistors (outside
  audio and VBUS paths, >= 10 ohm) and five 100 nF signal capacitors in
  0201 (BOM v1.16); schematic and board regenerated.
- Result: 1,012/1,012 placed, 98.8 % by the floorplan method (was 111 %),
  factor left 1.68 (was 1.49); DRC 0 errors, ERC 0 errors, 0 check
  findings, pcb tests 20/20, schematic craft Q1 met.
- Specs: PCB constraints v0.17 (M-01, M-02, M-08, Z-02, Z-06 to Z-09,
  R-07), placement v1.1 (section 3, decisions 4 and 13, checks, open
  items with the gated swaps and the reserve), floorplan v1 section 1,
  BOM v1.16.

Co-Authored-By: Claude Opus 5.5 <noreply@anthropic.com>
Claude-Session: https://claude.ai/code/session_01Ei262h3TpgY9vyfNLMi5Mn
Parts:
- R1320: footprint Resistor_SMD:R_0402_1005Metric -> Resistor_SMD:R_0201_0603Metric; MPN RC0402FR-07120RL -> RC0201FR-07120RL
Changed lines of the file:
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@@
   (property "Reference" "R1320" (at 46.99 199.39 0) (effects (font (size 1.27 1.27)) (justify left)))
   (property "Value" "120 Ω" (at 46.99 201.93 0) (effects (font (size 1.27 1.27)) (justify left)))
-  (property "Footprint" "Resistor_SMD:R_0402_1005Metric" (at 45.72 200.66 0) (effects (font (size 1.27 1.27))) (hide yes))
-  (property "Datasheet" "https://yageogroup.com/en/ProductSearch/PartNumberSearch?part=RC0402FR-07120RL" (at 45.72 200.66 0) (effects (font (size 1.27 1.27))) (hide yes))
-  (property "Description" "Resistor, 120 Ω, 1 %, 1/16 W, 0402" (at 45.72 200.66 0) (effects (font (size 1.27 1.27))) (hide yes))
+  (property "Footprint" "Resistor_SMD:R_0201_0603Metric" (at 45.72 200.66 0) (effects (font (size 1.27 1.27))) (hide yes))
+  (property "Datasheet" "https://yageogroup.com/en/ProductSearch/PartNumberSearch?part=RC0201FR-07120RL" (at 45.72 200.66 0) (effects (font (size 1.27 1.27))) (hide yes))
+  (property "Description" "Resistor, 120 Ω, 1 %, 1/20 W, 0201" (at 45.72 200.66 0) (effects (font (size 1.27 1.27))) (hide yes))
   (property "Manufacturer" "YAGEO" (at 45.72 200.66 0) (effects (font (size 1.27 1.27))) (hide yes))
-  (property "MPN" "RC0402FR-07120RL" (at 45.72 200.66 0) (effects (font (size 1.27 1.27))) (hide yes))
+  (property "MPN" "RC0201FR-07120RL" (at 45.72 200.66 0) (effects (font (size 1.27 1.27))) (hide yes))
   (property "Block" "blk.soc-ddr" (at 45.72 200.66 0) (effects (font (size 1.27 1.27))) (hide yes))
   (pin "1")
