File: board/hardware/t1-main-board/soc-pmuio.kicad_sch (KiCad schematic)
At the start: 28 parts, among them U1301 RK3566, Y1301 24 MHz

Commit message: Board on libs v0.2.0: lower-case kebab vendor keys (HL-13)
The libs submodule moves to v0.2.0 (5f24483). Every library nickname in
the generator, the placement tool and the floorplan study follows the
key table (Texas_Instruments -> texas-instruments, OpenDAP_Device ->
opendap-generic, Rockchip and Rockchip_PMIC -> rockchip, ...); the
library tables are written from the files. Schematic and board
regenerated.

Checks: ERC 0 errors (warnings unchanged); DRC 0 errors, 605 warnings,
the same counts by type, schematic parity 0; every placement identical;
craft Q1 met; pcb tests pass; STEP export resolves every libs 3D model
(the 27 parts without a model are KiCad stock lands that have none).

Co-Authored-By: Claude Opus 5.5 <noreply@anthropic.com>
Claude-Session: https://claude.ai/code/session_01Ei262h3TpgY9vyfNLMi5Mn
Parts:
- U1301: footprint Rockchip:Rockchip_FCCSP-565L_15.5x14.4mm_P0.4mm_P0.65mm_Ball0.25mm_Pad0.25mm_NSMD -> rockchip:Rockchip_FCCSP-565L_15.5x14.4mm_P0.4mm_P0.65mm_Ball0.25mm_Pad0.25mm_NSMD; symbol Rockchip:RK3566 -> rockchip:RK3566
- Y1301: symbol OpenDAP_Device:Crystal_GND24 -> opendap-generic:Crystal_GND24
Changed lines of the file:
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@@
 (paper "A3")
 (title_block (title "SoC: PMU IO domains, clock, reset and SARADC") (date "2026-10-25") (rev "A") (company "The OpenDAP Project") (comment 1 "blk.soc-pmuio") (comment 2 "RK3566 units on PMUIO0-2 and the SARADC, with the 24 MHz crystal, reset, straps and bus pull-ups"))
-(symbol (lib_id "Rockchip:RK3566") (at 92.71 59.69 0) (unit 4) (body_style 1) (exclude_from_sim no) (in_bom yes) (on_board yes) (dnp no)
+(symbol (lib_id "rockchip:RK3566") (at 92.71 59.69 0) (unit 4) (body_style 1) (exclude_from_sim no) (in_bom yes) (on_board yes) (dnp no)
   (property "Reference" "U1301" (at 50.8 35.56 0) (effects (font (size 1.27 1.27)) (justify left)))
   (property "Value" "RK3566" (at 50.8 33.02 0) (effects (font (size 1.27 1.27)) (justify left)))
-  (property "Footprint" "Rockchip:Rockchip_FCCSP-565L_15.5x14.4mm_P0.4mm_P0.65mm_Ball0.25mm_Pad0.25mm_NSMD" (at 92.71 59.69 0) (effects (font (size 1.27 1.27))) (hide yes))
+  (property "Footprint" "rockchip:Rockchip_FCCSP-565L_15.5x14.4mm_P0.4mm_P0.65mm_Ball0.25mm_Pad0.25mm_NSMD" (at 92.71 59.69 0) (effects (font (size 1.27 1.27))) (hide yes))
   (property "Datasheet" "https://dl.xkwy2018.com/downloads/RK3568/Rockchip-RK3566-Datasheet-V1.1-20210305.pdf" (at 92.71 59.69 0) (effects (font (size 1.27 1.27))) (hide yes))
   (property "Description" "Quad-core Arm Cortex-A55 application processor, LPDDR4X/DDR4 32-bit, eMMC 5.1, FCCSP565L 15.5 x 14.4 mm" (at 92.71 59.69 0) (effects (font (size 1.27 1.27))) (hide yes))
@@
 (wire (pts (xy 44.45 74.93) (xy 41.91 74.93)) (stroke (width 0) (type default)))
 (wire (pts (xy 140.97 41.91) (xy 143.51 41.91)) (stroke (width 0) (type default)))
-(symbol (lib_id "Rockchip:RK3566") (at 223.52 64.77 0) (unit 5) (body_style 1) (exclude_from_sim no) (in_bom yes) (on_board yes) (dnp no)
+(symbol (lib_id "rockchip:RK3566") (at 223.52 64.77 0) (unit 5) (body_style 1) (exclude_from_sim no) (in_bom yes) (on_board yes) (dnp no)
   (property "Reference" "U1301" (at 184.15 35.56 0) (effects (font (size 1.27 1.27)) (justify left)))
   (property "Value" "RK3566" (at 184.15 33.02 0) (effects (font (size 1.27 1.27)) (justify left)))
-  (property "Footprint" "Rockchip:Rockchip_FCCSP-565L_15.5x14.4mm_P0.4mm_P0.65mm_Ball0.25mm_Pad0.25mm_NSMD" (at 223.52 64.77 0) (effects (font (size 1.27 1.27))) (hide yes))
+  (property "Footprint" "rockchip:Rockchip_FCCSP-565L_15.5x14.4mm_P0.4mm_P0.65mm_Ball0.25mm_Pad0.25mm_NSMD" (at 223.52 64.77 0) (effects (font (size 1.27 1.27))) (hide yes))
   (property "Datasheet" "https://dl.xkwy2018.com/downloads/RK3568/Rockchip-RK3566-Datasheet-V1.1-20210305.pdf" (at 223.52 64.77 0) (effects (font (size 1.27 1.27))) (hide yes))
   (property "Description" "Quad-core Arm Cortex-A55 application processor, LPDDR4X/DDR4 32-bit, eMMC 5.1, FCCSP565L 15.5 x 14.4 mm" (at 223.52 64.77 0) (effects (font (size 1.27 1.27))) (hide yes))
@@
 (wire (pts (xy 177.8 82.55) (xy 175.26 82.55)) (stroke (width 0) (type default)))
 (wire (pts (xy 177.8 85.09) (xy 175.26 85.09)) (stroke (width 0) (type default)))
-(symbol (lib_id "Rockchip:RK3566") (at 311.15 46.99 0) (unit 19) (body_style 1) (exclude_from_sim no) (in_bom yes) (on_board yes) (dnp no)
+(symbol (lib_id "rockchip:RK3566") (at 311.15 46.99 0) (unit 19) (body_style 1) (exclude_from_sim no) (in_bom yes) (on_board yes) (dnp no)
   (property "Reference" "U1301" (at 299.72 35.56 0) (effects (font (size 1.27 1.27)) (justify left)))
   (property "Value" "RK3566" (at 299.72 33.02 0) (effects (font (size 1.27 1.27)) (justify left)))
-  (property "Footprint" "Rockchip:Rockchip_FCCSP-565L_15.5x14.4mm_P0.4mm_P0.65mm_Ball0.25mm_Pad0.25mm_NSMD" (at 311.15 46.99 0) (effects (font (size 1.27 1.27))) (hide yes))
+  (property "Footprint" "rockchip:Rockchip_FCCSP-565L_15.5x14.4mm_P0.4mm_P0.65mm_Ball0.25mm_Pad0.25mm_NSMD" (at 311.15 46.99 0) (effects (font (size 1.27 1.27))) (hide yes))
   (property "Datasheet" "https://dl.xkwy2018.com/downloads/RK3568/Rockchip-RK3566-Datasheet-V1.1-20210305.pdf" (at 311.15 46.99 0) (effects (font (size 1.27 1.27))) (hide yes))
   (property "Description" "Quad-core Arm Cortex-A55 application processor, LPDDR4X/DDR4 32-bit, eMMC 5.1, FCCSP565L 15.5 x 14.4 mm" (at 311.15 46.99 0) (effects (font (size 1.27 1.27))) (hide yes))
@@
 (rectangle (start 25.4 125.73) (end 129.54 171.45) (stroke (width 0) (type dash)) (fill (type none)))
 (text "24 MHz crystal (HDG 1.1 pp. 16-17)" (exclude_from_sim no) (at 26.67 124.46 0) (effects (font (size 2.54 2.54)) (justify left bottom)))
-(symbol (lib_id "OpenDAP_Device:Crystal_GND24") (at 76.2 148.59 0) (unit 1) (body_style 1) (exclude_from_sim no) (in_bom yes) (on_board yes) (dnp no)
+(symbol (lib_id "opendap-generic:Crystal_GND24") (at 76.2 148.59 0) (unit 1) (body_style 1) (exclude_from_sim no) (in_bom yes) (on_board yes) (dnp no)
   (property "Reference" "Y1301" (at 80.01 143.51 0) (effects (font (size 1.27 1.27)) (justify left)))
   (property "Value" "24 MHz" (at 80.01 154.94 0) (effects (font (size 1.27 1.27)) (justify left)))

Commit message: Board in the 62.5 x 95.0 mm body: ADR 0025, outline 59.1 x 91.6, 0201 swaps
ADR 0025 supersedes ADR 0016 for t1 ADR 0006's body: board outline from
the body, 1.2 mm walls and 0.5 mm clearance; height zones and stack
restated unchanged; the speaker on a case shelf (PCB-Z-09); pocket
reliefs at the 4.4 mm jack, the microSD (DM3AT push-push kept) and the
side buttons; the audio 0603 -> 0402 swap gated by t1 V2-A08; reserve
(NFC reader, then TPM) recorded, not applied.

- pcb/geometry.py derives the outline from BODY, WALL and CLEARANCE;
  the pocket, display and fixed parts keep their device-frame positions;
  holes keep their edge distance; the speaker shadow becomes a 1.5 mm
  shelf height area (placement, checks, occupancy).
- build.py reports pocket reliefs and routing room; C904 unfixed (it
  now finds back room, so PCB-Z-04 carries no part).
- Generator: parts.area_swap puts 121 generic 0402 resistors (outside
  audio and VBUS paths, >= 10 ohm) and five 100 nF signal capacitors in
  0201 (BOM v1.16); schematic and board regenerated.
- Result: 1,012/1,012 placed, 98.8 % by the floorplan method (was 111 %),
  factor left 1.68 (was 1.49); DRC 0 errors, ERC 0 errors, 0 check
  findings, pcb tests 20/20, schematic craft Q1 met.
- Specs: PCB constraints v0.17 (M-01, M-02, M-08, Z-02, Z-06 to Z-09,
  R-07), placement v1.1 (section 3, decisions 4 and 13, checks, open
  items with the gated swaps and the reserve), floorplan v1 section 1,
  BOM v1.16.

Co-Authored-By: Claude Opus 5.5 <noreply@anthropic.com>
Claude-Session: https://claude.ai/code/session_01Ei262h3TpgY9vyfNLMi5Mn
Parts:
- C1303: footprint Capacitor_SMD:C_0402_1005Metric -> Capacitor_SMD:C_0201_0603Metric; MPN GRM155R71C104KA88D -> GRM033R61A104KE15D
- R1301: footprint Resistor_SMD:R_0402_1005Metric -> Resistor_SMD:R_0201_0603Metric; MPN RC0402FR-071ML -> RC0201FR-071ML
- R1302: footprint Resistor_SMD:R_0402_1005Metric -> Resistor_SMD:R_0201_0603Metric; MPN RC0402FR-0722RL -> RC0201FR-0722RL
- R1303, R1304, R1312, R1319: footprint Resistor_SMD:R_0402_1005Metric -> Resistor_SMD:R_0201_0603Metric; MPN RC0402FR-0710KL -> RC0201FR-0710KL
- R1305, R1306, R1307, R1308, R1309, R1310: footprint Resistor_SMD:R_0402_1005Metric -> Resistor_SMD:R_0201_0603Metric; MPN RC0402FR-072K2L -> RC0201FR-072K2L
- R1311, R1313, R1314, R1315, R1316, R1317, R1318: footprint Resistor_SMD:R_0402_1005Metric -> Resistor_SMD:R_0201_0603Metric; MPN RC0402FR-074K7L -> RC0201FR-074K7L

Commit message: NFC reader withdrawn from the board, every model (BRD-057)
Maintainer decision 2026-10-27, reason: board area. blk.nfc-reader (#42)
withdrawn: PN7160, front end, crystal, antenna contacts, NFC_VBAT switch
and link #18 removed (35 parts). BRD-057 reworded: NFC as the dynamic tag
only; blk.nfc-tag stays. Pinout v1: 1N20, A37, B38 become unconnected
spares, expander P05 a spare. BOM v1.18 item 7 (line 50: 5 switches,
lines 127-128 withdrawn), power tree v0.10, variant files, feature blocks.

Sheets after the removed one move up a page; references renumbered in
plan.py, parts.py and the specs (J6201 -> J6101 and others).

Placement v1.4: 990 parts placed, board need 96.9 % (99.1 % before),
factor 1.72; 243 capacitors within bound; DRC 0 errors; ERC 0 errors;
craft Q1 met; overlaps 0; pcb tests pass; STEP exported.

Co-Authored-By: Claude Opus 5.5 <noreply@anthropic.com>
Claude-Session: https://claude.ai/code/session_01Ei262h3TpgY9vyfNLMi5Mn
Connections:
- net NFC_IRQ: no longer names the net of U1301.1N20 (GPIO0_D5_d)
- no-connect marks 0 -> 1
Changed lines of the file:
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@@
 (wire (pts (xy 44.45 46.99) (xy 41.91 46.99)) (stroke (width 0) (type default)))
 (wire (pts (xy 44.45 49.53) (xy 41.91 49.53)) (stroke (width 0) (type default)))
-(wire (pts (xy 44.45 52.07) (xy 41.91 52.07)) (stroke (width 0) (type default)))
+(no_connect (at 44.45 52.07))
 (wire (pts (xy 44.45 54.61) (xy 41.91 54.61)) (stroke (width 0) (type default)))
 (wire (pts (xy 44.45 57.15) (xy 41.91 57.15)) (stroke (width 0) (type default)))
@@
 (label "TPM_RST_N" (at 41.91 46.99 180) (effects (font (size 1.27 1.27)) (justify right bottom)))
 (label "NFC_FD_N" (at 41.91 49.53 180) (effects (font (size 1.27 1.27)) (justify right bottom)))
-(label "NFC_IRQ" (at 41.91 52.07 180) (effects (font (size 1.27 1.27)) (justify right bottom)))
 (label "EXP_INT_N" (at 41.91 54.61 180) (effects (font (size 1.27 1.27)) (justify right bottom)))
 (label "COVER_DET_N" (at 41.91 57.15 180) (effects (font (size 1.27 1.27)) (justify right bottom)))
