File: board/hardware/t1-main-board/audio-supply.kicad_sch (KiCad schematic)
At the start: 15 parts, among them U2301 TPS22919DCKR, U2302 TPS22919DCKR, U2303 TPS62840DLCR

Commit message: Board: capture blk.current-monitors
Five INA236 on I2C1 (0x40-0x43, 0x48) with their shunts, per power tree
§4.12 and BOM v1 lines 54 and 136. The measured branches are rails of
their own (VSYS_SRC, VSYS_LV_AUDIO, VSYS_AUDIO, VSYS_LV_BL, VSYS_P5V1),
fed through the shunts on this sheet; the charger, audio, backlight and
5.1 V sheets take them. The root's layout may leave a stack level empty,
so the block sits under the notes; IC bboxes hold turned rail values;
passive rows hold a bottom rail's text.

Co-Authored-By: Claude Opus 5.5 <noreply@anthropic.com>
Claude-Session: https://claude.ai/code/session_01Ei262h3TpgY9vyfNLMi5Mn
Connections:
- net VSYS_LV renamed VSYS_LV_AUDIO
Other:
- moved on the sheet: C2301, C2302, C2303, C2304, L2301, R2301, R2302, R2303, TP2301, TP2302, TP2303, TP2304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

Commit message: Board on libs v0.2.0: lower-case kebab vendor keys (HL-13)
The libs submodule moves to v0.2.0 (5f24483). Every library nickname in
the generator, the placement tool and the floorplan study follows the
key table (Texas_Instruments -> texas-instruments, OpenDAP_Device ->
opendap-generic, Rockchip and Rockchip_PMIC -> rockchip, ...); the
library tables are written from the files. Schematic and board
regenerated.

Checks: ERC 0 errors (warnings unchanged); DRC 0 errors, 605 warnings,
the same counts by type, schematic parity 0; every placement identical;
craft Q1 met; pcb tests pass; STEP export resolves every libs 3D model
(the 27 parts without a model are KiCad stock lands that have none).

Co-Authored-By: Claude Opus 5.5 <noreply@anthropic.com>
Claude-Session: https://claude.ai/code/session_01Ei262h3TpgY9vyfNLMi5Mn
Parts:
- U2301, U2302: footprint Texas_Instruments:Texas_DCK0006A_SC-70-6_1.25x2mm_P0.65mm -> texas-instruments:Texas_DCK0006A_SC-70-6_1.25x2mm_P0.65mm; symbol Texas_Instruments:TPS22919DCKR -> texas-instruments:TPS22919DCKR
- U2303: footprint Texas_Instruments:Texas_DLC0008B_VSON-HR-8_1.5x2mm_P0.5mm -> texas-instruments:Texas_DLC0008B_VSON-HR-8_1.5x2mm_P0.5mm; symbol Texas_Instruments:TPS62840DLCR -> texas-instruments:TPS62840DLCR
Changed lines of the file:
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@@
 (paper "A3")
 (title_block (title "Audio: DAC supplies") (date "2026-10-25") (rev "A") (company "The OpenDAP Project") (comment 1 "blk.audio-supply") (comment 2 "DAC_VP and DAC_DIG_1V8 load switches and the AUDIO_2V2 pre-buck, with their links"))
-(symbol (lib_id "Texas_Instruments:TPS22919DCKR") (at 55.88 58.42 0) (unit 1) (body_style 1) (exclude_from_sim no) (in_bom yes) (on_board yes) (dnp no)
+(symbol (lib_id "texas-instruments:TPS22919DCKR") (at 55.88 58.42 0) (unit 1) (body_style 1) (exclude_from_sim no) (in_bom yes) (on_board yes) (dnp no)
   (property "Reference" "U2301" (at 48.26 43.18 0) (effects (font (size 1.27 1.27)) (justify left)))
   (property "Value" "TPS22919DCKR" (at 48.26 40.64 0) (effects (font (size 1.27 1.27)) (justify left)))
-  (property "Footprint" "Texas_Instruments:Texas_DCK0006A_SC-70-6_1.25x2mm_P0.65mm" (at 55.88 58.42 0) (effects (font (size 1.27 1.27))) (hide yes))
+  (property "Footprint" "texas-instruments:Texas_DCK0006A_SC-70-6_1.25x2mm_P0.65mm" (at 55.88 58.42 0) (effects (font (size 1.27 1.27))) (hide yes))
   (property "Datasheet" "https://www.ti.com/lit/ds/symlink/tps22919.pdf" (at 55.88 58.42 0) (effects (font (size 1.27 1.27))) (hide yes))
   (property "Description" "Load switch, 1.6-5.5 V, 1.5 A, 90 mOhm, controlled rise time, short-circuit protection, adjustable quick output discharge, SOT/SC-70-6 (DCK0006A)" (at 55.88 58.42 0) (effects (font (size 1.27 1.27))) (hide yes))
@@
 (rectangle (start 22.86 35.56) (end 95.25 85.09) (stroke (width 0) (type dash)) (fill (type none)))
 (text "DAC_VP switch" (exclude_from_sim no) (at 24.13 34.29 0) (effects (font (size 2.54 2.54)) (justify left bottom)))
-(symbol (lib_id "Texas_Instruments:TPS22919DCKR") (at 128.27 58.42 0) (unit 1) (body_style 1) (exclude_from_sim no) (in_bom yes) (on_board yes) (dnp no)
+(symbol (lib_id "texas-instruments:TPS22919DCKR") (at 128.27 58.42 0) (unit 1) (body_style 1) (exclude_from_sim no) (in_bom yes) (on_board yes) (dnp no)
   (property "Reference" "U2302" (at 120.65 43.18 0) (effects (font (size 1.27 1.27)) (justify left)))
   (property "Value" "TPS22919DCKR" (at 120.65 40.64 0) (effects (font (size 1.27 1.27)) (justify left)))
-  (property "Footprint" "Texas_Instruments:Texas_DCK0006A_SC-70-6_1.25x2mm_P0.65mm" (at 128.27 58.42 0) (effects (font (size 1.27 1.27))) (hide yes))
+  (property "Footprint" "texas-instruments:Texas_DCK0006A_SC-70-6_1.25x2mm_P0.65mm" (at 128.27 58.42 0) (effects (font (size 1.27 1.27))) (hide yes))
   (property "Datasheet" "https://www.ti.com/lit/ds/symlink/tps22919.pdf" (at 128.27 58.42 0) (effects (font (size 1.27 1.27))) (hide yes))
   (property "Description" "Load switch, 1.6-5.5 V, 1.5 A, 90 mOhm, controlled rise time, short-circuit protection, adjustable quick output discharge, SOT/SC-70-6 (DCK0006A)" (at 128.27 58.42 0) (effects (font (size 1.27 1.27))) (hide yes))
@@
   (instances (project "t1-main-board" (path "/7746052e-d7f9-59ad-ba73-bd2b74439529/d6f0155c-678f-5298-bf09-6ea7c0e72438/0fd668ea-4b01-5ddb-ae91-3a6690d51f81" (reference "#FLG0017") (unit 1))))
 )
-(symbol (lib_id "Texas_Instruments:TPS62840DLCR") (at 59.69 125.73 0) (unit 1) (body_style 1) (exclude_from_sim no) (in_bom yes) (on_board yes) (dnp no)
+(symbol (lib_id "texas-instruments:TPS62840DLCR") (at 59.69 125.73 0) (unit 1) (body_style 1) (exclude_from_sim no) (in_bom yes) (on_board yes) (dnp no)
   (property "Reference" "U2303" (at 60.96 105.41 0) (effects (font (size 1.27 1.27)) (justify left)))
   (property "Value" "TPS62840DLCR" (at 60.96 102.87 0) (effects (font (size 1.27 1.27)) (justify left)))
-  (property "Footprint" "Texas_Instruments:Texas_DLC0008B_VSON-HR-8_1.5x2mm_P0.5mm" (at 59.69 125.73 0) (effects (font (size 1.27 1.27))) (hide yes))
+  (property "Footprint" "texas-instruments:Texas_DLC0008B_VSON-HR-8_1.5x2mm_P0.5mm" (at 59.69 125.73 0) (effects (font (size 1.27 1.27))) (hide yes))
   (property "Datasheet" "https://www.ti.com/lit/ds/symlink/tps62840.pdf" (at 59.69 125.73 0) (effects (font (size 1.27 1.27))) (hide yes))
   (property "Description" "750 mA step-down converter, 60 nA quiescent current, 1.8-6.5 V input, 1.8-3.3 V output set by one VSET resistor, MODE and STOP pins, output discharge, VSON-HR-8 (DLC0008B) 1.5 x 2 mm" (at 59.69 125.73 0) (effects (font (size 1.27 1.27))) (hide yes))

Commit message: Load switches in TPS22916C WCSP (BOM v1.17 item 3, libs v0.3.1)
The six TPS22919DCKR become the TPS22916CYFPR, the BOM's named second
source, now that kicad-lib v0.3.1 carries its land, symbol and model.
Each position's rise time and output discharge checked against the
data sheet (SLVSDO5F section 6.6): every sequencing rule holds; the
fixed 150 Ohm discharge is slower and the driver's delays follow it.
Power tree v0.9 restates the switch rows.

Co-Authored-By: Claude Opus 5.5 <noreply@anthropic.com>
Claude-Session: https://claude.ai/code/session_01Ei262h3TpgY9vyfNLMi5Mn
Parts:
- U2301, U2302: value TPS22919DCKR -> TPS22916CYFPR; footprint texas-instruments:Texas_DCK0006A_SC-70-6_1.25x2mm_P0.65mm -> texas-instruments:Texas_YFP0004_DSBGA-4_0.78x0.78mm_Layout2x2_P0.4mm; symbol texas-instruments:TPS22919DCKR -> texas-instruments:TPS22916CYFPR; MPN TPS22919DCKR -> TPS22916CYFPR; Second_Source Texas Instruments TPS22916CYFPR (WCSP, other land; BOM v1 l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 -> (none)
Connections:
- net DAC_DIG_1V8_SRC: now also U2302.A1 (VOUT); no longer U2302.5 (QOD), U2302.6 (VOUT)
- net DAC_DIG_EN: now also U2302.B2 (ON); no longer U2302.3 (ON)
- net DAC_VP: now also U2301.A1 (VOUT); no longer U2301.5 (QOD), U2301.6 (VOUT)
- net DAC_VP_EN: now also U2301.B2 (ON); no longer U2301.3 (ON)
- net GND: now also U2301.B1 (GND), U2302.B1 (GND); no longer U2301.2 (GND), U2302.2 (GND)
- net VSYS_LV_AUDIO: now also U2301.A2 (VIN); no longer U2301.1 (IN)
- net vcc_1v8: now also U2302.A2 (VIN); no longer U2302.1 (IN)
- no-connect marks 2 -> 0
Other:
- moved on the sheet: C2301, C2302, C2303, C2304, L2301, R2301, R2302, R2303, TP2301, TP2302, TP2303, TP2304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

Commit message: BOM v1.18 item 2: successors of the discontinued 1 uF 0402
GRM155R61A105KE15D is to be discontinued. 44 positions take
GRM155C71A105KE11D (1 uF 10 V X7S); the eight TPS7A20 positions take
GRM155R61C225KE11D (2.2 uF 16 V X5R) to keep the 0.47 uF effective
minimum with 10 % to spare at up to 3.8 V. Same land; sourcing pass.
Closes BOM §7 item 52; new item 55 lists the other capture parts outside
Murata's product data or near end of life.

Co-Authored-By: Claude Opus 5.5 <noreply@anthropic.com>
Claude-Session: https://claude.ai/code/session_01Ei262h3TpgY9vyfNLMi5Mn
Parts:
- C2301, C2302: MPN GRM155R61A105KE15D -> GRM155C71A105KE11D
