File: board/hardware/t1-main-board/cover-detect.kicad_sch (KiCad schematic)
At the start: 4 parts

Commit message: Board: capture blk.mic-ambient and links #34, #35
IM73D122 on PDM CLK1 and SDI1 (BOM v1 line 34, pinout v1 AK2 and 1P2),
LR to ground, 22 Ω clock series, VDD from MIC_1V8 through link #35.
Link #34 on blk.mic-main makes the faceplate branch the rail MIC_1V8_FP
for contact 40 (power tree §4.12, G10). kicad-lib moves to e46bda4 for
the IM73D122, TPS3808G01, SN74LVC1G58 and BAT54 parts.

Co-Authored-By: Claude Opus 5.5 <noreply@anthropic.com>
Claude-Session: https://claude.ai/code/session_01Ei262h3TpgY9vyfNLMi5Mn
Parts:
- removed D5701: TPD1E10B06, Package_SON:Texas_DPY0002A_0.6x1mm_P0.65mm, symbol Device:D_TVS
- removed R5701: 100 kΩ, Resistor_SMD:R_0402_1005Metric, symbol Device:R
- removed TP5701: COVER, TestPoint:TestPoint_Pad_2.0x2.0mm, symbol Connector:TestPoint
- removed TP5702: COVER_GND, TestPoint:TestPoint_Pad_2.0x2.0mm, symbol Connector:TestPoint
- added D5801: TPD1E10B06, Package_SON:Texas_DPY0002A_0.6x1mm_P0.65mm, symbol Device:D_TVS
- added R5801: 100 kΩ, Resistor_SMD:R_0402_1005Metric, symbol Device:R
- added TP5801: COVER, TestPoint:TestPoint_Pad_2.0x2.0mm, symbol Connector:TestPoint
- added TP5802: COVER_GND, TestPoint:TestPoint_Pad_2.0x2.0mm, symbol Connector:TestPoint
Connections:
- net COVER_DET_N: now also D5801.2 (A2), R5801.2, TP5801.1
- net GND: now also D5801.1 (A1), TP5802.1
- net vcc3v3_pmu: now also R5801.1
Changed lines of the file:
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@@
 (title_block (title "Cover detect") (date "2026-10-25") (rev "A") (company "The OpenDAP Project") (comment 1 "blk.cover-detect") (comment 2 "Back-cover detect input: board-edge contact pads, pull-up, ESD"))
 (symbol (lib_id "Connector:TestPoint") (at 39.37 45.72 0) (unit 1) (body_style 1) (exclude_from_sim no) (in_bom no) (on_board yes) (dnp no)
-  (property "Reference" "TP5701" (at 38.1 40.64 0) (effects (font (size 1.27 1.27)) (justify right)))
+  (property "Reference" "TP5801" (at 38.1 40.64 0) (effects (font (size 1.27 1.27)) (justify right)))
   (property "Value" "COVER" (at 38.1 43.18 0) (effects (font (size 1.27 1.27)) (justify right)))
   (property "Footprint" "TestPoint:TestPoint_Pad_2.0x2.0mm" (at 39.37 45.72 0) (effects (font (size 1.27 1.27))) (hide yes))
@@
   (property "Block" "blk.cover-detect" (at 39.37 45.72 0) (effects (font (size 1.27 1.27))) (hide yes))
   (pin "1")
-  (instances (project "t1-main-board" (path "/7746052e-d7f9-59ad-ba73-bd2b74439529/357cd0ed-ef3a-5696-a4d8-7fa96210e511" (reference "TP5701") (unit 1))))
+  (instances (project "t1-main-board" (path "/7746052e-d7f9-59ad-ba73-bd2b74439529/357cd0ed-ef3a-5696-a4d8-7fa96210e511" (reference "TP5801") (unit 1))))
 )
 (symbol (lib_id "Connector:TestPoint") (at 64.77 45.72 0) (unit 1) (body_style 1) (exclude_from_sim no) (in_bom no) (on_board yes) (dnp no)
-  (property "Reference" "TP5702" (at 63.5 40.64 0) (effects (font (size 1.27 1.27)) (justify right)))
+  (property "Reference" "TP5802" (at 63.5 40.64 0) (effects (font (size 1.27 1.27)) (justify right)))
   (property "Value" "COVER_GND" (at 63.5 43.18 0) (effects (font (size 1.27 1.27)) (justify right)))
   (property "Footprint" "TestPoint:TestPoint_Pad_2.0x2.0mm" (at 64.77 45.72 0) (effects (font (size 1.27 1.27))) (hide yes))
@@
   (property "Block" "blk.cover-detect" (at 64.77 45.72 0) (effects (font (size 1.27 1.27))) (hide yes))
   (pin "1")
-  (instances (project "t1-main-board" (path "/7746052e-d7f9-59ad-ba73-bd2b74439529/357cd0ed-ef3a-5696-a4d8-7fa96210e511" (reference "TP5702") (unit 1))))
+  (instances (project "t1-main-board" (path "/7746052e-d7f9-59ad-ba73-bd2b74439529/357cd0ed-ef3a-5696-a4d8-7fa96210e511" (reference "TP5802") (unit 1))))
 )
 (wire (pts (xy 64.77 45.72) (xy 64.77 48.26)) (stroke (width 0) (type default)))
 (symbol (lib_id "power:GND") (at 64.77 48.26 0) (unit 1) (body_style 1) (exclude_from_sim no) (in_bom yes) (on_board yes) (dnp no)
-  (property "Reference" "#PWR0929" (at 64.77 48.26 0) (effects (font (size 1.27 1.27))) (hide yes))
+  (property "Reference" "#PWR0931" (at 64.77 48.26 0) (effects (font (size 1.27 1.27))) (hide yes))
   (property "Value" "GND" (at 64.77 52.07 0) (effects (font (size 1.27 1.27))))
   (property "Footprint" "" (at 64.77 48.26 0) (effects (font (size 1.27 1.27))) (hide yes))
   (property "Datasheet" "" (at 64.77 48.26 0) (effects (font (size 1.27 1.27))) (hide yes))
   (pin "1")
-  (instances (project "t1-main-board" (path "/7746052e-d7f9-59ad-ba73-bd2b74439529/357cd0ed-ef3a-5696-a4d8-7fa96210e511" (reference "#PWR0929") (unit 1))))
+  (instances (project "t1-main-board" (path "/7746052e-d7f9-59ad-ba73-bd2b74439529/357cd0ed-ef3a-5696-a4d8-7fa96210e511" (reference "#PWR0931") (unit 1))))
 )
 (rectangle (start 22.86 35.56) (end 158.75 63.5) (stroke (width 0) (type dash)) (fill (type none)))
 (text "Contact pads at the board edge (BOM v1 line 143; PCB-L-10)" (exclude_from_sim no) (at 24.13 34.29 0) (effects (font (size 2.54 2.54)) (justify left bottom)))
 (symbol (lib_id "Device:R") (at 175.26 48.26 0) (unit 1) (body_style 1) (exclude_from_sim no) (in_bom yes) (on_board yes) (dnp no)
-  (property "Reference" "R5701" (at 176.53 46.99 0) (effects (font (size 1.27 1.27)) (justify left)))
+  (property "Reference" "R5801" (at 176.53 46.99 0) (effects (font (size 1.27 1.27)) (justify left)))
   (property "Value" "100 kΩ" (at 176.53 49.53 0) (effects (font (size 1.27 1.27)) (justify left)))
   (property "Footprint" "Resistor_SMD:R_0402_1005Metric" (at 175.26 48.26 0) (effects (font (size 1.27 1.27))) (hide yes))
@@
   (pin "1")
   (pin "2")
-  (instances (project "t1-main-board" (path "/7746052e-d7f9-59ad-ba73-bd2b74439529/357cd0ed-ef3a-5696-a4d8-7fa96210e511" (reference "R5701") (unit 1))))
+  (instances (project "t1-main-board" (path "/7746052e-d7f9-59ad-ba73-bd2b74439529/357cd0ed-ef3a-5696-a4d8-7fa96210e511" (reference "R5801") (unit 1))))
 )
 (wire (pts (xy 175.26 44.45) (xy 175.26 41.91)) (stroke (width 0) (type default)))
 (symbol (lib_id "power:VCC") (at 175.26 41.91 0) (unit 1) (body_style 1) (exclude_from_sim no) (in_bom yes) (on_board yes) (dnp no)
-  (property "Reference" "#PWR0930" (at 175.26 41.91 0) (effects (font (size 1.27 1.27))) (hide yes))
+  (property "Reference" "#PWR0932" (at 175.26 41.91 0) (effects (font (size 1.27 1.27))) (hide yes))
   (property "Value" "vcc3v3_pmu" (at 175.26 38.1 0) (effects (font (size 1.27 1.27))))
   (property "Footprint" "" (at 175.26 41.91 0) (effects (font (size 1.27 1.27))) (hide yes))
   (property "Datasheet" "" (at 175.26 41.91 0) (effects (font (size 1.27 1.27))) (hide yes))
   (pin "1")
-  (instances (project "t1-main-board" (path "/7746052e-d7f9-59ad-ba73-bd2b74439529/357cd0ed-ef3a-5696-a4d8-7fa96210e511" (reference "#PWR0930") (unit 1))))
+  (instances (project "t1-main-board" (path "/7746052e-d7f9-59ad-ba73-bd2b74439529/357cd0ed-ef3a-5696-a4d8-7fa96210e511" (reference "#PWR0932") (unit 1))))
 )
 (rectangle (start 163.83 35.56) (end 214.63 71.12) (stroke (width 0) (type dash)) (fill (type none)))
 (text "Pull-up to vcc3v3_pmu" (exclude_from_sim no) (at 165.1 34.29 0) (effects (font (size 2.54 2.54)) (justify left bottom)))
 (symbol (lib_id "Device:D_TVS") (at 30.48 104.14 90) (unit 1) (body_style 1) (exclude_from_sim no) (in_bom yes) (on_board yes) (dnp no)
-  (property "Reference" "D5701" (at 35.92 102.87 90) (effects (font (size 1.27 1.27))))
+  (property "Reference" "D5801" (at 35.92 102.87 90) (effects (font (size 1.27 1.27))))
   (property "Value" "TPD1E10B06" (at 38.82 105.41 90) (effects (font (size 1.27 1.27))))
   (property "Footprint" "Package_SON:Texas_DPY0002A_0.6x1mm_P0.65mm" (at 30.48 104.14 0) (effects (font (size 1.27 1.27))) (hide yes))
@@
   (pin "1")
   (pin "2")
-  (instances (project "t1-main-board" (path "/7746052e-d7f9-59ad-ba73-bd2b74439529/357cd0ed-ef3a-5696-a4d8-7fa96210e511" (reference "D5701") (unit 1))))
+  (instances (project "t1-main-board" (path "/7746052e-d7f9-59ad-ba73-bd2b74439529/357cd0ed-ef3a-5696-a4d8-7fa96210e511" (reference "D5801") (unit 1))))
 )
 (wire (pts (xy 30.48 100.33) (xy 30.48 97.79)) (stroke (width 0) (type default)))
 (wire (pts (xy 30.48 107.95) (xy 30.48 110.49)) (stroke (width 0) (type default)))
 (symbol (lib_id "power:GND") (at 30.48 110.49 0) (unit 1) (body_style 1) (exclude_from_sim no) (in_bom yes) (on_board yes) (dnp no)
-  (property "Reference" "#PWR0931" (at 30.48 110.49 0) (effects (font (size 1.27 1.27))) (hide yes))
+  (property "Reference" "#PWR0933" (at 30.48 110.49 0) (effects (font (size 1.27 1.27))) (hide yes))
   (property "Value" "GND" (at 30.48 114.3 0) (effects (font (size 1.27 1.27))))
   (property "Footprint" "" (at 30.48 110.49 0) (effects (font (size 1.27 1.27))) (hide yes))
   (property "Datasheet" "" (at 30.48 110.49 0) (effects (font (size 1.27 1.27))) (hide yes))
   (pin "1")
-  (instances (project "t1-main-board" (path "/7746052e-d7f9-59ad-ba73-bd2b74439529/357cd0ed-ef3a-5696-a4d8-7fa96210e511" (reference "#PWR0931") (unit 1))))
+  (instances (project "t1-main-board" (path "/7746052e-d7f9-59ad-ba73-bd2b74439529/357cd0ed-ef3a-5696-a4d8-7fa96210e511" (reference "#PWR0933") (unit 1))))
 )
 (rectangle (start 22.86 81.28) (end 87.63 119.38) (stroke (width 0) (type dash)) (fill (type none)))

Commit message: Board: capture blk.maskrom
Power + Vol- at a cold power-on pull eMMC D0 low inside the TPS3808G01
boot window (BOM v1 lines 35, 78, 97, 98; sim/maskrom): SENSE 280k/100k,
CT 390 nF, WINDOW_N with its pad, SN74LVC1G57 and SN74LVC1G58 on
vcca1v8_pmu, BAT54 from PWRON_N, DMG1012T through 1 kΩ to EMMC_D0.
Every block in use now has its sheet; the README states the remaining
single-pin nets.

Co-Authored-By: Claude Opus 5.5 <noreply@anthropic.com>
Claude-Session: https://claude.ai/code/session_01Ei262h3TpgY9vyfNLMi5Mn
Parts:
- removed D5801: TPD1E10B06, Package_SON:Texas_DPY0002A_0.6x1mm_P0.65mm, symbol Device:D_TVS
- removed R5801: 100 kΩ, Resistor_SMD:R_0402_1005Metric, symbol Device:R
- removed TP5801: COVER, TestPoint:TestPoint_Pad_2.0x2.0mm, symbol Connector:TestPoint
- removed TP5802: COVER_GND, TestPoint:TestPoint_Pad_2.0x2.0mm, symbol Connector:TestPoint
- added D5901: TPD1E10B06, Package_SON:Texas_DPY0002A_0.6x1mm_P0.65mm, symbol Device:D_TVS
- added R5901: 100 kΩ, Resistor_SMD:R_0402_1005Metric, symbol Device:R
- added TP5901: COVER, TestPoint:TestPoint_Pad_2.0x2.0mm, symbol Connector:TestPoint
- added TP5902: COVER_GND, TestPoint:TestPoint_Pad_2.0x2.0mm, symbol Connector:TestPoint
Connections:
- net COVER_DET_N: now also D5901.2 (A2), R5901.2, TP5901.1
- net GND: now also D5901.1 (A1), TP5902.1
- net vcc3v3_pmu: now also R5901.1
Changed lines of the file:
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@@
 (title_block (title "Cover detect") (date "2026-10-25") (rev "A") (company "The OpenDAP Project") (comment 1 "blk.cover-detect") (comment 2 "Back-cover detect input: board-edge contact pads, pull-up, ESD"))
 (symbol (lib_id "Connector:TestPoint") (at 39.37 45.72 0) (unit 1) (body_style 1) (exclude_from_sim no) (in_bom no) (on_board yes) (dnp no)
-  (property "Reference" "TP5801" (at 38.1 40.64 0) (effects (font (size 1.27 1.27)) (justify right)))
+  (property "Reference" "TP5901" (at 38.1 40.64 0) (effects (font (size 1.27 1.27)) (justify right)))
   (property "Value" "COVER" (at 38.1 43.18 0) (effects (font (size 1.27 1.27)) (justify right)))
   (property "Footprint" "TestPoint:TestPoint_Pad_2.0x2.0mm" (at 39.37 45.72 0) (effects (font (size 1.27 1.27))) (hide yes))
@@
   (property "Block" "blk.cover-detect" (at 39.37 45.72 0) (effects (font (size 1.27 1.27))) (hide yes))
   (pin "1")
-  (instances (project "t1-main-board" (path "/7746052e-d7f9-59ad-ba73-bd2b74439529/357cd0ed-ef3a-5696-a4d8-7fa96210e511" (reference "TP5801") (unit 1))))
+  (instances (project "t1-main-board" (path "/7746052e-d7f9-59ad-ba73-bd2b74439529/357cd0ed-ef3a-5696-a4d8-7fa96210e511" (reference "TP5901") (unit 1))))
 )
 (symbol (lib_id "Connector:TestPoint") (at 64.77 45.72 0) (unit 1) (body_style 1) (exclude_from_sim no) (in_bom no) (on_board yes) (dnp no)
-  (property "Reference" "TP5802" (at 63.5 40.64 0) (effects (font (size 1.27 1.27)) (justify right)))
+  (property "Reference" "TP5902" (at 63.5 40.64 0) (effects (font (size 1.27 1.27)) (justify right)))
   (property "Value" "COVER_GND" (at 63.5 43.18 0) (effects (font (size 1.27 1.27)) (justify right)))
   (property "Footprint" "TestPoint:TestPoint_Pad_2.0x2.0mm" (at 64.77 45.72 0) (effects (font (size 1.27 1.27))) (hide yes))
@@
   (property "Block" "blk.cover-detect" (at 64.77 45.72 0) (effects (font (size 1.27 1.27))) (hide yes))
   (pin "1")
-  (instances (project "t1-main-board" (path "/7746052e-d7f9-59ad-ba73-bd2b74439529/357cd0ed-ef3a-5696-a4d8-7fa96210e511" (reference "TP5802") (unit 1))))
+  (instances (project "t1-main-board" (path "/7746052e-d7f9-59ad-ba73-bd2b74439529/357cd0ed-ef3a-5696-a4d8-7fa96210e511" (reference "TP5902") (unit 1))))
 )
 (wire (pts (xy 64.77 45.72) (xy 64.77 48.26)) (stroke (width 0) (type default)))
@@
 (text "Contact pads at the board edge (BOM v1 line 143; PCB-L-10)" (exclude_from_sim no) (at 24.13 34.29 0) (effects (font (size 2.54 2.54)) (justify left bottom)))
 (symbol (lib_id "Device:R") (at 175.26 48.26 0) (unit 1) (body_style 1) (exclude_from_sim no) (in_bom yes) (on_board yes) (dnp no)
-  (property "Reference" "R5801" (at 176.53 46.99 0) (effects (font (size 1.27 1.27)) (justify left)))
+  (property "Reference" "R5901" (at 176.53 46.99 0) (effects (font (size 1.27 1.27)) (justify left)))
   (property "Value" "100 kΩ" (at 176.53 49.53 0) (effects (font (size 1.27 1.27)) (justify left)))
   (property "Footprint" "Resistor_SMD:R_0402_1005Metric" (at 175.26 48.26 0) (effects (font (size 1.27 1.27))) (hide yes))
@@
   (pin "1")
   (pin "2")
-  (instances (project "t1-main-board" (path "/7746052e-d7f9-59ad-ba73-bd2b74439529/357cd0ed-ef3a-5696-a4d8-7fa96210e511" (reference "R5801") (unit 1))))
+  (instances (project "t1-main-board" (path "/7746052e-d7f9-59ad-ba73-bd2b74439529/357cd0ed-ef3a-5696-a4d8-7fa96210e511" (reference "R5901") (unit 1))))
 )
 (wire (pts (xy 175.26 44.45) (xy 175.26 41.91)) (stroke (width 0) (type default)))
@@
 (text "Pull-up to vcc3v3_pmu" (exclude_from_sim no) (at 165.1 34.29 0) (effects (font (size 2.54 2.54)) (justify left bottom)))
 (symbol (lib_id "Device:D_TVS") (at 30.48 104.14 90) (unit 1) (body_style 1) (exclude_from_sim no) (in_bom yes) (on_board yes) (dnp no)
-  (property "Reference" "D5801" (at 35.92 102.87 90) (effects (font (size 1.27 1.27))))
+  (property "Reference" "D5901" (at 35.92 102.87 90) (effects (font (size 1.27 1.27))))
   (property "Value" "TPD1E10B06" (at 38.82 105.41 90) (effects (font (size 1.27 1.27))))
   (property "Footprint" "Package_SON:Texas_DPY0002A_0.6x1mm_P0.65mm" (at 30.48 104.14 0) (effects (font (size 1.27 1.27))) (hide yes))
@@
   (pin "1")
   (pin "2")
-  (instances (project "t1-main-board" (path "/7746052e-d7f9-59ad-ba73-bd2b74439529/357cd0ed-ef3a-5696-a4d8-7fa96210e511" (reference "D5801") (unit 1))))
+  (instances (project "t1-main-board" (path "/7746052e-d7f9-59ad-ba73-bd2b74439529/357cd0ed-ef3a-5696-a4d8-7fa96210e511" (reference "D5901") (unit 1))))
 )
 (wire (pts (xy 30.48 100.33) (xy 30.48 97.79)) (stroke (width 0) (type default)))

Commit message: Board in the 62.5 x 95.0 mm body: ADR 0025, outline 59.1 x 91.6, 0201 swaps
ADR 0025 supersedes ADR 0016 for t1 ADR 0006's body: board outline from
the body, 1.2 mm walls and 0.5 mm clearance; height zones and stack
restated unchanged; the speaker on a case shelf (PCB-Z-09); pocket
reliefs at the 4.4 mm jack, the microSD (DM3AT push-push kept) and the
side buttons; the audio 0603 -> 0402 swap gated by t1 V2-A08; reserve
(NFC reader, then TPM) recorded, not applied.

- pcb/geometry.py derives the outline from BODY, WALL and CLEARANCE;
  the pocket, display and fixed parts keep their device-frame positions;
  holes keep their edge distance; the speaker shadow becomes a 1.5 mm
  shelf height area (placement, checks, occupancy).
- build.py reports pocket reliefs and routing room; C904 unfixed (it
  now finds back room, so PCB-Z-04 carries no part).
- Generator: parts.area_swap puts 121 generic 0402 resistors (outside
  audio and VBUS paths, >= 10 ohm) and five 100 nF signal capacitors in
  0201 (BOM v1.16); schematic and board regenerated.
- Result: 1,012/1,012 placed, 98.8 % by the floorplan method (was 111 %),
  factor left 1.68 (was 1.49); DRC 0 errors, ERC 0 errors, 0 check
  findings, pcb tests 20/20, schematic craft Q1 met.
- Specs: PCB constraints v0.17 (M-01, M-02, M-08, Z-02, Z-06 to Z-09,
  R-07), placement v1.1 (section 3, decisions 4 and 13, checks, open
  items with the gated swaps and the reserve), floorplan v1 section 1,
  BOM v1.16.

Co-Authored-By: Claude Opus 5.5 <noreply@anthropic.com>
Claude-Session: https://claude.ai/code/session_01Ei262h3TpgY9vyfNLMi5Mn
Parts:
- R5901: footprint Resistor_SMD:R_0402_1005Metric -> Resistor_SMD:R_0201_0603Metric; MPN RC0402FR-07100KL -> RC0201FR-07100KL
Changed lines of the file:
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@@
   (property "Reference" "R5901" (at 176.53 46.99 0) (effects (font (size 1.27 1.27)) (justify left)))
   (property "Value" "100 kΩ" (at 176.53 49.53 0) (effects (font (size 1.27 1.27)) (justify left)))
-  (property "Footprint" "Resistor_SMD:R_0402_1005Metric" (at 175.26 48.26 0) (effects (font (size 1.27 1.27))) (hide yes))
-  (property "Datasheet" "https://yageogroup.com/en/ProductSearch/PartNumberSearch?part=RC0402FR-07100KL" (at 175.26 48.26 0) (effects (font (size 1.27 1.27))) (hide yes))
-  (property "Description" "Resistor, 100 kΩ, 1 %, 1/16 W, 0402" (at 175.26 48.26 0) (effects (font (size 1.27 1.27))) (hide yes))
+  (property "Footprint" "Resistor_SMD:R_0201_0603Metric" (at 175.26 48.26 0) (effects (font (size 1.27 1.27))) (hide yes))
+  (property "Datasheet" "https://yageogroup.com/en/ProductSearch/PartNumberSearch?part=RC0201FR-07100KL" (at 175.26 48.26 0) (effects (font (size 1.27 1.27))) (hide yes))
+  (property "Description" "Resistor, 100 kΩ, 1 %, 1/20 W, 0201" (at 175.26 48.26 0) (effects (font (size 1.27 1.27))) (hide yes))
   (property "Manufacturer" "YAGEO" (at 175.26 48.26 0) (effects (font (size 1.27 1.27))) (hide yes))
-  (property "MPN" "RC0402FR-07100KL" (at 175.26 48.26 0) (effects (font (size 1.27 1.27))) (hide yes))
+  (property "MPN" "RC0201FR-07100KL" (at 175.26 48.26 0) (effects (font (size 1.27 1.27))) (hide yes))
   (property "Block" "blk.cover-detect" (at 175.26 48.26 0) (effects (font (size 1.27 1.27))) (hide yes))
   (pin "1")
