File: board/hardware/t1-main-board/emmc.kicad_sch (KiCad schematic)
At the start: 12 parts, among them U3801 KLMBG2JETD-B041

Commit message: Board on libs v0.2.0: lower-case kebab vendor keys (HL-13)
The libs submodule moves to v0.2.0 (5f24483). Every library nickname in
the generator, the placement tool and the floorplan study follows the
key table (Texas_Instruments -> texas-instruments, OpenDAP_Device ->
opendap-generic, Rockchip and Rockchip_PMIC -> rockchip, ...); the
library tables are written from the files. Schematic and board
regenerated.

Checks: ERC 0 errors (warnings unchanged); DRC 0 errors, 605 warnings,
the same counts by type, schematic parity 0; every placement identical;
craft Q1 met; pcb tests pass; STEP export resolves every libs 3D model
(the 27 parts without a model are KiCad stock lands that have none).

Co-Authored-By: Claude Opus 5.5 <noreply@anthropic.com>
Claude-Session: https://claude.ai/code/session_01Ei262h3TpgY9vyfNLMi5Mn
Parts:
- U3801: footprint Samsung:Samsung_FBGA-153_11.5x13.0mm_Layout14x14_P0.5mm_Ball0.3mm_Pad0.25mm_NSMD -> samsung:Samsung_FBGA-153_11.5x13.0mm_Layout14x14_P0.5mm_Ball0.3mm_Pad0.25mm_NSMD; symbol Samsung:KLMBG2JETD-B041 -> samsung:KLMBG2JETD-B041
Changed lines of the file:
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@@
   (instances (project "t1-main-board" (path "/7746052e-d7f9-59ad-ba73-bd2b74439529/f5764254-5d4c-5116-a59d-bc4db1d1e41c" (reference "#PWR0352") (unit 1))))
 )
-(symbol (lib_id "Samsung:KLMBG2JETD-B041") (at 149.86 58.42 0) (unit 1) (body_style 1) (exclude_from_sim no) (in_bom yes) (on_board yes) (dnp no)
+(symbol (lib_id "samsung:KLMBG2JETD-B041") (at 149.86 58.42 0) (unit 1) (body_style 1) (exclude_from_sim no) (in_bom yes) (on_board yes) (dnp no)
   (property "Reference" "U3801" (at 137.16 40.64 0) (effects (font (size 1.27 1.27)) (justify left)))
   (property "Value" "KLMBG2JETD-B041" (at 137.16 38.1 0) (effects (font (size 1.27 1.27)) (justify left)))
-  (property "Footprint" "Samsung:Samsung_FBGA-153_11.5x13.0mm_Layout14x14_P0.5mm_Ball0.3mm_Pad0.25mm_NSMD" (at 149.86 58.42 0) (effects (font (size 1.27 1.27))) (hide yes))
+  (property "Footprint" "samsung:Samsung_FBGA-153_11.5x13.0mm_Layout14x14_P0.5mm_Ball0.3mm_Pad0.25mm_NSMD" (at 149.86 58.42 0) (effects (font (size 1.27 1.27))) (hide yes))
   (property "Datasheet" "https://datasheet.lcsc.com/datasheet/pdf/8cca530d6d5054b226dcd9a69d076028.pdf?productCode=C2803245" (at 149.86 58.42 0) (effects (font (size 1.27 1.27))) (hide yes))
   (property "Description" "eMMC 5.1 managed NAND, 32 GB, HS400, VCCQ 1.70-1.95 V or 2.7-3.6 V, VCC 2.7-3.6 V, 153FBGA 11.5 x 13 x 0.8 mm" (at 149.86 58.42 0) (effects (font (size 1.27 1.27))) (hide yes))
@@
 (wire (pts (xy 132.08 68.58) (xy 129.54 68.58)) (stroke (width 0) (type default)))
 (wire (pts (xy 167.64 45.72) (xy 170.18 45.72)) (stroke (width 0) (type default)))
-(symbol (lib_id "Samsung:KLMBG2JETD-B041") (at 142.24 88.9 0) (unit 2) (body_style 1) (exclude_from_sim no) (in_bom yes) (on_board yes) (dnp no)
+(symbol (lib_id "samsung:KLMBG2JETD-B041") (at 142.24 88.9 0) (unit 2) (body_style 1) (exclude_from_sim no) (in_bom yes) (on_board yes) (dnp no)
   (property "Reference" "U3801" (at 134.62 83.82 0) (effects (font (size 1.27 1.27)) (justify left)))
   (property "Value" "KLMBG2JETD-B041" (at 134.62 81.28 0) (effects (font (size 1.27 1.27)) (justify left)))
-  (property "Footprint" "Samsung:Samsung_FBGA-153_11.5x13.0mm_Layout14x14_P0.5mm_Ball0.3mm_Pad0.25mm_NSMD" (at 142.24 88.9 0) (effects (font (size 1.27 1.27))) (hide yes))
+  (property "Footprint" "samsung:Samsung_FBGA-153_11.5x13.0mm_Layout14x14_P0.5mm_Ball0.3mm_Pad0.25mm_NSMD" (at 142.24 88.9 0) (effects (font (size 1.27 1.27))) (hide yes))
   (property "Datasheet" "https://datasheet.lcsc.com/datasheet/pdf/8cca530d6d5054b226dcd9a69d076028.pdf?productCode=C2803245" (at 142.24 88.9 0) (effects (font (size 1.27 1.27))) (hide yes))
   (property "Description" "eMMC 5.1 managed NAND, 32 GB, HS400, VCCQ 1.70-1.95 V or 2.7-3.6 V, VCC 2.7-3.6 V, 153FBGA 11.5 x 13 x 0.8 mm" (at 142.24 88.9 0) (effects (font (size 1.27 1.27))) (hide yes))
@@
   (instances (project "t1-main-board" (path "/7746052e-d7f9-59ad-ba73-bd2b74439529/f5764254-5d4c-5116-a59d-bc4db1d1e41c" (reference "#PWR0355") (unit 1))))
 )
-(symbol (lib_id "Samsung:KLMBG2JETD-B041") (at 114.3 148.59 0) (unit 3) (body_style 1) (exclude_from_sim no) (in_bom yes) (on_board yes) (dnp no)
+(symbol (lib_id "samsung:KLMBG2JETD-B041") (at 114.3 148.59 0) (unit 3) (body_style 1) (exclude_from_sim no) (in_bom yes) (on_board yes) (dnp no)
   (property "Reference" "U3801" (at 101.6 161.29 0) (effects (font (size 1.27 1.27)) (justify left)))
   (property "Value" "KLMBG2JETD-B041" (at 101.6 158.75 0) (effects (font (size 1.27 1.27)) (justify left)))
-  (property "Footprint" "Samsung:Samsung_FBGA-153_11.5x13.0mm_Layout14x14_P0.5mm_Ball0.3mm_Pad0.25mm_NSMD" (at 114.3 148.59 0) (effects (font (size 1.27 1.27))) (hide yes))
+  (property "Footprint" "samsung:Samsung_FBGA-153_11.5x13.0mm_Layout14x14_P0.5mm_Ball0.3mm_Pad0.25mm_NSMD" (at 114.3 148.59 0) (effects (font (size 1.27 1.27))) (hide yes))
   (property "Datasheet" "https://datasheet.lcsc.com/datasheet/pdf/8cca530d6d5054b226dcd9a69d076028.pdf?productCode=C2803245" (at 114.3 148.59 0) (effects (font (size 1.27 1.27))) (hide yes))
   (property "Description" "eMMC 5.1 managed NAND, 32 GB, HS400, VCCQ 1.70-1.95 V or 2.7-3.6 V, VCC 2.7-3.6 V, 153FBGA 11.5 x 13 x 0.8 mm" (at 114.3 148.59 0) (effects (font (size 1.27 1.27))) (hide yes))
@@
 (junction (at 116.84 133.35) (diameter 0) (color 0 0 0 0))
 (wire (pts (xy 132.08 151.13) (xy 134.62 151.13)) (stroke (width 0) (type default)))
-(symbol (lib_id "Samsung:KLMBG2JETD-B041") (at 116.84 185.42 0) (unit 4) (body_style 1) (exclude_from_sim no) (in_bom yes) (on_board yes) (dnp no)
+(symbol (lib_id "samsung:KLMBG2JETD-B041") (at 116.84 185.42 0) (unit 4) (body_style 1) (exclude_from_sim no) (in_bom yes) (on_board yes) (dnp no)
   (property "Reference" "U3801" (at 101.6 175.26 0) (effects (font (size 1.27 1.27)) (justify left)))
   (property "Value" "KLMBG2JETD-B041" (at 101.6 172.72 0) (effects (font (size 1.27 1.27)) (justify left)))
-  (property "Footprint" "Samsung:Samsung_FBGA-153_11.5x13.0mm_Layout14x14_P0.5mm_Ball0.3mm_Pad0.25mm_NSMD" (at 116.84 185.42 0) (effects (font (size 1.27 1.27))) (hide yes))
+  (property "Footprint" "samsung:Samsung_FBGA-153_11.5x13.0mm_Layout14x14_P0.5mm_Ball0.3mm_Pad0.25mm_NSMD" (at 116.84 185.42 0) (effects (font (size 1.27 1.27))) (hide yes))
   (property "Datasheet" "https://datasheet.lcsc.com/datasheet/pdf/8cca530d6d5054b226dcd9a69d076028.pdf?productCode=C2803245" (at 116.84 185.42 0) (effects (font (size 1.27 1.27))) (hide yes))
   (property "Description" "eMMC 5.1 managed NAND, 32 GB, HS400, VCCQ 1.70-1.95 V or 2.7-3.6 V, VCC 2.7-3.6 V, 153FBGA 11.5 x 13 x 0.8 mm" (at 116.84 185.42 0) (effects (font (size 1.27 1.27))) (hide yes))
@@
 (rectangle (start 22.86 114.3) (end 187.96 209.55) (stroke (width 0) (type dash)) (fill (type none)))
 (text "Supplies (power tree §4.12 #14, #15)" (exclude_from_sim no) (at 24.13 113.03 0) (effects (font (size 2.54 2.54)) (justify left bottom)))
-(symbol (lib_id "Samsung:KLMBG2JETD-B041") (at 241.3 121.92 0) (unit 5) (body_style 1) (exclude_from_sim no) (in_bom yes) (on_board yes) (dnp no)
+(symbol (lib_id "samsung:KLMBG2JETD-B041") (at 241.3 121.92 0) (unit 5) (body_style 1) (exclude_from_sim no) (in_bom yes) (on_board yes) (dnp no)
   (property "Reference" "U3801" (at 233.68 40.64 0) (effects (font (size 1.27 1.27)) (justify left)))
   (property "Value" "KLMBG2JETD-B041" (at 233.68 38.1 0) (effects (font (size 1.27 1.27)) (justify left)))
-  (property "Footprint" "Samsung:Samsung_FBGA-153_11.5x13.0mm_Layout14x14_P0.5mm_Ball0.3mm_Pad0.25mm_NSMD" (at 241.3 121.92 0) (effects (font (size 1.27 1.27))) (hide yes))
+  (property "Footprint" "samsung:Samsung_FBGA-153_11.5x13.0mm_Layout14x14_P0.5mm_Ball0.3mm_Pad0.25mm_NSMD" (at 241.3 121.92 0) (effects (font (size 1.27 1.27))) (hide yes))
   (property "Datasheet" "https://datasheet.lcsc.com/datasheet/pdf/8cca530d6d5054b226dcd9a69d076028.pdf?productCode=C2803245" (at 241.3 121.92 0) (effects (font (size 1.27 1.27))) (hide yes))
   (property "Description" "eMMC 5.1 managed NAND, 32 GB, HS400, VCCQ 1.70-1.95 V or 2.7-3.6 V, VCC 2.7-3.6 V, 153FBGA 11.5 x 13 x 0.8 mm" (at 241.3 121.92 0) (effects (font (size 1.27 1.27))) (hide yes))
@@
 (no_connect (at 228.6 195.58))
 (no_connect (at 228.6 198.12))
-(symbol (lib_id "Samsung:KLMBG2JETD-B041") (at 287.02 119.38 0) (unit 6) (body_style 1) (exclude_from_sim no) (in_bom yes) (on_board yes) (dnp no)
+(symbol (lib_id "samsung:KLMBG2JETD-B041") (at 287.02 119.38 0) (unit 6) (body_style 1) (exclude_from_sim no) (in_bom yes) (on_board yes) (dnp no)
   (property "Reference" "U3801" (at 279.4 40.64 0) (effects (font (size 1.27 1.27)) (justify left)))
   (property "Value" "KLMBG2JETD-B041" (at 279.4 38.1 0) (effects (font (size 1.27 1.27)) (justify left)))
-  (property "Footprint" "Samsung:Samsung_FBGA-153_11.5x13.0mm_Layout14x14_P0.5mm_Ball0.3mm_Pad0.25mm_NSMD" (at 287.02 119.38 0) (effects (font (size 1.27 1.27))) (hide yes))
+  (property "Footprint" "samsung:Samsung_FBGA-153_11.5x13.0mm_Layout14x14_P0.5mm_Ball0.3mm_Pad0.25mm_NSMD" (at 287.02 119.38 0) (effects (font (size 1.27 1.27))) (hide yes))
   (property "Datasheet" "https://datasheet.lcsc.com/datasheet/pdf/8cca530d6d5054b226dcd9a69d076028.pdf?productCode=C2803245" (at 287.02 119.38 0) (effects (font (size 1.27 1.27))) (hide yes))
   (property "Description" "eMMC 5.1 managed NAND, 32 GB, HS400, VCCQ 1.70-1.95 V or 2.7-3.6 V, VCC 2.7-3.6 V, 153FBGA 11.5 x 13 x 0.8 mm" (at 287.02 119.38 0) (effects (font (size 1.27 1.27))) (hide yes))

Commit message: Board in the 62.5 x 95.0 mm body: ADR 0025, outline 59.1 x 91.6, 0201 swaps
ADR 0025 supersedes ADR 0016 for t1 ADR 0006's body: board outline from
the body, 1.2 mm walls and 0.5 mm clearance; height zones and stack
restated unchanged; the speaker on a case shelf (PCB-Z-09); pocket
reliefs at the 4.4 mm jack, the microSD (DM3AT push-push kept) and the
side buttons; the audio 0603 -> 0402 swap gated by t1 V2-A08; reserve
(NFC reader, then TPM) recorded, not applied.

- pcb/geometry.py derives the outline from BODY, WALL and CLEARANCE;
  the pocket, display and fixed parts keep their device-frame positions;
  holes keep their edge distance; the speaker shadow becomes a 1.5 mm
  shelf height area (placement, checks, occupancy).
- build.py reports pocket reliefs and routing room; C904 unfixed (it
  now finds back room, so PCB-Z-04 carries no part).
- Generator: parts.area_swap puts 121 generic 0402 resistors (outside
  audio and VBUS paths, >= 10 ohm) and five 100 nF signal capacitors in
  0201 (BOM v1.16); schematic and board regenerated.
- Result: 1,012/1,012 placed, 98.8 % by the floorplan method (was 111 %),
  factor left 1.68 (was 1.49); DRC 0 errors, ERC 0 errors, 0 check
  findings, pcb tests 20/20, schematic craft Q1 met.
- Specs: PCB constraints v0.17 (M-01, M-02, M-08, Z-02, Z-06 to Z-09,
  R-07), placement v1.1 (section 3, decisions 4 and 13, checks, open
  items with the gated swaps and the reserve), floorplan v1 section 1,
  BOM v1.16.

Co-Authored-By: Claude Opus 5.5 <noreply@anthropic.com>
Claude-Session: https://claude.ai/code/session_01Ei262h3TpgY9vyfNLMi5Mn
Parts:
- R3801: footprint Resistor_SMD:R_0402_1005Metric -> Resistor_SMD:R_0201_0603Metric; MPN RC0402FR-0722RL -> RC0201FR-0722RL
- R3802, R3803, R3804: footprint Resistor_SMD:R_0402_1005Metric -> Resistor_SMD:R_0201_0603Metric; MPN RC0402FR-0710KL -> RC0201FR-0710KL
Changed lines of the file:
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@@
   (property "Reference" "R3801" (at 45.72 38.1 90) (effects (font (size 1.27 1.27))))
   (property "Value" "22 Ω" (at 45.72 43.18 90) (effects (font (size 1.27 1.27))))
-  (property "Footprint" "Resistor_SMD:R_0402_1005Metric" (at 45.72 40.64 0) (effects (font (size 1.27 1.27))) (hide yes))
-  (property "Datasheet" "https://yageogroup.com/en/ProductSearch/PartNumberSearch?part=RC0402FR-0722RL" (at 45.72 40.64 0) (effects (font (size 1.27 1.27))) (hide yes))
-  (property "Description" "Resistor, 22 Ω, 1 %, 1/16 W, 0402" (at 45.72 40.64 0) (effects (font (size 1.27 1.27))) (hide yes))
+  (property "Footprint" "Resistor_SMD:R_0201_0603Metric" (at 45.72 40.64 0) (effects (font (size 1.27 1.27))) (hide yes))
+  (property "Datasheet" "https://yageogroup.com/en/ProductSearch/PartNumberSearch?part=RC0201FR-0722RL" (at 45.72 40.64 0) (effects (font (size 1.27 1.27))) (hide yes))
+  (property "Description" "Resistor, 22 Ω, 1 %, 1/20 W, 0201" (at 45.72 40.64 0) (effects (font (size 1.27 1.27))) (hide yes))
   (property "Manufacturer" "YAGEO" (at 45.72 40.64 0) (effects (font (size 1.27 1.27))) (hide yes))
-  (property "MPN" "RC0402FR-0722RL" (at 45.72 40.64 0) (effects (font (size 1.27 1.27))) (hide yes))
+  (property "MPN" "RC0201FR-0722RL" (at 45.72 40.64 0) (effects (font (size 1.27 1.27))) (hide yes))
   (property "Block" "blk.emmc" (at 45.72 40.64 0) (effects (font (size 1.27 1.27))) (hide yes))
   (pin "1")
@@
   (property "Reference" "R3802" (at 72.39 54.61 0) (effects (font (size 1.27 1.27)) (justify left)))
   (property "Value" "10 kΩ" (at 72.39 57.15 0) (effects (font (size 1.27 1.27)) (justify left)))
-  (property "Footprint" "Resistor_SMD:R_0402_1005Metric" (at 71.12 55.88 0) (effects (font (size 1.27 1.27))) (hide yes))
-  (property "Datasheet" "https://yageogroup.com/en/ProductSearch/PartNumberSearch?part=RC0402FR-0710KL" (at 71.12 55.88 0) (effects (font (size 1.27 1.27))) (hide yes))
-  (property "Description" "Resistor, 10 kΩ, 1 %, 1/16 W, 0402" (at 71.12 55.88 0) (effects (font (size 1.27 1.27))) (hide yes))
+  (property "Footprint" "Resistor_SMD:R_0201_0603Metric" (at 71.12 55.88 0) (effects (font (size 1.27 1.27))) (hide yes))
+  (property "Datasheet" "https://yageogroup.com/en/ProductSearch/PartNumberSearch?part=RC0201FR-0710KL" (at 71.12 55.88 0) (effects (font (size 1.27 1.27))) (hide yes))
+  (property "Description" "Resistor, 10 kΩ, 1 %, 1/20 W, 0201" (at 71.12 55.88 0) (effects (font (size 1.27 1.27))) (hide yes))
   (property "Manufacturer" "YAGEO" (at 71.12 55.88 0) (effects (font (size 1.27 1.27))) (hide yes))
-  (property "MPN" "RC0402FR-0710KL" (at 71.12 55.88 0) (effects (font (size 1.27 1.27))) (hide yes))
+  (property "MPN" "RC0201FR-0710KL" (at 71.12 55.88 0) (effects (font (size 1.27 1.27))) (hide yes))
   (property "Block" "blk.emmc" (at 71.12 55.88 0) (effects (font (size 1.27 1.27))) (hide yes))
   (pin "1")
@@
   (property "Reference" "R3803" (at 85.09 54.61 0) (effects (font (size 1.27 1.27)) (justify left)))
   (property "Value" "10 kΩ" (at 85.09 57.15 0) (effects (font (size 1.27 1.27)) (justify left)))
-  (property "Footprint" "Resistor_SMD:R_0402_1005Metric" (at 83.82 55.88 0) (effects (font (size 1.27 1.27))) (hide yes))
-  (property "Datasheet" "https://yageogroup.com/en/ProductSearch/PartNumberSearch?part=RC0402FR-0710KL" (at 83.82 55.88 0) (effects (font (size 1.27 1.27))) (hide yes))
-  (property "Description" "Resistor, 10 kΩ, 1 %, 1/16 W, 0402" (at 83.82 55.88 0) (effects (font (size 1.27 1.27))) (hide yes))
+  (property "Footprint" "Resistor_SMD:R_0201_0603Metric" (at 83.82 55.88 0) (effects (font (size 1.27 1.27))) (hide yes))
+  (property "Datasheet" "https://yageogroup.com/en/ProductSearch/PartNumberSearch?part=RC0201FR-0710KL" (at 83.82 55.88 0) (effects (font (size 1.27 1.27))) (hide yes))
+  (property "Description" "Resistor, 10 kΩ, 1 %, 1/20 W, 0201" (at 83.82 55.88 0) (effects (font (size 1.27 1.27))) (hide yes))
   (property "Manufacturer" "YAGEO" (at 83.82 55.88 0) (effects (font (size 1.27 1.27))) (hide yes))
-  (property "MPN" "RC0402FR-0710KL" (at 83.82 55.88 0) (effects (font (size 1.27 1.27))) (hide yes))
+  (property "MPN" "RC0201FR-0710KL" (at 83.82 55.88 0) (effects (font (size 1.27 1.27))) (hide yes))
   (property "Block" "blk.emmc" (at 83.82 55.88 0) (effects (font (size 1.27 1.27))) (hide yes))
   (pin "1")
@@
   (property "Reference" "R3804" (at 97.79 54.61 0) (effects (font (size 1.27 1.27)) (justify left)))
   (property "Value" "10 kΩ" (at 97.79 57.15 0) (effects (font (size 1.27 1.27)) (justify left)))
-  (property "Footprint" "Resistor_SMD:R_0402_1005Metric" (at 96.52 55.88 0) (effects (font (size 1.27 1.27))) (hide yes))
-  (property "Datasheet" "https://yageogroup.com/en/ProductSearch/PartNumberSearch?part=RC0402FR-0710KL" (at 96.52 55.88 0) (effects (font (size 1.27 1.27))) (hide yes))
-  (property "Description" "Resistor, 10 kΩ, 1 %, 1/16 W, 0402" (at 96.52 55.88 0) (effects (font (size 1.27 1.27))) (hide yes))
+  (property "Footprint" "Resistor_SMD:R_0201_0603Metric" (at 96.52 55.88 0) (effects (font (size 1.27 1.27))) (hide yes))
+  (property "Datasheet" "https://yageogroup.com/en/ProductSearch/PartNumberSearch?part=RC0201FR-0710KL" (at 96.52 55.88 0) (effects (font (size 1.27 1.27))) (hide yes))
+  (property "Description" "Resistor, 10 kΩ, 1 %, 1/20 W, 0201" (at 96.52 55.88 0) (effects (font (size 1.27 1.27))) (hide yes))
   (property "Manufacturer" "YAGEO" (at 96.52 55.88 0) (effects (font (size 1.27 1.27))) (hide yes))
-  (property "MPN" "RC0402FR-0710KL" (at 96.52 55.88 0) (effects (font (size 1.27 1.27))) (hide yes))
+  (property "MPN" "RC0201FR-0710KL" (at 96.52 55.88 0) (effects (font (size 1.27 1.27))) (hide yes))
   (property "Block" "blk.emmc" (at 96.52 55.88 0) (effects (font (size 1.27 1.27))) (hide yes))
   (pin "1")
