File: board/hardware/t1-main-board/hpa-rails-pre.kicad_sch (KiCad schematic)
At the start: 35 parts, among them Q2801 DMG1012T, Q2802 DMP3099L, U2801 TPS65131RGER, U2802 LMR33630CRNXR

Commit message: Board: capture blk.current-monitors
Five INA236 on I2C1 (0x40-0x43, 0x48) with their shunts, per power tree
§4.12 and BOM v1 lines 54 and 136. The measured branches are rails of
their own (VSYS_SRC, VSYS_LV_AUDIO, VSYS_AUDIO, VSYS_LV_BL, VSYS_P5V1),
fed through the shunts on this sheet; the charger, audio, backlight and
5.1 V sheets take them. The root's layout may leave a stack level empty,
so the block sits under the notes; IC bboxes hold turned rail values;
passive rows hold a bottom rail's text.

Co-Authored-By: Claude Opus 5.5 <noreply@anthropic.com>
Claude-Session: https://claude.ai/code/session_01Ei262h3TpgY9vyfNLMi5Mn
Connections:
- net VSYS renamed VSYS_AUDIO
- net VSYS_LV renamed VSYS_LV_AUDIO
Other:
- moved on the sheet: C2801, C2802, C2803, C2805, C2806, C2807, C2808, C2809, C2810, C2811, C2812, C2813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

Commit message: Board on libs v0.2.0: lower-case kebab vendor keys (HL-13)
The libs submodule moves to v0.2.0 (5f24483). Every library nickname in
the generator, the placement tool and the floorplan study follows the
key table (Texas_Instruments -> texas-instruments, OpenDAP_Device ->
opendap-generic, Rockchip and Rockchip_PMIC -> rockchip, ...); the
library tables are written from the files. Schematic and board
regenerated.

Checks: ERC 0 errors (warnings unchanged); DRC 0 errors, 605 warnings,
the same counts by type, schematic parity 0; every placement identical;
craft Q1 met; pcb tests pass; STEP export resolves every libs 3D model
(the 27 parts without a model are KiCad stock lands that have none).

Co-Authored-By: Claude Opus 5.5 <noreply@anthropic.com>
Claude-Session: https://claude.ai/code/session_01Ei262h3TpgY9vyfNLMi5Mn
Parts:
- U2801: footprint Texas_Instruments:Texas_RGE0024B_VQFN-24-1EP_4x4mm_P0.5mm_EP2.45x2.45mm_ThermalVias -> texas-instruments:Texas_RGE0024B_VQFN-24-1EP_4x4mm_P0.5mm_EP2.45x2.45mm_ThermalVias; symbol Texas_Instruments:TPS65131RGER -> texas-instruments:TPS65131RGER
- U2802: footprint Texas_Instruments:Texas_RNX0012B_VQFN-HR-12_2x3mm_P0.5mm -> texas-instruments:Texas_RNX0012B_VQFN-HR-12_2x3mm_P0.5mm; symbol Texas_Instruments:LMR33630CRNXR -> texas-instruments:LMR33630CRNXR
Changed lines of the file:
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@@
 (paper "A3")
 (title_block (title "Amplifier rails: +-7 V pre-rails") (date "2026-10-25") (rev "A") (company "The OpenDAP Project") (comment 1 "blk.hpa-rails-pre") (comment 2 "+7 V TPS65131 boost, -7 V LMR33630C inverting buck-boost and its enable shifter"))
-(symbol (lib_id "Texas_Instruments:TPS65131RGER") (at 66.04 87.63 0) (unit 1) (body_style 1) (exclude_from_sim no) (in_bom yes) (on_board yes) (dnp no)
+(symbol (lib_id "texas-instruments:TPS65131RGER") (at 66.04 87.63 0) (unit 1) (body_style 1) (exclude_from_sim no) (in_bom yes) (on_board yes) (dnp no)
   (property "Reference" "U2801" (at 67.31 58.42 0) (effects (font (size 1.27 1.27)) (justify left)))
   (property "Value" "TPS65131RGER" (at 67.31 55.88 0) (effects (font (size 1.27 1.27)) (justify left)))
-  (property "Footprint" "Texas_Instruments:Texas_RGE0024B_VQFN-24-1EP_4x4mm_P0.5mm_EP2.45x2.45mm_ThermalVias" (at 66.04 87.63 0) (effects (font (size 1.27 1.27))) (hide yes))
+  (property "Footprint" "texas-instruments:Texas_RGE0024B_VQFN-24-1EP_4x4mm_P0.5mm_EP2.45x2.45mm_ThermalVias" (at 66.04 87.63 0) (effects (font (size 1.27 1.27))) (hide yes))
   (property "Datasheet" "https://www.ti.com/lit/ds/symlink/tps65131.pdf" (at 66.04 87.63 0) (effects (font (size 1.27 1.27))) (hide yes))
   (property "Description" "Dual-output DC-DC converter, boost up to 15 V and inverter down to -15 V, 2.7-5.5 V input, 1.95 A switch limit, power save, VQFN-24 (RGE0024B) 4 x 4 mm with exposed pad" (at 66.04 87.63 0) (effects (font (size 1.27 1.27))) (hide yes))
@@
 (rectangle (start 22.86 35.56) (end 195.58 157.48) (stroke (width 0) (type dash)) (fill (type none)))
 (text "+7 V pre-rail: TPS65131 boost (ADR 0015 item 2)" (exclude_from_sim no) (at 24.13 34.29 0) (effects (font (size 2.54 2.54)) (justify left bottom)))
-(symbol (lib_id "Texas_Instruments:LMR33630CRNXR") (at 236.22 82.55 0) (unit 1) (body_style 1) (exclude_from_sim no) (in_bom yes) (on_board yes) (dnp no)
+(symbol (lib_id "texas-instruments:LMR33630CRNXR") (at 236.22 82.55 0) (unit 1) (body_style 1) (exclude_from_sim no) (in_bom yes) (on_board yes) (dnp no)
   (property "Reference" "U2802" (at 240.03 60.96 0) (effects (font (size 1.27 1.27)) (justify left)))
   (property "Value" "LMR33630CRNXR" (at 240.03 58.42 0) (effects (font (size 1.27 1.27)) (justify left)))
-  (property "Footprint" "Texas_Instruments:Texas_RNX0012B_VQFN-HR-12_2x3mm_P0.5mm" (at 236.22 82.55 0) (effects (font (size 1.27 1.27))) (hide yes))
+  (property "Footprint" "texas-instruments:Texas_RNX0012B_VQFN-HR-12_2x3mm_P0.5mm" (at 236.22 82.55 0) (effects (font (size 1.27 1.27))) (hide yes))
   (property "Datasheet" "https://www.ti.com/lit/ds/symlink/lmr33630.pdf" (at 236.22 82.55 0) (effects (font (size 1.27 1.27))) (hide yes))
   (property "Description" "3.8-36 V, 3 A synchronous step-down converter, 2.1 MHz (C version), power good, VQFN-HR-12 (RNX0012B) 2 x 3 mm" (at 236.22 82.55 0) (effects (font (size 1.27 1.27))) (hide yes))

Commit message: BOM v1.18 item 2: successors of the discontinued 1 uF 0402
GRM155R61A105KE15D is to be discontinued. 44 positions take
GRM155C71A105KE11D (1 uF 10 V X7S); the eight TPS7A20 positions take
GRM155R61C225KE11D (2.2 uF 16 V X5R) to keep the 0.47 uF effective
minimum with 10 % to spare at up to 3.8 V. Same land; sourcing pass.
Closes BOM §7 item 52; new item 55 lists the other capture parts outside
Murata's product data or near end of life.

Co-Authored-By: Claude Opus 5.5 <noreply@anthropic.com>
Claude-Session: https://claude.ai/code/session_01Ei262h3TpgY9vyfNLMi5Mn
Parts:
- C2813: MPN GRM155R61A105KE15D -> GRM155C71A105KE11D
Changed lines of the file:
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@@
   (property "Value" "1 µF" (at 337.82 72.39 0) (effects (font (size 1.27 1.27)) (justify left)))
   (property "Footprint" "Capacitor_SMD:C_0402_1005Metric" (at 335.28 71.12 0) (effects (font (size 1.27 1.27))) (hide yes))
-  (property "Datasheet" "https://www.murata.com/en-us/products/productdetail?partno=GRM155R61A105KE15D" (at 335.28 71.12 0) (effects (font (size 1.27 1.27))) (hide yes))
-  (property "Description" "Capacitor, 1 µF, 10 V, X5R, 0402" (at 335.28 71.12 0) (effects (font (size 1.27 1.27))) (hide yes))
+  (property "Datasheet" "https://www.murata.com/en-us/products/productdetail?partno=GRM155C71A105KE11D" (at 335.28 71.12 0) (effects (font (size 1.27 1.27))) (hide yes))
+  (property "Description" "Capacitor, 1 µF, 10 V, X7S, 0402" (at 335.28 71.12 0) (effects (font (size 1.27 1.27))) (hide yes))
   (property "Manufacturer" "Murata" (at 335.28 71.12 0) (effects (font (size 1.27 1.27))) (hide yes))
-  (property "MPN" "GRM155R61A105KE15D" (at 335.28 71.12 0) (effects (font (size 1.27 1.27))) (hide yes))
+  (property "MPN" "GRM155C71A105KE11D" (at 335.28 71.12 0) (effects (font (size 1.27 1.27))) (hide yes))
   (property "Block" "blk.hpa-rails-pre" (at 335.28 71.12 0) (effects (font (size 1.27 1.27))) (hide yes))
   (pin "1")

Commit message: Variants: devicetree nodes, host-side absent pulls, board variant data
Feature blocks: every record with a devicetree node names it; Sub-blocks
rows for the 16 sheet IDs. The RP2354 and HPA_RAIL_EN absent-state
pull-downs move to blk.soc-vccio-b, so they stay when the block is not
fitted; cover detect relies on the ball's own pull-down. pcb/variants.py
copies the schematic's production data onto the board. odapkit variant
check: full and production pass, reproducible.

The PTS815 land drawn from the C&K data sheet (p. B-44); the side buttons
respaced for it (PCB-Z-08 updated). Studies find repos.tsv by walking up
and use libs' rockchip.pretty. DRC 0 errors, ERC 0 errors, craft Q1 met,
pcb tests pass (33), 994 parts placed, 99.7 % board need, factor 1.64.

Co-Authored-By: Claude Opus 5.5 <noreply@anthropic.com>
Claude-Session: https://claude.ai/code/session_013P6pW9LdyEMFishwCcZGUr
Parts:
- removed R2809: 100 kΩ, Resistor_SMD:R_0402_1005Metric, symbol Device:R
Connections:
- net AUDIO_N7V0: now also R2808.2
- net GND: no longer R2806.2
- net HPA_N7_EN: now also R2807.2, R2808.1; no longer R2808.2
- net HPA_N7_LS_D: now also R2807.1; no longer R2808.1
- net HPA_N7_LS_G: now also R2806.2; no longer R2807.2
- net HPA_RAIL_EN: no longer R2806.1
- net VSYS_AUDIO: now also R2806.1; no longer R2807.1
Other:
- moved on the sheet: Q2801, Q2802, R2806, R2807, R2808
