File: board/hardware/t1-main-board/soc-ground.kicad_sch (KiCad schematic)
At the start: 1 part, among them U1301 RK3566

Commit message: Board on libs v0.2.0: lower-case kebab vendor keys (HL-13)
The libs submodule moves to v0.2.0 (5f24483). Every library nickname in
the generator, the placement tool and the floorplan study follows the
key table (Texas_Instruments -> texas-instruments, OpenDAP_Device ->
opendap-generic, Rockchip and Rockchip_PMIC -> rockchip, ...); the
library tables are written from the files. Schematic and board
regenerated.

Checks: ERC 0 errors (warnings unchanged); DRC 0 errors, 605 warnings,
the same counts by type, schematic parity 0; every placement identical;
craft Q1 met; pcb tests pass; STEP export resolves every libs 3D model
(the 27 parts without a model are KiCad stock lands that have none).

Co-Authored-By: Claude Opus 5.5 <noreply@anthropic.com>
Claude-Session: https://claude.ai/code/session_01Ei262h3TpgY9vyfNLMi5Mn
Parts:
- U1301: footprint Rockchip:Rockchip_FCCSP-565L_15.5x14.4mm_P0.4mm_P0.65mm_Ball0.25mm_Pad0.25mm_NSMD -> rockchip:Rockchip_FCCSP-565L_15.5x14.4mm_P0.4mm_P0.65mm_Ball0.25mm_Pad0.25mm_NSMD; symbol Rockchip:RK3566 -> rockchip:RK3566
Changed lines of the file:
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@@
 (paper "A3")
 (title_block (title "SoC: ground") (date "2026-10-25") (rev "A") (company "The OpenDAP Project") (comment 1 "blk.soc-ground") (comment 2 "RK3566 ground balls"))
-(symbol (lib_id "Rockchip:RK3566") (at 110.49 46.99 0) (unit 23) (body_style 1) (exclude_from_sim no) (in_bom yes) (on_board yes) (dnp no)
+(symbol (lib_id "rockchip:RK3566") (at 110.49 46.99 0) (unit 23) (body_style 1) (exclude_from_sim no) (in_bom yes) (on_board yes) (dnp no)
   (property "Reference" "U1301" (at 25.4 35.56 0) (effects (font (size 1.27 1.27)) (justify left)))
   (property "Value" "RK3566" (at 25.4 33.02 0) (effects (font (size 1.27 1.27)) (justify left)))
-  (property "Footprint" "Rockchip:Rockchip_FCCSP-565L_15.5x14.4mm_P0.4mm_P0.65mm_Ball0.25mm_Pad0.25mm_NSMD" (at 110.49 46.99 0) (effects (font (size 1.27 1.27))) (hide yes))
+  (property "Footprint" "rockchip:Rockchip_FCCSP-565L_15.5x14.4mm_P0.4mm_P0.65mm_Ball0.25mm_Pad0.25mm_NSMD" (at 110.49 46.99 0) (effects (font (size 1.27 1.27))) (hide yes))
   (property "Datasheet" "https://dl.xkwy2018.com/downloads/RK3568/Rockchip-RK3566-Datasheet-V1.1-20210305.pdf" (at 110.49 46.99 0) (effects (font (size 1.27 1.27))) (hide yes))
   (property "Description" "Quad-core Arm Cortex-A55 application processor, LPDDR4X/DDR4 32-bit, eMMC 5.1, FCCSP565L 15.5 x 14.4 mm" (at 110.49 46.99 0) (effects (font (size 1.27 1.27))) (hide yes))
@@
   (instances (project "t1-main-board" (path "/7746052e-d7f9-59ad-ba73-bd2b74439529/8302eaa7-1fc9-5a34-8a84-8a9171d22bdf/04e4d217-3e36-5614-b369-f64dc9d56988" (reference "#PWR0315") (unit 1))))
 )
-(symbol (lib_id "Rockchip:RK3566") (at 288.29 49.53 0) (unit 24) (body_style 1) (exclude_from_sim no) (in_bom yes) (on_board yes) (dnp no)
+(symbol (lib_id "rockchip:RK3566") (at 288.29 49.53 0) (unit 24) (body_style 1) (exclude_from_sim no) (in_bom yes) (on_board yes) (dnp no)
   (property "Reference" "U1301" (at 203.2 35.56 0) (effects (font (size 1.27 1.27)) (justify left)))
   (property "Value" "RK3566" (at 203.2 33.02 0) (effects (font (size 1.27 1.27)) (justify left)))
-  (property "Footprint" "Rockchip:Rockchip_FCCSP-565L_15.5x14.4mm_P0.4mm_P0.65mm_Ball0.25mm_Pad0.25mm_NSMD" (at 288.29 49.53 0) (effects (font (size 1.27 1.27))) (hide yes))
+  (property "Footprint" "rockchip:Rockchip_FCCSP-565L_15.5x14.4mm_P0.4mm_P0.65mm_Ball0.25mm_Pad0.25mm_NSMD" (at 288.29 49.53 0) (effects (font (size 1.27 1.27))) (hide yes))
   (property "Datasheet" "https://dl.xkwy2018.com/downloads/RK3568/Rockchip-RK3566-Datasheet-V1.1-20210305.pdf" (at 288.29 49.53 0) (effects (font (size 1.27 1.27))) (hide yes))
   (property "Description" "Quad-core Arm Cortex-A55 application processor, LPDDR4X/DDR4 32-bit, eMMC 5.1, FCCSP565L 15.5 x 14.4 mm" (at 288.29 49.53 0) (effects (font (size 1.27 1.27))) (hide yes))
@@
   (instances (project "t1-main-board" (path "/7746052e-d7f9-59ad-ba73-bd2b74439529/8302eaa7-1fc9-5a34-8a84-8a9171d22bdf/04e4d217-3e36-5614-b369-f64dc9d56988" (reference "#PWR0316") (unit 1))))
 )
-(symbol (lib_id "Rockchip:RK3566") (at 105.41 105.41 0) (unit 25) (body_style 1) (exclude_from_sim no) (in_bom yes) (on_board yes) (dnp no)
+(symbol (lib_id "rockchip:RK3566") (at 105.41 105.41 0) (unit 25) (body_style 1) (exclude_from_sim no) (in_bom yes) (on_board yes) (dnp no)
   (property "Reference" "U1301" (at 25.4 88.9 0) (effects (font (size 1.27 1.27)) (justify left)))
   (property "Value" "RK3566" (at 25.4 86.36 0) (effects (font (size 1.27 1.27)) (justify left)))
-  (property "Footprint" "Rockchip:Rockchip_FCCSP-565L_15.5x14.4mm_P0.4mm_P0.65mm_Ball0.25mm_Pad0.25mm_NSMD" (at 105.41 105.41 0) (effects (font (size 1.27 1.27))) (hide yes))
+  (property "Footprint" "rockchip:Rockchip_FCCSP-565L_15.5x14.4mm_P0.4mm_P0.65mm_Ball0.25mm_Pad0.25mm_NSMD" (at 105.41 105.41 0) (effects (font (size 1.27 1.27))) (hide yes))
   (property "Datasheet" "https://dl.xkwy2018.com/downloads/RK3568/Rockchip-RK3566-Datasheet-V1.1-20210305.pdf" (at 105.41 105.41 0) (effects (font (size 1.27 1.27))) (hide yes))
   (property "Description" "Quad-core Arm Cortex-A55 application processor, LPDDR4X/DDR4 32-bit, eMMC 5.1, FCCSP565L 15.5 x 14.4 mm" (at 105.41 105.41 0) (effects (font (size 1.27 1.27))) (hide yes))
