File: board/hardware/t1-main-board/hpa-bal-l.kicad_sch (KiCad schematic)
At the start: 34 parts, among them U3201 OPA1622IDRCR, U3202 OPA1622IDRCR

Commit message: Board on libs v0.2.0: lower-case kebab vendor keys (HL-13)
The libs submodule moves to v0.2.0 (5f24483). Every library nickname in
the generator, the placement tool and the floorplan study follows the
key table (Texas_Instruments -> texas-instruments, OpenDAP_Device ->
opendap-generic, Rockchip and Rockchip_PMIC -> rockchip, ...); the
library tables are written from the files. Schematic and board
regenerated.

Checks: ERC 0 errors (warnings unchanged); DRC 0 errors, 605 warnings,
the same counts by type, schematic parity 0; every placement identical;
craft Q1 met; pcb tests pass; STEP export resolves every libs 3D model
(the 27 parts without a model are KiCad stock lands that have none).

Co-Authored-By: Claude Opus 5.5 <noreply@anthropic.com>
Claude-Session: https://claude.ai/code/session_01Ei262h3TpgY9vyfNLMi5Mn
Parts:
- U3201, U3202: footprint Texas_Instruments:VSON-10-1EP_3x3mm_P0.5mm_EP1.65x2.4mm_ThermalVias -> texas-instruments:VSON-10-1EP_3x3mm_P0.5mm_EP1.65x2.4mm_ThermalVias; symbol Texas_Instruments:OPA1622IDRCR -> texas-instruments:OPA1622IDRCR
Changed lines of the file:
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@@
 (wire (pts (xy 132.08 109.22) (xy 132.08 111.76)) (stroke (width 0) (type default)))
 (wire (pts (xy 132.08 111.76) (xy 127 111.76)) (stroke (width 0) (type default)))
-(symbol (lib_id "Texas_Instruments:OPA1622IDRCR") (at 193.04 78.74 0) (unit 1) (body_style 1) (exclude_from_sim no) (in_bom yes) (on_board yes) (dnp no)
+(symbol (lib_id "texas-instruments:OPA1622IDRCR") (at 193.04 78.74 0) (unit 1) (body_style 1) (exclude_from_sim no) (in_bom yes) (on_board yes) (dnp no)
   (property "Reference" "U3201" (at 194.31 57.15 0) (effects (font (size 1.27 1.27)) (justify left)))
   (property "Value" "OPA1622IDRCR" (at 194.31 54.61 0) (effects (font (size 1.27 1.27)) (justify left)))
-  (property "Footprint" "Texas_Instruments:VSON-10-1EP_3x3mm_P0.5mm_EP1.65x2.4mm_ThermalVias" (at 193.04 78.74 0) (effects (font (size 1.27 1.27))) (hide yes))
+  (property "Footprint" "texas-instruments:VSON-10-1EP_3x3mm_P0.5mm_EP1.65x2.4mm_ThermalVias" (at 193.04 78.74 0) (effects (font (size 1.27 1.27))) (hide yes))
   (property "Datasheet" "https://www.ti.com/lit/ds/symlink/opa1622.pdf" (at 193.04 78.74 0) (effects (font (size 1.27 1.27))) (hide yes))
   (property "Description" "Dual bipolar-input audio operational amplifier, high-current output, enable pin, VSON-10 (DRC) 3 x 3 mm with thermal pad" (at 193.04 78.74 0) (effects (font (size 1.27 1.27))) (hide yes))
@@
 (wire (pts (xy 132.08 203.2) (xy 132.08 205.74)) (stroke (width 0) (type default)))
 (wire (pts (xy 132.08 205.74) (xy 127 205.74)) (stroke (width 0) (type default)))
-(symbol (lib_id "Texas_Instruments:OPA1622IDRCR") (at 193.04 172.72 0) (unit 1) (body_style 1) (exclude_from_sim no) (in_bom yes) (on_board yes) (dnp no)
+(symbol (lib_id "texas-instruments:OPA1622IDRCR") (at 193.04 172.72 0) (unit 1) (body_style 1) (exclude_from_sim no) (in_bom yes) (on_board yes) (dnp no)
   (property "Reference" "U3202" (at 194.31 151.13 0) (effects (font (size 1.27 1.27)) (justify left)))
   (property "Value" "OPA1622IDRCR" (at 194.31 148.59 0) (effects (font (size 1.27 1.27)) (justify left)))
-  (property "Footprint" "Texas_Instruments:VSON-10-1EP_3x3mm_P0.5mm_EP1.65x2.4mm_ThermalVias" (at 193.04 172.72 0) (effects (font (size 1.27 1.27))) (hide yes))
+  (property "Footprint" "texas-instruments:VSON-10-1EP_3x3mm_P0.5mm_EP1.65x2.4mm_ThermalVias" (at 193.04 172.72 0) (effects (font (size 1.27 1.27))) (hide yes))
   (property "Datasheet" "https://www.ti.com/lit/ds/symlink/opa1622.pdf" (at 193.04 172.72 0) (effects (font (size 1.27 1.27))) (hide yes))
   (property "Description" "Dual bipolar-input audio operational amplifier, high-current output, enable pin, VSON-10 (DRC) 3 x 3 mm with thermal pad" (at 193.04 172.72 0) (effects (font (size 1.27 1.27))) (hide yes))
