File: board/hardware/t1-main-board/hpa-rails-ldo.kicad_sch (KiCad schematic)
At the start: 28 parts, among them U2901 LT3045EDD, U2902 LT3045EDD, U2903 LT3094EDD, U2904 LT3094EDD

Commit message: Board on libs v0.2.0: lower-case kebab vendor keys (HL-13)
The libs submodule moves to v0.2.0 (5f24483). Every library nickname in
the generator, the placement tool and the floorplan study follows the
key table (Texas_Instruments -> texas-instruments, OpenDAP_Device ->
opendap-generic, Rockchip and Rockchip_PMIC -> rockchip, ...); the
library tables are written from the files. Schematic and board
regenerated.

Checks: ERC 0 errors (warnings unchanged); DRC 0 errors, 605 warnings,
the same counts by type, schematic parity 0; every placement identical;
craft Q1 met; pcb tests pass; STEP export resolves every libs 3D model
(the 27 parts without a model are KiCad stock lands that have none).

Co-Authored-By: Claude Opus 5.5 <noreply@anthropic.com>
Claude-Session: https://claude.ai/code/session_01Ei262h3TpgY9vyfNLMi5Mn
Parts:
- U2901, U2902: footprint Analog_Devices:Analog_DD_DFN-10-1EP_3x3mm_P0.5mm_EP1.65x2.38mm -> analog-devices:Analog_DD_DFN-10-1EP_3x3mm_P0.5mm_EP1.65x2.38mm; symbol Analog_Devices:LT3045EDD -> analog-devices:LT3045EDD
- U2903, U2904: footprint Analog_Devices:Analog_DD_DFN-12-1EP_3x3mm_P0.45mm_EP1.65x2.38mm -> analog-devices:Analog_DD_DFN-12-1EP_3x3mm_P0.45mm_EP1.65x2.38mm; symbol Analog_Devices:LT3094EDD -> analog-devices:LT3094EDD
Changed lines of the file:
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@@
 (paper "A3")
 (title_block (title "Amplifier rails: +-6 V LDOs") (date "2026-10-25") (rev "A") (company "The OpenDAP Project") (comment 1 "blk.hpa-rails-ldo") (comment 2 "Two LT3045 and two LT3094 in parallel with trace ballasts (ADR 0015 item 3)"))
-(symbol (lib_id "Analog_Devices:LT3045EDD") (at 67.31 64.77 0) (unit 1) (body_style 1) (exclude_from_sim no) (in_bom yes) (on_board yes) (dnp no)
+(symbol (lib_id "analog-devices:LT3045EDD") (at 67.31 64.77 0) (unit 1) (body_style 1) (exclude_from_sim no) (in_bom yes) (on_board yes) (dnp no)
   (property "Reference" "U2901" (at 58.42 43.18 0) (effects (font (size 1.27 1.27)) (justify left)))
   (property "Value" "LT3045EDD" (at 58.42 40.64 0) (effects (font (size 1.27 1.27)) (justify left)))
-  (property "Footprint" "Analog_Devices:Analog_DD_DFN-10-1EP_3x3mm_P0.5mm_EP1.65x2.38mm" (at 67.31 64.77 0) (effects (font (size 1.27 1.27))) (hide yes))
+  (property "Footprint" "analog-devices:Analog_DD_DFN-10-1EP_3x3mm_P0.5mm_EP1.65x2.38mm" (at 67.31 64.77 0) (effects (font (size 1.27 1.27))) (hide yes))
   (property "Datasheet" "https://www.analog.com/media/en/technical-documentation/data-sheets/lt3045.pdf" (at 67.31 64.77 0) (effects (font (size 1.27 1.27))) (hide yes))
   (property "Description" "LDO regulator, 20 V, 500 mA, 0.8 uVrms noise, 76 dB PSRR at 1 MHz, programmable current limit and power good, single-resistor output set, DFN-10 (DD) 3 x 3 mm with exposed pad" (at 67.31 64.77 0) (effects (font (size 1.27 1.27))) (hide yes))
@@
   (instances (project "t1-main-board" (path "/7746052e-d7f9-59ad-ba73-bd2b74439529/d6f0155c-678f-5298-bf09-6ea7c0e72438/cbed7f0f-43ec-5b1b-b7a5-569b0b608c26/0c52ca39-f442-51ee-bc92-c47d67c8d1a4" (reference "#PWR0512") (unit 1))))
 )
-(symbol (lib_id "Analog_Devices:LT3045EDD") (at 151.13 64.77 0) (unit 1) (body_style 1) (exclude_from_sim no) (in_bom yes) (on_board yes) (dnp no)
+(symbol (lib_id "analog-devices:LT3045EDD") (at 151.13 64.77 0) (unit 1) (body_style 1) (exclude_from_sim no) (in_bom yes) (on_board yes) (dnp no)
   (property "Reference" "U2902" (at 142.24 43.18 0) (effects (font (size 1.27 1.27)) (justify left)))
   (property "Value" "LT3045EDD" (at 142.24 40.64 0) (effects (font (size 1.27 1.27)) (justify left)))
-  (property "Footprint" "Analog_Devices:Analog_DD_DFN-10-1EP_3x3mm_P0.5mm_EP1.65x2.38mm" (at 151.13 64.77 0) (effects (font (size 1.27 1.27))) (hide yes))
+  (property "Footprint" "analog-devices:Analog_DD_DFN-10-1EP_3x3mm_P0.5mm_EP1.65x2.38mm" (at 151.13 64.77 0) (effects (font (size 1.27 1.27))) (hide yes))
   (property "Datasheet" "https://www.analog.com/media/en/technical-documentation/data-sheets/lt3045.pdf" (at 151.13 64.77 0) (effects (font (size 1.27 1.27))) (hide yes))
   (property "Description" "LDO regulator, 20 V, 500 mA, 0.8 uVrms noise, 76 dB PSRR at 1 MHz, programmable current limit and power good, single-resistor output set, DFN-10 (DD) 3 x 3 mm with exposed pad" (at 151.13 64.77 0) (effects (font (size 1.27 1.27))) (hide yes))
@@
 (rectangle (start 22.86 35.56) (end 205.74 166.37) (stroke (width 0) (type dash)) (fill (type none)))
 (text "+6 V: two LT3045 in parallel (ADR 0015 item 3)" (exclude_from_sim no) (at 24.13 34.29 0) (effects (font (size 2.54 2.54)) (justify left bottom)))
-(symbol (lib_id "Analog_Devices:LT3094EDD") (at 255.27 64.77 0) (unit 1) (body_style 1) (exclude_from_sim no) (in_bom yes) (on_board yes) (dnp no)
+(symbol (lib_id "analog-devices:LT3094EDD") (at 255.27 64.77 0) (unit 1) (body_style 1) (exclude_from_sim no) (in_bom yes) (on_board yes) (dnp no)
   (property "Reference" "U2903" (at 246.38 43.18 0) (effects (font (size 1.27 1.27)) (justify left)))
   (property "Value" "LT3094EDD" (at 246.38 40.64 0) (effects (font (size 1.27 1.27)) (justify left)))
-  (property "Footprint" "Analog_Devices:Analog_DD_DFN-12-1EP_3x3mm_P0.45mm_EP1.65x2.38mm" (at 255.27 64.77 0) (effects (font (size 1.27 1.27))) (hide yes))
+  (property "Footprint" "analog-devices:Analog_DD_DFN-12-1EP_3x3mm_P0.45mm_EP1.65x2.38mm" (at 255.27 64.77 0) (effects (font (size 1.27 1.27))) (hide yes))
   (property "Datasheet" "https://www.analog.com/media/en/technical-documentation/data-sheets/lt3094.pdf" (at 255.27 64.77 0) (effects (font (size 1.27 1.27))) (hide yes))
   (property "Description" "Negative LDO regulator, -20 V, -500 mA, 0.8 uVrms noise, 74 dB PSRR at 1 MHz, programmable current limit, power good, VIOC tracking, DFN-12 (DD) 3 x 3 mm with exposed pad (IN)" (at 255.27 64.77 0) (effects (font (size 1.27 1.27))) (hide yes))
@@
   (instances (project "t1-main-board" (path "/7746052e-d7f9-59ad-ba73-bd2b74439529/d6f0155c-678f-5298-bf09-6ea7c0e72438/cbed7f0f-43ec-5b1b-b7a5-569b0b608c26/0c52ca39-f442-51ee-bc92-c47d67c8d1a4" (reference "#PWR0532") (unit 1))))
 )
-(symbol (lib_id "Analog_Devices:LT3094EDD") (at 339.09 64.77 0) (unit 1) (body_style 1) (exclude_from_sim no) (in_bom yes) (on_board yes) (dnp no)
+(symbol (lib_id "analog-devices:LT3094EDD") (at 339.09 64.77 0) (unit 1) (body_style 1) (exclude_from_sim no) (in_bom yes) (on_board yes) (dnp no)
   (property "Reference" "U2904" (at 330.2 43.18 0) (effects (font (size 1.27 1.27)) (justify left)))
   (property "Value" "LT3094EDD" (at 330.2 40.64 0) (effects (font (size 1.27 1.27)) (justify left)))
-  (property "Footprint" "Analog_Devices:Analog_DD_DFN-12-1EP_3x3mm_P0.45mm_EP1.65x2.38mm" (at 339.09 64.77 0) (effects (font (size 1.27 1.27))) (hide yes))
+  (property "Footprint" "analog-devices:Analog_DD_DFN-12-1EP_3x3mm_P0.45mm_EP1.65x2.38mm" (at 339.09 64.77 0) (effects (font (size 1.27 1.27))) (hide yes))
   (property "Datasheet" "https://www.analog.com/media/en/technical-documentation/data-sheets/lt3094.pdf" (at 339.09 64.77 0) (effects (font (size 1.27 1.27))) (hide yes))
   (property "Description" "Negative LDO regulator, -20 V, -500 mA, 0.8 uVrms noise, 74 dB PSRR at 1 MHz, programmable current limit, power good, VIOC tracking, DFN-12 (DD) 3 x 3 mm with exposed pad (IN)" (at 339.09 64.77 0) (effects (font (size 1.27 1.27))) (hide yes))

Commit message: BOM v1.18 item 3: 22 uF X7R 1210 at the LT3045 and LT3094
GRM21BR71C106KE51L is not in Murata's product data. GRM32ER71C226KEA8L
keeps 11.1 uF effective at 6.04 V (one per output) and 10.4 uF at
7.06 V (two per LT3094 input) against the 10 uF stability minimum; no
10 uF X7R 0805 or 1206 passes. Sourcing pass. Closes BOM §7 item 53.

Co-Authored-By: Claude Opus 5.5 <noreply@anthropic.com>
Claude-Session: https://claude.ai/code/session_01Ei262h3TpgY9vyfNLMi5Mn
Parts:
- added C2913, C2914: 470 nF, Capacitor_SMD:C_0603_1608Metric, symbol Device:C
- C2902, C2904, C2907, C2908, C2909, C2910: value 10 µF -> 22 µF; footprint Capacitor_SMD:C_0805_2012Metric -> Capacitor_SMD:C_1210_3225Metric; MPN GRM21BR71C106KE51L -> GRM32ER71C226KEA8L
- C2911, C2912: value 470 nF -> 22 µF; footprint Capacitor_SMD:C_0603_1608Metric -> Capacitor_SMD:C_1210_3225Metric; MPN GRM188R71C474KA88D -> GRM32ER71C226KEA8L
Connections:
- net AUDIO_N7V0: now also C2908.1, C2910.1, C2911.1; no longer C2909.1
- net GND: now also C2913.2, C2914.2
- net HPA_N6_A: now also C2909.1; no longer C2908.1
- net HPA_N6_B: now also C2912.1; no longer C2910.1
- net HPA_N6_SET: now also C2913.1, C2914.1; no longer C2911.1, C2912.1
Other:
- moved on the sheet: C2909, C2910, C2911, C2912

Commit message: Placement v1.3: capacitor proximity rule, checked and met
pcb/proximity.py assigns every converter's input and output capacitors
(from pin functions and types) and every IC's decoupling (block rule and
the generator's new Decoupling field) and checks each within its bound
of the pins it serves (input 3, output 5, decoupling 4, bulk 6 mm); the
build fails otherwise. The placer places each IC's capacitors right
after it, keeps room for them, reorders, swaps and repairs; a search
radius bug (mm used as cells) that blocked rotations is fixed. RK809
moved 1.2 mm right and 1.1 mm down off the radio zone edge.

Fixes found: C901 was 29 mm from U901; 136 of 237 capacitors were beyond
their bound. Now 248 checked, none beyond. BOM v1.18 items 3 (revised:
3 x GRM219R61C226ME15L per LDO position), 5 (C4403 as 2 x 0805) and 6.
Tests: test_proximity (6).

Co-Authored-By: Claude Opus 5.5 <noreply@anthropic.com>
Claude-Session: https://claude.ai/code/session_01Ei262h3TpgY9vyfNLMi5Mn
Parts:
- added C2915, C2916, C2917, C2918, C2919, C2920, C2921, C2922: 22 µF, Capacitor_SMD:C_0805_2012Metric, symbol Device:C
- added C2923, C2924: 470 nF, Capacitor_SMD:C_0603_1608Metric, symbol Device:C
- C2902, C2904, C2907, C2908, C2911, C2912: footprint Capacitor_SMD:C_1210_3225Metric -> Capacitor_SMD:C_0805_2012Metric; MPN GRM32ER71C226KEA8L -> GRM219R61C226ME15L; Spec 16 V X7R -> 16 V X5R
- C2903: value 4.7 µF -> 22 µF; MPN GRM21BR71C475KA73L -> GRM219R61C226ME15L; Spec 16 V X7R -> 16 V X5R
- C2905: value 470 nF -> 4.7 µF; footprint Capacitor_SMD:C_0603_1608Metric -> Capacitor_SMD:C_0805_2012Metric; MPN GRM188R71C474KA88D -> GRM21BR71C475KA73L
- C2906, C2913, C2914: value 470 nF -> 22 µF; footprint Capacitor_SMD:C_0603_1608Metric -> Capacitor_SMD:C_0805_2012Metric; MPN GRM188R71C474KA88D -> GRM219R61C226ME15L; Spec 16 V X7R -> 16 V X5R
- C2909, C2910: value 22 µF -> 470 nF; footprint Capacitor_SMD:C_1210_3225Metric -> Capacitor_SMD:C_0603_1608Metric; MPN GRM32ER71C226KEA8L -> GRM188R71C474KA88D
Connections:
- net AUDIO_N7V0: now also C2912.1, C2913.1, C2917.1, C2918.1, C2919.1; no longer C2907.1, C2908.1, C2910.1
- net AUDIO_P7V0: now also C2905.1; no longer C2903.1
- net GND: now also C2915.2, C2916.2, C2917.2, C2918.2, C2919.2, C2920.2, C2921.2, C2922.2, C2923.2, C2924.2
- net HPA_N6_A: now also C2914.1, C2915.1, C2916.1; no longer C2909.1
- net HPA_N6_B: now also C2920.1, C2921.1, C2922.1; no longer C2912.1
- net HPA_N6_SET: now also C2923.1, C2924.1; no longer C2913.1, C2914.1
- net HPA_P6_A: now also C2903.1, C2904.1
- net HPA_P6_B: now also C2906.1, C2907.1, C2908.1; no longer C2904.1
- net HPA_P6_SET: now also C2909.1, C2910.1; no longer C2905.1, C2906.1
Other:
- moved on the sheet: C2902, C2903, C2904, C2905, C2906, C2907, C2908, C2909, C2910, C2911, C2912, C2913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
