File: board/hardware/t1-main-board/hpa-se.kicad_sch (KiCad schematic)
At the start: 40 parts, among them U3001 OPA1622IDRCR, U3002 OPA1622IDRCR

Commit message: Board on libs v0.2.0: lower-case kebab vendor keys (HL-13)
The libs submodule moves to v0.2.0 (5f24483). Every library nickname in
the generator, the placement tool and the floorplan study follows the
key table (Texas_Instruments -> texas-instruments, OpenDAP_Device ->
opendap-generic, Rockchip and Rockchip_PMIC -> rockchip, ...); the
library tables are written from the files. Schematic and board
regenerated.

Checks: ERC 0 errors (warnings unchanged); DRC 0 errors, 605 warnings,
the same counts by type, schematic parity 0; every placement identical;
craft Q1 met; pcb tests pass; STEP export resolves every libs 3D model
(the 27 parts without a model are KiCad stock lands that have none).

Co-Authored-By: Claude Opus 5.5 <noreply@anthropic.com>
Claude-Session: https://claude.ai/code/session_01Ei262h3TpgY9vyfNLMi5Mn
Parts:
- U3001, U3002: footprint Texas_Instruments:VSON-10-1EP_3x3mm_P0.5mm_EP1.65x2.4mm_ThermalVias -> texas-instruments:VSON-10-1EP_3x3mm_P0.5mm_EP1.65x2.4mm_ThermalVias; symbol Texas_Instruments:OPA1622IDRCR -> texas-instruments:OPA1622IDRCR
Changed lines of the file:
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@@
 (wire (pts (xy 130.81 107.95) (xy 130.81 110.49)) (stroke (width 0) (type default)))
 (wire (pts (xy 130.81 110.49) (xy 125.73 110.49)) (stroke (width 0) (type default)))
-(symbol (lib_id "Texas_Instruments:OPA1622IDRCR") (at 190.5 77.47 0) (unit 1) (body_style 1) (exclude_from_sim no) (in_bom yes) (on_board yes) (dnp no)
+(symbol (lib_id "texas-instruments:OPA1622IDRCR") (at 190.5 77.47 0) (unit 1) (body_style 1) (exclude_from_sim no) (in_bom yes) (on_board yes) (dnp no)
   (property "Reference" "U3001" (at 191.77 55.88 0) (effects (font (size 1.27 1.27)) (justify left)))
   (property "Value" "OPA1622IDRCR" (at 191.77 53.34 0) (effects (font (size 1.27 1.27)) (justify left)))
-  (property "Footprint" "Texas_Instruments:VSON-10-1EP_3x3mm_P0.5mm_EP1.65x2.4mm_ThermalVias" (at 190.5 77.47 0) (effects (font (size 1.27 1.27))) (hide yes))
+  (property "Footprint" "texas-instruments:VSON-10-1EP_3x3mm_P0.5mm_EP1.65x2.4mm_ThermalVias" (at 190.5 77.47 0) (effects (font (size 1.27 1.27))) (hide yes))
   (property "Datasheet" "https://www.ti.com/lit/ds/symlink/opa1622.pdf" (at 190.5 77.47 0) (effects (font (size 1.27 1.27))) (hide yes))
   (property "Description" "Dual bipolar-input audio operational amplifier, high-current output, enable pin, VSON-10 (DRC) 3 x 3 mm with thermal pad" (at 190.5 77.47 0) (effects (font (size 1.27 1.27))) (hide yes))
@@
 (wire (pts (xy 130.81 200.66) (xy 130.81 203.2)) (stroke (width 0) (type default)))
 (wire (pts (xy 130.81 203.2) (xy 125.73 203.2)) (stroke (width 0) (type default)))
-(symbol (lib_id "Texas_Instruments:OPA1622IDRCR") (at 190.5 170.18 0) (unit 1) (body_style 1) (exclude_from_sim no) (in_bom yes) (on_board yes) (dnp no)
+(symbol (lib_id "texas-instruments:OPA1622IDRCR") (at 190.5 170.18 0) (unit 1) (body_style 1) (exclude_from_sim no) (in_bom yes) (on_board yes) (dnp no)
   (property "Reference" "U3002" (at 191.77 148.59 0) (effects (font (size 1.27 1.27)) (justify left)))
   (property "Value" "OPA1622IDRCR" (at 191.77 146.05 0) (effects (font (size 1.27 1.27)) (justify left)))
-  (property "Footprint" "Texas_Instruments:VSON-10-1EP_3x3mm_P0.5mm_EP1.65x2.4mm_ThermalVias" (at 190.5 170.18 0) (effects (font (size 1.27 1.27))) (hide yes))
+  (property "Footprint" "texas-instruments:VSON-10-1EP_3x3mm_P0.5mm_EP1.65x2.4mm_ThermalVias" (at 190.5 170.18 0) (effects (font (size 1.27 1.27))) (hide yes))
   (property "Datasheet" "https://www.ti.com/lit/ds/symlink/opa1622.pdf" (at 190.5 170.18 0) (effects (font (size 1.27 1.27))) (hide yes))
   (property "Description" "Dual bipolar-input audio operational amplifier, high-current output, enable pin, VSON-10 (DRC) 3 x 3 mm with thermal pad" (at 190.5 170.18 0) (effects (font (size 1.27 1.27))) (hide yes))
