File: board/hardware/t1-main-board/maskrom.kicad_sch (KiCad schematic)
At the start: 16 parts, among them Q4101 DMG1012T, U4101 TPS3808G01DBVR, U4102 SN74LVC1G57DCKR, U4103 SN74LVC1G58DCKR

Commit message: Compaction: lower inductors, 0201 decoupling, 0.8 mm signal test pads
A matrix tool (hardware/studies/compaction) checks each candidate against
the design's stresses: same inductance, design peak <= 70 % and the
converter's maximum limit <= 100 % of Isat (30 % drop), height zones,
ratings at least twice the rail, PCB-D-06; sourcing outcome per part.

Applied (placement v1 decision 12, BOM v1.15):
- L601, L4401: XGL4015-102MEC (1.5 mm) for XAL/XGL4020-102MEC (2.1 mm);
- L1001, L5101: XGL4015-471MEC (1.5 mm) for Wurth 744373240047, on the
  stock XxL4020 land (the Wurth land was never drawn);
- L1201 is 1.2 mm (XGL4012, per-MPN heights): it moves next to the SoC;
- 58 x 100 nF decoupling on rails <= 3.3 V in core/IO/radio: 0201;
- 51 test pads on signal nets: 0.8 mm (PCB-D-06 v0.16, JLCPCB guide).
Kept: L901, L2802 (XGL4015 at 103 % of Isat at the limit); no thinner
0805/1206 capacitor passes (obsolete, NRND or unlisted).

Board need 113 % -> 111 % (core band 227 -> 203 %, power band 258 ->
233 %, radio band 19 -> 0 %); only C904 still relies on PCB-Z-04.
ERC 0 errors, craft Q1 met, DRC 0 errors (605 warnings), pcb and study
tests pass, rules test board PASS.

Co-Authored-By: Claude Opus 5.5 <noreply@anthropic.com>
Claude-Session: https://claude.ai/code/session_01Ei262h3TpgY9vyfNLMi5Mn
Parts:
- C4101, C4103, C4104: footprint Capacitor_SMD:C_0402_1005Metric -> Capacitor_SMD:C_0201_0603Metric; MPN GRM155R71C104KA88D -> GRM033R61A104KE15D
- TP4101: footprint TestPoint:TestPoint_Pad_D1.0mm -> T1_Main_Board:TestPoint_Pad_D0.8mm
Changed lines of the file:
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@@
   (property "Reference" "C4101" (at 85.09 46.99 0) (effects (font (size 1.27 1.27)) (justify left)))
   (property "Value" "100 nF" (at 85.09 49.53 0) (effects (font (size 1.27 1.27)) (justify left)))
-  (property "Footprint" "Capacitor_SMD:C_0402_1005Metric" (at 82.55 48.26 0) (effects (font (size 1.27 1.27))) (hide yes))
-  (property "Datasheet" "https://www.murata.com/en-us/products/productdetail?partno=GRM155R71C104KA88D" (at 82.55 48.26 0) (effects (font (size 1.27 1.27))) (hide yes))
-  (property "Description" "Capacitor, 100 nF, 16 V, X7R, 0402" (at 82.55 48.26 0) (effects (font (size 1.27 1.27))) (hide yes))
+  (property "Footprint" "Capacitor_SMD:C_0201_0603Metric" (at 82.55 48.26 0) (effects (font (size 1.27 1.27))) (hide yes))
+  (property "Datasheet" "https://www.murata.com/en-us/products/productdetail?partno=GRM033R61A104KE15D" (at 82.55 48.26 0) (effects (font (size 1.27 1.27))) (hide yes))
+  (property "Description" "Capacitor, 100 nF, 10 V, X5R, 0201" (at 82.55 48.26 0) (effects (font (size 1.27 1.27))) (hide yes))
   (property "Manufacturer" "Murata" (at 82.55 48.26 0) (effects (font (size 1.27 1.27))) (hide yes))
-  (property "MPN" "GRM155R71C104KA88D" (at 82.55 48.26 0) (effects (font (size 1.27 1.27))) (hide yes))
+  (property "MPN" "GRM033R61A104KE15D" (at 82.55 48.26 0) (effects (font (size 1.27 1.27))) (hide yes))
   (property "Block" "blk.maskrom" (at 82.55 48.26 0) (effects (font (size 1.27 1.27))) (hide yes))
   (pin "1")
@@
   (property "Reference" "C4103" (at 217.17 46.99 0) (effects (font (size 1.27 1.27)) (justify left)))
   (property "Value" "100 nF" (at 217.17 49.53 0) (effects (font (size 1.27 1.27)) (justify left)))
-  (property "Footprint" "Capacitor_SMD:C_0402_1005Metric" (at 214.63 48.26 0) (effects (font (size 1.27 1.27))) (hide yes))
-  (property "Datasheet" "https://www.murata.com/en-us/products/productdetail?partno=GRM155R71C104KA88D" (at 214.63 48.26 0) (effects (font (size 1.27 1.27))) (hide yes))
-  (property "Description" "Capacitor, 100 nF, 16 V, X7R, 0402" (at 214.63 48.26 0) (effects (font (size 1.27 1.27))) (hide yes))
+  (property "Footprint" "Capacitor_SMD:C_0201_0603Metric" (at 214.63 48.26 0) (effects (font (size 1.27 1.27))) (hide yes))
+  (property "Datasheet" "https://www.murata.com/en-us/products/productdetail?partno=GRM033R61A104KE15D" (at 214.63 48.26 0) (effects (font (size 1.27 1.27))) (hide yes))
+  (property "Description" "Capacitor, 100 nF, 10 V, X5R, 0201" (at 214.63 48.26 0) (effects (font (size 1.27 1.27))) (hide yes))
   (property "Manufacturer" "Murata" (at 214.63 48.26 0) (effects (font (size 1.27 1.27))) (hide yes))
-  (property "MPN" "GRM155R71C104KA88D" (at 214.63 48.26 0) (effects (font (size 1.27 1.27))) (hide yes))
+  (property "MPN" "GRM033R61A104KE15D" (at 214.63 48.26 0) (effects (font (size 1.27 1.27))) (hide yes))
   (property "Block" "blk.maskrom" (at 214.63 48.26 0) (effects (font (size 1.27 1.27))) (hide yes))
   (pin "1")
@@
   (property "Reference" "C4104" (at 97.79 137.16 0) (effects (font (size 1.27 1.27)) (justify left)))
   (property "Value" "100 nF" (at 97.79 139.7 0) (effects (font (size 1.27 1.27)) (justify left)))
-  (property "Footprint" "Capacitor_SMD:C_0402_1005Metric" (at 95.25 138.43 0) (effects (font (size 1.27 1.27))) (hide yes))
-  (property "Datasheet" "https://www.murata.com/en-us/products/productdetail?partno=GRM155R71C104KA88D" (at 95.25 138.43 0) (effects (font (size 1.27 1.27))) (hide yes))
-  (property "Description" "Capacitor, 100 nF, 16 V, X7R, 0402" (at 95.25 138.43 0) (effects (font (size 1.27 1.27))) (hide yes))
+  (property "Footprint" "Capacitor_SMD:C_0201_0603Metric" (at 95.25 138.43 0) (effects (font (size 1.27 1.27))) (hide yes))
+  (property "Datasheet" "https://www.murata.com/en-us/products/productdetail?partno=GRM033R61A104KE15D" (at 95.25 138.43 0) (effects (font (size 1.27 1.27))) (hide yes))
+  (property "Description" "Capacitor, 100 nF, 10 V, X5R, 0201" (at 95.25 138.43 0) (effects (font (size 1.27 1.27))) (hide yes))
   (property "Manufacturer" "Murata" (at 95.25 138.43 0) (effects (font (size 1.27 1.27))) (hide yes))
-  (property "MPN" "GRM155R71C104KA88D" (at 95.25 138.43 0) (effects (font (size 1.27 1.27))) (hide yes))
+  (property "MPN" "GRM033R61A104KE15D" (at 95.25 138.43 0) (effects (font (size 1.27 1.27))) (hide yes))
   (property "Block" "blk.maskrom" (at 95.25 138.43 0) (effects (font (size 1.27 1.27))) (hide yes))
   (pin "1")
@@
   (property "Reference" "TP4101" (at 261.62 130.81 0) (effects (font (size 1.27 1.27)) (justify right)))
   (property "Value" "WINDOW_N" (at 261.62 133.35 0) (effects (font (size 1.27 1.27)) (justify right)))
-  (property "Footprint" "TestPoint:TestPoint_Pad_D1.0mm" (at 262.89 135.89 0) (effects (font (size 1.27 1.27))) (hide yes))
+  (property "Footprint" "T1_Main_Board:TestPoint_Pad_D0.8mm" (at 262.89 135.89 0) (effects (font (size 1.27 1.27))) (hide yes))
   (property "Datasheet" "~" (at 262.89 135.89 0) (effects (font (size 1.27 1.27))) (hide yes))
-  (property "Description" "Test pad, 1.0 mm" (at 262.89 135.89 0) (effects (font (size 1.27 1.27))) (hide yes))
+  (property "Description" "Test pad, 0.8 mm, signal net" (at 262.89 135.89 0) (effects (font (size 1.27 1.27))) (hide yes))
   (property "Block" "blk.maskrom" (at 262.89 135.89 0) (effects (font (size 1.27 1.27))) (hide yes))
   (pin "1")

Commit message: Board on libs v0.2.0: lower-case kebab vendor keys (HL-13)
The libs submodule moves to v0.2.0 (5f24483). Every library nickname in
the generator, the placement tool and the floorplan study follows the
key table (Texas_Instruments -> texas-instruments, OpenDAP_Device ->
opendap-generic, Rockchip and Rockchip_PMIC -> rockchip, ...); the
library tables are written from the files. Schematic and board
regenerated.

Checks: ERC 0 errors (warnings unchanged); DRC 0 errors, 605 warnings,
the same counts by type, schematic parity 0; every placement identical;
craft Q1 met; pcb tests pass; STEP export resolves every libs 3D model
(the 27 parts without a model are KiCad stock lands that have none).

Co-Authored-By: Claude Opus 5.5 <noreply@anthropic.com>
Claude-Session: https://claude.ai/code/session_01Ei262h3TpgY9vyfNLMi5Mn
Parts:
- D4101: footprint Nexperia:Nexperia_SOT23_TO-236AB_2.9x1.3mm_P1.9mm -> nexperia:Nexperia_SOT23_TO-236AB_2.9x1.3mm_P1.9mm; symbol Nexperia:BAT54 -> nexperia:BAT54
- U4101: footprint Texas_Instruments:Texas_DBV0006A_SOT-23-6_1.6x2.9mm_P0.95mm -> texas-instruments:Texas_DBV0006A_SOT-23-6_1.6x2.9mm_P0.95mm; symbol Texas_Instruments:TPS3808G01DBVR -> texas-instruments:TPS3808G01DBVR
- U4102: footprint Texas_Instruments:Texas_DCK0006A_SC-70-6_1.25x2mm_P0.65mm -> texas-instruments:Texas_DCK0006A_SC-70-6_1.25x2mm_P0.65mm; symbol Texas_Instruments:SN74LVC1G57DCKR -> texas-instruments:SN74LVC1G57DCKR
- U4103: footprint Texas_Instruments:Texas_DCK0006A_SC-70-6_1.25x2mm_P0.65mm -> texas-instruments:Texas_DCK0006A_SC-70-6_1.25x2mm_P0.65mm; symbol Texas_Instruments:SN74LVC1G58DCKR -> texas-instruments:SN74LVC1G58DCKR
Changed lines of the file:
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@@
 (paper "A3")
 (title_block (title "MaskROM entry") (date "2026-10-25") (rev "A") (company "The OpenDAP Project") (comment 1 "blk.maskrom") (comment 2 "Power + Vol- at power-on pull eMMC D0 low inside a boot window: TPS3808, two gates, BAT54, FET"))
-(symbol (lib_id "Texas_Instruments:TPS3808G01DBVR") (at 54.61 60.96 0) (unit 1) (body_style 1) (exclude_from_sim no) (in_bom yes) (on_board yes) (dnp no)
+(symbol (lib_id "texas-instruments:TPS3808G01DBVR") (at 54.61 60.96 0) (unit 1) (body_style 1) (exclude_from_sim no) (in_bom yes) (on_board yes) (dnp no)
   (property "Reference" "U4101" (at 55.88 45.72 0) (effects (font (size 1.27 1.27)) (justify left)))
   (property "Value" "TPS3808G01DBVR" (at 55.88 43.18 0) (effects (font (size 1.27 1.27)) (justify left)))
-  (property "Footprint" "Texas_Instruments:Texas_DBV0006A_SOT-23-6_1.6x2.9mm_P0.95mm" (at 54.61 60.96 0) (effects (font (size 1.27 1.27))) (hide yes))
+  (property "Footprint" "texas-instruments:Texas_DBV0006A_SOT-23-6_1.6x2.9mm_P0.95mm" (at 54.61 60.96 0) (effects (font (size 1.27 1.27))) (hide yes))
   (property "Datasheet" "https://www.ti.com/lit/ds/symlink/tps3808.pdf" (at 54.61 60.96 0) (effects (font (size 1.27 1.27))) (hide yes))
   (property "Description" "Voltage supervisor, adjustable threshold (0.405 V SENSE), programmable reset delay (CT), manual reset, open-drain active-low RESET, 1.7-6.5 V, SOT-23-6 (DBV0006A)" (at 54.61 60.96 0) (effects (font (size 1.27 1.27))) (hide yes))
@@
 (rectangle (start 22.86 35.56) (end 147.32 115.57) (stroke (width 0) (type dash)) (fill (type none)))
 (text "Boot window: TPS3808G01, 1.21-3.43 s (BOM v1 line 97)" (exclude_from_sim no) (at 24.13 34.29 0) (effects (font (size 2.54 2.54)) (justify left bottom)))
-(symbol (lib_id "Texas_Instruments:SN74LVC1G57DCKR") (at 184.15 60.96 0) (unit 1) (body_style 1) (exclude_from_sim no) (in_bom yes) (on_board yes) (dnp no)
+(symbol (lib_id "texas-instruments:SN74LVC1G57DCKR") (at 184.15 60.96 0) (unit 1) (body_style 1) (exclude_from_sim no) (in_bom yes) (on_board yes) (dnp no)
   (property "Reference" "U4102" (at 185.42 45.72 0) (effects (font (size 1.27 1.27)) (justify left)))
   (property "Value" "SN74LVC1G57DCKR" (at 185.42 43.18 0) (effects (font (size 1.27 1.27)) (justify left)))
-  (property "Footprint" "Texas_Instruments:Texas_DCK0006A_SC-70-6_1.25x2mm_P0.65mm" (at 184.15 60.96 0) (effects (font (size 1.27 1.27))) (hide yes))
+  (property "Footprint" "texas-instruments:Texas_DCK0006A_SC-70-6_1.25x2mm_P0.65mm" (at 184.15 60.96 0) (effects (font (size 1.27 1.27))) (hide yes))
   (property "Datasheet" "https://www.ti.com/lit/ds/symlink/sn74lvc1g57.pdf" (at 184.15 60.96 0) (effects (font (size 1.27 1.27))) (hide yes))
   (property "Description" "Configurable multiple-function gate (AND, OR, NAND, NOR, XNOR, inverter, buffer by wiring), Schmitt-trigger inputs, 1.65-5.5 V, Ioff, SOT/SC-70-6 (DCK0006A)" (at 184.15 60.96 0) (effects (font (size 1.27 1.27))) (hide yes))
@@
 (rectangle (start 152.4 35.56) (end 245.11 87.63) (stroke (width 0) (type dash)) (fill (type none)))
 (text "Both keys: SN74LVC1G57 (BOM v1 line 98)" (exclude_from_sim no) (at 153.67 34.29 0) (effects (font (size 2.54 2.54)) (justify left bottom)))
-(symbol (lib_id "Nexperia:BAT54") (at 276.86 53.34 0) (unit 1) (body_style 1) (exclude_from_sim no) (in_bom yes) (on_board yes) (dnp no)
+(symbol (lib_id "nexperia:BAT54") (at 276.86 53.34 0) (unit 1) (body_style 1) (exclude_from_sim no) (in_bom yes) (on_board yes) (dnp no)
   (property "Reference" "D4101" (at 271.78 43.18 0) (effects (font (size 1.27 1.27)) (justify left)))
   (property "Value" "BAT54" (at 271.78 40.64 0) (effects (font (size 1.27 1.27)) (justify left)))
-  (property "Footprint" "Nexperia:Nexperia_SOT23_TO-236AB_2.9x1.3mm_P1.9mm" (at 276.86 53.34 0) (effects (font (size 1.27 1.27))) (hide yes))
+  (property "Footprint" "nexperia:Nexperia_SOT23_TO-236AB_2.9x1.3mm_P1.9mm" (at 276.86 53.34 0) (effects (font (size 1.27 1.27))) (hide yes))
   (property "Datasheet" "https://assets.nexperia.com/documents/data-sheet/BAT54_SER.pdf" (at 276.86 53.34 0) (effects (font (size 1.27 1.27))) (hide yes))
   (property "Description" "Schottky barrier diode, single, 30 V, 200 mA, VF 320 mV max at 1 mA, SOT23 (TO-236AB)" (at 276.86 53.34 0) (effects (font (size 1.27 1.27))) (hide yes))
@@
 (rectangle (start 250.19 35.56) (end 342.9 63.5) (stroke (width 0) (type dash)) (fill (type none)))
 (text "PWRON isolation: BAT54 (BOM v1 line 78)" (exclude_from_sim no) (at 251.46 34.29 0) (effects (font (size 2.54 2.54)) (justify left bottom)))
-(symbol (lib_id "Texas_Instruments:SN74LVC1G58DCKR") (at 64.77 151.13 0) (unit 1) (body_style 1) (exclude_from_sim no) (in_bom yes) (on_board yes) (dnp no)
+(symbol (lib_id "texas-instruments:SN74LVC1G58DCKR") (at 64.77 151.13 0) (unit 1) (body_style 1) (exclude_from_sim no) (in_bom yes) (on_board yes) (dnp no)
   (property "Reference" "U4103" (at 66.04 135.89 0) (effects (font (size 1.27 1.27)) (justify left)))
   (property "Value" "SN74LVC1G58DCKR" (at 66.04 133.35 0) (effects (font (size 1.27 1.27)) (justify left)))
-  (property "Footprint" "Texas_Instruments:Texas_DCK0006A_SC-70-6_1.25x2mm_P0.65mm" (at 64.77 151.13 0) (effects (font (size 1.27 1.27))) (hide yes))
+  (property "Footprint" "texas-instruments:Texas_DCK0006A_SC-70-6_1.25x2mm_P0.65mm" (at 64.77 151.13 0) (effects (font (size 1.27 1.27))) (hide yes))
   (property "Datasheet" "https://www.ti.com/lit/ds/symlink/sn74lvc1g58.pdf" (at 64.77 151.13 0) (effects (font (size 1.27 1.27))) (hide yes))
   (property "Description" "Configurable multiple-function gate (AND, OR, NAND, NOR, XOR, inverter, buffer by wiring), Schmitt-trigger inputs, 1.65-5.5 V, Ioff, SOT/SC-70-6 (DCK0006A)" (at 64.77 151.13 0) (effects (font (size 1.27 1.27))) (hide yes))
