File: board/hardware/t1-main-board/mic-ambient.kicad_sch (KiCad schematic)
At the start: 7 parts

Commit message: Board on libs v0.2.0: lower-case kebab vendor keys (HL-13)
The libs submodule moves to v0.2.0 (5f24483). Every library nickname in
the generator, the placement tool and the floorplan study follows the
key table (Texas_Instruments -> texas-instruments, OpenDAP_Device ->
opendap-generic, Rockchip and Rockchip_PMIC -> rockchip, ...); the
library tables are written from the files. Schematic and board
regenerated.

Checks: ERC 0 errors (warnings unchanged); DRC 0 errors, 605 warnings,
the same counts by type, schematic parity 0; every placement identical;
craft Q1 met; pcb tests pass; STEP export resolves every libs 3D model
(the 27 parts without a model are KiCad stock lands that have none).

Co-Authored-By: Claude Opus 5.5 <noreply@anthropic.com>
Claude-Session: https://claude.ai/code/session_01Ei262h3TpgY9vyfNLMi5Mn
Parts:
- MK3901: footprint Infineon:Infineon_PG-LLGA-5-3_3x4mm_P0.7mm_BottomPort -> infineon:Infineon_PG-LLGA-5-3_3x4mm_P0.7mm_BottomPort; symbol Infineon:IM73D122V01XTMA1 -> infineon:IM73D122V01XTMA1
Changed lines of the file:
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@@
 (paper "A4")
 (title_block (title "Ambient microphone") (date "2026-10-25") (rev "A") (company "The OpenDAP Project") (comment 1 "blk.mic-ambient") (comment 2 "IM73D122 PDM microphone on PDM CLK1 and SDI1, on its own MIC_1V8 branch (link #35)"))
-(symbol (lib_id "Infineon:IM73D122V01XTMA1") (at 52.07 69.85 0) (unit 1) (body_style 1) (exclude_from_sim no) (in_bom yes) (on_board yes) (dnp no)
+(symbol (lib_id "infineon:IM73D122V01XTMA1") (at 52.07 69.85 0) (unit 1) (body_style 1) (exclude_from_sim no) (in_bom yes) (on_board yes) (dnp no)
   (property "Reference" "MK3901" (at 53.34 54.61 0) (effects (font (size 1.27 1.27)) (justify left)))
   (property "Value" "IM73D122V01XTMA1" (at 53.34 52.07 0) (effects (font (size 1.27 1.27)) (justify left)))
-  (property "Footprint" "Infineon:Infineon_PG-LLGA-5-3_3x4mm_P0.7mm_BottomPort" (at 52.07 69.85 0) (effects (font (size 1.27 1.27))) (hide yes))
+  (property "Footprint" "infineon:Infineon_PG-LLGA-5-3_3x4mm_P0.7mm_BottomPort" (at 52.07 69.85 0) (effects (font (size 1.27 1.27))) (hide yes))
   (property "Datasheet" "https://www.infineon.com/assets/row/public/documents/24/49/infineon-im73d122-datasheet-en.pdf" (at 52.07 69.85 0) (effects (font (size 1.27 1.27))) (hide yes))
   (property "Description" "Digital PDM MEMS microphone, bottom port, 73 dB(A) SNR, -26 dBFS, 122 dBSPL AOP, 1.62-3.6 V, PG-LLGA-5-3 (4 x 3 x 1.2 mm)" (at 52.07 69.85 0) (effects (font (size 1.27 1.27))) (hide yes))

Commit message: Board in the 62.5 x 95.0 mm body: ADR 0025, outline 59.1 x 91.6, 0201 swaps
ADR 0025 supersedes ADR 0016 for t1 ADR 0006's body: board outline from
the body, 1.2 mm walls and 0.5 mm clearance; height zones and stack
restated unchanged; the speaker on a case shelf (PCB-Z-09); pocket
reliefs at the 4.4 mm jack, the microSD (DM3AT push-push kept) and the
side buttons; the audio 0603 -> 0402 swap gated by t1 V2-A08; reserve
(NFC reader, then TPM) recorded, not applied.

- pcb/geometry.py derives the outline from BODY, WALL and CLEARANCE;
  the pocket, display and fixed parts keep their device-frame positions;
  holes keep their edge distance; the speaker shadow becomes a 1.5 mm
  shelf height area (placement, checks, occupancy).
- build.py reports pocket reliefs and routing room; C904 unfixed (it
  now finds back room, so PCB-Z-04 carries no part).
- Generator: parts.area_swap puts 121 generic 0402 resistors (outside
  audio and VBUS paths, >= 10 ohm) and five 100 nF signal capacitors in
  0201 (BOM v1.16); schematic and board regenerated.
- Result: 1,012/1,012 placed, 98.8 % by the floorplan method (was 111 %),
  factor left 1.68 (was 1.49); DRC 0 errors, ERC 0 errors, 0 check
  findings, pcb tests 20/20, schematic craft Q1 met.
- Specs: PCB constraints v0.17 (M-01, M-02, M-08, Z-02, Z-06 to Z-09,
  R-07), placement v1.1 (section 3, decisions 4 and 13, checks, open
  items with the gated swaps and the reserve), floorplan v1 section 1,
  BOM v1.16.

Co-Authored-By: Claude Opus 5.5 <noreply@anthropic.com>
Claude-Session: https://claude.ai/code/session_01Ei262h3TpgY9vyfNLMi5Mn
Parts:
- R3902: footprint Resistor_SMD:R_0402_1005Metric -> Resistor_SMD:R_0201_0603Metric; MPN RC0402FR-0722RL -> RC0201FR-0722RL
Changed lines of the file:
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@@
   (property "Reference" "R3902" (at 168.91 78.74 90) (effects (font (size 1.27 1.27))))
   (property "Value" "22 Ω" (at 168.91 83.82 90) (effects (font (size 1.27 1.27))))
-  (property "Footprint" "Resistor_SMD:R_0402_1005Metric" (at 168.91 81.28 0) (effects (font (size 1.27 1.27))) (hide yes))
-  (property "Datasheet" "https://yageogroup.com/en/ProductSearch/PartNumberSearch?part=RC0402FR-0722RL" (at 168.91 81.28 0) (effects (font (size 1.27 1.27))) (hide yes))
-  (property "Description" "Resistor, 22 Ω, 1 %, 1/16 W, 0402" (at 168.91 81.28 0) (effects (font (size 1.27 1.27))) (hide yes))
+  (property "Footprint" "Resistor_SMD:R_0201_0603Metric" (at 168.91 81.28 0) (effects (font (size 1.27 1.27))) (hide yes))
+  (property "Datasheet" "https://yageogroup.com/en/ProductSearch/PartNumberSearch?part=RC0201FR-0722RL" (at 168.91 81.28 0) (effects (font (size 1.27 1.27))) (hide yes))
+  (property "Description" "Resistor, 22 Ω, 1 %, 1/20 W, 0201" (at 168.91 81.28 0) (effects (font (size 1.27 1.27))) (hide yes))
   (property "Manufacturer" "YAGEO" (at 168.91 81.28 0) (effects (font (size 1.27 1.27))) (hide yes))
-  (property "MPN" "RC0402FR-0722RL" (at 168.91 81.28 0) (effects (font (size 1.27 1.27))) (hide yes))
+  (property "MPN" "RC0201FR-0722RL" (at 168.91 81.28 0) (effects (font (size 1.27 1.27))) (hide yes))
   (property "Block" "blk.mic-ambient" (at 168.91 81.28 0) (effects (font (size 1.27 1.27))) (hide yes))
   (pin "1")

Commit message: BOM v1.18 item 2: successors of the discontinued 1 uF 0402
GRM155R61A105KE15D is to be discontinued. 44 positions take
GRM155C71A105KE11D (1 uF 10 V X7S); the eight TPS7A20 positions take
GRM155R61C225KE11D (2.2 uF 16 V X5R) to keep the 0.47 uF effective
minimum with 10 % to spare at up to 3.8 V. Same land; sourcing pass.
Closes BOM §7 item 52; new item 55 lists the other capture parts outside
Murata's product data or near end of life.

Co-Authored-By: Claude Opus 5.5 <noreply@anthropic.com>
Claude-Session: https://claude.ai/code/session_01Ei262h3TpgY9vyfNLMi5Mn
Parts:
- C3901: MPN GRM155R61A105KE15D -> GRM155C71A105KE11D
Changed lines of the file:
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@@
   (property "Value" "1 µF" (at 83.82 59.69 0) (effects (font (size 1.27 1.27)) (justify left)))
   (property "Footprint" "Capacitor_SMD:C_0402_1005Metric" (at 81.28 58.42 0) (effects (font (size 1.27 1.27))) (hide yes))
-  (property "Datasheet" "https://www.murata.com/en-us/products/productdetail?partno=GRM155R61A105KE15D" (at 81.28 58.42 0) (effects (font (size 1.27 1.27))) (hide yes))
-  (property "Description" "Capacitor, 1 µF, 10 V, X5R, 0402" (at 81.28 58.42 0) (effects (font (size 1.27 1.27))) (hide yes))
+  (property "Datasheet" "https://www.murata.com/en-us/products/productdetail?partno=GRM155C71A105KE11D" (at 81.28 58.42 0) (effects (font (size 1.27 1.27))) (hide yes))
+  (property "Description" "Capacitor, 1 µF, 10 V, X7S, 0402" (at 81.28 58.42 0) (effects (font (size 1.27 1.27))) (hide yes))
   (property "Manufacturer" "Murata" (at 81.28 58.42 0) (effects (font (size 1.27 1.27))) (hide yes))
-  (property "MPN" "GRM155R61A105KE15D" (at 81.28 58.42 0) (effects (font (size 1.27 1.27))) (hide yes))
+  (property "MPN" "GRM155C71A105KE11D" (at 81.28 58.42 0) (effects (font (size 1.27 1.27))) (hide yes))
   (property "Block" "blk.mic-ambient" (at 81.28 58.42 0) (effects (font (size 1.27 1.27))) (hide yes))
   (pin "1")
