File: board/hardware/t1-main-board/t1-main-board.kicad_pcb (KiCad board)
At the start: 6 copper layers, 59.1 x 91.6 mm, 1005 parts, among them J3401 SJ2-35954D-SMT-TR, J4001 GT-3321667P-01, J4601 USB4105-GF-A, J4701 DF40C-50DS-0.4V(51), J5201 U.FL-R-SMT-1, J5202 U.FL-R-SMT-1, J5301 FH35C-51S-0.3SHW, J6201 DM3AT-SF-PEJM5, J701 70-9258-001-120-006, J702 70-9258-001-120-006, J703 70-9258-001-120-006, J704 70-9258-001-120-006, J705 70-9258-001-120-006, J706 70-9258-001-120-006, Q2801 DMG1012T, Q2802 DMP3099L, Q3501 DMG1012T, Q4101 DMG1012T, Q4801 DMG1012T, Q701 CSD17575Q3, SW6901 PTS815, SW6902 PTS815, SW6903 PTS815, SW6904 Action (part open), U1001 TPS62827DMQR, U1101 RK809-5, U1201 TPS62870Z4WRXSR, U1301 RK3566, U1302 SN74LVC2G66DCUR, U2101 MT53E1G32D2FW-046, U2102 TPS7A1006PDSER, U2301 TPS22916CYFPR, U2302 TPS22916CYFPR, U2303 TPS62840DLCR, U2401 SN74LVC1G57DCKR, U2402 TPS7A2031PDBVR, U2403 TPS7A2018PDBVR, U2404 SN74AUC1G74DCUR, U2405 SN74AUC1G74DCUR, U2501 CS43198-CNZR, U2502 TPS7A2018PDBVR, U2601 CS43198-CNZR, U2602 TPS7A2018PDBVR, U2801 TPS65131RGER, U2802 LMR33630CRNXR, U2901 LT3045EDD, U2902 LT3045EDD, U2903 LT3094EDD, U2904 LT3094EDD, U3001 OPA1622IDRCR, U3002 OPA1622IDRCR, U3201 OPA1622IDRCR, U3202 OPA1622IDRCR, U3301 OPA1622IDRCR, U3302 OPA1622IDRCR, U3501 RP2354A, U3502 TPS22916CYFPR, U3503 TPS22916CYFPR, U3801 KLMBG2JETD-B041, U4101 TPS3808G01DBVR, U4102 SN74LVC1G57DCKR, U4103 SN74LVC1G58DCKR, U4201 INA236AIDDFR, U4202 INA236AIDDFR, U4203 INA236AIDDFR, U4204 INA236AIDDFR, U4205 INA236BIDDFR, U4401 TPS62903RPJR, U4501 TPS259470ARPWR, U4502 TPS259470ARPWR, U4601 TVS2200DRVR, U4602 TPD8S300ARUKR, U4603 TPD4E05U06DQAR, U4604 FUSB302BMPX, U4801 TPS259470ARPWR, U4802 FUSB302B01MPX, U5001 LBES5PL2EL-923, U501 TPS2121RUXR, U5101 SN74AXC1T45DCKR, U5102 TPS22916CYFPR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

Commit message: Board: faceplate DSI ESD captured, FP_GPIO1 on a single TPD1E10B06 (BOM v1.21)
Line 72's three TPD4E05U06 stand on blk.fp-connector next to the FH35C
contacts (U5306-U5308, one pair per two channels); the sixth low-speed
array, one channel used, becomes one TPD1E10B06 (sourcing check passed).
Catalog records 21 and 22 follow; placement rebuilt (need 99.2 %).

Co-Authored-By: Claude Opus 5.5 <noreply@anthropic.com>
Claude-Session: https://claude.ai/code/session_013P6pW9LdyEMFishwCcZGUr
Parts:
- removed the D5801 at (127.7, 114.0)
- added D5301: TPD1E10B06, Package_SON:Texas_DPY0002A_0.6x1mm_P0.65mm, F.Cu at (93.0, 132.2)
- added D6901: TPD1E10B06, Package_SON:Texas_DPY0002A_0.6x1mm_P0.65mm, F.Cu at (128.7, 72.8)
- added U5309: TPS22950YBHR, texas-instruments:Texas_YBH0006_DSBGA-6_0.706x1.106mm_Layout2x3_P0.4mm, F.Cu at (97.2, 111.2)
- added U5310: TPS22945DCKR, texas-instruments:Texas_DCK0005A_SC-70-5_1.25x2mm_P0.65mm, B.Cu at (96.1, 111.9)
- R5301: value 10 kΩ -> 3.57 kΩ
- R5302: moved to F.Cu
- R5303: value 100 kΩ -> 100 mΩ; footprint Resistor_SMD:R_0201_0603Metric -> Resistor_SMD:R_0603_1608Metric; moved to F.Cu
- R5304: value 3.57 kΩ -> 1 Ω; footprint Resistor_SMD:R_0201_0603Metric -> Resistor_SMD:R_0603_1608Metric
- R5305: value 100 kΩ -> 10 kΩ; moved to B.Cu
- R5306: value 100 mΩ -> 10 kΩ; footprint Resistor_SMD:R_0603_1608Metric -> Resistor_SMD:R_0201_0603Metric
- R5307: value 1 Ω -> 100 kΩ; footprint Resistor_SMD:R_0603_1608Metric -> Resistor_SMD:R_0201_0603Metric; moved to B.Cu
- R5308: value 10 kΩ -> 100 kΩ
- U5307: value TPS22950YBHR -> TPD4E05U06DQAR; footprint texas-instruments:Texas_YBH0006_DSBGA-6_0.706x1.106mm_Layout2x3_P0.4mm -> texas-instruments:Texas_DQA0010A_USON-10_1x2.5mm_P0.5mm
- U5308: value TPS22945DCKR -> TPD4E05U06DQAR; footprint texas-instruments:Texas_DCK0005A_SC-70-5_1.25x2mm_P0.65mm -> texas-instruments:Texas_DQA0010A_USON-10_1x2.5mm_P0.5mm; moved to F.Cu
- moved D5801 41.3 mm to (127.7, 114.0), turned to 0 degrees
- moved U5308 30.2 mm to (106.5, 140.2), turned to 90 degrees
- moved U5307 29.0 mm to (108.0, 138.2)
- moved R5302 23.4 mm to (97.0, 113.5), turned to 0 degrees
- moved R5303 17.8 mm to (97.2, 120.7), turned to 0 degrees
- moved R5307 14.9 mm to (94.2, 136.8), turned to 90 degrees
- moved R5301 14.5 mm to (97.5, 109.0)
- moved R5304 13.3 mm to (97.9, 122.3)
- moved U5306 9.58 mm to (107.8, 136.2)
- moved R5308 9.25 mm to (94.6, 125.8)
- moved R5305 3.94 mm to (94.5, 116.5), turned to 90 degrees
- moved R5306 2.80 mm to (97.2, 123.5)
- renumbered D6901 to D5801
Connections:
- D5801 pad 2: /PWRON_N -> /COVER_DET_N
- R5301 pad 1: vcc3v3_sys -> /Faceplate connector/FP3V3_ILIM
- R5301 pad 2: /FP_DET_N -> GND
- R5302 pad 1: /FP_GPIO0 -> /FP_IO_EN
- R5303 pad 1: /FP_GPIO1 -> /Faceplate connector/FP_3V3_SRC
- R5303 pad 2: GND -> FP_3V3
- R5304 pad 1: /Faceplate connector/FP3V3_ILIM -> /Faceplate connector/FP_1V8_SRC
- R5304 pad 2: GND -> FP_1V8
- R5305 pad 1: /FP_IO_EN -> /Faceplate connector/FP_1V8_SRC
- R5306 pad 1: /Faceplate connector/FP_3V3_SRC -> vcc3v3_sys
- R5306 pad 2: FP_3V3 -> /FP_DET_N
- R5307 pad 1: /Faceplate connector/FP_1V8_SRC -> /FP_GPIO0
- R5307 pad 2: FP_1V8 -> GND
- R5308 pad 1: /Faceplate connector/FP_1V8_SRC -> /FP_GPIO1
- U5306 pad 1: /FP_GPIO1 -> /FP_DSI_D0_P
- U5306 pad 2: unconnected-(U5306-D1--Pad2) -> /FP_DSI_D0_N
- U5306 pad 4: unconnected-(U5306-D2+-Pad4) -> /FP_DSI_D1_P
- U5306 pad 5: unconnected-(U5306-D2--Pad5) -> /FP_DSI_D1_N
- U5308 pad 1: /Faceplate connector/FP_1V8_SRC -> /FP_DSI_CLK_P
- U5308 pad 2: GND -> /FP_DSI_CLK_N
- U5308 pad 3: unconnected-(U5308-OC-Pad3) -> GND
- U5308 pad 4: /FP_IO_EN -> unconnected-(U5308-D2+-Pad4)
- U5308 pad 5: vcc_1v8 -> unconnected-(U5308-D2--Pad5)

Commit message: Board: test pads on either side for flying-probe test (ADR 0027)
Prototypes and first runs are tested by flying probe, so flat test pads
may stand on the back where their net's zone allows (placement v1.8
decision 9 revised, new PCB-D-11, plan.TEST_PAD_SIDES). 18 of 156 pads
take the back; the placer refills the front cells with passives, so the
front courtyard (about 2,800 mm2) and the board need (99.2 %) do not
change. Placement v1.8 also places the DSI ESD of BOM v1.21.

Co-Authored-By: Claude Opus 5.5 <noreply@anthropic.com>
Claude-Session: https://claude.ai/code/session_013P6pW9LdyEMFishwCcZGUr
Parts:
- C2513, C3203, C3301, C3503, C3902, C5402, NT3402, R1323, R1326, R2302, R2601, R2603, R2903, R2906, R3308, R3501, R507, R6704, TP1001, TP1101, TP2301, TP2303, TP2403, TP2404, TP2601, TP3102, TP3104, TP3505, TP4344, TP4349, TP4350, TP4353, TP4501, TP5303, TP6503, TP6602: moved to B.Cu
- C2910, C2923, C3201, C3204, C3208, C3308, C3309, C3510, C602, C603, NT2901, NT2904, R1314, R1315, R1319, R1322, R1325, R1329, R2403, R2404, R2802, R2803, R2904, R2907, R3206, R3217, R3309, R3504, R3512, R3902, R4501, R503, R504, R505, R506, R5305, R5502, R6002, R603, R604, R6502, R6801: moved to F.Cu
- moved R3219 44.5 mm to (77.5, 88.5)
- moved R3214 41.3 mm to (77.5, 90.0)
- moved R3211 41.1 mm to (88.0, 132.8), turned to 0 degrees
- moved R3215 40.8 mm to (77.6, 130.8)
- moved R3207 40.6 mm to (88.0, 130.4), turned to 90 degrees
- moved R3216 40.4 mm to (74.2, 130.3)
- moved R3209 39.6 mm to (77.8, 126.5), turned to 90 degrees
- moved R3204 38.8 mm to (90.3, 129.8), turned to 0 degrees
- moved R3217 38.3 mm to (74.4, 90.0)
- moved R3203 37.8 mm to (88.5, 127.3)
- moved R3212 37.8 mm to (77.3, 129.2)
- moved R3213 34.9 mm to (72.8, 92.0), turned to 0 degrees
- moved R3512 27.9 mm to (76.1, 84.5)
- moved C3507 27.4 mm to (74.8, 81.0), turned to 90 degrees
- moved C3506 27.2 mm to (74.5, 79.5), turned to 90 degrees
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