File: board/hardware/t1-main-board/gauge.kicad_sch (KiCad schematic)
At the start: 16 parts, among them U801 BQ28Z610DRZR-R1

Commit message: Board on libs v0.2.0: lower-case kebab vendor keys (HL-13)
The libs submodule moves to v0.2.0 (5f24483). Every library nickname in
the generator, the placement tool and the floorplan study follows the
key table (Texas_Instruments -> texas-instruments, OpenDAP_Device ->
opendap-generic, Rockchip and Rockchip_PMIC -> rockchip, ...); the
library tables are written from the files. Schematic and board
regenerated.

Checks: ERC 0 errors (warnings unchanged); DRC 0 errors, 605 warnings,
the same counts by type, schematic parity 0; every placement identical;
craft Q1 met; pcb tests pass; STEP export resolves every libs 3D model
(the 27 parts without a model are KiCad stock lands that have none).

Co-Authored-By: Claude Opus 5.5 <noreply@anthropic.com>
Claude-Session: https://claude.ai/code/session_01Ei262h3TpgY9vyfNLMi5Mn
Parts:
- RT801: symbol OpenDAP_Device:Thermistor_NTC -> opendap-generic:Thermistor_NTC
- U801: footprint Texas_Instruments:VSON-12-1EP_4x2.5mm_P0.4mm_EP2.45x1.95mm_ThermalVias -> texas-instruments:VSON-12-1EP_4x2.5mm_P0.4mm_EP2.45x1.95mm_ThermalVias; symbol Texas_Instruments:BQ28Z610DRZR-R1 -> texas-instruments:BQ28Z610DRZR-R1
Changed lines of the file:
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@@
 (paper "A3")
 (title_block (title "Fuel gauge") (date "2026-10-25") (rev "A") (company "The OpenDAP Project") (comment 1 "blk.gauge") (comment 2 "BQ28Z610-R1 on the pack side, its 3 mΩ sense resistor and board NTC (ADR 0017)"))
-(symbol (lib_id "Texas_Instruments:BQ28Z610DRZR-R1") (at 52.07 77.47 0) (unit 1) (body_style 1) (exclude_from_sim no) (in_bom yes) (on_board yes) (dnp no)
+(symbol (lib_id "texas-instruments:BQ28Z610DRZR-R1") (at 52.07 77.47 0) (unit 1) (body_style 1) (exclude_from_sim no) (in_bom yes) (on_board yes) (dnp no)
   (property "Reference" "U801" (at 55.88 53.34 0) (effects (font (size 1.27 1.27)) (justify left)))
   (property "Value" "BQ28Z610DRZR-R1" (at 55.88 50.8 0) (effects (font (size 1.27 1.27)) (justify left)))
-  (property "Footprint" "Texas_Instruments:VSON-12-1EP_4x2.5mm_P0.4mm_EP2.45x1.95mm_ThermalVias" (at 52.07 77.47 0) (effects (font (size 1.27 1.27))) (hide yes))
+  (property "Footprint" "texas-instruments:VSON-12-1EP_4x2.5mm_P0.4mm_EP2.45x1.95mm_ThermalVias" (at 52.07 77.47 0) (effects (font (size 1.27 1.27))) (hide yes))
   (property "Datasheet" "https://www.ti.com/lit/ds/symlink/bq28z610-r1.pdf" (at 52.07 77.47 0) (effects (font (size 1.27 1.27))) (hide yes))
   (property "Description" "Impedance Track gas gauge and protection controller for 1-2 series Li-ion packs, high-side N-FET drive, cell balancing, I2C, VSON-12 (DRZ) 4 x 2.5 mm" (at 52.07 77.47 0) (effects (font (size 1.27 1.27))) (hide yes))
@@
 )
 (wire (pts (xy 113.03 90.17) (xy 113.03 87.63)) (stroke (width 0) (type default)))
-(symbol (lib_id "OpenDAP_Device:Thermistor_NTC") (at 130.81 93.98 0) (unit 1) (body_style 1) (exclude_from_sim no) (in_bom yes) (on_board yes) (dnp no)
+(symbol (lib_id "opendap-generic:Thermistor_NTC") (at 130.81 93.98 0) (unit 1) (body_style 1) (exclude_from_sim no) (in_bom yes) (on_board yes) (dnp no)
   (property "Reference" "RT801" (at 133.35 92.71 0) (effects (font (size 1.27 1.27)) (justify left)))
   (property "Value" "10 kΩ" (at 133.35 95.25 0) (effects (font (size 1.27 1.27)) (justify left)))

Commit message: Board in the 62.5 x 95.0 mm body: ADR 0025, outline 59.1 x 91.6, 0201 swaps
ADR 0025 supersedes ADR 0016 for t1 ADR 0006's body: board outline from
the body, 1.2 mm walls and 0.5 mm clearance; height zones and stack
restated unchanged; the speaker on a case shelf (PCB-Z-09); pocket
reliefs at the 4.4 mm jack, the microSD (DM3AT push-push kept) and the
side buttons; the audio 0603 -> 0402 swap gated by t1 V2-A08; reserve
(NFC reader, then TPM) recorded, not applied.

- pcb/geometry.py derives the outline from BODY, WALL and CLEARANCE;
  the pocket, display and fixed parts keep their device-frame positions;
  holes keep their edge distance; the speaker shadow becomes a 1.5 mm
  shelf height area (placement, checks, occupancy).
- build.py reports pocket reliefs and routing room; C904 unfixed (it
  now finds back room, so PCB-Z-04 carries no part).
- Generator: parts.area_swap puts 121 generic 0402 resistors (outside
  audio and VBUS paths, >= 10 ohm) and five 100 nF signal capacitors in
  0201 (BOM v1.16); schematic and board regenerated.
- Result: 1,012/1,012 placed, 98.8 % by the floorplan method (was 111 %),
  factor left 1.68 (was 1.49); DRC 0 errors, ERC 0 errors, 0 check
  findings, pcb tests 20/20, schematic craft Q1 met.
- Specs: PCB constraints v0.17 (M-01, M-02, M-08, Z-02, Z-06 to Z-09,
  R-07), placement v1.1 (section 3, decisions 4 and 13, checks, open
  items with the gated swaps and the reserve), floorplan v1 section 1,
  BOM v1.16.

Co-Authored-By: Claude Opus 5.5 <noreply@anthropic.com>
Claude-Session: https://claude.ai/code/session_01Ei262h3TpgY9vyfNLMi5Mn
Parts:
- R801, R804, R805, R806, R807: footprint Resistor_SMD:R_0402_1005Metric -> Resistor_SMD:R_0201_0603Metric; MPN RC0402FR-07100RL -> RC0201FR-07100RL
- R803: footprint Resistor_SMD:R_0402_1005Metric -> Resistor_SMD:R_0201_0603Metric; MPN RC0402FR-0710RL -> RC0201FR-0710RL
Changed lines of the file:
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@@
   (property "Reference" "R801" (at 167.64 43.18 90) (effects (font (size 1.27 1.27))))
   (property "Value" "100 Ω" (at 167.64 48.26 90) (effects (font (size 1.27 1.27))))
-  (property "Footprint" "Resistor_SMD:R_0402_1005Metric" (at 167.64 45.72 0) (effects (font (size 1.27 1.27))) (hide yes))
-  (property "Datasheet" "https://yageogroup.com/en/ProductSearch/PartNumberSearch?part=RC0402FR-07100RL" (at 167.64 45.72 0) (effects (font (size 1.27 1.27))) (hide yes))
-  (property "Description" "Resistor, 100 Ω, 1 %, 1/16 W, 0402" (at 167.64 45.72 0) (effects (font (size 1.27 1.27))) (hide yes))
+  (property "Footprint" "Resistor_SMD:R_0201_0603Metric" (at 167.64 45.72 0) (effects (font (size 1.27 1.27))) (hide yes))
+  (property "Datasheet" "https://yageogroup.com/en/ProductSearch/PartNumberSearch?part=RC0201FR-07100RL" (at 167.64 45.72 0) (effects (font (size 1.27 1.27))) (hide yes))
+  (property "Description" "Resistor, 100 Ω, 1 %, 1/20 W, 0201" (at 167.64 45.72 0) (effects (font (size 1.27 1.27))) (hide yes))
   (property "Manufacturer" "YAGEO" (at 167.64 45.72 0) (effects (font (size 1.27 1.27))) (hide yes))
-  (property "MPN" "RC0402FR-07100RL" (at 167.64 45.72 0) (effects (font (size 1.27 1.27))) (hide yes))
+  (property "MPN" "RC0201FR-07100RL" (at 167.64 45.72 0) (effects (font (size 1.27 1.27))) (hide yes))
   (property "Block" "blk.gauge" (at 167.64 45.72 0) (effects (font (size 1.27 1.27))) (hide yes))
   (pin "1")
@@
   (property "Reference" "R803" (at 167.64 68.58 90) (effects (font (size 1.27 1.27))))
   (property "Value" "10 Ω" (at 167.64 73.66 90) (effects (font (size 1.27 1.27))))
-  (property "Footprint" "Resistor_SMD:R_0402_1005Metric" (at 167.64 71.12 0) (effects (font (size 1.27 1.27))) (hide yes))
-  (property "Datasheet" "https://yageogroup.com/en/ProductSearch/PartNumberSearch?part=RC0402FR-0710RL" (at 167.64 71.12 0) (effects (font (size 1.27 1.27))) (hide yes))
-  (property "Description" "Resistor, 10 Ω, 1 %, 1/16 W, 0402" (at 167.64 71.12 0) (effects (font (size 1.27 1.27))) (hide yes))
+  (property "Footprint" "Resistor_SMD:R_0201_0603Metric" (at 167.64 71.12 0) (effects (font (size 1.27 1.27))) (hide yes))
+  (property "Datasheet" "https://yageogroup.com/en/ProductSearch/PartNumberSearch?part=RC0201FR-0710RL" (at 167.64 71.12 0) (effects (font (size 1.27 1.27))) (hide yes))
+  (property "Description" "Resistor, 10 Ω, 1 %, 1/20 W, 0201" (at 167.64 71.12 0) (effects (font (size 1.27 1.27))) (hide yes))
   (property "Manufacturer" "YAGEO" (at 167.64 71.12 0) (effects (font (size 1.27 1.27))) (hide yes))
-  (property "MPN" "RC0402FR-0710RL" (at 167.64 71.12 0) (effects (font (size 1.27 1.27))) (hide yes))
+  (property "MPN" "RC0201FR-0710RL" (at 167.64 71.12 0) (effects (font (size 1.27 1.27))) (hide yes))
   (property "Block" "blk.gauge" (at 167.64 71.12 0) (effects (font (size 1.27 1.27))) (hide yes))
   (pin "1")
@@
   (property "Reference" "R804" (at 167.64 78.74 90) (effects (font (size 1.27 1.27))))
   (property "Value" "100 Ω" (at 167.64 83.82 90) (effects (font (size 1.27 1.27))))
-  (property "Footprint" "Resistor_SMD:R_0402_1005Metric" (at 167.64 81.28 0) (effects (font (size 1.27 1.27))) (hide yes))
-  (property "Datasheet" "https://yageogroup.com/en/ProductSearch/PartNumberSearch?part=RC0402FR-07100RL" (at 167.64 81.28 0) (effects (font (size 1.27 1.27))) (hide yes))
-  (property "Description" "Resistor, 100 Ω, 1 %, 1/16 W, 0402" (at 167.64 81.28 0) (effects (font (size 1.27 1.27))) (hide yes))
+  (property "Footprint" "Resistor_SMD:R_0201_0603Metric" (at 167.64 81.28 0) (effects (font (size 1.27 1.27))) (hide yes))
+  (property "Datasheet" "https://yageogroup.com/en/ProductSearch/PartNumberSearch?part=RC0201FR-07100RL" (at 167.64 81.28 0) (effects (font (size 1.27 1.27))) (hide yes))
+  (property "Description" "Resistor, 100 Ω, 1 %, 1/20 W, 0201" (at 167.64 81.28 0) (effects (font (size 1.27 1.27))) (hide yes))
   (property "Manufacturer" "YAGEO" (at 167.64 81.28 0) (effects (font (size 1.27 1.27))) (hide yes))
-  (property "MPN" "RC0402FR-07100RL" (at 167.64 81.28 0) (effects (font (size 1.27 1.27))) (hide yes))
+  (property "MPN" "RC0201FR-07100RL" (at 167.64 81.28 0) (effects (font (size 1.27 1.27))) (hide yes))
   (property "Block" "blk.gauge" (at 167.64 81.28 0) (effects (font (size 1.27 1.27))) (hide yes))
   (pin "1")
@@
   (property "Reference" "R805" (at 167.64 88.9 90) (effects (font (size 1.27 1.27))))
   (property "Value" "100 Ω" (at 167.64 93.98 90) (effects (font (size 1.27 1.27))))
-  (property "Footprint" "Resistor_SMD:R_0402_1005Metric" (at 167.64 91.44 0) (effects (font (size 1.27 1.27))) (hide yes))
-  (property "Datasheet" "https://yageogroup.com/en/ProductSearch/PartNumberSearch?part=RC0402FR-07100RL" (at 167.64 91.44 0) (effects (font (size 1.27 1.27))) (hide yes))
-  (property "Description" "Resistor, 100 Ω, 1 %, 1/16 W, 0402" (at 167.64 91.44 0) (effects (font (size 1.27 1.27))) (hide yes))
+  (property "Footprint" "Resistor_SMD:R_0201_0603Metric" (at 167.64 91.44 0) (effects (font (size 1.27 1.27))) (hide yes))
+  (property "Datasheet" "https://yageogroup.com/en/ProductSearch/PartNumberSearch?part=RC0201FR-07100RL" (at 167.64 91.44 0) (effects (font (size 1.27 1.27))) (hide yes))
+  (property "Description" "Resistor, 100 Ω, 1 %, 1/20 W, 0201" (at 167.64 91.44 0) (effects (font (size 1.27 1.27))) (hide yes))
   (property "Manufacturer" "YAGEO" (at 167.64 91.44 0) (effects (font (size 1.27 1.27))) (hide yes))
-  (property "MPN" "RC0402FR-07100RL" (at 167.64 91.44 0) (effects (font (size 1.27 1.27))) (hide yes))
+  (property "MPN" "RC0201FR-07100RL" (at 167.64 91.44 0) (effects (font (size 1.27 1.27))) (hide yes))
   (property "Block" "blk.gauge" (at 167.64 91.44 0) (effects (font (size 1.27 1.27))) (hide yes))
   (pin "1")
@@
   (property "Reference" "R806" (at 167.64 99.06 90) (effects (font (size 1.27 1.27))))
   (property "Value" "100 Ω" (at 167.64 104.14 90) (effects (font (size 1.27 1.27))))
-  (property "Footprint" "Resistor_SMD:R_0402_1005Metric" (at 167.64 101.6 0) (effects (font (size 1.27 1.27))) (hide yes))
-  (property "Datasheet" "https://yageogroup.com/en/ProductSearch/PartNumberSearch?part=RC0402FR-07100RL" (at 167.64 101.6 0) (effects (font (size 1.27 1.27))) (hide yes))
-  (property "Description" "Resistor, 100 Ω, 1 %, 1/16 W, 0402" (at 167.64 101.6 0) (effects (font (size 1.27 1.27))) (hide yes))
+  (property "Footprint" "Resistor_SMD:R_0201_0603Metric" (at 167.64 101.6 0) (effects (font (size 1.27 1.27))) (hide yes))
+  (property "Datasheet" "https://yageogroup.com/en/ProductSearch/PartNumberSearch?part=RC0201FR-07100RL" (at 167.64 101.6 0) (effects (font (size 1.27 1.27))) (hide yes))
+  (property "Description" "Resistor, 100 Ω, 1 %, 1/20 W, 0201" (at 167.64 101.6 0) (effects (font (size 1.27 1.27))) (hide yes))
   (property "Manufacturer" "YAGEO" (at 167.64 101.6 0) (effects (font (size 1.27 1.27))) (hide yes))
-  (property "MPN" "RC0402FR-07100RL" (at 167.64 101.6 0) (effects (font (size 1.27 1.27))) (hide yes))
+  (property "MPN" "RC0201FR-07100RL" (at 167.64 101.6 0) (effects (font (size 1.27 1.27))) (hide yes))
   (property "Block" "blk.gauge" (at 167.64 101.6 0) (effects (font (size 1.27 1.27))) (hide yes))
   (pin "1")
@@
   (property "Reference" "R807" (at 167.64 109.22 90) (effects (font (size 1.27 1.27))))
   (property "Value" "100 Ω" (at 167.64 114.3 90) (effects (font (size 1.27 1.27))))
-  (property "Footprint" "Resistor_SMD:R_0402_1005Metric" (at 167.64 111.76 0) (effects (font (size 1.27 1.27))) (hide yes))
-  (property "Datasheet" "https://yageogroup.com/en/ProductSearch/PartNumberSearch?part=RC0402FR-07100RL" (at 167.64 111.76 0) (effects (font (size 1.27 1.27))) (hide yes))
-  (property "Description" "Resistor, 100 Ω, 1 %, 1/16 W, 0402" (at 167.64 111.76 0) (effects (font (size 1.27 1.27))) (hide yes))
+  (property "Footprint" "Resistor_SMD:R_0201_0603Metric" (at 167.64 111.76 0) (effects (font (size 1.27 1.27))) (hide yes))
+  (property "Datasheet" "https://yageogroup.com/en/ProductSearch/PartNumberSearch?part=RC0201FR-07100RL" (at 167.64 111.76 0) (effects (font (size 1.27 1.27))) (hide yes))
+  (property "Description" "Resistor, 100 Ω, 1 %, 1/20 W, 0201" (at 167.64 111.76 0) (effects (font (size 1.27 1.27))) (hide yes))
   (property "Manufacturer" "YAGEO" (at 167.64 111.76 0) (effects (font (size 1.27 1.27))) (hide yes))
-  (property "MPN" "RC0402FR-07100RL" (at 167.64 111.76 0) (effects (font (size 1.27 1.27))) (hide yes))
+  (property "MPN" "RC0201FR-07100RL" (at 167.64 111.76 0) (effects (font (size 1.27 1.27))) (hide yes))
   (property "Block" "blk.gauge" (at 167.64 111.76 0) (effects (font (size 1.27 1.27))) (hide yes))
   (pin "1")

Commit message: Board: pre-PCB schematic items closed with datasheets (BOM v1.22)
Display INA236 to 0x49 (INA236B, A0 = VS): no A0 = SDA strap, so the
address no longer depends on the host's I2C hold time. The 18 WSL
shunts and links on Vishay's doc 30100 lands. 24 MHz crystal NDK
NX3225GA (CL 8 pF) with 2 x 10 pF. Backlight inductor Coilcraft
XFL3012-223MEC on its published land (no placeholder left). Action
button PTS815 G code on the side-button land. Cover-detect leakage,
TPS3808 spread, RP2354A supply pins and the USB series scheme closed
without change. Placement v1.9: 100.2 % need, factor 1.64, DRC 0
errors; power tree v0.12; PCB-Z-08 and CB-08 strip values.

Co-Authored-By: Claude Opus 5.5 <noreply@anthropic.com>
Claude-Session: https://claude.ai/code/session_013P6pW9LdyEMFishwCcZGUr
Parts:
- R808: footprint Resistor_SMD:R_1206_3216Metric -> T1_Main_Board:R_Vishay_WSL1206_2m-5m9
Changed lines of the file:
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@@
   (property "Value" "3 mΩ" (at 242.57 48.26 90) (effects (font (size 1.27 1.27))))
   (property "Spec" "1206" (at 242.57 50.8 90) (effects (font (size 1.27 1.27))))
-  (property "Footprint" "Resistor_SMD:R_1206_3216Metric" (at 242.57 45.72 0) (effects (font (size 1.27 1.27))) (hide yes))
+  (property "Footprint" "T1_Main_Board:R_Vishay_WSL1206_2m-5m9" (at 242.57 45.72 0) (effects (font (size 1.27 1.27))) (hide yes))
   (property "Datasheet" "https://www.vishay.com/docs/30100/wsl.pdf" (at 242.57 45.72 0) (effects (font (size 1.27 1.27))) (hide yes))
   (property "Description" "Current-sense resistor, 3 mOhm, 1 %, 0.25 W, 1206 metal strip" (at 242.57 45.72 0) (effects (font (size 1.27 1.27))) (hide yes))
