File: board/hardware/t1-main-board/pwr-3v3-sys.kicad_sch (KiCad schematic)
At the start: 13 parts, among them U1001 TPS62827DMQR

Commit message: Zone net classes and named switch nodes from the generator
Every net but GND now carries the ZONE_<NAME> class of each zone whose
blocks it touches (block zones from pcb/plan.py; the faceplate connector's
sheet also the faceplate zone); a rail used in more than one zone carries
ZONE_SHARED. Nets KiCad names from a pin take their part's sheet zone.
1,080 nets: 911 in one zone, 104 in two, 36 in three, 28 shared rails.

Switch nodes are named *_SW (VSYS_LV_SW, VCC3V3_SYS_SW, VDD_CPU_SW,
RP_VREG_SW); the display switch output is FP_VCI_OUT, so SW_NODE holds
the 18 switch nodes only. Board rebuilt: DRC 0 errors, 607 warnings
(the six PCB-I-09 gone), ERC 0 errors, craft Q1 met, pcb tests pass.
Closes placement v1 open items 2 and 3, floorplan v1 item 6.

Co-Authored-By: Claude Opus 5.5 <noreply@anthropic.com>
Claude-Session: https://claude.ai/code/session_01Ei262h3TpgY9vyfNLMi5Mn
Connections:
- net VCC3V3_SYS_SW: now reaches L1001.1, U1001.5 (SW)
Changed lines of the file:
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@@
 (table (column_count 3) (border (external yes) (header yes) (stroke (width 0) (type solid))) (separators (rows yes) (cols yes) (stroke (width 0) (type solid))) (column_widths 45.72 25.4 50.8) (row_heights 5.08 5.08 5.08) (cells (table_cell "Net" (exclude_from_sim no) (at 22.86 149.86 0) (size 45.72 5.08) (margins 0.9525 0.9525 0.9525 0.9525) (span 1 1) (fill (type none)) (effects (font (size 1.27 1.27) (bold yes)) (justify left top))) (table_cell "Direction" (exclude_from_sim no) (at 68.58 149.86 0) (size 25.4 5.08) (margins 0.9525 0.9525 0.9525 0.9525) (span 1 1) (fill (type none)) (effects (font (size 1.27 1.27) (bold yes)) (justify left top))) (table_cell "Absent state (block not fitted)" (exclude_from_sim no) (at 93.98 149.86 0) (size 50.8 5.08) (margins 0.9525 0.9525 0.9525 0.9525) (span 1 1) (fill (type none)) (effects (font (size 1.27 1.27) (bold yes)) (justify left top))) (table_cell "VSYS_LV" (exclude_from_sim no) (at 22.86 154.94 0) (size 45.72 5.08) (margins 0.9525 0.9525 0.9525 0.9525) (span 1 1) (fill (type none)) (effects (font (size 1.27 1.27)) (justify left top))) (table_cell "Supply in" (exclude_from_sim no) (at 68.58 154.94 0) (size 25.4 5.08) (margins 0.9525 0.9525 0.9525 0.9525) (span 1 1) (fill (type none)) (effects (font (size 1.27 1.27)) (justify left top))) (table_cell "Not applicable: never omitted" (exclude_from_sim no) (at 93.98 154.94 0) (size 50.8 5.08) (margins 0.9525 0.9525 0.9525 0.9525) (span 1 1) (fill (type none)) (effects (font (size 1.27 1.27)) (justify left top))) (table_cell "vcc3v3_sys" (exclude_from_sim no) (at 22.86 160.02 0) (size 45.72 5.08) (margins 0.9525 0.9525 0.9525 0.9525) (span 1 1) (fill (type none)) (effects (font (size 1.27 1.27)) (justify left top))) (table_cell "Supply out" (exclude_from_sim no) (at 68.58 160.02 0) (size 25.4 5.08) (margins 0.9525 0.9525 0.9525 0.9525) (span 1 1) (fill (type none)) (effects (font (size 1.27 1.27)) (justify left top))) (table_cell "Not applicable: always on (EN = VSYS_LV)" (exclude_from_sim no) (at 93.98 160.02 0) (size 50.8 5.08) (margins 0.9525 0.9525 0.9525 0.9525) (span 1 1) (fill (type none)) (effects (font (size 1.27 1.27)) (justify left top)))))
 (label "VCC3V3_SYS_PG" (at 116.84 91.44 270) (effects (font (size 1.27 1.27)) (justify right bottom)))
+(label "VCC3V3_SYS_SW" (at 116.84 81.28 90) (effects (font (size 1.27 1.27)) (justify left bottom)))
 (label "VCC3V3_SYS_PG" (at 195.58 105.41 270) (effects (font (size 1.27 1.27)) (justify right bottom)))
 (embedded_fonts no))

Commit message: Compaction: lower inductors, 0201 decoupling, 0.8 mm signal test pads
A matrix tool (hardware/studies/compaction) checks each candidate against
the design's stresses: same inductance, design peak <= 70 % and the
converter's maximum limit <= 100 % of Isat (30 % drop), height zones,
ratings at least twice the rail, PCB-D-06; sourcing outcome per part.

Applied (placement v1 decision 12, BOM v1.15):
- L601, L4401: XGL4015-102MEC (1.5 mm) for XAL/XGL4020-102MEC (2.1 mm);
- L1001, L5101: XGL4015-471MEC (1.5 mm) for Wurth 744373240047, on the
  stock XxL4020 land (the Wurth land was never drawn);
- L1201 is 1.2 mm (XGL4012, per-MPN heights): it moves next to the SoC;
- 58 x 100 nF decoupling on rails <= 3.3 V in core/IO/radio: 0201;
- 51 test pads on signal nets: 0.8 mm (PCB-D-06 v0.16, JLCPCB guide).
Kept: L901, L2802 (XGL4015 at 103 % of Isat at the limit); no thinner
0805/1206 capacitor passes (obsolete, NRND or unlisted).

Board need 113 % -> 111 % (core band 227 -> 203 %, power band 258 ->
233 %, radio band 19 -> 0 %); only C904 still relies on PCB-Z-04.
ERC 0 errors, craft Q1 met, DRC 0 errors (605 warnings), pcb and study
tests pass, rules test board PASS.

Co-Authored-By: Claude Opus 5.5 <noreply@anthropic.com>
Claude-Session: https://claude.ai/code/session_01Ei262h3TpgY9vyfNLMi5Mn
Parts:
- L1001: footprint T1_Main_Board:L_Wuerth_WE-LHMI_4020 -> Inductor_SMD:L_Coilcraft_XxL4020; MPN 744373240047 -> XGL4015-471MEC; Manufacturer Wurth Elektronik -> Coilcraft; Second_Source Coilcraft XFL4015-471MEC (land compatibility UNVERIFIED, BO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 -> Wurth 744373240047 (other land, 1.8 mm: bands only; BOM v1 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; Spec Isat 10.4 A -> Isat 10.5 A
- TP1001: footprint TestPoint:TestPoint_Pad_D1.0mm -> T1_Main_Board:TestPoint_Pad_D0.8mm
Changed lines of the file:
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@@
   (property "Reference" "L1001" (at 129.54 73.66 90) (effects (font (size 1.27 1.27))))
   (property "Value" "470 nH" (at 129.54 76.2 90) (effects (font (size 1.27 1.27))))
-  (property "Spec" "Isat 10.4 A" (at 129.54 78.74 90) (effects (font (size 1.27 1.27))))
-  (property "Footprint" "T1_Main_Board:L_Wuerth_WE-LHMI_4020" (at 129.54 81.28 0) (effects (font (size 1.27 1.27))) (hide yes))
-  (property "Datasheet" "https://www.we-online.com/components/products/datasheet/744373240047.pdf" (at 129.54 81.28 0) (effects (font (size 1.27 1.27))) (hide yes))
-  (property "Description" "Power inductor, 0.47 uH, IR 8.7 A, Isat 10.4 A (10 % drop), 4.45 x 4.06 x 1.8 mm" (at 129.54 81.28 0) (effects (font (size 1.27 1.27))) (hide yes))
-  (property "Manufacturer" "Wurth Elektronik" (at 129.54 81.28 0) (effects (font (size 1.27 1.27))) (hide yes))
-  (property "MPN" "744373240047" (at 129.54 81.28 0) (effects (font (size 1.27 1.27))) (hide yes))
-  (property "Second_Source" "Coilcraft XFL4015-471MEC (land compatibility UNVERIFIED, BOM v1 line 106)" (at 129.54 81.28 0) (effects (font (size 1.27 1.27))) (hide yes))
+  (property "Spec" "Isat 10.5 A" (at 129.54 78.74 90) (effects (font (size 1.27 1.27))))
+  (property "Footprint" "Inductor_SMD:L_Coilcraft_XxL4020" (at 129.54 81.28 0) (effects (font (size 1.27 1.27))) (hide yes))
+  (property "Datasheet" "https://coilcraft.com/getmedia/c5d04454-742d-473e-8b80-06c97338c587/xgl4015.pdf" (at 129.54 81.28 0) (effects (font (size 1.27 1.27))) (hide yes))
+  (property "Description" "Power inductor, 0.47 uH 20 %, Isat 10.5 A (30 % drop), Irms 9.6 A, 4.0 x 4.0 x 1.5 mm" (at 129.54 81.28 0) (effects (font (size 1.27 1.27))) (hide yes))
+  (property "Manufacturer" "Coilcraft" (at 129.54 81.28 0) (effects (font (size 1.27 1.27))) (hide yes))
+  (property "MPN" "XGL4015-471MEC" (at 129.54 81.28 0) (effects (font (size 1.27 1.27))) (hide yes))
+  (property "Second_Source" "Wurth 744373240047 (other land, 1.8 mm: bands only; BOM v1 line 106)" (at 129.54 81.28 0) (effects (font (size 1.27 1.27))) (hide yes))
   (property "Block" "blk.pwr-3v3-sys" (at 129.54 81.28 0) (effects (font (size 1.27 1.27))) (hide yes))
   (pin "1")
@@
   (property "Reference" "TP1001" (at 189.23 99.06 0) (effects (font (size 1.27 1.27)) (justify right)))
   (property "Value" "VCC3V3_SYS_PG" (at 189.23 101.6 0) (effects (font (size 1.27 1.27)) (justify right)))
-  (property "Footprint" "TestPoint:TestPoint_Pad_D1.0mm" (at 190.5 104.14 0) (effects (font (size 1.27 1.27))) (hide yes))
+  (property "Footprint" "T1_Main_Board:TestPoint_Pad_D0.8mm" (at 190.5 104.14 0) (effects (font (size 1.27 1.27))) (hide yes))
   (property "Datasheet" "~" (at 190.5 104.14 0) (effects (font (size 1.27 1.27))) (hide yes))
-  (property "Description" "Test pad, 1.0 mm" (at 190.5 104.14 0) (effects (font (size 1.27 1.27))) (hide yes))
+  (property "Description" "Test pad, 0.8 mm, signal net" (at 190.5 104.14 0) (effects (font (size 1.27 1.27))) (hide yes))
   (property "Block" "blk.pwr-3v3-sys" (at 190.5 104.14 0) (effects (font (size 1.27 1.27))) (hide yes))
   (pin "1")
@@
   (instances (project "t1-main-board" (path "/7746052e-d7f9-59ad-ba73-bd2b74439529/e24a57d0-1408-545b-9ef7-83abcf0ce576" (reference "#FLG0005") (unit 1))))
 )
-(text_box "Notes\n1. Function: TI TPS62827DMQR, VSYS_LV to vcc3v3_sys 3.3 V, 4 A, always on (BOM v1\n   line 6): RK809 VCC5-9, eMMC, SoC IO banks, radio switch (power tree §3).\n2. Absent state: not applicable. EN tied to VSYS_LV (RK809 EXT_EN unused).\n3. Feedback: 453 kΩ / 100 kΩ with VFB 0.6 V: 3.318 V (SLVSEF9I Eq. 4; the 450 kΩ\n   of Eq. 4 is not an E96 value). C3 120 pF = 12 µs / R2 (Eq. 5).\n4. L: Würth 744373240047 0.47 µH (BOM v1 line 106). Open: its footprint\n   T1_Main_Board:L_Wuerth_WE-LHMI_4020 is not drawn (data sheet not retrieved).\n5. Link H5 5 mΩ in every variant (power tree §4.12 #4); feedback on its source side.\n6. Unless noted: resistors 1 % 0402; capacitors X5R/X7R, at least twice the rail." (exclude_from_sim no) (at 152.4 137.16 0) (size 129.54 24.13) (margins 1.905 1.905 1.905 1.905) (stroke (width 0) (type default)) (fill (type none)) (effects (font (size 1.27 1.27)) (justify left top)))
+(text_box "Notes\n1. Function: TI TPS62827DMQR, VSYS_LV to vcc3v3_sys 3.3 V, 4 A, always on (BOM v1\n   line 6): RK809 VCC5-9, eMMC, SoC IO banks, radio switch (power tree §3).\n2. Absent state: not applicable. EN tied to VSYS_LV (RK809 EXT_EN unused).\n3. Feedback: 453 kΩ / 100 kΩ with VFB 0.6 V: 3.318 V (SLVSEF9I Eq. 4; the 450 kΩ\n   of Eq. 4 is not an E96 value). C3 120 pF = 12 µs / R2 (Eq. 5).\n4. L: Coilcraft XGL4015-471MEC 0.47 µH, 1.5 mm (compaction study, 2026-10-27; was\n   Würth 744373240047 of BOM v1 line 106, 1.8 mm, kept as the other-land alternate).\n5. Link H5 5 mΩ in every variant (power tree §4.12 #4); feedback on its source side.\n6. Unless noted: resistors 1 % 0402; capacitors X5R/X7R, at least twice the rail." (exclude_from_sim no) (at 152.4 137.16 0) (size 129.54 24.13) (margins 1.905 1.905 1.905 1.905) (stroke (width 0) (type default)) (fill (type none)) (effects (font (size 1.27 1.27)) (justify left top)))
 (text "Rails" (exclude_from_sim no) (at 22.86 171.45 0) (effects (font (size 2.54 2.54)) (justify left bottom)))
 (table (column_count 3) (border (external yes) (header yes) (stroke (width 0) (type solid))) (separators (rows yes) (cols yes) (stroke (width 0) (type solid))) (column_widths 27.94 39.37 54.61) (row_heights 5.08 7.62 7.62) (cells (table_cell "Rail" (exclude_from_sim no) (at 22.86 172.72 0) (size 27.94 5.08) (margins 0.9525 0.9525 0.9525 0.9525) (span 1 1) (fill (type none)) (effects (font (size 1.27 1.27) (bold yes)) (justify left top))) (table_cell "Capacitors" (exclude_from_sim no) (at 50.8 172.72 0) (size 39.37 5.08) (margins 0.9525 0.9525 0.9525 0.9525) (span 1 1) (fill (type none)) (effects (font (size 1.27 1.27) (bold yes)) (justify left top))) (table_cell "Requirement and source" (exclude_from_sim no) (at 90.17 172.72 0) (size 54.61 5.08) (margins 0.9525 0.9525 0.9525 0.9525) (span 1 1) (fill (type none)) (effects (font (size 1.27 1.27) (bold yes)) (justify left top))) (table_cell "VSYS_LV" (exclude_from_sim no) (at 22.86 177.8 0) (size 27.94 7.62) (margins 0.9525 0.9525 0.9525 0.9525) (span 1 1) (fill (type none)) (effects (font (size 1.27 1.27)) (justify left top))) (table_cell "4.7 µF 6.3 V X7R 0603" (exclude_from_sim no) (at 50.8 177.8 0) (size 39.37 7.62) (margins 0.9525 0.9525 0.9525 0.9525) (span 1 1) (fill (type none)) (effects (font (size 1.27 1.27)) (justify left top))) (table_cell "C1 4.7 µF (SLVSEF9I Fig. 8-2); >= 3 µF effective (p. 14)" (exclude_from_sim no) (at 90.17 177.8 0) (size 54.61 7.62) (margins 0.9525 0.9525 0.9525 0.9525) (span 1 1) (fill (type none)) (effects (font (size 1.27 1.27)) (justify left top))) (table_cell "vcc3v3_sys" (exclude_from_sim no) (at 22.86 185.42 0) (size 27.94 7.62) (margins 0.9525 0.9525 0.9525 0.9525) (span 1 1) (fill (type none)) (effects (font (size 1.27 1.27)) (justify left top))) (table_cell "22 µF + 10 µF 0603" (exclude_from_sim no) (at 50.8 185.42 0) (size 39.37 7.62) (margins 0.9525 0.9525 0.9525 0.9525) (span 1 1) (fill (type none)) (effects (font (size 1.27 1.27)) (justify left top))) (table_cell ">= 20 µF effective for the TPS62827 (p. 14; BOM D26); DC bias UNVERIFIED" (exclude_from_sim no) (at 90.17 185.42 0) (size 54.61 7.62) (margins 0.9525 0.9525 0.9525 0.9525) (span 1 1) (fill (type none)) (effects (font (size 1.27 1.27)) (justify left top)))))

Commit message: Board on libs v0.2.0: lower-case kebab vendor keys (HL-13)
The libs submodule moves to v0.2.0 (5f24483). Every library nickname in
the generator, the placement tool and the floorplan study follows the
key table (Texas_Instruments -> texas-instruments, OpenDAP_Device ->
opendap-generic, Rockchip and Rockchip_PMIC -> rockchip, ...); the
library tables are written from the files. Schematic and board
regenerated.

Checks: ERC 0 errors (warnings unchanged); DRC 0 errors, 605 warnings,
the same counts by type, schematic parity 0; every placement identical;
craft Q1 met; pcb tests pass; STEP export resolves every libs 3D model
(the 27 parts without a model are KiCad stock lands that have none).

Co-Authored-By: Claude Opus 5.5 <noreply@anthropic.com>
Claude-Session: https://claude.ai/code/session_01Ei262h3TpgY9vyfNLMi5Mn
Parts:
- U1001: footprint Texas_Instruments:Texas_DMQ0006A_VSON-HR-6_1.5x1.5mm_P0.5mm -> texas-instruments:Texas_DMQ0006A_VSON-HR-6_1.5x1.5mm_P0.5mm; symbol Texas_Instruments:TPS62827DMQR -> texas-instruments:TPS62827DMQR
Changed lines of the file:
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@@
 (paper "A4")
 (title_block (title "3.3 V system rail") (date "2026-10-25") (rev "A") (company "The OpenDAP Project") (comment 1 "blk.pwr-3v3-sys") (comment 2 "VSYS_LV to the always-on vcc3v3_sys 3.3 V rail, 4 A"))
-(symbol (lib_id "Texas_Instruments:TPS62827DMQR") (at 101.6 83.82 0) (unit 1) (body_style 1) (exclude_from_sim no) (in_bom yes) (on_board yes) (dnp no)
+(symbol (lib_id "texas-instruments:TPS62827DMQR") (at 101.6 83.82 0) (unit 1) (body_style 1) (exclude_from_sim no) (in_bom yes) (on_board yes) (dnp no)
   (property "Reference" "U1001" (at 102.87 66.04 0) (effects (font (size 1.27 1.27)) (justify left)))
   (property "Value" "TPS62827DMQR" (at 102.87 63.5 0) (effects (font (size 1.27 1.27)) (justify left)))
-  (property "Footprint" "Texas_Instruments:Texas_DMQ0006A_VSON-HR-6_1.5x1.5mm_P0.5mm" (at 101.6 83.82 0) (effects (font (size 1.27 1.27))) (hide yes))
+  (property "Footprint" "texas-instruments:Texas_DMQ0006A_VSON-HR-6_1.5x1.5mm_P0.5mm" (at 101.6 83.82 0) (effects (font (size 1.27 1.27))) (hide yes))
   (property "Datasheet" "https://www.ti.com/lit/ds/symlink/tps62826.pdf" (at 101.6 83.82 0) (effects (font (size 1.27 1.27))) (hide yes))
   (property "Description" "4 A synchronous step-down converter, 2.5-5.5 V input, 0.6-4.0 V adjustable output, power save mode, power good, 100 % duty cycle, VSON-HR-6 (DMQ0006A) 1.5 x 1.5 mm" (at 101.6 83.82 0) (effects (font (size 1.27 1.27))) (hide yes))

Commit message: Board in the 62.5 x 95.0 mm body: ADR 0025, outline 59.1 x 91.6, 0201 swaps
ADR 0025 supersedes ADR 0016 for t1 ADR 0006's body: board outline from
the body, 1.2 mm walls and 0.5 mm clearance; height zones and stack
restated unchanged; the speaker on a case shelf (PCB-Z-09); pocket
reliefs at the 4.4 mm jack, the microSD (DM3AT push-push kept) and the
side buttons; the audio 0603 -> 0402 swap gated by t1 V2-A08; reserve
(NFC reader, then TPM) recorded, not applied.

- pcb/geometry.py derives the outline from BODY, WALL and CLEARANCE;
  the pocket, display and fixed parts keep their device-frame positions;
  holes keep their edge distance; the speaker shadow becomes a 1.5 mm
  shelf height area (placement, checks, occupancy).
- build.py reports pocket reliefs and routing room; C904 unfixed (it
  now finds back room, so PCB-Z-04 carries no part).
- Generator: parts.area_swap puts 121 generic 0402 resistors (outside
  audio and VBUS paths, >= 10 ohm) and five 100 nF signal capacitors in
  0201 (BOM v1.16); schematic and board regenerated.
- Result: 1,012/1,012 placed, 98.8 % by the floorplan method (was 111 %),
  factor left 1.68 (was 1.49); DRC 0 errors, ERC 0 errors, 0 check
  findings, pcb tests 20/20, schematic craft Q1 met.
- Specs: PCB constraints v0.17 (M-01, M-02, M-08, Z-02, Z-06 to Z-09,
  R-07), placement v1.1 (section 3, decisions 4 and 13, checks, open
  items with the gated swaps and the reserve), floorplan v1 section 1,
  BOM v1.16.

Co-Authored-By: Claude Opus 5.5 <noreply@anthropic.com>
Claude-Session: https://claude.ai/code/session_01Ei262h3TpgY9vyfNLMi5Mn
Parts:
- R1001: footprint Resistor_SMD:R_0402_1005Metric -> Resistor_SMD:R_0201_0603Metric; MPN RC0402FR-07453KL -> RC0201FR-07453KL
- R1002, R1003: footprint Resistor_SMD:R_0402_1005Metric -> Resistor_SMD:R_0201_0603Metric; MPN RC0402FR-07100KL -> RC0201FR-07100KL
Changed lines of the file:
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@@
   (property "Reference" "R1001" (at 143.51 85.09 0) (effects (font (size 1.27 1.27)) (justify left)))
   (property "Value" "453 kΩ" (at 143.51 87.63 0) (effects (font (size 1.27 1.27)) (justify left)))
-  (property "Footprint" "Resistor_SMD:R_0402_1005Metric" (at 142.24 86.36 0) (effects (font (size 1.27 1.27))) (hide yes))
-  (property "Datasheet" "https://yageogroup.com/en/ProductSearch/PartNumberSearch?part=RC0402FR-07453KL" (at 142.24 86.36 0) (effects (font (size 1.27 1.27))) (hide yes))
-  (property "Description" "Resistor, 453 kΩ, 1 %, 1/16 W, 0402" (at 142.24 86.36 0) (effects (font (size 1.27 1.27))) (hide yes))
+  (property "Footprint" "Resistor_SMD:R_0201_0603Metric" (at 142.24 86.36 0) (effects (font (size 1.27 1.27))) (hide yes))
+  (property "Datasheet" "https://yageogroup.com/en/ProductSearch/PartNumberSearch?part=RC0201FR-07453KL" (at 142.24 86.36 0) (effects (font (size 1.27 1.27))) (hide yes))
+  (property "Description" "Resistor, 453 kΩ, 1 %, 1/20 W, 0201" (at 142.24 86.36 0) (effects (font (size 1.27 1.27))) (hide yes))
   (property "Manufacturer" "YAGEO" (at 142.24 86.36 0) (effects (font (size 1.27 1.27))) (hide yes))
-  (property "MPN" "RC0402FR-07453KL" (at 142.24 86.36 0) (effects (font (size 1.27 1.27))) (hide yes))
+  (property "MPN" "RC0201FR-07453KL" (at 142.24 86.36 0) (effects (font (size 1.27 1.27))) (hide yes))
   (property "Block" "blk.pwr-3v3-sys" (at 142.24 86.36 0) (effects (font (size 1.27 1.27))) (hide yes))
   (pin "1")
@@
   (property "Reference" "R1002" (at 143.51 100.33 0) (effects (font (size 1.27 1.27)) (justify left)))
   (property "Value" "100 kΩ" (at 143.51 102.87 0) (effects (font (size 1.27 1.27)) (justify left)))
-  (property "Footprint" "Resistor_SMD:R_0402_1005Metric" (at 142.24 101.6 0) (effects (font (size 1.27 1.27))) (hide yes))
-  (property "Datasheet" "https://yageogroup.com/en/ProductSearch/PartNumberSearch?part=RC0402FR-07100KL" (at 142.24 101.6 0) (effects (font (size 1.27 1.27))) (hide yes))
-  (property "Description" "Resistor, 100 kΩ, 1 %, 1/16 W, 0402" (at 142.24 101.6 0) (effects (font (size 1.27 1.27))) (hide yes))
+  (property "Footprint" "Resistor_SMD:R_0201_0603Metric" (at 142.24 101.6 0) (effects (font (size 1.27 1.27))) (hide yes))
+  (property "Datasheet" "https://yageogroup.com/en/ProductSearch/PartNumberSearch?part=RC0201FR-07100KL" (at 142.24 101.6 0) (effects (font (size 1.27 1.27))) (hide yes))
+  (property "Description" "Resistor, 100 kΩ, 1 %, 1/20 W, 0201" (at 142.24 101.6 0) (effects (font (size 1.27 1.27))) (hide yes))
   (property "Manufacturer" "YAGEO" (at 142.24 101.6 0) (effects (font (size 1.27 1.27))) (hide yes))
-  (property "MPN" "RC0402FR-07100KL" (at 142.24 101.6 0) (effects (font (size 1.27 1.27))) (hide yes))
+  (property "MPN" "RC0201FR-07100KL" (at 142.24 101.6 0) (effects (font (size 1.27 1.27))) (hide yes))
   (property "Block" "blk.pwr-3v3-sys" (at 142.24 101.6 0) (effects (font (size 1.27 1.27))) (hide yes))
   (pin "1")
@@
   (property "Reference" "R1003" (at 196.85 85.09 0) (effects (font (size 1.27 1.27)) (justify left)))
   (property "Value" "100 kΩ" (at 196.85 87.63 0) (effects (font (size 1.27 1.27)) (justify left)))
-  (property "Footprint" "Resistor_SMD:R_0402_1005Metric" (at 195.58 86.36 0) (effects (font (size 1.27 1.27))) (hide yes))
-  (property "Datasheet" "https://yageogroup.com/en/ProductSearch/PartNumberSearch?part=RC0402FR-07100KL" (at 195.58 86.36 0) (effects (font (size 1.27 1.27))) (hide yes))
-  (property "Description" "Resistor, 100 kΩ, 1 %, 1/16 W, 0402" (at 195.58 86.36 0) (effects (font (size 1.27 1.27))) (hide yes))
+  (property "Footprint" "Resistor_SMD:R_0201_0603Metric" (at 195.58 86.36 0) (effects (font (size 1.27 1.27))) (hide yes))
+  (property "Datasheet" "https://yageogroup.com/en/ProductSearch/PartNumberSearch?part=RC0201FR-07100KL" (at 195.58 86.36 0) (effects (font (size 1.27 1.27))) (hide yes))
+  (property "Description" "Resistor, 100 kΩ, 1 %, 1/20 W, 0201" (at 195.58 86.36 0) (effects (font (size 1.27 1.27))) (hide yes))
   (property "Manufacturer" "YAGEO" (at 195.58 86.36 0) (effects (font (size 1.27 1.27))) (hide yes))
-  (property "MPN" "RC0402FR-07100KL" (at 195.58 86.36 0) (effects (font (size 1.27 1.27))) (hide yes))
+  (property "MPN" "RC0201FR-07100KL" (at 195.58 86.36 0) (effects (font (size 1.27 1.27))) (hide yes))
   (property "Block" "blk.pwr-3v3-sys" (at 195.58 86.36 0) (effects (font (size 1.27 1.27))) (hide yes))
   (pin "1")
