File: board/hardware/t1-main-board/pwr-3v3-sys.kicad_sch (KiCad schematic)
At the start: 13 parts, among them U1001 TPS62827DMQR

Commit message: Board: pre-PCB schematic items closed with datasheets (BOM v1.22)
Display INA236 to 0x49 (INA236B, A0 = VS): no A0 = SDA strap, so the
address no longer depends on the host's I2C hold time. The 18 WSL
shunts and links on Vishay's doc 30100 lands. 24 MHz crystal NDK
NX3225GA (CL 8 pF) with 2 x 10 pF. Backlight inductor Coilcraft
XFL3012-223MEC on its published land (no placeholder left). Action
button PTS815 G code on the side-button land. Cover-detect leakage,
TPS3808 spread, RP2354A supply pins and the USB series scheme closed
without change. Placement v1.9: 100.2 % need, factor 1.64, DRC 0
errors; power tree v0.12; PCB-Z-08 and CB-08 strip values.

Co-Authored-By: Claude Opus 5.5 <noreply@anthropic.com>
Claude-Session: https://claude.ai/code/session_013P6pW9LdyEMFishwCcZGUr
Parts:
- R1004: footprint Resistor_SMD:R_1206_3216Metric -> T1_Main_Board:R_Vishay_WSL1206_2m-5m9
Changed lines of the file:
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@@
   (property "Value" "5 mΩ" (at 231.14 83.82 90) (effects (font (size 1.27 1.27))))
   (property "Spec" "1206" (at 231.14 86.36 90) (effects (font (size 1.27 1.27))))
-  (property "Footprint" "Resistor_SMD:R_1206_3216Metric" (at 233.68 81.28 0) (effects (font (size 1.27 1.27))) (hide yes))
+  (property "Footprint" "T1_Main_Board:R_Vishay_WSL1206_2m-5m9" (at 233.68 81.28 0) (effects (font (size 1.27 1.27))) (hide yes))
   (property "Datasheet" "https://www.vishay.com/docs/30100/wsl.pdf" (at 233.68 81.28 0) (effects (font (size 1.27 1.27))) (hide yes))
   (property "Description" "Current-sense resistor, 5 mOhm, 1 %, 0.5 W, 1206 metal strip: measurement link H5" (at 233.68 81.28 0) (effects (font (size 1.27 1.27))) (hide yes))
