File: board/hardware/t1-main-board/soc-power.kicad_sch (KiCad schematic)
At the start: 45 parts, among them U1301 RK3566

Commit message: Compaction: lower inductors, 0201 decoupling, 0.8 mm signal test pads
A matrix tool (hardware/studies/compaction) checks each candidate against
the design's stresses: same inductance, design peak <= 70 % and the
converter's maximum limit <= 100 % of Isat (30 % drop), height zones,
ratings at least twice the rail, PCB-D-06; sourcing outcome per part.

Applied (placement v1 decision 12, BOM v1.15):
- L601, L4401: XGL4015-102MEC (1.5 mm) for XAL/XGL4020-102MEC (2.1 mm);
- L1001, L5101: XGL4015-471MEC (1.5 mm) for Wurth 744373240047, on the
  stock XxL4020 land (the Wurth land was never drawn);
- L1201 is 1.2 mm (XGL4012, per-MPN heights): it moves next to the SoC;
- 58 x 100 nF decoupling on rails <= 3.3 V in core/IO/radio: 0201;
- 51 test pads on signal nets: 0.8 mm (PCB-D-06 v0.16, JLCPCB guide).
Kept: L901, L2802 (XGL4015 at 103 % of Isat at the limit); no thinner
0805/1206 capacitor passes (obsolete, NRND or unlisted).

Board need 113 % -> 111 % (core band 227 -> 203 %, power band 258 ->
233 %, radio band 19 -> 0 %); only C904 still relies on PCB-Z-04.
ERC 0 errors, craft Q1 met, DRC 0 errors (605 warnings), pcb and study
tests pass, rules test board PASS.

Co-Authored-By: Claude Opus 5.5 <noreply@anthropic.com>
Claude-Session: https://claude.ai/code/session_01Ei262h3TpgY9vyfNLMi5Mn
Parts:
- C1333, C1335, C1337, C1338, C1339, C1340, C1341, C1342, C1343, C1344, C1345, C1346, C1347, C1348: footprint Capacitor_SMD:C_0402_1005Metric -> Capacitor_SMD:C_0201_0603Metric; MPN GRM155R71C104KA88D -> GRM033R61A104KE15D

Commit message: Board on libs v0.2.0: lower-case kebab vendor keys (HL-13)
The libs submodule moves to v0.2.0 (5f24483). Every library nickname in
the generator, the placement tool and the floorplan study follows the
key table (Texas_Instruments -> texas-instruments, OpenDAP_Device ->
opendap-generic, Rockchip and Rockchip_PMIC -> rockchip, ...); the
library tables are written from the files. Schematic and board
regenerated.

Checks: ERC 0 errors (warnings unchanged); DRC 0 errors, 605 warnings,
the same counts by type, schematic parity 0; every placement identical;
craft Q1 met; pcb tests pass; STEP export resolves every libs 3D model
(the 27 parts without a model are KiCad stock lands that have none).

Co-Authored-By: Claude Opus 5.5 <noreply@anthropic.com>
Claude-Session: https://claude.ai/code/session_01Ei262h3TpgY9vyfNLMi5Mn
Parts:
- U1301: footprint Rockchip:Rockchip_FCCSP-565L_15.5x14.4mm_P0.4mm_P0.65mm_Ball0.25mm_Pad0.25mm_NSMD -> rockchip:Rockchip_FCCSP-565L_15.5x14.4mm_P0.4mm_P0.65mm_Ball0.25mm_Pad0.25mm_NSMD; symbol Rockchip:RK3566 -> rockchip:RK3566
Changed lines of the file:
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@@
 (paper "A3")
 (title_block (title "SoC: supplies and decoupling") (date "2026-10-25") (rev "A") (company "The OpenDAP Project") (comment 1 "blk.soc-power") (comment 2 "RK3566 supply units with the decoupling of the hardware design guide, grouped by rail"))
-(symbol (lib_id "Rockchip:RK3566") (at 67.31 81.28 0) (unit 20) (body_style 1) (exclude_from_sim no) (in_bom yes) (on_board yes) (dnp no)
+(symbol (lib_id "rockchip:RK3566") (at 67.31 81.28 0) (unit 20) (body_style 1) (exclude_from_sim no) (in_bom yes) (on_board yes) (dnp no)
   (property "Reference" "U1301" (at 25.4 102.87 0) (effects (font (size 1.27 1.27)) (justify left)))
   (property "Value" "RK3566" (at 25.4 100.33 0) (effects (font (size 1.27 1.27)) (justify left)))
-  (property "Footprint" "Rockchip:Rockchip_FCCSP-565L_15.5x14.4mm_P0.4mm_P0.65mm_Ball0.25mm_Pad0.25mm_NSMD" (at 67.31 81.28 0) (effects (font (size 1.27 1.27))) (hide yes))
+  (property "Footprint" "rockchip:Rockchip_FCCSP-565L_15.5x14.4mm_P0.4mm_P0.65mm_Ball0.25mm_Pad0.25mm_NSMD" (at 67.31 81.28 0) (effects (font (size 1.27 1.27))) (hide yes))
   (property "Datasheet" "https://dl.xkwy2018.com/downloads/RK3568/Rockchip-RK3566-Datasheet-V1.1-20210305.pdf" (at 67.31 81.28 0) (effects (font (size 1.27 1.27))) (hide yes))
   (property "Description" "Quad-core Arm Cortex-A55 application processor, LPDDR4X/DDR4 32-bit, eMMC 5.1, FCCSP565L 15.5 x 14.4 mm" (at 67.31 81.28 0) (effects (font (size 1.27 1.27))) (hide yes))
@@
   (instances (project "t1-main-board" (path "/7746052e-d7f9-59ad-ba73-bd2b74439529/8302eaa7-1fc9-5a34-8a84-8a9171d22bdf/84b45083-7f8c-57ed-8ede-15f51b372710" (reference "#PWR0223") (unit 1))))
 )
-(symbol (lib_id "Rockchip:RK3566") (at 151.13 80.01 0) (unit 21) (body_style 1) (exclude_from_sim no) (in_bom yes) (on_board yes) (dnp no)
+(symbol (lib_id "rockchip:RK3566") (at 151.13 80.01 0) (unit 21) (body_style 1) (exclude_from_sim no) (in_bom yes) (on_board yes) (dnp no)
   (property "Reference" "U1301" (at 116.84 99.06 0) (effects (font (size 1.27 1.27)) (justify left)))
   (property "Value" "RK3566" (at 116.84 96.52 0) (effects (font (size 1.27 1.27)) (justify left)))
-  (property "Footprint" "Rockchip:Rockchip_FCCSP-565L_15.5x14.4mm_P0.4mm_P0.65mm_Ball0.25mm_Pad0.25mm_NSMD" (at 151.13 80.01 0) (effects (font (size 1.27 1.27))) (hide yes))
+  (property "Footprint" "rockchip:Rockchip_FCCSP-565L_15.5x14.4mm_P0.4mm_P0.65mm_Ball0.25mm_Pad0.25mm_NSMD" (at 151.13 80.01 0) (effects (font (size 1.27 1.27))) (hide yes))
   (property "Datasheet" "https://dl.xkwy2018.com/downloads/RK3568/Rockchip-RK3566-Datasheet-V1.1-20210305.pdf" (at 151.13 80.01 0) (effects (font (size 1.27 1.27))) (hide yes))
   (property "Description" "Quad-core Arm Cortex-A55 application processor, LPDDR4X/DDR4 32-bit, eMMC 5.1, FCCSP565L 15.5 x 14.4 mm" (at 151.13 80.01 0) (effects (font (size 1.27 1.27))) (hide yes))
@@
   (instances (project "t1-main-board" (path "/7746052e-d7f9-59ad-ba73-bd2b74439529/8302eaa7-1fc9-5a34-8a84-8a9171d22bdf/84b45083-7f8c-57ed-8ede-15f51b372710" (reference "#PWR0234") (unit 1))))
 )
-(symbol (lib_id "Rockchip:RK3566") (at 227.33 90.17 0) (unit 22) (body_style 1) (exclude_from_sim no) (in_bom yes) (on_board yes) (dnp no)
+(symbol (lib_id "rockchip:RK3566") (at 227.33 90.17 0) (unit 22) (body_style 1) (exclude_from_sim no) (in_bom yes) (on_board yes) (dnp no)
   (property "Reference" "U1301" (at 193.04 119.38 0) (effects (font (size 1.27 1.27)) (justify left)))
   (property "Value" "RK3566" (at 193.04 116.84 0) (effects (font (size 1.27 1.27)) (justify left)))
-  (property "Footprint" "Rockchip:Rockchip_FCCSP-565L_15.5x14.4mm_P0.4mm_P0.65mm_Ball0.25mm_Pad0.25mm_NSMD" (at 227.33 90.17 0) (effects (font (size 1.27 1.27))) (hide yes))
+  (property "Footprint" "rockchip:Rockchip_FCCSP-565L_15.5x14.4mm_P0.4mm_P0.65mm_Ball0.25mm_Pad0.25mm_NSMD" (at 227.33 90.17 0) (effects (font (size 1.27 1.27))) (hide yes))
   (property "Datasheet" "https://dl.xkwy2018.com/downloads/RK3568/Rockchip-RK3566-Datasheet-V1.1-20210305.pdf" (at 227.33 90.17 0) (effects (font (size 1.27 1.27))) (hide yes))
   (property "Description" "Quad-core Arm Cortex-A55 application processor, LPDDR4X/DDR4 32-bit, eMMC 5.1, FCCSP565L 15.5 x 14.4 mm" (at 227.33 90.17 0) (effects (font (size 1.27 1.27))) (hide yes))

Commit message: BOM v1.18 item 2: successors of the discontinued 1 uF 0402
GRM155R61A105KE15D is to be discontinued. 44 positions take
GRM155C71A105KE11D (1 uF 10 V X7S); the eight TPS7A20 positions take
GRM155R61C225KE11D (2.2 uF 16 V X5R) to keep the 0.47 uF effective
minimum with 10 % to spare at up to 3.8 V. Same land; sourcing pass.
Closes BOM §7 item 52; new item 55 lists the other capture parts outside
Murata's product data or near end of life.

Co-Authored-By: Claude Opus 5.5 <noreply@anthropic.com>
Claude-Session: https://claude.ai/code/session_01Ei262h3TpgY9vyfNLMi5Mn
Parts:
- C1334, C1336: MPN GRM155R61A105KE15D -> GRM155C71A105KE11D
Changed lines of the file:
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@@
   (property "Value" "1 µF" (at 45.72 205.74 0) (effects (font (size 1.27 1.27)) (justify left)))
   (property "Footprint" "Capacitor_SMD:C_0402_1005Metric" (at 43.18 204.47 0) (effects (font (size 1.27 1.27))) (hide yes))
-  (property "Datasheet" "https://www.murata.com/en-us/products/productdetail?partno=GRM155R61A105KE15D" (at 43.18 204.47 0) (effects (font (size 1.27 1.27))) (hide yes))
-  (property "Description" "Capacitor, 1 µF, 10 V, X5R, 0402" (at 43.18 204.47 0) (effects (font (size 1.27 1.27))) (hide yes))
+  (property "Datasheet" "https://www.murata.com/en-us/products/productdetail?partno=GRM155C71A105KE11D" (at 43.18 204.47 0) (effects (font (size 1.27 1.27))) (hide yes))
+  (property "Description" "Capacitor, 1 µF, 10 V, X7S, 0402" (at 43.18 204.47 0) (effects (font (size 1.27 1.27))) (hide yes))
   (property "Manufacturer" "Murata" (at 43.18 204.47 0) (effects (font (size 1.27 1.27))) (hide yes))
-  (property "MPN" "GRM155R61A105KE15D" (at 43.18 204.47 0) (effects (font (size 1.27 1.27))) (hide yes))
+  (property "MPN" "GRM155C71A105KE11D" (at 43.18 204.47 0) (effects (font (size 1.27 1.27))) (hide yes))
   (property "Block" "blk.soc-power" (at 43.18 204.47 0) (effects (font (size 1.27 1.27))) (hide yes))
   (pin "1")
@@
   (property "Value" "1 µF" (at 83.82 205.74 0) (effects (font (size 1.27 1.27)) (justify left)))
   (property "Footprint" "Capacitor_SMD:C_0402_1005Metric" (at 81.28 204.47 0) (effects (font (size 1.27 1.27))) (hide yes))
-  (property "Datasheet" "https://www.murata.com/en-us/products/productdetail?partno=GRM155R61A105KE15D" (at 81.28 204.47 0) (effects (font (size 1.27 1.27))) (hide yes))
-  (property "Description" "Capacitor, 1 µF, 10 V, X5R, 0402" (at 81.28 204.47 0) (effects (font (size 1.27 1.27))) (hide yes))
+  (property "Datasheet" "https://www.murata.com/en-us/products/productdetail?partno=GRM155C71A105KE11D" (at 81.28 204.47 0) (effects (font (size 1.27 1.27))) (hide yes))
+  (property "Description" "Capacitor, 1 µF, 10 V, X7S, 0402" (at 81.28 204.47 0) (effects (font (size 1.27 1.27))) (hide yes))
   (property "Manufacturer" "Murata" (at 81.28 204.47 0) (effects (font (size 1.27 1.27))) (hide yes))
-  (property "MPN" "GRM155R61A105KE15D" (at 81.28 204.47 0) (effects (font (size 1.27 1.27))) (hide yes))
+  (property "MPN" "GRM155C71A105KE11D" (at 81.28 204.47 0) (effects (font (size 1.27 1.27))) (hide yes))
   (property "Block" "blk.soc-power" (at 81.28 204.47 0) (effects (font (size 1.27 1.27))) (hide yes))
   (pin "1")

Commit message: Placement v1.3: capacitor proximity rule, checked and met
pcb/proximity.py assigns every converter's input and output capacitors
(from pin functions and types) and every IC's decoupling (block rule and
the generator's new Decoupling field) and checks each within its bound
of the pins it serves (input 3, output 5, decoupling 4, bulk 6 mm); the
build fails otherwise. The placer places each IC's capacitors right
after it, keeps room for them, reorders, swaps and repairs; a search
radius bug (mm used as cells) that blocked rotations is fixed. RK809
moved 1.2 mm right and 1.1 mm down off the radio zone edge.

Fixes found: C901 was 29 mm from U901; 136 of 237 capacitors were beyond
their bound. Now 248 checked, none beyond. BOM v1.18 items 3 (revised:
3 x GRM219R61C226ME15L per LDO position), 5 (C4403 as 2 x 0805) and 6.
Tests: test_proximity (6).

Co-Authored-By: Claude Opus 5.5 <noreply@anthropic.com>
Claude-Session: https://claude.ai/code/session_01Ei262h3TpgY9vyfNLMi5Mn
Parts:
- C1309, C1310, C1311, C1312: Decoupling (none) -> vdd_cpu
- C1313, C1314, C1315, C1316, C1317: Decoupling (none) -> vdd_logic
- C1318, C1319, C1320: Decoupling (none) -> vdd_gpu
- C1321, C1322: Decoupling (none) -> vdd_npu
- C1323, C1324, C1325, C1326, C1327: Decoupling (none) -> vcc_ddr
- C1328, C1329, C1330, C1331, C1332: Decoupling (none) -> vcc0v6_ddr
- C1333, C1334: Decoupling (none) -> vdda_0v9
- C1335, C1336: Decoupling (none) -> vcca_1v8
- C1337, C1338, C1339, C1340: Decoupling (none) -> vcc3v3_sys
- C1341, C1342: Decoupling (none) -> vcc_1v8
- C1343: Decoupling (none) -> vccio_sd
- C1344, C1345: Decoupling (none) -> vccio6_1v8
- C1346: Decoupling (none) -> vcc3v3_pmu
- C1347, C1348: Decoupling (none) -> vcca1v8_pmu

Commit message: vdd_cpu on the TPS62870Z4 (ADR 0026, placement v1.5)
ADR 0026 supersedes ADR 0023: TPS62870Z4WRXSR at I2C0 0x42 with the
Coilcraft XEL4012-920NE, 3 MHz, MODE/SYNC to ground with forced PWM by
register, differential sense from the 22 uF at the SoC. Output capacitance
sized at the 1.1 V devicetree cap for the 4.8 A worst-case step (peak
1.149 V, DC-bias effective values); 1800 MHz kept as a verification row.

Submodule at libs v0.3.2 (the RXS0016A land). BOM v1.18 item 8, power
tree v0.10, pinout v1 I2C0 note, feature blocks #13, placement v1.5.
Schematic regenerated, board rebuilt: 991 parts placed, 97.0 % board need,
factor 1.71, 244 capacitors within their bound, DRC 0 errors, ERC 0
errors, craft Q1 met, pcb tests pass, STEP exported (27 parts without a
model in KiCad's library, as before).

Co-Authored-By: Claude Opus 5.5 <noreply@anthropic.com>
Claude-Session: https://claude.ai/code/session_013P6pW9LdyEMFishwCcZGUr
Parts:
- added C1349: 100 nF, Capacitor_SMD:C_0201_0603Metric, symbol Device:C
- C1313: value 100 nF -> 22 µF; footprint Capacitor_SMD:C_0201_0603Metric -> Capacitor_SMD:C_0603_1608Metric; Decoupling vdd_logic -> vdd_cpu; MPN GRM033R61A104KE15D -> GRM188R60J226MEA0D; Spec 10 V X5R -> 6.3 V X5R
- C1314, C1319, C1326, C1331: value 4.7 µF -> 100 nF; footprint Capacitor_SMD:C_0402_1005Metric -> Capacitor_SMD:C_0201_0603Metric; MPN GRM155R60J475ME47D -> GRM033R61A104KE15D; Spec 6.3 V X5R -> 10 V X5R
- C1317, C1320: value 22 µF -> 4.7 µF; footprint Capacitor_SMD:C_0603_1608Metric -> Capacitor_SMD:C_0402_1005Metric; MPN GRM188R60J226MEA0D -> GRM155R60J475ME47D
- C1318: value 100 nF -> 22 µF; footprint Capacitor_SMD:C_0201_0603Metric -> Capacitor_SMD:C_0603_1608Metric; Decoupling vdd_gpu -> vdd_logic; MPN GRM033R61A104KE15D -> GRM188R60J226MEA0D; Spec 10 V X5R -> 6.3 V X5R
- C1321: value 100 nF -> 22 µF; footprint Capacitor_SMD:C_0201_0603Metric -> Capacitor_SMD:C_0603_1608Metric; Decoupling vdd_npu -> vdd_gpu; MPN GRM033R61A104KE15D -> GRM188R60J226MEA0D; Spec 10 V X5R -> 6.3 V X5R
- C1322: value 22 µF -> 100 nF; footprint Capacitor_SMD:C_0603_1608Metric -> Capacitor_SMD:C_0201_0603Metric; MPN GRM188R60J226MEA0D -> GRM033R61A104KE15D; Spec 6.3 V X5R -> 10 V X5R
- C1323: value 100 nF -> 22 µF; footprint Capacitor_SMD:C_0201_0603Metric -> Capacitor_SMD:C_0603_1608Metric; Decoupling vcc_ddr -> vdd_npu; MPN GRM033R61A104KE15D -> GRM188R60J226MEA0D; Spec 10 V X5R -> 6.3 V X5R
- C1327: value 10 µF -> 4.7 µF; footprint Capacitor_SMD:C_0603_1608Metric -> Capacitor_SMD:C_0402_1005Metric; MPN GRM188R61A106KE69D -> GRM155R60J475ME47D; Spec 10 V X5R -> 6.3 V X5R
- C1328: value 100 nF -> 10 µF; footprint Capacitor_SMD:C_0201_0603Metric -> Capacitor_SMD:C_0603_1608Metric; Decoupling vcc0v6_ddr -> vcc_ddr; MPN GRM033R61A104KE15D -> GRM188R61A106KE69D
- C1333: value 100 nF -> 4.7 µF; footprint Capacitor_SMD:C_0201_0603Metric -> Capacitor_SMD:C_0402_1005Metric; Decoupling vdda_0v9 -> vcc0v6_ddr; MPN GRM033R61A104KE15D -> GRM155R60J475ME47D; Spec (none) -> 6.3 V X5R
- C1334, C1336: value 1 µF -> 100 nF; footprint Capacitor_SMD:C_0402_1005Metric -> Capacitor_SMD:C_0201_0603Metric; MPN GRM155C71A105KE11D -> GRM033R61A104KE15D
- C1335: value 100 nF -> 1 µF; footprint Capacitor_SMD:C_0201_0603Metric -> Capacitor_SMD:C_0402_1005Metric; Decoupling vcca_1v8 -> vdda_0v9; MPN GRM033R61A104KE15D -> GRM155C71A105KE11D
- C1337: value 100 nF -> 1 µF; footprint Capacitor_SMD:C_0201_0603Metric -> Capacitor_SMD:C_0402_1005Metric; Decoupling vcc3v3_sys -> vcca_1v8; MPN GRM033R61A104KE15D -> GRM155C71A105KE11D
- C1341: Decoupling vcc_1v8 -> vcc3v3_sys
- C1343: Decoupling vccio_sd -> vcc_1v8
- C1344: Decoupling vccio6_1v8 -> vccio_sd
- C1346: Decoupling vcc3v3_pmu -> vccio6_1v8
- C1347: Decoupling vcca1v8_pmu -> vcc3v3_pmu
Connections:
- net GND: now also C1349.2
- net vcc0v6_ddr: now also C1333.1; no longer C1328.1
- net vcc3v3_pmu: now also C1347.1; no longer C1346.1
- net vcc3v3_sys: now also C1341.1; no longer C1337.1
- net vcc_1v8: now also C1343.1; no longer C1341.1
- net vcc_ddr: now also C1328.1; no longer C1323.1
- net vcca1v8_pmu: now also C1349.1; no longer C1347.1
- net vcca_1v8: now also C1337.1; no longer C1335.1
- net vccio6_1v8: now also C1346.1; no longer C1344.1
- net vccio_sd: now also C1344.1; no longer C1343.1
- net vdd_cpu: now also C1313.1
- net vdd_gpu: now also C1321.1; no longer C1318.1
- net vdd_logic: now also C1318.1; no longer C1313.1
- net vdd_npu: now also C1323.1; no longer C1321.1
- net vdda_0v9: now also C1335.1; no longer C1333.1
Other:
- moved on the sheet: C1313, C1314, C1315, C1316, C1317, C1318, C1319, C1320, C1321, C1322, C1323, C1324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

Commit message: Variants: devicetree nodes, host-side absent pulls, board variant data
Feature blocks: every record with a devicetree node names it; Sub-blocks
rows for the 16 sheet IDs. The RP2354 and HPA_RAIL_EN absent-state
pull-downs move to blk.soc-vccio-b, so they stay when the block is not
fitted; cover detect relies on the ball's own pull-down. pcb/variants.py
copies the schematic's production data onto the board. odapkit variant
check: full and production pass, reproducible.

The PTS815 land drawn from the C&K data sheet (p. B-44); the side buttons
respaced for it (PCB-Z-08 updated). Studies find repos.tsv by walking up
and use libs' rockchip.pretty. DRC 0 errors, ERC 0 errors, craft Q1 met,
pcb tests pass (33), 994 parts placed, 99.7 % board need, factor 1.64.

Co-Authored-By: Claude Opus 5.5 <noreply@anthropic.com>
Claude-Session: https://claude.ai/code/session_013P6pW9LdyEMFishwCcZGUr
Parts:
- removed R1336: 5 mΩ, Resistor_SMD:R_1206_3216Metric, symbol Device:R
- removed R1337: 0 Ω, Resistor_SMD:R_0603_1608Metric, symbol Device:R
- added R1339: 5 mΩ, Resistor_SMD:R_1206_3216Metric, symbol Device:R
- added R1340: 0 Ω, Resistor_SMD:R_0603_1608Metric, symbol Device:R
Connections:
- net VDD_LOGIC_SRC: now also R1339.1
- net vcc_1v8: now also R1340.1
- net vccio6_1v8: now also R1340.2
- net vdd_logic: now also R1339.2

Commit message: Board: pre-PCB schematic items closed with datasheets (BOM v1.22)
Display INA236 to 0x49 (INA236B, A0 = VS): no A0 = SDA strap, so the
address no longer depends on the host's I2C hold time. The 18 WSL
shunts and links on Vishay's doc 30100 lands. 24 MHz crystal NDK
NX3225GA (CL 8 pF) with 2 x 10 pF. Backlight inductor Coilcraft
XFL3012-223MEC on its published land (no placeholder left). Action
button PTS815 G code on the side-button land. Cover-detect leakage,
TPS3808 spread, RP2354A supply pins and the USB series scheme closed
without change. Placement v1.9: 100.2 % need, factor 1.64, DRC 0
errors; power tree v0.12; PCB-Z-08 and CB-08 strip values.

Co-Authored-By: Claude Opus 5.5 <noreply@anthropic.com>
Claude-Session: https://claude.ai/code/session_013P6pW9LdyEMFishwCcZGUr
Parts:
- R1339: footprint Resistor_SMD:R_1206_3216Metric -> T1_Main_Board:R_Vishay_WSL1206_2m-5m9
Changed lines of the file:
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@@
   (property "Value" "5 mΩ" (at 73.66 266.7 90) (effects (font (size 1.27 1.27))))
   (property "Spec" "1206" (at 73.66 269.24 90) (effects (font (size 1.27 1.27))))
-  (property "Footprint" "Resistor_SMD:R_1206_3216Metric" (at 76.2 264.16 0) (effects (font (size 1.27 1.27))) (hide yes))
+  (property "Footprint" "T1_Main_Board:R_Vishay_WSL1206_2m-5m9" (at 76.2 264.16 0) (effects (font (size 1.27 1.27))) (hide yes))
   (property "Datasheet" "https://www.vishay.com/docs/30100/wsl.pdf" (at 76.2 264.16 0) (effects (font (size 1.27 1.27))) (hide yes))
   (property "Description" "Current-sense resistor, 5 mOhm, 1 %, 0.5 W, 1206 metal strip: measurement link H5" (at 76.2 264.16 0) (effects (font (size 1.27 1.27))) (hide yes))
