File: board/hardware/t1-main-board/vdd-cpu.kicad_sch (KiCad schematic)
At the start: 20 parts, among them U1201 TPS6286910CRQYR

Commit message: Zone net classes and named switch nodes from the generator
Every net but GND now carries the ZONE_<NAME> class of each zone whose
blocks it touches (block zones from pcb/plan.py; the faceplate connector's
sheet also the faceplate zone); a rail used in more than one zone carries
ZONE_SHARED. Nets KiCad names from a pin take their part's sheet zone.
1,080 nets: 911 in one zone, 104 in two, 36 in three, 28 shared rails.

Switch nodes are named *_SW (VSYS_LV_SW, VCC3V3_SYS_SW, VDD_CPU_SW,
RP_VREG_SW); the display switch output is FP_VCI_OUT, so SW_NODE holds
the 18 switch nodes only. Board rebuilt: DRC 0 errors, 607 warnings
(the six PCB-I-09 gone), ERC 0 errors, craft Q1 met, pcb tests pass.
Closes placement v1 open items 2 and 3, floorplan v1 item 6.

Co-Authored-By: Claude Opus 5.5 <noreply@anthropic.com>
Claude-Session: https://claude.ai/code/session_01Ei262h3TpgY9vyfNLMi5Mn
Connections:
- net VDD_CPU_SW: now reaches L1201.1, U1201.7 (SW)
Changed lines of the file:
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@@
 (label "I2C0_SCL" (at 104.14 81.28 180) (effects (font (size 1.27 1.27)) (justify right bottom)))
 (label "VDD_CPU_PG" (at 129.54 93.98 270) (effects (font (size 1.27 1.27)) (justify right bottom)))
+(label "VDD_CPU_SW" (at 134.62 76.2 90) (effects (font (size 1.27 1.27)) (justify left bottom)))
 (label "VDD_CPU_PG" (at 40.64 134.62 180) (effects (font (size 1.27 1.27)) (justify right bottom)))
 (bus (pts (xy 45.72 247.65) (xy 50.8 247.65)) (stroke (width 0) (type default)))

Commit message: Compaction: lower inductors, 0201 decoupling, 0.8 mm signal test pads
A matrix tool (hardware/studies/compaction) checks each candidate against
the design's stresses: same inductance, design peak <= 70 % and the
converter's maximum limit <= 100 % of Isat (30 % drop), height zones,
ratings at least twice the rail, PCB-D-06; sourcing outcome per part.

Applied (placement v1 decision 12, BOM v1.15):
- L601, L4401: XGL4015-102MEC (1.5 mm) for XAL/XGL4020-102MEC (2.1 mm);
- L1001, L5101: XGL4015-471MEC (1.5 mm) for Wurth 744373240047, on the
  stock XxL4020 land (the Wurth land was never drawn);
- L1201 is 1.2 mm (XGL4012, per-MPN heights): it moves next to the SoC;
- 58 x 100 nF decoupling on rails <= 3.3 V in core/IO/radio: 0201;
- 51 test pads on signal nets: 0.8 mm (PCB-D-06 v0.16, JLCPCB guide).
Kept: L901, L2802 (XGL4015 at 103 % of Isat at the limit); no thinner
0805/1206 capacitor passes (obsolete, NRND or unlisted).

Board need 113 % -> 111 % (core band 227 -> 203 %, power band 258 ->
233 %, radio band 19 -> 0 %); only C904 still relies on PCB-Z-04.
ERC 0 errors, craft Q1 met, DRC 0 errors (605 warnings), pcb and study
tests pass, rules test board PASS.

Co-Authored-By: Claude Opus 5.5 <noreply@anthropic.com>
Claude-Session: https://claude.ai/code/session_01Ei262h3TpgY9vyfNLMi5Mn
Parts:
- TP1201, TP1204: footprint TestPoint:TestPoint_Pad_D1.0mm -> T1_Main_Board:TestPoint_Pad_D0.8mm
Changed lines of the file:
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@@
   (property "Reference" "TP1201" (at 207.01 86.36 0) (effects (font (size 1.27 1.27)) (justify left)))
   (property "Value" "VDD_CPU_VOS" (at 207.01 88.9 0) (effects (font (size 1.27 1.27)) (justify left)))
-  (property "Footprint" "TestPoint:TestPoint_Pad_D1.0mm" (at 205.74 91.44 0) (effects (font (size 1.27 1.27))) (hide yes))
+  (property "Footprint" "T1_Main_Board:TestPoint_Pad_D0.8mm" (at 205.74 91.44 0) (effects (font (size 1.27 1.27))) (hide yes))
   (property "Datasheet" "~" (at 205.74 91.44 0) (effects (font (size 1.27 1.27))) (hide yes))
-  (property "Description" "Test pad, 1.0 mm" (at 205.74 91.44 0) (effects (font (size 1.27 1.27))) (hide yes))
+  (property "Description" "Test pad, 0.8 mm, signal net" (at 205.74 91.44 0) (effects (font (size 1.27 1.27))) (hide yes))
   (property "Block" "blk.vdd-cpu" (at 205.74 91.44 0) (effects (font (size 1.27 1.27))) (hide yes))
   (pin "1")
@@
   (property "Reference" "TP1204" (at 72.39 127 0) (effects (font (size 1.27 1.27)) (justify left)))
   (property "Value" "VDD_CPU_PG" (at 72.39 129.54 0) (effects (font (size 1.27 1.27)) (justify left)))
-  (property "Footprint" "TestPoint:TestPoint_Pad_D1.0mm" (at 71.12 132.08 0) (effects (font (size 1.27 1.27))) (hide yes))
+  (property "Footprint" "T1_Main_Board:TestPoint_Pad_D0.8mm" (at 71.12 132.08 0) (effects (font (size 1.27 1.27))) (hide yes))
   (property "Datasheet" "~" (at 71.12 132.08 0) (effects (font (size 1.27 1.27))) (hide yes))
-  (property "Description" "Test pad, 1.0 mm" (at 71.12 132.08 0) (effects (font (size 1.27 1.27))) (hide yes))
+  (property "Description" "Test pad, 0.8 mm, signal net" (at 71.12 132.08 0) (effects (font (size 1.27 1.27))) (hide yes))
   (property "Block" "blk.vdd-cpu" (at 71.12 132.08 0) (effects (font (size 1.27 1.27))) (hide yes))
   (pin "1")

Commit message: Board on libs v0.2.0: lower-case kebab vendor keys (HL-13)
The libs submodule moves to v0.2.0 (5f24483). Every library nickname in
the generator, the placement tool and the floorplan study follows the
key table (Texas_Instruments -> texas-instruments, OpenDAP_Device ->
opendap-generic, Rockchip and Rockchip_PMIC -> rockchip, ...); the
library tables are written from the files. Schematic and board
regenerated.

Checks: ERC 0 errors (warnings unchanged); DRC 0 errors, 605 warnings,
the same counts by type, schematic parity 0; every placement identical;
craft Q1 met; pcb tests pass; STEP export resolves every libs 3D model
(the 27 parts without a model are KiCad stock lands that have none).

Co-Authored-By: Claude Opus 5.5 <noreply@anthropic.com>
Claude-Session: https://claude.ai/code/session_01Ei262h3TpgY9vyfNLMi5Mn
Parts:
- U1201: footprint Texas_Instruments:Texas_RQY0009A_VQFN-HR-9_1.5x2.5mm_P0.5mm -> texas-instruments:Texas_RQY0009A_VQFN-HR-9_1.5x2.5mm_P0.5mm; symbol Texas_Instruments:TPS6286910CRQYR -> texas-instruments:TPS6286910CRQYR
Changed lines of the file:
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@@
 (paper "A3")
 (title_block (title "CPU core supply") (date "2026-10-25") (rev "A") (company "The OpenDAP Project") (comment 1 "blk.vdd-cpu") (comment 2 "vdd_cpu 0.85-1.15 V for the RK3566 CPU cluster, I2C DVS on I2C0 at 0x42, 6 A"))
-(symbol (lib_id "Texas_Instruments:TPS6286910CRQYR") (at 116.84 78.74 0) (unit 1) (body_style 1) (exclude_from_sim no) (in_bom yes) (on_board yes) (dnp no)
+(symbol (lib_id "texas-instruments:TPS6286910CRQYR") (at 116.84 78.74 0) (unit 1) (body_style 1) (exclude_from_sim no) (in_bom yes) (on_board yes) (dnp no)
   (property "Reference" "U1201" (at 118.11 60.96 0) (effects (font (size 1.27 1.27)) (justify left)))
   (property "Value" "TPS6286910CRQYR" (at 118.11 58.42 0) (effects (font (size 1.27 1.27)) (justify left)))
-  (property "Footprint" "Texas_Instruments:Texas_RQY0009A_VQFN-HR-9_1.5x2.5mm_P0.5mm" (at 116.84 78.74 0) (effects (font (size 1.27 1.27))) (hide yes))
+  (property "Footprint" "texas-instruments:Texas_RQY0009A_VQFN-HR-9_1.5x2.5mm_P0.5mm" (at 116.84 78.74 0) (effects (font (size 1.27 1.27))) (hide yes))
   (property "Datasheet" "https://www.ti.com/lit/ds/symlink/tps62869.pdf" (at 116.84 78.74 0) (effects (font (size 1.27 1.27))) (hide yes))
   (property "Description" "6 A synchronous step-down converter with I2C DVS, 2.4-5.5 V input, 0.4-1.675 V in 5 mV steps, 0.9 V start-up, address 0x42, power good, VQFN-HR-9 (RQY0009A) 1.5 x 2.5 mm" (at 116.84 78.74 0) (effects (font (size 1.27 1.27))) (hide yes))

Commit message: Board in the 62.5 x 95.0 mm body: ADR 0025, outline 59.1 x 91.6, 0201 swaps
ADR 0025 supersedes ADR 0016 for t1 ADR 0006's body: board outline from
the body, 1.2 mm walls and 0.5 mm clearance; height zones and stack
restated unchanged; the speaker on a case shelf (PCB-Z-09); pocket
reliefs at the 4.4 mm jack, the microSD (DM3AT push-push kept) and the
side buttons; the audio 0603 -> 0402 swap gated by t1 V2-A08; reserve
(NFC reader, then TPM) recorded, not applied.

- pcb/geometry.py derives the outline from BODY, WALL and CLEARANCE;
  the pocket, display and fixed parts keep their device-frame positions;
  holes keep their edge distance; the speaker shadow becomes a 1.5 mm
  shelf height area (placement, checks, occupancy).
- build.py reports pocket reliefs and routing room; C904 unfixed (it
  now finds back room, so PCB-Z-04 carries no part).
- Generator: parts.area_swap puts 121 generic 0402 resistors (outside
  audio and VBUS paths, >= 10 ohm) and five 100 nF signal capacitors in
  0201 (BOM v1.16); schematic and board regenerated.
- Result: 1,012/1,012 placed, 98.8 % by the floorplan method (was 111 %),
  factor left 1.68 (was 1.49); DRC 0 errors, ERC 0 errors, 0 check
  findings, pcb tests 20/20, schematic craft Q1 met.
- Specs: PCB constraints v0.17 (M-01, M-02, M-08, Z-02, Z-06 to Z-09,
  R-07), placement v1.1 (section 3, decisions 4 and 13, checks, open
  items with the gated swaps and the reserve), floorplan v1 section 1,
  BOM v1.16.

Co-Authored-By: Claude Opus 5.5 <noreply@anthropic.com>
Claude-Session: https://claude.ai/code/session_01Ei262h3TpgY9vyfNLMi5Mn
Parts:
- C1204, C1207: footprint Capacitor_SMD:C_0402_1005Metric -> Capacitor_SMD:C_0201_0603Metric; MPN GRM155R71C104KA88D -> GRM033R61A104KE15D
- R1201: footprint Resistor_SMD:R_0402_1005Metric -> Resistor_SMD:R_0201_0603Metric; MPN RC0402FR-0751KL -> RC0201FR-0751KL
- R1202: footprint Resistor_SMD:R_0402_1005Metric -> Resistor_SMD:R_0201_0603Metric; MPN RC0402FR-07100RL -> RC0201FR-07100RL
- R1205: footprint Resistor_SMD:R_0402_1005Metric -> Resistor_SMD:R_0201_0603Metric; MPN RC0402FR-07100KL -> RC0201FR-07100KL
- R1206: footprint Resistor_SMD:R_0402_1005Metric -> Resistor_SMD:R_0201_0603Metric; MPN RC0402FR-0786K6L -> RC0201FR-0786K6L
Changed lines of the file:
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@@
   (property "Reference" "R1201" (at 77.47 64.77 0) (effects (font (size 1.27 1.27)) (justify right)))
   (property "Value" "51 kΩ" (at 77.47 67.31 0) (effects (font (size 1.27 1.27)) (justify right)))
-  (property "Footprint" "Resistor_SMD:R_0402_1005Metric" (at 78.74 66.04 0) (effects (font (size 1.27 1.27))) (hide yes))
-  (property "Datasheet" "https://yageogroup.com/en/ProductSearch/PartNumberSearch?part=RC0402FR-0751KL" (at 78.74 66.04 0) (effects (font (size 1.27 1.27))) (hide yes))
-  (property "Description" "Resistor, 51 kΩ, 1 %, 1/16 W, 0402" (at 78.74 66.04 0) (effects (font (size 1.27 1.27))) (hide yes))
+  (property "Footprint" "Resistor_SMD:R_0201_0603Metric" (at 78.74 66.04 0) (effects (font (size 1.27 1.27))) (hide yes))
+  (property "Datasheet" "https://yageogroup.com/en/ProductSearch/PartNumberSearch?part=RC0201FR-0751KL" (at 78.74 66.04 0) (effects (font (size 1.27 1.27))) (hide yes))
+  (property "Description" "Resistor, 51 kΩ, 1 %, 1/20 W, 0201" (at 78.74 66.04 0) (effects (font (size 1.27 1.27))) (hide yes))
   (property "Manufacturer" "YAGEO" (at 78.74 66.04 0) (effects (font (size 1.27 1.27))) (hide yes))
-  (property "MPN" "RC0402FR-0751KL" (at 78.74 66.04 0) (effects (font (size 1.27 1.27))) (hide yes))
+  (property "MPN" "RC0201FR-0751KL" (at 78.74 66.04 0) (effects (font (size 1.27 1.27))) (hide yes))
   (property "Block" "blk.vdd-cpu" (at 78.74 66.04 0) (effects (font (size 1.27 1.27))) (hide yes))
   (pin "1")
@@
   (property "Reference" "C1204" (at 88.9 87.63 0) (effects (font (size 1.27 1.27)) (justify left)))
   (property "Value" "100 nF" (at 88.9 90.17 0) (effects (font (size 1.27 1.27)) (justify left)))
-  (property "Footprint" "Capacitor_SMD:C_0402_1005Metric" (at 86.36 88.9 0) (effects (font (size 1.27 1.27))) (hide yes))
-  (property "Datasheet" "https://www.murata.com/en-us/products/productdetail?partno=GRM155R71C104KA88D" (at 86.36 88.9 0) (effects (font (size 1.27 1.27))) (hide yes))
-  (property "Description" "Capacitor, 100 nF, 16 V, X7R, 0402" (at 86.36 88.9 0) (effects (font (size 1.27 1.27))) (hide yes))
+  (property "Footprint" "Capacitor_SMD:C_0201_0603Metric" (at 86.36 88.9 0) (effects (font (size 1.27 1.27))) (hide yes))
+  (property "Datasheet" "https://www.murata.com/en-us/products/productdetail?partno=GRM033R61A104KE15D" (at 86.36 88.9 0) (effects (font (size 1.27 1.27))) (hide yes))
+  (property "Description" "Capacitor, 100 nF, 10 V, X5R, 0201" (at 86.36 88.9 0) (effects (font (size 1.27 1.27))) (hide yes))
   (property "Manufacturer" "Murata" (at 86.36 88.9 0) (effects (font (size 1.27 1.27))) (hide yes))
-  (property "MPN" "GRM155R71C104KA88D" (at 86.36 88.9 0) (effects (font (size 1.27 1.27))) (hide yes))
+  (property "MPN" "GRM033R61A104KE15D" (at 86.36 88.9 0) (effects (font (size 1.27 1.27))) (hide yes))
   (property "Block" "blk.vdd-cpu" (at 86.36 88.9 0) (effects (font (size 1.27 1.27))) (hide yes))
   (pin "1")
@@
   (property "Reference" "R1202" (at 184.15 83.82 0) (effects (font (size 1.27 1.27)) (justify left)))
   (property "Value" "100 Ω" (at 184.15 86.36 0) (effects (font (size 1.27 1.27)) (justify left)))
-  (property "Footprint" "Resistor_SMD:R_0402_1005Metric" (at 182.88 85.09 0) (effects (font (size 1.27 1.27))) (hide yes))
-  (property "Datasheet" "https://yageogroup.com/en/ProductSearch/PartNumberSearch?part=RC0402FR-07100RL" (at 182.88 85.09 0) (effects (font (size 1.27 1.27))) (hide yes))
-  (property "Description" "Resistor, 100 Ω, 1 %, 1/16 W, 0402" (at 182.88 85.09 0) (effects (font (size 1.27 1.27))) (hide yes))
+  (property "Footprint" "Resistor_SMD:R_0201_0603Metric" (at 182.88 85.09 0) (effects (font (size 1.27 1.27))) (hide yes))
+  (property "Datasheet" "https://yageogroup.com/en/ProductSearch/PartNumberSearch?part=RC0201FR-07100RL" (at 182.88 85.09 0) (effects (font (size 1.27 1.27))) (hide yes))
+  (property "Description" "Resistor, 100 Ω, 1 %, 1/20 W, 0201" (at 182.88 85.09 0) (effects (font (size 1.27 1.27))) (hide yes))
   (property "Manufacturer" "YAGEO" (at 182.88 85.09 0) (effects (font (size 1.27 1.27))) (hide yes))
-  (property "MPN" "RC0402FR-07100RL" (at 182.88 85.09 0) (effects (font (size 1.27 1.27))) (hide yes))
+  (property "MPN" "RC0201FR-07100RL" (at 182.88 85.09 0) (effects (font (size 1.27 1.27))) (hide yes))
   (property "Block" "blk.vdd-cpu" (at 182.88 85.09 0) (effects (font (size 1.27 1.27))) (hide yes))
   (pin "1")
@@
   (property "Reference" "C1207" (at 203.2 101.6 0) (effects (font (size 1.27 1.27)) (justify left)))
   (property "Value" "100 nF" (at 203.2 104.14 0) (effects (font (size 1.27 1.27)) (justify left)))
-  (property "Footprint" "Capacitor_SMD:C_0402_1005Metric" (at 200.66 102.87 0) (effects (font (size 1.27 1.27))) (hide yes))
-  (property "Datasheet" "https://www.murata.com/en-us/products/productdetail?partno=GRM155R71C104KA88D" (at 200.66 102.87 0) (effects (font (size 1.27 1.27))) (hide yes))
-  (property "Description" "Capacitor, 100 nF, 16 V, X7R, 0402" (at 200.66 102.87 0) (effects (font (size 1.27 1.27))) (hide yes))
+  (property "Footprint" "Capacitor_SMD:C_0201_0603Metric" (at 200.66 102.87 0) (effects (font (size 1.27 1.27))) (hide yes))
+  (property "Datasheet" "https://www.murata.com/en-us/products/productdetail?partno=GRM033R61A104KE15D" (at 200.66 102.87 0) (effects (font (size 1.27 1.27))) (hide yes))
+  (property "Description" "Capacitor, 100 nF, 10 V, X5R, 0201" (at 200.66 102.87 0) (effects (font (size 1.27 1.27))) (hide yes))
   (property "Manufacturer" "Murata" (at 200.66 102.87 0) (effects (font (size 1.27 1.27))) (hide yes))
-  (property "MPN" "GRM155R71C104KA88D" (at 200.66 102.87 0) (effects (font (size 1.27 1.27))) (hide yes))
+  (property "MPN" "GRM033R61A104KE15D" (at 200.66 102.87 0) (effects (font (size 1.27 1.27))) (hide yes))
   (property "Block" "blk.vdd-cpu" (at 200.66 102.87 0) (effects (font (size 1.27 1.27))) (hide yes))
   (pin "1")
@@
   (property "Reference" "R1205" (at 57.15 129.54 0) (effects (font (size 1.27 1.27)) (justify left)))
   (property "Value" "100 kΩ" (at 57.15 132.08 0) (effects (font (size 1.27 1.27)) (justify left)))
-  (property "Footprint" "Resistor_SMD:R_0402_1005Metric" (at 55.88 130.81 0) (effects (font (size 1.27 1.27))) (hide yes))
-  (property "Datasheet" "https://yageogroup.com/en/ProductSearch/PartNumberSearch?part=RC0402FR-07100KL" (at 55.88 130.81 0) (effects (font (size 1.27 1.27))) (hide yes))
-  (property "Description" "Resistor, 100 kΩ, 1 %, 1/16 W, 0402" (at 55.88 130.81 0) (effects (font (size 1.27 1.27))) (hide yes))
+  (property "Footprint" "Resistor_SMD:R_0201_0603Metric" (at 55.88 130.81 0) (effects (font (size 1.27 1.27))) (hide yes))
+  (property "Datasheet" "https://yageogroup.com/en/ProductSearch/PartNumberSearch?part=RC0201FR-07100KL" (at 55.88 130.81 0) (effects (font (size 1.27 1.27))) (hide yes))
+  (property "Description" "Resistor, 100 kΩ, 1 %, 1/20 W, 0201" (at 55.88 130.81 0) (effects (font (size 1.27 1.27))) (hide yes))
   (property "Manufacturer" "YAGEO" (at 55.88 130.81 0) (effects (font (size 1.27 1.27))) (hide yes))
-  (property "MPN" "RC0402FR-07100KL" (at 55.88 130.81 0) (effects (font (size 1.27 1.27))) (hide yes))
+  (property "MPN" "RC0201FR-07100KL" (at 55.88 130.81 0) (effects (font (size 1.27 1.27))) (hide yes))
   (property "Block" "blk.vdd-cpu" (at 55.88 130.81 0) (effects (font (size 1.27 1.27))) (hide yes))
   (pin "1")
@@
   (property "Reference" "R1206" (at 92.71 137.16 0) (effects (font (size 1.27 1.27)) (justify left)))
   (property "Value" "86.6 kΩ" (at 92.71 139.7 0) (effects (font (size 1.27 1.27)) (justify left)))
-  (property "Footprint" "Resistor_SMD:R_0402_1005Metric" (at 91.44 138.43 0) (effects (font (size 1.27 1.27))) (hide yes))
-  (property "Datasheet" "https://yageogroup.com/en/ProductSearch/PartNumberSearch?part=RC0402FR-0786K6L" (at 91.44 138.43 0) (effects (font (size 1.27 1.27))) (hide yes))
-  (property "Description" "Resistor, 86.6 kΩ, 1 %, 1/16 W, 0402" (at 91.44 138.43 0) (effects (font (size 1.27 1.27))) (hide yes))
+  (property "Footprint" "Resistor_SMD:R_0201_0603Metric" (at 91.44 138.43 0) (effects (font (size 1.27 1.27))) (hide yes))
+  (property "Datasheet" "https://yageogroup.com/en/ProductSearch/PartNumberSearch?part=RC0201FR-0786K6L" (at 91.44 138.43 0) (effects (font (size 1.27 1.27))) (hide yes))
+  (property "Description" "Resistor, 86.6 kΩ, 1 %, 1/20 W, 0201" (at 91.44 138.43 0) (effects (font (size 1.27 1.27))) (hide yes))
   (property "Manufacturer" "YAGEO" (at 91.44 138.43 0) (effects (font (size 1.27 1.27))) (hide yes))
-  (property "MPN" "RC0402FR-0786K6L" (at 91.44 138.43 0) (effects (font (size 1.27 1.27))) (hide yes))
+  (property "MPN" "RC0201FR-0786K6L" (at 91.44 138.43 0) (effects (font (size 1.27 1.27))) (hide yes))
   (property "Block" "blk.vdd-cpu" (at 91.44 138.43 0) (effects (font (size 1.27 1.27))) (hide yes))
   (property "Alternate" "tps628691a" (at 91.44 138.43 0) (effects (font (size 1.27 1.27))) (hide yes))
